Commit message: some minor changes to atlas_robot.urdf
git-svn-id: https://svn.csail.mit.edu/drc@62 c7283977-0100-402a-a91a-fa70b306dbfe

File: ros_workspace/atlas_description/urdf/atlas_robot.urdf (robot description, URDF)
Before this commit: robot atlas, 36 links, 35 joints
Links:
- removed link Lankle
- removed link Lfoot
- removed link Rankle
- removed link Rfoot
- removed link back
- removed link pelvis-link1
- removed link pelvis-link2
- removed link torso
- added link Back, mass 0.01
- added link LAnkle, mass 0.01
- added link LFoot, mass 2.0; collision box size=0.224276512 0.06 0.015; visual box size=0.224276512 0.06 0.015
- added link Pelvis-link1, mass 5.7; collision cylinder length=0.152491948 radius=0.025; visual cylinder length=0.112491948 radius=0.025
- added link Pelvis-link2, mass 0.01; collision cylinder length=0.21784564 radius=0.025; visual cylinder length=0.17784564 radius=0.025
- added link RAnkle, mass 0.01
- added link RFoot, mass 2.0; collision box size=0.224276512 0.06 0.015; visual box size=0.224276512 0.06 0.015
- added link Torso, mass 19.267; collision box size=0.178562 0.4999736 0.47854616; visual cylinder length=0.47854616 radius=0.025
Joints:
- removed joint Lankle_joint
- removed joint Lfoot_joint
- removed joint Rankle_joint
- removed joint Rfoot_joint
- removed joint back_pelvis
- removed joint mid_pelvis_dummy
- added joint Back_Pelvis_Joint: type fixed, parent Back, child Pelvis-link1, origin xyz=0 0 0 rpy=0 0 0
- added joint LAnkle_joint: type fixed, parent LAnklePitch_link, child LAnkle, origin xyz=0 0 0
- added joint LFoot_joint: type fixed, parent LAnkle, child LFoot, origin xyz=0 0 -0.04519
- added joint Mid_Pelvis_Joint: type fixed, parent Pelvis-link1, child Pelvis-link2, origin xyz=0 0 -0.152491948 rpy=0 0 0
- added joint RAnkle_joint: type fixed, parent RAnklePitch_link, child RAnkle, origin xyz=0 0 0
- added joint RFoot_joint: type fixed, parent RAnkle, child RFoot, origin xyz=0 0 -0.04519
- joint BackRoll_Torso_joint: child torso -> Torso
- joint BackYaw: parent back -> Back
- joint LHipYaw: parent pelvis-link2 -> Pelvis-link2
- joint NeckYaw: parent torso -> Torso
- joint RHipYaw: parent pelvis-link2 -> Pelvis-link2
- joint base_joint: child back -> Back

File: ros_workspace/atlas_description/urdf/atlas_structure.urdf.xacro (robot description, xacro)
@@ -89,8 +89,8 @@
     <xacro:insert_visualization_ankle side="${side}"/>
   </link>
-  <link name="${side}ankle">
-    <xacro:insert_small_inertial />
-  </link>
-  <link name="${side}foot">
+  <link name="${side}Ankle">
+    <xacro:insert_small_inertial />
+  </link>
+  <link name="${side}Foot">
    <xacro:insert_inertial_cuboid mass="${mass_foot}" l_x="${l_foot*height}" l_y="0.06" l_z="0.015"/>
     <xacro:insert_visualization_foot side="${side}"/>
@@ -106,5 +106,5 @@
   </joint>
   <joint name="BackYaw" type="revolute">
-    <parent link="back"/>
+    <parent link="Back"/>
     <child link="BackYaw_link"/>
     <origin xyz="0 0 0.0" rpy="0 0 0" />
@@ -127,5 +127,5 @@
   </joint>
   <joint name="BackRoll_Torso_joint" type="fixed">
-    <child link="torso"/>
+    <child link="Torso"/>
     <parent link="BackRoll_link"/>
     <origin xyz="0 0 0" rpy="0 0 0" />
@@ -234,5 +234,5 @@
   </joint>
  <!-- <joint name="LHipYaw" type="revolute">
-    <parent link="back"/>
+    <parent link="Back"/>
     <child link="LHipYaw_link"/>
     <origin xyz="0 ${-1*-(o_back_hip_y*height)} ${-o_back_hip_z*height}" rpy="0 0 0"/>
@@ -241,5 +241,5 @@
   </joint>
   <joint name="RHipYaw" type="revolute">
-    <parent link="back"/>
+    <parent link="Back"/>
     <child link="RHipYaw_link"/>
     <origin xyz="0 ${1*-(o_back_hip_y*height)} ${-o_back_hip_z*height}" rpy="0 0 0"/>
@@ -276,12 +276,12 @@
     <limit velocity="3.0" effort="30" lower="${ankle_flexion_limit*pi_180}" upper="${ankle_extension_limit*pi_180}"/>
   </joint>
-  <joint name="${side}ankle_joint" type="fixed">
+  <joint name="${side}Ankle_joint" type="fixed">
     <parent link="${side}AnklePitch_link" />
-    <child link="${side}ankle" />
+    <child link="${side}Ankle" />
     <origin xyz="0 0 0" />
   </joint>
-  <joint name="${side}foot_joint" type="fixed">
-    <parent link="${side}ankle" />
-    <child link="${side}foot" />
+  <joint name="${side}Foot_joint" type="fixed">
+    <parent link="${side}Ankle" />
+    <child link="${side}Foot" />
     <origin xyz="0 0 -0.04519" />
   </joint>
