Commit message: git-svn-id: https://svn.csail.mit.edu/drc@60 c7283977-0100-402a-a91a-fa70b306dbfe

File: ros_workspace/atlas_description/urdf/atlas_structure.urdf.xacro (robot description, xacro)
@@ -11,12 +11,12 @@
     <xacro:insert_small_inertial />
   </link>
-  <link name="back">
-    <xacro:insert_small_inertial />
-  </link>
-  <link name="pelvis-link1">
+  <link name="Back">
+    <xacro:insert_small_inertial />
+  </link>
+  <link name="Pelvis-link1">
    <xacro:insert_inertial_cuboid mass="${mass_pelvis}" l_x="${0.1*height}" l_y="${w_pelvis*height}" l_z="${l_pelvis*height}"/>
    <xacro:insert_visualization_pelvis1/>
   </link>
-  <link name="pelvis-link2">
+  <link name="Pelvis-link2">
    <xacro:insert_small_inertial />
    <xacro:insert_visualization_pelvis2/>
@@ -31,5 +31,5 @@
     <xacro:insert_small_inertial />
   </link>
- <link name="torso" >
+ <link name="Torso" >
    <!-- assuming the rotational inertia of the torso is of a cuboid -->
   <xacro:insert_inertial_cuboid mass="${mass_torso_back+mass_misc_div_3}" l_x="${0.1*height}" l_y="${0.28*height}" l_z="${0.268*height}"/>
@@ -101,5 +101,5 @@
 <!--   Joints following below -->
   <joint name="base_joint" type="fixed">
-    <child link="back"/>
+    <child link="Back"/>
     <parent link="base_link"/>
     <origin xyz="0 0 0" rpy="0 0 0" />
@@ -133,5 +133,5 @@
 <!-- Neck joints -->
   <joint name="NeckYaw" type="revolute">
-    <parent link="torso"/>
+    <parent link="Torso"/>
     <child link="NeckYaw_link"/>
     <origin xyz="0 0 ${(l_torso)*height}" rpy="0 0 0" />
@@ -208,17 +208,17 @@
   </joint>
 <!-- Pelvis joints -->
- <joint name="back_pelvis" type="fixed">
-    <parent link="back"/>
-    <child link="pelvis-link1"/>
-    <origin xyz="0 0 0" rpy="0 0 0" />
-  </joint>
- <joint name="mid_pelvis_dummy" type="fixed">
-    <parent link="pelvis-link1"/>
-    <child link="pelvis-link2"/>
+ <joint name="Back_Pelvis_Joint" type="fixed">
+    <parent link="Back"/>
+    <child link="Pelvis-link1"/>
+    <origin xyz="0 0 0" rpy="0 0 0" />
+  </joint>
+ <joint name="Mid_Pelvis_Joint" type="fixed">
+    <parent link="Pelvis-link1"/>
+    <child link="Pelvis-link2"/>
     <origin xyz="0 0 ${-l_pelvis*height}" rpy="0 0 0" />
   </joint>
 <!-- Leg joints -->
  <joint name="LHipYaw" type="revolute">
-    <parent link="pelvis-link2"/>
+    <parent link="Pelvis-link2"/>
     <child link="LHipYaw_link"/>
     <origin xyz="0 ${-1*-(o_back_hip_y*height)} 0" rpy="0 0 0"/>
@@ -227,5 +227,5 @@
   </joint>
   <joint name="RHipYaw" type="revolute">
-    <parent link="pelvis-link2"/>
+    <parent link="Pelvis-link2"/>
     <child link="RHipYaw_link"/>
     <origin xyz="0 ${1*-(o_back_hip_y*height)} 0" rpy="0 0 0"/>

Commit message: git-svn-id: https://svn.csail.mit.edu/drc@84 c7283977-0100-402a-a91a-fa70b306dbfe

File: ros_workspace/atlas_description/urdf/atlas_structure.urdf.xacro (robot description, xacro)
@@ -151,5 +151,5 @@
     <child link="LShoulderRoll_link"/>
     <origin xyz="0 0 0" rpy="0 0 0" />
-    <axis xyz="0 0 1"/>
+    <axis xyz="1 0 0"/>
 <limit velocity="3.0" effort="30" lower="${shoulder_adduction_limit*pi_180}" upper="${shoulder_abduction_limit*pi_180}" />
   </joint>
@@ -158,6 +158,6 @@
     <child link="RShoulderRoll_link"/>
     <origin xyz="0 0 0" rpy="0 0 0" />
-    <axis xyz="0 0 1"/>
-<limit velocity="3.0" effort="30" lower="${-shoulder_abduction_limit*pi_180}" upper="${-shoulder_adduction_limit*pi_180}" />
+    <axis xyz="1 0 0"/>
+<limit velocity="3.0" effort="30" lower="-${shoulder_abduction_limit*pi_180}" upper="-${shoulder_adduction_limit*pi_180}" />
   </joint>
  <xacro:macro name="arm_joints" params="side reflect">
@@ -166,5 +166,5 @@
     <child link="${side}ShoulderYaw_link"/>
     <origin xyz="0 ${reflect*-(o_back_shoulder_y*height)} ${o_back_shoulder_z*height}" rpy="0 0 0"/>
-    <axis xyz="1 0 0"/>
+    <axis xyz="0 0 1"/>
     <limit velocity="3.0" effort="30" lower="${shoulder_int_rotation_limit*pi_180}" upper="${shoulder_ext_rotation_limit*pi_180}" />
   </joint>
@@ -187,5 +187,5 @@
     <child link="${side}WristYaw_link"/>
     <origin xyz="0 0 -${(l_lower_arm)*height}" rpy="0 0 0"/>
-    <axis xyz="1 0 0"/>
+    <axis xyz="0 0 1"/>
     <limit velocity="3.0" effort="30" lower="${wrist_int_rotation_limit*pi_180}" upper="${wrist_ext_rotation_limit*pi_180}" />
   </joint>
@@ -197,5 +197,5 @@
     <child link="LWristRoll_link"/>
     <origin xyz="0 0 0" rpy="0 0 0"/>
-    <axis xyz="0 0 1"/>
+    <axis xyz="1 0 0"/>
 <limit velocity="3.0" effort="30" lower="${wrist_adduction_limit*pi_180}" upper="${wrist_abduction_limit*pi_180}" />
   </joint>
@@ -204,5 +204,5 @@
     <child link="RWristRoll_link"/>
     <origin xyz="0 0 0" rpy="0 0 0"/>
-    <axis xyz="0 0 1"/>
+    <axis xyz="1 0 0"/>
 <limit velocity="3.0" effort="30" lower="${-wrist_abduction_limit*pi_180}" upper="${-wrist_adduction_limit*pi_180}" />
   </joint>
@@ -233,19 +233,12 @@
   <limit velocity="3.0" effort="30" lower="${-hip_ext_rotation_limit*pi_180}" upper="${-hip_int_rotation_limit*pi_180}" />
   </joint>
- <!-- <joint name="LHipYaw" type="revolute">
-    <parent link="Back"/>
-    <child link="LHipYaw_link"/>
-    <origin xyz="0 ${-1*-(o_back_hip_y*height)} ${-o_back_hip_z*height}" rpy="0 0 0"/>
+<xacro:macro name="leg_joints" params="side reflect">
+ <!-- <joint name="${side}HipYaw" type="revolute">
+    <parent link="Pelvis-link2"/>
+    <child link="${side}HipYaw_link"/>
+    <origin xyz="0 ${reflect*(o_back_hip_y*height)} 0" rpy="0 0 0"/>
     <axis xyz="0 0 1"/>
   <limit velocity="3.0" effort="30" lower="${hip_int_rotation_limit*pi_180}" upper="${hip_ext_rotation_limit*pi_180}" />
-  </joint>
-  <joint name="RHipYaw" type="revolute">
-    <parent link="Back"/>
-    <child link="RHipYaw_link"/>
-    <origin xyz="0 ${1*-(o_back_hip_y*height)} ${-o_back_hip_z*height}" rpy="0 0 0"/>
-    <axis xyz="0 0 1"/>
-  <limit velocity="3.0" effort="30" lower="${-hip_ext_rotation_limit*pi_180}" upper="${-hip_int_rotation_limit*pi_180}" />
-  </joint> -->
-<xacro:macro name="leg_joints" params="side reflect">
+  </joint>-->
   <joint name="${side}HipPitch" type="revolute">
     <parent link="${side}HipYaw_link"/>
