Commit message: Adding a hovering altas model to atlas_description ros package
git-svn-id: https://svn.csail.mit.edu/drc@130 c7283977-0100-402a-a91a-fa70b306dbfe

File: ros_workspace/atlas_description/urdf/hoveringAtlas.urdf (robot description, URDF)
Before this commit: robot wheeled_atlas, 20 links, 19 joints
Links:
- removed link LbackWheel
- removed link LfrontWheel
- removed link RbackWheel
- removed link RfrontWheel
- added link X_link, mass 121.06
- added link Y_link, mass 121.06
- added link base, mass 121.06; collision box size=0.4 0.4 0.3; visual box size=0.4 0.4 0.3
- link base_link: mass 121.06 -> 10000; geometry collision box size=0.8 0.8 0.02; visual box size=0.8 0.8 0.02
Joints:
- removed joint LbackWheel_joint
- removed joint LfrontWheel_joint
- removed joint RbackWheel_joint
- removed joint RfrontWheel_joint
- added joint Theta_Joint: type continuous, parent Y_link, child base, origin xyz=0 0 0.0 rpy=0 0 0, axis 0 0 1
- added joint X_Joint: type prismatic, parent base_link, child X_link, origin xyz=0 0 0.15 rpy=0 0 0, axis 1 0 0, limit lower=-50 upper=50 effort=200 velocity=30.0
- added joint Y_Joint: type prismatic, parent X_link, child Y_link, origin xyz=0 0 0.0 rpy=0 0 0, axis 0 1 0, limit lower=-50 upper=50 effort=200 velocity=30.0
- joint Base_Torso_joint: parent base_link -> base
- joint LShoulderYaw: parent base_link -> base
- joint RShoulderYaw: parent base_link -> base
