Commit message: added pelvis links to the biped urdf
git-svn-id: https://svn.csail.mit.edu/drc@39 c7283977-0100-402a-a91a-fa70b306dbfe

File: ros_workspace/atlas_description/urdf/atlas_properties.xacro (robot description, xacro)
@@ -20,4 +20,5 @@
 <xacro:property name="mass_power_plant" value="22.0" />
 <xacro:property name="mass_total" value="102.9" />
+<xacro:property name="mass_pelvis" value="5.7" />
 <xacro:property name="mass_foot" value="2.0"/> <!-- made up a value for the foot mass -->
 <!-- proportions -->
@@ -33,8 +34,10 @@
 <xacro:property name="l_ankle" value="0.0243" />
 <xacro:property name="l_foot" value="0.0976" />
+<xacro:property name="l_pelvis" value="0.0854" />
 <!-- guessing the width of stuff -->
 <xacro:property name="w_head" value="0.075" />
 <xacro:property name="w_arm" value="0.02" />
 <xacro:property name="w_leg" value="0.02" />
+<xacro:property name="w_pelvis" value="0.122" />
 <!-- offsets (meters)  -->
 <xacro:property name="o_back_shoulder_y" value="0.135" />

File: ros_workspace/atlas_description/urdf/atlas_robot.urdf (robot description, URDF)
Before this commit: robot atlas, 34 links, 33 joints
Links:
- added link pelvis-link1, mass 5.7; collision cylinder length=0.152491948 radius=0.025; visual cylinder length=0.112491948 radius=0.025
- added link pelvis-link2, mass 0.01; collision cylinder length=0.21784564 radius=0.025; visual cylinder length=0.17784564 radius=0.025
- link LHipRoll_link: mass 9.04175 -> 7.61675
- link LKneePitch_link: mass 9.04175 -> 7.61675
- link RHipRoll_link: mass 9.04175 -> 7.61675
- link RKneePitch_link: mass 9.04175 -> 7.61675
Joints:
- added joint back_pelvis: type fixed, parent back, child pelvis-link1, origin xyz=0 0 0 rpy=0 0 0
- added joint mid_pelvis_dummy: type fixed, parent pelvis-link1, child pelvis-link2, origin xyz=0 0 -0.152491948 rpy=0 0 0
- joint LHipYaw: origin xyz=0 0.10892282 -0.152491948 rpy=0 0 0 -> xyz=0 0.10892282 0 rpy=0 0 0; parent back -> pelvis-link2
- joint RHipYaw: origin xyz=0 -0.10892282 -0.152491948 rpy=0 0 0 -> xyz=0 -0.10892282 0 rpy=0 0 0; parent back -> pelvis-link2

File: ros_workspace/atlas_description/urdf/atlas_structure.urdf.xacro (robot description, xacro)
@@ -14,4 +14,12 @@
     <xacro:insert_small_inertial />
   </link>
+  <link name="pelvis-link1">
+   <xacro:insert_inertial_cuboid mass="${mass_pelvis}" l_x="${0.1*height}" l_y="${w_pelvis*height}" l_z="${l_pelvis*height}"/>
+   <xacro:insert_visualization_pelvis1/>
+  </link>
+  <link name="pelvis-link2">
+   <xacro:insert_small_inertial />
+   <xacro:insert_visualization_pelvis2/>
+  </link>
   <link name="BackYaw_link">
     <xacro:insert_small_inertial />
@@ -70,9 +78,9 @@
   </link>
   <link name="${side}HipRoll_link">
-   <xacro:insert_inertial_cylinder mass="${((mass_pelvis_legs-(2*mass_foot)+mass_misc_div_3)/4)}" r="${(w_leg/2)*height}" l="${l_thigh*height}"/>
+   <xacro:insert_inertial_cylinder mass="${((mass_pelvis_legs-(2*mass_foot)-mass_pelvis+mass_misc_div_3)/4)}" r="${(w_leg/2)*height}" l="${l_thigh*height}"/>
     <xacro:insert_visualization_thigh side="${side}"/>
   </link>
   <link name="${side}KneePitch_link">
-     <xacro:insert_inertial_cylinder mass="${((mass_pelvis_legs-(2*mass_foot)+mass_misc_div_3)/4)}" r="${(w_leg/2)*height}" l="${l_shin*height}"/>
+     <xacro:insert_inertial_cylinder mass="${((mass_pelvis_legs-(2*mass_foot)-mass_pelvis+mass_misc_div_3)/4)}" r="${(w_leg/2)*height}" l="${l_shin*height}"/>
     <xacro:insert_visualization_shin side="${side}"/>
   </link>
@@ -199,6 +207,31 @@
 <limit velocity="3.0" effort="30" lower="${-wrist_abduction_limit*pi_180}" upper="${-wrist_adduction_limit*pi_180}" />
   </joint>
+<!-- Pelvis joints -->
+ <joint name="back_pelvis" type="fixed">
+    <parent link="back"/>
+    <child link="pelvis-link1"/>
+    <origin xyz="0 0 0" rpy="0 0 0" />
+  </joint>
+ <joint name="mid_pelvis_dummy" type="fixed">
+    <parent link="pelvis-link1"/>
+    <child link="pelvis-link2"/>
+    <origin xyz="0 0 ${-l_pelvis*height}" rpy="0 0 0" />
+  </joint>
 <!-- Leg joints -->
-  <joint name="LHipYaw" type="revolute">
+ <joint name="LHipYaw" type="revolute">
+    <parent link="pelvis-link2"/>
+    <child link="LHipYaw_link"/>
+    <origin xyz="0 ${-1*-(o_back_hip_y*height)} 0" rpy="0 0 0"/>
+    <axis xyz="0 0 1"/>
+  <limit velocity="3.0" effort="30" lower="${hip_int_rotation_limit*pi_180}" upper="${hip_ext_rotation_limit*pi_180}" />
+  </joint>
+  <joint name="RHipYaw" type="revolute">
+    <parent link="pelvis-link2"/>
+    <child link="RHipYaw_link"/>
+    <origin xyz="0 ${1*-(o_back_hip_y*height)} 0" rpy="0 0 0"/>
+    <axis xyz="0 0 1"/>
+  <limit velocity="3.0" effort="30" lower="${-hip_ext_rotation_limit*pi_180}" upper="${-hip_int_rotation_limit*pi_180}" />
+  </joint>
+ <!-- <joint name="LHipYaw" type="revolute">
     <parent link="back"/>
     <child link="LHipYaw_link"/>
@@ -213,5 +246,5 @@
     <axis xyz="0 0 1"/>
   <limit velocity="3.0" effort="30" lower="${-hip_ext_rotation_limit*pi_180}" upper="${-hip_int_rotation_limit*pi_180}" />
-  </joint>
+  </joint> -->
 <xacro:macro name="leg_joints" params="side reflect">
   <joint name="${side}HipPitch" type="revolute">

File: ros_workspace/atlas_description/urdf/atlas_visualsandcollision.xacro (robot description, xacro)
@@ -92,4 +92,34 @@
         </collision>
     </xacro:macro>
+    <xacro:macro name="insert_visualization_pelvis1" params="">
+        <visual>
+            <origin xyz="0 0 -${(l_pelvis/2)*height}" rpy="0 0 0"/>
+            <geometry>
+               <cylinder radius="${cylinder_radius}" length="${l_pelvis*height-buffer}"/>
+            </geometry>
+            <material name="LightGrey"/>
+        </visual>
+       <collision>
+            <origin xyz="0 0 -${(l_pelvis/2)*height}" rpy="0 0 0"/>
+            <geometry>
+                <cylinder radius="${cylinder_radius}" length="${l_pelvis*height}"/>
+            </geometry>
+        </collision>
+    </xacro:macro>
+    <xacro:macro name="insert_visualization_pelvis2" params="">
+        <visual>
+            <origin xyz="0 0 0" rpy="${pi_2} 0 0"/>
+            <geometry>
+               <cylinder radius="${cylinder_radius}" length="${w_pelvis*height-buffer}"/>
+            </geometry>
+            <material name="LightGrey"/>
+        </visual>
+       <collision>
+            <origin xyz="0 0 0" rpy="${pi_2} 0 0"/>
+            <geometry>
+                <cylinder radius="${cylinder_radius}" length="${w_pelvis*height}"/>
+            </geometry>
+        </collision>
+    </xacro:macro>
     <xacro:macro name="insert_visualization_thigh" params="side">
         <visual>

Commit message: fixing back joint limits in urdf
git-svn-id: https://svn.csail.mit.edu/drc@65 c7283977-0100-402a-a91a-fa70b306dbfe

File: ros_workspace/atlas_description/urdf/atlas_properties.xacro (robot description, xacro)
@@ -71,5 +71,5 @@
 <xacro:property name="ankle_flexion_limit" value="-40"/>
 <xacro:property name="ankle_extension_limit" value="40"/>
-<xacro:property name="back_flexion_limit" value="-25"/>
+<xacro:property name="back_flexion_limit" value="-35"/>
 <xacro:property name="back_extension_limit" value="25"/>
 <xacro:property name="neck_flexion_limit" value="-45"/>

File: ros_workspace/atlas_description/urdf/atlas_robot.urdf (robot description, URDF)
Before this commit: robot atlas, 36 links, 35 joints
Joints:
- joint BackPitch: limit lower=-0.43633231275 upper=0.43633231275 effort=30 velocity=3.0 -> lower=-0.61086523785 upper=0.43633231275 effort=30 velocity=3.0

Commit message: git-svn-id: https://svn.csail.mit.edu/drc@67 c7283977-0100-402a-a91a-fa70b306dbfe

File: ros_workspace/atlas_description/urdf/atlas_properties.xacro (robot description, xacro)
@@ -76,6 +76,6 @@
 <xacro:property name="neck_extension_limit" value="45"/>
 <!-- The Boston Dynamics slide says flexion is -90 and extension is 50. But the other way makes more sense -->
-<xacro:property name="shoulder_flexion_limit" value="-50"/>
-<xacro:property name="shoulder_extension_limit" value="90"/>
+<xacro:property name="shoulder_flexion_limit" value="-90"/>
+<xacro:property name="shoulder_extension_limit" value="50"/>
 <xacro:property name="elbow_flexion_limit" value="-135"/>
 <xacro:property name="elbow_extension_limit" value="0"/>

File: ros_workspace/atlas_description/urdf/atlas_robot.urdf (robot description, URDF)
Before this commit: robot atlas, 36 links, 35 joints
Joints:
- joint LElbowPitch: origin xyz=0.3481959 0 0 rpy=0 0 0 -> xyz=0 0 -0.3481959 rpy=0 0 0
- joint LShoulderPitch: limit lower=-0.8726646255 upper=1.5707963259 effort=30 velocity=3.0 -> lower=-1.5707963259 upper=0.8726646255 effort=30 velocity=3.0
- joint LWristYaw: origin xyz=0.3035554 0 0 rpy=0 0 0 -> xyz=0 0 -0.3035554 rpy=0 0 0
- joint RElbowPitch: origin xyz=0.3481959 0 0 rpy=0 0 0 -> xyz=0 0 -0.3481959 rpy=0 0 0
- joint RShoulderPitch: limit lower=-0.8726646255 upper=1.5707963259 effort=30 velocity=3.0 -> lower=-1.5707963259 upper=0.8726646255 effort=30 velocity=3.0
- joint RWristYaw: origin xyz=0.3035554 0 0 rpy=0 0 0 -> xyz=0 0 -0.3035554 rpy=0 0 0

File: ros_workspace/atlas_description/urdf/atlas_structure.urdf.xacro (robot description, xacro)
@@ -179,5 +179,5 @@
     <parent link="${side}ShoulderRoll_link"/>
     <child link="${side}ElbowPitch_link"/>
-    <origin xyz="${(l_upper_arm)*height} 0 0" rpy="0 0 0"/>
+    <origin xyz="0 0 -${(l_upper_arm)*height}" rpy="0 0 0"/>
     <axis xyz="0 1 0"/>
     <limit velocity="3.0" effort="30" lower="${elbow_flexion_limit*pi_180}" upper="${elbow_extension_limit*pi_180}"/>
@@ -186,5 +186,5 @@
     <parent link="${side}ElbowPitch_link"/>
     <child link="${side}WristYaw_link"/>
-    <origin xyz="${(l_lower_arm)*height} 0 0" rpy="0 0 0"/>
+    <origin xyz="0 0 -${(l_lower_arm)*height}" rpy="0 0 0"/>
     <axis xyz="1 0 0"/>
     <limit velocity="3.0" effort="30" lower="${wrist_int_rotation_limit*pi_180}" upper="${wrist_ext_rotation_limit*pi_180}" />

File: ros_workspace/atlas_description/urdf/atlas_visualsandcollision.xacro (robot description, xacro)
@@ -49,5 +49,5 @@
     <xacro:macro name="insert_visualization_upper_arm" params="side">
         <visual>
-            <origin xyz="${(l_upper_arm/2)*height} 0 0" rpy="${pi_2} 0 ${pi_2}"/>
+            <origin xyz="0 0 -${(l_upper_arm/2)*height}" rpy="0 0 0"/>
             <geometry>
                 <cylinder radius="${cylinder_radius}" length="${l_upper_arm*height-buffer}"/>
@@ -56,5 +56,5 @@
         </visual>
        <collision>
-            <origin xyz="${(l_upper_arm/2)*height} 0 0" rpy="${pi_2} 0 ${pi_2}"/>
+            <origin xyz="0 0 -${(l_upper_arm/2)*height}" rpy="0 0 0"/>
             <geometry>
                 <cylinder radius="${cylinder_radius}" length="${l_upper_arm*height}"/>
@@ -64,5 +64,5 @@
     <xacro:macro name="insert_visualization_lower_arm" params="side">
         <visual>
-            <origin xyz="${(l_lower_arm/2)*height} 0 0"  rpy="${pi_2} 0 ${pi_2}"/>
+            <origin xyz="0 0 -${(l_lower_arm/2)*height}"  rpy="0 0 0"/>
             <geometry>
                <cylinder radius="${cylinder_radius}" length="${l_lower_arm*height-buffer}"/>
@@ -71,5 +71,5 @@
         </visual>
        <collision>
-            <origin xyz="${(l_lower_arm/2)*height} 0 0"  rpy="${pi_2} 0 ${pi_2}"/>
+            <origin xyz="0 0 -${(l_lower_arm/2)*height}"  rpy="0 0 0"/>
             <geometry>
                 <cylinder radius="${cylinder_radius}" length="${l_lower_arm*height}"/>
@@ -79,5 +79,5 @@
     <xacro:macro name="insert_visualization_hand" params="side">
  	<visual>
-            <origin xyz="${(l_hand/2)*height} 0 0"  rpy="${pi_2} 0 ${pi_2}"/>
+            <origin xyz="0 0 -${(l_hand/2)*height}"  rpy="0 0 0"/>
             <geometry>
                <cylinder radius="${cylinder_radius}" length="${l_hand*height-buffer}"/>
@@ -86,5 +86,5 @@
         </visual>
        <collision>
-            <origin xyz="${(l_hand/2)*height} 0 0"  rpy="${pi_2} 0 ${pi_2}"/>
+             <origin xyz="0 0 -${(l_hand/2)*height}"  rpy="0 0 0"/>
             <geometry>
                 <cylinder radius="${cylinder_radius}" length="${l_hand*height}"/>

Commit message: Modified launch files to suit the latest updates within gazebo
git-svn-id: https://svn.csail.mit.edu/drc@145 c7283977-0100-402a-a91a-fa70b306dbfe

File: ros_workspace/atlas_description/urdf/atlas_properties.xacro (robot description, xacro)
@@ -22,4 +22,5 @@
 <xacro:property name="mass_pelvis" value="5.7" />
 <xacro:property name="mass_foot" value="2.0"/> <!-- made up a value for the foot mass -->
+<xacro:property name="mass_wrist" value="2.0"/> <!-- made up a value for the foot mass -->
 <!-- proportions -->
 <xacro:property name="l_neck_head" value="0.134" />
@@ -37,6 +38,6 @@
 <!-- guessing the width of stuff -->
 <xacro:property name="w_head" value="0.075" />
-<xacro:property name="w_arm" value="0.02" />
-<xacro:property name="w_leg" value="0.02" />
+<xacro:property name="w_arm" value="0.05" />
+<xacro:property name="w_leg" value="0.06" />
 <xacro:property name="w_pelvis" value="0.122" />
 <!-- offsets (meters)  -->
@@ -91,4 +92,27 @@
 <xacro:property name="wrist_int_rotation_limit" value="-85"/>
 <xacro:property name="wrist_ext_rotation_limit" value="85"/>
+<!-- Torque Limits -->
+<xacro:property name="hip_adduction_abduction_torque_limit" value="180"/>
+<xacro:property name="hip_flexion_extension_torque_limit" value="260"/>
+<xacro:property name="hip_int_ext_rotation_torque_limit" value="110"/>
+<xacro:property name="knee_flexion_extension_torque_limit" value="220"/>
+<xacro:property name="ankle_flexion_extension_torque_limit" value="220"/>
+<xacro:property name="back_adduction_abduction_torque_limit" value="100"/>
+<xacro:property name="back_flexion_extension_torque_limit" value="180"/>
+<xacro:property name="back_int_ext_rotation_torque_limit" value="110"/>
+<xacro:property name="neck_flexion_extension_torque_limit" value="25"/>
+<xacro:property name="neck_int_ext_rotation_torque_limit" value="54"/>
+<xacro:property name="shoulder_adduction_abduction_torque_limit" value="110"/>
+<xacro:property name="shoulder_flexion_extension_torque_limit" value="110"/>
+<xacro:property name="shoulder_int_ext_rotation_torque_limit" value="80"/>
+<xacro:property name="elbow_flexion_extension_torque_limit" value="100"/>
+<xacro:property name="wrist_adduction_abduction_torque_limit" value="30"/>
+<xacro:property name="wrist_int_ext_rotation_torque_limit" value="15"/>
+<!-- Velocity Limit -->
+<xacro:property name="joint_velocity_limit" value="3"/>
+<!-- Damping and friction in joints -->
+<!-- Maybe we need one for each type of joint -->
+<xacro:property name="joint_damping" value="100"/>
+<xacro:property name="joint_friction" value="10"/>
 <!-- Macros for inertial properties of simple geometries -->
  <xacro:macro name="insert_inertial_cylinder" params="mass r l">
@@ -127,3 +151,12 @@
     </inertial>
 </xacro:macro>
+ <xacro:macro name="insert_inertial_cylinder2" params="mass mass4inertiatensor r l">
+   <!-- Useful when specifying inertia of multiDOF joints if they are subdivided into individual links, shoulder yaw,pitch,roll-->
+      <inertial>
+         <mass value="${mass}" />
+          <inertia ixx="${(mass4inertiatensor/12)*((3*r*r) + (l*l))}" ixy="0.0" ixz="0.0"
+                   iyy="${(mass4inertiatensor/12)*((3*r*r) + (l*l))}" iyz="0.0"
+                   izz="${(mass4inertiatensor/2)*(r*r)}" />
+        </inertial>
+</xacro:macro>
 </robot>

File: ros_workspace/atlas_description/urdf/atlas_robot.urdf (robot description, URDF)
Before this commit: robot atlas, 36 links, 35 joints
Links:
- link Back: mass 0.01 -> 0.98
- link BackPitch_link: mass 0.01 -> 0.98
- link BackRoll_link: mass 0.01 -> 0.98
- link BackYaw_link: mass 0.01 -> 0.98
- link LAnkle: mass 0.01 -> 1.0
- link LAnklePitch_link: mass 0.01 -> 1.0
- link LElbowPitch_link: mass 4.91675 -> 3.27783333333
- link LHipPitch_link: mass 0.01 -> 3.38522222222
- link LHipRoll_link: mass 7.61675 -> 3.38522222222
- link LHipYaw_link: mass 0.01 -> 3.38522222222
- link LKneePitch_link: mass 7.61675 -> 5.07783333333
- link LShoulderPitch_link: mass 0.01 -> 2.18522222222
- link LShoulderRoll_link: mass 4.91675 -> 2.18522222222
- link LShoulderYaw_link: mass 0.01 -> 2.18522222222
- link LWristRoll_link: mass 0.01 -> 1.0
- link LWristYaw_link: mass 0.01 -> 1.0
- link NeckPitch_link: mass 1.8 -> 0.9
- link NeckYaw_link: mass 0.01 -> 0.9
- link Pelvis-link1: mass 5.7 -> 2.85
- link Pelvis-link2: mass 0.01 -> 2.85
- link RAnkle: mass 0.01 -> 1.0
- link RAnklePitch_link: mass 0.01 -> 1.0
- link RElbowPitch_link: mass 4.91675 -> 3.27783333333
- link RHipPitch_link: mass 0.01 -> 3.38522222222
- link RHipRoll_link: mass 7.61675 -> 3.38522222222
- link RHipYaw_link: mass 0.01 -> 3.38522222222
- link RKneePitch_link: mass 7.61675 -> 5.07783333333
- link RShoulderPitch_link: mass 0.01 -> 2.18522222222
- link RShoulderRoll_link: mass 4.91675 -> 2.18522222222
- link RShoulderYaw_link: mass 0.01 -> 2.18522222222
- link RWristRoll_link: mass 0.01 -> 1.0
- link RWristYaw_link: mass 0.01 -> 1.0
- link Torso: mass 19.267 -> 15.347
Joints:
- joint BackPitch: limit lower=-0.61086523785 upper=0.43633231275 effort=30 velocity=3.0 -> lower=-0.61086523785 upper=0.43633231275 effort=180 velocity=3
- joint BackRoll: limit lower=-0.6981317004 upper=0.6981317004 effort=30 velocity=3.0 -> lower=-0.6981317004 upper=0.6981317004 effort=100 velocity=3
- joint BackYaw: limit lower=-0.78539816295 upper=0.78539816295 effort=30 velocity=3.0 -> lower=-0.78539816295 upper=0.78539816295 effort=110 velocity=3
- joint LAnklePitch: limit lower=-0.6981317004 upper=0.6981317004 effort=30 velocity=3.0 -> lower=-0.6981317004 upper=0.6981317004 effort=220 velocity=3
- joint LElbowPitch: limit lower=-2.35619448885 upper=0.0 effort=30 velocity=3.0 -> lower=-2.35619448885 upper=0.0 effort=100 velocity=3
- joint LHipPitch: limit lower=-1.745329251 upper=0.3490658502 effort=30 velocity=3.0 -> lower=-1.745329251 upper=0.3490658502 effort=260 velocity=3
- joint LHipRoll: limit lower=-0.3490658502 upper=0.3490658502 effort=30 velocity=3.0 -> lower=-0.3490658502 upper=0.3490658502 effort=180 velocity=3
- joint LHipYaw: limit lower=-0.1745329251 upper=1.2217304757 effort=30 velocity=3.0 -> lower=-0.1745329251 upper=1.2217304757 effort=110 velocity=3
- joint LKneePitch: limit lower=0.0 upper=2.35619448885 effort=30 velocity=3.0 -> lower=0.0 upper=2.35619448885 effort=220 velocity=3
- joint LShoulderPitch: limit lower=-1.5707963259 upper=0.8726646255 effort=30 velocity=3.0 -> lower=-1.5707963259 upper=0.8726646255 effort=110 velocity=3
- joint LShoulderRoll: limit lower=0.0 upper=2.00712863865 effort=30 velocity=3.0 -> lower=0.0 upper=2.00712863865 effort=110 velocity=3
- joint LShoulderYaw: limit lower=-0.6981317004 upper=1.745329251 effort=30 velocity=3.0 -> lower=-0.6981317004 upper=1.745329251 effort=80 velocity=3
- joint LWristRoll: limit lower=-0.5235987753 upper=1.0471975506 effort=30 velocity=3.0 -> lower=-0.5235987753 upper=1.0471975506 effort=30 velocity=3
- joint LWristYaw: limit lower=-1.48352986335 upper=1.48352986335 effort=30 velocity=3.0 -> lower=-1.48352986335 upper=1.48352986335 effort=15 velocity=3
- joint NeckPitch: limit lower=-0.78539816295 upper=0.78539816295 effort=30 velocity=3.0 -> lower=-0.78539816295 upper=0.78539816295 effort=25 velocity=3
- joint NeckYaw: limit lower=-1.5707963259 upper=1.5707963259 effort=30 velocity=3.0 -> lower=-1.5707963259 upper=1.5707963259 effort=54 velocity=3
- joint RAnklePitch: limit lower=-0.6981317004 upper=0.6981317004 effort=30 velocity=3.0 -> lower=-0.6981317004 upper=0.6981317004 effort=220 velocity=3
- joint RElbowPitch: limit lower=-2.35619448885 upper=0.0 effort=30 velocity=3.0 -> lower=-2.35619448885 upper=0.0 effort=100 velocity=3
- joint RHipPitch: limit lower=-1.745329251 upper=0.3490658502 effort=30 velocity=3.0 -> lower=-1.745329251 upper=0.3490658502 effort=260 velocity=3
- joint RHipRoll: limit lower=-0.3490658502 upper=0.3490658502 effort=30 velocity=3.0 -> lower=-0.3490658502 upper=0.3490658502 effort=180 velocity=3
- joint RHipYaw: limit lower=-1.2217304757 upper=0.1745329251 effort=30 velocity=3.0 -> lower=-1.2217304757 upper=0.1745329251 effort=110 velocity=3
- joint RKneePitch: limit lower=0.0 upper=2.35619448885 effort=30 velocity=3.0 -> lower=0.0 upper=2.35619448885 effort=220 velocity=3
- joint RShoulderPitch: limit lower=-1.5707963259 upper=0.8726646255 effort=30 velocity=3.0 -> lower=-1.5707963259 upper=0.8726646255 effort=110 velocity=3
- joint RShoulderRoll: limit lower=-2.00712863865 upper=-0.0 effort=30 velocity=3.0 -> lower=-2.00712863865 upper=-0.0 effort=110 velocity=3
- joint RShoulderYaw: limit lower=-0.6981317004 upper=1.745329251 effort=30 velocity=3.0 -> lower=-0.6981317004 upper=1.745329251 effort=80 velocity=3
- joint RWristRoll: limit lower=-1.0471975506 upper=0.5235987753 effort=30 velocity=3.0 -> lower=-1.0471975506 upper=0.5235987753 effort=30 velocity=3
- joint RWristYaw: limit lower=-1.48352986335 upper=1.48352986335 effort=30 velocity=3.0 -> lower=-1.48352986335 upper=1.48352986335 effort=15 velocity=3
