Commit message: Modified launch files to suit the latest updates within gazebo
git-svn-id: https://svn.csail.mit.edu/drc@145 c7283977-0100-402a-a91a-fa70b306dbfe

File: ros_workspace/atlas_description/urdf/atlas_structure.urdf.xacro (robot description, xacro)
@@ -12,56 +12,57 @@
   </link>
   <link name="Back">
-    <xacro:insert_small_inertial />
+   <xacro:insert_inertial_cylinder mass="${0.1*mass_torso_back}" r="${w_pelvis*height}" l="${0.1*height}"/>
   </link>
   <link name="Pelvis-link1">
-   <xacro:insert_inertial_cuboid mass="${mass_pelvis}" l_x="${0.1*height}" l_y="${w_pelvis*height}" l_z="${l_pelvis*height}"/>
+   <xacro:insert_inertial_cuboid mass="${0.5*mass_pelvis}" l_x="${0.1*height}" l_y="${w_pelvis*height}" l_z="${l_pelvis*height}"/>
    <xacro:insert_visualization_pelvis1/>
   </link>
   <link name="Pelvis-link2">
-   <xacro:insert_small_inertial />
+   <xacro:insert_inertial_cuboid mass="${0.5*mass_pelvis}" l_x="${0.1*height}" l_y="${l_pelvis*height}" l_z="${w_pelvis*height}"/>
    <xacro:insert_visualization_pelvis2/>
   </link>
   <link name="BackYaw_link">
-    <xacro:insert_small_inertial />
+   <xacro:insert_inertial_cylinder mass="${0.1*mass_torso_back}" r="${o_back_shoulder_y*height}" l="${0.1*height}"/>
   </link>
   <link name="BackPitch_link">
-    <xacro:insert_small_inertial />
+  <xacro:insert_inertial_cuboid mass="${0.1*mass_torso_back}" l_x="${0.1*height}" l_y="${0.28*height}" l_z="${0.268*height}"/>
   </link>
   <link name="BackRoll_link">
-    <xacro:insert_small_inertial />
+  <xacro:insert_inertial_cuboid mass="${0.1*mass_torso_back}" l_x="${0.1*height}" l_y="${0.28*height}" l_z="${0.268*height}"/>
   </link>
  <link name="Torso" >
    <!-- assuming the rotational inertia of the torso is of a cuboid -->
-  <xacro:insert_inertial_cuboid mass="${mass_torso_back+mass_misc_div_3}" l_x="${0.1*height}" l_y="${0.28*height}" l_z="${0.268*height}"/>
+  <xacro:insert_inertial_cuboid mass="${0.6*mass_torso_back+mass_misc_div_3}" l_x="${0.1*height}" l_y="${0.28*height}" l_z="${0.268*height}"/>
    <xacro:insert_visualization_torso/>
   </link>
   <link name="NeckYaw_link">
-    <xacro:insert_small_inertial />
+  <xacro:insert_inertial_cylinder mass="${0.5*mass_head_neck}" r="${(w_head/2)*height}" l="${l_neck_head*height}"/>
   </link>
   <link name="NeckPitch_link">
-  <xacro:insert_inertial_cylinder mass="${mass_head_neck}" r="${(w_head/2)*height}" l="${l_neck_head*height}"/>
+  <xacro:insert_inertial_cylinder mass="${0.5*mass_head_neck}" r="${(w_head/2)*height}" l="${l_neck_head*height}"/>
   <xacro:insert_visualization_head/>
   </link>
-  <!-- Arms -->
+  <!-- Arms, 2/3 of the weight is in the shoulders and upper arm. 1/3 is in the lower arm -->
   <xacro:macro name="arm_links" params="side reflect">
   <link name = "${side}ShoulderYaw_link">
-   <xacro:insert_small_inertial />
+  <xacro:insert_inertial_cylinder mass="${((mass_arms_hands+mass_misc_div_3)/9)}"
+ r="${(w_arm/2)*height}" l="${l_upper_arm*height}"/>
   </link>
   <link name = "${side}ShoulderPitch_link">
-    <xacro:insert_small_inertial />
-  </link>
+  <xacro:insert_inertial_cylinder mass="${((mass_arms_hands+mass_misc_div_3)/9)}"  r="${(w_arm/2)*height}" l="${l_upper_arm*height}"/>
+   </link>
   <link name = "${side}ShoulderRoll_link">
-  <xacro:insert_inertial_cylinder mass="${((mass_arms_hands+mass_misc_div_3)/4)}" r="${(w_arm/2)*height}" l="${l_upper_arm*height}"/>
+  <xacro:insert_inertial_cylinder mass="${((mass_arms_hands+mass_misc_div_3)/9)}" r="${(w_arm/2)*height}" l="${l_upper_arm*height}"/>
     <xacro:insert_visualization_upper_arm side="${side}"/>
   </link>
   <link name = "${side}ElbowPitch_link">
-  <xacro:insert_inertial_cylinder mass="${((mass_arms_hands+mass_misc_div_3)/4)}" r="${(w_arm/2)*height}" l="${l_lower_arm*height}"/>
+  <xacro:insert_inertial_cylinder mass="${((mass_arms_hands+mass_misc_div_3)/6)}" r="${(w_arm/2)*height}" l="${l_lower_arm*height}"/>
     <xacro:insert_visualization_lower_arm side="${side}"/>
   </link>
   <link name = "${side}WristYaw_link">
-    <xacro:insert_small_inertial />
+    <xacro:insert_inertial_cylinder2 mass="${mass_wrist*0.5}" mass4inertiatensor="${mass_wrist}" r="${(w_arm/2)*height}" l="${l_hand*height}"/>
   </link>
   <link name = "${side}WristRoll_link">
-   <xacro:insert_inertial_cylinder mass="0.01" r="${(w_arm/2)*height}" l="${l_hand*height}"/>
+   <xacro:insert_inertial_cylinder2 mass="${mass_wrist*0.5}" mass4inertiatensor="${mass_wrist}" r="${(w_arm/2)*height}" l="${l_hand*height}"/>
    <xacro:insert_visualization_hand side="${side}"/>
   </link>
@@ -69,26 +70,26 @@
   <xacro:arm_links side="L" reflect="-1"/>
   <xacro:arm_links side="R" reflect="1"/>
-<!-- Legs  -->
+<!-- Legs, 2/3 of the weight is in the hips and thigh and other 1/3 is in the lower leg  -->
 <xacro:macro name="leg_links" params="side reflect">
   <link name="${side}HipYaw_link" >
- 	<xacro:insert_small_inertial />
+   <xacro:insert_inertial_cylinder mass="${((mass_pelvis_legs-(2*mass_foot)-mass_pelvis+mass_misc_div_3)/9)}" r="${(w_leg/2)*height}" l="${l_thigh*height}"/>
   </link>
   <link name="${side}HipPitch_link">
- 	<xacro:insert_small_inertial />
+   <xacro:insert_inertial_cylinder mass="${((mass_pelvis_legs-(2*mass_foot)-mass_pelvis+mass_misc_div_3)/9)}" r="${(w_leg/2)*height}" l="${l_thigh*height}"/>
   </link>
   <link name="${side}HipRoll_link">
-   <xacro:insert_inertial_cylinder mass="${((mass_pelvis_legs-(2*mass_foot)-mass_pelvis+mass_misc_div_3)/4)}" r="${(w_leg/2)*height}" l="${l_thigh*height}"/>
+   <xacro:insert_inertial_cylinder mass="${((mass_pelvis_legs-(2*mass_foot)-mass_pelvis+mass_misc_div_3)/9)}" r="${(w_leg/2)*height}" l="${l_thigh*height}"/>
     <xacro:insert_visualization_thigh side="${side}"/>
   </link>
   <link name="${side}KneePitch_link">
-     <xacro:insert_inertial_cylinder mass="${((mass_pelvis_legs-(2*mass_foot)-mass_pelvis+mass_misc_div_3)/4)}" r="${(w_leg/2)*height}" l="${l_shin*height}"/>
+     <xacro:insert_inertial_cylinder mass="${((mass_pelvis_legs-(2*mass_foot)-mass_pelvis+mass_misc_div_3)/6)}" r="${(w_leg/2)*height}" l="${l_shin*height}"/>
     <xacro:insert_visualization_shin side="${side}"/>
   </link>
   <link name="${side}AnklePitch_link">
-    <xacro:insert_small_inertial />
+    <xacro:insert_inertial_cylinder mass="${1}" r="${cylinder_radius}" l="${l_ankle*height}"/>
     <xacro:insert_visualization_ankle side="${side}"/>
   </link>
   <link name="${side}Ankle">
-    <xacro:insert_small_inertial />
+    <xacro:insert_inertial_cylinder mass="${1}" r="${cylinder_radius}" l="${l_ankle*height}"/>
   </link>
   <link name="${side}Foot">
@@ -110,5 +111,6 @@
     <origin xyz="0 0 0.0" rpy="0 0 0" />
     <axis xyz="0 0 1" />
-    <limit velocity="3.0" effort="30" lower="${back_int_rotation_limit*pi_180}" upper="${back_ext_rotation_limit*pi_180}" />
+    <limit velocity="${joint_velocity_limit}" effort="${back_int_ext_rotation_torque_limit}" lower="${back_int_rotation_limit*pi_180}" upper="${back_ext_rotation_limit*pi_180}" />
+     <dynamics damping="${joint_damping}" friction = "${joint_friction}"/>
   </joint>
   <joint name="BackPitch" type="revolute">
@@ -117,5 +119,6 @@
     <origin xyz="0 0 0" rpy="0 0 0" />
     <axis xyz="0 1 0" />
-    <limit velocity="3.0" effort="30" lower="${back_flexion_limit*pi_180}" upper="${back_extension_limit*pi_180}" />
+    <limit velocity="${joint_velocity_limit}" effort="${back_flexion_extension_torque_limit}" lower="${back_flexion_limit*pi_180}" upper="${back_extension_limit*pi_180}" />
+     <dynamics damping="${joint_damping}" friction = "${joint_friction}"/>
   </joint>
   <joint name="BackRoll" type="revolute">
@@ -124,5 +127,6 @@
     <origin xyz="0 0 0" rpy="0 0 0" />
     <axis xyz="1 0 0" />
-    <limit velocity="3.0" effort="30" lower="${back_adduction_limit*pi_180}" upper="${back_abduction_limit*pi_180}" />
+    <limit velocity="${joint_velocity_limit}" effort="${back_adduction_abduction_torque_limit}" lower="${back_adduction_limit*pi_180}" upper="${back_abduction_limit*pi_180}" />
+     <dynamics damping="${joint_damping}" friction = "${joint_friction}"/>
   </joint>
   <joint name="BackRoll_Torso_joint" type="fixed">
@@ -137,5 +141,6 @@
     <origin xyz="0 0 ${(l_torso)*height}" rpy="0 0 0" />
     <axis xyz="0 0 1" />
-    <limit velocity="3.0" effort="30" lower="${neck_int_rotation_limit*pi_180}" upper="${neck_ext_rotation_limit*pi_180}" />
+    <limit velocity="${joint_velocity_limit}" effort="${neck_int_ext_rotation_torque_limit}" lower="${neck_int_rotation_limit*pi_180}" upper="${neck_ext_rotation_limit*pi_180}" />
+     <dynamics damping="${joint_damping}" friction = "${joint_friction}"/>
   </joint>
   <joint name="NeckPitch" type="revolute">
@@ -144,5 +149,6 @@
     <origin xyz="0 0 0" rpy="0 0 0" />
     <axis xyz="0 1 0" />
-    <limit velocity="3.0" effort="30" lower="${neck_flexion_limit*pi_180}" upper="${neck_extension_limit*pi_180}"/>
+    <limit velocity="${joint_velocity_limit}" effort="${neck_flexion_extension_torque_limit}" lower="${neck_flexion_limit*pi_180}" upper="${neck_extension_limit*pi_180}"/>
+     <dynamics damping="${joint_damping}" friction = "${joint_friction}"/>
   </joint>
 <!-- Arm joints -->
@@ -152,5 +158,6 @@
     <origin xyz="0 0 0" rpy="0 0 0" />
     <axis xyz="1 0 0"/>
-<limit velocity="3.0" effort="30" lower="${shoulder_adduction_limit*pi_180}" upper="${shoulder_abduction_limit*pi_180}" />
+<limit velocity="${joint_velocity_limit}" effort="${shoulder_adduction_abduction_torque_limit}" lower="${shoulder_adduction_limit*pi_180}" upper="${shoulder_abduction_limit*pi_180}" />
+     <dynamics damping="${joint_damping}" friction = "${joint_friction}"/>
   </joint>
   <joint name="RShoulderRoll" type="revolute">
@@ -159,5 +166,6 @@
     <origin xyz="0 0 0" rpy="0 0 0" />
     <axis xyz="1 0 0"/>
-<limit velocity="3.0" effort="30" lower="-${shoulder_abduction_limit*pi_180}" upper="-${shoulder_adduction_limit*pi_180}" />
+<limit velocity="${joint_velocity_limit}" effort="${shoulder_adduction_abduction_torque_limit}" lower="-${shoulder_abduction_limit*pi_180}" upper="-${shoulder_adduction_limit*pi_180}" />
+     <dynamics damping="${joint_damping}" friction = "${joint_friction}"/>
   </joint>
  <xacro:macro name="arm_joints" params="side reflect">
@@ -167,5 +175,6 @@
     <origin xyz="0 ${reflect*-(o_back_shoulder_y*height)} ${o_back_shoulder_z*height}" rpy="0 0 0"/>
     <axis xyz="0 0 1"/>
-    <limit velocity="3.0" effort="30" lower="${shoulder_int_rotation_limit*pi_180}" upper="${shoulder_ext_rotation_limit*pi_180}" />
+    <limit velocity="${joint_velocity_limit}" effort="${shoulder_int_ext_rotation_torque_limit}" lower="${shoulder_int_rotation_limit*pi_180}" upper="${shoulder_ext_rotation_limit*pi_180}" />
+     <dynamics damping="${joint_damping}" friction = "${joint_friction}"/>
   </joint>
   <joint name="${side}ShoulderPitch" type="revolute">
@@ -174,5 +183,6 @@
     <origin xyz="0 0 0" rpy="0 0 0" />
     <axis xyz="0 1 0"/>
-   <limit velocity="3.0" effort="30" lower="${shoulder_flexion_limit*pi_180}" upper="${shoulder_extension_limit*pi_180}" />
+   <limit velocity="${joint_velocity_limit}" effort="${shoulder_flexion_extension_torque_limit}" lower="${shoulder_flexion_limit*pi_180}" upper="${shoulder_extension_limit*pi_180}" />
+     <dynamics damping="${joint_damping}" friction = "${joint_friction}"/>
   </joint>
   <joint name="${side}ElbowPitch" type="revolute">
@@ -181,5 +191,6 @@
     <origin xyz="0 0 -${(l_upper_arm)*height}" rpy="0 0 0"/>
     <axis xyz="0 1 0"/>
-    <limit velocity="3.0" effort="30" lower="${elbow_flexion_limit*pi_180}" upper="${elbow_extension_limit*pi_180}"/>
+    <limit velocity="${joint_velocity_limit}" effort="${elbow_flexion_extension_torque_limit}" lower="${elbow_flexion_limit*pi_180}" upper="${elbow_extension_limit*pi_180}"/>
+     <dynamics damping="${joint_damping}" friction = "${joint_friction}"/>
   </joint>
   <joint name="${side}WristYaw" type="revolute">
@@ -188,5 +199,6 @@
     <origin xyz="0 0 -${(l_lower_arm)*height}" rpy="0 0 0"/>
     <axis xyz="0 0 1"/>
-    <limit velocity="3.0" effort="30" lower="${wrist_int_rotation_limit*pi_180}" upper="${wrist_ext_rotation_limit*pi_180}" />
+    <limit velocity="${joint_velocity_limit}" effort="${wrist_int_ext_rotation_torque_limit}" lower="${wrist_int_rotation_limit*pi_180}" upper="${wrist_ext_rotation_limit*pi_180}" />
+     <dynamics damping="${joint_damping}" friction = "${joint_friction}"/>
   </joint>
   </xacro:macro>
@@ -198,5 +210,6 @@
     <origin xyz="0 0 0" rpy="0 0 0"/>
     <axis xyz="1 0 0"/>
-<limit velocity="3.0" effort="30" lower="${wrist_adduction_limit*pi_180}" upper="${wrist_abduction_limit*pi_180}" />
+<limit velocity="${joint_velocity_limit}" effort="${wrist_adduction_abduction_torque_limit}" lower="${wrist_adduction_limit*pi_180}" upper="${wrist_abduction_limit*pi_180}" />
+     <dynamics damping="${joint_damping}" friction = "${joint_friction}"/>
   </joint>
   <joint name="RWristRoll" type="revolute">
@@ -205,5 +218,6 @@
     <origin xyz="0 0 0" rpy="0 0 0"/>
     <axis xyz="1 0 0"/>
-<limit velocity="3.0" effort="30" lower="${-wrist_abduction_limit*pi_180}" upper="${-wrist_adduction_limit*pi_180}" />
+<limit velocity="${joint_velocity_limit}" effort="${wrist_adduction_abduction_torque_limit}" lower="${-wrist_abduction_limit*pi_180}" upper="${-wrist_adduction_limit*pi_180}" />
+     <dynamics damping="${joint_damping}" friction = "${joint_friction}"/>
   </joint>
 <!-- Pelvis joints -->
@@ -224,5 +238,6 @@
     <origin xyz="0 ${-1*-(o_back_hip_y*height)} 0" rpy="0 0 0"/>
     <axis xyz="0 0 1"/>
-  <limit velocity="3.0" effort="30" lower="${hip_int_rotation_limit*pi_180}" upper="${hip_ext_rotation_limit*pi_180}" />
+  <limit velocity="${joint_velocity_limit}" effort="${hip_int_ext_rotation_torque_limit}" lower="${hip_int_rotation_limit*pi_180}" upper="${hip_ext_rotation_limit*pi_180}" />
+     <dynamics damping="${joint_damping}" friction = "${joint_friction}"/>
   </joint>
   <joint name="RHipYaw" type="revolute">
@@ -231,5 +246,6 @@
     <origin xyz="0 ${1*-(o_back_hip_y*height)} 0" rpy="0 0 0"/>
     <axis xyz="0 0 1"/>
-  <limit velocity="3.0" effort="30" lower="${-hip_ext_rotation_limit*pi_180}" upper="${-hip_int_rotation_limit*pi_180}" />
+  <limit velocity="${joint_velocity_limit}" effort="${hip_int_ext_rotation_torque_limit}" lower="${-hip_ext_rotation_limit*pi_180}" upper="${-hip_int_rotation_limit*pi_180}" />
+     <dynamics damping="${joint_damping}" friction = "${joint_friction}"/>
   </joint>
 <xacro:macro name="leg_joints" params="side reflect">
@@ -239,5 +255,6 @@
     <origin xyz="0 ${reflect*(o_back_hip_y*height)} 0" rpy="0 0 0"/>
     <axis xyz="0 0 1"/>
-  <limit velocity="3.0" effort="30" lower="${hip_int_rotation_limit*pi_180}" upper="${hip_ext_rotation_limit*pi_180}" />
+  <limit velocity="${joint_velocity_limit}" effort="${hip_int_ext_rotation_torque_limit}" lower="${hip_int_rotation_limit*pi_180}" upper="${hip_ext_rotation_limit*pi_180}" />
+     <dynamics damping="${joint_damping}" friction = "${joint_friction}"/>
   </joint>-->
   <joint name="${side}HipPitch" type="revolute">
@@ -246,5 +263,6 @@
     <origin xyz="0 0 0" rpy="0 0 0"/>
     <axis xyz="0 1 0"/>
-      <limit velocity="3.0" effort="30" lower="${hip_flexion_limit*pi_180}" upper="${hip_extension_limit*pi_180}" />
+      <limit velocity="${joint_velocity_limit}" effort="${hip_flexion_extension_torque_limit}" lower="${hip_flexion_limit*pi_180}" upper="${hip_extension_limit*pi_180}" />
+     <dynamics damping="${joint_damping}" friction = "${joint_friction}"/>
   </joint>
   <joint name="${side}HipRoll" type="revolute">
@@ -253,5 +271,6 @@
     <origin xyz="0 0 0" rpy="0 0 0"/>
     <axis xyz="1 0 0"/>
-    <limit velocity="3.0" effort="30" lower="${hip_adduction_limit*pi_180}" upper="${hip_abduction_limit*pi_180}" />
+    <limit velocity="${joint_velocity_limit}" effort="${hip_adduction_abduction_torque_limit}" lower="${hip_adduction_limit*pi_180}" upper="${hip_abduction_limit*pi_180}" />
+     <dynamics damping="${joint_damping}" friction = "${joint_friction}"/>
   </joint>
   <joint name="${side}KneePitch" type="revolute">
@@ -260,5 +279,6 @@
     <origin xyz="0 0 -${(l_thigh)*height}" rpy="0 0 0"/>
     <axis xyz="0 1 0"/>
-    <limit velocity="3.0" effort="30" lower="${knee_flexion_limit*pi_180}" upper="${knee_extension_limit*pi_180}"/>
+    <limit velocity="${joint_velocity_limit}" effort="${knee_flexion_extension_torque_limit}" lower="${knee_flexion_limit*pi_180}" upper="${knee_extension_limit*pi_180}"/>
+     <dynamics damping="${joint_damping}" friction = "${joint_friction}"/>
   </joint>
   <joint name="${side}AnklePitch" type="revolute">
@@ -267,5 +287,6 @@
     <origin xyz="0 0 -${(l_shin)*height}" rpy="0 0 0"/>
     <axis xyz="0 1 0"/>
-    <limit velocity="3.0" effort="30" lower="${ankle_flexion_limit*pi_180}" upper="${ankle_extension_limit*pi_180}"/>
+    <limit velocity="${joint_velocity_limit}" effort="${ankle_flexion_extension_torque_limit}" lower="${ankle_flexion_limit*pi_180}" upper="${ankle_extension_limit*pi_180}"/>
+     <dynamics damping="${joint_damping}" friction = "${joint_friction}"/>
   </joint>
   <joint name="${side}Ankle_joint" type="fixed">

File: ros_workspace/atlas_description/urdf/hoveringAtlas.urdf (robot description, URDF)
Before this commit: robot hovering_atlas, 19 links, 18 joints
Links:
- link LElbowPitch_link: mass 4.91675 -> 3.27783333333
- link LShoulderPitch_link: mass 0.01 -> 2.18522222222
- link LShoulderRoll_link: mass 4.91675 -> 2.18522222222
- link LShoulderYaw_link: mass 0.01 -> 2.18522222222
- link LWristRoll_link: mass 0.01 -> 1.0
- link LWristYaw_link: mass 0.01 -> 1.0
- link NeckPitch_link: mass 1.8 -> 0.9
- link NeckYaw_link: mass 0.01 -> 0.9
- link RElbowPitch_link: mass 4.91675 -> 3.27783333333
- link RShoulderPitch_link: mass 0.01 -> 2.18522222222
- link RShoulderRoll_link: mass 4.91675 -> 2.18522222222
- link RShoulderYaw_link: mass 0.01 -> 2.18522222222
- link RWristRoll_link: mass 0.01 -> 1.0
- link RWristYaw_link: mass 0.01 -> 1.0
Joints:
- joint LElbowPitch: limit lower=-2.35619448885 upper=0.0 effort=30 velocity=3.0 -> lower=-2.35619448885 upper=0.0 effort=100 velocity=3
- joint LShoulderPitch: limit lower=-1.5707963259 upper=0.8726646255 effort=30 velocity=3.0 -> lower=-1.5707963259 upper=0.8726646255 effort=110 velocity=3
- joint LShoulderRoll: limit lower=0.0 upper=2.00712863865 effort=30 velocity=3.0 -> lower=0.0 upper=2.00712863865 effort=110 velocity=3
- joint LShoulderYaw: limit lower=-0.6981317004 upper=1.745329251 effort=30 velocity=3.0 -> lower=-0.6981317004 upper=1.745329251 effort=80 velocity=3
- joint LWristRoll: limit lower=-0.5235987753 upper=1.0471975506 effort=30 velocity=3.0 -> lower=-0.5235987753 upper=1.0471975506 effort=30 velocity=3
- joint LWristYaw: limit lower=-1.48352986335 upper=1.48352986335 effort=30 velocity=3.0 -> lower=-1.48352986335 upper=1.48352986335 effort=15 velocity=3
- joint NeckPitch: limit lower=-0.78539816295 upper=0.78539816295 effort=30 velocity=3.0 -> lower=-0.78539816295 upper=0.78539816295 effort=25 velocity=3
- joint NeckYaw: limit lower=-1.5707963259 upper=1.5707963259 effort=30 velocity=3.0 -> lower=-1.5707963259 upper=1.5707963259 effort=54 velocity=3
- joint RElbowPitch: limit lower=-2.35619448885 upper=0.0 effort=30 velocity=3.0 -> lower=-2.35619448885 upper=0.0 effort=100 velocity=3
- joint RShoulderPitch: limit lower=-1.5707963259 upper=0.8726646255 effort=30 velocity=3.0 -> lower=-1.5707963259 upper=0.8726646255 effort=110 velocity=3
- joint RShoulderRoll: limit lower=-2.00712863865 upper=-0.0 effort=30 velocity=3.0 -> lower=-2.00712863865 upper=-0.0 effort=110 velocity=3
- joint RShoulderYaw: limit lower=-0.6981317004 upper=1.745329251 effort=30 velocity=3.0 -> lower=-0.6981317004 upper=1.745329251 effort=80 velocity=3
- joint RWristRoll: limit lower=-1.0471975506 upper=0.5235987753 effort=30 velocity=3.0 -> lower=-1.0471975506 upper=0.5235987753 effort=30 velocity=3
- joint RWristYaw: limit lower=-1.48352986335 upper=1.48352986335 effort=30 velocity=3.0 -> lower=-1.48352986335 upper=1.48352986335 effort=15 velocity=3
