Commit message: Modified launch files to suit the latest updates within gazebo
git-svn-id: https://svn.csail.mit.edu/drc@145 c7283977-0100-402a-a91a-fa70b306dbfe

File: ros_workspace/atlas_description/urdf/wheeledAtlas.urdf (robot description, URDF)
Before this commit: robot wheeled_atlas, 20 links, 19 joints
Links:
- added link base, mass 121.06; collision box size=0.4 0.4 0.3; visual box size=0.4 0.4 0.3
- link LElbowPitch_link: mass 4.91675 -> 3.27783333333
- link LShoulderPitch_link: mass 0.01 -> 2.18522222222
- link LShoulderRoll_link: mass 4.91675 -> 2.18522222222
- link LShoulderYaw_link: mass 0.01 -> 2.18522222222
- link LWristRoll_link: mass 0.01 -> 1.0
- link LWristYaw_link: mass 0.01 -> 1.0
- link NeckPitch_link: mass 1.8 -> 0.9
- link NeckYaw_link: mass 0.01 -> 0.9
- link RElbowPitch_link: mass 4.91675 -> 3.27783333333
- link RShoulderPitch_link: mass 0.01 -> 2.18522222222
- link RShoulderRoll_link: mass 4.91675 -> 2.18522222222
- link RShoulderYaw_link: mass 0.01 -> 2.18522222222
- link RWristRoll_link: mass 0.01 -> 1.0
- link RWristYaw_link: mass 0.01 -> 1.0
- link base_link: mass 121.06 -> 0.01; geometry 
Joints:
- added joint base_joint: type fixed, parent base_link, child base, origin xyz=0 0 0 rpy=0 0 0
- joint Base_Torso_joint: parent base_link -> base
- joint LElbowPitch: limit lower=-2.35619448885 upper=0.0 effort=30 velocity=3.0 -> lower=-2.35619448885 upper=0.0 effort=100 velocity=3
- joint LShoulderPitch: limit lower=-1.5707963259 upper=0.8726646255 effort=30 velocity=3.0 -> lower=-1.5707963259 upper=0.8726646255 effort=110 velocity=3
- joint LShoulderRoll: limit lower=0.0 upper=2.00712863865 effort=30 velocity=3.0 -> lower=0.0 upper=2.00712863865 effort=110 velocity=3
- joint LShoulderYaw: limit lower=-0.6981317004 upper=1.745329251 effort=30 velocity=3.0 -> lower=-0.6981317004 upper=1.745329251 effort=80 velocity=3; parent base_link -> base
- joint LWristRoll: limit lower=-0.5235987753 upper=1.0471975506 effort=30 velocity=3.0 -> lower=-0.5235987753 upper=1.0471975506 effort=30 velocity=3
- joint LWristYaw: limit lower=-1.48352986335 upper=1.48352986335 effort=30 velocity=3.0 -> lower=-1.48352986335 upper=1.48352986335 effort=15 velocity=3
- joint LbackWheel_joint: parent base_link -> base
- joint LfrontWheel_joint: parent base_link -> base
- joint NeckPitch: limit lower=-0.78539816295 upper=0.78539816295 effort=30 velocity=3.0 -> lower=-0.78539816295 upper=0.78539816295 effort=25 velocity=3
- joint NeckYaw: limit lower=-1.5707963259 upper=1.5707963259 effort=30 velocity=3.0 -> lower=-1.5707963259 upper=1.5707963259 effort=54 velocity=3
- joint RElbowPitch: limit lower=-2.35619448885 upper=0.0 effort=30 velocity=3.0 -> lower=-2.35619448885 upper=0.0 effort=100 velocity=3
- joint RShoulderPitch: limit lower=-1.5707963259 upper=0.8726646255 effort=30 velocity=3.0 -> lower=-1.5707963259 upper=0.8726646255 effort=110 velocity=3
- joint RShoulderRoll: limit lower=-2.00712863865 upper=-0.0 effort=30 velocity=3.0 -> lower=-2.00712863865 upper=-0.0 effort=110 velocity=3
- joint RShoulderYaw: limit lower=-0.6981317004 upper=1.745329251 effort=30 velocity=3.0 -> lower=-0.6981317004 upper=1.745329251 effort=80 velocity=3; parent base_link -> base
- joint RWristRoll: limit lower=-1.0471975506 upper=0.5235987753 effort=30 velocity=3.0 -> lower=-1.0471975506 upper=0.5235987753 effort=30 velocity=3
- joint RWristYaw: limit lower=-1.48352986335 upper=1.48352986335 effort=30 velocity=3.0 -> lower=-1.48352986335 upper=1.48352986335 effort=15 velocity=3
- joint RbackWheel_joint: parent base_link -> base
- joint RfrontWheel_joint: parent base_link -> base

Commit message: added transmission elements to atlas model.  added simple reaching example.  it's painfully slow right now, because it's doing symbolic differentiation of the entire 54-link chain for every timestep for every iteration of the optimization.  will get a lot faster when i implement the analytic gradients (e.g. from posadev)
git-svn-id: https://svn.csail.mit.edu/drc@163 c7283977-0100-402a-a91a-fa70b306dbfe

File: ros_workspace/atlas_description/urdf/atlas_properties.xacro (robot description, xacro)
@@ -113,5 +113,5 @@
 <!-- Damping and friction in joints -->
 <!-- Maybe we need one for each type of joint -->
-<xacro:property name="joint_damping" value="100"/>
+<xacro:property name="joint_damping" value="1"/>
 <xacro:property name="joint_friction" value="10"/>
 <!-- Macros for inertial properties of simple geometries -->

File: ros_workspace/atlas_description/urdf/atlas_structure.urdf.xacro (robot description, xacro)
@@ -101,4 +101,11 @@
   <xacro:leg_links side="R" reflect="1"/>
 <!--   Joints following below -->
+<xacro:macro name="joint_trans" params="joint_name">
+  <transmission type="SimpleTransmission" name="${joint_name}_trans">
+    <actuator name="${joint_name}Torque" />
+    <joint name="${joint_name}" />
+    <mechanicalReduction>1</mechanicalReduction>
+  </transmission>
+</xacro:macro>
   <joint name="base_joint" type="fixed">
     <child link="Back"/>
@@ -114,4 +121,5 @@
      <dynamics damping="${joint_damping}" friction = "${joint_friction}"/>
   </joint>
+  <xacro:joint_trans joint_name="BackYaw"/>
   <joint name="BackPitch" type="revolute">
     <parent link="BackYaw_link"/>
@@ -122,4 +130,5 @@
      <dynamics damping="${joint_damping}" friction = "${joint_friction}"/>
   </joint>
+  <xacro:joint_trans joint_name="BackPitch"/>
   <joint name="BackRoll" type="revolute">
     <parent link="BackPitch_link"/>
@@ -130,4 +139,5 @@
      <dynamics damping="${joint_damping}" friction = "${joint_friction}"/>
   </joint>
+  <xacro:joint_trans joint_name="BackRoll"/>
   <joint name="BackRoll_Torso_joint" type="fixed">
     <child link="Torso"/>
@@ -144,4 +154,5 @@
      <dynamics damping="${joint_damping}" friction = "${joint_friction}"/>
   </joint>
+  <xacro:joint_trans joint_name="NeckYaw"/>
   <joint name="NeckPitch" type="revolute">
     <parent link="NeckYaw_link"/>
@@ -152,4 +163,5 @@
      <dynamics damping="${joint_damping}" friction = "${joint_friction}"/>
   </joint>
+  <xacro:joint_trans joint_name="NeckPitch"/>
 <!-- Arm joints -->
   <joint name="LShoulderRoll" type="revolute">
@@ -161,4 +173,5 @@
      <dynamics damping="${joint_damping}" friction = "${joint_friction}"/>
   </joint>
+  <xacro:joint_trans joint_name="LShoulderRoll"/>
   <joint name="RShoulderRoll" type="revolute">
     <parent link="RShoulderPitch_link"/>
@@ -169,4 +182,5 @@
      <dynamics damping="${joint_damping}" friction = "${joint_friction}"/>
   </joint>
+  <xacro:joint_trans joint_name="RShoulderRoll"/>
  <xacro:macro name="arm_joints" params="side reflect">
   <joint name="${side}ShoulderYaw" type="revolute">
@@ -178,4 +192,5 @@
      <dynamics damping="${joint_damping}" friction = "${joint_friction}"/>
   </joint>
+  <xacro:joint_trans joint_name="${side}ShoulderYaw"/>
   <joint name="${side}ShoulderPitch" type="revolute">
     <parent link="${side}ShoulderYaw_link"/>
@@ -186,4 +201,5 @@
      <dynamics damping="${joint_damping}" friction = "${joint_friction}"/>
   </joint>
+  <xacro:joint_trans joint_name="${side}ShoulderPitch"/>
   <joint name="${side}ElbowPitch" type="revolute">
     <parent link="${side}ShoulderRoll_link"/>
@@ -194,4 +210,5 @@
      <dynamics damping="${joint_damping}" friction = "${joint_friction}"/>
   </joint>
+  <xacro:joint_trans joint_name="${side}ElbowPitch"/>
   <joint name="${side}WristYaw" type="revolute">
     <parent link="${side}ElbowPitch_link"/>
@@ -202,4 +219,5 @@
      <dynamics damping="${joint_damping}" friction = "${joint_friction}"/>
   </joint>
+  <xacro:joint_trans joint_name="${side}WristYaw"/>
   </xacro:macro>
   <xacro:arm_joints side="L" reflect="-1"/>
@@ -213,4 +231,5 @@
      <dynamics damping="${joint_damping}" friction = "${joint_friction}"/>
   </joint>
+  <xacro:joint_trans joint_name="LWristRoll"/>
   <joint name="RWristRoll" type="revolute">
     <parent link="RWristYaw_link"/>
@@ -221,4 +240,5 @@
      <dynamics damping="${joint_damping}" friction = "${joint_friction}"/>
   </joint>
+  <xacro:joint_trans joint_name="RWristRoll"/>
 <!-- Pelvis joints -->
  <joint name="Back_Pelvis_Joint" type="fixed">
@@ -241,4 +261,5 @@
      <dynamics damping="${joint_damping}" friction = "${joint_friction}"/>
   </joint>
+  <xacro:joint_trans joint_name="LHipYaw"/>
   <joint name="RHipYaw" type="revolute">
     <parent link="Pelvis-link2"/>
@@ -249,4 +270,5 @@
      <dynamics damping="${joint_damping}" friction = "${joint_friction}"/>
   </joint>
+  <xacro:joint_trans joint_name="RHipYaw"/>
 <xacro:macro name="leg_joints" params="side reflect">
  <!-- <joint name="${side}HipYaw" type="revolute">
@@ -266,4 +288,5 @@
      <dynamics damping="${joint_damping}" friction = "${joint_friction}"/>
   </joint>
+  <xacro:joint_trans joint_name="${side}HipPitch"/>
   <joint name="${side}HipRoll" type="revolute">
     <parent link="${side}HipPitch_link"/>
@@ -274,4 +297,5 @@
      <dynamics damping="${joint_damping}" friction = "${joint_friction}"/>
   </joint>
+  <xacro:joint_trans joint_name="${side}HipRoll"/>
   <joint name="${side}KneePitch" type="revolute">
     <parent link="${side}HipRoll_link"/>
@@ -282,4 +306,5 @@
      <dynamics damping="${joint_damping}" friction = "${joint_friction}"/>
   </joint>
+  <xacro:joint_trans joint_name="${side}KneePitch"/>
   <joint name="${side}AnklePitch" type="revolute">
     <parent link="${side}KneePitch_link"/>
@@ -290,4 +315,5 @@
      <dynamics damping="${joint_damping}" friction = "${joint_friction}"/>
   </joint>
+  <xacro:joint_trans joint_name="${side}AnklePitch"/>
   <joint name="${side}Ankle_joint" type="fixed">
     <parent link="${side}AnklePitch_link" />
