Commit message: adding a hovering atlas model and plugin code for electric
git-svn-id: https://svn.csail.mit.edu/drc@210 c7283977-0100-402a-a91a-fa70b306dbfe

File: ros_workspace/atlas_description/urdf/hoveringAtlas_pre_fuerte.urdf (robot description, URDF)
Before this commit: robot hovering_atlas, 19 links, 18 joints
Joints:
- joint Theta_Joint: origin xyz=0 0 0.15 rpy=0 0 0 -> xyz=0 0 0.17 rpy=0 0 0
