Commit message: git-svn-id: https://svn.csail.mit.edu/drc@216 c7283977-0100-402a-a91a-fa70b306dbfe

File: ros_workspace/atlas_description/urdf/Pendulum.urdf (robot description, URDF)
Before this commit: robot Pendulum, 2 links, 1 joints
Links:
- removed link world
- added link arm, mass 0.5; visual cylinder length=.75 radius=.01
- added link arm_com, mass 0.5; visual sphere radius=.025
- added link base, mass 100000; visual box size=1 1 1
Joints:
- added joint arm_weld: type fixed, parent arm, child arm_com
- added joint theta: type continuous, parent base, child arm, axis 0 1 0
- joint base_weld: parent world -> base

Commit message: now Gazebo can spawn the pendulum. It is crucial to add the collision tag
git-svn-id: https://svn.csail.mit.edu/drc@217 c7283977-0100-402a-a91a-fa70b306dbfe

File: ros_workspace/atlas_description/urdf/Pendulum.urdf (robot description, URDF)
Before this commit: robot Pendulum, 4 links, 3 joints
Links:
- removed link base
- added link world
- link arm: geometry collision cylinder length=.75 radius=.01; visual cylinder length=.75 radius=.01
- link arm_com: geometry collision sphere radius=.025; visual sphere radius=.025
- link base_part2: geometry collision sphere radius=.015; visual sphere radius=.015
Joints:
- joint base_weld: origin (none) -> xyz=0 0 1; parent base -> world
- joint theta: parent base -> base_part2
