Commit message: Updated ATLAS models to include contact links at the four corners of the foot. Ground reaction force sensing isnt working yet. To be continued...
git-svn-id: https://svn.csail.mit.edu/drc@311 c7283977-0100-402a-a91a-fa70b306dbfe

File: ros_workspace/atlas_description/urdf/atlas_controllers.xacro (robot description, xacro)
@@ -5,7 +5,54 @@
 <robot xmlns:sensor="http://playerstage.sourceforge.net/gazebo/xmlschema/#sensor"
        xmlns:controller="http://playerstage.sourceforge.net/gazebo/xmlschema/#controller"
-       xmlns:interface="http://playerstage.sourceforge.net/gazebo/xmlschema/#interface">
-        <gazebo>
-            <!--<controller:gazebo_ros_p3d name="p3d_base_controller" plugin="libgazebo_ros_p3d.so">
+       xmlns:interface="http://playerstage.sourceforge.net/gazebo/xmlschema/#interface"
+       xmlns:xacro="http://ros.org/wiki/xacro">
+<!--
+    <xacro:macro name="foot_bumpers" params="name">
+	<gazebo reference="${name}_link">
+	<selfCollide>true</selfCollide>
+    	<sensor:contact name="${name}_contact_sensor">
+        <geom>${name}_link_geom</geom>
+       	<updateRate>1.0</updateRate>
+       	<controller:gazebo_ros_bumper name="${name}_gazebo_ros_bumper_controller" plugin="libgazebo_ros_bumper.so">
+       		<alwaysOn>true</alwaysOn>
+       		<updateRate>100.0</updateRate>
+       		<bumperTopicName>${name}_bumper</bumperTopicName>
+       		<interface:bumper name="${name}_bumper_iface" />
+       	</controller:gazebo_ros_bumper>
+   	</sensor:contact>
+	</gazebo>
+	</xacro:macro>
+	<xacro:foot_bumpers name="RHipRoll"/>
+	<xacro:foot_bumpers name="RShoulderRoll"/>
+	<xacro:foot_bumpers name="LFootToeIn"/>
+	<xacro:foot_bumpers name="LFootToeOut"/>
+	<xacro:foot_bumpers name="LFootHeelIn"/>
+	<xacro:foot_bumpers name="LFootHeelOut"/>
+	<xacro:foot_bumpers name="RFootToeIn"/>
+	<xacro:foot_bumpers name="RFootToeOut"/>
+	<xacro:foot_bumpers name="RFootHeelIn"/>
+	<xacro:foot_bumpers name="RFootHeelOut"/>
+-->
+    <xacro:macro name="foot_contact_force" params="name">
+	<gazebo reference="${name}_link">
+        <controller:gazebo_ros_f3d name="${name}_gazebo_ros_f3d_controller" plugin="libgazebo_ros_f3d.so">
+            <alwaysOn>true</alwaysOn>
+            <updateRate>100.0</updateRate>
+            <bodyName>${name}_link</bodyName>
+            <topicName>${name}_f3d</topicName>
+            <interface:position name="{name}_gazebo_ros_f3d_position" />
+        </controller:gazebo_ros_f3d>
+    </gazebo>
+	</xacro:macro>
+	<xacro:foot_contact_force name="LFootToeIn"/>
+	<xacro:foot_contact_force name="LFootToeOut"/>
+	<xacro:foot_contact_force name="LFootHeelIn"/>
+	<xacro:foot_contact_force name="LFootHeelOut"/>
+	<xacro:foot_contact_force name="RFootToeIn"/>
+	<xacro:foot_contact_force name="RFootToeOut"/>
+	<xacro:foot_contact_force name="RFootHeelIn"/>
+	<xacro:foot_contact_force name="RFootHeelOut"/>
+	<gazebo>
+        <!--<controller:gazebo_ros_p3d name="p3d_base_controller" plugin="libgazebo_ros_p3d.so">
                 <alwaysOn>true</alwaysOn>
                 <updateRate>100.0</updateRate>
@@ -30,9 +77,9 @@
        <topicName>actuator_cmd</topicName>
     </controller:joint_actuation_plugin>
-      <controller:gazebo_ros_pub_robot_state name="gazebo_ros_pub_robot_controller" plugin="libgazebo_ros_pub_robot_state.so">
-        <alwaysOn>true</alwaysOn>
-        <updateRate>100.0</updateRate>
-     <topicName>true_robot_state</topicName>
-      </controller:gazebo_ros_pub_robot_state>
-        </gazebo>
+    <controller:gazebo_ros_pub_robot_state name="gazebo_ros_pub_robot_controller" plugin="libgazebo_ros_pub_robot_state.so">
+       <alwaysOn>true</alwaysOn>
+       <updateRate>100.0</updateRate>
+       <topicName>true_robot_state</topicName>
+    </controller:gazebo_ros_pub_robot_state>
+    </gazebo>
 </robot>

File: ros_workspace/atlas_description/urdf/atlas_properties.xacro (robot description, xacro)
@@ -41,4 +41,5 @@
 <xacro:property name="w_leg" value="0.06" />
 <xacro:property name="w_pelvis" value="0.122" />
+<xacro:property name="w_foot" value="0.06" />
 <!-- offsets (meters)  -->
 <xacro:property name="o_back_shoulder_y" value="0.135" />

File: ros_workspace/atlas_description/urdf/atlas_robot.urdf (robot description, URDF)
Before this commit: robot atlas, 36 links, 35 joints
Links:
- added link LFootHeelIn_link, mass 0.01; collision sphere radius=0.0001; visual sphere radius=0.001
- added link LFootHeelOut_link, mass 0.01; collision sphere radius=0.0001; visual sphere radius=0.001
- added link LFootToeIn_link, mass 0.01; collision sphere radius=0.0001; visual sphere radius=0.001
- added link LFootToeOut_link, mass 0.01; collision sphere radius=0.0001; visual sphere radius=0.001
- added link RFootHeelIn_link, mass 0.01; collision sphere radius=0.0001; visual sphere radius=0.001
- added link RFootHeelOut_link, mass 0.01; collision sphere radius=0.0001; visual sphere radius=0.001
- added link RFootToeIn_link, mass 0.01; collision sphere radius=0.0001; visual sphere radius=0.001
- added link RFootToeOut_link, mass 0.01; collision sphere radius=0.0001; visual sphere radius=0.001
Joints:
- added joint LFootHeelIn_joint: type fixed, parent LAnklePitch_link, child LFootHeelIn_link, origin xyz=-0.025 -0.03 -0.04519
- added joint LFootHeelOut_joint: type fixed, parent LAnklePitch_link, child LFootHeelOut_link, origin xyz=-0.025 0.03 -0.04519
- added joint LFootToeIn_joint: type fixed, parent LAnklePitch_link, child LFootToeIn_link, origin xyz=0.199276512 -0.03 -0.04519
- added joint LFootToeOut_joint: type fixed, parent LAnklePitch_link, child LFootToeOut_link, origin xyz=0.199276512 0.03 -0.04519
- added joint RFootHeelIn_joint: type fixed, parent RAnklePitch_link, child RFootHeelIn_link, origin xyz=-0.025 0.03 -0.04519
- added joint RFootHeelOut_joint: type fixed, parent RAnklePitch_link, child RFootHeelOut_link, origin xyz=-0.025 -0.03 -0.04519
- added joint RFootToeIn_joint: type fixed, parent RAnklePitch_link, child RFootToeIn_link, origin xyz=0.199276512 0.03 -0.04519
- added joint RFootToeOut_joint: type fixed, parent RAnklePitch_link, child RFootToeOut_link, origin xyz=0.199276512 -0.03 -0.04519
- joint LFoot_joint: parent LAnkle -> LAnklePitch_link
- joint RFoot_joint: parent RAnkle -> RAnklePitch_link

File: ros_workspace/atlas_description/urdf/atlas_structure.urdf.xacro (robot description, xacro)
@@ -94,7 +94,23 @@
   </link>
   <link name="${side}Foot">
-   <xacro:insert_inertial_cuboid mass="${mass_foot}" l_x="${l_foot*height}" l_y="0.06" l_z="0.015"/>
+    <xacro:insert_inertial_cuboid mass="${mass_foot}" l_x="${l_foot*height}" l_y="0.06" l_z="0.015"/>
     <xacro:insert_visualization_foot side="${side}"/>
-    </link>
+  </link>
+  <link name="${side}FootToeIn_link">
+    <xacro:insert_small_inertial />
+    <xacro:insert_visualization_foot_contact_point side="${side}"/>
+  </link>
+  <link name="${side}FootToeOut_link">
+    <xacro:insert_small_inertial />
+    <xacro:insert_visualization_foot_contact_point side="${side}"/>
+  </link>
+  <link name="${side}FootHeelIn_link">
+    <xacro:insert_small_inertial />
+    <xacro:insert_visualization_foot_contact_point side="${side}"/>
+  </link>
+  <link name="${side}FootHeelOut_link">
+    <xacro:insert_small_inertial />
+    <xacro:insert_visualization_foot_contact_point side="${side}"/>
+  </link>
  </xacro:macro>
   <xacro:leg_links side="L" reflect="-1"/>
@@ -322,7 +338,27 @@
   </joint>
   <joint name="${side}Foot_joint" type="fixed">
-    <parent link="${side}Ankle" />
+    <parent link="${side}AnklePitch_link" />
     <child link="${side}Foot" />
     <origin xyz="0 0 -0.04519" />
+  </joint>
+  <joint name="${side}FootToeIn_joint" type="fixed">
+    <parent link="${side}AnklePitch_link" />
+    <child link="${side}FootToeIn_link" />
+    <origin xyz="${l_foot*height+0.025} ${reflect*w_foot/2} -0.04519" />
+  </joint>
+  <joint name="${side}FootToeOut_joint" type="fixed">
+    <parent link="${side}AnklePitch_link" />
+    <child link="${side}FootToeOut_link" />
+    <origin xyz="${l_foot*height+0.025} ${-reflect*w_foot/2} -0.04519" />
+  </joint>
+  <joint name="${side}FootHeelIn_joint" type="fixed">
+    <parent link="${side}AnklePitch_link" />
+    <child link="${side}FootHeelIn_link" />
+    <origin xyz="-0.025 ${reflect*w_foot/2} -0.04519" />
+  </joint>
+  <joint name="${side}FootHeelOut_joint" type="fixed">
+    <parent link="${side}AnklePitch_link" />
+    <child link="${side}FootHeelOut_link" />
+    <origin xyz="-0.025 ${-reflect*w_foot/2} -0.04519" />
   </joint>
 </xacro:macro>

File: ros_workspace/atlas_description/urdf/atlas_visualsandcollision.xacro (robot description, xacro)
@@ -171,5 +171,5 @@
             <origin xyz="${(l_foot/2)*height} 0 0.0075" rpy="0 0 0"/>
             <geometry>
-                <box size="${l_foot*height+0.05} 0.06 0.015"/>
+                <box size="${l_foot*height+0.05} ${w_foot} 0.015"/>
             </geometry>
             <material name="LightGrey"/>
@@ -178,5 +178,20 @@
            <origin xyz="${(l_foot/2)*height} 0 0.0075" rpy="0 0 0"/>
             <geometry>
-                <box size="${l_foot*height+0.05} 0.06 0.015"/>
+                <box size="${l_foot*height+0.05} ${w_foot} 0.015"/>
+            </geometry>
+        </collision>
+    </xacro:macro>
+    <xacro:macro name="insert_visualization_foot_contact_point" params="side">
+        <visual>
+            <origin xyz="0 0 0" rpy="0 0 0"/>
+            <geometry>
+                <sphere radius="0.001"/>
+            </geometry>
+            <material name="LightGrey"/>
+        </visual>
+       <collision>
+           <origin xyz="0 0 0" rpy="0 0 0"/>
+            <geometry>
+                <sphere radius="0.0001"/> <!-- ~=point contact -->
             </geometry>
         </collision>

Commit message: Some comments in est_robot_state_publisher for Scott
git-svn-id: https://svn.csail.mit.edu/drc@315 c7283977-0100-402a-a91a-fa70b306dbfe

File: ros_workspace/atlas_description/urdf/atlas_controllers.xacro (robot description, xacro)
@@ -7,8 +7,7 @@
        xmlns:interface="http://playerstage.sourceforge.net/gazebo/xmlschema/#interface"
        xmlns:xacro="http://ros.org/wiki/xacro">
-<!--
     <xacro:macro name="foot_bumpers" params="name">
 	<gazebo reference="${name}_link">
-	<selfCollide>true</selfCollide>
+	<selfCollide>false</selfCollide>
     	<sensor:contact name="${name}_contact_sensor">
         <geom>${name}_link_geom</geom>
@@ -23,6 +22,6 @@
 	</gazebo>
 	</xacro:macro>
-	<xacro:foot_bumpers name="RHipRoll"/>
-	<xacro:foot_bumpers name="RShoulderRoll"/>
+<!--	<xacro:foot_bumpers name="RHipRoll"/>-->
+<!--	<xacro:foot_bumpers name="RShoulderRoll"/>-->
 	<xacro:foot_bumpers name="LFootToeIn"/>
 	<xacro:foot_bumpers name="LFootToeOut"/>
@@ -33,24 +32,23 @@
 	<xacro:foot_bumpers name="RFootHeelIn"/>
 	<xacro:foot_bumpers name="RFootHeelOut"/>
--->
-    <xacro:macro name="foot_contact_force" params="name">
-	<gazebo reference="${name}_link">
-        <controller:gazebo_ros_f3d name="${name}_gazebo_ros_f3d_controller" plugin="libgazebo_ros_f3d.so">
-            <alwaysOn>true</alwaysOn>
-            <updateRate>100.0</updateRate>
-            <bodyName>${name}_link</bodyName>
-            <topicName>${name}_f3d</topicName>
-            <interface:position name="{name}_gazebo_ros_f3d_position" />
-        </controller:gazebo_ros_f3d>
-    </gazebo>
-	</xacro:macro>
-	<xacro:foot_contact_force name="LFootToeIn"/>
-	<xacro:foot_contact_force name="LFootToeOut"/>
-	<xacro:foot_contact_force name="LFootHeelIn"/>
-	<xacro:foot_contact_force name="LFootHeelOut"/>
-	<xacro:foot_contact_force name="RFootToeIn"/>
-	<xacro:foot_contact_force name="RFootToeOut"/>
-	<xacro:foot_contact_force name="RFootHeelIn"/>
-	<xacro:foot_contact_force name="RFootHeelOut"/>
+<!--    <xacro:macro name="foot_contact_force" params="name">-->
+<!--	<gazebo reference="${name}_link">-->
+<!--        <controller:gazebo_ros_f3d name="${name}_gazebo_ros_f3d_controller" plugin="libgazebo_ros_f3d.so">-->
+<!--            <alwaysOn>true</alwaysOn>-->
+<!--            <updateRate>100.0</updateRate>-->
+<!--            <bodyName>${name}_link</bodyName>-->
+<!--            <topicName>${name}_f3d</topicName>-->
+<!--            <interface:position name="{name}_gazebo_ros_f3d_position" />-->
+<!--        </controller:gazebo_ros_f3d>-->
+<!--    </gazebo>-->
+<!--	</xacro:macro>-->
+<!--	<xacro:foot_contact_force name="LFootToeIn"/>-->
+<!--	<xacro:foot_contact_force name="LFootToeOut"/>-->
+<!--	<xacro:foot_contact_force name="LFootHeelIn"/>-->
+<!--	<xacro:foot_contact_force name="LFootHeelOut"/>-->
+<!--	<xacro:foot_contact_force name="RFootToeIn"/>-->
+<!--	<xacro:foot_contact_force name="RFootToeOut"/>-->
+<!--	<xacro:foot_contact_force name="RFootHeelIn"/>-->
+<!--	<xacro:foot_contact_force name="RFootHeelOut"/>-->
 	<gazebo>
         <!--<controller:gazebo_ros_p3d name="p3d_base_controller" plugin="libgazebo_ros_p3d.so">

File: ros_workspace/atlas_description/urdf/atlas_controllers_pre_fuerte.xacro (robot description, xacro)
@@ -5,5 +5,31 @@
 <robot xmlns:sensor="http://playerstage.sourceforge.net/gazebo/xmlschema/#sensor"
        xmlns:controller="http://playerstage.sourceforge.net/gazebo/xmlschema/#controller"
-       xmlns:interface="http://playerstage.sourceforge.net/gazebo/xmlschema/#interface">
+       xmlns:interface="http://playerstage.sourceforge.net/gazebo/xmlschema/#interface"
+       xmlns:xacro="http://ros.org/wiki/xacro">
+    <xacro:macro name="foot_bumpers" params="name">
+	<gazebo reference="${name}_link">
+	<selfCollide>false</selfCollide>
+    	<sensor:contact name="${name}_contact_sensor">
+        <geom>${name}_link_geom</geom>
+       	<updateRate>1.0</updateRate>
+       	<controller:gazebo_ros_bumper name="${name}_gazebo_ros_bumper_controller" plugin="libgazebo_ros_bumper.so">
+       		<alwaysOn>true</alwaysOn>
+       		<updateRate>100.0</updateRate>
+       		<bumperTopicName>${name}_bumper</bumperTopicName>
+       		<interface:bumper name="${name}_bumper_iface" />
+       	</controller:gazebo_ros_bumper>
+   	</sensor:contact>
+	</gazebo>
+	</xacro:macro>
+<!--	<xacro:foot_bumpers name="RHipRoll"/>-->
+<!--	<xacro:foot_bumpers name="RShoulderRoll"/>-->
+	<xacro:foot_bumpers name="LFootToeIn"/>
+	<xacro:foot_bumpers name="LFootToeOut"/>
+	<xacro:foot_bumpers name="LFootHeelIn"/>
+	<xacro:foot_bumpers name="LFootHeelOut"/>
+	<xacro:foot_bumpers name="RFootToeIn"/>
+	<xacro:foot_bumpers name="RFootToeOut"/>
+	<xacro:foot_bumpers name="RFootHeelIn"/>
+	<xacro:foot_bumpers name="RFootHeelOut"/>
         <gazebo>
 	<!--

Commit message: added drakeIgnore attribute to foot contact links
git-svn-id: https://svn.csail.mit.edu/drc@382 c7283977-0100-402a-a91a-fa70b306dbfe

File: ros_workspace/atlas_description/urdf/atlas_controllers.xacro (robot description, xacro)
@@ -7,27 +7,4 @@
        xmlns:interface="http://playerstage.sourceforge.net/gazebo/xmlschema/#interface"
        xmlns:xacro="http://ros.org/wiki/xacro">
-    <xacro:macro name="foot_bumpers" params="name">
-	<gazebo reference="${name}_link">
-	<selfCollide>false</selfCollide>
-    	<sensor:contact name="${name}_contact_sensor">
-        <geom>${name}_link_geom</geom>
-        <updateRate>100.0</updateRate>
-       	<controller:gazebo_ros_bumper name="${name}_gazebo_ros_bumper_controller" plugin="libgazebo_ros_bumper.so">
-       		<alwaysOn>true</alwaysOn>
-       		<updateRate>100.0</updateRate>
-       		<bumperTopicName>${name}_bumper</bumperTopicName>
-       		<interface:bumper name="${name}_bumper_iface" />
-       	</controller:gazebo_ros_bumper>
-   	</sensor:contact>
-	</gazebo>
-	</xacro:macro>
-	<xacro:foot_bumpers name="LFootToeIn"/>
-	<xacro:foot_bumpers name="LFootToeOut"/>
-	<xacro:foot_bumpers name="LFootHeelIn"/>
-	<xacro:foot_bumpers name="LFootHeelOut"/>
-	<xacro:foot_bumpers name="RFootToeIn"/>
-	<xacro:foot_bumpers name="RFootToeOut"/>
-	<xacro:foot_bumpers name="RFootHeelIn"/>
-	<xacro:foot_bumpers name="RFootHeelOut"/>
 	<gazebo>
         <!--<controller:gazebo_ros_p3d name="p3d_base_controller" plugin="libgazebo_ros_p3d.so">

File: ros_workspace/atlas_description/urdf/atlas_structure.urdf.xacro (robot description, xacro)
@@ -97,17 +97,17 @@
     <xacro:insert_visualization_foot side="${side}"/>
   </link>
-  <link name="${side}FootToeIn_link">
+  <link name="${side}FootToeIn_link" drakeIgnore="True">
     <xacro:insert_small_inertial />
     <xacro:insert_visualization_foot_contact_point side="${side}"/>
   </link>
-  <link name="${side}FootToeOut_link">
+  <link name="${side}FootToeOut_link" drakeIgnore="True">
     <xacro:insert_small_inertial />
     <xacro:insert_visualization_foot_contact_point side="${side}"/>
   </link>
-  <link name="${side}FootHeelIn_link">
+  <link name="${side}FootHeelIn_link" drakeIgnore="True">
     <xacro:insert_small_inertial />
     <xacro:insert_visualization_foot_contact_point side="${side}"/>
   </link>
-  <link name="${side}FootHeelOut_link">
+  <link name="${side}FootHeelOut_link" drakeIgnore="True">
     <xacro:insert_small_inertial />
     <xacro:insert_visualization_foot_contact_point side="${side}"/>
@@ -342,20 +342,20 @@
     <origin xyz="0 0 -0.04519" />
   </joint>
-  <joint name="${side}FootToeIn_joint" type="fixed">
+  <joint name="${side}FootToeIn_joint" type="fixed" drakeIgnore="True">
     <parent link="${side}AnklePitch_link" />
     <child link="${side}FootToeIn_link" />
     <origin xyz="${l_foot*height+0.025} ${reflect*w_foot/2} -0.04519" />
   </joint>
-  <joint name="${side}FootToeOut_joint" type="fixed">
+  <joint name="${side}FootToeOut_joint" type="fixed" drakeIgnore="True">
     <parent link="${side}AnklePitch_link" />
     <child link="${side}FootToeOut_link" />
     <origin xyz="${l_foot*height+0.025} ${-reflect*w_foot/2} -0.04519" />
   </joint>
-  <joint name="${side}FootHeelIn_joint" type="fixed">
+  <joint name="${side}FootHeelIn_joint" type="fixed" drakeIgnore="True">
     <parent link="${side}AnklePitch_link" />
     <child link="${side}FootHeelIn_link" />
     <origin xyz="-0.025 ${reflect*w_foot/2} -0.04519" />
   </joint>
-  <joint name="${side}FootHeelOut_joint" type="fixed">
+  <joint name="${side}FootHeelOut_joint" type="fixed" drakeIgnore="True">
     <parent link="${side}AnklePitch_link" />
     <child link="${side}FootHeelOut_link" />
