Commit message: Adding two ROS compatible models and changing inertial tag of dummy links
git-svn-id: https://svn.csail.mit.edu/drc@85 c7283977-0100-402a-a91a-fa70b306dbfe

File: ros_workspace/atlas_precursor_models/ROShover.urdf (robot description, URDF)
Before this commit: robot simpleHoverBot, 4 links, 3 joints
Joints:
- joint X: limit effort=200 velocity=30.0 -> lower=-100 upper=100 effort=200 velocity=30.0
- joint Z: limit effort=200 velocity=30.0 -> lower=-100 upper=100 effort=200 velocity=30.0

File: ros_workspace/atlas_precursor_models/ROShover.urdf.xacro (robot description, xacro)
@@ -70,5 +70,5 @@
     <child link="Z_link"/>
     <axis xyz="0 0 1"/>
-    <limit effort="200" velocity="30.0"/>
+    <limit effort="200" velocity="30.0" lower="-100" upper="100"/>
   </joint>
   <joint name="X" type="prismatic">
@@ -76,5 +76,5 @@
     <child link="X_link"/>
     <axis xyz="1 0 0"/>
-    <limit effort="200" velocity="30.0"/>
+    <limit effort="200" velocity="30.0" lower="-100" upper="100"/>
   </joint>
   <joint name="Theta" type="continuous">
