Commit message: correction to atlas urdf
git-svn-id: https://svn.csail.mit.edu/drc@111 c7283977-0100-402a-a91a-fa70b306dbfe

File: models/atlas_robot.urdf (robot description, URDF)
Before this commit: robot atlas, 36 links, 35 joints
Joints:
- joint LShoulderRoll: axis 0 0 1 -> 1 0 0
- joint LShoulderYaw: axis 1 0 0 -> 0 0 1
- joint LWristRoll: axis 0 0 1 -> 1 0 0
- joint LWristYaw: axis 1 0 0 -> 0 0 1
- joint RShoulderRoll: axis 0 0 1 -> 1 0 0
- joint RShoulderYaw: axis 1 0 0 -> 0 0 1
- joint RWristRoll: axis 0 0 1 -> 1 0 0
- joint RWristYaw: axis 1 0 0 -> 0 0 1
