Commit message: Updated diff drive plugins in Electric. The physics for electric and fuerte are like chalk and cheese, this is an issue for tuning controllers.
git-svn-id: https://svn.csail.mit.edu/drc@268 c7283977-0100-402a-a91a-fa70b306dbfe

File: models/wheeledAtlas_pre_fuerte.urdf (robot description, URDF)
Before this commit: robot wheeled_atlas, 21 links, 20 joints
Links:
- link LElbowPitch_link: mass 4.91675 -> 3.27783333333
- link LShoulderPitch_link: mass 0.01 -> 2.18522222222
- link LShoulderRoll_link: mass 4.91675 -> 2.18522222222
- link LShoulderYaw_link: mass 0.01 -> 2.18522222222
- link LWristRoll_link: mass 0.01 -> 1.0
- link LWristYaw_link: mass 0.01 -> 1.0
- link LbackWheel: mass 13.51 -> 103.51
- link LfrontWheel: mass 13.51 -> 103.51
- link NeckPitch_link: mass 1.8 -> 0.9
- link NeckYaw_link: mass 0.01 -> 0.9
- link RElbowPitch_link: mass 4.91675 -> 3.27783333333
- link RShoulderPitch_link: mass 0.01 -> 2.18522222222
- link RShoulderRoll_link: mass 4.91675 -> 2.18522222222
- link RShoulderYaw_link: mass 0.01 -> 2.18522222222
- link RWristRoll_link: mass 0.01 -> 1.0
- link RWristYaw_link: mass 0.01 -> 1.0
- link RbackWheel: mass 13.51 -> 103.51
- link RfrontWheel: mass 13.51 -> 103.51
- link base_link: mass .01 -> 0.01
Joints:
- joint LElbowPitch: limit lower=-2.35619448885 upper=0.0 effort=30 velocity=3.0 -> lower=-2.35619448885 upper=0.0 effort=100 velocity=3
- joint LShoulderPitch: limit lower=-1.5707963259 upper=0.8726646255 effort=30 velocity=3.0 -> lower=-1.5707963259 upper=0.8726646255 effort=110 velocity=3
- joint LShoulderRoll: limit lower=0.0 upper=2.00712863865 effort=30 velocity=3.0 -> lower=0.0 upper=2.00712863865 effort=110 velocity=3
- joint LShoulderYaw: limit lower=-0.6981317004 upper=1.745329251 effort=30 velocity=3.0 -> lower=-0.6981317004 upper=1.745329251 effort=80 velocity=3
- joint LWristRoll: limit lower=-0.5235987753 upper=1.0471975506 effort=30 velocity=3.0 -> lower=-0.5235987753 upper=1.0471975506 effort=30 velocity=3
- joint LWristYaw: limit lower=-1.48352986335 upper=1.48352986335 effort=30 velocity=3.0 -> lower=-1.48352986335 upper=1.48352986335 effort=15 velocity=3
- joint NeckPitch: limit lower=-0.78539816295 upper=0.78539816295 effort=30 velocity=3.0 -> lower=-0.78539816295 upper=0.78539816295 effort=25 velocity=3
- joint NeckYaw: limit lower=-1.5707963259 upper=1.5707963259 effort=30 velocity=3.0 -> lower=-1.5707963259 upper=1.5707963259 effort=54 velocity=3
- joint RElbowPitch: limit lower=-2.35619448885 upper=0.0 effort=30 velocity=3.0 -> lower=-2.35619448885 upper=0.0 effort=100 velocity=3
- joint RShoulderPitch: limit lower=-1.5707963259 upper=0.8726646255 effort=30 velocity=3.0 -> lower=-1.5707963259 upper=0.8726646255 effort=110 velocity=3
- joint RShoulderRoll: limit lower=-2.00712863865 upper=-0.0 effort=30 velocity=3.0 -> lower=-2.00712863865 upper=-0.0 effort=110 velocity=3
- joint RShoulderYaw: limit lower=-0.6981317004 upper=1.745329251 effort=30 velocity=3.0 -> lower=-0.6981317004 upper=1.745329251 effort=80 velocity=3
- joint RWristRoll: limit lower=-1.0471975506 upper=0.5235987753 effort=30 velocity=3.0 -> lower=-1.0471975506 upper=0.5235987753 effort=30 velocity=3
- joint RWristYaw: limit lower=-1.48352986335 upper=1.48352986335 effort=30 velocity=3.0 -> lower=-1.48352986335 upper=1.48352986335 effort=15 velocity=3
