Commit message: changes to ros2lcm_translator_combined to include foot contact sensors. adding a new config file for atlas_robot in electric. Changes to atlas_robot.urdf.xacro
git-svn-id: https://svn.csail.mit.edu/drc@320 c7283977-0100-402a-a91a-fa70b306dbfe

File: models/atlas_robot_pre_fuerte.urdf (robot description, URDF)
Before this commit: robot atlas, 36 links, 35 joints
Links:
- added link LFootHeelIn_link, mass 0.01; collision sphere radius=0.0001; visual sphere radius=0.001
- added link LFootHeelOut_link, mass 0.01; collision sphere radius=0.0001; visual sphere radius=0.001
- added link LFootToeIn_link, mass 0.01; collision sphere radius=0.0001; visual sphere radius=0.001
- added link LFootToeOut_link, mass 0.01; collision sphere radius=0.0001; visual sphere radius=0.001
- added link RFootHeelIn_link, mass 0.01; collision sphere radius=0.0001; visual sphere radius=0.001
- added link RFootHeelOut_link, mass 0.01; collision sphere radius=0.0001; visual sphere radius=0.001
- added link RFootToeIn_link, mass 0.01; collision sphere radius=0.0001; visual sphere radius=0.001
- added link RFootToeOut_link, mass 0.01; collision sphere radius=0.0001; visual sphere radius=0.001
- link Back: mass 0.01 -> 0.98
- link BackPitch_link: mass 0.01 -> 0.98
- link BackRoll_link: mass 0.01 -> 0.98
- link BackYaw_link: mass 0.01 -> 0.98
- link LAnkle: mass 0.01 -> 1.0
- link LAnklePitch_link: mass 0.01 -> 1.0
- link LElbowPitch_link: mass 4.91675 -> 3.27783333333
- link LHipPitch_link: mass 0.01 -> 3.38522222222
- link LHipRoll_link: mass 7.61675 -> 3.38522222222
- link LHipYaw_link: mass 0.01 -> 3.38522222222
- link LKneePitch_link: mass 7.61675 -> 5.07783333333
- link LShoulderPitch_link: mass 0.01 -> 2.18522222222
- link LShoulderRoll_link: mass 4.91675 -> 2.18522222222
- link LShoulderYaw_link: mass 0.01 -> 2.18522222222
- link LWristRoll_link: mass 0.01 -> 1.0
- link LWristYaw_link: mass 0.01 -> 1.0
- link NeckPitch_link: mass 1.8 -> 0.9
- link NeckYaw_link: mass 0.01 -> 0.9
- link Pelvis-link1: mass 5.7 -> 2.85
- link Pelvis-link2: mass 0.01 -> 2.85
- link RAnkle: mass 0.01 -> 1.0
- link RAnklePitch_link: mass 0.01 -> 1.0
- link RElbowPitch_link: mass 4.91675 -> 3.27783333333
- link RHipPitch_link: mass 0.01 -> 3.38522222222
- link RHipRoll_link: mass 7.61675 -> 3.38522222222
- link RHipYaw_link: mass 0.01 -> 3.38522222222
- link RKneePitch_link: mass 7.61675 -> 5.07783333333
- link RShoulderPitch_link: mass 0.01 -> 2.18522222222
- link RShoulderRoll_link: mass 4.91675 -> 2.18522222222
- link RShoulderYaw_link: mass 0.01 -> 2.18522222222
- link RWristRoll_link: mass 0.01 -> 1.0
- link RWristYaw_link: mass 0.01 -> 1.0
- link Torso: mass 19.267 -> 15.347
Joints:
- added joint LFootHeelIn_joint: type fixed, parent LAnklePitch_link, child LFootHeelIn_link, origin xyz=-0.025 -0.03 -0.04519
- added joint LFootHeelOut_joint: type fixed, parent LAnklePitch_link, child LFootHeelOut_link, origin xyz=-0.025 0.03 -0.04519
- added joint LFootToeIn_joint: type fixed, parent LAnklePitch_link, child LFootToeIn_link, origin xyz=0.199276512 -0.03 -0.04519
- added joint LFootToeOut_joint: type fixed, parent LAnklePitch_link, child LFootToeOut_link, origin xyz=0.199276512 0.03 -0.04519
- added joint RFootHeelIn_joint: type fixed, parent RAnklePitch_link, child RFootHeelIn_link, origin xyz=-0.025 0.03 -0.04519
- added joint RFootHeelOut_joint: type fixed, parent RAnklePitch_link, child RFootHeelOut_link, origin xyz=-0.025 -0.03 -0.04519
- added joint RFootToeIn_joint: type fixed, parent RAnklePitch_link, child RFootToeIn_link, origin xyz=0.199276512 0.03 -0.04519
- added joint RFootToeOut_joint: type fixed, parent RAnklePitch_link, child RFootToeOut_link, origin xyz=0.199276512 -0.03 -0.04519
- joint BackPitch: limit lower=-0.61086523785 upper=0.43633231275 effort=30 velocity=3.0 -> lower=-0.61086523785 upper=0.43633231275 effort=180 velocity=3
- joint BackRoll: limit lower=-0.6981317004 upper=0.6981317004 effort=30 velocity=3.0 -> lower=-0.6981317004 upper=0.6981317004 effort=100 velocity=3
- joint BackYaw: limit lower=-0.78539816295 upper=0.78539816295 effort=30 velocity=3.0 -> lower=-0.78539816295 upper=0.78539816295 effort=110 velocity=3
- joint LAnklePitch: limit lower=-0.6981317004 upper=0.6981317004 effort=30 velocity=3.0 -> lower=-0.6981317004 upper=0.6981317004 effort=220 velocity=3
- joint LElbowPitch: limit lower=-2.35619448885 upper=0.0 effort=30 velocity=3.0 -> lower=-2.35619448885 upper=0.0 effort=100 velocity=3
- joint LFoot_joint: parent LAnkle -> LAnklePitch_link
- joint LHipPitch: limit lower=-1.745329251 upper=0.3490658502 effort=30 velocity=3.0 -> lower=-1.745329251 upper=0.3490658502 effort=260 velocity=3
- joint LHipRoll: limit lower=-0.3490658502 upper=0.3490658502 effort=30 velocity=3.0 -> lower=-0.3490658502 upper=0.3490658502 effort=180 velocity=3
- joint LHipYaw: limit lower=-0.1745329251 upper=1.2217304757 effort=30 velocity=3.0 -> lower=-0.1745329251 upper=1.2217304757 effort=110 velocity=3
- joint LKneePitch: limit lower=0.0 upper=2.35619448885 effort=30 velocity=3.0 -> lower=0.0 upper=2.35619448885 effort=220 velocity=3
- joint LShoulderPitch: limit lower=-1.5707963259 upper=0.8726646255 effort=30 velocity=3.0 -> lower=-1.5707963259 upper=0.8726646255 effort=110 velocity=3
- joint LShoulderRoll: limit lower=0.0 upper=2.00712863865 effort=30 velocity=3.0 -> lower=0.0 upper=2.00712863865 effort=110 velocity=3
- joint LShoulderYaw: limit lower=-0.6981317004 upper=1.745329251 effort=30 velocity=3.0 -> lower=-0.6981317004 upper=1.745329251 effort=80 velocity=3
- joint LWristRoll: limit lower=-0.5235987753 upper=1.0471975506 effort=30 velocity=3.0 -> lower=-0.5235987753 upper=1.0471975506 effort=30 velocity=3
- joint LWristYaw: limit lower=-1.48352986335 upper=1.48352986335 effort=30 velocity=3.0 -> lower=-1.48352986335 upper=1.48352986335 effort=15 velocity=3
- joint NeckPitch: limit lower=-0.78539816295 upper=0.78539816295 effort=30 velocity=3.0 -> lower=-0.78539816295 upper=0.78539816295 effort=25 velocity=3
- joint NeckYaw: limit lower=-1.5707963259 upper=1.5707963259 effort=30 velocity=3.0 -> lower=-1.5707963259 upper=1.5707963259 effort=54 velocity=3
- joint RAnklePitch: limit lower=-0.6981317004 upper=0.6981317004 effort=30 velocity=3.0 -> lower=-0.6981317004 upper=0.6981317004 effort=220 velocity=3
- joint RElbowPitch: limit lower=-2.35619448885 upper=0.0 effort=30 velocity=3.0 -> lower=-2.35619448885 upper=0.0 effort=100 velocity=3
- joint RFoot_joint: parent RAnkle -> RAnklePitch_link
- joint RHipPitch: limit lower=-1.745329251 upper=0.3490658502 effort=30 velocity=3.0 -> lower=-1.745329251 upper=0.3490658502 effort=260 velocity=3
- joint RHipRoll: limit lower=-0.3490658502 upper=0.3490658502 effort=30 velocity=3.0 -> lower=-0.3490658502 upper=0.3490658502 effort=180 velocity=3
- joint RHipYaw: limit lower=-1.2217304757 upper=0.1745329251 effort=30 velocity=3.0 -> lower=-1.2217304757 upper=0.1745329251 effort=110 velocity=3
- joint RKneePitch: limit lower=0.0 upper=2.35619448885 effort=30 velocity=3.0 -> lower=0.0 upper=2.35619448885 effort=220 velocity=3
- joint RShoulderPitch: limit lower=-1.5707963259 upper=0.8726646255 effort=30 velocity=3.0 -> lower=-1.5707963259 upper=0.8726646255 effort=110 velocity=3
- joint RShoulderRoll: limit lower=-2.00712863865 upper=-0.0 effort=30 velocity=3.0 -> lower=-2.00712863865 upper=-0.0 effort=110 velocity=3
- joint RShoulderYaw: limit lower=-0.6981317004 upper=1.745329251 effort=30 velocity=3.0 -> lower=-0.6981317004 upper=1.745329251 effort=80 velocity=3
- joint RWristRoll: limit lower=-1.0471975506 upper=0.5235987753 effort=30 velocity=3.0 -> lower=-1.0471975506 upper=0.5235987753 effort=30 velocity=3
- joint RWristYaw: limit lower=-1.48352986335 upper=1.48352986335 effort=30 velocity=3.0 -> lower=-1.48352986335 upper=1.48352986335 effort=15 velocity=3

File: ros_workspace/atlas_description/urdf/atlas_controllers.xacro (robot description, xacro)
@@ -12,5 +12,5 @@
     	<sensor:contact name="${name}_contact_sensor">
         <geom>${name}_link_geom</geom>
-       	<updateRate>1.0</updateRate>
+        <updateRate>100.0</updateRate>
        	<controller:gazebo_ros_bumper name="${name}_gazebo_ros_bumper_controller" plugin="libgazebo_ros_bumper.so">
        		<alwaysOn>true</alwaysOn>
@@ -22,6 +22,4 @@
 	</gazebo>
 	</xacro:macro>
-<!--	<xacro:foot_bumpers name="RHipRoll"/>-->
-<!--	<xacro:foot_bumpers name="RShoulderRoll"/>-->
 	<xacro:foot_bumpers name="LFootToeIn"/>
 	<xacro:foot_bumpers name="LFootToeOut"/>
@@ -32,23 +30,4 @@
 	<xacro:foot_bumpers name="RFootHeelIn"/>
 	<xacro:foot_bumpers name="RFootHeelOut"/>
-<!--    <xacro:macro name="foot_contact_force" params="name">-->
-<!--	<gazebo reference="${name}_link">-->
-<!--        <controller:gazebo_ros_f3d name="${name}_gazebo_ros_f3d_controller" plugin="libgazebo_ros_f3d.so">-->
-<!--            <alwaysOn>true</alwaysOn>-->
-<!--            <updateRate>100.0</updateRate>-->
-<!--            <bodyName>${name}_link</bodyName>-->
-<!--            <topicName>${name}_f3d</topicName>-->
-<!--            <interface:position name="{name}_gazebo_ros_f3d_position" />-->
-<!--        </controller:gazebo_ros_f3d>-->
-<!--    </gazebo>-->
-<!--	</xacro:macro>-->
-<!--	<xacro:foot_contact_force name="LFootToeIn"/>-->
-<!--	<xacro:foot_contact_force name="LFootToeOut"/>-->
-<!--	<xacro:foot_contact_force name="LFootHeelIn"/>-->
-<!--	<xacro:foot_contact_force name="LFootHeelOut"/>-->
-<!--	<xacro:foot_contact_force name="RFootToeIn"/>-->
-<!--	<xacro:foot_contact_force name="RFootToeOut"/>-->
-<!--	<xacro:foot_contact_force name="RFootHeelIn"/>-->
-<!--	<xacro:foot_contact_force name="RFootHeelOut"/>-->
 	<gazebo>
         <!--<controller:gazebo_ros_p3d name="p3d_base_controller" plugin="libgazebo_ros_p3d.so">

File: ros_workspace/atlas_description/urdf/atlas_controllers_pre_fuerte.xacro (robot description, xacro)
@@ -12,5 +12,5 @@
     	<sensor:contact name="${name}_contact_sensor">
         <geom>${name}_link_geom</geom>
-       	<updateRate>1.0</updateRate>
+        <updateRate>100.0</updateRate>
        	<controller:gazebo_ros_bumper name="${name}_gazebo_ros_bumper_controller" plugin="libgazebo_ros_bumper.so">
        		<alwaysOn>true</alwaysOn>
@@ -22,6 +22,4 @@
 	</gazebo>
 	</xacro:macro>
-<!--	<xacro:foot_bumpers name="RHipRoll"/>-->
-<!--	<xacro:foot_bumpers name="RShoulderRoll"/>-->
 	<xacro:foot_bumpers name="LFootToeIn"/>
 	<xacro:foot_bumpers name="LFootToeOut"/>
