Commit message: moved the laser and head forward 10cm
git-svn-id: https://svn.csail.mit.edu/drc@805 c7283977-0100-402a-a91a-fa70b306dbfe

File: software/models/mit_gazebo_models/mit_robot/xacro/drc_skeleton.urdf (robot description, URDF)
Before this commit: robot drc_skeleton, 29 links, 28 joints
Joints:
- joint neck_ay: origin xyz=0.011 0 0.44 rpy=0 -0 0 -> xyz=0.021 0 0.44 rpy=0 -0 0
