Commit message: updating atlas models for drcsim 2.3. includes some significant changes to link masses, inertias, and damping coefficients
git-svn-id: https://svn.csail.mit.edu/drc@2782 c7283977-0100-402a-a91a-fa70b306dbfe

File: software/models/mit_gazebo_models/mit_robot/xacro/atlas_skeleton.urdf (robot description, URDF)
Before this commit: robot drc_skeleton, 28 links, 28 joints
Links:
- link l_foot: mass 0.817 -> 0.867
- link l_lglut: mass 0.69 -> 0.803
- link l_talus: mass 0.817 -> 0.867
- link l_uglut: mass 0.5166 -> 1.51622
- link l_uleg: mass 7.34 -> 7.227
- link ltorso: mass 1.92 -> 1.62729
- link mtorso: mass 0.55 -> 3.8068
- link pelvis: mass 14.2529 -> 12.54638
- link r_foot: mass 0.817 -> 0.867
- link r_lglut: mass 0.69 -> 0.803
- link r_talus: mass 0.817 -> 0.867
- link r_uglut: mass 0.5166 -> 1.51622
- link r_uleg: mass 7.34 -> 7.227
- link utorso: mass 18.484 -> 15.2272

File: software/models/mit_gazebo_models/mit_robot_drake/model_minimal_contact.urdf (robot description, URDF)
Before this commit: robot atlas, 29 links, 28 joints
Links:
- link l_foot: mass 0.817 -> 0.867
- link l_lglut: mass 0.69 -> 0.803
- link l_talus: mass 0.817 -> 0.867
- link l_uglut: mass 0.5166 -> 1.51622
- link l_uleg: mass 7.34 -> 7.227
- link ltorso: mass 1.92 -> 1.62729
- link mtorso: mass 0.55 -> 3.8068
- link pelvis: mass 14.2529 -> 12.54638
- link r_foot: mass 0.817 -> 0.867
- link r_lglut: mass 0.69 -> 0.803
- link r_talus: mass 0.817 -> 0.867
- link r_uglut: mass 0.5166 -> 1.51622
- link r_uleg: mass 7.34 -> 7.227
- link utorso: mass 18.484 -> 15.2272

File: software/models/mit_gazebo_models/mit_robot_drake/model_minimal_contact_with_hands.urdf (robot description, URDF)
Before this commit: robot atlas, 101 links, 100 joints
Links:
- link l_foot: mass 0.817 -> 0.867
- link l_lglut: mass 0.69 -> 0.803
- link l_talus: mass 0.817 -> 0.867
- link l_uglut: mass 0.5166 -> 1.51622
- link l_uleg: mass 7.34 -> 7.227
- link ltorso: mass 1.92 -> 1.62729
- link mtorso: mass 0.55 -> 3.8068
- link pelvis: mass 14.2529 -> 12.54638
- link r_foot: mass 0.817 -> 0.867
- link r_lglut: mass 0.69 -> 0.803
- link r_talus: mass 0.817 -> 0.867
- link r_uglut: mass 0.5166 -> 1.51622
- link r_uleg: mass 7.34 -> 7.227
- link utorso: mass 18.484 -> 15.2272

File: software/models/mit_gazebo_models/mit_robot_drake/xacro/atlas_skeleton_minimal_contact.urdf (robot description, URDF)
Before this commit: robot drc_skeleton, 28 links, 28 joints
Links:
- link l_foot: mass 0.817 -> 0.867
- link l_lglut: mass 0.69 -> 0.803
- link l_talus: mass 0.817 -> 0.867
- link l_uglut: mass 0.5166 -> 1.51622
- link l_uleg: mass 7.34 -> 7.227
- link ltorso: mass 1.92 -> 1.62729
- link mtorso: mass 0.55 -> 3.8068
- link pelvis: mass 14.2529 -> 12.54638
- link r_foot: mass 0.817 -> 0.867
- link r_lglut: mass 0.69 -> 0.803
- link r_talus: mass 0.817 -> 0.867
- link r_uglut: mass 0.5166 -> 1.51622
- link r_uleg: mass 7.34 -> 7.227
- link utorso: mass 18.484 -> 15.2272

File: software/models/mit_gazebo_models/mit_robot_nohands/model.urdf (robot description, URDF)
Before this commit: robot atlas, 41 links, 40 joints
Links:
- link ltorso: mass 1.92 -> 2.0
