Commit message: irobot and sandia fixes
git-svn-id: https://svn.csail.mit.edu/drc/trunk@6719 c7283977-0100-402a-a91a-fa70b306dbfe

File: software/models/mit_gazebo_models/mit_robot/xacro/atlas_irobot_hands.urdf.xacro (robot description, xacro)
@@ -3,4 +3,11 @@
   <include filename="$(find mit_drcsim_scripts)/models/mit_robot/xacro/atlas.transmission" />
   <include filename="$(find mit_drcsim_scripts)/models/multisense_sl/multisense_sl.urdf" />
+  <xacro:include filename="$(find handle_description)/src/irobot_hand_simple.urdf.xacro" />
+  <xacro:irobot_hand side="right" parent="r_hand" reflect="1">
+    <origin rpy="1.57079 0 0" xyz="0 -0.08516 0"/>
+  </xacro:irobot_hand>
+  <xacro:irobot_hand side="left" parent="l_hand" reflect="-1">
+    <origin rpy="1.57079 3.14159 3.14159" xyz="0 0.11516 0"/>
+  </xacro:irobot_hand>
 <!--
 05 sept: Sisir added an offset of 0.045 in the urdf to account
@@ -11,11 +18,7 @@
 0.05 + 0.03516 = 0.08516
 0.1  + 0.03516 = 0.13516
+27 sept: mfallon tested with the left irobot hand on the robot and found
+significant errors in yaw and y. fixed them as best as I could (3-4cm)
+needs to be improved further
 -->
-  <include filename="$(find handle_description)/src/irobot_hand_simple.urdf.xacro" />
-  <xacro:irobot_hand side="right" parent="r_hand" reflect="1">
-    <origin rpy="1.57079 0 0" xyz="0 -0.08516 0"/>
-  </xacro:irobot_hand>
-  <xacro:irobot_hand side="left" parent="l_hand" reflect="-1">
-    <origin rpy="1.57079 0 3.14159" xyz="0 0.08516 0"/>
-  </xacro:irobot_hand>
 </robot>

File: software/models/mit_gazebo_models/mit_robot/xacro/atlas_irobot_left_sandia_right.urdf.xacro (robot description, xacro)
@@ -1,9 +1,10 @@
 <robot xmlns:xacro="http://www.ros.org/wiki/xacro" name="atlas" >
   <xacro:include filename="$(find sandia_hand_description)/urdf/sandia_hand_simple_shapes.urdf.xacro" />
+  <xacro:include filename="$(find handle_description)/src/irobot_hand_simple.urdf.xacro" />
   <xacro:sandia_hand side="right" parent="r_hand" reflect="1" joint_type="revolute" thumb_angle="0">
     <origin xyz="-0.00179 -0.13516 0.01176" rpy="0 0 -1.57079"/>
   </xacro:sandia_hand>
   <xacro:irobot_hand side="left" parent="l_hand" reflect="-1">
-    <origin rpy="1.57079 0 3.14159" xyz="0 0.08516 0"/>
+    <origin rpy="1.57079 3.14159 3.14159" xyz="0 0.11516 0"/>
   </xacro:irobot_hand>
   <include filename="$(find mit_drcsim_scripts)/models/mit_robot/xacro/atlas_skeleton.urdf" />

File: software/models/mit_gazebo_models/mit_robot/xacro/atlas_sandia_left_irobot_right.urdf.xacro (robot description, xacro)
@@ -1,5 +1,5 @@
 <robot xmlns:xacro="http://www.ros.org/wiki/xacro" name="atlas" >
   <xacro:include filename="$(find sandia_hand_description)/urdf/sandia_hand_simple_shapes.urdf.xacro" />
-  <include filename="$(find handle_description)/src/irobot_hand_simple.urdf.xacro" />
+  <xacro:include filename="$(find handle_description)/src/irobot_hand_simple.urdf.xacro" />
   <xacro:sandia_hand side="left" parent="l_hand" reflect="-1" joint_type="revolute" thumb_angle="0">
     <origin xyz="0.00179  0.13516 0.01176" rpy="0 0  1.57079"/>
