Commit message: Added LQ_RH model.  Updated LH_RQ to work with modified pointer xacro
git-svn-id: https://svn.csail.mit.edu/drc/trunk@7908 c7283977-0100-402a-a91a-fa70b306dbfe

File: software/models/mit_gazebo_models/mit_robot/xacro/atlas_LQ_RH.urdf.xacro (robot description, xacro)
@@ -5,16 +5,16 @@
   <xacro:include filename="$(find robotiq_hand_description)/cfg/robotiq_hand.urdf.xacro" />
   <xacro:include filename="$(find hook_description)/src/hook_hand_simple.urdf.xacro" />
-  <link name="right_base_link"/>
-  <joint name="right_base_link_fix" type="fixed">
-    <parent link="r_hand"/>
-    <child link="right_base_link"/>
-    <origin rpy="0 -.5236 3.141" xyz="0 -.19016 -0.015"/>
+  <link name="left_base_link"/>
+  <joint name="left_base_link_fix" type="fixed">
+    <parent link="l_hand"/>
+    <child link="left_base_link"/>
+    <origin rpy="0 -.5236 0" xyz="0 .19016 0.015"/>
   </joint>
-  <xacro:robotiq_hand side="right" parent="right_base_link" reflect="1">
+  <xacro:robotiq_hand side="left" parent="left_base_link" reflect="-1">
 <!--    <origin rpy="0 -.5236 3.141" xyz="0 -.19016 -0.015"/>-->
     <origin rpy="0 0 0" xyz="0 0 0"/>
   </xacro:robotiq_hand>
-  <xacro:hook_hand side="left" parent="l_hand" reflect="-1"  hookflip="1" noof30degoffset="0">
-    <origin rpy="1.57079 3.14159 3.14159" xyz="0 0.11516 0.015"/>
+  <xacro:hook_hand side="right" parent="r_hand" reflect="1"  hookflip="1" noof30degoffset="0">
+    <origin rpy="1.57079 3.14159 0" xyz="0 -0.11516 -0.015"/>
   </xacro:hook_hand>
 </robot>
