Commit message: working towards final hands
git-svn-id: https://svn.csail.mit.edu/drc/trunk@7936 c7283977-0100-402a-a91a-fa70b306dbfe

File: software/models/mit_gazebo_models/mit_robot/xacro/atlas_LI_RR.urdf.xacro (robot description, xacro)
@@ -4,10 +4,10 @@
   <include filename="$(find mit_drcsim_scripts)/models/multisense_sl/multisense_sl.urdf" />
   <xacro:include filename="$(find handle_description)/src/irobot_hand_simple.urdf.xacro" />
-  <xacro:include filename="$(find hook_description)/src/hook_hand_simple.urdf.xacro" />
-  <xacro:irobot_hand side="right" parent="r_hand" reflect="1">
-    <origin rpy="1.57079 2.0944 0" xyz="0 -0.11516 -0.015"/>
+  <xacro:include filename="$(find robotiq_hand_description)/cfg/robotiq_hand.urdf.xacro" />
+  <xacro:irobot_hand side="left" parent="l_hand" reflect="-1">
+    <origin rpy="1.57079 3.14159 3.14159" xyz="0 0.11516 0.015"/>
   </xacro:irobot_hand>
-  <xacro:hook_hand side="left" parent="l_hand" reflect="-1"  hookflip="1"  noof30degoffset="0">
-    <origin rpy="1.57079 3.14159 3.14159" xyz="0 0.11516 0.015"/>
-  </xacro:hook_hand>
+  <xacro:robotiq_hand side="right" parent="r_hand" reflect="1">
+    <origin rpy="0 3.141 3.141" xyz="0 -0.11516 -0.015"/>
+  </xacro:robotiq_hand>
 </robot>

Commit message: removed depreciated hand usages

File: software/models/mit_gazebo_models/mit_robot/xacro/atlas_LI_RR.urdf.xacro (robot description, xacro)
@@ -9,6 +9,6 @@
     <origin rpy="1.57079 3.14159 3.14159" xyz="0 0.11516 0.015"/>
   </xacro:irobot_hand>
-  <xacro:robotiq_hand side="right" parent="r_hand" reflect="1">
-    <origin rpy="0 1.57079 3.141" xyz="0 -0.19016 -0.015"/>
+  <xacro:robotiq_hand side="right" parent="r_hand_force_torque" reflect="1">
+    <origin rpy="0 -1.57079 0" xyz="0 0.06566 0.0"/>
   </xacro:robotiq_hand>
 </robot>

File: software/models/mit_gazebo_models/mit_robot/xacro/atlas_LN_RR.urdf.xacro (robot description, xacro)
@@ -5,6 +5,6 @@
   <include filename="$(find mit_drcsim_scripts)/models/mit_robot/xacro/hand_force_torque.urdf" />
   <xacro:include filename="$(find robotiq_hand_description)/cfg/robotiq_hand.urdf.xacro" />
-  <xacro:robotiq_hand side="right" parent="r_hand" reflect="1">
-    <origin rpy="0 3.141 3.141" xyz="0 -0.11516 -0.015"/>
+  <xacro:robotiq_hand side="right" parent="r_hand_force_torque" reflect="1">
+    <origin rpy="0 -1.57079 0" xyz="0 0.06566 0.0"/>
   </xacro:robotiq_hand>
 </robot>

File: software/models/mit_gazebo_models/mit_robot/xacro/atlas_LP_RR.urdf.xacro (robot description, xacro)
@@ -5,10 +5,10 @@
   <include filename="$(find mit_drcsim_scripts)/models/mit_robot/xacro/hand_force_torque.urdf" />
   <xacro:include filename="$(find hook_description)/src/hook_hand_simple.urdf.xacro" />
-  <xacro:include filename="$(find robotiq_hand_description)/cfg/robotiq_hand.urdf.xacro" />
   <xacro:hook_hand side="left" parent="l_hand" reflect="-1"  hookflip="1"  noof30degoffset="0">
     <origin rpy="1.57079 3.14159 3.14159" xyz="0 0.11516 0.015"/>
   </xacro:hook_hand>
-  <xacro:robotiq_hand side="right" parent="r_hand" reflect="1">
-    <origin rpy="0 3.141 3.141" xyz="0 -0.19016 -0.015"/>
+  <xacro:include filename="$(find robotiq_hand_description)/cfg/robotiq_hand.urdf.xacro" />
+  <xacro:robotiq_hand side="right" parent="r_hand_force_torque" reflect="1">
+    <origin rpy="0 -1.57079 0" xyz="0 0.06566 0.0"/>
   </xacro:robotiq_hand>
 </robot>
