Commit message: Revert "more tweaking URDF stuff for testing"
This reverts commit e345620ef8ccfedfce6b4847732320bd138ed659.

File: software/models/mit_gazebo_models/mit_robot/xacro/hand_force_torque.urdf (robot description, URDF)
Before this commit: robot hand_force_torque, 2 links, 2 joints
Joints:
- joint l_hand_force_torque_joint: origin xyz=0 0.2773 0.0112 rpy=0 0 0 -> xyz=0 0.1245 0.0112 rpy=0 0 0
