Commit message: more tweaking URDF stuff for testing

File: software/models/mit_gazebo_models/mit_robot/xacro/atlas_LR_RR.urdf.xacro (robot description, xacro)
@@ -7,6 +7,5 @@
   <xacro:include filename="$(find robotiq_hand_description)/cfg/robotiq_hand.urdf.xacro" />
   <xacro:robotiq_hand side="left" parent="l_hand_force_torque" reflect="1">
-    <!--origin rpy="0 -1.57079 0" xyz="0 0.06566 0.0"/-->
-    <origin rpy="0 -1.57079 0" xyz="0 0.21846 0.0"/>
+    <origin rpy="0 -1.57079 0" xyz="0 0.06566 0.0"/>
   </xacro:robotiq_hand>
   <xacro:robotiq_hand side="right" parent="r_hand_force_torque" reflect="1">

File: software/models/mit_gazebo_models/mit_robot/xacro/hand_force_torque.urdf (robot description, URDF)
Before this commit: robot hand_force_torque, 2 links, 2 joints
Joints:
- joint l_hand_force_torque_joint: origin xyz=0 0.1245 0.0112 rpy=0 0 0 -> xyz=0 0.2773 0.0112 rpy=0 0 0

Commit message: Removing more un-needed testing changes for URDF

File: software/models/mit_gazebo_models/mit_robot/xacro/atlas_LR_RR.urdf.xacro (robot description, xacro)
@@ -7,6 +7,5 @@
   <xacro:include filename="$(find robotiq_hand_description)/cfg/robotiq_hand.urdf.xacro" />
   <xacro:robotiq_hand side="left" parent="l_hand_force_torque" reflect="1">
-    <!--origin rpy="0 -1.57079 0" xyz="0 0.06566 0.0"/-->
-    <origin rpy="0 -1.57079 0" xyz="0 0.21846 0.0"/>
+    <origin rpy="0 -1.57079 0" xyz="0 0.06566 0.0"/>
   </xacro:robotiq_hand>
   <xacro:robotiq_hand side="right" parent="r_hand_force_torque" reflect="1">
