Commit message: functional sequence of actions to raise the drill and press the button
with a poker ... but beyond basic

File: software/models/mit_gazebo_models/mit_robot/xacro/atlas_LR_RP.urdf.xacro (robot description, xacro)
@@ -7,12 +7,12 @@
   <xacro:include filename="$(find robotiq_camera)/urdf/robotiq_camera.urdf.xacro" />
   <xacro:include filename="$(find hook_description)/src/hook_hand_simple.urdf.xacro" />
-  <xacro:hook_hand side="left" parent="l_hand_force_torque">
+  <xacro:robotiq_hand side="left" parent="l_hand_force_torque" reflect="1">
+    <origin rpy="0 -1.57079 0" xyz="0 0.06566 0.0"/>
+  </xacro:robotiq_hand>
+  <xacro:robotiq_camera  side_letter="l" reflect="1" parent="l_hand_force_torque" >
+    <origin xyz="0.0  0.0 0.0" rpy="0.0 0  0.0"/>
+  </xacro:robotiq_camera>
+  <xacro:hook_hand side="right" parent="r_hand_force_torque">
     <origin rpy="1.57079 3.14159 3.14159" xyz="0 0.0 0.0"/>
   </xacro:hook_hand>
-  <xacro:robotiq_hand side="right" parent="r_hand_force_torque" reflect="1">
-    <origin rpy="0 -1.57079 0" xyz="0 0.06566 0.0"/>
-  </xacro:robotiq_hand>
-  <xacro:robotiq_camera  side_letter="r" reflect="-1" parent="r_hand_force_torque" >
-    <origin xyz="0.0  0.0 0.0" rpy="0.0 0  0.0"/>
-  </xacro:robotiq_camera>
 </robot>
