Commit message: update to planning and control atlas models
git-svn-id: https://svn.csail.mit.edu/drc@885 c7283977-0100-402a-a91a-fa70b306dbfe

File: software/models/mit_gazebo_models/mit_robot_PnC/xacro/atlas.model.xacro (robot description, xacro)
@@ -8,4 +8,5 @@
   <include filename="$(find atlas_utils)/urdf/atlas.transmission" />
   <include filename="$(find atlas_utils)/urdf/atlas.sensors" />
-  <include filename="$(find mit_drcsim_scripts)/models/mit_robot_PnC/xacro/mit_atlas.gazebo" />
+<!--  <include filename="$(find mit_drcsim_scripts)/models/mit_robot_PnC/xacro/mit_atlas.gazebo" /> -->
+  <include filename="$(find mit_drcsim_scripts)/models/mit_robot_PnC/xacro/mit_atlas_position_control.gazebo" />
 </robot>

File: software/models/mit_gazebo_models/mit_robot_PnC/xacro/atlas_skeleton_minimal_contact.urdf (robot description, URDF)
Before this commit: robot drc_skeleton, 29 links, 28 joints
Links:
- added link l_foot_c1, mass 0.001; collision sphere radius=0.001; visual sphere radius=0.001
- added link l_foot_c2, mass 0.001; collision sphere radius=0.001; visual sphere radius=0.001
- added link l_foot_c3, mass 0.001; collision sphere radius=0.001; visual sphere radius=0.001
- added link l_foot_c4, mass 0.001; collision sphere radius=0.001; visual sphere radius=0.001
- added link r_foot_c1, mass 0.001; collision sphere radius=0.001; visual sphere radius=0.001
- added link r_foot_c2, mass 0.001; collision sphere radius=0.001; visual sphere radius=0.001
- added link r_foot_c3, mass 0.001; collision sphere radius=0.001; visual sphere radius=0.001
- added link r_foot_c4, mass 0.001; collision sphere radius=0.001; visual sphere radius=0.001
- link l_foot: geometry visual mesh filename=package://mit_robot/meshes/l_foot.dae scale=1 1 1
- link r_foot: geometry visual mesh filename=package://mit_robot/meshes/r_foot.dae scale=1 1 1
Joints:
- added joint l_foot_j1: type fixed, parent l_foot, child l_foot_c1, origin xyz=0.178 0.032 -0.080 rpy=0 0 0
- added joint l_foot_j2: type fixed, parent l_foot, child l_foot_c2, origin xyz=0.178 -0.032 -0.080 rpy=0 0 0
- added joint l_foot_j3: type fixed, parent l_foot, child l_foot_c3, origin xyz=-0.075 -0.047 -0.081 rpy=0 0 0
- added joint l_foot_j4: type fixed, parent l_foot, child l_foot_c4, origin xyz=-0.075 0.048 -0.081 rpy=0 0 0
- added joint r_foot_j1: type fixed, parent r_foot, child r_foot_c1, origin xyz=0.178 0.032 -0.080 rpy=0 0 0
- added joint r_foot_j2: type fixed, parent r_foot, child r_foot_c2, origin xyz=0.178 -0.032 -0.080 rpy=0 0 0
- added joint r_foot_j3: type fixed, parent r_foot, child r_foot_c3, origin xyz=-0.075 -0.047 -0.081 rpy=0 0 0
- added joint r_foot_j4: type fixed, parent r_foot, child r_foot_c4, origin xyz=-0.075 0.048 -0.081 rpy=0 0 0
