Commit message: committing models for hand
git-svn-id: https://svn.csail.mit.edu/drc@1783 c7283977-0100-402a-a91a-fa70b306dbfe

File: software/models/mit_gazebo_models/mit_robot_PnC/xacro/atlas_sandia_hands.urdf.xacro (robot description, xacro)
@@ -8,7 +8,7 @@
     <origin xyz="0  0.1 0" rpy=" 1.57079 0  1.57079"/>
   </xacro:sandia_hand>
+  <include filename="$(find atlas_description)/urdf/atlas.transmission" />
+  <include filename="$(find mit_drcsim_scripts)/models/multisense_sl/multisense_sl.urdf" />
   <include filename="$(find mit_drcsim_scripts)/models/mit_robot_PnC/xacro/mit_atlas.gazebo" />
-  <include filename="$(find atlas_description)/urdf/atlas.transmission" />
-  <include filename="$(find multisense_sl_description)/urdf/multisense_sl.urdf" />
   <gazebo>
     <!-- include plugin for snadia hands -->

File: software/models/mit_gazebo_models/mit_robot_drake/model_minimal_contact.urdf (robot description, URDF)
Before this commit: robot atlas, 31 links, 30 joints
Links:
- link head: geometry visual mesh filename=/home/mfallon/drc/ros_workspace/mit_drcsim_scripts/models/m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
- link l_clav: geometry visual mesh filename=/home/mfallon/drc/ros_workspace/mit_drcsim_scripts/models/m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 scale=1 1 1
- link l_farm: geometry visual mesh filename=/home/mfallon/drc/ros_workspace/mit_drcsim_scripts/models/m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 scale=1 1 1
- link l_foot: geometry collision sphere radius=0; collision sphere radius=0
- link l_hand: geometry visual mesh filename=/home/mfallon/drc/ros_workspace/mit_drcsim_scripts/models/m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 scale=1 1 1
- link l_larm: geometry visual mesh filename=/home/mfallon/drc/ros_workspace/mit_drcsim_scripts/models/m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 scale=1 1 1
- link l_lglut: geometry visual mesh filename=/home/mfallon/drc/ros_workspace/mit_drcsim_scripts/models/m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 scale=1 1 1
- link l_lleg: geometry visual mesh filename=/home/mfallon/drc/ros_workspace/mit_drcsim_scripts/models/m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 scale=1 1 1
- link l_scap: geometry visual mesh filename=/home/mfallon/drc/ros_workspace/mit_drcsim_scripts/models/m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 scale=1 1 1
- link l_talus: geometry visual mesh filename=/home/mfallon/drc/ros_workspace/mit_drcsim_scripts/models/m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 scale=1 1 1
- link l_uarm: geometry visual mesh filename=/home/mfallon/drc/ros_workspace/mit_drcsim_scripts/models/m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 scale=1 1 1
- link l_uglut: geometry visual mesh filename=/home/mfallon/drc/ros_workspace/mit_drcsim_scripts/models/m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 scale=1 1 1
- link l_uleg: geometry visual mesh filename=/home/mfallon/drc/ros_workspace/mit_drcsim_scripts/models/m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 scale=1 1 1
- link ltorso: geometry visual mesh filename=/home/mfallon/drc/ros_workspace/mit_drcsim_scripts/models/m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 scale=1 1 1
- link mtorso: geometry visual mesh filename=/home/mfallon/drc/ros_workspace/mit_drcsim_scripts/models/m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 scale=1 1 1
- link pelvis: geometry visual mesh filename=/home/mfallon/drc/ros_workspace/mit_drcsim_scripts/models/m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 scale=1 1 1
- link r_clav: geometry visual mesh filename=/home/mfallon/drc/ros_workspace/mit_drcsim_scripts/models/m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 scale=1 1 1
- link r_farm: geometry visual mesh filename=/home/mfallon/drc/ros_workspace/mit_drcsim_scripts/models/m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 scale=1 1 1
- link r_foot: geometry collision sphere radius=0; collision sphere radius=0
- link r_hand: geometry visual mesh filename=/home/mfallon/drc/ros_workspace/mit_drcsim_scripts/models/m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 scale=1 1 1
- link r_larm: geometry visual mesh filename=/home/mfallon/drc/ros_workspace/mit_drcsim_scripts/models/m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 scale=1 1 1
- link r_lglut: geometry visual mesh filename=/home/mfallon/drc/ros_workspace/mit_drcsim_scripts/models/m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 scale=1 1 1
- link r_lleg: geometry visual mesh filename=/home/mfallon/drc/ros_workspace/mit_drcsim_scripts/models/m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 scale=1 1 1
- link r_scap: geometry visual mesh filename=/home/mfallon/drc/ros_workspace/mit_drcsim_scripts/models/m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 scale=1 1 1
- link r_talus: geometry visual mesh filename=/home/mfallon/drc/ros_workspace/mit_drcsim_scripts/models/m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 scale=1 1 1
- link r_uarm: geometry visual mesh filename=/home/mfallon/drc/ros_workspace/mit_drcsim_scripts/models/m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 scale=1 1 1
- link r_uglut: geometry visual mesh filename=/home/mfallon/drc/ros_workspace/mit_drcsim_scripts/models/m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 scale=1 1 1
- link r_uleg: geometry visual mesh filename=/home/mfallon/drc/ros_workspace/mit_drcsim_scripts/models/m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 scale=1 1 1
- link utorso: geometry visual mesh filename=/home/mfallon/drc/ros_workspace/mit_drcsim_scripts/models/m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 scale=1 1 1
