Commit message: removed redundant gazebo include
git-svn-id: https://svn.csail.mit.edu/drc@1838 c7283977-0100-402a-a91a-fa70b306dbfe

File: software/models/mit_gazebo_models/mit_robot_PnC/xacro/atlas.urdf.xacro (robot description, xacro)
@@ -1,17 +1,6 @@
 <robot xmlns:xacro="http://playerstage.sourceforge.net/gazebo/xmlschema/#interface" name="atlas" >
   <include filename="$(find mit_drcsim_scripts)/models/mit_robot_PnC/xacro/atlas_skeleton.urdf" />
-  <include filename="$(find sandia_hand_description)/urdf/sandia_hand_simple_shapes.urdf.xacro" />
-  <xacro:sandia_hand side="right" parent="r_hand" reflect="1">
-    <origin xyz="0 -0.1 0" rpy="-1.57079 0 -1.57079"/>
-  </xacro:sandia_hand>
-  <xacro:sandia_hand side="left" parent="l_hand" reflect="-1">
-    <origin xyz="0  0.1 0" rpy=" 1.57079 0  1.57079"/>
-  </xacro:sandia_hand>
   <include filename="$(find atlas_description)/urdf/atlas.transmission" />
   <include filename="$(find mit_drcsim_scripts)/models/multisense_sl/multisense_sl.urdf" />
   <include filename="$(find mit_drcsim_scripts)/models/mit_robot_PnC/xacro/mit_atlas.gazebo" />
-  <gazebo>
-    <!-- include plugin for snadia hands -->
-    <plugin name="sandia_hand_plugin" filename="libSandiaHandPlugin.so"/>
-  </gazebo>
 </robot>
