Commit message: minor modifications to xacro
git-svn-id: https://svn.csail.mit.edu/drc@1213 c7283977-0100-402a-a91a-fa70b306dbfe

File: software/models/mit_gazebo_models/mit_robot_hands/xacro/sandia_hand_left.urdf.xacro (robot description, xacro)
@@ -25,5 +25,5 @@
   </link>
   <xacro:sandia_hand side="left" parent="base">
-    <origin xyz="0 0 0.5" rpy="0 -1.57079 0"/>
+    <origin xyz="0 0 0.0" rpy="0 -1.57079 0"/>
   </xacro:sandia_hand>
 </robot>

File: software/models/mit_gazebo_models/mit_robot_hands/xacro/sandia_hand_right.urdf.xacro (robot description, xacro)
@@ -25,5 +25,5 @@
   </link>
   <xacro:sandia_hand side="right" parent="base">
-    <origin xyz="0 0 0.5" rpy="0 -1.57079 0"/>
+    <origin xyz="0 0 0.0" rpy="0 -1.57079 0"/>
   </xacro:sandia_hand>
 </robot>
