Commit message: added files to support floating base for sandia hand
git-svn-id: https://svn.csail.mit.edu/drc@1335 c7283977-0100-402a-a91a-fa70b306dbfe

File: software/models/mit_gazebo_models/mit_robot_hands/xacro/sandia_hand_right.urdf.xacro (robot description, xacro)
@@ -3,7 +3,7 @@
        xmlns:interface="http://playerstage.sourceforge.net/gazebo/xmlschema/#interface"
        xmlns:xacro="http://playerstage.sourceforge.net/gazebo/xmlschema/#interface"
-       name="humanoid" >
-  <include filename="$(find sandia_hand_utils)/urdf/sandia_hand.urdf.xacro" />
-  <link name="base">
+       name="sandia_hand" >
+  <include filename="$(find mit_drcsim_scripts)/models/mit_robot_hands/xacro/sandia_hand.xacro" />
+ <!-- <link name="base">
     <inertial>
         <mass value="0.1" />
@@ -11,5 +11,5 @@
         <inertia ixx="0.01" ixy="0" ixz="0" iyy="0.01" iyz="0" izz="0.01" />
     </inertial>
-    <!--<visual>
+    <visual>
         <origin xyz="0 0 0.25" rpy="0 0 0" />
         <geometry>
@@ -22,8 +22,8 @@
             <box size="0.5 0.5 0.5" />
         </geometry>
-    </collision>-->
-  </link>
-  <xacro:sandia_hand side="right" parent="base">
-    <origin xyz="0 0 0.0" rpy="0 -1.57079 0"/>
+    </collision>
+  </link>-->
+  <xacro:sandia_hand side="right" parent="right_base_yaw">
+    <origin xyz="0 0 0" rpy="0 -1.57079 0"/>
   </xacro:sandia_hand>
 </robot>

Commit message: <robot xmlns:sensor="http://playerstage.sourceforge.net/gazebo/xmlschema/#sensor"        xmlns:controller="http://playerstage.sourceforge.net/gazebo/xmlschema/#controller"        xmlns:interface="http://playerstage.sourceforge.net/gazebo/xmlschema/#interface"        xmlns:xacro="http://playerstage.sourceforge.net/gazebo/xmlschema/#interface"        name="sandia_hand" >
  <include filename="$(find sandia_hand_utils)/urdf/sandia_hand.urdf.xacro" />

  <link name="base">
    <inertial>
        <mass value="0.1" />
        <origin xyz="0 0 0.25" rpy="0 0 0" />
        <inertia ixx="0.01" ixy="0" ixz="0" iyy="0.01" iyz="0" izz="0.01" />
    </inertial>
 <!--   <visual>
        <origin xyz="0 0 0.25" rpy="0 0 0" />
        <geometry>
            <box size="0.5 0.5 0.5" />
        </geometry>
    </visual>
    <collision>
        <origin xyz="0 0 0.25" rpy="0 0 0" />
        <geometry>
            <box size="0.5 0.5 0.5" />
        </geometry>
    </collision> -->
  </link>
  <xacro:sandia_hand side="right" parent="base">
    <origin xyz="0 0 0" rpy="0 -1.57079 0"/>
  </xacro:sandia_hand>
</robot>


git-svn-id: https://svn.csail.mit.edu/drc@1344 c7283977-0100-402a-a91a-fa70b306dbfe

File: software/models/mit_gazebo_models/mit_robot_hands/xacro/sandia_hand_right.urdf.xacro (robot description, xacro)
@@ -4,6 +4,6 @@
        xmlns:xacro="http://playerstage.sourceforge.net/gazebo/xmlschema/#interface"
        name="sandia_hand" >
-  <include filename="$(find mit_drcsim_scripts)/models/mit_robot_hands/xacro/sandia_hand.xacro" />
- <!-- <link name="base">
+  <include filename="$(find sandia_hand_utils)/urdf/sandia_hand.urdf.xacro" />
+  <link name="base">
     <inertial>
         <mass value="0.1" />
@@ -11,5 +11,5 @@
         <inertia ixx="0.01" ixy="0" ixz="0" iyy="0.01" iyz="0" izz="0.01" />
     </inertial>
-    <visual>
+ <!--   <visual>
         <origin xyz="0 0 0.25" rpy="0 0 0" />
         <geometry>
@@ -22,7 +22,7 @@
             <box size="0.5 0.5 0.5" />
         </geometry>
-    </collision>
-  </link>-->
-  <xacro:sandia_hand side="right" parent="right_base_yaw">
+    </collision> -->
+  </link>
+  <xacro:sandia_hand side="right" parent="base">
     <origin xyz="0 0 0" rpy="0 -1.57079 0"/>
   </xacro:sandia_hand>
