Commit message: removing an offset in inertial origin. Never used anyway
git-svn-id: https://svn.csail.mit.edu/drc/trunk@6736 c7283977-0100-402a-a91a-fa70b306dbfe

File: software/models/mit_gazebo_models/mit_robot_hands/xacro/irobot_hand_left.urdf.xacro (robot description, xacro)
@@ -8,5 +8,5 @@
     <inertial>
         <mass value="0.1" />
-        <origin xyz="0 0 0.25" rpy="0 0 0" />
+        <origin xyz="0 0 0.0" rpy="0 0 0" />
         <inertia ixx="0.01" ixy="0" ixz="0" iyy="0.01" iyz="0" izz="0.01" />
     </inertial>

File: software/models/mit_gazebo_models/mit_robot_hands/xacro/irobot_hand_right.urdf.xacro (robot description, xacro)
@@ -8,5 +8,5 @@
     <inertial>
         <mass value="0.1" />
-        <origin xyz="0 0 0.25" rpy="0 0 0" />
+        <origin xyz="0 0 0.0" rpy="0 0 0" />
         <inertia ixx="0.01" ixy="0" ixz="0" iyy="0.01" iyz="0" izz="0.01" />
     </inertial>

File: software/models/mit_gazebo_models/mit_robot_hands/xacro/sandia_hand_left.urdf.xacro (robot description, xacro)
@@ -11,5 +11,5 @@
     <inertial>
         <mass value="0.1" />
-        <origin xyz="0 0 0.25" rpy="0 0 0" />
+        <origin xyz="0 0 0.0" rpy="0 0 0" />
         <inertia ixx="0.01" ixy="0" ixz="0" iyy="0.01" iyz="0" izz="0.01" />
     </inertial>

File: software/models/mit_gazebo_models/mit_robot_hands/xacro/sandia_hand_right.urdf.xacro (robot description, xacro)
@@ -11,5 +11,5 @@
     <inertial>
         <mass value="0.1" />
-        <origin xyz="0 0 0.25" rpy="0 0 0" />
+        <origin xyz="0 0 0.0" rpy="0 0 0" />
         <inertia ixx="0.01" ixy="0" ixz="0" iyy="0.01" iyz="0" izz="0.01" />
     </inertial>
