Commit message: git-svn-id: https://svn.csail.mit.edu/drc/trunk@7755 c7283977-0100-402a-a91a-fa70b306dbfe

File: software/models/mit_gazebo_models/mit_robot_hands/xacro/inert_hand_left.urdf.xacro (robot description, xacro)
@@ -11,11 +11,7 @@
     </inertial>
   </link>
- <xacro:include filename="$(find hook_description)/src/hook_hand_simple.urdf.xacro" />
+ <xacro:include filename="$(find hook_description)/src/bdihook_hand.urdf.xacro" />
   <xacro:hook_hand side="left" parent="plane::xy::base" reflect="-1" hookflip="1">
     <origin rpy="1.57 0.0 -1.57" xyz="0.0 0.0 0.0"/>
-  </xacro:hook_hand>
-<!-- <xacro:include filename="$(find hook_description)/src/bdihook_hand.urdf.xacro" />-->
-<!--  <xacro:hook_hand side="left" parent="plane::xy::base" reflect="-1" hookflip="1">-->
-<!--    <origin rpy="1.57 0.0 -1.57" xyz="0.0 0.0 0.0"/>-->
-<!--  </xacro:hook_hand>-->
+ </xacro:hook_hand>
 </robot>

File: software/models/mit_gazebo_models/mit_robot_hands/xacro/new_not_integrated/pointer_hand_left.urdf.xacro (robot description, xacro)
@@ -3,5 +3,5 @@
        xmlns:interface="http://playerstage.sourceforge.net/gazebo/xmlschema/#interface"
        xmlns:xacro="http://playerstage.sourceforge.net/gazebo/xmlschema/#interface"
-       name="inert_hand_right" >
+       name="inert_hand_left" >
   <link name="plane::xy::base">
     <inertial>
@@ -11,7 +11,7 @@
     </inertial>
   </link>
-  <xacro:include filename="$(find hook_description)/src/bdihook_hand.urdf.xacro" />
-   <xacro:hook_hand side="right" parent="plane::xy::base" reflect="1" hookflip="1">
-     <origin rpy="1.57 3.14 -1.57" xyz="0 0 0"/>
+ <xacro:include filename="$(find hook_description)/src/hook_hand_simple.urdf.xacro" />
+  <xacro:hook_hand side="left" parent="plane::xy::base" reflect="-1" hookflip="1">
+    <origin rpy="1.57 0.0 -1.57" xyz="0.0 0.0 0.0"/>
   </xacro:hook_hand>
 </robot>

File: software/models/mit_gazebo_models/mit_robot_hands/xacro/new_not_integrated/pointer_hand_right.urdf.xacro (robot description, xacro)
@@ -11,7 +11,7 @@
     </inertial>
   </link>
-  <xacro:include filename="$(find hook_description)/src/bdihook_hand.urdf.xacro" />
-   <xacro:hook_hand side="right" parent="plane::xy::base" reflect="1" hookflip="1">
-     <origin rpy="1.57 3.14 -1.57" xyz="0 0 0"/>
+ <xacro:include filename="$(find hook_description)/src/hook_hand_simple.urdf.xacro" />
+  <xacro:hook_hand side="right" parent="plane::xy::base" reflect="1" hookflip="1">
+    <origin rpy="1.57 0.0 -1.57" xyz="0 0 0"/>
   </xacro:hook_hand>
 </robot>
