Commit message: significant clean up to remove all the unnecessary hand models
replaced with a script and removed from the build

File: software/models/mit_gazebo_models/mit_robot_hands/xacro/pointer_hand_left.urdf.xacro (robot description, xacro)
@@ -3,5 +3,5 @@
        xmlns:interface="http://playerstage.sourceforge.net/gazebo/xmlschema/#interface"
        xmlns:xacro="http://playerstage.sourceforge.net/gazebo/xmlschema/#interface"
-       name="inert_hand_right" >
+       name="pointer_hand_left" >
   <link name="plane::xy::base">
     <inertial>
@@ -11,8 +11,7 @@
     </inertial>
   </link>
-<!--  <xacro:include filename="$(find hook_description)/src/bdihook_hand.urdf.xacro" />  -->
   <xacro:include filename="$(find hook_description)/src/hook_hand_simple.urdf.xacro" />
-   <xacro:hook_hand side="right" parent="plane::xy::base">
-     <origin rpy="1.57 3.14 -1.57" xyz="0.243 0.0 -0.127"/>
+   <xacro:hook_hand side="left" parent="plane::xy::base" >
+     <origin rpy="1.57 0.0 -1.57" xyz="0.243 0.0 -0.127"/>
   </xacro:hook_hand>
 </robot>

File: software/models/mit_gazebo_models/mit_robot_hands/xacro/pointer_hand_right.urdf.xacro (robot description, xacro)
@@ -3,5 +3,5 @@
        xmlns:interface="http://playerstage.sourceforge.net/gazebo/xmlschema/#interface"
        xmlns:xacro="http://playerstage.sourceforge.net/gazebo/xmlschema/#interface"
-       name="inert_hand_left" >
+       name="pointer_hand_right" >
   <link name="plane::xy::base">
     <inertial>
@@ -11,8 +11,7 @@
     </inertial>
   </link>
-<!-- <xacro:include filename="$(find hook_description)/src/bdihook_hand.urdf.xacro" />  -->
- <xacro:include filename="$(find hook_description)/src/hook_hand_simple.urdf.xacro" />
-  <xacro:hook_hand side="left" parent="plane::xy::base" >
-    <origin rpy="1.57 0.0 -1.57" xyz="0.243 0.0 -0.127"/>
- </xacro:hook_hand>
+  <xacro:include filename="$(find hook_description)/src/hook_hand_simple.urdf.xacro" />
+   <xacro:hook_hand side="right" parent="plane::xy::base">
+     <origin rpy="1.57 3.14 -1.57" xyz="0.243 0.0 -0.127"/>
+  </xacro:hook_hand>
 </robot>
