Commit message: git-svn-id: https://svn.csail.mit.edu/drc@943 c7283977-0100-402a-a91a-fa70b306dbfe

File: software/models/mit_gazebo_models/mit_robot_hands/drake_urdfs/xacro/sandia_hand_drake.xacro (robot description, xacro)
@@ -37,10 +37,10 @@
         </material>
       </visual>
-      <collision>
+  <!-- <collision>
         <origin xyz="0 0 0" rpy="0 0 0"/>
         <geometry>
           <mesh filename="$(find mit_drcsim_scripts)/models/sandia_hand/meshes/f0.stl"/>
         </geometry>
-      </collision>
+  </collision> -->
     </link>
     <link name="${side}_f${idx}_1">
@@ -60,10 +60,10 @@
         </material>
       </visual>
-      <collision>
+  <!-- <collision>
         <origin xyz="0 0 0" rpy="0 0 0"/>
         <geometry>
           <mesh filename="$(find mit_drcsim_scripts)/models/sandia_hand/meshes/f1.stl"/>
         </geometry>
-      </collision>
+  </collision> -->
     </link>
     <link name="${side}_f${idx}_1_accel">
@@ -91,18 +91,30 @@
         </material>
       </visual>
+  <!-- <collision>
+        <origin xyz="0 0 0" rpy="0 0 0"/>
+        <geometry>
+          <mesh filename="$(find mit_drcsim_scripts)/models/sandia_hand/meshes/f2.stl"/>
+        </geometry>
+  </collision> -->
+    </link>
+    <link name="${side}_f${idx}_2_accel">
+      <origin xyz="0 0 0" rpy="0 0 0"/>
+      <inertial>
+        <mass value="0.1"/>
+        <origin xyz="0 0 0"/>
+        <inertia ixx="0.01" ixy="0" ixz="0" iyy="0.01" iyz="0" izz="0.01"/>
+      </inertial>
+     <visual>
+      <origin  xyz="0 0 0" rpy="0 0 0"/>
+      <geometry>
+        <sphere radius="0.001"/>
+      </geometry>
+    </visual>
       <collision>
-        <origin xyz="0 0 0" rpy="0 0 0"/>
-        <geometry>
-          <mesh filename="$(find mit_drcsim_scripts)/models/sandia_hand/meshes/f2.stl"/>
-        </geometry>
-      </collision>
-    </link>
-    <link name="${side}_f${idx}_2_accel">
-      <origin xyz="0 0 0" rpy="0 0 0"/>
-      <inertial>
-        <mass value="0.1"/>
-        <origin xyz="0 0 0"/>
-        <inertia ixx="0.01" ixy="0" ixz="0" iyy="0.01" iyz="0" izz="0.01"/>
-      </inertial>
+      <origin  xyz="0 0 0" rpy="0 0 0"/>
+      <geometry>
+        <sphere radius="0"/>
+      </geometry>
+    </collision>
     </link>
     <joint name="${side}_f${idx}_base" type="fixed">
@@ -172,10 +184,10 @@
         </material>
       </visual>
-      <collision>
+  <!-- <collision>
         <origin xyz="0 0 0" rpy="0 0 0"/>
         <geometry>
           <mesh filename="$(find mit_drcsim_scripts)/models/sandia_hand/meshes/palm.stl"/>
         </geometry>
-      </collision>
+  </collision> -->
     </link>
     <joint name="${side}_sandia_hand_joint" type="fixed">

File: software/models/mit_gazebo_models/mit_robot_hands/drake_urdfs/xacro/sandia_hand_drake_test.xacro (robot description, xacro)
@@ -20,4 +20,16 @@
         <inertia ixx="0.01" ixy="0" ixz="0" iyy="0.01" iyz="0" izz="0.01"/>
       </inertial>
+       <visual>
+      <origin rpy="0 0 0" xyz="0 0 0.055 "/>
+      <geometry>
+        <sphere radius="0.005"/>
+      </geometry>
+    </visual>
+    <collision>
+      <origin rpy="0 0 0" xyz="0 0 0"/>
+      <geometry>
+        <sphere radius="0"/>
+      </geometry>
+    </collision>
     </link>
     <link name="${side}_f${idx}_0">
@@ -74,4 +86,16 @@
         <inertia ixx="0.01" ixy="0" ixz="0" iyy="0.01" iyz="0" izz="0.01"/>
       </inertial>
+      <visual>
+      <origin rpy="0 0 0" xyz="0 0 0.01 "/>
+      <geometry>
+        <sphere radius="0.005"/>
+      </geometry>
+    </visual>
+    <collision>
+      <origin rpy="0 0 0" xyz="0 0 0"/>
+      <geometry>
+        <sphere radius="0"/>
+      </geometry>
+    </collision>
     </link>
     <link name="${side}_f${idx}_2">
@@ -105,4 +129,16 @@
         <inertia ixx="0.01" ixy="0" ixz="0" iyy="0.01" iyz="0" izz="0.01"/>
       </inertial>
+     <visual>
+      <origin rpy="0 0 0" xyz="0 0 0.01 "/>
+      <geometry>
+        <sphere radius="0.005"/>
+      </geometry>
+    </visual>
+    <collision>
+      <origin rpy="0 0 0" xyz="0 0 0"/>
+      <geometry>
+        <sphere radius="0"/>
+      </geometry>
+    </collision>
     </link>
     <joint name="${side}_f${idx}_base" type="fixed">

File: software/models/mit_gazebo_models/mit_robot_hands/drake_urdfs/xacro/sandia_hand_left_drake.urdf.xacro (robot description, xacro)
@@ -25,5 +25,5 @@
   </link>
   <xacro:sandia_hand side="left" parent="base">
-    <origin xyz="0 0 0.5" rpy="0 -1.57079 0"/>
+    <origin xyz="0 0 0.0" rpy="0 -1.57079 0"/>
   </xacro:sandia_hand>
 </robot>

File: software/models/mit_gazebo_models/mit_robot_hands/drake_urdfs/xacro/sandia_hand_right_drake.urdf.xacro (robot description, xacro)
@@ -25,5 +25,5 @@
   </link>
   <xacro:sandia_hand side="right" parent="base">
-    <origin xyz="0 0 0.5" rpy="0 -1.57079 0"/>
+    <origin xyz="0 0 0.0" rpy="0 -1.57079 0"/>
   </xacro:sandia_hand>
 </robot>

Commit message: git-svn-id: https://svn.csail.mit.edu/drc@960 c7283977-0100-402a-a91a-fa70b306dbfe

File: software/models/mit_gazebo_models/mit_robot_hands/drake_urdfs/xacro/sandia_hand_drake.xacro (robot description, xacro)
@@ -20,5 +20,25 @@
         <inertia ixx="0.01" ixy="0" ixz="0" iyy="0.01" iyz="0" izz="0.01"/>
       </inertial>
-    </link>
+      <collision>
+      <origin  xyz="0 0 0.05" rpy="0 0 0"/>
+      <geometry>
+        <sphere radius="0"/>
+      </geometry>
+    </collision>
+    </link>
+    <link name="${side}_f${idx}_knuckle_dummy_contact">
+    <origin rpy="0 0 0" xyz="0 0 0"/>
+    <inertial>
+      <mass value="0.001"/>
+      <origin xyz="0 0 0"/>
+      <inertia ixx="0.001" ixy="0" ixz="0" iyy="0.001" iyz="0" izz="0.001"/>
+    </inertial>
+    <collision>
+      <origin rpy="0 0 0" xyz="0.1 0 0.05"/>
+      <geometry>
+        <sphere radius="0"/>
+      </geometry>
+    </collision>
+  </link>
     <link name="${side}_f${idx}_0">
       <origin xyz="0 0 0" rpy="0 0 0"/>
@@ -74,4 +94,10 @@
         <inertia ixx="0.01" ixy="0" ixz="0" iyy="0.01" iyz="0" izz="0.01"/>
       </inertial>
+      <collision>
+      <origin  xyz="0 0 0.01" rpy="0 0 0"/>
+      <geometry>
+        <sphere radius="0"/>
+      </geometry>
+    </collision>
     </link>
     <link name="${side}_f${idx}_2">
@@ -105,12 +131,6 @@
         <inertia ixx="0.01" ixy="0" ixz="0" iyy="0.01" iyz="0" izz="0.01"/>
       </inertial>
-     <visual>
-      <origin  xyz="0 0 0" rpy="0 0 0"/>
-      <geometry>
-        <sphere radius="0.001"/>
-      </geometry>
-    </visual>
       <collision>
-      <origin  xyz="0 0 0" rpy="0 0 0"/>
+      <origin  xyz="0 0 0.01" rpy="0 0 0"/>
       <geometry>
         <sphere radius="0"/>
@@ -155,4 +175,9 @@
       <origin xyz="-0.05 0 0" rpy="0 0 0"/>
     </joint>
+   <joint name="${side}_f${idx}_knuckle_dummy_contact" type="fixed">
+    <parent link="${side}_f${idx}_base"/>
+    <child link="${side}_f${idx}_knuckle_dummy_contact"/>
+    <origin rpy="0 0 0" xyz="-0.05 0 0"/>
+  </joint>
     <joint name="${side}_f${idx}_1_accel" type="fixed">
       <parent link="${side}_f${idx}_1"/>

Commit message: Added xacro that includes x,y,z,roll,pitch,yaw to the base of the sandia hand
git-svn-id: https://svn.csail.mit.edu/drc@1309 c7283977-0100-402a-a91a-fa70b306dbfe

File: software/models/mit_gazebo_models/mit_robot_hands/drake_urdfs/xacro/sandia_hand_drake.xacro (robot description, xacro)
@@ -4,4 +4,5 @@
   <include filename="$(find sandia_hand_utils)/urdf/sandia_hand.gazebo.xacro" />
   <include filename="$(find sandia_hand_utils)/urdf/sandia_hand.transmission.xacro" />
+  <include filename="$(find mit_drcsim_scripts)/models/mit_robot_hands/drake_urdfs/xacro/sandia_hand_floating_base.xacro"/>
   <xacro:macro name="finger" params="idx x y z r p yaw side">
     <link name="${side}_f${idx}_base">
@@ -225,4 +226,5 @@
     <xacro:finger side="${side}" idx="2" x="0.090" y="0.06245" z="0" r="0" p="0" yaw="0.3"/>
     <xacro:finger side="${side}" idx="3" x="0.03995" y="-0.04383" z="0.014" r="0" p="-1.57079" yaw="-2.3562"/>
+    <xacro:base_links side ="${side}"/>
     <!-- not needed unless simulating the hand by itself
     <xacro:sandia_hand_gazebo side="${side}" />

File: software/models/mit_gazebo_models/mit_robot_hands/drake_urdfs/xacro/sandia_hand_right_drake.urdf.xacro (robot description, xacro)
@@ -5,5 +5,5 @@
        name="sandia_hand_right" >
   <include filename="$(find mit_drcsim_scripts)/models/mit_robot_hands/drake_urdfs/xacro/sandia_hand_drake.xacro" />
-  <link name="base">
+<!--  <link name="base">
     <inertial>
         <mass value="0.1" />
@@ -11,5 +11,5 @@
         <inertia ixx="0.01" ixy="0" ixz="0" iyy="0.01" iyz="0" izz="0.01" />
     </inertial>
-   <!-- <visual>
+    <visual>
         <origin xyz="0 0 0.25" rpy="0 0 0" />
         <geometry>
@@ -22,8 +22,8 @@
             <box size="0.5 0.5 0.5" />
         </geometry>
-    </collision> -->
-  </link>
-  <xacro:sandia_hand side="right" parent="base">
-    <origin xyz="0 0 0.0" rpy="0 -1.57079 0"/>
+    </collision>
+  </link> -->
+  <xacro:sandia_hand side="right" parent="right_base_yaw">
+    <origin xyz="0 0 0" rpy="0 0 0"/>
   </xacro:sandia_hand>
 </robot>

Commit message: <?xml version="1.0"?>
<robot name="sandia_hand"
       xmlns:xacro="http://www.ros.org/wiki/xacro">

  <include filename="$(find sandia_hand_utils)/urdf/sandia_hand.gazebo.xacro" />
  <include filename="$(find sandia_hand_utils)/urdf/sandia_hand.transmission.xacro" />

  <xacro:macro name="finger" params="idx x y z r p yaw side">
    <link name="${side}_f${idx}_base">
      <origin xyz="0 0 0" rpy="0 0 0"/>
      <inertial>
        <mass value="0.1"/>
        <origin xyz="0 0 0"/>
        <inertia ixx="0.01" ixy="0" ixz="0" iyy="0.01" iyz="0" izz="0.01"/>
      </inertial>
    </link>
   <link name="${side}_f${idx}_fixed_accel">
      <origin xyz="0 0 0" rpy="0 0 0"/>
      <inertial>
        <mass value="0.1"/>
        <origin xyz="0 0 0"/>
        <inertia ixx="0.01" ixy="0" ixz="0" iyy="0.01" iyz="0" izz="0.01"/>
      </inertial>
      <collision>
      <origin  xyz="0 0 0.05" rpy="0 0 0"/>
      <geometry>
        <sphere radius="0"/>
      </geometry>
    </collision>
    </link> 
    
    <link name="${side}_f${idx}_knuckle_dummy_contact">
    <origin rpy="0 0 0" xyz="0 0 0"/>
    <inertial>
      <mass value="0.001"/>
      <origin xyz="0 0 0"/>
      <inertia ixx="0.001" ixy="0" ixz="0" iyy="0.001" iyz="0" izz="0.001"/>
    </inertial>
    <collision>
      <origin rpy="0 0 0" xyz="0.1 0 0.05"/>
      <geometry>
        <sphere radius="0"/>
      </geometry>
    </collision>
  </link>

    
    <link name="${side}_f${idx}_0">
      <origin xyz="0 0 0" rpy="0 0 0"/>
      <inertial>
        <mass value="0.1"/>
        <origin xyz="0 0 0"/>
        <inertia ixx="0.01" ixy="0" ixz="0" iyy="0.01" iyz="0" izz="0.01"/>
      </inertial>
      <visual>
        <origin xyz="0 0 0" rpy="0 0 0"/>
        <geometry>
          <mesh filename="$(find mit_drcsim_scripts)/models/sandia_hand/meshes/f0.wrl"/>
        </geometry>
        <material name="${side}_sandia_hand_skin_suntan">
          <color rgba="0.7 0.4 0.2 1.0"/>
        </material>
      </visual>
  <!-- <collision>
        <origin xyz="0 0 0" rpy="0 0 0"/>
        <geometry>
          <mesh filename="$(find mit_drcsim_scripts)/models/sandia_hand/meshes/f0.stl"/>
        </geometry>
  </collision> -->
    </link>
    <link name="${side}_f${idx}_1">
      <origin xyz="0 0 0" rpy="0 0 0"/>
      <inertial>
        <mass value="0.1"/>
        <origin xyz="0 0 0"/>
        <inertia ixx="0.01" ixy="0" ixz="0" iyy="0.01" iyz="0" izz="0.01"/>
      </inertial>
      <visual>
        <origin xyz="0 0 0" rpy="0 0 0"/>
        <geometry>
          <mesh filename="$(find mit_drcsim_scripts)/models/sandia_hand/meshes/f1.wrl"/>
        </geometry>
        <material name="${side}_sandia_hand_skin">
          <color rgba="0.835 0.655 0.345 1.0"/>
        </material>
      </visual>
  <!-- <collision>
        <origin xyz="0 0 0" rpy="0 0 0"/>
        <geometry>
          <mesh filename="$(find mit_drcsim_scripts)/models/sandia_hand/meshes/f1.stl"/>
        </geometry>
  </collision> -->
    </link>
    <link name="${side}_f${idx}_1_accel">
      <origin xyz="0 0 0" rpy="0 0 0"/>
      <inertial>
        <mass value="0.1"/>
        <origin xyz="0 0 0"/>
        <inertia ixx="0.01" ixy="0" ixz="0" iyy="0.01" iyz="0" izz="0.01"/>
      </inertial>
      <collision>
      <origin  xyz="0 0 0.01" rpy="0 0 0"/>
      <geometry>
        <sphere radius="0"/>
      </geometry>
    </collision>
    </link> 
    <link name="${side}_f${idx}_2">
      <origin xyz="0 0 0" rpy="0 0 0"/>
      <inertial>
        <mass value="0.1"/>
        <origin xyz="0 0 0"/>
        <inertia ixx="0.01" ixy="0" ixz="0" iyy="0.01" iyz="0" izz="0.01"/>
      </inertial>
      <visual>
        <origin xyz="0 0 0" rpy="0 0 0"/>
        <geometry>
          <mesh filename="$(find mit_drcsim_scripts)/models/sandia_hand/meshes/f2.wrl"/>
        </geometry>
        <material name="${side}_sandia_hand_skin_suntan">
          <color rgba="0.8 0.6 0.3 1.0"/>
        </material>
      </visual>
  <!-- <collision>
        <origin xyz="0 0 0" rpy="0 0 0"/>
        <geometry>
          <mesh filename="$(find mit_drcsim_scripts)/models/sandia_hand/meshes/f2.stl"/>
        </geometry>
  </collision> -->      
    </link>
    <link name="${side}_f${idx}_2_accel">
      <origin xyz="0 0 0" rpy="0 0 0"/>
      <inertial>
        <mass value="0.1"/>
        <origin xyz="0 0 0"/>
        <inertia ixx="0.01" ixy="0" ixz="0" iyy="0.01" iyz="0" izz="0.01"/>
      </inertial>
      <collision>
      <origin  xyz="0 0 0.01" rpy="0 0 0"/>
      <geometry>
        <sphere radius="0"/>
      </geometry>
    </collision>
    </link>
    <joint name="${side}_f${idx}_base" type="fixed">
      <parent link="${side}_palm"/>
      <child link="${side}_f${idx}_base"/>
      <origin xyz="${x} ${y} ${z}" rpy="${r} ${p} ${yaw}"/>
    </joint>
    <joint name="${side}_f${idx}_j0" type="revolute">
      <axis xyz="0 0 1"/>
      <parent link="${side}_f${idx}_base"/>
      <child link="${side}_f${idx}_0"/>
      <limit lower="-1.57079" upper="1.57079" effort="1" velocity="1"/>
      <safety_controller soft_lower_limit="${-1.57079-10.0}" soft_upper_limit="${1.57079+10.0}" k_position="1000.0" k_velocity="1000.0"/>
      <dynamics damping="0.1"/>
      <origin xyz="0 0 0" rpy="0 0 0"/>
    </joint>
    <joint name="${side}_f${idx}_j1" type="revolute">
      <axis xyz="0 0 1"/>
      <parent link="${side}_f${idx}_0"/>
      <child link="${side}_f${idx}_1"/>
      <limit lower="-1.57079" upper="1.57079" effort="1" velocity="1"/>
      <safety_controller soft_lower_limit="${-1.57079-10.0}" soft_upper_limit="${1.57079+10.0}" k_position="1000.0" k_velocity="1000.0"/>
      <dynamics damping="0.1"/>
      <origin xyz="0.028 0 0" rpy="1.57079 0 0"/>
    </joint>
    <joint name="${side}_f${idx}_j2" type="revolute">
      <axis xyz="0 0 1"/>
      <parent link="${side}_f${idx}_1"/>
      <child link="${side}_f${idx}_2"/>
      <origin xyz="0.05 0 0" rpy="0 0 0"/>
      <safety_controller soft_lower_limit="${-1.57079-10.0}" soft_upper_limit="${1.57079+10.0}" k_position="1000.0" k_velocity="1000.0"/>
      <dynamics damping="0.1"/>
      <limit lower="-1.57079" upper="1.57079" effort="1" velocity="1"/>
    </joint>

   <joint name="${side}_f${idx}_fixed_accel" type="fixed">
      <parent link="${side}_f${idx}_base"/>
      <child link="${side}_f${idx}_fixed_accel"/>
      <origin xyz="-0.05 0 0" rpy="0 0 0"/>
    </joint>
    
        
   <joint name="${side}_f${idx}_knuckle_dummy_contact" type="fixed">
    <parent link="${side}_f${idx}_base"/>
    <child link="${side}_f${idx}_knuckle_dummy_contact"/>
    <origin rpy="0 0 0" xyz="-0.05 0 0"/>
  </joint>
  
    
    <joint name="${side}_f${idx}_1_accel" type="fixed">
      <parent link="${side}_f${idx}_1"/>
      <child link="${side}_f${idx}_1_accel"/>
      <origin xyz="0.03 0 0" rpy="-1.5709 0 0"/>
    </joint>
    <joint name="${side}_f${idx}_2_accel" type="fixed">
      <parent link="${side}_f${idx}_2"/>
      <child link="${side}_f${idx}_2_accel"/>
      <origin xyz="0.04 0 0" rpy="-1.5709 0 0"/>
    </joint>
    
    <xacro:finger_transmission side="${side}" idx="${idx}" x="${x}" y="${y}" z="${z}" r="${r}" p="${p}" yaw="${yaw}"/>
  </xacro:macro>

  <xacro:macro name="sandia_hand" params="side parent *origin">
    <link name="${side}_palm">
      <origin xyz="0 0 0" rpy="0 0 0"/>
      <inertial>
        <mass value="0.1"/>
        <origin xyz="0 0 0"/>
        <inertia ixx="0.01" ixy="0" ixz="0" iyy="0.01" iyz="0" izz="0.01"/>
      </inertial>
      <visual>
        <origin xyz="0 0 0" rpy="0 0 0"/>
        <geometry>
          <mesh filename="$(find mit_drcsim_scripts)/models/sandia_hand/meshes/palm.wrl"/>
        </geometry>
        <material name="${side}_sandia_hand_skin">
          <color rgba="0.835 0.655 0.345 1.0"/>
        </material>
      </visual>
  <!-- <collision>
        <origin xyz="0 0 0" rpy="0 0 0"/>
        <geometry>
          <mesh filename="$(find mit_drcsim_scripts)/models/sandia_hand/meshes/palm.stl"/>
        </geometry>
  </collision> -->      
    </link>

    <joint name="${side}_sandia_hand_joint" type="fixed">
      <parent link="${parent}"/>
      <child link="${side}_palm"/>
      <insert_block name="origin" />
    </joint>

    <xacro:finger side="${side}" idx="0" x="0.140" y="0.00000" z="0" r="0" p="0" yaw="0.3"/>
    <xacro:finger side="${side}" idx="1" x="0.115" y="0.03122" z="0" r="0" p="0" yaw="0.3"/>
    <xacro:finger side="${side}" idx="2" x="0.090" y="0.06245" z="0" r="0" p="0" yaw="0.3"/>
    <xacro:finger side="${side}" idx="3" x="0.03995" y="-0.04383" z="0.014" r="0" p="-1.57079" yaw="-2.3562"/>

    <!-- not needed unless simulating the hand by itself
    <xacro:sandia_hand_gazebo side="${side}" />
    -->

  </xacro:macro>
</robot>



git-svn-id: https://svn.csail.mit.edu/drc@1347 c7283977-0100-402a-a91a-fa70b306dbfe

File: software/models/mit_gazebo_models/mit_robot_hands/drake_urdfs/xacro/sandia_hand_drake.xacro (robot description, xacro)
@@ -4,5 +4,4 @@
   <include filename="$(find sandia_hand_utils)/urdf/sandia_hand.gazebo.xacro" />
   <include filename="$(find sandia_hand_utils)/urdf/sandia_hand.transmission.xacro" />
-  <include filename="$(find mit_drcsim_scripts)/models/mit_robot_hands/drake_urdfs/xacro/sandia_hand_floating_base.xacro"/>
   <xacro:macro name="finger" params="idx x y z r p yaw side">
     <link name="${side}_f${idx}_base">
@@ -226,5 +225,4 @@
     <xacro:finger side="${side}" idx="2" x="0.090" y="0.06245" z="0" r="0" p="0" yaw="0.3"/>
     <xacro:finger side="${side}" idx="3" x="0.03995" y="-0.04383" z="0.014" r="0" p="-1.57079" yaw="-2.3562"/>
-    <xacro:base_links side ="${side}"/>
     <!-- not needed unless simulating the hand by itself
     <xacro:sandia_hand_gazebo side="${side}" />

File: software/models/mit_gazebo_models/mit_robot_hands/drake_urdfs/xacro/sandia_hand_right_drake.urdf.xacro (robot description, xacro)
@@ -4,6 +4,6 @@
        xmlns:xacro="http://playerstage.sourceforge.net/gazebo/xmlschema/#interface"
        name="sandia_hand_right" >
-  <include filename="$(find mit_drcsim_scripts)/models/mit_robot_hands/drake_urdfs/xacro/sandia_hand_drake_floating.xacro" />
-<!--  <link name="base">
+  <include filename="$(find mit_drcsim_scripts)/models/mit_robot_hands/drake_urdfs/xacro/sandia_hand_drake.xacro" />
+  <link name="base">
     <inertial>
         <mass value="0.1" />
@@ -11,5 +11,5 @@
         <inertia ixx="0.01" ixy="0" ixz="0" iyy="0.01" iyz="0" izz="0.01" />
     </inertial>
-    <visual>
+    <!-- <visual>
         <origin xyz="0 0 0.25" rpy="0 0 0" />
         <geometry>
@@ -22,7 +22,7 @@
             <box size="0.5 0.5 0.5" />
         </geometry>
-    </collision>
-  </link> -->
-  <xacro:sandia_hand side="right" parent="right_base_yaw">
+    </collision> -->
+  </link>
+  <xacro:sandia_hand side="right" parent="base">
     <origin xyz="0 0 0" rpy="0 0 0"/>
   </xacro:sandia_hand>
