Commit message: Changes to sticky hand urdf's as joint names in the robot urdf use l_ and r_ instead of left_ and right_
git-svn-id: https://svn.csail.mit.edu/drc@1476 c7283977-0100-402a-a91a-fa70b306dbfe

File: software/models/mit_gazebo_models/mit_robot_hands/drake_urdfs/xacro/sandia_hand_drake.xacro (robot description, xacro)
@@ -147,5 +147,7 @@
       <parent link="${side}_f${idx}_base"/>
       <child link="${side}_f${idx}_0"/>
-      <limit lower="-1.57079" upper="1.57079" effort="1" velocity="1"/>
+      <limit effort="1" lower="-1.57079" upper="1.57079" velocity="1"/>
+ <!-- limits are customized in the urdf, no point setting limits in xacro as they differ for each finger  -->
+ <!--      <limit effort="1" lower="-1.57079" upper="0" velocity="1"/>-->
       <safety_controller soft_lower_limit="${-1.57079-10.0}" soft_upper_limit="${1.57079+10.0}" k_position="1000.0" k_velocity="1000.0"/>
       <dynamics damping="0.1"/>

File: software/models/mit_gazebo_models/mit_robot_hands/drake_urdfs/xacro/sandia_hand_left_drake.urdf.xacro (robot description, xacro)
@@ -4,4 +4,7 @@
        xmlns:xacro="http://playerstage.sourceforge.net/gazebo/xmlschema/#interface"
        name="sandia_hand_left" >
+<!--  TODO: sandia_hand_drake.xacro needs to be editted to properly include
+customized joints limits for grasp optimization, these change for each finger,
+so finger generic sandia_hand_drake.xacro is no good. For the moment manually editting urdf files-->
   <include filename="$(find mit_drcsim_scripts)/models/mit_robot_hands/drake_urdfs/xacro/sandia_hand_drake.xacro" />
   <link name="base">
@@ -24,5 +27,5 @@
     </collision> -->
   </link>
-  <xacro:sandia_hand side="left" parent="base">
+  <xacro:sandia_hand side="l" parent="base">
     <origin xyz="0 0 0.0" rpy="0 -1.57079 0"/>
   </xacro:sandia_hand>

File: software/models/mit_gazebo_models/mit_robot_hands/drake_urdfs/xacro/sandia_hand_right_drake.urdf.xacro (robot description, xacro)
@@ -24,5 +24,5 @@
     </collision> -->
   </link>
-  <xacro:sandia_hand side="right" parent="base">
+  <xacro:sandia_hand side="r" parent="base">
     <origin xyz="0 0 0.0" rpy="0 -1.57079 0"/>
   </xacro:sandia_hand>

File: software/models/mit_gazebo_models/mit_robot_hands/xacro/sandia_hand_left.urdf.xacro (robot description, xacro)
@@ -3,5 +3,5 @@
        xmlns:interface="http://playerstage.sourceforge.net/gazebo/xmlschema/#interface"
        xmlns:xacro="http://playerstage.sourceforge.net/gazebo/xmlschema/#interface"
-       name="humanoid" >
+       name="sandia_hand_left" >
   <include filename="$(find sandia_hand_utils)/urdf/sandia_hand.urdf.xacro" />
   <link name="base">
@@ -24,6 +24,6 @@
     </collision> -->
   </link>
-  <xacro:sandia_hand side="left" parent="base">
-    <origin xyz="0 0 0.5" rpy="0 -1.57079 0"/>
+  <xacro:sandia_hand side="l" parent="base">
+    <origin xyz="0 0 0.0" rpy="0 -1.57079 0"/>
   </xacro:sandia_hand>
 </robot>

File: software/models/mit_gazebo_models/mit_robot_hands/xacro/sandia_hand_right.urdf.xacro (robot description, xacro)
@@ -3,5 +3,5 @@
        xmlns:interface="http://playerstage.sourceforge.net/gazebo/xmlschema/#interface"
        xmlns:xacro="http://playerstage.sourceforge.net/gazebo/xmlschema/#interface"
-       name="humanoid" >
+       name="sandia_hand_right" >
   <include filename="$(find sandia_hand_utils)/urdf/sandia_hand.urdf.xacro" />
   <link name="base">
@@ -24,6 +24,6 @@
     </collision> -->
   </link>
-  <xacro:sandia_hand side="right" parent="base">
-    <origin xyz="0 0 0.5" rpy="0 -1.57079 0"/>
+  <xacro:sandia_hand side="r" parent="base">
+    <origin xyz="0 0 0.0" rpy="0 -1.57079 0"/>
   </xacro:sandia_hand>
 </robot>
