Commit message: minor modifications to hands
git-svn-id: https://svn.csail.mit.edu/drc@1759 c7283977-0100-402a-a91a-fa70b306dbfe

File: software/models/mit_gazebo_models/mit_robot_hands/drake_urdfs/xacro/sandia_hand_simple_shapes_drake.urdf.xacro (robot description, xacro)
@@ -232,5 +232,5 @@
       <!-- ############ MIT ADDITION ############ -->
       <collision>
-        <origin rpy="0 0 0" xyz="0 0 0.01"/>
+        <origin rpy="0 0 0" xyz="0 0 0.001"/>
         <geometry>
           <sphere radius="0"/>
@@ -318,5 +318,5 @@
     </inertial>
     <collision>
-      <origin rpy="0 0 0" xyz="0.058 0 0.034"/> <!--TODO: THERE IS A ERROR HERE: xyz needs to be "0.058 0 0.034" instead of "0.1 0 0.05"-->
+      <origin rpy="0 0 0" xyz="0.058 0 0.034"/>
       <geometry>
         <sphere radius="0"/>
@@ -533,5 +533,5 @@
       <!-- ############ MIT ADDITION ############ -->
       <collision>
-        <origin rpy="0 0 0" xyz="0 0 0.01"/>
+        <origin rpy="0 0 0" xyz="0 0 0.001"/>
         <geometry>
           <sphere radius="0"/>
