Commit message: =
git-svn-id: https://svn.csail.mit.edu/drc@4052 c7283977-0100-402a-a91a-fa70b306dbfe

File: software/models/mit_gazebo_models/mit_robot_hands/drake_urdfs/xacro/sandia_palm_simple_shapes_drake.urdf.xacro (robot description, xacro)
@@ -55,17 +55,5 @@
       </collision>
       <collision group="knuckle">
-        <origin xyz="0.155 0 -0.01" rpy="0 0 0"/>
-        <geometry>
-          <sphere radius="0"/>
-        </geometry>
-      </collision>
-      <collision group="knuckle">
-        <origin xyz="0.155 0 0.01" rpy="0 0 0"/>
-        <geometry>
-          <sphere radius="0"/>
-        </geometry>
-      </collision>
-      <collision group="knuckle">
-        <origin xyz="0.15 0.01 0" rpy="0 0 0"/>
+        <origin xyz="0.155 0 0" rpy="0 0 0"/>
         <geometry>
           <sphere radius="0"/>
@@ -73,17 +61,5 @@
       </collision>
       <visual group="knuckle">
-        <origin xyz="0.155 0 -0.01" rpy="0 0 0"/>
-        <geometry>
-          <sphere radius="0.005"/>
-        </geometry>
-      </visual>
-      <visual group="knuckle">
-        <origin xyz="0.155 0 0.01" rpy="0 0 0"/>
-        <geometry>
-          <sphere radius="0.005"/>
-        </geometry>
-      </visual>
-      <visual group="knuckle">
-        <origin xyz="0.15 0.01 0" rpy="0 0 0"/>
+        <origin xyz="0.155 0 0" rpy="0 0 0"/>
         <geometry>
           <sphere radius="0.005"/>

Commit message: Update contact groups for pelvis and sandia knuckle
git-svn-id: https://svn.csail.mit.edu/drc@4229 c7283977-0100-402a-a91a-fa70b306dbfe

File: software/models/mit_gazebo_models/mit_robot_hands/drake_urdfs/xacro/sandia_palm_simple_shapes_drake.urdf.xacro (robot description, xacro)
@@ -55,5 +55,5 @@
       </collision>
       <collision group="knuckle">
-        <origin xyz="0.155 0 0" rpy="0 0 0"/>
+        <origin xyz="0.175 0 0" rpy="0 0 0"/>
         <geometry>
           <sphere radius="0"/>
@@ -61,5 +61,5 @@
       </collision>
       <visual group="knuckle">
-        <origin xyz="0.155 0 0" rpy="0 0 0"/>
+        <origin xyz="0.175 0 0" rpy="0 0 0"/>
         <geometry>
           <sphere radius="0.005"/>
