Commit message: adding combined model
git-svn-id: https://svn.csail.mit.edu/drc@1504 c7283977-0100-402a-a91a-fa70b306dbfe

File: software/models/mit_gazebo_models/mit_robotWhands_PnC/model.urdf (robot description, URDF)
Before this commit: robot atlas, 93 links, 92 joints
Links:
- added link center_bottom_led_frame, mass 0.1
- added link center_top_led_frame, mass 0.1
- added link head_imu_link, mass 0.1; collision box size=0.01 0.01 0.01; visual box size=0.01 0.01 0.01
- added link hokuyo_link, mass 0.057664; collision mesh filename=package://multisense_sl/meshes/hokuyo_link.STL; visual mesh filename=package://multisense_sl/meshes/hokuyo_link.STL
- added link left_led_frame, mass 0.1
- added link right_led_frame, mass 0.1
- link head: mass 2.6 -> 1.4199; geometry collision mesh filename=package://multisense_sl/meshes/base_link.STL; visual mesh filename=package://multisense_sl/meshes/base_link.STL
- link head_hokuyo: mass 0.1 -> 0.01
Joints:
- added joint center_bottom_led_frame_joint: type fixed, parent head, child center_bottom_led_frame, origin xyz=0.01125 0.0 -0.0155
- added joint center_top_led_frame_joint: type fixed, parent head, child center_top_led_frame, origin xyz=0.01125 0.0 0.0105
- added joint head_imu_joint: type revolute, parent head, child head_imu_link, origin xyz=0 0 0 rpy=0 0 0, axis 0 0 1, limit lower=0 upper=0 effort=0 velocity=0
- added joint hokuyo_joint: type continuous, parent head, child hokuyo_link, origin xyz=-0.0446 0 0.0880 rpy=0 0 0, axis 1 0 0
- added joint left_led_frame_joint: type fixed, parent head, child left_led_frame, origin xyz=-0.01443 0.07452 0.050346 rpy=0 -0.15 0.53
- added joint right_led_frame_joint: type fixed, parent head, child right_led_frame, origin xyz=-0.01443 -0.07452 0.050346 rpy=0 -0.15 -0.53
- joint head_hokuyo_joint: origin xyz=0.03 0 0.13 rpy=0 0 0 -> xyz=0.03 0 0.015 rpy=0 0 0; parent head -> hokuyo_link
- joint left_camera_frame_joint: origin xyz=0.03 0.1 0.1 -> xyz=0.0 0.035 -0.002
- joint neck_ay: limit lower=-0.785398 upper=0.785398 effort=5 velocity=12 -> lower=-0.610865238 upper=1.13446401 effort=5 velocity=12; origin xyz=0.011 0 0.44 rpy=0 -0 0 -> xyz=0.16555 0 0.50823 rpy=0 0 0
- joint right_camera_frame_joint: origin xyz=0.03 -0.1 0.1 -> xyz=0.0 -0.035 -0.002

File: software/models/mit_gazebo_models/mit_robot_PnC/model.urdf (robot description, URDF)
Before this commit: robot atlas, 35 links, 34 joints
Links:
- added link center_bottom_led_frame, mass 0.1
- added link center_top_led_frame, mass 0.1
- added link head_imu_link, mass 0.1; collision box size=0.01 0.01 0.01; visual box size=0.01 0.01 0.01
- added link hokuyo_link, mass 0.057664; collision mesh filename=package://multisense_sl/meshes/hokuyo_link.STL; visual mesh filename=package://multisense_sl/meshes/hokuyo_link.STL
- added link left_led_frame, mass 0.1
- added link right_led_frame, mass 0.1
- link head: mass 2.6 -> 1.4199; geometry collision mesh filename=package://multisense_sl/meshes/base_link.STL; visual mesh filename=package://multisense_sl/meshes/base_link.STL
- link head_hokuyo: mass 0.1 -> 0.01
Joints:
- added joint center_bottom_led_frame_joint: type fixed, parent head, child center_bottom_led_frame, origin xyz=0.01125 0.0 -0.0155
- added joint center_top_led_frame_joint: type fixed, parent head, child center_top_led_frame, origin xyz=0.01125 0.0 0.0105
- added joint head_imu_joint: type revolute, parent head, child head_imu_link, origin xyz=0 0 0 rpy=0 0 0, axis 0 0 1, limit lower=0 upper=0 effort=0 velocity=0
- added joint hokuyo_joint: type continuous, parent head, child hokuyo_link, origin xyz=-0.0446 0 0.0880 rpy=0 0 0, axis 1 0 0
- added joint left_led_frame_joint: type fixed, parent head, child left_led_frame, origin xyz=-0.01443 0.07452 0.050346 rpy=0 -0.15 0.53
- added joint right_led_frame_joint: type fixed, parent head, child right_led_frame, origin xyz=-0.01443 -0.07452 0.050346 rpy=0 -0.15 -0.53
- joint head_hokuyo_joint: origin xyz=0.03 0 0.13 rpy=0 0 0 -> xyz=0.03 0 0.015 rpy=0 0 0; parent head -> hokuyo_link
- joint left_camera_frame_joint: origin xyz=0.03 0.1 0.1 -> xyz=0.0 0.035 -0.002
- joint neck_ay: limit lower=-0.785398 upper=0.785398 effort=5 velocity=12 -> lower=-0.610865238 upper=1.13446401 effort=5 velocity=12; origin xyz=0.011 0 0.44 rpy=0 -0 0 -> xyz=0.16555 0 0.50823 rpy=0 0 0
- joint right_camera_frame_joint: origin xyz=0.03 -0.1 0.1 -> xyz=0.0 -0.035 -0.002

File: software/models/mit_gazebo_models/mit_robot_PnC/xacro/atlas.model.xacro (robot description, xacro)
@@ -7,5 +7,8 @@
 <!--  <include filename="$(find mit_drcsim_scripts)/models/mit_robot_PnC/xacro/atlas_skeleton_minimal_contact.urdf" /> -->
   <include filename="$(find atlas_utils)/urdf/atlas.transmission" />
-  <include filename="$(find atlas_utils)/urdf/atlas.sensors" />
+<!-- was: -->
+<!--  <include filename="$(find atlas_utils)/urdf/atlas.sensors" /> -->
+<!-- now: -->
+  <include filename="$(find mit_drcsim_scripts)/models/mit_robot_PnC/xacro/atlas.sensors" />
 <!--  <include filename="$(find mit_drcsim_scripts)/models/mit_robot_PnC/xacro/mit_atlas.gazebo" /> -->
   <include filename="$(find mit_drcsim_scripts)/models/mit_robot_PnC/xacro/mit_atlas_position_control.gazebo" />

File: software/models/mit_gazebo_models/mit_robot_PnC/xacro/atlas_sandia_hands.model.xacro (robot description, xacro)
@@ -13,5 +13,8 @@
   </xacro:sandia_hand>
   <include filename="$(find atlas_utils)/urdf/atlas.transmission" />
-  <include filename="$(find atlas_utils)/urdf/atlas.sensors" />
+<!-- was: -->
+<!--  <include filename="$(find atlas_utils)/urdf/atlas.sensors" /> -->
+<!-- now: -->
+  <include filename="$(find mit_drcsim_scripts)/models/mit_robot_PnC/xacro/atlas.sensors" />
 <!--  <include filename="$(find mit_drcsim_scripts)/models/mit_robot_PnC/xacro/mit_atlas.gazebo" /> -->
   <include filename="$(find mit_drcsim_scripts)/models/mit_robot_PnC/xacro/mit_atlas_position_control.gazebo" />

File: software/models/mit_gazebo_models/mit_robot_PnC/xacro/atlas_skeleton.urdf (robot description, URDF)
Before this commit: robot drc_skeleton, 29 links, 28 joints
Links:
- added link hokuyo_link, mass 0.057664; collision mesh filename=package://multisense_sl/meshes/hokuyo_link.STL; visual mesh filename=package://multisense_sl/meshes/hokuyo_link.STL
- link head: mass 2.6 -> 1.4199; geometry collision mesh filename=package://multisense_sl/meshes/base_link.STL; visual mesh filename=package://multisense_sl/meshes/base_link.STL
Joints:
- added joint hokuyo_joint: type continuous, parent head, child hokuyo_link, origin xyz=-0.0446 0 0.0880 rpy=0 0 0, axis 1 0 0
- joint neck_ay: limit lower=-0.785398 upper=0.785398 effort=5 velocity=12 -> lower=-0.610865238 upper=1.13446401 effort=5 velocity=12; origin xyz=0.011 0 0.44 rpy=0 -0 0 -> xyz=0.16555 0 0.50823 rpy=0 0 0
