Commit message: use lowercase extension
git-svn-id: https://svn.csail.mit.edu/drc@1579 c7283977-0100-402a-a91a-fa70b306dbfe

File: software/models/mit_gazebo_models/multisense_sl/MultiSense-SL_simplified2.URDF (robot description, URDF)
Before this commit: robot multisense_sl, 2 links, 1 joints
Links:
- link base_link: geometry collision mesh filename=package://multisense_sl/meshes/base_link.stl; visual mesh filename=package://multisense_sl/meshes/base_link.stl
