Commit message: updating multisense head to 2.2
git-svn-id: https://svn.csail.mit.edu/drc@2280 c7283977-0100-402a-a91a-fa70b306dbfe

File: software/models/mit_gazebo_models/multisense_sl/multisense_sl.urdf (robot description, URDF)
Before this commit: robot multisense_sl, 11 links, 10 joints
Links:
- added link head_imu_link, mass 0.1; visual box size=0.01 0.01 0.01
Joints:
- added joint head_imu_joint: type fixed, parent head, child head_imu_link, origin xyz=-0.0475 0.035 0.0 rpy=0 0 0
