Commit message: use lowercase extension
git-svn-id: https://svn.csail.mit.edu/drc@1578 c7283977-0100-402a-a91a-fa70b306dbfe

File: ros_workspace/multisense/multisense/multisense_description/robots/MultiSense-SL_simplified2.URDF (robot description, URDF)
Before this commit: robot MultiSense-SL_simplified2, 2 links, 1 joints
Links:
- link base_link: geometry collision mesh filename=package://MultiSense-SL_simplified2/meshes/base_link.stl; visual mesh filename=package://MultiSense-SL_simplified2/meshes/base_link.stl

Commit message: use lowercase extension
git-svn-id: https://svn.csail.mit.edu/drc@1582 c7283977-0100-402a-a91a-fa70b306dbfe

File: ros_workspace/multisense/multisense/multisense_description/robots/MultiSense-SL_simplified2.URDF (robot description, URDF)
Before this commit: robot MultiSense-SL_simplified2, 2 links, 1 joints
Links:
- link hokuyo_link: geometry collision mesh filename=package://MultiSense-SL_simplified2/meshes/hokuyo_link.stl; visual mesh filename=package://MultiSense-SL_simplified2/meshes/hokuyo_link.stl
