Commit message: git-svn-id: https://svn.csail.mit.edu/drc@1677 c7283977-0100-402a-a91a-fa70b306dbfe

File: software/models/mit_gazebo_models/mit_robot_hands/floatingbase_urdfs/sandia_hand_drake_left_floating.urdf (robot description, URDF)
Before this commit: robot sandia_hand_left, 39 links, 38 joints
Links:
- added link left_f0_2_accel_dummy1, mass 0.001; collision sphere radius=0
- added link left_f1_2_accel_dummy1, mass 0.001; collision sphere radius=0
- added link left_f2_2_accel_dummy1, mass 0.001; collision sphere radius=0
- added link left_f3_2_accel_dummy1, mass 0.001; collision sphere radius=0
- link left_f0_1_accel: geometry 
- link left_f1_1_accel: geometry 
- link left_f2_1_accel: geometry 
Joints:
- added joint left_f0_2_accel_dummy1: type fixed, parent left_f0_2, child left_f0_2_accel_dummy1, origin xyz=0.04 0 0 rpy=-1.57079632679 0 0
- added joint left_f1_2_accel_dummy1: type fixed, parent left_f1_2, child left_f1_2_accel_dummy1, origin xyz=0.04 0 0 rpy=-1.57079632679 0 0
- added joint left_f2_2_accel_dummy1: type fixed, parent left_f2_2, child left_f2_2_accel_dummy1, origin xyz=0.04 0 0 rpy=-1.57079632679 0 0
- added joint left_f3_2_accel_dummy1: type fixed, parent left_f3_2, child left_f3_2_accel_dummy1, origin xyz=0.04 0 0 rpy=-1.57079632679 0 0

File: software/models/mit_gazebo_models/mit_robot_hands/floatingbase_urdfs/sandia_hand_drake_right_floating.urdf (robot description, URDF)
Before this commit: robot sandia_hand_right, 39 links, 38 joints
Links:
- added link right_f0_2_accel_dummy1, mass 0.001; collision sphere radius=0
- added link right_f1_2_accel_dummy1, mass 0.001; collision sphere radius=0
- added link right_f2_2_accel_dummy1, mass 0.001; collision sphere radius=0
- added link right_f3_2_accel_dummy1, mass 0.001; collision sphere radius=0
- link right_f0_1_accel: geometry 
- link right_f1_1_accel: geometry 
- link right_f2_1_accel: geometry 
Joints:
- added joint right_f0_2_accel_dummy1: type fixed, parent right_f0_2, child right_f0_2_accel_dummy1, origin xyz=0.04 0 0 rpy=-1.57079632679 0 0
- added joint right_f1_2_accel_dummy1: type fixed, parent right_f1_2, child right_f1_2_accel_dummy1, origin xyz=0.04 0 0 rpy=-1.57079632679 0 0
- added joint right_f2_2_accel_dummy1: type fixed, parent right_f2_2, child right_f2_2_accel_dummy1, origin xyz=0.04 0 0 rpy=-1.57079632679 0 0
- added joint right_f3_2_accel_dummy1: type fixed, parent right_f3_2, child right_f3_2_accel_dummy1, origin xyz=0.04 0 0 rpy=-1.57079632679 0 0

File: software/models/mit_gazebo_models/mit_robot_hands/floatingbase_urdfs/xacro/sandia_hand_drake_left_w_floating_base.urdf.xacro (robot description, xacro)
@@ -6,6 +6,6 @@
 <!-- derived from /usr/share/sandia-hand-5.1/ros/sandia_hand_description/robots/sandia_hand_left_on_box.urdf.xacro-->
   <!-- Commenting out urdf with meshes, using simple collision shapes instead -->
-  <!--<include filename="$(find mit_drcsim_scripts)/models/mit_robot_hands/drake_urdfs/new_xacro/sandia_hand_drake.urdf.xacro" />-->
-  <include filename="$(find mit_drcsim_scripts)/models/mit_robot_hands/drake_urdfs/new_xacro/sandia_hand_simple_shapes_drake.urdf.xacro" />
+  <!--<include filename="$(find mit_drcsim_scripts)/models/mit_robot_hands/drake_urdfs/xacro/sandia_hand_drake.urdf.xacro" />-->
+  <include filename="$(find mit_drcsim_scripts)/models/mit_robot_hands/drake_urdfs/xacro/sandia_hand_simple_shapes_drake.urdf.xacro" />
   <include filename="$(find mit_drcsim_scripts)/models/mit_robot_hands/floatingbase_urdfs/xacro/floating_base.urdf.xacro" />
   <link name="world">

File: software/models/mit_gazebo_models/mit_robot_hands/floatingbase_urdfs/xacro/sandia_hand_drake_right_w_floating_base.urdf.xacro (robot description, xacro)
@@ -6,6 +6,6 @@
 <!--  derived from /usr/share/sandia-hand-5.1/ros/sandia_hand_description/robots/sandia_hand_right_on_box.urdf.xacro-->
   <!-- Commenting out urdf with meshes, using simple collision shapes instead -->
-  <!--<include filename="$(find mit_drcsim_scripts)/models/mit_robot_hands/drake_urdfs/new_xacro/sandia_hand_drake.urdf.xacro" />-->
-  <include filename="$(find mit_drcsim_scripts)/models/mit_robot_hands/drake_urdfs/new_xacro/sandia_hand_simple_shapes_drake.urdf.xacro" />
+  <!--<include filename="$(find mit_drcsim_scripts)/models/mit_robot_hands/drake_urdfs/xacro/sandia_hand_drake.urdf.xacro" />-->
+  <include filename="$(find mit_drcsim_scripts)/models/mit_robot_hands/drake_urdfs/xacro/sandia_hand_simple_shapes_drake.urdf.xacro" />
   <include filename="$(find mit_drcsim_scripts)/models/mit_robot_hands/floatingbase_urdfs/xacro/floating_base.urdf.xacro" />
   <link name="world">

Commit message: git-svn-id: https://svn.csail.mit.edu/drc@1725 c7283977-0100-402a-a91a-fa70b306dbfe

File: software/models/mit_gazebo_models/mit_robot_hands/floatingbase_urdfs/sandia_hand_drake_left_floating.urdf (robot description, URDF)
Before this commit: robot sandia_hand_left, 43 links, 42 joints
Joints:
- joint left_base_pitch: limit lower=-1.57079 upper=1.57079 effort=1 velocity=1 -> lower=-6.2832 upper=6.2832 effort=1 velocity=1
- joint left_base_roll: limit lower=-1.57079 upper=1.57079 effort=1 velocity=1 -> lower=-6.2832 upper=6.2832 effort=1 velocity=1
- joint left_base_yaw: limit lower=-1.57079 upper=1.57079 effort=1 velocity=1 -> lower=-6.2832 upper=6.2832 effort=1 velocity=1

File: software/models/mit_gazebo_models/mit_robot_hands/floatingbase_urdfs/sandia_hand_drake_right_floating.urdf (robot description, URDF)
Before this commit: robot sandia_hand_right, 43 links, 42 joints
Joints:
- joint right_base_pitch: limit lower=-1.57079 upper=1.57079 effort=1 velocity=1 -> lower=-6.2832 upper=6.2832 effort=1 velocity=1
- joint right_base_roll: limit lower=-1.57079 upper=1.57079 effort=1 velocity=1 -> lower=-6.2832 upper=6.2832 effort=1 velocity=1
- joint right_base_yaw: limit lower=-1.57079 upper=1.57079 effort=1 velocity=1 -> lower=-6.2832 upper=6.2832 effort=1 velocity=1

File: software/models/mit_gazebo_models/mit_robot_hands/floatingbase_urdfs/sandia_hands_floating.urdf (robot description, URDF)
Before this commit: robot sandia_hands, 71 links, 70 joints
Joints:
- joint left_base_pitch: limit lower=-1.57079 upper=1.57079 effort=1 velocity=1 -> lower=-6.2832 upper=6.2832 effort=1 velocity=1
- joint left_base_roll: limit lower=-1.57079 upper=1.57079 effort=1 velocity=1 -> lower=-6.2832 upper=6.2832 effort=1 velocity=1
- joint left_base_yaw: limit lower=-1.57079 upper=1.57079 effort=1 velocity=1 -> lower=-6.2832 upper=6.2832 effort=1 velocity=1
- joint right_base_pitch: limit lower=-1.57079 upper=1.57079 effort=1 velocity=1 -> lower=-6.2832 upper=6.2832 effort=1 velocity=1
- joint right_base_roll: limit lower=-1.57079 upper=1.57079 effort=1 velocity=1 -> lower=-6.2832 upper=6.2832 effort=1 velocity=1
- joint right_base_yaw: limit lower=-1.57079 upper=1.57079 effort=1 velocity=1 -> lower=-6.2832 upper=6.2832 effort=1 velocity=1

File: software/models/mit_gazebo_models/mit_robot_hands/floatingbase_urdfs/xacro/floating_base.urdf.xacro (robot description, xacro)
@@ -82,5 +82,5 @@
       <parent link="${side}_base_z"/>
       <child link="${side}_base_roll"/>
-      <limit lower="-1.57079" upper="1.57079" effort="1" velocity="1"/>
+      <limit lower="-6.2832" upper="6.2832" effort="1" velocity="1"/>
       <safety_controller soft_lower_limit="${-1.57079-10.0}" soft_upper_limit="${1.57079+10.0}" k_position="1000.0" k_velocity="1000.0"/>
       <dynamics damping="0.1"/>
@@ -91,5 +91,5 @@
       <parent link="${side}_base_roll"/>
       <child link="${side}_base_pitch"/>
-      <limit lower="-1.57079" upper="1.57079" effort="1" velocity="1"/>
+      <limit lower="-6.2832" upper="6.2832" effort="1" velocity="1"/>
       <safety_controller soft_lower_limit="${-1.57079-10.0}" soft_upper_limit="${1.57079+10.0}" k_position="1000.0" k_velocity="1000.0"/>
       <dynamics damping="0.1"/>
@@ -100,5 +100,5 @@
       <parent link="${side}_base_pitch"/>
       <child link="${side}_base_yaw"/>
-      <limit lower="-1.57079" upper="1.57079" effort="1" velocity="1"/>
+      <limit lower="-6.2832" upper="6.2832" effort="1" velocity="1"/>
       <safety_controller soft_lower_limit="${-1.57079-10.0}" soft_upper_limit="${1.57079+10.0}" k_position="1000.0" k_velocity="1000.0"/>
       <dynamics damping="0.1"/>
