Commit message: git-svn-id: https://svn.csail.mit.edu/drc@2613 c7283977-0100-402a-a91a-fa70b306dbfe

File: software/models/mit_gazebo_models/mit_robot_hands/floatingbase_urdfs/sandia_hands_floating.urdf (robot description, URDF)
Before this commit: robot sandia_hands, 71 links, 70 joints
Joints:
- joint left_f0_j0: limit lower=-1.57079632679 upper=1.57079632679 effort=1 velocity=1 -> lower=-1.57079632679 upper=1.57079632679 effort=11 velocity=1
- joint left_f0_j1: limit lower=-1.57079632679 upper=1.57079632679 effort=1 velocity=1 -> lower=-1.57079632679 upper=1.57079632679 effort=28 velocity=1
- joint left_f0_j2: limit lower=-1.57079632679 upper=1.57079632679 effort=1 velocity=1 -> lower=-1.57079632679 upper=1.57079632679 effort=28 velocity=1
- joint left_f1_j0: limit lower=-1.57079632679 upper=1.57079632679 effort=1 velocity=1 -> lower=-1.57079632679 upper=1.57079632679 effort=11 velocity=1
- joint left_f1_j1: limit lower=-1.57079632679 upper=1.57079632679 effort=1 velocity=1 -> lower=-1.57079632679 upper=1.57079632679 effort=28 velocity=1
- joint left_f1_j2: limit lower=-1.57079632679 upper=1.57079632679 effort=1 velocity=1 -> lower=-1.57079632679 upper=1.57079632679 effort=28 velocity=1
- joint left_f2_j0: limit lower=-1.57079632679 upper=1.57079632679 effort=1 velocity=1 -> lower=-1.57079632679 upper=1.57079632679 effort=11 velocity=1
- joint left_f2_j1: limit lower=-1.57079632679 upper=1.57079632679 effort=1 velocity=1 -> lower=-1.57079632679 upper=1.57079632679 effort=28 velocity=1
- joint left_f2_j2: limit lower=-1.57079632679 upper=1.57079632679 effort=1 velocity=1 -> lower=-1.57079632679 upper=1.57079632679 effort=28 velocity=1
- joint left_f3_j0: limit lower=-1.57079632679 upper=1.57079632679 effort=1 velocity=1 -> lower=-1.57079632679 upper=1.57079632679 effort=11 velocity=1
- joint left_f3_j1: limit lower=-1.57079632679 upper=1.57079632679 effort=1 velocity=1 -> lower=-1.57079632679 upper=1.57079632679 effort=28 velocity=1
- joint left_f3_j2: limit lower=-1.57079632679 upper=1.57079632679 effort=1 velocity=1 -> lower=-1.57079632679 upper=1.57079632679 effort=28 velocity=1
- joint right_f0_j0: limit lower=-1.57079632679 upper=1.57079632679 effort=1 velocity=1 -> lower=-1.57079632679 upper=1.57079632679 effort=11 velocity=1
- joint right_f0_j1: limit lower=-1.57079632679 upper=1.57079632679 effort=1 velocity=1 -> lower=-1.57079632679 upper=1.57079632679 effort=28 velocity=1
- joint right_f0_j2: limit lower=-1.57079632679 upper=1.57079632679 effort=1 velocity=1 -> lower=-1.57079632679 upper=1.57079632679 effort=28 velocity=1
- joint right_f1_j0: limit lower=-1.57079632679 upper=1.57079632679 effort=1 velocity=1 -> lower=-1.57079632679 upper=1.57079632679 effort=11 velocity=1
- joint right_f1_j1: limit lower=-1.57079632679 upper=1.57079632679 effort=1 velocity=1 -> lower=-1.57079632679 upper=1.57079632679 effort=28 velocity=1
- joint right_f1_j2: limit lower=-1.57079632679 upper=1.57079632679 effort=1 velocity=1 -> lower=-1.57079632679 upper=1.57079632679 effort=28 velocity=1
- joint right_f2_j0: limit lower=-1.57079632679 upper=1.57079632679 effort=1 velocity=1 -> lower=-1.57079632679 upper=1.57079632679 effort=11 velocity=1
- joint right_f2_j1: limit lower=-1.57079632679 upper=1.57079632679 effort=1 velocity=1 -> lower=-1.57079632679 upper=1.57079632679 effort=28 velocity=1
- joint right_f2_j2: limit lower=-1.57079632679 upper=1.57079632679 effort=1 velocity=1 -> lower=-1.57079632679 upper=1.57079632679 effort=28 velocity=1
- joint right_f3_j0: limit lower=-1.57079632679 upper=1.57079632679 effort=1 velocity=1 -> lower=-1.57079632679 upper=1.57079632679 effort=11 velocity=1
- joint right_f3_j1: limit lower=-1.57079632679 upper=1.57079632679 effort=1 velocity=1 -> lower=-1.57079632679 upper=1.57079632679 effort=28 velocity=1
- joint right_f3_j2: limit lower=-1.57079632679 upper=1.57079632679 effort=1 velocity=1 -> lower=-1.57079632679 upper=1.57079632679 effort=28 velocity=1
