Commit message: updated drake model to atlas 2.2.0
git-svn-id: https://svn.csail.mit.edu/drc@2274 c7283977-0100-402a-a91a-fa70b306dbfe

File: software/models/mit_gazebo_models/mit_robot_drake/model_foot_contact.urdf (robot description, URDF)
Before this commit: robot atlas, 29 links, 28 joints
Links:
- link l_foot: mass 1.634 -> 0.817
- link l_talus: mass 0.1 -> 0.817
- link r_foot: mass 1.634 -> 0.817
- link r_talus: mass 0.1 -> 0.817

File: software/models/mit_gazebo_models/mit_robot_drake/model_minimal_contact.urdf (robot description, URDF)
Before this commit: robot atlas, 29 links, 28 joints
Links:
- link l_foot: mass 1.634 -> 0.817
- link l_talus: mass 0.1 -> 0.817
- link r_foot: mass 1.634 -> 0.817
- link r_talus: mass 0.1 -> 0.817

File: software/models/mit_gazebo_models/mit_robot_drake/model_minimal_contact_with_hands.urdf (robot description, URDF)
Before this commit: robot atlas, 101 links, 100 joints
Links:
- link l_foot: mass 1.634 -> 0.817
- link l_talus: mass 0.1 -> 0.817
- link r_foot: mass 1.634 -> 0.817
- link r_talus: mass 0.1 -> 0.817

File: software/models/mit_gazebo_models/mit_robot_drake/xacro/atlas_skeleton_foot_contact.urdf (robot description, URDF)
Before this commit: robot drc_skeleton, 28 links, 28 joints
Links:
- link l_foot: mass 1.634 -> 0.817
- link l_talus: mass 0.1 -> 0.817
- link r_foot: mass 1.634 -> 0.817
- link r_talus: mass 0.1 -> 0.817

File: software/models/mit_gazebo_models/mit_robot_drake/xacro/atlas_skeleton_minimal_contact.urdf (robot description, URDF)
Before this commit: robot drc_skeleton, 28 links, 28 joints
Links:
- link l_foot: mass 1.634 -> 0.817
- link l_talus: mass 0.1 -> 0.817
- link r_foot: mass 1.634 -> 0.817
- link r_talus: mass 0.1 -> 0.817
