Commit message: added toenails to simple visuals model
git-svn-id: https://svn.csail.mit.edu/drc@4736 c7283977-0100-402a-a91a-fa70b306dbfe

File: software/models/mit_gazebo_models/mit_robot_drake/model_simple_visuals_point_hands.urdf (robot description, URDF)
Before this commit: robot atlas, 31 links, 30 joints
Links:
- link l_foot: geometry collision box size=0.26 0.124887 0.05; collision sphere radius=0
- link r_foot: geometry collision box size=0.26 0.124887 0.05; collision sphere radius=0
