Commit message: Adds "hook" contact group to Drake atlas models
git-svn-id: https://svn.csail.mit.edu/drc@4761 c7283977-0100-402a-a91a-fa70b306dbfe

File: software/models/mit_gazebo_models/mit_robot_drake/model_minimal_contact_with_hands.urdf (robot description, URDF)
Before this commit: robot atlas, 101 links, 100 joints
Links:
- added link left_hook; collision sphere radius=0; collision sphere radius=0
- added link right_hook; collision sphere radius=0; collision sphere radius=0
Joints:
- added joint left_hook_joint: type fixed, parent left_palm, child left_hook, origin xyz=0.044 0.04 -0.005 rpy=0 0 -0.79
- added joint right_hook_joint: type fixed, parent right_palm, child right_hook, origin xyz=0.044 -0.04 -0.005 rpy=0 0 0.79

File: software/models/mit_gazebo_models/mit_robot_drake/model_simple_visuals.urdf (robot description, URDF)
Before this commit: robot atlas, 31 links, 30 joints
Links:
- added link left_hook; collision sphere radius=0; collision sphere radius=0
- added link right_hook; collision sphere radius=0; collision sphere radius=0
Joints:
- added joint left_hook_joint: type fixed, parent left_palm, child left_hook, origin xyz=0.044 0.04 -0.005 rpy=0 0 -0.79
- added joint right_hook_joint: type fixed, parent right_palm, child right_hook, origin xyz=0.044 -0.04 -0.005 rpy=0 0 0.79

File: software/models/mit_gazebo_models/mit_robot_hands/drake_urdfs/sandia_hand_drake_left.urdf (robot description, URDF)
Before this commit: robot sandia_hand_left, 37 links, 36 joints
Links:
- added link left_hook; collision sphere radius=0; collision sphere radius=0
Joints:
- added joint left_hook_joint: type fixed, parent left_palm, child left_hook, origin xyz=0.044 0.04 -0.005 rpy=0 0 -0.79

File: software/models/mit_gazebo_models/mit_robot_hands/drake_urdfs/sandia_hand_drake_right.urdf (robot description, URDF)
Before this commit: robot sandia_hand_right, 37 links, 36 joints
Links:
- added link right_hook; collision sphere radius=0; collision sphere radius=0
Joints:
- added joint right_hook_joint: type fixed, parent right_palm, child right_hook, origin xyz=0.044 -0.04 -0.005 rpy=0 0 0.79

File: software/models/mit_gazebo_models/mit_robot_hands/drake_urdfs/xacro/sandia_hand_simple_shapes_drake.urdf.xacro (robot description, xacro)
@@ -15,4 +15,18 @@
   <include filename="$(find sandia_hand_description)/urdf/sandia_hand.transmission.xacro" />
   <xacro:property name="M_pi" value="3.1415926535897931" />
+  <xacro:macro name="collision_point" params="group xyz visualize">
+    <collision group="${group}">
+      <origin rpy="0 0 0" xyz="${xyz}"/>
+      <geometry>
+        <sphere radius="0"/>
+      </geometry>
+    </collision>
+    <visual>
+      <origin rpy="0 0 0" xyz="${xyz}"/>
+      <geometry>
+        <sphere radius="${visualize*0.01}"/>
+      </geometry>
+    </visual>
+  </xacro:macro>
   <xacro:macro name="finger" params="idx x y z r p yaw side reflect">
     <link name="${side}_f${idx}_base">
@@ -751,4 +765,13 @@
       <child link="${side}_palm"/>
       <insert_block name="origin" />
+    </joint>
+    <link name="${side}_hook">
+      <xacro:collision_point group="default" xyz="-0.045 ${reflect*0.015} -0.03" visualize="1"/>
+      <xacro:collision_point group="default" xyz="-0.045 ${reflect*0.015} 0.03" visualize="1"/>
+    </link>
+    <joint name="${side}_hook_joint" type="fixed">
+      <origin xyz="0.044 ${-0.04*reflect} -0.005" rpy="0 0 ${0.79*reflect}"/>
+      <parent link="${side}_palm"/>
+      <child link="${side}_hook"/>
     </joint>
     <xacro:finger side="${side}" idx="0" x="0.140" y="0.00000" z="0" r="0" p="0" yaw="${0.3*reflect}" reflect="${reflect}" />

File: software/models/mit_gazebo_models/mit_robot_hands/drake_urdfs/xacro/sandia_palm_simple_shapes_drake.urdf.xacro (robot description, xacro)
@@ -169,4 +169,13 @@
       <insert_block name="origin" />
     </joint>
+    <link name="${side}_hook">
+      <xacro:collision_point group="default" xyz="-0.045 ${reflect*0.015} -0.03" visualize="1"/>
+      <xacro:collision_point group="default" xyz="-0.045 ${reflect*0.015} 0.03" visualize="1"/>
+    </link>
+    <joint name="${side}_hook_joint" type="fixed">
+      <origin xyz="0.044 ${-0.04*reflect} -0.005" rpy="0 0 ${0.79*reflect}"/>
+      <parent link="${side}_palm"/>
+      <child link="${side}_hook"/>
+    </joint>
     <!-- not needed unless simulating the hand by itself
     <xacro:sandia_hand_gazebo side="${side}" />

File: software/models/mit_gazebo_models/mit_robot_hands/floatingbase_urdfs/sandia_hand_drake_left_floating.urdf (robot description, URDF)
Before this commit: robot sandia_hand_left, 43 links, 42 joints
Links:
- added link left_hook; collision sphere radius=0; collision sphere radius=0
Joints:
- added joint left_hook_joint: type fixed, parent left_palm, child left_hook, origin xyz=0.044 0.04 -0.005 rpy=0 0 -0.79

File: software/models/mit_gazebo_models/mit_robot_hands/floatingbase_urdfs/sandia_hand_drake_right_floating.urdf (robot description, URDF)
Before this commit: robot sandia_hand_right, 43 links, 42 joints
Links:
- added link right_hook; collision sphere radius=0; collision sphere radius=0
Joints:
- added joint right_hook_joint: type fixed, parent right_palm, child right_hook, origin xyz=0.044 -0.04 -0.005 rpy=0 0 0.79
