Commit message: Adds model_simple_visuals.urdf.
git-svn-id: https://svn.csail.mit.edu/drc@4856 c7283977-0100-402a-a91a-fa70b306dbfe

File: software/models/mit_gazebo_models/mit_robot_drake/model_simple_visuals.urdf (robot description, URDF)
Before this commit: robot atlas, 33 links, 32 joints
Links:
- link l_foot: geometry collision box size=0.26 0.124887 0.05; collision sphere radius=0
- link l_larm: geometry collision box size=0.135 0.15 0.06; collision cylinder length=0.125 radius=0.045
- link pelvis: geometry collision box size=0.1 0.15 0.2; collision box size=0.1 0.15 0.2
- link r_foot: geometry collision box size=0.26 0.124887 0.05; collision sphere radius=0
- link r_larm: geometry collision box size=0.135 0.15 0.06; collision cylinder length=0.125 radius=0.045
