Commit message: updating palm to hand transform to the correct one in xacro files for fixed joint hands and sandia hands
git-svn-id: https://svn.csail.mit.edu/drc/trunk@6347 c7283977-0100-402a-a91a-fa70b306dbfe

File: software/models/mit_gazebo_models/mit_robot_drake/model_minimal_contact_fixedjoint_hands.urdf (robot description, URDF)
Before this commit: robot atlas, 95 links, 94 joints
Joints:
- joint left_sandia_hand_joint: origin xyz=0  0.1 0 rpy= 1.57079 0  1.57079 -> xyz=0  0.145 0 rpy=0 0  1.57079
- joint right_sandia_hand_joint: origin xyz=0 -0.1 0 rpy=-1.57079 0 -1.57079 -> xyz=0 -0.145 0 rpy=0.0 0 -1.57079

File: software/models/mit_gazebo_models/mit_robot_drake/xacro/atlas_fixedjoint_hands.urdf.xacro (robot description, xacro)
@@ -3,8 +3,8 @@
   <include filename="$(find sandia_hand_description)/urdf/sandia_hand_simple_shapes.urdf.xacro" />
   <xacro:sandia_hand side="right" parent="r_hand" reflect="1" joint_type="fixed" thumb_angle="0">
-	<origin xyz="0 -0.1 0" rpy="-1.57079 0 -1.57079"/>
+	 <origin xyz="0 -0.145 0" rpy="0.0 0 -1.57079"/>
   </xacro:sandia_hand>
   <xacro:sandia_hand side="left" parent="l_hand" reflect="-1" joint_type="fixed" thumb_angle="0">
-	<origin xyz="0  0.1 0" rpy=" 1.57079 0  1.57079"/>
+	 <origin xyz="0  0.145 0" rpy="0 0  1.57079"/>
   </xacro:sandia_hand>
   <include filename="$(find mit_drcsim_scripts)/models/mit_robot_drake/xacro/atlas.transmission" />

File: software/models/mit_gazebo_models/mit_robot_drake/xacro/atlas_sandia_hands.urdf.xacro (robot description, xacro)
@@ -4,8 +4,8 @@
   <!-- adding an offset in the urdf to account for the ft sensor and the coupling plate, chaning origin form 0.1 to 0.145 for sandia, and 0.05 to 0.095 for irobot-->
   <xacro:sandia_hand side="right" parent="r_hand" reflect="1" joint_type="revolute" thumb_angle="0">
-	<origin xyz="0 -0.145 0" rpy="-1.57079 0 -1.57079"/>
+    <origin xyz="0 -0.145 0" rpy="0.0 0 -1.57079"/>
   </xacro:sandia_hand>
   <xacro:sandia_hand side="left" parent="l_hand" reflect="-1" joint_type="revolute" thumb_angle="0">
-	<origin xyz="0  0.145 0" rpy=" 1.57079 0  1.57079"/>
+    <origin xyz="0  0.145 0" rpy="0 0  1.57079"/>
   </xacro:sandia_hand>
   <include filename="$(find mit_drcsim_scripts)/models/mit_robot_drake/xacro/atlas.transmission" />
