Commit message: Added collision groups to drake Atlas model feet
git-svn-id: https://svn.csail.mit.edu/drc@1498 c7283977-0100-402a-a91a-fa70b306dbfe

File: software/models/mit_gazebo_models/mit_robot_drake/model_minimal_contact.urdf (robot description, URDF)
Before this commit: robot atlas, 29 links, 28 joints
Links:
- link head: geometry visual mesh filename=/home/rdeits/drc/ros_workspace/mit_drcsim_scripts/models/mi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 scale=1 1 1
- link l_clav: geometry visual mesh filename=/home/rdeits/drc/ros_workspace/mit_drcsim_scripts/models/mi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 scale=1 1 1
- link l_farm: geometry visual mesh filename=/home/rdeits/drc/ros_workspace/mit_drcsim_scripts/models/mi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 scale=1 1 1
- link l_foot: geometry collision sphere radius=0; collision sphere radius=0
- link l_hand: geometry visual mesh filename=/home/rdeits/drc/ros_workspace/mit_drcsim_scripts/models/mi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 scale=1 1 1
- link l_larm: geometry visual mesh filename=/home/rdeits/drc/ros_workspace/mit_drcsim_scripts/models/mi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 scale=1 1 1
- link l_lglut: geometry visual mesh filename=/home/rdeits/drc/ros_workspace/mit_drcsim_scripts/models/mi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 scale=1 1 1
- link l_lleg: geometry visual mesh filename=/home/rdeits/drc/ros_workspace/mit_drcsim_scripts/models/mi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 scale=1 1 1
- link l_scap: geometry visual mesh filename=/home/rdeits/drc/ros_workspace/mit_drcsim_scripts/models/mi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 scale=1 1 1
- link l_talus: geometry visual mesh filename=/home/rdeits/drc/ros_workspace/mit_drcsim_scripts/models/mi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 scale=1 1 1
- link l_uarm: geometry visual mesh filename=/home/rdeits/drc/ros_workspace/mit_drcsim_scripts/models/mi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 scale=1 1 1
- link l_uglut: geometry visual mesh filename=/home/rdeits/drc/ros_workspace/mit_drcsim_scripts/models/mi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 scale=1 1 1
- link l_uleg: geometry visual mesh filename=/home/rdeits/drc/ros_workspace/mit_drcsim_scripts/models/mi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 scale=1 1 1
- link ltorso: geometry visual mesh filename=/home/rdeits/drc/ros_workspace/mit_drcsim_scripts/models/mi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 scale=1 1 1
- link mtorso: geometry visual mesh filename=/home/rdeits/drc/ros_workspace/mit_drcsim_scripts/models/mi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 scale=1 1 1
- link pelvis: geometry visual mesh filename=/home/rdeits/drc/ros_workspace/mit_drcsim_scripts/models/mi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 scale=1 1 1
- link r_clav: geometry visual mesh filename=/home/rdeits/drc/ros_workspace/mit_drcsim_scripts/models/mi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 scale=1 1 1
- link r_farm: geometry visual mesh filename=/home/rdeits/drc/ros_workspace/mit_drcsim_scripts/models/mi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 scale=1 1 1
- link r_foot: geometry collision sphere radius=0; collision sphere radius=0
- link r_hand: geometry visual mesh filename=/home/rdeits/drc/ros_workspace/mit_drcsim_scripts/models/mi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 scale=1 1 1
- link r_larm: geometry visual mesh filename=/home/rdeits/drc/ros_workspace/mit_drcsim_scripts/models/mi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 scale=1 1 1
- link r_lglut: geometry visual mesh filename=/home/rdeits/drc/ros_workspace/mit_drcsim_scripts/models/mi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 scale=1 1 1
- link r_lleg: geometry visual mesh filename=/home/rdeits/drc/ros_workspace/mit_drcsim_scripts/models/mi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 scale=1 1 1
- link r_scap: geometry visual mesh filename=/home/rdeits/drc/ros_workspace/mit_drcsim_scripts/models/mi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 scale=1 1 1
- link r_talus: geometry visual mesh filename=/home/rdeits/drc/ros_workspace/mit_drcsim_scripts/models/mi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 scale=1 1 1
- link r_uarm: geometry visual mesh filename=/home/rdeits/drc/ros_workspace/mit_drcsim_scripts/models/mi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 scale=1 1 1
- link r_uglut: geometry visual mesh filename=/home/rdeits/drc/ros_workspace/mit_drcsim_scripts/models/mi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 scale=1 1 1
- link r_uleg: geometry visual mesh filename=/home/rdeits/drc/ros_workspace/mit_drcsim_scripts/models/mi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 scale=1 1 1
- link utorso: geometry visual mesh filename=/home/rdeits/drc/ros_workspace/mit_drcsim_scripts/models/mi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 scale=1 1 1

Commit message: various commits and updates
git-svn-id: https://svn.csail.mit.edu/drc@1546 c7283977-0100-402a-a91a-fa70b306dbfe

File: software/models/mit_gazebo_models/mit_robot_drake/model_minimal_contact.urdf (robot description, URDF)
Before this commit: robot atlas, 29 links, 28 joints
Links:
- link head: geometry visual mesh filename=/home/mfallon/drc/ros_workspace/mit_drcsim_scripts/models/m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 scale=1 1 1
- link l_clav: geometry visual mesh filename=/home/mfallon/drc/ros_workspace/mit_drcsim_scripts/models/m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 scale=1 1 1
- link l_farm: geometry visual mesh filename=/home/mfallon/drc/ros_workspace/mit_drcsim_scripts/models/m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 scale=1 1 1
- link l_foot: geometry collision sphere radius=0; collision sphere radius=0
- link l_hand: geometry visual mesh filename=/home/mfallon/drc/ros_workspace/mit_drcsim_scripts/models/m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 scale=1 1 1
- link l_larm: geometry visual mesh filename=/home/mfallon/drc/ros_workspace/mit_drcsim_scripts/models/m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 scale=1 1 1
- link l_lglut: geometry visual mesh filename=/home/mfallon/drc/ros_workspace/mit_drcsim_scripts/models/m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 scale=1 1 1
- link l_lleg: geometry visual mesh filename=/home/mfallon/drc/ros_workspace/mit_drcsim_scripts/models/m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 scale=1 1 1
- link l_scap: geometry visual mesh filename=/home/mfallon/drc/ros_workspace/mit_drcsim_scripts/models/m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 scale=1 1 1
- link l_talus: geometry visual mesh filename=/home/mfallon/drc/ros_workspace/mit_drcsim_scripts/models/m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 scale=1 1 1
- link l_uarm: geometry visual mesh filename=/home/mfallon/drc/ros_workspace/mit_drcsim_scripts/models/m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 scale=1 1 1
- link l_uglut: geometry visual mesh filename=/home/mfallon/drc/ros_workspace/mit_drcsim_scripts/models/m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 scale=1 1 1
- link l_uleg: geometry visual mesh filename=/home/mfallon/drc/ros_workspace/mit_drcsim_scripts/models/m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 scale=1 1 1
- link ltorso: geometry visual mesh filename=/home/mfallon/drc/ros_workspace/mit_drcsim_scripts/models/m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 scale=1 1 1
- link mtorso: geometry visual mesh filename=/home/mfallon/drc/ros_workspace/mit_drcsim_scripts/models/m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 scale=1 1 1
- link pelvis: geometry visual mesh filename=/home/mfallon/drc/ros_workspace/mit_drcsim_scripts/models/m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 scale=1 1 1
- link r_clav: geometry visual mesh filename=/home/mfallon/drc/ros_workspace/mit_drcsim_scripts/models/m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 scale=1 1 1
- link r_farm: geometry visual mesh filename=/home/mfallon/drc/ros_workspace/mit_drcsim_scripts/models/m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 scale=1 1 1
- link r_foot: geometry collision sphere radius=0; collision sphere radius=0
- link r_hand: geometry visual mesh filename=/home/mfallon/drc/ros_workspace/mit_drcsim_scripts/models/m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 scale=1 1 1
- link r_larm: geometry visual mesh filename=/home/mfallon/drc/ros_workspace/mit_drcsim_scripts/models/m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 scale=1 1 1
- link r_lglut: geometry visual mesh filename=/home/mfallon/drc/ros_workspace/mit_drcsim_scripts/models/m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 scale=1 1 1
- link r_lleg: geometry visual mesh filename=/home/mfallon/drc/ros_workspace/mit_drcsim_scripts/models/m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 scale=1 1 1
- link r_scap: geometry visual mesh filename=/home/mfallon/drc/ros_workspace/mit_drcsim_scripts/models/m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 scale=1 1 1
- link r_talus: geometry visual mesh filename=/home/mfallon/drc/ros_workspace/mit_drcsim_scripts/models/m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 scale=1 1 1
- link r_uarm: geometry visual mesh filename=/home/mfallon/drc/ros_workspace/mit_drcsim_scripts/models/m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 scale=1 1 1
- link r_uglut: geometry visual mesh filename=/home/mfallon/drc/ros_workspace/mit_drcsim_scripts/models/m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 scale=1 1 1
- link r_uleg: geometry visual mesh filename=/home/mfallon/drc/ros_workspace/mit_drcsim_scripts/models/m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 scale=1 1 1
- link utorso: geometry visual mesh filename=/home/mfallon/drc/ros_workspace/mit_drcsim_scripts/models/m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 scale=1 1 1

Commit message: updated to latest atlas model specs
git-svn-id: https://svn.csail.mit.edu/drc@1570 c7283977-0100-402a-a91a-fa70b306dbfe

File: software/models/mit_gazebo_models/mit_robot_drake/model_minimal_contact.urdf (robot description, URDF)
Before this commit: robot atlas, 29 links, 28 joints
Links:
- link head: mass 2.6 -> 1.4199; geometry visual mesh filename=/home/scottk/drc/ros_workspace/mit_drcsim_scripts/models/mu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
- link l_clav: geometry visual mesh filename=/home/scottk/drc/ros_workspace/mit_drcsim_scripts/models/mi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 scale=1 1 1
- link l_farm: geometry visual mesh filename=/home/scottk/drc/ros_workspace/mit_drcsim_scripts/models/mi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 scale=1 1 1
- link l_foot: geometry collision sphere radius=0; collision sphere radius=0
- link l_hand: geometry visual mesh filename=/home/scottk/drc/ros_workspace/mit_drcsim_scripts/models/mi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 scale=1 1 1
- link l_larm: geometry visual mesh filename=/home/scottk/drc/ros_workspace/mit_drcsim_scripts/models/mi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 scale=1 1 1
- link l_lglut: geometry visual mesh filename=/home/scottk/drc/ros_workspace/mit_drcsim_scripts/models/mi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 scale=1 1 1
- link l_lleg: geometry visual mesh filename=/home/scottk/drc/ros_workspace/mit_drcsim_scripts/models/mi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 scale=1 1 1
- link l_scap: geometry visual mesh filename=/home/scottk/drc/ros_workspace/mit_drcsim_scripts/models/mi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 scale=1 1 1
- link l_talus: geometry visual mesh filename=/home/scottk/drc/ros_workspace/mit_drcsim_scripts/models/mi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 scale=1 1 1
- link l_uarm: geometry visual mesh filename=/home/scottk/drc/ros_workspace/mit_drcsim_scripts/models/mi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 scale=1 1 1
- link l_uglut: geometry visual mesh filename=/home/scottk/drc/ros_workspace/mit_drcsim_scripts/models/mi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 scale=1 1 1
- link l_uleg: geometry visual mesh filename=/home/scottk/drc/ros_workspace/mit_drcsim_scripts/models/mi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 scale=1 1 1
- link ltorso: geometry visual mesh filename=/home/scottk/drc/ros_workspace/mit_drcsim_scripts/models/mi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 scale=1 1 1
- link mtorso: geometry visual mesh filename=/home/scottk/drc/ros_workspace/mit_drcsim_scripts/models/mi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 scale=1 1 1
- link pelvis: geometry visual mesh filename=/home/scottk/drc/ros_workspace/mit_drcsim_scripts/models/mi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 scale=1 1 1
- link r_clav: geometry visual mesh filename=/home/scottk/drc/ros_workspace/mit_drcsim_scripts/models/mi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 scale=1 1 1
- link r_farm: geometry visual mesh filename=/home/scottk/drc/ros_workspace/mit_drcsim_scripts/models/mi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 scale=1 1 1
- link r_foot: geometry collision sphere radius=0; collision sphere radius=0
- link r_hand: geometry visual mesh filename=/home/scottk/drc/ros_workspace/mit_drcsim_scripts/models/mi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 scale=1 1 1
- link r_larm: geometry visual mesh filename=/home/scottk/drc/ros_workspace/mit_drcsim_scripts/models/mi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 scale=1 1 1
- link r_lglut: geometry visual mesh filename=/home/scottk/drc/ros_workspace/mit_drcsim_scripts/models/mi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 scale=1 1 1
- link r_lleg: geometry visual mesh filename=/home/scottk/drc/ros_workspace/mit_drcsim_scripts/models/mi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 scale=1 1 1
- link r_scap: geometry visual mesh filename=/home/scottk/drc/ros_workspace/mit_drcsim_scripts/models/mi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 scale=1 1 1
- link r_talus: geometry visual mesh filename=/home/scottk/drc/ros_workspace/mit_drcsim_scripts/models/mi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 scale=1 1 1
- link r_uarm: geometry visual mesh filename=/home/scottk/drc/ros_workspace/mit_drcsim_scripts/models/mi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 scale=1 1 1
- link r_uglut: geometry visual mesh filename=/home/scottk/drc/ros_workspace/mit_drcsim_scripts/models/mi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 scale=1 1 1
- link r_uleg: geometry visual mesh filename=/home/scottk/drc/ros_workspace/mit_drcsim_scripts/models/mi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 scale=1 1 1
- link utorso: geometry visual mesh filename=/home/scottk/drc/ros_workspace/mit_drcsim_scripts/models/mi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 scale=1 1 1
Joints:
- joint neck_ay: limit lower=-0.785398 upper=0.785398 effort=5 velocity=12 -> lower=-0.610865238 upper=1.13446401 effort=5 velocity=12; origin xyz=0.011 0 0.44 rpy=0 -0 0 -> xyz=0.16555 0 0.50823 rpy=0 -0 0
- joint r_arm_usy: axis 0 -0.5 0.866025 -> 0 0.5 -0.866025

File: software/models/mit_gazebo_models/mit_robot_drake/xacro/atlas.model.xacro (robot description, xacro)
@@ -1,9 +1,5 @@
-<robot xmlns:sensor="http://playerstage.sourceforge.net/gazebo/xmlschema/#sensor"
-       xmlns:controller="http://playerstage.sourceforge.net/gazebo/xmlschema/#controller"
-       xmlns:interface="http://playerstage.sourceforge.net/gazebo/xmlschema/#interface"
-       xmlns:xacro="http://playerstage.sourceforge.net/gazebo/xmlschema/#interface"
-       name="atlas" >
+<robot name="atlas" >
   <include filename="$(find mit_drcsim_scripts)/models/mit_robot_drake/xacro/atlas_skeleton_minimal_contact.urdf" />
-<!--  <include filename="$(find mit_drcsim_scripts)/models/mit_robot_drake/xacro/atlas_skeleton.urdf" /> -->
-  <include filename="$(find atlas_utils)/urdf/atlas.transmission" />
+  <include filename="$(find mit_drcsim_scripts)/models/mit_robot_drake/xacro/atlas.transmission" />
+  <include filename="$(find mit_drcsim_scripts)/models/mit_robot_drake/xacro/multisense_sl_no_contact.urdf" />
 </robot>

File: software/models/mit_gazebo_models/mit_robot_drake/xacro/atlas_skeleton_minimal_contact.urdf (robot description, URDF)
Before this commit: robot drc_skeleton, 29 links, 28 joints
Links:
- removed link head
- link l_foot: geometry collision sphere radius=0; collision sphere radius=0
- link r_foot: geometry collision sphere radius=0; collision sphere radius=0
Joints:
- joint neck_ay: limit lower=-0.785398 upper=0.785398 effort=5 velocity=12 -> lower=-0.610865238 upper=1.13446401 effort=5 velocity=12; origin xyz=0.011 0 0.44 rpy=0 -0 0 -> xyz=0.16555 0 0.50823 rpy=0 -0 0
- joint r_arm_usy: axis 0 -0.5 0.866025 -> 0 0.5 -0.866025

Commit message: point hands are included by default
git-svn-id: https://svn.csail.mit.edu/drc@1575 c7283977-0100-402a-a91a-fa70b306dbfe

File: software/models/mit_gazebo_models/mit_robot_drake/model_minimal_contact.urdf (robot description, URDF)
Before this commit: robot atlas, 29 links, 28 joints
Links:
- added link l_hand_point_mass, mass 2.9; visual sphere radius=0.03
- added link r_hand_point_mass, mass 2.9; visual sphere radius=0.03
Joints:
- added joint l_hand_joint: type fixed, parent l_hand, child l_hand_point_mass, origin xyz=0.0089 0.1855 0.0047 rpy=0 0 0
- added joint r_hand_joint: type fixed, parent r_hand, child r_hand_point_mass, origin xyz=0.0089 -0.1855 -0.0047 rpy=0 0 0

File: software/models/mit_gazebo_models/mit_robot_drake/xacro/atlas.model.xacro (robot description, xacro)
@@ -1,4 +1,5 @@
 <robot name="atlas" >
   <include filename="$(find mit_drcsim_scripts)/models/mit_robot_drake/xacro/atlas_skeleton_minimal_contact.urdf" />
+  <include filename="$(find mit_drcsim_scripts)/models/mit_robot_drake/xacro/atlas_point_mass_hands.urdf" />
   <include filename="$(find mit_drcsim_scripts)/models/mit_robot_drake/xacro/atlas.transmission" />
   <include filename="$(find mit_drcsim_scripts)/models/mit_robot_drake/xacro/multisense_sl_no_contact.urdf" />

File: software/models/mit_gazebo_models/mit_robot_drake/xacro/atlas_point_mass_hands.urdf (robot description, URDF)
Before this commit: robot atlas, 2 links, 2 joints
Links:
- link l_hand_point_mass: geometry visual sphere radius=0.03
- link r_hand_point_mass: geometry visual sphere radius=0.03

Commit message: working on changes to structure
git-svn-id: https://svn.csail.mit.edu/drc@1652 c7283977-0100-402a-a91a-fa70b306dbfe

File: software/models/mit_gazebo_models/mit_robot_drake/model_minimal_contact.urdf (robot description, URDF)
Before this commit: robot atlas, 31 links, 30 joints
Links:
- link head: geometry visual mesh filename=/home/mfallon/drc/ros_workspace/mit_drcsim_scripts/models/m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
- link l_clav: geometry visual mesh filename=/home/mfallon/drc/ros_workspace/mit_drcsim_scripts/models/m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 scale=1 1 1
- link l_farm: geometry visual mesh filename=/home/mfallon/drc/ros_workspace/mit_drcsim_scripts/models/m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 scale=1 1 1
- link l_foot: geometry collision sphere radius=0; collision sphere radius=0
- link l_hand: geometry visual mesh filename=/home/mfallon/drc/ros_workspace/mit_drcsim_scripts/models/m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 scale=1 1 1
- link l_larm: geometry visual mesh filename=/home/mfallon/drc/ros_workspace/mit_drcsim_scripts/models/m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 scale=1 1 1
- link l_lglut: geometry visual mesh filename=/home/mfallon/drc/ros_workspace/mit_drcsim_scripts/models/m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 scale=1 1 1
- link l_lleg: geometry visual mesh filename=/home/mfallon/drc/ros_workspace/mit_drcsim_scripts/models/m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 scale=1 1 1
- link l_scap: geometry visual mesh filename=/home/mfallon/drc/ros_workspace/mit_drcsim_scripts/models/m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 scale=1 1 1
- link l_talus: geometry visual mesh filename=/home/mfallon/drc/ros_workspace/mit_drcsim_scripts/models/m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 scale=1 1 1
- link l_uarm: geometry visual mesh filename=/home/mfallon/drc/ros_workspace/mit_drcsim_scripts/models/m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 scale=1 1 1
- link l_uglut: geometry visual mesh filename=/home/mfallon/drc/ros_workspace/mit_drcsim_scripts/models/m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 scale=1 1 1
- link l_uleg: geometry visual mesh filename=/home/mfallon/drc/ros_workspace/mit_drcsim_scripts/models/m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 scale=1 1 1
- link ltorso: geometry visual mesh filename=/home/mfallon/drc/ros_workspace/mit_drcsim_scripts/models/m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 scale=1 1 1
- link mtorso: geometry visual mesh filename=/home/mfallon/drc/ros_workspace/mit_drcsim_scripts/models/m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 scale=1 1 1
- link pelvis: geometry visual mesh filename=/home/mfallon/drc/ros_workspace/mit_drcsim_scripts/models/m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 scale=1 1 1
- link r_clav: geometry visual mesh filename=/home/mfallon/drc/ros_workspace/mit_drcsim_scripts/models/m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 scale=1 1 1
- link r_farm: geometry visual mesh filename=/home/mfallon/drc/ros_workspace/mit_drcsim_scripts/models/m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 scale=1 1 1
- link r_foot: geometry collision sphere radius=0; collision sphere radius=0
- link r_hand: geometry visual mesh filename=/home/mfallon/drc/ros_workspace/mit_drcsim_scripts/models/m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 scale=1 1 1
- link r_larm: geometry visual mesh filename=/home/mfallon/drc/ros_workspace/mit_drcsim_scripts/models/m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 scale=1 1 1
- link r_lglut: geometry visual mesh filename=/home/mfallon/drc/ros_workspace/mit_drcsim_scripts/models/m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 scale=1 1 1
- link r_lleg: geometry visual mesh filename=/home/mfallon/drc/ros_workspace/mit_drcsim_scripts/models/m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 scale=1 1 1
- link r_scap: geometry visual mesh filename=/home/mfallon/drc/ros_workspace/mit_drcsim_scripts/models/m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 scale=1 1 1
- link r_talus: geometry visual mesh filename=/home/mfallon/drc/ros_workspace/mit_drcsim_scripts/models/m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 scale=1 1 1
- link r_uarm: geometry visual mesh filename=/home/mfallon/drc/ros_workspace/mit_drcsim_scripts/models/m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 scale=1 1 1
- link r_uglut: geometry visual mesh filename=/home/mfallon/drc/ros_workspace/mit_drcsim_scripts/models/m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 scale=1 1 1
- link r_uleg: geometry visual mesh filename=/home/mfallon/drc/ros_workspace/mit_drcsim_scripts/models/m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 scale=1 1 1
- link utorso: geometry visual mesh filename=/home/mfallon/drc/ros_workspace/mit_drcsim_scripts/models/m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 scale=1 1 1

Commit message: urdf files are now regenerated on make
git-svn-id: https://svn.csail.mit.edu/drc@1732 c7283977-0100-402a-a91a-fa70b306dbfe

File: software/models/mit_gazebo_models/mit_robot_drake/model_minimal_contact.urdf (robot description, URDF)
Before this commit: robot atlas, 31 links, 30 joints
Links:
- link head: geometry visual mesh filename=/home/drc/drc/ros_workspace/mit_drcsim_scripts/models/multi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
- link l_clav: geometry visual mesh filename=/home/drc/drc/ros_workspace/mit_drcsim_scripts/models/mit_r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 scale=1 1 1
- link l_farm: geometry visual mesh filename=/home/drc/drc/ros_workspace/mit_drcsim_scripts/models/mit_r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 scale=1 1 1
- link l_foot: geometry collision sphere radius=0; collision sphere radius=0
- link l_hand: geometry visual mesh filename=/home/drc/drc/ros_workspace/mit_drcsim_scripts/models/mit_r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 scale=1 1 1
- link l_larm: geometry visual mesh filename=/home/drc/drc/ros_workspace/mit_drcsim_scripts/models/mit_r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 scale=1 1 1
- link l_lglut: geometry visual mesh filename=/home/drc/drc/ros_workspace/mit_drcsim_scripts/models/mit_r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 scale=1 1 1
- link l_lleg: geometry visual mesh filename=/home/drc/drc/ros_workspace/mit_drcsim_scripts/models/mit_r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 scale=1 1 1
- link l_scap: geometry visual mesh filename=/home/drc/drc/ros_workspace/mit_drcsim_scripts/models/mit_r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 scale=1 1 1
- link l_talus: geometry visual mesh filename=/home/drc/drc/ros_workspace/mit_drcsim_scripts/models/mit_r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 scale=1 1 1
- link l_uarm: geometry visual mesh filename=/home/drc/drc/ros_workspace/mit_drcsim_scripts/models/mit_r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 scale=1 1 1
- link l_uglut: geometry visual mesh filename=/home/drc/drc/ros_workspace/mit_drcsim_scripts/models/mit_r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 scale=1 1 1
- link l_uleg: geometry visual mesh filename=/home/drc/drc/ros_workspace/mit_drcsim_scripts/models/mit_r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 scale=1 1 1
- link ltorso: geometry visual mesh filename=/home/drc/drc/ros_workspace/mit_drcsim_scripts/models/mit_r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 scale=1 1 1
- link mtorso: geometry visual mesh filename=/home/drc/drc/ros_workspace/mit_drcsim_scripts/models/mit_r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 scale=1 1 1
- link pelvis: geometry visual mesh filename=/home/drc/drc/ros_workspace/mit_drcsim_scripts/models/mit_r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 scale=1 1 1
- link r_clav: geometry visual mesh filename=/home/drc/drc/ros_workspace/mit_drcsim_scripts/models/mit_r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 scale=1 1 1
- link r_farm: geometry visual mesh filename=/home/drc/drc/ros_workspace/mit_drcsim_scripts/models/mit_r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 scale=1 1 1
- link r_foot: geometry collision sphere radius=0; collision sphere radius=0
- link r_hand: geometry visual mesh filename=/home/drc/drc/ros_workspace/mit_drcsim_scripts/models/mit_r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 scale=1 1 1
- link r_larm: geometry visual mesh filename=/home/drc/drc/ros_workspace/mit_drcsim_scripts/models/mit_r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 scale=1 1 1
- link r_lglut: geometry visual mesh filename=/home/drc/drc/ros_workspace/mit_drcsim_scripts/models/mit_r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 scale=1 1 1
- link r_lleg: geometry visual mesh filename=/home/drc/drc/ros_workspace/mit_drcsim_scripts/models/mit_r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 scale=1 1 1
- link r_scap: geometry visual mesh filename=/home/drc/drc/ros_workspace/mit_drcsim_scripts/models/mit_r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 scale=1 1 1
- link r_talus: geometry visual mesh filename=/home/drc/drc/ros_workspace/mit_drcsim_scripts/models/mit_r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 scale=1 1 1
- link r_uarm: geometry visual mesh filename=/home/drc/drc/ros_workspace/mit_drcsim_scripts/models/mit_r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 scale=1 1 1
- link r_uglut: geometry visual mesh filename=/home/drc/drc/ros_workspace/mit_drcsim_scripts/models/mit_r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 scale=1 1 1
- link r_uleg: geometry visual mesh filename=/home/drc/drc/ros_workspace/mit_drcsim_scripts/models/mit_r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 scale=1 1 1
- link utorso: geometry visual mesh filename=/home/drc/drc/ros_workspace/mit_drcsim_scripts/models/mit_r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 scale=1 1 1

File: software/models/mit_gazebo_models/mit_robot_drake/xacro/atlas_with_hands.model.xacro (robot description, xacro)
@@ -8,10 +8,9 @@
   <!-- <include filename="$(find mit_drcsim_scripts)/models/mit_robot_hands/drake_urdfs/xacro/atlas_left_hand_drake.xacro" />
   <include filename="$(find mit_drcsim_scripts)/models/mit_robot_hands/drake_urdfs/xacro/atlas_right_hand_drake.xacro" /> -->
-  <include filename="$(find atlas_utils)/urdf/atlas.transmission" />
-  <include filename="$(find mit_drcsim_scripts)/models/mit_robot_hands/drake_urdfs/xacro/sandia_hand_drake.xacro" />
-  <xacro:sandia_hand side="l" parent="l_hand">
+ <include filename="$(find mit_drcsim_scripts)/models/mit_robot_hands/drake_urdfs/xacro/sandia_hand_simple_shapes_drake.urdf.xacro" />
+  <xacro:sandia_hand side="left" parent="l_hand" reflect="-1">
     <origin xyz="0 0.1 -0.03" rpy="0 3.1416  -1.57079"/>
   </xacro:sandia_hand>
-  <xacro:sandia_hand side="r" parent="r_hand">
+  <xacro:sandia_hand side="right" parent="r_hand" reflect="1">
     <origin xyz="0 -0.1 -0.03" rpy="0 3.1416  1.57079"/>
   </xacro:sandia_hand>
@@ -28,3 +27,5 @@
 <child link='left_palm'/>
 </joint> -->
+  <include filename="$(find mit_drcsim_scripts)/models/mit_robot_drake/xacro/atlas.transmission" />
+  <include filename="$(find mit_drcsim_scripts)/models/mit_robot_drake/xacro/multisense_sl_no_contact.urdf" />
 </robot>
