Commit message: merged ros minimal contact model with the non-ros version. the resulting model inherets the package notation and hand/leg contact points from the ros model. It uses the simpler foot 4 contact point layout from the non-ros model (that is consistent with the block feet being used in DRCSIM 2.0)
git-svn-id: https://svn.csail.mit.edu/drc@1841 c7283977-0100-402a-a91a-fa70b306dbfe

File: software/models/mit_gazebo_models/mit_robot_drake/model_minimal_contact.urdf (robot description, URDF)
Before this commit: robot atlas, 31 links, 30 joints
Links:
- removed link l_hand_point_mass
- removed link r_hand_point_mass
- link head: geometry visual mesh filename=package://multisense_sl/meshes/base_link.wrl
- link l_clav: geometry visual mesh filename=package://mit_robot/meshes/l_clav.wrl scale=1 1 1
- link l_farm: geometry visual mesh filename=package://mit_robot/meshes/l_farm.wrl scale=1 1 1
- link l_foot: geometry collision sphere radius=0; collision sphere radius=0
- link l_hand: geometry collision sphere radius=0; visual mesh filename=package://mit_robot/meshes/l_hand.wrl scale=1 1 1
- link l_larm: geometry visual mesh filename=package://mit_robot/meshes/l_larm.wrl scale=1 1 1
- link l_lglut: geometry visual mesh filename=package://mit_robot/meshes/l_lglut.wrl scale=1 1 1
- link l_lleg: geometry collision sphere radius=0; collision sphere radius=0
- link l_scap: geometry visual mesh filename=package://mit_robot/meshes/l_scap.wrl scale=1 1 1
- link l_talus: geometry visual mesh filename=package://mit_robot/meshes/l_talus.wrl scale=1 1 1
- link l_uarm: geometry visual mesh filename=package://mit_robot/meshes/l_uarm.wrl scale=1 1 1
- link l_uglut: geometry visual mesh filename=package://mit_robot/meshes/l_uglut.wrl scale=1 1 1
- link l_uleg: geometry visual mesh filename=package://mit_robot/meshes/l_uleg.wrl scale=1 1 1
- link ltorso: geometry visual mesh filename=package://mit_robot/meshes/ltorso.wrl scale=1 1 1
- link mtorso: geometry visual mesh filename=package://mit_robot/meshes/mtorso.wrl scale=1 1 1
- link pelvis: geometry visual mesh filename=package://mit_robot/meshes/pelvis.wrl scale=1 1 1
- link r_clav: geometry visual mesh filename=package://mit_robot/meshes/r_clav.wrl scale=1 1 1
- link r_farm: geometry visual mesh filename=package://mit_robot/meshes/r_farm.wrl scale=1 1 1
- link r_foot: geometry collision sphere radius=0; collision sphere radius=0
- link r_hand: geometry collision sphere radius=0; visual mesh filename=package://mit_robot/meshes/r_hand.wrl scale=1 1 1
- link r_larm: geometry visual mesh filename=package://mit_robot/meshes/r_larm.wrl scale=1 1 1
- link r_lglut: geometry visual mesh filename=package://mit_robot/meshes/r_lglut.wrl scale=1 1 1
- link r_lleg: geometry collision sphere radius=0; collision sphere radius=0
- link r_scap: geometry visual mesh filename=package://mit_robot/meshes/r_scap.wrl scale=1 1 1
- link r_talus: geometry visual mesh filename=package://mit_robot/meshes/r_talus.wrl scale=1 1 1
- link r_uarm: geometry visual mesh filename=package://mit_robot/meshes/r_uarm.wrl scale=1 1 1
- link r_uglut: geometry visual mesh filename=package://mit_robot/meshes/r_uglut.wrl scale=1 1 1
- link r_uleg: geometry visual mesh filename=package://mit_robot/meshes/r_uleg.wrl scale=1 1 1
- link utorso: geometry visual mesh filename=package://mit_robot/meshes/utorso.wrl scale=1 1 1
Joints:
- removed joint l_hand_joint
- removed joint r_hand_joint

File: software/models/mit_gazebo_models/mit_robot_drake/xacro/atlas.urdf.xacro (robot description, xacro)
@@ -1,5 +1,5 @@
 <robot name="atlas" >
   <include filename="$(find mit_drcsim_scripts)/models/mit_robot_drake/xacro/atlas_skeleton_minimal_contact.urdf" />
-  <include filename="$(find mit_drcsim_scripts)/models/mit_robot_drake/xacro/atlas_point_mass_hands.urdf" />
+<!--  <include filename="$(find mit_drcsim_scripts)/models/mit_robot_drake/xacro/point_mass_hands.urdf" />-->
   <include filename="$(find mit_drcsim_scripts)/models/mit_robot_drake/xacro/atlas.transmission" />
   <include filename="$(find mit_drcsim_scripts)/models/mit_robot_drake/xacro/multisense_sl_no_contact.urdf" />

File: software/models/mit_gazebo_models/mit_robot_drake/xacro/atlas_skeleton_minimal_contact.urdf (robot description, URDF)
Before this commit: robot drc_skeleton, 28 links, 28 joints
Links:
- link l_clav: geometry visual mesh filename=package://mit_robot/meshes/l_clav.wrl scale=1 1 1
- link l_farm: geometry visual mesh filename=package://mit_robot/meshes/l_farm.wrl scale=1 1 1
- link l_foot: geometry collision sphere radius=0; collision sphere radius=0
- link l_hand: geometry collision sphere radius=0; visual mesh filename=package://mit_robot/meshes/l_hand.wrl scale=1 1 1
- link l_larm: geometry visual mesh filename=package://mit_robot/meshes/l_larm.wrl scale=1 1 1
- link l_lglut: geometry visual mesh filename=package://mit_robot/meshes/l_lglut.wrl scale=1 1 1
- link l_lleg: geometry collision sphere radius=0; collision sphere radius=0
- link l_scap: geometry visual mesh filename=package://mit_robot/meshes/l_scap.wrl scale=1 1 1
- link l_talus: geometry visual mesh filename=package://mit_robot/meshes/l_talus.wrl scale=1 1 1
- link l_uarm: geometry visual mesh filename=package://mit_robot/meshes/l_uarm.wrl scale=1 1 1
- link l_uglut: geometry visual mesh filename=package://mit_robot/meshes/l_uglut.wrl scale=1 1 1
- link l_uleg: geometry visual mesh filename=package://mit_robot/meshes/l_uleg.wrl scale=1 1 1
- link ltorso: geometry visual mesh filename=package://mit_robot/meshes/ltorso.wrl scale=1 1 1
- link mtorso: geometry visual mesh filename=package://mit_robot/meshes/mtorso.wrl scale=1 1 1
- link pelvis: geometry visual mesh filename=package://mit_robot/meshes/pelvis.wrl scale=1 1 1
- link r_clav: geometry visual mesh filename=package://mit_robot/meshes/r_clav.wrl scale=1 1 1
- link r_farm: geometry visual mesh filename=package://mit_robot/meshes/r_farm.wrl scale=1 1 1
- link r_foot: geometry collision sphere radius=0; collision sphere radius=0
- link r_hand: geometry collision sphere radius=0; visual mesh filename=package://mit_robot/meshes/r_hand.wrl scale=1 1 1
- link r_larm: geometry visual mesh filename=package://mit_robot/meshes/r_larm.wrl scale=1 1 1
- link r_lglut: geometry visual mesh filename=package://mit_robot/meshes/r_lglut.wrl scale=1 1 1
- link r_lleg: geometry collision sphere radius=0; collision sphere radius=0
- link r_scap: geometry visual mesh filename=package://mit_robot/meshes/r_scap.wrl scale=1 1 1
- link r_talus: geometry visual mesh filename=package://mit_robot/meshes/r_talus.wrl scale=1 1 1
- link r_uarm: geometry visual mesh filename=package://mit_robot/meshes/r_uarm.wrl scale=1 1 1
- link r_uglut: geometry visual mesh filename=package://mit_robot/meshes/r_uglut.wrl scale=1 1 1
- link r_uleg: geometry visual mesh filename=package://mit_robot/meshes/r_uleg.wrl scale=1 1 1
- link utorso: geometry visual mesh filename=package://mit_robot/meshes/utorso.wrl scale=1 1 1

File: software/models/mit_gazebo_models/mit_robot_drake/xacro/multisense_sl_no_contact.urdf (robot description, URDF)
Before this commit: robot multisense_sl, 1 links, 0 joints
Links:
- link head: geometry visual mesh filename=package://multisense_sl/meshes/base_link.wrl

Commit message: uses mit_drcsim_scripts for package path
git-svn-id: https://svn.csail.mit.edu/drc@1842 c7283977-0100-402a-a91a-fa70b306dbfe

File: software/models/mit_gazebo_models/mit_robot_drake/model_minimal_contact.urdf (robot description, URDF)
Before this commit: robot atlas, 29 links, 28 joints
Links:
- link head: geometry visual mesh filename=package://mit_drcsim_scripts/models/multisense_sl/meshes/ba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
- link l_clav: geometry visual mesh filename=package://mit_drcsim_scripts/models/mit_robot/meshes/l_clav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 scale=1 1 1
- link l_farm: geometry visual mesh filename=package://mit_drcsim_scripts/models/mit_robot/meshes/l_farm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 scale=1 1 1
- link l_foot: geometry collision sphere radius=0; collision sphere radius=0
- link l_hand: geometry collision sphere radius=0; visual mesh filename=package://mit_drcsim_scripts/models/mit_robot/meshes/l_hand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 scale=1 1 1
- link l_larm: geometry visual mesh filename=package://mit_drcsim_scripts/models/mit_robot/meshes/l_larm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 scale=1 1 1
- link l_lglut: geometry visual mesh filename=package://mit_drcsim_scripts/models/mit_robot/meshes/l_lglu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 scale=1 1 1
- link l_lleg: geometry collision sphere radius=0; collision sphere radius=0
- link l_scap: geometry visual mesh filename=package://mit_drcsim_scripts/models/mit_robot/meshes/l_scap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 scale=1 1 1
- link l_talus: geometry visual mesh filename=package://mit_drcsim_scripts/models/mit_robot/meshes/l_talu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 scale=1 1 1
- link l_uarm: geometry visual mesh filename=package://mit_drcsim_scripts/models/mit_robot/meshes/l_uarm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 scale=1 1 1
- link l_uglut: geometry visual mesh filename=package://mit_drcsim_scripts/models/mit_robot/meshes/l_uglu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 scale=1 1 1
- link l_uleg: geometry visual mesh filename=package://mit_drcsim_scripts/models/mit_robot/meshes/l_uleg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 scale=1 1 1
- link ltorso: geometry visual mesh filename=package://mit_drcsim_scripts/models/mit_robot/meshes/ltorso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 scale=1 1 1
- link mtorso: geometry visual mesh filename=package://mit_drcsim_scripts/models/mit_robot/meshes/mtorso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 scale=1 1 1
- link pelvis: geometry visual mesh filename=package://mit_drcsim_scripts/models/mit_robot/meshes/pelvis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 scale=1 1 1
- link r_clav: geometry visual mesh filename=package://mit_drcsim_scripts/models/mit_robot/meshes/r_clav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 scale=1 1 1
- link r_farm: geometry visual mesh filename=package://mit_drcsim_scripts/models/mit_robot/meshes/r_farm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 scale=1 1 1
- link r_foot: geometry collision sphere radius=0; collision sphere radius=0
- link r_hand: geometry collision sphere radius=0; visual mesh filename=package://mit_drcsim_scripts/models/mit_robot/meshes/r_hand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 scale=1 1 1
- link r_larm: geometry visual mesh filename=package://mit_drcsim_scripts/models/mit_robot/meshes/r_larm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 scale=1 1 1
- link r_lglut: geometry visual mesh filename=package://mit_drcsim_scripts/models/mit_robot/meshes/r_lglu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 scale=1 1 1
- link r_lleg: geometry collision sphere radius=0; collision sphere radius=0
- link r_scap: geometry visual mesh filename=package://mit_drcsim_scripts/models/mit_robot/meshes/r_scap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 scale=1 1 1
- link r_talus: geometry visual mesh filename=package://mit_drcsim_scripts/models/mit_robot/meshes/r_talu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 scale=1 1 1
- link r_uarm: geometry visual mesh filename=package://mit_drcsim_scripts/models/mit_robot/meshes/r_uarm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 scale=1 1 1
- link r_uglut: geometry visual mesh filename=package://mit_drcsim_scripts/models/mit_robot/meshes/r_uglu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 scale=1 1 1
- link r_uleg: geometry visual mesh filename=package://mit_drcsim_scripts/models/mit_robot/meshes/r_uleg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 scale=1 1 1
- link utorso: geometry visual mesh filename=package://mit_drcsim_scripts/models/mit_robot/meshes/utorso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 scale=1 1 1

File: software/models/mit_gazebo_models/mit_robot_drake/xacro/atlas_skeleton_minimal_contact.urdf (robot description, URDF)
Before this commit: robot drc_skeleton, 28 links, 28 joints
Links:
- link l_clav: geometry visual mesh filename=package://mit_drcsim_scripts/models/mit_robot/meshes/l_clav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 scale=1 1 1
- link l_farm: geometry visual mesh filename=package://mit_drcsim_scripts/models/mit_robot/meshes/l_farm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 scale=1 1 1
- link l_foot: geometry collision sphere radius=0; collision sphere radius=0
- link l_hand: geometry collision sphere radius=0; visual mesh filename=package://mit_drcsim_scripts/models/mit_robot/meshes/l_hand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 scale=1 1 1
- link l_larm: geometry visual mesh filename=package://mit_drcsim_scripts/models/mit_robot/meshes/l_larm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 scale=1 1 1
- link l_lglut: geometry visual mesh filename=package://mit_drcsim_scripts/models/mit_robot/meshes/l_lglu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 scale=1 1 1
- link l_lleg: geometry collision sphere radius=0; collision sphere radius=0
- link l_scap: geometry visual mesh filename=package://mit_drcsim_scripts/models/mit_robot/meshes/l_scap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 scale=1 1 1
- link l_talus: geometry visual mesh filename=package://mit_drcsim_scripts/models/mit_robot/meshes/l_talu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 scale=1 1 1
- link l_uarm: geometry visual mesh filename=package://mit_drcsim_scripts/models/mit_robot/meshes/l_uarm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 scale=1 1 1
- link l_uglut: geometry visual mesh filename=package://mit_drcsim_scripts/models/mit_robot/meshes/l_uglu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 scale=1 1 1
- link l_uleg: geometry visual mesh filename=package://mit_drcsim_scripts/models/mit_robot/meshes/l_uleg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 scale=1 1 1
- link ltorso: geometry visual mesh filename=package://mit_drcsim_scripts/models/mit_robot/meshes/ltorso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 scale=1 1 1
- link mtorso: geometry visual mesh filename=package://mit_drcsim_scripts/models/mit_robot/meshes/mtorso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 scale=1 1 1
- link pelvis: geometry visual mesh filename=package://mit_drcsim_scripts/models/mit_robot/meshes/pelvis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 scale=1 1 1
- link r_clav: geometry visual mesh filename=package://mit_drcsim_scripts/models/mit_robot/meshes/r_clav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 scale=1 1 1
- link r_farm: geometry visual mesh filename=package://mit_drcsim_scripts/models/mit_robot/meshes/r_farm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 scale=1 1 1
- link r_foot: geometry collision sphere radius=0; collision sphere radius=0
- link r_hand: geometry collision sphere radius=0; visual mesh filename=package://mit_drcsim_scripts/models/mit_robot/meshes/r_hand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 scale=1 1 1
- link r_larm: geometry visual mesh filename=package://mit_drcsim_scripts/models/mit_robot/meshes/r_larm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 scale=1 1 1
- link r_lglut: geometry visual mesh filename=package://mit_drcsim_scripts/models/mit_robot/meshes/r_lglu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 scale=1 1 1
- link r_lleg: geometry collision sphere radius=0; collision sphere radius=0
- link r_scap: geometry visual mesh filename=package://mit_drcsim_scripts/models/mit_robot/meshes/r_scap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 scale=1 1 1
- link r_talus: geometry visual mesh filename=package://mit_drcsim_scripts/models/mit_robot/meshes/r_talu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 scale=1 1 1
- link r_uarm: geometry visual mesh filename=package://mit_drcsim_scripts/models/mit_robot/meshes/r_uarm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 scale=1 1 1
- link r_uglut: geometry visual mesh filename=package://mit_drcsim_scripts/models/mit_robot/meshes/r_uglu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 scale=1 1 1
- link r_uleg: geometry visual mesh filename=package://mit_drcsim_scripts/models/mit_robot/meshes/r_uleg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 scale=1 1 1
- link utorso: geometry visual mesh filename=package://mit_drcsim_scripts/models/mit_robot/meshes/utorso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 scale=1 1 1

File: software/models/mit_gazebo_models/mit_robot_drake/xacro/multisense_sl_no_contact.urdf (robot description, URDF)
Before this commit: robot multisense_sl, 1 links, 0 joints
Links:
- link head: geometry visual mesh filename=package://mit_drcsim_scripts/models/multisense_sl/meshes/ba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

Commit message: knee now has only 1 contact point
git-svn-id: https://svn.csail.mit.edu/drc@1847 c7283977-0100-402a-a91a-fa70b306dbfe

File: software/models/mit_gazebo_models/mit_robot_drake/model_minimal_contact.urdf (robot description, URDF)
Before this commit: robot atlas, 29 links, 28 joints
Links:
- link l_lleg: geometry collision sphere radius=0; visual mesh filename=package://mit_drcsim_scripts/models/mit_robot/meshes/l_lleg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 scale=1 1 1
- link r_lleg: geometry collision sphere radius=0; visual mesh filename=package://mit_drcsim_scripts/models/mit_robot/meshes/r_lleg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 scale=1 1 1

File: software/models/mit_gazebo_models/mit_robot_drake/xacro/atlas_skeleton_minimal_contact.urdf (robot description, URDF)
Before this commit: robot drc_skeleton, 28 links, 28 joints
Links:
- link l_lleg: geometry collision sphere radius=0; visual mesh filename=package://mit_drcsim_scripts/models/mit_robot/meshes/l_lleg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 scale=1 1 1
- link r_lleg: geometry collision sphere radius=0; visual mesh filename=package://mit_drcsim_scripts/models/mit_robot/meshes/r_lleg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 scale=1 1 1

Commit message: switching package names back
git-svn-id: https://svn.csail.mit.edu/drc@1870 c7283977-0100-402a-a91a-fa70b306dbfe

File: software/models/mit_gazebo_models/mit_robot_drake/model_minimal_contact.urdf (robot description, URDF)
Before this commit: robot atlas, 29 links, 28 joints
Links:
- link head: geometry visual mesh filename=package://multisense_sl/meshes/base_link.wrl
- link l_clav: geometry visual mesh filename=package://mit_robot/meshes/l_clav.wrl scale=1 1 1
- link l_farm: geometry visual mesh filename=package://mit_robot/meshes/l_farm.wrl scale=1 1 1
- link l_foot: geometry collision sphere radius=0; collision sphere radius=0
- link l_hand: geometry collision sphere radius=0; visual mesh filename=package://mit_robot/meshes/l_hand.wrl scale=1 1 1
- link l_larm: geometry visual mesh filename=package://mit_robot/meshes/l_larm.wrl scale=1 1 1
- link l_lglut: geometry visual mesh filename=package://mit_robot/meshes/l_lglut.wrl scale=1 1 1
- link l_lleg: geometry collision sphere radius=0; visual mesh filename=package://mit_robot/meshes/l_lleg.wrl scale=1 1 1
- link l_scap: geometry visual mesh filename=package://mit_robot/meshes/l_scap.wrl scale=1 1 1
- link l_talus: geometry visual mesh filename=package://mit_robot/meshes/l_talus.wrl scale=1 1 1
- link l_uarm: geometry visual mesh filename=package://mit_robot/meshes/l_uarm.wrl scale=1 1 1
- link l_uglut: geometry visual mesh filename=package://mit_robot/meshes/l_uglut.wrl scale=1 1 1
- link l_uleg: geometry visual mesh filename=package://mit_robot/meshes/l_uleg.wrl scale=1 1 1
- link ltorso: geometry visual mesh filename=package://mit_robot/meshes/ltorso.wrl scale=1 1 1
- link mtorso: geometry visual mesh filename=package://mit_robot/meshes/mtorso.wrl scale=1 1 1
- link pelvis: geometry visual mesh filename=package://mit_robot/meshes/pelvis.wrl scale=1 1 1
- link r_clav: geometry visual mesh filename=package://mit_robot/meshes/r_clav.wrl scale=1 1 1
- link r_farm: geometry visual mesh filename=package://mit_robot/meshes/r_farm.wrl scale=1 1 1
- link r_foot: geometry collision sphere radius=0; collision sphere radius=0
- link r_hand: geometry collision sphere radius=0; visual mesh filename=package://mit_robot/meshes/r_hand.wrl scale=1 1 1
- link r_larm: geometry visual mesh filename=package://mit_robot/meshes/r_larm.wrl scale=1 1 1
- link r_lglut: geometry visual mesh filename=package://mit_robot/meshes/r_lglut.wrl scale=1 1 1
- link r_lleg: geometry collision sphere radius=0; visual mesh filename=package://mit_robot/meshes/r_lleg.wrl scale=1 1 1
- link r_scap: geometry visual mesh filename=package://mit_robot/meshes/r_scap.wrl scale=1 1 1
- link r_talus: geometry visual mesh filename=package://mit_robot/meshes/r_talus.wrl scale=1 1 1
- link r_uarm: geometry visual mesh filename=package://mit_robot/meshes/r_uarm.wrl scale=1 1 1
- link r_uglut: geometry visual mesh filename=package://mit_robot/meshes/r_uglut.wrl scale=1 1 1
- link r_uleg: geometry visual mesh filename=package://mit_robot/meshes/r_uleg.wrl scale=1 1 1
- link utorso: geometry visual mesh filename=package://mit_robot/meshes/utorso.wrl scale=1 1 1

File: software/models/mit_gazebo_models/mit_robot_drake/xacro/atlas_skeleton_minimal_contact.urdf (robot description, URDF)
Before this commit: robot drc_skeleton, 28 links, 28 joints
Links:
- link l_clav: geometry visual mesh filename=package://mit_robot/meshes/l_clav.wrl scale=1 1 1
- link l_farm: geometry visual mesh filename=package://mit_robot/meshes/l_farm.wrl scale=1 1 1
- link l_foot: geometry collision sphere radius=0; collision sphere radius=0
- link l_hand: geometry collision sphere radius=0; visual mesh filename=package://mit_robot/meshes/l_hand.wrl scale=1 1 1
- link l_larm: geometry visual mesh filename=package://mit_robot/meshes/l_larm.wrl scale=1 1 1
- link l_lglut: geometry visual mesh filename=package://mit_robot/meshes/l_lglut.wrl scale=1 1 1
- link l_lleg: geometry collision sphere radius=0; visual mesh filename=package://mit_robot/meshes/l_lleg.wrl scale=1 1 1
- link l_scap: geometry visual mesh filename=package://mit_robot/meshes/l_scap.wrl scale=1 1 1
- link l_talus: geometry visual mesh filename=package://mit_robot/meshes/l_talus.wrl scale=1 1 1
- link l_uarm: geometry visual mesh filename=package://mit_robot/meshes/l_uarm.wrl scale=1 1 1
- link l_uglut: geometry visual mesh filename=package://mit_robot/meshes/l_uglut.wrl scale=1 1 1
- link l_uleg: geometry visual mesh filename=package://mit_robot/meshes/l_uleg.wrl scale=1 1 1
- link ltorso: geometry visual mesh filename=package://mit_robot/meshes/ltorso.wrl scale=1 1 1
- link mtorso: geometry visual mesh filename=package://mit_robot/meshes/mtorso.wrl scale=1 1 1
- link pelvis: geometry visual mesh filename=package://mit_robot/meshes/pelvis.wrl scale=1 1 1
- link r_clav: geometry visual mesh filename=package://mit_robot/meshes/r_clav.wrl scale=1 1 1
- link r_farm: geometry visual mesh filename=package://mit_robot/meshes/r_farm.wrl scale=1 1 1
- link r_foot: geometry collision sphere radius=0; collision sphere radius=0
- link r_hand: geometry collision sphere radius=0; visual mesh filename=package://mit_robot/meshes/r_hand.wrl scale=1 1 1
- link r_larm: geometry visual mesh filename=package://mit_robot/meshes/r_larm.wrl scale=1 1 1
- link r_lglut: geometry visual mesh filename=package://mit_robot/meshes/r_lglut.wrl scale=1 1 1
- link r_lleg: geometry collision sphere radius=0; visual mesh filename=package://mit_robot/meshes/r_lleg.wrl scale=1 1 1
- link r_scap: geometry visual mesh filename=package://mit_robot/meshes/r_scap.wrl scale=1 1 1
- link r_talus: geometry visual mesh filename=package://mit_robot/meshes/r_talus.wrl scale=1 1 1
- link r_uarm: geometry visual mesh filename=package://mit_robot/meshes/r_uarm.wrl scale=1 1 1
- link r_uglut: geometry visual mesh filename=package://mit_robot/meshes/r_uglut.wrl scale=1 1 1
- link r_uleg: geometry visual mesh filename=package://mit_robot/meshes/r_uleg.wrl scale=1 1 1
- link utorso: geometry visual mesh filename=package://mit_robot/meshes/utorso.wrl scale=1 1 1

File: software/models/mit_gazebo_models/mit_robot_drake/xacro/multisense_sl_no_contact.urdf (robot description, URDF)
Before this commit: robot multisense_sl, 1 links, 0 joints
Links:
- link head: geometry visual mesh filename=package://multisense_sl/meshes/base_link.wrl
