Commit message: reverting
git-svn-id: https://svn.csail.mit.edu/drc@1871 c7283977-0100-402a-a91a-fa70b306dbfe

File: software/models/mit_gazebo_models/mit_robot_drake/model_minimal_contact.urdf (robot description, URDF)
Before this commit: robot atlas, 29 links, 28 joints
Links:
- link head: geometry visual mesh filename=package://mit_drcsim_scripts/models/multisense_sl/meshes/ba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
- link l_clav: geometry visual mesh filename=package://mit_drcsim_scripts/models/mit_robot/meshes/l_clav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 scale=1 1 1
- link l_farm: geometry visual mesh filename=package://mit_drcsim_scripts/models/mit_robot/meshes/l_farm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 scale=1 1 1
- link l_foot: geometry collision sphere radius=0; collision sphere radius=0
- link l_hand: geometry collision sphere radius=0; visual mesh filename=package://mit_drcsim_scripts/models/mit_robot/meshes/l_hand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 scale=1 1 1
- link l_larm: geometry visual mesh filename=package://mit_drcsim_scripts/models/mit_robot/meshes/l_larm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 scale=1 1 1
- link l_lglut: geometry visual mesh filename=package://mit_drcsim_scripts/models/mit_robot/meshes/l_lglu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 scale=1 1 1
- link l_lleg: geometry collision sphere radius=0; visual mesh filename=package://mit_drcsim_scripts/models/mit_robot/meshes/l_lleg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 scale=1 1 1
- link l_scap: geometry visual mesh filename=package://mit_drcsim_scripts/models/mit_robot/meshes/l_scap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 scale=1 1 1
- link l_talus: geometry visual mesh filename=package://mit_drcsim_scripts/models/mit_robot/meshes/l_talu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 scale=1 1 1
- link l_uarm: geometry visual mesh filename=package://mit_drcsim_scripts/models/mit_robot/meshes/l_uarm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 scale=1 1 1
- link l_uglut: geometry visual mesh filename=package://mit_drcsim_scripts/models/mit_robot/meshes/l_uglu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 scale=1 1 1
- link l_uleg: geometry visual mesh filename=package://mit_drcsim_scripts/models/mit_robot/meshes/l_uleg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 scale=1 1 1
- link ltorso: geometry visual mesh filename=package://mit_drcsim_scripts/models/mit_robot/meshes/ltorso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 scale=1 1 1
- link mtorso: geometry visual mesh filename=package://mit_drcsim_scripts/models/mit_robot/meshes/mtorso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 scale=1 1 1
- link pelvis: geometry visual mesh filename=package://mit_drcsim_scripts/models/mit_robot/meshes/pelvis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 scale=1 1 1
- link r_clav: geometry visual mesh filename=package://mit_drcsim_scripts/models/mit_robot/meshes/r_clav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 scale=1 1 1
- link r_farm: geometry visual mesh filename=package://mit_drcsim_scripts/models/mit_robot/meshes/r_farm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 scale=1 1 1
- link r_foot: geometry collision sphere radius=0; collision sphere radius=0
- link r_hand: geometry collision sphere radius=0; visual mesh filename=package://mit_drcsim_scripts/models/mit_robot/meshes/r_hand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 scale=1 1 1
- link r_larm: geometry visual mesh filename=package://mit_drcsim_scripts/models/mit_robot/meshes/r_larm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 scale=1 1 1
- link r_lglut: geometry visual mesh filename=package://mit_drcsim_scripts/models/mit_robot/meshes/r_lglu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 scale=1 1 1
- link r_lleg: geometry collision sphere radius=0; visual mesh filename=package://mit_drcsim_scripts/models/mit_robot/meshes/r_lleg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 scale=1 1 1
- link r_scap: geometry visual mesh filename=package://mit_drcsim_scripts/models/mit_robot/meshes/r_scap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 scale=1 1 1
- link r_talus: geometry visual mesh filename=package://mit_drcsim_scripts/models/mit_robot/meshes/r_talu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 scale=1 1 1
- link r_uarm: geometry visual mesh filename=package://mit_drcsim_scripts/models/mit_robot/meshes/r_uarm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 scale=1 1 1
- link r_uglut: geometry visual mesh filename=package://mit_drcsim_scripts/models/mit_robot/meshes/r_uglu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 scale=1 1 1
- link r_uleg: geometry visual mesh filename=package://mit_drcsim_scripts/models/mit_robot/meshes/r_uleg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 scale=1 1 1
- link utorso: geometry visual mesh filename=package://mit_drcsim_scripts/models/mit_robot/meshes/utorso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 scale=1 1 1

File: software/models/mit_gazebo_models/mit_robot_drake/xacro/atlas_skeleton_minimal_contact.urdf (robot description, URDF)
Before this commit: robot drc_skeleton, 28 links, 28 joints
Links:
- link l_clav: geometry visual mesh filename=package://mit_drcsim_scripts/models/mit_robot/meshes/l_clav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 scale=1 1 1
- link l_farm: geometry visual mesh filename=package://mit_drcsim_scripts/models/mit_robot/meshes/l_farm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 scale=1 1 1
- link l_foot: geometry collision sphere radius=0; collision sphere radius=0
- link l_hand: geometry collision sphere radius=0; visual mesh filename=package://mit_drcsim_scripts/models/mit_robot/meshes/l_hand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 scale=1 1 1
- link l_larm: geometry visual mesh filename=package://mit_drcsim_scripts/models/mit_robot/meshes/l_larm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 scale=1 1 1
- link l_lglut: geometry visual mesh filename=package://mit_drcsim_scripts/models/mit_robot/meshes/l_lglu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 scale=1 1 1
- link l_lleg: geometry collision sphere radius=0; visual mesh filename=package://mit_drcsim_scripts/models/mit_robot/meshes/l_lleg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 scale=1 1 1
- link l_scap: geometry visual mesh filename=package://mit_drcsim_scripts/models/mit_robot/meshes/l_scap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 scale=1 1 1
- link l_talus: geometry visual mesh filename=package://mit_drcsim_scripts/models/mit_robot/meshes/l_talu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 scale=1 1 1
- link l_uarm: geometry visual mesh filename=package://mit_drcsim_scripts/models/mit_robot/meshes/l_uarm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 scale=1 1 1
- link l_uglut: geometry visual mesh filename=package://mit_drcsim_scripts/models/mit_robot/meshes/l_uglu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 scale=1 1 1
- link l_uleg: geometry visual mesh filename=package://mit_drcsim_scripts/models/mit_robot/meshes/l_uleg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 scale=1 1 1
- link ltorso: geometry visual mesh filename=package://mit_drcsim_scripts/models/mit_robot/meshes/ltorso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 scale=1 1 1
- link mtorso: geometry visual mesh filename=package://mit_drcsim_scripts/models/mit_robot/meshes/mtorso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 scale=1 1 1
- link pelvis: geometry visual mesh filename=package://mit_drcsim_scripts/models/mit_robot/meshes/pelvis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 scale=1 1 1
- link r_clav: geometry visual mesh filename=package://mit_drcsim_scripts/models/mit_robot/meshes/r_clav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 scale=1 1 1
- link r_farm: geometry visual mesh filename=package://mit_drcsim_scripts/models/mit_robot/meshes/r_farm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 scale=1 1 1
- link r_foot: geometry collision sphere radius=0; collision sphere radius=0
- link r_hand: geometry collision sphere radius=0; visual mesh filename=package://mit_drcsim_scripts/models/mit_robot/meshes/r_hand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 scale=1 1 1
- link r_larm: geometry visual mesh filename=package://mit_drcsim_scripts/models/mit_robot/meshes/r_larm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 scale=1 1 1
- link r_lglut: geometry visual mesh filename=package://mit_drcsim_scripts/models/mit_robot/meshes/r_lglu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 scale=1 1 1
- link r_lleg: geometry collision sphere radius=0; visual mesh filename=package://mit_drcsim_scripts/models/mit_robot/meshes/r_lleg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 scale=1 1 1
- link r_scap: geometry visual mesh filename=package://mit_drcsim_scripts/models/mit_robot/meshes/r_scap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 scale=1 1 1
- link r_talus: geometry visual mesh filename=package://mit_drcsim_scripts/models/mit_robot/meshes/r_talu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 scale=1 1 1
- link r_uarm: geometry visual mesh filename=package://mit_drcsim_scripts/models/mit_robot/meshes/r_uarm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 scale=1 1 1
- link r_uglut: geometry visual mesh filename=package://mit_drcsim_scripts/models/mit_robot/meshes/r_uglu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 scale=1 1 1
- link r_uleg: geometry visual mesh filename=package://mit_drcsim_scripts/models/mit_robot/meshes/r_uleg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 scale=1 1 1
- link utorso: geometry visual mesh filename=package://mit_drcsim_scripts/models/mit_robot/meshes/utorso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 scale=1 1 1

Commit message: and the corresponding updated model files
git-svn-id: https://svn.csail.mit.edu/drc@3411 c7283977-0100-402a-a91a-fa70b306dbfe

File: software/models/mit_gazebo_models/mit_robot_drake/model_minimal_contact.urdf (robot description, URDF)
Before this commit: robot atlas, 29 links, 28 joints
Links:
- link head: mass 1.4199 -> 1.477574
- link pelvis: mass 12.54638 -> 12.64638

File: software/models/mit_gazebo_models/mit_robot_drake/model_minimal_contact_point_hands.urdf (robot description, URDF)
Before this commit: robot atlas, 31 links, 30 joints
Links:
- link l_hand_point_mass: mass 2.312 -> 3.111
- link r_hand_point_mass: mass 2.312 -> 3.111

File: software/models/mit_gazebo_models/mit_robot_drake/model_minimal_contact_with_hands.urdf (robot description, URDF)
Before this commit: robot atlas, 101 links, 100 joints
Links:
- link head: mass 1.4199 -> 1.477574
- link pelvis: mass 12.54638 -> 12.64638

Commit message: updated mesh scalings in drake model
git-svn-id: https://svn.csail.mit.edu/drc@3764 c7283977-0100-402a-a91a-fa70b306dbfe

File: software/models/mit_gazebo_models/mit_robot_drake/model_minimal_contact.urdf (robot description, URDF)
Before this commit: robot atlas, 29 links, 28 joints
Links:
- link l_uleg: geometry visual mesh filename=package://mit_drcsim_scripts/models/mit_robot/meshes/l_uleg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 scale=1. 1. 1.
- link pelvis: geometry visual mesh filename=package://mit_drcsim_scripts/models/mit_robot/meshes/pelvis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 scale=1. 1. 1.
- link r_larm: geometry visual mesh filename=package://mit_drcsim_scripts/models/mit_robot/meshes/r_larm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 scale=1. 1. 1.
- link r_lglut: geometry visual mesh filename=package://mit_drcsim_scripts/models/mit_robot/meshes/r_lglu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 scale=1. 1. 1.
- link r_lleg: geometry collision sphere radius=0; visual mesh filename=package://mit_drcsim_scripts/models/mit_robot/meshes/r_lleg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 scale=1. 1. 1.
- link r_uarm: geometry visual mesh filename=package://mit_drcsim_scripts/models/mit_robot/meshes/r_uarm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 scale=1. 1. 1.
- link r_uglut: geometry visual mesh filename=package://mit_drcsim_scripts/models/mit_robot/meshes/r_uglu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 scale=1. 1. 1.
- link r_uleg: geometry visual mesh filename=package://mit_drcsim_scripts/models/mit_robot/meshes/r_uleg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 scale=1. 1. 1.

File: software/models/mit_gazebo_models/mit_robot_drake/model_minimal_contact_point_hands.urdf (robot description, URDF)
Before this commit: robot atlas, 31 links, 30 joints
Links:
- link l_uleg: geometry visual mesh filename=package://mit_drcsim_scripts/models/mit_robot/meshes/l_uleg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 scale=1. 1. 1.
- link pelvis: geometry visual mesh filename=package://mit_drcsim_scripts/models/mit_robot/meshes/pelvis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 scale=1. 1. 1.
- link r_larm: geometry visual mesh filename=package://mit_drcsim_scripts/models/mit_robot/meshes/r_larm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 scale=1. 1. 1.
- link r_lglut: geometry visual mesh filename=package://mit_drcsim_scripts/models/mit_robot/meshes/r_lglu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 scale=1. 1. 1.
- link r_lleg: geometry collision sphere radius=0; visual mesh filename=package://mit_drcsim_scripts/models/mit_robot/meshes/r_lleg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 scale=1. 1. 1.
- link r_uarm: geometry visual mesh filename=package://mit_drcsim_scripts/models/mit_robot/meshes/r_uarm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 scale=1. 1. 1.
- link r_uglut: geometry visual mesh filename=package://mit_drcsim_scripts/models/mit_robot/meshes/r_uglu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 scale=1. 1. 1.
- link r_uleg: geometry visual mesh filename=package://mit_drcsim_scripts/models/mit_robot/meshes/r_uleg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 scale=1. 1. 1.

File: software/models/mit_gazebo_models/mit_robot_drake/xacro/atlas_skeleton_minimal_contact.urdf (robot description, URDF)
Before this commit: robot drc_skeleton, 28 links, 28 joints
Links:
- link l_uleg: geometry visual mesh filename=package://mit_drcsim_scripts/models/mit_robot/meshes/l_uleg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 scale=1. 1. 1.
- link pelvis: geometry visual mesh filename=package://mit_drcsim_scripts/models/mit_robot/meshes/pelvis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 scale=1. 1. 1.
- link r_larm: geometry visual mesh filename=package://mit_drcsim_scripts/models/mit_robot/meshes/r_larm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 scale=1. 1. 1.
- link r_lglut: geometry visual mesh filename=package://mit_drcsim_scripts/models/mit_robot/meshes/r_lglu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 scale=1. 1. 1.
- link r_lleg: geometry collision sphere radius=0; visual mesh filename=package://mit_drcsim_scripts/models/mit_robot/meshes/r_lleg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 scale=1. 1. 1.
- link r_uarm: geometry visual mesh filename=package://mit_drcsim_scripts/models/mit_robot/meshes/r_uarm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 scale=1. 1. 1.
- link r_uglut: geometry visual mesh filename=package://mit_drcsim_scripts/models/mit_robot/meshes/r_uglu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 scale=1. 1. 1.
- link r_uleg: geometry visual mesh filename=package://mit_drcsim_scripts/models/mit_robot/meshes/r_uleg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 scale=1. 1. 1.

Commit message: Adds 'butt' contact group to 'pelvis' link. Contact points are at the back corners of the box collision element.
git-svn-id: https://svn.csail.mit.edu/drc@3857 c7283977-0100-402a-a91a-fa70b306dbfe

File: software/models/mit_gazebo_models/mit_robot_drake/model_minimal_contact.urdf (robot description, URDF)
Before this commit: robot atlas, 29 links, 28 joints
Links:
- link pelvis: geometry collision sphere radius=0; collision sphere radius=0

File: software/models/mit_gazebo_models/mit_robot_drake/model_minimal_contact_point_hands.urdf (robot description, URDF)
Before this commit: robot atlas, 31 links, 30 joints
Links:
- link pelvis: geometry collision sphere radius=0; collision sphere radius=0

File: software/models/mit_gazebo_models/mit_robot_drake/model_minimal_contact_with_hands.urdf (robot description, URDF)
Before this commit: robot atlas, 101 links, 100 joints
Links:
- link pelvis: geometry collision sphere radius=0; collision sphere radius=0

File: software/models/mit_gazebo_models/mit_robot_drake/xacro/atlas_skeleton_minimal_contact.urdf (robot description, URDF)
Before this commit: robot drc_skeleton, 28 links, 28 joints
Links:
- link pelvis: geometry collision sphere radius=0; collision sphere radius=0

Commit message: Adds additional contact points to atlas_skeleton_minimal_contact
git-svn-id: https://svn.csail.mit.edu/drc@3907 c7283977-0100-402a-a91a-fa70b306dbfe

File: software/models/mit_gazebo_models/mit_robot_drake/model_minimal_contact.urdf (robot description, URDF)
Before this commit: robot atlas, 29 links, 28 joints
Links:
- link l_foot: geometry collision sphere radius=0; collision sphere radius=0
- link l_hand: geometry collision sphere radius=0; visual mesh filename=package://mit_drcsim_scripts/models/mit_robot/meshes/l_hand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 scale=1 1 1
- link l_lleg: geometry collision sphere radius=0; visual mesh filename=package://mit_drcsim_scripts/models/mit_robot/meshes/l_lleg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 scale=100. 100. 100.
- link l_uleg: geometry collision sphere radius=0; collision sphere radius=0
- link pelvis: geometry collision sphere radius=0; collision sphere radius=0
- link r_foot: geometry collision sphere radius=0; collision sphere radius=0
- link r_hand: geometry collision sphere radius=0; visual mesh filename=package://mit_drcsim_scripts/models/mit_robot/meshes/r_hand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 scale=1 1 1
- link r_lleg: geometry collision sphere radius=0; visual mesh filename=package://mit_drcsim_scripts/models/mit_robot/meshes/r_lleg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 scale=1. 1. 1.
- link r_uleg: geometry collision sphere radius=0; collision sphere radius=0
- link utorso: geometry collision sphere radius=0; collision sphere radius=0

File: software/models/mit_gazebo_models/mit_robot_drake/model_minimal_contact_point_hands.urdf (robot description, URDF)
Before this commit: robot atlas, 31 links, 30 joints
Links:
- link l_foot: geometry collision sphere radius=0; collision sphere radius=0
- link l_hand: geometry collision sphere radius=0; visual mesh filename=package://mit_drcsim_scripts/models/mit_robot/meshes/l_hand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 scale=1 1 1
- link l_lleg: geometry collision sphere radius=0; visual mesh filename=package://mit_drcsim_scripts/models/mit_robot/meshes/l_lleg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 scale=100. 100. 100.
- link l_uleg: geometry collision sphere radius=0; collision sphere radius=0
- link pelvis: geometry collision sphere radius=0; collision sphere radius=0
- link r_foot: geometry collision sphere radius=0; collision sphere radius=0
- link r_hand: geometry collision sphere radius=0; visual mesh filename=package://mit_drcsim_scripts/models/mit_robot/meshes/r_hand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 scale=1 1 1
- link r_lleg: geometry collision sphere radius=0; visual mesh filename=package://mit_drcsim_scripts/models/mit_robot/meshes/r_lleg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 scale=1. 1. 1.
- link r_uleg: geometry collision sphere radius=0; collision sphere radius=0
- link utorso: geometry collision sphere radius=0; collision sphere radius=0

File: software/models/mit_gazebo_models/mit_robot_drake/model_minimal_contact_with_hands.urdf (robot description, URDF)
Before this commit: robot atlas, 101 links, 100 joints
Links:
- link l_foot: geometry collision sphere radius=0; collision sphere radius=0
- link l_hand: geometry collision sphere radius=0; visual mesh filename=package://mit_drcsim_scripts/models/mit_robot/meshes/l_hand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 scale=1 1 1
- link l_lleg: geometry collision sphere radius=0; visual mesh filename=package://mit_drcsim_scripts/models/mit_robot/meshes/l_lleg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 scale=100. 100. 100.
- link l_uleg: geometry collision sphere radius=0; collision sphere radius=0
- link pelvis: geometry collision sphere radius=0; collision sphere radius=0
- link r_foot: geometry collision sphere radius=0; collision sphere radius=0
- link r_hand: geometry collision sphere radius=0; visual mesh filename=package://mit_drcsim_scripts/models/mit_robot/meshes/r_hand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 scale=1 1 1
- link r_lleg: geometry collision sphere radius=0; visual mesh filename=package://mit_drcsim_scripts/models/mit_robot/meshes/r_lleg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 scale=1. 1. 1.
- link r_uleg: geometry collision sphere radius=0; collision sphere radius=0
- link utorso: geometry collision sphere radius=0; collision sphere radius=0

File: software/models/mit_gazebo_models/mit_robot_drake/xacro/atlas_skeleton_minimal_contact.urdf (robot description, URDF)
Before this commit: robot drc_skeleton, 28 links, 28 joints
Links:
- link l_foot: geometry visual mesh filename=package://mit_drcsim_scripts/models/mit_robot/meshes/l_foot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 scale=1 1 1
- link l_hand: geometry visual mesh filename=package://mit_drcsim_scripts/models/mit_robot/meshes/l_hand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 scale=1 1 1
- link l_lleg: geometry visual mesh filename=package://mit_drcsim_scripts/models/mit_robot/meshes/l_lleg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 scale=100. 100. 100.
- link pelvis: geometry visual mesh filename=package://mit_drcsim_scripts/models/mit_robot/meshes/pelvis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 scale=1. 1. 1.
- link r_foot: geometry visual mesh filename=package://mit_drcsim_scripts/models/mit_robot/meshes/r_foot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 scale=1 1 1
- link r_hand: geometry visual mesh filename=package://mit_drcsim_scripts/models/mit_robot/meshes/r_hand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 scale=1 1 1
- link r_lleg: geometry visual mesh filename=package://mit_drcsim_scripts/models/mit_robot/meshes/r_lleg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 scale=1. 1. 1.

File: software/models/mit_gazebo_models/mit_robot_drake/xacro/atlas_skeleton_simple_visuals.urdf (robot description, URDF)
Before this commit: robot drc_skeleton, 28 links, 28 joints
Links:
- link r_uleg: geometry collision cylinder length=0.10 radius=0.1; collision cylinder length=0.15 radius=0.07
- link utorso: geometry collision box size=0.3188 0.24 0.3162; collision cylinder length=0.22375 radius=0.0363

Commit message: Update urdfs to match changes introduced in r4229.
git-svn-id: https://svn.csail.mit.edu/drc@4230 c7283977-0100-402a-a91a-fa70b306dbfe

File: software/models/mit_gazebo_models/mit_robot_drake/model_minimal_contact.urdf (robot description, URDF)
Before this commit: robot atlas, 29 links, 28 joints
Links:
- link pelvis: geometry collision sphere radius=0; collision sphere radius=0

File: software/models/mit_gazebo_models/mit_robot_drake/model_minimal_contact_with_hands.urdf (robot description, URDF)
Before this commit: robot atlas, 101 links, 100 joints
Links:
- link pelvis: geometry collision sphere radius=0; collision sphere radius=0

File: software/models/mit_gazebo_models/mit_robot_drake/model_simple_visuals_point_hands.urdf (robot description, URDF)
Before this commit: robot atlas, 31 links, 30 joints
Links:
- removed link l_hand_point_mass
- removed link r_hand_point_mass
- added link left_palm, mass 0.3; collision box size=0.09 .03 .06; collision box size=0.09 .03 .06
- added link right_palm, mass 0.3; collision box size=0.09 .03 .06; collision box size=0.09 .03 .06
- link head: geometry collision box size=0.0468 0.12 0.1184; collision box size=0.1311 0.12 0.0591
- link l_clav: geometry collision box size=0.13 0.15 0.05; collision cylinder length=0.1525 radius=0.045
- link l_farm: geometry collision box size=0.135 0.1 0.045; collision cylinder length=0.125 radius=0.045
- link l_foot: geometry collision box size=0.26 0.124887 0.05; collision sphere radius=0
- link l_hand: geometry collision box size=0.13 0.09 0.07; collision cylinder length=0.05 radius=0.03
- link l_larm: geometry collision box size=0.135 0.15 0.06; collision cylinder length=0.125 radius=0.045
- link l_lglut: geometry collision cylinder length=0.060306 radius=0.02009687; collision cylinder length=0.12 radius=0.02
- link l_lleg: geometry collision cylinder length=0.40 radius=0.07; collision sphere radius=0
- link l_scap: geometry collision cylinder length=0.125 radius=0.045; visual box size=0.15 0.15 0.06
- link l_talus: geometry collision cylinder length=0.029542 radius=0.010181; visual cylinder length=0.010059 radius=0.010348
- link l_uarm: geometry collision cylinder length=0.125 radius=0.045; visual box size=0.04 0.07 0.13
- link l_uglut: geometry collision cylinder length=0.078396 radius=0.019096; visual cylinder length=0.078396 radius=0.019096
- link l_uleg: geometry collision cylinder length=0.10 radius=0.1; collision cylinder length=0.15 radius=0.07
- link ltorso: geometry 
- link mtorso: geometry collision cylinder length=0.02 radius=0.015; collision cylinder length=0.02 radius=0.015
- link pelvis: mass 12.64638 -> 12.54638; geometry collision box size=0.1 0.15 0.2; collision box size=0.1 0.15 0.2
- link r_clav: geometry collision box size=0.13 0.15 0.05; collision cylinder length=0.1525 radius=0.045
- link r_farm: geometry collision box size=0.135 0.1 0.045; collision cylinder length=0.125 radius=0.045
- link r_foot: geometry collision box size=0.26 0.124887 0.05; collision sphere radius=0
- link r_hand: geometry collision box size=0.13 0.09 0.07; collision cylinder length=0.05 radius=0.03
- link r_larm: geometry collision box size=0.135 0.15 0.06; collision cylinder length=0.125 radius=0.045
- link r_lglut: geometry collision cylinder length=0.060306 radius=0.02009687; collision cylinder length=0.12 radius=0.02
- link r_lleg: geometry collision cylinder length=0.40 radius=0.07; collision sphere radius=0
- link r_scap: geometry collision box size=0.15 0.15 0.06; collision cylinder length=0.125 radius=0.045
- link r_talus: geometry collision cylinder length=0.010059 radius=0.010348; collision cylinder length=0.029542 radius=0.010181
- link r_uarm: geometry collision box size=0.04 0.07 0.13; collision cylinder length=0.125 radius=0.045
- link r_uglut: geometry collision cylinder length=0.078396 radius=0.019096; collision cylinder length=0.080842 radius=0.019841
- link r_uleg: geometry collision cylinder length=0.10 radius=0.1; collision cylinder length=0.15 radius=0.07
- link utorso: geometry collision box size=0.3188 0.24 0.3162; collision cylinder length=0.22375 radius=0.0363
Joints:
- removed joint l_hand_joint
- removed joint r_hand_joint
- added joint left_sandia_hand_joint: type fixed, parent l_hand, child left_palm, origin xyz=0  0.1 0 rpy= 1.57079 0  1.57079
- added joint right_sandia_hand_joint: type fixed, parent r_hand, child right_palm, origin xyz=0 -0.1 0 rpy=-1.57079 0 -1.57079
