Commit message: fixed scaling of mesh in leg link--should have no effect
git-svn-id: https://svn.csail.mit.edu/drc@4256 c7283977-0100-402a-a91a-fa70b306dbfe

File: software/models/mit_gazebo_models/mit_robot_drake/model_minimal_contact.urdf (robot description, URDF)
Before this commit: robot atlas, 29 links, 28 joints
Links:
- link l_lleg: geometry collision sphere radius=0; visual mesh filename=package://mit_drcsim_scripts/models/mit_robot/meshes/l_lleg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 scale=1 1 1

File: software/models/mit_gazebo_models/mit_robot_drake/model_minimal_contact_point_hands.urdf (robot description, URDF)
Before this commit: robot atlas, 31 links, 30 joints
Links:
- link l_lleg: geometry collision sphere radius=0; visual mesh filename=package://mit_drcsim_scripts/models/mit_robot/meshes/l_lleg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 scale=1 1 1

File: software/models/mit_gazebo_models/mit_robot_drake/model_minimal_contact_with_hands.urdf (robot description, URDF)
Before this commit: robot atlas, 101 links, 100 joints
Links:
- link l_lleg: geometry collision sphere radius=0; visual mesh filename=package://mit_drcsim_scripts/models/mit_robot/meshes/l_lleg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 scale=1 1 1

File: software/models/mit_gazebo_models/mit_robot_drake/xacro/atlas_skeleton_minimal_contact.urdf (robot description, URDF)
Before this commit: robot drc_skeleton, 28 links, 28 joints
Links:
- link l_lleg: geometry visual mesh filename=package://mit_drcsim_scripts/models/mit_robot/meshes/l_lleg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 scale=1 1 1

Commit message: adding foot inner contact group. deleting models that are no longer generated by make
git-svn-id: https://svn.csail.mit.edu/drc@4876 c7283977-0100-402a-a91a-fa70b306dbfe

File: software/models/mit_gazebo_models/mit_robot_drake/model_minimal_contact.urdf (robot description, URDF)
Before this commit: robot atlas, 29 links, 28 joints
Links:
- link l_foot: geometry collision sphere radius=0; collision sphere radius=0
- link r_foot: geometry collision sphere radius=0; collision sphere radius=0

File: software/models/mit_gazebo_models/mit_robot_drake/model_minimal_contact_fixedjoint_hands.urdf (robot description, URDF)
Before this commit: robot atlas, 103 links, 102 joints
Links:
- removed link left_f0_2_accel_dummy1
- removed link left_f0_knuckle_dummy_contact
- removed link left_f1_2_accel_dummy1
- removed link left_f1_knuckle_dummy_contact
- removed link left_f2_2_accel_dummy1
- removed link left_f2_knuckle_dummy_contact
- removed link left_f3_2_accel_dummy1
- removed link left_hook
- removed link right_f0_2_accel_dummy1
- removed link right_f0_knuckle_dummy_contact
- removed link right_f1_2_accel_dummy1
- removed link right_f1_knuckle_dummy_contact
- removed link right_f2_2_accel_dummy1
- removed link right_f2_knuckle_dummy_contact
- removed link right_f3_2_accel_dummy1
- removed link right_hook
- added link left_palm_left_camera_frame, mass 0.01; visual box size=0.003 0.010 0.007
- added link left_palm_left_camera_optical_frame
- added link left_palm_right_camera_frame, mass 0.01; visual box size=0.003 0.010 0.007
- added link left_palm_right_camera_optical_frame
- added link right_palm_left_camera_frame, mass 0.01; visual box size=0.003 0.010 0.007
- added link right_palm_left_camera_optical_frame
- added link right_palm_right_camera_frame, mass 0.01; visual box size=0.003 0.010 0.007
- added link right_palm_right_camera_optical_frame
- link l_foot: geometry collision sphere radius=0; collision sphere radius=0
- link left_f0_0: mass 0.05 -> 0.106; geometry collision cylinder length=0.023 radius=0.01; collision cylinder length=0.023 radius=0.015
- link left_f0_1: mass 0.05 -> 0.033; geometry collision cylinder length=0.067 radius=0.01; visual cylinder length=0.067 radius=0.01
- link left_f0_1_accel: mass 0.001 -> 0.01
- link left_f0_2: mass 0.05 -> 0.033; geometry collision cylinder length=0.057 radius=0.009; collision sphere radius=0.009
- link left_f0_2_accel: mass 0.001 -> 0.01; geometry 
- link left_f0_base: mass 0.35 -> 0.250
- link left_f0_fixed_accel: mass 0.001 -> 0.01; geometry 
- link left_f1_0: mass 0.05 -> 0.106; geometry collision cylinder length=0.023 radius=0.01; collision cylinder length=0.023 radius=0.015
- link left_f1_1: mass 0.05 -> 0.033; geometry collision cylinder length=0.067 radius=0.01; visual cylinder length=0.067 radius=0.01
- link left_f1_1_accel: mass 0.001 -> 0.01
- link left_f1_2: mass 0.05 -> 0.033; geometry collision cylinder length=0.057 radius=0.009; collision sphere radius=0.009
- link left_f1_2_accel: mass 0.001 -> 0.01; geometry 
- link left_f1_base: mass 0.35 -> 0.250
- link left_f1_fixed_accel: mass 0.001 -> 0.01; geometry 
- link left_f2_0: mass 0.05 -> 0.106; geometry collision cylinder length=0.023 radius=0.01; collision cylinder length=0.023 radius=0.015
- link left_f2_1: mass 0.05 -> 0.033; geometry collision cylinder length=0.067 radius=0.01; visual cylinder length=0.067 radius=0.01
- link left_f2_1_accel: mass 0.001 -> 0.01
- link left_f2_2: mass 0.05 -> 0.033; geometry collision cylinder length=0.057 radius=0.009; collision sphere radius=0.009
- link left_f2_2_accel: mass 0.001 -> 0.01; geometry 
- link left_f2_base: mass 0.35 -> 0.250
- link left_f2_fixed_accel: mass 0.001 -> 0.01; geometry 
- link left_f3_0: mass 0.05 -> 0.106; geometry collision cylinder length=0.023 radius=0.01; collision cylinder length=0.023 radius=0.015
- link left_f3_1: mass 0.05 -> 0.033; geometry collision cylinder length=0.067 radius=0.01; visual cylinder length=0.067 radius=0.01
- link left_f3_1_accel: mass 0.001 -> 0.01
- link left_f3_2: mass 0.05 -> 0.033; geometry collision cylinder length=0.057 radius=0.009; collision sphere radius=0.009
- link left_f3_2_accel: mass 0.001 -> 0.01; geometry 
- link left_f3_base: mass 0.35 -> 0.250
- link left_f3_fixed_accel: mass 0.001 -> 0.01
- link left_palm: mass 0.3 -> 1.303; geometry collision box size=0.09 .03 .06; collision box size=0.09 .03 .06
- link r_foot: geometry collision sphere radius=0; collision sphere radius=0
- link right_f0_0: mass 0.05 -> 0.106; geometry collision cylinder length=0.023 radius=0.01; collision cylinder length=0.023 radius=0.015
- link right_f0_1: mass 0.05 -> 0.033; geometry collision cylinder length=0.067 radius=0.01; visual cylinder length=0.067 radius=0.01
- link right_f0_1_accel: mass 0.001 -> 0.01
- link right_f0_2: mass 0.05 -> 0.033; geometry collision cylinder length=0.057 radius=0.009; collision sphere radius=0.009
- link right_f0_2_accel: mass 0.001 -> 0.01; geometry 
- link right_f0_base: mass 0.35 -> 0.250
- link right_f0_fixed_accel: mass 0.001 -> 0.01; geometry 
- link right_f1_0: mass 0.05 -> 0.106; geometry collision cylinder length=0.023 radius=0.01; collision cylinder length=0.023 radius=0.015
- link right_f1_1: mass 0.05 -> 0.033; geometry collision cylinder length=0.067 radius=0.01; visual cylinder length=0.067 radius=0.01
- link right_f1_1_accel: mass 0.001 -> 0.01
- link right_f1_2: mass 0.05 -> 0.033; geometry collision cylinder length=0.057 radius=0.009; collision sphere radius=0.009
- link right_f1_2_accel: mass 0.001 -> 0.01; geometry 
- link right_f1_base: mass 0.35 -> 0.250
- link right_f1_fixed_accel: mass 0.001 -> 0.01; geometry 
- link right_f2_0: mass 0.05 -> 0.106; geometry collision cylinder length=0.023 radius=0.01; collision cylinder length=0.023 radius=0.015
- link right_f2_1: mass 0.05 -> 0.033; geometry collision cylinder length=0.067 radius=0.01; visual cylinder length=0.067 radius=0.01
- link right_f2_1_accel: mass 0.001 -> 0.01
- link right_f2_2: mass 0.05 -> 0.033; geometry collision cylinder length=0.057 radius=0.009; collision sphere radius=0.009
- link right_f2_2_accel: mass 0.001 -> 0.01; geometry 
- link right_f2_base: mass 0.35 -> 0.250
- link right_f2_fixed_accel: mass 0.001 -> 0.01; geometry 
- link right_f3_0: mass 0.05 -> 0.106; geometry collision cylinder length=0.023 radius=0.01; collision cylinder length=0.023 radius=0.015
- link right_f3_1: mass 0.05 -> 0.033; geometry collision cylinder length=0.067 radius=0.01; visual cylinder length=0.067 radius=0.01
- link right_f3_1_accel: mass 0.001 -> 0.01
- link right_f3_2: mass 0.05 -> 0.033; geometry collision cylinder length=0.057 radius=0.009; collision sphere radius=0.009
- link right_f3_2_accel: mass 0.001 -> 0.01; geometry 
- link right_f3_base: mass 0.35 -> 0.250
- link right_f3_fixed_accel: mass 0.001 -> 0.01
- link right_palm: mass 0.3 -> 1.303; geometry collision box size=0.09 .03 .06; collision box size=0.09 .03 .06
Joints:
- removed joint left_f0_2_accel_dummy1
- removed joint left_f0_knuckle_dummy_contact
- removed joint left_f1_2_accel_dummy1
- removed joint left_f1_knuckle_dummy_contact
- removed joint left_f2_2_accel_dummy1
- removed joint left_f2_knuckle_dummy_contact
- removed joint left_f3_2_accel_dummy1
- removed joint left_hook_joint
- removed joint right_f0_2_accel_dummy1
- removed joint right_f0_knuckle_dummy_contact
- removed joint right_f1_2_accel_dummy1
- removed joint right_f1_knuckle_dummy_contact
- removed joint right_f2_2_accel_dummy1
- removed joint right_f2_knuckle_dummy_contact
- removed joint right_f3_2_accel_dummy1
- removed joint right_hook_joint
- added joint left_palm_left_camera_frame_joint: type fixed, parent left_palm, child left_palm_left_camera_frame, origin xyz=0.0435128991906 -0.0451672761576 0.025 rpy=-0.6708 -1.57079632679 3.14159265359
- added joint left_palm_left_camera_optical_frame_joint: type fixed, parent left_palm_left_camera_frame, child left_palm_left_camera_optical_frame, origin xyz=0 0 0 rpy=-1.57079632679 0.0 -1.57079632679
- added joint left_palm_right_camera_frame_joint: type fixed, parent left_palm, child left_palm_right_camera_frame, origin xyz=0.0683774130138 -0.0138342911048 0.025 rpy=-0.6708 -1.57079632679 3.14159265359
- added joint left_palm_right_camera_optical_frame_joint: type fixed, parent left_palm_right_camera_frame, child left_palm_right_camera_optical_frame, origin xyz=0 0 0 rpy=-1.57079632679 0.0 -1.57079632679
- added joint right_palm_left_camera_frame_joint: type fixed, parent right_palm, child right_palm_left_camera_frame, origin xyz=0.0683774130138 0.0138342911048 0.025 rpy=0.6708 -1.57079632679 3.14159265359
- added joint right_palm_left_camera_optical_frame_joint: type fixed, parent right_palm_left_camera_frame, child right_palm_left_camera_optical_frame, origin xyz=0 0 0 rpy=-1.57079632679 0.0 -1.57079632679
- added joint right_palm_right_camera_frame_joint: type fixed, parent right_palm, child right_palm_right_camera_frame, origin xyz=0.0435128991906 0.0451672761576 0.025 rpy=0.6708 -1.57079632679 3.14159265359
- added joint right_palm_right_camera_optical_frame_joint: type fixed, parent right_palm_right_camera_frame, child right_palm_right_camera_optical_frame, origin xyz=0 0 0 rpy=-1.57079632679 0.0 -1.57079632679
- joint left_f0_j0: limit lower=-1.57079632679 upper=0 effort=1 velocity=1 -> lower=-1.57079632679 upper=1.57079632679 effort=11 velocity=-1; type revolute -> fixed
- joint left_f0_j1: limit lower=-1.57079632679 upper=1.57079632679 effort=1 velocity=1 -> lower=-1.57079632679 upper=1.57079632679 effort=28 velocity=-1; type revolute -> fixed
- joint left_f0_j2: limit lower=-1.57079632679 upper=1.57079632679 effort=1 velocity=1 -> lower=-1.57079632679 upper=1.57079632679 effort=28 velocity=-1; type revolute -> fixed
- joint left_f1_j0: limit lower=-0.09 upper=0.09 effort=1 velocity=1 -> lower=-1.57079632679 upper=1.57079632679 effort=11 velocity=-1; type revolute -> fixed
- joint left_f1_j1: limit lower=-1.57079632679 upper=1.57079632679 effort=1 velocity=1 -> lower=-1.57079632679 upper=1.57079632679 effort=28 velocity=-1; type revolute -> fixed
- joint left_f1_j2: limit lower=-1.57079632679 upper=1.57079632679 effort=1 velocity=1 -> lower=-1.57079632679 upper=1.57079632679 effort=28 velocity=-1; type revolute -> fixed
- joint left_f2_j0: limit lower=0 upper=1.57079632679 effort=1 velocity=1 -> lower=-1.57079632679 upper=1.57079632679 effort=11 velocity=-1; type revolute -> fixed
- joint left_f2_j1: limit lower=-1.57079632679 upper=1.57079632679 effort=1 velocity=1 -> lower=-1.57079632679 upper=1.57079632679 effort=28 velocity=-1; type revolute -> fixed
- joint left_f2_j2: limit lower=-1.57079632679 upper=1.57079632679 effort=1 velocity=1 -> lower=-1.57079632679 upper=1.57079632679 effort=28 velocity=-1; type revolute -> fixed
- joint left_f3_j0: limit lower=-1.57079632679 upper=1.57079632679 effort=1 velocity=1 -> lower=-1.57079632679 upper=1.57079632679 effort=11 velocity=-1; type revolute -> fixed
- joint left_f3_j1: limit lower=-1.57079632679 upper=1.57079632679 effort=1 velocity=1 -> lower=-1.57079632679 upper=1.57079632679 effort=28 velocity=-1; type revolute -> fixed
- joint left_f3_j2: limit lower=-1.57079632679 upper=1.57079632679 effort=1 velocity=1 -> lower=-1.57079632679 upper=1.57079632679 effort=28 velocity=-1; type revolute -> fixed
- joint right_f0_j0: limit lower=-1.57079632679 upper=0 effort=1 velocity=1 -> lower=-1.57079632679 upper=1.57079632679 effort=11 velocity=-1; type revolute -> fixed
- joint right_f0_j1: limit lower=-1.57079632679 upper=1.57079632679 effort=1 velocity=1 -> lower=-1.57079632679 upper=1.57079632679 effort=28 velocity=-1; type revolute -> fixed
- joint right_f0_j2: limit lower=-1.57079632679 upper=1.57079632679 effort=1 velocity=1 -> lower=-1.57079632679 upper=1.57079632679 effort=28 velocity=-1; type revolute -> fixed
- joint right_f1_j0: limit lower=-0.09 upper=0.09 effort=1 velocity=1 -> lower=-1.57079632679 upper=1.57079632679 effort=11 velocity=-1; type revolute -> fixed
- joint right_f1_j1: limit lower=-1.57079632679 upper=1.57079632679 effort=1 velocity=1 -> lower=-1.57079632679 upper=1.57079632679 effort=28 velocity=-1; type revolute -> fixed
- joint right_f1_j2: limit lower=-1.57079632679 upper=1.57079632679 effort=1 velocity=1 -> lower=-1.57079632679 upper=1.57079632679 effort=28 velocity=-1; type revolute -> fixed
- joint right_f2_j0: limit lower=0 upper=1.57079632679 effort=1 velocity=1 -> lower=-1.57079632679 upper=1.57079632679 effort=11 velocity=-1; type revolute -> fixed
- joint right_f2_j1: limit lower=-1.57079632679 upper=1.57079632679 effort=1 velocity=1 -> lower=-1.57079632679 upper=1.57079632679 effort=28 velocity=-1; type revolute -> fixed
- joint right_f2_j2: limit lower=-1.57079632679 upper=1.57079632679 effort=1 velocity=1 -> lower=-1.57079632679 upper=1.57079632679 effort=28 velocity=-1; type revolute -> fixed
- joint right_f3_j0: limit lower=-1.57079632679 upper=1.57079632679 effort=1 velocity=1 -> lower=-1.57079632679 upper=1.57079632679 effort=11 velocity=-1; type revolute -> fixed
- joint right_f3_j1: limit lower=-1.57079632679 upper=1.57079632679 effort=1 velocity=1 -> lower=-1.57079632679 upper=1.57079632679 effort=28 velocity=-1; type revolute -> fixed
- joint right_f3_j2: limit lower=-1.57079632679 upper=1.57079632679 effort=1 velocity=1 -> lower=-1.57079632679 upper=1.57079632679 effort=28 velocity=-1; type revolute -> fixed

File: software/models/mit_gazebo_models/mit_robot_drake/model_minimal_contact_point_hands.urdf (robot description, URDF)
Before this commit: robot atlas, 31 links, 30 joints
Links:
- link l_foot: geometry collision sphere radius=0; collision sphere radius=0
- link r_foot: geometry collision sphere radius=0; collision sphere radius=0

Commit message: Adds knuckle contact points to l_hand and r_hand
git-svn-id: https://svn.csail.mit.edu/drc@4993 c7283977-0100-402a-a91a-fa70b306dbfe

File: software/models/mit_gazebo_models/mit_robot_drake/model_minimal_contact.urdf (robot description, URDF)
Before this commit: robot atlas, 29 links, 28 joints
Links:
- link l_hand: geometry collision sphere radius=0; collision sphere radius=0
- link r_hand: geometry collision sphere radius=0; collision sphere radius=0

File: software/models/mit_gazebo_models/mit_robot_drake/model_minimal_contact_point_hands.urdf (robot description, URDF)
Before this commit: robot atlas, 31 links, 30 joints
Links:
- link l_hand: geometry collision sphere radius=0; collision sphere radius=0
- link r_hand: geometry collision sphere radius=0; collision sphere radius=0

Commit message: Adds toe_mid and heel_mid contact points to minimal_contact models
git-svn-id: https://svn.csail.mit.edu/drc@4994 c7283977-0100-402a-a91a-fa70b306dbfe

File: software/models/mit_gazebo_models/mit_robot_drake/model_minimal_contact.urdf (robot description, URDF)
Before this commit: robot atlas, 29 links, 28 joints
Links:
- link l_foot: geometry collision sphere radius=0; collision sphere radius=0
- link r_foot: geometry collision sphere radius=0; collision sphere radius=0

File: software/models/mit_gazebo_models/mit_robot_drake/model_minimal_contact_point_hands.urdf (robot description, URDF)
Before this commit: robot atlas, 31 links, 30 joints
Links:
- link l_foot: geometry collision sphere radius=0; collision sphere radius=0
- link r_foot: geometry collision sphere radius=0; collision sphere radius=0

Commit message: Comment out toe_mid and heel_mid contact points
git-svn-id: https://svn.csail.mit.edu/drc@5071 c7283977-0100-402a-a91a-fa70b306dbfe

File: software/models/mit_gazebo_models/mit_robot_drake/model_minimal_contact.urdf (robot description, URDF)
Before this commit: robot atlas, 29 links, 28 joints
Links:
- link l_foot: geometry collision sphere radius=0; collision sphere radius=0
- link r_foot: geometry collision sphere radius=0; collision sphere radius=0

File: software/models/mit_gazebo_models/mit_robot_drake/model_minimal_contact_fixedjoint_hands.urdf (robot description, URDF)
Before this commit: robot atlas, 95 links, 94 joints
Links:
- link l_hand: geometry collision sphere radius=0; collision sphere radius=0
- link r_hand: geometry collision sphere radius=0; collision sphere radius=0

File: software/models/mit_gazebo_models/mit_robot_drake/model_minimal_contact_point_hands.urdf (robot description, URDF)
Before this commit: robot atlas, 31 links, 30 joints
Links:
- link l_foot: geometry collision sphere radius=0; collision sphere radius=0
- link r_foot: geometry collision sphere radius=0; collision sphere radius=0

Commit message: updating drake model shx joint limits
git-svn-id: https://svn.csail.mit.edu/drc/trunk@5957 c7283977-0100-402a-a91a-fa70b306dbfe

File: software/models/mit_gazebo_models/mit_robot_drake/model_minimal_contact.urdf (robot description, URDF)
Before this commit: robot atlas, 29 links, 28 joints
Joints:
- joint l_arm_shx: limit lower=-1.39626 upper=1.74533 effort=170 velocity=12 -> lower=-1.5 upper=1.74533 effort=170 velocity=12
- joint r_arm_shx: limit lower=-1.74533 upper=1.39626 effort=170 velocity=12 -> lower=-1.74533 upper=1.5 effort=170 velocity=12

File: software/models/mit_gazebo_models/mit_robot_drake/model_minimal_contact_fixedjoint_hands.urdf (robot description, URDF)
Before this commit: robot atlas, 95 links, 94 joints
Joints:
- joint l_arm_shx: limit lower=-1.39626 upper=1.74533 effort=170 velocity=12 -> lower=-1.5 upper=1.74533 effort=170 velocity=12
- joint r_arm_shx: limit lower=-1.74533 upper=1.39626 effort=170 velocity=12 -> lower=-1.74533 upper=1.5 effort=170 velocity=12

File: software/models/mit_gazebo_models/mit_robot_drake/model_minimal_contact_point_hands.urdf (robot description, URDF)
Before this commit: robot atlas, 31 links, 30 joints
Joints:
- joint l_arm_shx: limit lower=-1.39626 upper=1.74533 effort=170 velocity=12 -> lower=-1.5 upper=1.74533 effort=170 velocity=12
- joint r_arm_shx: limit lower=-1.74533 upper=1.39626 effort=170 velocity=12 -> lower=-1.74533 upper=1.5 effort=170 velocity=12

File: software/models/mit_gazebo_models/mit_robot_drake/model_simple_visuals.urdf (robot description, URDF)
Before this commit: robot atlas, 33 links, 32 joints
Joints:
- joint l_arm_shx: limit lower=-1.39626 upper=1.74533 effort=170 velocity=12 -> lower=-1.5 upper=1.74533 effort=170 velocity=12
- joint r_arm_shx: limit lower=-1.74533 upper=1.39626 effort=170 velocity=12 -> lower=-1.74533 upper=1.5 effort=170 velocity=12

File: software/models/mit_gazebo_models/mit_robot_drake/xacro/atlas_skeleton_minimal_contact.urdf (robot description, URDF)
Before this commit: robot drc_skeleton, 28 links, 28 joints
Joints:
- joint l_arm_shx: limit lower=-1.39626 upper=1.74533 effort=170 velocity=12 -> lower=-1.5 upper=1.74533 effort=170 velocity=12
- joint r_arm_shx: limit lower=-1.74533 upper=1.39626 effort=170 velocity=12 -> lower=-1.74533 upper=1.5 effort=170 velocity=12

File: software/models/mit_gazebo_models/mit_robot_drake/xacro/atlas_skeleton_simple_visuals.urdf (robot description, URDF)
Before this commit: robot drc_skeleton, 28 links, 28 joints
Joints:
- joint l_arm_shx: limit lower=-1.39626 upper=1.74533 effort=170 velocity=12 -> lower=-1.5 upper=1.74533 effort=170 velocity=12
- joint r_arm_shx: limit lower=-1.74533 upper=1.39626 effort=170 velocity=12 -> lower=-1.74533 upper=1.5 effort=170 velocity=12

File: software/models/mit_gazebo_models/mit_robot_drake/xacro/atlas_skeleton_simple_visuals_minimal_contact.urdf (robot description, URDF)
Before this commit: robot drc_skeleton, 28 links, 28 joints
Joints:
- joint l_arm_shx: limit lower=-1.39626 upper=1.74533 effort=170 velocity=12 -> lower=-1.5 upper=1.74533 effort=170 velocity=12
- joint r_arm_shx: limit lower=-1.74533 upper=1.39626 effort=170 velocity=12 -> lower=-1.74533 upper=1.5 effort=170 velocity=12

Commit message: updated leg friction params

File: software/models/mit_gazebo_models/mit_robot_drake/model_minimal_contact.urdf (robot description, URDF)
Before this commit: robot atlas, 29 links, 28 joints
Links:
- link utorso: mass 52.007 -> 55

File: software/models/mit_gazebo_models/mit_robot_drake/model_minimal_contact_fixedjoint_hands.urdf (robot description, URDF)
Before this commit: robot atlas, 95 links, 94 joints
Links:
- link utorso: mass 52.007 -> 55

File: software/models/mit_gazebo_models/mit_robot_drake/model_minimal_contact_point_hands.urdf (robot description, URDF)
Before this commit: robot atlas, 31 links, 30 joints
Links:
- link utorso: mass 52.007 -> 55

File: software/models/mit_gazebo_models/mit_robot_drake/model_minimal_contact_point_stumps.urdf (robot description, URDF)
Before this commit: robot atlas, 31 links, 30 joints
Links:
- link utorso: mass 52.007 -> 55

File: software/models/mit_gazebo_models/mit_robot_drake/xacro/atlas_skeleton_minimal_contact.urdf (robot description, URDF)
Before this commit: robot drc_skeleton, 28 links, 28 joints
Links:
- link utorso: mass 52.007 -> 55
