Commit message: fixed utorso mass

File: software/models/mit_gazebo_models/mit_robot_drake/model_minimal_contact.urdf (robot description, URDF)
Before this commit: robot atlas, 29 links, 28 joints
Links:
- link utorso: mass 60 -> 52.007

File: software/models/mit_gazebo_models/mit_robot_drake/model_minimal_contact_fixedjoint_hands.urdf (robot description, URDF)
Before this commit: robot atlas, 95 links, 94 joints
Links:
- link utorso: mass 60 -> 52.007

File: software/models/mit_gazebo_models/mit_robot_drake/model_minimal_contact_point_hands.urdf (robot description, URDF)
Before this commit: robot atlas, 31 links, 30 joints
Links:
- link utorso: mass 60 -> 52.007

File: software/models/mit_gazebo_models/mit_robot_drake/model_minimal_contact_point_stumps.urdf (robot description, URDF)
Before this commit: robot atlas, 31 links, 30 joints
Links:
- link utorso: mass 60 -> 52.007

File: software/models/mit_gazebo_models/mit_robot_drake/xacro/atlas_skeleton_minimal_contact.urdf (robot description, URDF)
Before this commit: robot drc_skeleton, 28 links, 28 joints
Links:
- link utorso: mass 60 -> 52.007

Commit message: pulling out friction params. reduced torso mass in minimal contact skeleton

File: software/models/mit_gazebo_models/mit_robot_drake/model_minimal_contact.urdf (robot description, URDF)
Before this commit: robot atlas, 29 links, 28 joints
Links:
- link utorso: mass 55 -> 52

File: software/models/mit_gazebo_models/mit_robot_drake/model_minimal_contact_fixedjoint_hands.urdf (robot description, URDF)
Before this commit: robot atlas, 95 links, 94 joints
Links:
- link utorso: mass 55 -> 52

File: software/models/mit_gazebo_models/mit_robot_drake/model_minimal_contact_point_hands.urdf (robot description, URDF)
Before this commit: robot atlas, 31 links, 30 joints
Links:
- link utorso: mass 55 -> 52

File: software/models/mit_gazebo_models/mit_robot_drake/model_minimal_contact_point_stumps.urdf (robot description, URDF)
Before this commit: robot atlas, 31 links, 30 joints
Links:
- link utorso: mass 55 -> 52

File: software/models/mit_gazebo_models/mit_robot_drake/xacro/atlas_skeleton_minimal_contact.urdf (robot description, URDF)
Before this commit: robot drc_skeleton, 28 links, 28 joints
Links:
- link utorso: mass 55 -> 52
