Commit message: adding a drake-compatible version of the latest atlas model
git-svn-id: https://svn.csail.mit.edu/drc@875 c7283977-0100-402a-a91a-fa70b306dbfe

File: software/models/mit_gazebo_models/mit_robot_drake/model.urdf (robot description, URDF)
Before this commit: robot mit_drc_robot, 29 links, 28 joints
Links:
- link head: geometry collision mesh filename=/home/scottk/drc/ros_workspace/mit_drcsim_scripts/models/mi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 scale=1 1 1; visual mesh filename=/home/scottk/drc/ros_workspace/mit_drcsim_scripts/models/mi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 scale=1 1 1
- link l_clav: geometry collision mesh filename=/home/scottk/drc/ros_workspace/mit_drcsim_scripts/models/mi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 scale=1 1 1; visual mesh filename=/home/scottk/drc/ros_workspace/mit_drcsim_scripts/models/mi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 scale=1 1 1
- link l_farm: geometry collision mesh filename=/home/scottk/drc/ros_workspace/mit_drcsim_scripts/models/mi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 scale=1 1 1; visual mesh filename=/home/scottk/drc/ros_workspace/mit_drcsim_scripts/models/mi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 scale=1 1 1
- link l_foot: geometry collision mesh filename=/home/scottk/drc/ros_workspace/mit_drcsim_scripts/models/mi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 scale=1 1 1; visual mesh filename=/home/scottk/drc/ros_workspace/mit_drcsim_scripts/models/mi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 scale=1 1 1
- link l_hand: geometry collision mesh filename=/home/scottk/drc/ros_workspace/mit_drcsim_scripts/models/mi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 scale=1 1 1; visual mesh filename=/home/scottk/drc/ros_workspace/mit_drcsim_scripts/models/mi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 scale=1 1 1
- link l_larm: geometry collision mesh filename=/home/scottk/drc/ros_workspace/mit_drcsim_scripts/models/mi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 scale=1 1 1; visual mesh filename=/home/scottk/drc/ros_workspace/mit_drcsim_scripts/models/mi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 scale=1 1 1
- link l_lglut: geometry collision mesh filename=/home/scottk/drc/ros_workspace/mit_drcsim_scripts/models/mi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 scale=1 1 1; visual mesh filename=/home/scottk/drc/ros_workspace/mit_drcsim_scripts/models/mi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 scale=1 1 1
- link l_lleg: geometry collision mesh filename=/home/scottk/drc/ros_workspace/mit_drcsim_scripts/models/mi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 scale=1 1 1; visual mesh filename=/home/scottk/drc/ros_workspace/mit_drcsim_scripts/models/mi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 scale=1 1 1
- link l_scap: geometry collision mesh filename=/home/scottk/drc/ros_workspace/mit_drcsim_scripts/models/mi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 scale=1 1 1; visual mesh filename=/home/scottk/drc/ros_workspace/mit_drcsim_scripts/models/mi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 scale=1 1 1
- link l_talus: geometry collision mesh filename=/home/scottk/drc/ros_workspace/mit_drcsim_scripts/models/mi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 scale=1 1 1; visual mesh filename=/home/scottk/drc/ros_workspace/mit_drcsim_scripts/models/mi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 scale=1 1 1
- link l_uarm: geometry collision mesh filename=/home/scottk/drc/ros_workspace/mit_drcsim_scripts/models/mi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 scale=1 1 1; visual mesh filename=/home/scottk/drc/ros_workspace/mit_drcsim_scripts/models/mi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 scale=1 1 1
- link l_uglut: geometry collision mesh filename=/home/scottk/drc/ros_workspace/mit_drcsim_scripts/models/mi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 scale=1 1 1; visual mesh filename=/home/scottk/drc/ros_workspace/mit_drcsim_scripts/models/mi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 scale=1 1 1
- link l_uleg: geometry collision mesh filename=/home/scottk/drc/ros_workspace/mit_drcsim_scripts/models/mi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 scale=1 1 1; visual mesh filename=/home/scottk/drc/ros_workspace/mit_drcsim_scripts/models/mi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 scale=1 1 1
- link ltorso: geometry collision mesh filename=/home/scottk/drc/ros_workspace/mit_drcsim_scripts/models/mi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 scale=1 1 1; visual mesh filename=/home/scottk/drc/ros_workspace/mit_drcsim_scripts/models/mi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 scale=1 1 1
- link mtorso: geometry collision mesh filename=/home/scottk/drc/ros_workspace/mit_drcsim_scripts/models/mi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 scale=1 1 1; visual mesh filename=/home/scottk/drc/ros_workspace/mit_drcsim_scripts/models/mi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 scale=1 1 1
- link pelvis: geometry collision mesh filename=/home/scottk/drc/ros_workspace/mit_drcsim_scripts/models/mi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 scale=1 1 1; visual mesh filename=/home/scottk/drc/ros_workspace/mit_drcsim_scripts/models/mi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 scale=1 1 1
- link r_clav: geometry collision mesh filename=/home/scottk/drc/ros_workspace/mit_drcsim_scripts/models/mi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 scale=1 1 1; visual mesh filename=/home/scottk/drc/ros_workspace/mit_drcsim_scripts/models/mi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 scale=1 1 1
- link r_farm: geometry collision mesh filename=/home/scottk/drc/ros_workspace/mit_drcsim_scripts/models/mi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 scale=1 1 1; visual mesh filename=/home/scottk/drc/ros_workspace/mit_drcsim_scripts/models/mi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 scale=1 1 1
- link r_foot: geometry collision mesh filename=/home/scottk/drc/ros_workspace/mit_drcsim_scripts/models/mi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 scale=1 1 1; visual mesh filename=/home/scottk/drc/ros_workspace/mit_drcsim_scripts/models/mi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 scale=1 1 1
- link r_hand: geometry collision mesh filename=/home/scottk/drc/ros_workspace/mit_drcsim_scripts/models/mi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 scale=1 1 1; visual mesh filename=/home/scottk/drc/ros_workspace/mit_drcsim_scripts/models/mi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 scale=1 1 1
- link r_larm: geometry collision mesh filename=/home/scottk/drc/ros_workspace/mit_drcsim_scripts/models/mi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 scale=1 1 1; visual mesh filename=/home/scottk/drc/ros_workspace/mit_drcsim_scripts/models/mi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 scale=1 1 1
- link r_lglut: geometry collision mesh filename=/home/scottk/drc/ros_workspace/mit_drcsim_scripts/models/mi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 scale=1 1 1; visual mesh filename=/home/scottk/drc/ros_workspace/mit_drcsim_scripts/models/mi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 scale=1 1 1
- link r_lleg: geometry collision mesh filename=/home/scottk/drc/ros_workspace/mit_drcsim_scripts/models/mi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 scale=1 1 1; visual mesh filename=/home/scottk/drc/ros_workspace/mit_drcsim_scripts/models/mi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 scale=1 1 1
- link r_scap: geometry collision mesh filename=/home/scottk/drc/ros_workspace/mit_drcsim_scripts/models/mi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 scale=1 1 1; visual mesh filename=/home/scottk/drc/ros_workspace/mit_drcsim_scripts/models/mi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 scale=1 1 1
- link r_talus: geometry collision mesh filename=/home/scottk/drc/ros_workspace/mit_drcsim_scripts/models/mi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 scale=1 1 1; visual mesh filename=/home/scottk/drc/ros_workspace/mit_drcsim_scripts/models/mi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 scale=1 1 1
- link r_uarm: geometry collision mesh filename=/home/scottk/drc/ros_workspace/mit_drcsim_scripts/models/mi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 scale=1 1 1; visual mesh filename=/home/scottk/drc/ros_workspace/mit_drcsim_scripts/models/mi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 scale=1 1 1
- link r_uglut: geometry collision mesh filename=/home/scottk/drc/ros_workspace/mit_drcsim_scripts/models/mi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 scale=1 1 1; visual mesh filename=/home/scottk/drc/ros_workspace/mit_drcsim_scripts/models/mi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 scale=1 1 1
- link r_uleg: geometry collision mesh filename=/home/scottk/drc/ros_workspace/mit_drcsim_scripts/models/mi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 scale=1 1 1; visual mesh filename=/home/scottk/drc/ros_workspace/mit_drcsim_scripts/models/mi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 scale=1 1 1
- link utorso: geometry collision mesh filename=/home/scottk/drc/ros_workspace/mit_drcsim_scripts/models/mi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 scale=1 1 1; visual mesh filename=/home/scottk/drc/ros_workspace/mit_drcsim_scripts/models/mi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 scale=1 1 1

File: software/models/mit_gazebo_models/mit_robot_drake/model_minimal_contact.urdf (robot description, URDF)
Before this commit: robot mit_drc_robot, 29 links, 28 joints
Links:
- link head: geometry visual mesh filename=/home/scottk/drc/ros_workspace/mit_drcsim_scripts/models/mi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 scale=1 1 1
- link l_clav: geometry visual mesh filename=/home/scottk/drc/ros_workspace/mit_drcsim_scripts/models/mi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 scale=1 1 1
- link l_farm: geometry visual mesh filename=/home/scottk/drc/ros_workspace/mit_drcsim_scripts/models/mi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 scale=1 1 1
- link l_foot: geometry collision sphere radius=0; collision sphere radius=0
- link l_hand: geometry visual mesh filename=/home/scottk/drc/ros_workspace/mit_drcsim_scripts/models/mi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 scale=1 1 1
- link l_larm: geometry visual mesh filename=/home/scottk/drc/ros_workspace/mit_drcsim_scripts/models/mi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 scale=1 1 1
- link l_lglut: geometry visual mesh filename=/home/scottk/drc/ros_workspace/mit_drcsim_scripts/models/mi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 scale=1 1 1
- link l_lleg: geometry visual mesh filename=/home/scottk/drc/ros_workspace/mit_drcsim_scripts/models/mi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 scale=1 1 1
- link l_scap: geometry visual mesh filename=/home/scottk/drc/ros_workspace/mit_drcsim_scripts/models/mi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 scale=1 1 1
- link l_talus: geometry visual mesh filename=/home/scottk/drc/ros_workspace/mit_drcsim_scripts/models/mi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 scale=1 1 1
- link l_uarm: geometry visual mesh filename=/home/scottk/drc/ros_workspace/mit_drcsim_scripts/models/mi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 scale=1 1 1
- link l_uglut: geometry visual mesh filename=/home/scottk/drc/ros_workspace/mit_drcsim_scripts/models/mi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 scale=1 1 1
- link l_uleg: geometry visual mesh filename=/home/scottk/drc/ros_workspace/mit_drcsim_scripts/models/mi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 scale=1 1 1
- link ltorso: geometry visual mesh filename=/home/scottk/drc/ros_workspace/mit_drcsim_scripts/models/mi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 scale=1 1 1
- link mtorso: geometry visual mesh filename=/home/scottk/drc/ros_workspace/mit_drcsim_scripts/models/mi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 scale=1 1 1
- link pelvis: geometry visual mesh filename=/home/scottk/drc/ros_workspace/mit_drcsim_scripts/models/mi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 scale=1 1 1
- link r_clav: geometry visual mesh filename=/home/scottk/drc/ros_workspace/mit_drcsim_scripts/models/mi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 scale=1 1 1
- link r_farm: geometry visual mesh filename=/home/scottk/drc/ros_workspace/mit_drcsim_scripts/models/mi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 scale=1 1 1
- link r_foot: geometry collision sphere radius=0; collision sphere radius=0
- link r_hand: geometry visual mesh filename=/home/scottk/drc/ros_workspace/mit_drcsim_scripts/models/mi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 scale=1 1 1
- link r_larm: geometry visual mesh filename=/home/scottk/drc/ros_workspace/mit_drcsim_scripts/models/mi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 scale=1 1 1
- link r_lglut: geometry visual mesh filename=/home/scottk/drc/ros_workspace/mit_drcsim_scripts/models/mi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 scale=1 1 1
- link r_lleg: geometry visual mesh filename=/home/scottk/drc/ros_workspace/mit_drcsim_scripts/models/mi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 scale=1 1 1
- link r_scap: geometry visual mesh filename=/home/scottk/drc/ros_workspace/mit_drcsim_scripts/models/mi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 scale=1 1 1
- link r_talus: geometry visual mesh filename=/home/scottk/drc/ros_workspace/mit_drcsim_scripts/models/mi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 scale=1 1 1
- link r_uarm: geometry visual mesh filename=/home/scottk/drc/ros_workspace/mit_drcsim_scripts/models/mi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 scale=1 1 1
- link r_uglut: geometry visual mesh filename=/home/scottk/drc/ros_workspace/mit_drcsim_scripts/models/mi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 scale=1 1 1
- link r_uleg: geometry visual mesh filename=/home/scottk/drc/ros_workspace/mit_drcsim_scripts/models/mi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 scale=1 1 1
- link utorso: geometry visual mesh filename=/home/scottk/drc/ros_workspace/mit_drcsim_scripts/models/mi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 scale=1 1 1

Commit message: new directory for robot with hands, xacro file is in rit_robot_PnC
git-svn-id: https://svn.csail.mit.edu/drc@1399 c7283977-0100-402a-a91a-fa70b306dbfe

File: software/models/mit_gazebo_models/mit_robot_drake/model.urdf (robot description, URDF)
Before this commit: robot atlas, 29 links, 28 joints
Links:
- link head: geometry collision mesh filename=/home/ceci91/drc/ros_workspace/mit_drcsim_scripts/models/mi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 scale=1 1 1; visual mesh filename=/home/ceci91/drc/ros_workspace/mit_drcsim_scripts/models/mi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 scale=1 1 1
- link l_clav: geometry collision mesh filename=/home/ceci91/drc/ros_workspace/mit_drcsim_scripts/models/mi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 scale=1 1 1; visual mesh filename=/home/ceci91/drc/ros_workspace/mit_drcsim_scripts/models/mi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 scale=1 1 1
- link l_farm: geometry collision mesh filename=/home/ceci91/drc/ros_workspace/mit_drcsim_scripts/models/mi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 scale=1 1 1; visual mesh filename=/home/ceci91/drc/ros_workspace/mit_drcsim_scripts/models/mi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 scale=1 1 1
- link l_foot: geometry collision mesh filename=/home/ceci91/drc/ros_workspace/mit_drcsim_scripts/models/mi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 scale=1 1 1; visual mesh filename=/home/ceci91/drc/ros_workspace/mit_drcsim_scripts/models/mi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 scale=1 1 1
- link l_hand: geometry collision mesh filename=/home/ceci91/drc/ros_workspace/mit_drcsim_scripts/models/mi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 scale=1 1 1; visual mesh filename=/home/ceci91/drc/ros_workspace/mit_drcsim_scripts/models/mi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 scale=1 1 1
- link l_larm: geometry collision mesh filename=/home/ceci91/drc/ros_workspace/mit_drcsim_scripts/models/mi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 scale=1 1 1; visual mesh filename=/home/ceci91/drc/ros_workspace/mit_drcsim_scripts/models/mi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 scale=1 1 1
- link l_lglut: geometry collision mesh filename=/home/ceci91/drc/ros_workspace/mit_drcsim_scripts/models/mi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 scale=1 1 1; visual mesh filename=/home/ceci91/drc/ros_workspace/mit_drcsim_scripts/models/mi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 scale=1 1 1
- link l_lleg: geometry collision mesh filename=/home/ceci91/drc/ros_workspace/mit_drcsim_scripts/models/mi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 scale=1 1 1; visual mesh filename=/home/ceci91/drc/ros_workspace/mit_drcsim_scripts/models/mi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 scale=1 1 1
- link l_scap: geometry collision mesh filename=/home/ceci91/drc/ros_workspace/mit_drcsim_scripts/models/mi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 scale=1 1 1; visual mesh filename=/home/ceci91/drc/ros_workspace/mit_drcsim_scripts/models/mi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 scale=1 1 1
- link l_talus: geometry collision mesh filename=/home/ceci91/drc/ros_workspace/mit_drcsim_scripts/models/mi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 scale=1 1 1; visual mesh filename=/home/ceci91/drc/ros_workspace/mit_drcsim_scripts/models/mi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 scale=1 1 1
- link l_uarm: geometry collision mesh filename=/home/ceci91/drc/ros_workspace/mit_drcsim_scripts/models/mi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 scale=1 1 1; visual mesh filename=/home/ceci91/drc/ros_workspace/mit_drcsim_scripts/models/mi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 scale=1 1 1
- link l_uglut: geometry collision mesh filename=/home/ceci91/drc/ros_workspace/mit_drcsim_scripts/models/mi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 scale=1 1 1; visual mesh filename=/home/ceci91/drc/ros_workspace/mit_drcsim_scripts/models/mi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 scale=1 1 1
- link l_uleg: geometry collision mesh filename=/home/ceci91/drc/ros_workspace/mit_drcsim_scripts/models/mi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 scale=1 1 1; visual mesh filename=/home/ceci91/drc/ros_workspace/mit_drcsim_scripts/models/mi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 scale=1 1 1
- link ltorso: geometry collision mesh filename=/home/ceci91/drc/ros_workspace/mit_drcsim_scripts/models/mi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 scale=1 1 1; visual mesh filename=/home/ceci91/drc/ros_workspace/mit_drcsim_scripts/models/mi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 scale=1 1 1
- link mtorso: geometry collision mesh filename=/home/ceci91/drc/ros_workspace/mit_drcsim_scripts/models/mi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 scale=1 1 1; visual mesh filename=/home/ceci91/drc/ros_workspace/mit_drcsim_scripts/models/mi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 scale=1 1 1
- link pelvis: geometry collision mesh filename=/home/ceci91/drc/ros_workspace/mit_drcsim_scripts/models/mi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 scale=1 1 1; visual mesh filename=/home/ceci91/drc/ros_workspace/mit_drcsim_scripts/models/mi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 scale=1 1 1
- link r_clav: geometry collision mesh filename=/home/ceci91/drc/ros_workspace/mit_drcsim_scripts/models/mi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 scale=1 1 1; visual mesh filename=/home/ceci91/drc/ros_workspace/mit_drcsim_scripts/models/mi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 scale=1 1 1
- link r_farm: geometry collision mesh filename=/home/ceci91/drc/ros_workspace/mit_drcsim_scripts/models/mi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 scale=1 1 1; visual mesh filename=/home/ceci91/drc/ros_workspace/mit_drcsim_scripts/models/mi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 scale=1 1 1
- link r_foot: geometry collision mesh filename=/home/ceci91/drc/ros_workspace/mit_drcsim_scripts/models/mi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 scale=1 1 1; visual mesh filename=/home/ceci91/drc/ros_workspace/mit_drcsim_scripts/models/mi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 scale=1 1 1
- link r_hand: geometry collision mesh filename=/home/ceci91/drc/ros_workspace/mit_drcsim_scripts/models/mi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 scale=1 1 1; visual mesh filename=/home/ceci91/drc/ros_workspace/mit_drcsim_scripts/models/mi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 scale=1 1 1
- link r_larm: geometry collision mesh filename=/home/ceci91/drc/ros_workspace/mit_drcsim_scripts/models/mi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 scale=1 1 1; visual mesh filename=/home/ceci91/drc/ros_workspace/mit_drcsim_scripts/models/mi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 scale=1 1 1
- link r_lglut: geometry collision mesh filename=/home/ceci91/drc/ros_workspace/mit_drcsim_scripts/models/mi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 scale=1 1 1; visual mesh filename=/home/ceci91/drc/ros_workspace/mit_drcsim_scripts/models/mi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 scale=1 1 1
- link r_lleg: geometry collision mesh filename=/home/ceci91/drc/ros_workspace/mit_drcsim_scripts/models/mi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 scale=1 1 1; visual mesh filename=/home/ceci91/drc/ros_workspace/mit_drcsim_scripts/models/mi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 scale=1 1 1
- link r_scap: geometry collision mesh filename=/home/ceci91/drc/ros_workspace/mit_drcsim_scripts/models/mi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 scale=1 1 1; visual mesh filename=/home/ceci91/drc/ros_workspace/mit_drcsim_scripts/models/mi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 scale=1 1 1
- link r_talus: geometry collision mesh filename=/home/ceci91/drc/ros_workspace/mit_drcsim_scripts/models/mi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 scale=1 1 1; visual mesh filename=/home/ceci91/drc/ros_workspace/mit_drcsim_scripts/models/mi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 scale=1 1 1
- link r_uarm: geometry collision mesh filename=/home/ceci91/drc/ros_workspace/mit_drcsim_scripts/models/mi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 scale=1 1 1; visual mesh filename=/home/ceci91/drc/ros_workspace/mit_drcsim_scripts/models/mi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 scale=1 1 1
- link r_uglut: geometry collision mesh filename=/home/ceci91/drc/ros_workspace/mit_drcsim_scripts/models/mi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 scale=1 1 1; visual mesh filename=/home/ceci91/drc/ros_workspace/mit_drcsim_scripts/models/mi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 scale=1 1 1
- link r_uleg: geometry collision mesh filename=/home/ceci91/drc/ros_workspace/mit_drcsim_scripts/models/mi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 scale=1 1 1; visual mesh filename=/home/ceci91/drc/ros_workspace/mit_drcsim_scripts/models/mi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 scale=1 1 1
- link utorso: geometry collision mesh filename=/home/ceci91/drc/ros_workspace/mit_drcsim_scripts/models/mi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 scale=1 1 1; visual mesh filename=/home/ceci91/drc/ros_workspace/mit_drcsim_scripts/models/mi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 scale=1 1 1

File: software/models/mit_gazebo_models/mit_robot_hands/drake_urdfs/xacro/sandia_hand_drake_floating.xacro (robot description, xacro)
@@ -4,5 +4,7 @@
   <include filename="$(find sandia_hand_utils)/urdf/sandia_hand.gazebo.xacro" />
   <include filename="$(find sandia_hand_utils)/urdf/sandia_hand.transmission.xacro" />
-  <include filename="$(find mit_drcsim_scripts)/models/mit_robot_hands/drake_urdfs/xacro/sandia_hand_floating_base.xacro"/>
+  <include filename="$(find mit_drcsim_scripts)/models/mit_robot_hands/drake_urdfs/xacro/sandia_hand_floating_base.xacro"/>\
+ <!-- If the following line is uncommented then the grasp controller will fail // Not true anyore -->
+  <include filename="$(find mit_drcsim_scripts)/models/mit_robot_hands/xacro/sandia_base_transmissions.xacro"/>
   <xacro:macro name="finger" params="idx x y z r p yaw side">
     <link name="${side}_f${idx}_base">

File: software/models/mit_gazebo_models/mit_robot_hands/drake_urdfs/xacro/sandia_hand_right_drake.urdf.xacro (robot description, xacro)
@@ -11,5 +11,5 @@
         <inertia ixx="0.01" ixy="0" ixz="0" iyy="0.01" iyz="0" izz="0.01" />
     </inertial>
-    <!-- <visual>
+   <!-- <visual>
         <origin xyz="0 0 0.25" rpy="0 0 0" />
         <geometry>
@@ -25,5 +25,5 @@
   </link>
   <xacro:sandia_hand side="right" parent="base">
-    <origin xyz="0 0 0" rpy="0 0 0"/>
+    <origin xyz="0 0 0.0" rpy="0 -1.57079 0"/>
   </xacro:sandia_hand>
 </robot>

File: software/models/mit_gazebo_models/mit_robot_hands/xacro/sandia_hand_left.urdf.xacro (robot description, xacro)
@@ -25,5 +25,5 @@
   </link>
   <xacro:sandia_hand side="left" parent="base">
-    <origin xyz="0 0 0.0" rpy="0 -1.57079 0"/>
+    <origin xyz="0 0 0.5" rpy="0 -1.57079 0"/>
   </xacro:sandia_hand>
 </robot>

File: software/models/mit_gazebo_models/mit_robot_hands/xacro/sandia_hand_right.urdf.xacro (robot description, xacro)
@@ -3,5 +3,5 @@
        xmlns:interface="http://playerstage.sourceforge.net/gazebo/xmlschema/#interface"
        xmlns:xacro="http://playerstage.sourceforge.net/gazebo/xmlschema/#interface"
-       name="sandia_hand" >
+       name="humanoid" >
   <include filename="$(find sandia_hand_utils)/urdf/sandia_hand.urdf.xacro" />
   <link name="base">
@@ -25,5 +25,5 @@
   </link>
   <xacro:sandia_hand side="right" parent="base">
-    <origin xyz="0 0 0" rpy="0 -1.57079 0"/>
+    <origin xyz="0 0 0.5" rpy="0 -1.57079 0"/>
   </xacro:sandia_hand>
 </robot>
