Commit message: git-svn-id: https://svn.csail.mit.edu/drc@1400 c7283977-0100-402a-a91a-fa70b306dbfe

File: software/models/mit_gazebo_models/mit_robot_drake/model.urdf (robot description, URDF)
Before this commit: robot atlas, 29 links, 28 joints
Links:
- link head: geometry visual mesh filename=/home/scottk/drc/ros_workspace/mit_drcsim_scripts/models/mi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 scale=1 1 1
- link l_clav: geometry visual mesh filename=/home/scottk/drc/ros_workspace/mit_drcsim_scripts/models/mi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 scale=1 1 1
- link l_farm: geometry visual mesh filename=/home/scottk/drc/ros_workspace/mit_drcsim_scripts/models/mi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 scale=1 1 1
- link l_foot: geometry collision sphere radius=0; collision sphere radius=0
- link l_hand: geometry visual mesh filename=/home/scottk/drc/ros_workspace/mit_drcsim_scripts/models/mi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 scale=1 1 1
- link l_larm: geometry visual mesh filename=/home/scottk/drc/ros_workspace/mit_drcsim_scripts/models/mi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 scale=1 1 1
- link l_lglut: geometry visual mesh filename=/home/scottk/drc/ros_workspace/mit_drcsim_scripts/models/mi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 scale=1 1 1
- link l_lleg: geometry visual mesh filename=/home/scottk/drc/ros_workspace/mit_drcsim_scripts/models/mi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 scale=1 1 1
- link l_scap: geometry visual mesh filename=/home/scottk/drc/ros_workspace/mit_drcsim_scripts/models/mi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 scale=1 1 1
- link l_talus: geometry visual mesh filename=/home/scottk/drc/ros_workspace/mit_drcsim_scripts/models/mi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 scale=1 1 1
- link l_uarm: geometry visual mesh filename=/home/scottk/drc/ros_workspace/mit_drcsim_scripts/models/mi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 scale=1 1 1
- link l_uglut: geometry visual mesh filename=/home/scottk/drc/ros_workspace/mit_drcsim_scripts/models/mi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 scale=1 1 1
- link l_uleg: geometry visual mesh filename=/home/scottk/drc/ros_workspace/mit_drcsim_scripts/models/mi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 scale=1 1 1
- link ltorso: geometry visual mesh filename=/home/scottk/drc/ros_workspace/mit_drcsim_scripts/models/mi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 scale=1 1 1
- link mtorso: geometry visual mesh filename=/home/scottk/drc/ros_workspace/mit_drcsim_scripts/models/mi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 scale=1 1 1
- link pelvis: geometry visual mesh filename=/home/scottk/drc/ros_workspace/mit_drcsim_scripts/models/mi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 scale=1 1 1
- link r_clav: geometry visual mesh filename=/home/scottk/drc/ros_workspace/mit_drcsim_scripts/models/mi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 scale=1 1 1
- link r_farm: geometry visual mesh filename=/home/scottk/drc/ros_workspace/mit_drcsim_scripts/models/mi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 scale=1 1 1
- link r_foot: geometry collision sphere radius=0; collision sphere radius=0
- link r_hand: geometry visual mesh filename=/home/scottk/drc/ros_workspace/mit_drcsim_scripts/models/mi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 scale=1 1 1
- link r_larm: geometry visual mesh filename=/home/scottk/drc/ros_workspace/mit_drcsim_scripts/models/mi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 scale=1 1 1
- link r_lglut: geometry visual mesh filename=/home/scottk/drc/ros_workspace/mit_drcsim_scripts/models/mi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 scale=1 1 1
- link r_lleg: geometry visual mesh filename=/home/scottk/drc/ros_workspace/mit_drcsim_scripts/models/mi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 scale=1 1 1
- link r_scap: geometry visual mesh filename=/home/scottk/drc/ros_workspace/mit_drcsim_scripts/models/mi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 scale=1 1 1
- link r_talus: geometry visual mesh filename=/home/scottk/drc/ros_workspace/mit_drcsim_scripts/models/mi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 scale=1 1 1
- link r_uarm: geometry visual mesh filename=/home/scottk/drc/ros_workspace/mit_drcsim_scripts/models/mi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 scale=1 1 1
- link r_uglut: geometry visual mesh filename=/home/scottk/drc/ros_workspace/mit_drcsim_scripts/models/mi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 scale=1 1 1
- link r_uleg: geometry visual mesh filename=/home/scottk/drc/ros_workspace/mit_drcsim_scripts/models/mi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 scale=1 1 1
- link utorso: geometry visual mesh filename=/home/scottk/drc/ros_workspace/mit_drcsim_scripts/models/mi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 scale=1 1 1

File: software/models/mit_gazebo_models/mit_robot_drake/model_minimal_contact.urdf (robot description, URDF)
Before this commit: robot atlas, 29 links, 28 joints
Links:
- link head: geometry visual mesh filename=/home/scottk/drc/ros_workspace/mit_drcsim_scripts/models/mi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 scale=1 1 1
- link l_clav: geometry visual mesh filename=/home/scottk/drc/ros_workspace/mit_drcsim_scripts/models/mi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 scale=1 1 1
- link l_farm: geometry visual mesh filename=/home/scottk/drc/ros_workspace/mit_drcsim_scripts/models/mi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 scale=1 1 1
- link l_foot: geometry collision sphere radius=0; collision sphere radius=0
- link l_hand: geometry visual mesh filename=/home/scottk/drc/ros_workspace/mit_drcsim_scripts/models/mi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 scale=1 1 1
- link l_larm: geometry visual mesh filename=/home/scottk/drc/ros_workspace/mit_drcsim_scripts/models/mi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 scale=1 1 1
- link l_lglut: geometry visual mesh filename=/home/scottk/drc/ros_workspace/mit_drcsim_scripts/models/mi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 scale=1 1 1
- link l_lleg: geometry visual mesh filename=/home/scottk/drc/ros_workspace/mit_drcsim_scripts/models/mi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 scale=1 1 1
- link l_scap: geometry visual mesh filename=/home/scottk/drc/ros_workspace/mit_drcsim_scripts/models/mi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 scale=1 1 1
- link l_talus: geometry visual mesh filename=/home/scottk/drc/ros_workspace/mit_drcsim_scripts/models/mi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 scale=1 1 1
- link l_uarm: geometry visual mesh filename=/home/scottk/drc/ros_workspace/mit_drcsim_scripts/models/mi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 scale=1 1 1
- link l_uglut: geometry visual mesh filename=/home/scottk/drc/ros_workspace/mit_drcsim_scripts/models/mi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 scale=1 1 1
- link l_uleg: geometry visual mesh filename=/home/scottk/drc/ros_workspace/mit_drcsim_scripts/models/mi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 scale=1 1 1
- link ltorso: geometry visual mesh filename=/home/scottk/drc/ros_workspace/mit_drcsim_scripts/models/mi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 scale=1 1 1
- link mtorso: geometry visual mesh filename=/home/scottk/drc/ros_workspace/mit_drcsim_scripts/models/mi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 scale=1 1 1
- link pelvis: geometry visual mesh filename=/home/scottk/drc/ros_workspace/mit_drcsim_scripts/models/mi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 scale=1 1 1
- link r_clav: geometry visual mesh filename=/home/scottk/drc/ros_workspace/mit_drcsim_scripts/models/mi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 scale=1 1 1
- link r_farm: geometry visual mesh filename=/home/scottk/drc/ros_workspace/mit_drcsim_scripts/models/mi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 scale=1 1 1
- link r_foot: geometry collision sphere radius=0; collision sphere radius=0
- link r_hand: geometry visual mesh filename=/home/scottk/drc/ros_workspace/mit_drcsim_scripts/models/mi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 scale=1 1 1
- link r_larm: geometry visual mesh filename=/home/scottk/drc/ros_workspace/mit_drcsim_scripts/models/mi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 scale=1 1 1
- link r_lglut: geometry visual mesh filename=/home/scottk/drc/ros_workspace/mit_drcsim_scripts/models/mi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 scale=1 1 1
- link r_lleg: geometry visual mesh filename=/home/scottk/drc/ros_workspace/mit_drcsim_scripts/models/mi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 scale=1 1 1
- link r_scap: geometry visual mesh filename=/home/scottk/drc/ros_workspace/mit_drcsim_scripts/models/mi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 scale=1 1 1
- link r_talus: geometry visual mesh filename=/home/scottk/drc/ros_workspace/mit_drcsim_scripts/models/mi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 scale=1 1 1
- link r_uarm: geometry visual mesh filename=/home/scottk/drc/ros_workspace/mit_drcsim_scripts/models/mi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 scale=1 1 1
- link r_uglut: geometry visual mesh filename=/home/scottk/drc/ros_workspace/mit_drcsim_scripts/models/mi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 scale=1 1 1
- link r_uleg: geometry visual mesh filename=/home/scottk/drc/ros_workspace/mit_drcsim_scripts/models/mi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 scale=1 1 1
- link utorso: geometry visual mesh filename=/home/scottk/drc/ros_workspace/mit_drcsim_scripts/models/mi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 scale=1 1 1

Commit message: adding friction parameters for arms. updating hand point mass model for robot stumps
git-svn-id: https://svn.csail.mit.edu/drc/trunk@6309 c7283977-0100-402a-a91a-fa70b306dbfe

File: software/models/mit_gazebo_models/mit_robot_drake/model.urdf (robot description, URDF)
Before this commit: robot atlas, 95 links, 94 joints
Links:
- link l_clav: geometry collision mesh filename=package://mit_drcsim_scripts/models/mit_robot/meshes/l_clav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 scale=1 1 1; visual mesh filename=package://mit_drcsim_scripts/models/mit_robot/meshes/l_clav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 scale=1 1 1
- link l_farm: geometry collision mesh filename=package://mit_drcsim_scripts/models/mit_robot/meshes/l_farm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 scale=1 1 1; visual mesh filename=package://mit_drcsim_scripts/models/mit_robot/meshes/l_farm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 scale=1 1 1
- link l_foot: geometry collision box size=0.26 0.124887 0.05; collision sphere radius=0
- link l_hand: geometry collision mesh filename=package://mit_drcsim_scripts/models/mit_robot/meshes/l_hand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 scale=1 1 1; visual mesh filename=package://mit_drcsim_scripts/models/mit_robot/meshes/l_hand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 scale=1 1 1
- link l_larm: geometry collision mesh filename=package://mit_drcsim_scripts/models/mit_robot/meshes/l_elbo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 scale=1 1 1; visual mesh filename=package://mit_drcsim_scripts/models/mit_robot/meshes/l_elbo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 scale=1 1 1
- link l_lleg: geometry collision mesh filename=package://mit_drcsim_scripts/models/mit_robot/meshes/l_lleg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 scale=1 1 1; visual mesh filename=package://mit_drcsim_scripts/models/mit_robot/meshes/l_lleg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 scale=1 1 1
- link l_scap: geometry collision mesh filename=package://mit_drcsim_scripts/models/mit_robot/meshes/l_sh_r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 scale=1 1 1; visual mesh filename=package://mit_drcsim_scripts/models/mit_robot/meshes/l_sh_r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 scale=1 1 1
- link l_uarm: geometry collision mesh filename=package://mit_drcsim_scripts/models/mit_robot/meshes/l_elbo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 scale=1 1 1; visual mesh filename=package://mit_drcsim_scripts/models/mit_robot/meshes/l_elbo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 scale=1 1 1
- link l_uleg: geometry collision mesh filename=package://mit_drcsim_scripts/models/mit_robot/meshes/l_uleg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 scale=1 1 1; visual mesh filename=package://mit_drcsim_scripts/models/mit_robot/meshes/l_uleg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 scale=1 1 1
- link pelvis: geometry collision mesh filename=package://mit_drcsim_scripts/models/mit_robot/meshes/pelvis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 scale=1 1 1; visual mesh filename=package://mit_drcsim_scripts/models/mit_robot/meshes/pelvis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 scale=1 1 1
- link r_clav: geometry collision mesh filename=package://mit_drcsim_scripts/models/mit_robot/meshes/r_clav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 scale=1 1 1; visual mesh filename=package://mit_drcsim_scripts/models/mit_robot/meshes/r_clav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 scale=1 1 1
- link r_farm: geometry collision mesh filename=package://mit_drcsim_scripts/models/mit_robot/meshes/r_farm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 scale=1 1 1; visual mesh filename=package://mit_drcsim_scripts/models/mit_robot/meshes/r_farm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 scale=1 1 1
- link r_foot: geometry collision box size=0.26 0.124887 0.05; collision sphere radius=0
- link r_hand: geometry collision mesh filename=package://mit_drcsim_scripts/models/mit_robot/meshes/r_hand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 scale=1 1 1; visual mesh filename=package://mit_drcsim_scripts/models/mit_robot/meshes/r_hand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 scale=1 1 1
- link r_larm: geometry collision mesh filename=package://mit_drcsim_scripts/models/mit_robot/meshes/r_elbo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 scale=1 1 1; visual mesh filename=package://mit_drcsim_scripts/models/mit_robot/meshes/r_elbo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 scale=1 1 1
- link r_lleg: geometry collision mesh filename=package://mit_drcsim_scripts/models/mit_robot/meshes/r_lleg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 scale=1 1 1; visual mesh filename=package://mit_drcsim_scripts/models/mit_robot/meshes/r_lleg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 scale=1 1 1
- link r_scap: geometry collision mesh filename=package://mit_drcsim_scripts/models/mit_robot/meshes/r_sh_r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 scale=1 1 1; visual mesh filename=package://mit_drcsim_scripts/models/mit_robot/meshes/r_sh_r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 scale=1 1 1
- link r_uarm: geometry collision mesh filename=package://mit_drcsim_scripts/models/mit_robot/meshes/r_elbo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 scale=1 1 1; visual mesh filename=package://mit_drcsim_scripts/models/mit_robot/meshes/r_elbo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 scale=1 1 1
- link r_uleg: geometry collision mesh filename=package://mit_drcsim_scripts/models/mit_robot/meshes/r_uleg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 scale=1 1 1; visual mesh filename=package://mit_drcsim_scripts/models/mit_robot/meshes/r_uleg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 scale=1 1 1
- link utorso: geometry collision mesh filename=package://mit_drcsim_scripts/models/mit_robot/meshes/utorso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 scale=1 1 1; collision mesh filename=package://mit_drcsim_scripts/models/mit_robot/meshes/utorso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 scale=1 1 1
Joints:
- joint left_f0_j0: type fixed -> revolute
- joint left_f0_j1: type fixed -> revolute
- joint left_f0_j2: type fixed -> revolute
- joint left_f1_j0: type fixed -> revolute
- joint left_f1_j1: type fixed -> revolute
- joint left_f1_j2: type fixed -> revolute
- joint left_f2_j0: type fixed -> revolute
- joint left_f2_j1: type fixed -> revolute
- joint left_f2_j2: type fixed -> revolute
- joint left_f3_j0: type fixed -> revolute
- joint left_f3_j1: type fixed -> revolute
- joint left_f3_j2: type fixed -> revolute
- joint right_f0_j0: type fixed -> revolute
- joint right_f0_j1: type fixed -> revolute
- joint right_f0_j2: type fixed -> revolute
- joint right_f1_j0: type fixed -> revolute
- joint right_f1_j1: type fixed -> revolute
- joint right_f1_j2: type fixed -> revolute
- joint right_f2_j0: type fixed -> revolute
- joint right_f2_j1: type fixed -> revolute
- joint right_f2_j2: type fixed -> revolute
- joint right_f3_j0: type fixed -> revolute
- joint right_f3_j1: type fixed -> revolute
- joint right_f3_j2: type fixed -> revolute

File: software/models/mit_gazebo_models/mit_robot_drake/model_minimal_contact_point_hands.urdf (robot description, URDF)
Before this commit: robot atlas, 31 links, 30 joints
Links:
- link l_hand_point_mass: mass 3.131 -> 2.25
- link r_hand_point_mass: mass 3.131 -> 2.25
Joints:
- joint l_hand_joint: origin xyz=0.0037 0.1603 -0.0087 rpy=0 0 0 -> xyz=0.0 0.15 0.01 rpy=0 0 0
- joint r_hand_joint: origin xyz=0.0037 -0.1603 -0.0087 rpy=0 0 0 -> xyz=0.0 -0.15 0.01 rpy=0 0 0

File: software/models/mit_gazebo_models/mit_robot_drake/xacro/point_mass_hands.urdf (robot description, URDF)
Before this commit: robot drc_skeleton, 2 links, 2 joints
Links:
- link l_hand_point_mass: mass 3.131 -> 2.25
- link r_hand_point_mass: mass 3.131 -> 2.25
Joints:
- joint l_hand_joint: origin xyz=0.0037 0.1603 -0.0087 rpy=0 0 0 -> xyz=0.0 0.15 0.01 rpy=0 0 0
- joint r_hand_joint: origin xyz=0.0037 -0.1603 -0.0087 rpy=0 0 0 -> xyz=0.0 -0.15 0.01 rpy=0 0 0

Commit message: small changes to leg friction
git-svn-id: https://svn.csail.mit.edu/drc/trunk@6615 c7283977-0100-402a-a91a-fa70b306dbfe

File: software/models/mit_gazebo_models/mit_robot_drake/model.urdf (robot description, URDF)
Before this commit: robot atlas, 95 links, 94 joints
Joints:
- joint r_leg_kny: limit lower=0 upper=2.38569 effort=220 velocity=12 -> lower=0 upper=2.38569 effort=220 velocity=11

File: software/models/mit_gazebo_models/mit_robot_drake/model_minimal_contact.urdf (robot description, URDF)
Before this commit: robot atlas, 29 links, 28 joints
Links:
- link utorso: mass 52.007 -> 60
Joints:
- joint r_leg_kny: limit lower=0 upper=2.38569 effort=220 velocity=12 -> lower=0 upper=2.38569 effort=220 velocity=11

File: software/models/mit_gazebo_models/mit_robot_drake/model_minimal_contact_fixedjoint_hands.urdf (robot description, URDF)
Before this commit: robot atlas, 95 links, 94 joints
Links:
- link utorso: mass 52.007 -> 60
Joints:
- joint r_leg_kny: limit lower=0 upper=2.38569 effort=220 velocity=12 -> lower=0 upper=2.38569 effort=220 velocity=11

File: software/models/mit_gazebo_models/mit_robot_drake/model_minimal_contact_point_hands.urdf (robot description, URDF)
Before this commit: robot atlas, 31 links, 30 joints
Links:
- link utorso: mass 52.007 -> 60
Joints:
- joint r_leg_kny: limit lower=0 upper=2.38569 effort=220 velocity=12 -> lower=0 upper=2.38569 effort=220 velocity=11

File: software/models/mit_gazebo_models/mit_robot_drake/model_minimal_contact_point_stumps.urdf (robot description, URDF)
Before this commit: robot atlas, 31 links, 30 joints
Links:
- link utorso: mass 52.007 -> 60
Joints:
- joint r_leg_kny: limit lower=0 upper=2.38569 effort=220 velocity=12 -> lower=0 upper=2.38569 effort=220 velocity=11

File: software/models/mit_gazebo_models/mit_robot_drake/xacro/atlas_skeleton.urdf (robot description, URDF)
Before this commit: robot drc_skeleton, 28 links, 28 joints
Joints:
- joint r_leg_kny: limit lower=0 upper=2.38569 effort=220 velocity=12 -> lower=0 upper=2.38569 effort=220 velocity=11

File: software/models/mit_gazebo_models/mit_robot_drake/xacro/atlas_skeleton_minimal_contact.urdf (robot description, URDF)
Before this commit: robot drc_skeleton, 28 links, 28 joints
Links:
- link utorso: mass 52.007 -> 60
Joints:
- joint r_leg_kny: limit lower=0 upper=2.38569 effort=220 velocity=12 -> lower=0 upper=2.38569 effort=220 velocity=11
