Commit message: more reasonable input limits for the legs

File: software/models/mit_gazebo_models/mit_robot_drake/model.urdf (robot description, URDF)
Before this commit: robot atlas, 29 links, 28 joints
Joints:
- joint l_leg_akx: limit lower=-0.8 upper=0.8 effort=90 velocity=12 -> lower=-0.8 upper=0.8 effort=130 velocity=12
- joint l_leg_aky: limit lower=-1 upper=0.7 effort=700 velocity=12 -> lower=-1 upper=0.7 effort=350 velocity=12
- joint l_leg_hpx: limit lower=-0.523599 upper=0.523599 effort=180 velocity=12 -> lower=-0.523599 upper=0.523599 effort=250 velocity=12
- joint l_leg_hpz: limit lower=-0.174533 upper=1.22173 effort=110 velocity=12 -> lower=-0.174533 upper=1.22173 effort=68 velocity=12
- joint r_leg_akx: limit lower=-0.8 upper=0.8 effort=90 velocity=12 -> lower=-0.8 upper=0.8 effort=130 velocity=12
- joint r_leg_aky: limit lower=-1 upper=0.7 effort=700 velocity=12 -> lower=-1 upper=0.7 effort=350 velocity=12
- joint r_leg_hpx: limit lower=-0.523599 upper=0.523599 effort=180 velocity=12 -> lower=-0.523599 upper=0.523599 effort=250 velocity=12
- joint r_leg_hpz: limit lower=-1.22173 upper=0.174533 effort=110 velocity=12 -> lower=-1.22173 upper=0.174533 effort=68 velocity=12
- joint r_leg_kny: limit lower=0 upper=2.38569 effort=220 velocity=11 -> lower=0 upper=2.38569 effort=220 velocity=12

File: software/models/mit_gazebo_models/mit_robot_drake/model_minimal_contact.urdf (robot description, URDF)
Before this commit: robot atlas, 29 links, 28 joints
Joints:
- joint l_leg_akx: limit lower=-0.8 upper=0.8 effort=90 velocity=12 -> lower=-0.8 upper=0.8 effort=130 velocity=12
- joint l_leg_aky: limit lower=-1 upper=0.7 effort=700 velocity=12 -> lower=-1 upper=0.7 effort=350 velocity=12
- joint l_leg_hpx: limit lower=-0.523599 upper=0.523599 effort=180 velocity=12 -> lower=-0.523599 upper=0.523599 effort=250 velocity=12
- joint l_leg_hpz: limit lower=-0.174533 upper=1.22173 effort=110 velocity=12 -> lower=-0.174533 upper=1.22173 effort=68 velocity=12
- joint r_leg_akx: limit lower=-0.8 upper=0.8 effort=90 velocity=12 -> lower=-0.8 upper=0.8 effort=130 velocity=12
- joint r_leg_aky: limit lower=-1 upper=0.7 effort=700 velocity=12 -> lower=-1 upper=0.7 effort=350 velocity=12
- joint r_leg_hpx: limit lower=-0.523599 upper=0.523599 effort=180 velocity=12 -> lower=-0.523599 upper=0.523599 effort=250 velocity=12
- joint r_leg_hpz: limit lower=-1.22173 upper=0.174533 effort=110 velocity=12 -> lower=-1.22173 upper=0.174533 effort=68 velocity=12
- joint r_leg_kny: limit lower=0 upper=2.38569 effort=220 velocity=11 -> lower=0 upper=2.38569 effort=220 velocity=12

File: software/models/mit_gazebo_models/mit_robot_drake/model_minimal_contact_fixedjoint_hands.urdf (robot description, URDF)
Before this commit: robot atlas, 95 links, 94 joints
Joints:
- joint l_leg_akx: limit lower=-0.8 upper=0.8 effort=90 velocity=12 -> lower=-0.8 upper=0.8 effort=130 velocity=12
- joint l_leg_aky: limit lower=-1 upper=0.7 effort=700 velocity=12 -> lower=-1 upper=0.7 effort=350 velocity=12
- joint l_leg_hpx: limit lower=-0.523599 upper=0.523599 effort=180 velocity=12 -> lower=-0.523599 upper=0.523599 effort=250 velocity=12
- joint l_leg_hpz: limit lower=-0.174533 upper=1.22173 effort=110 velocity=12 -> lower=-0.174533 upper=1.22173 effort=68 velocity=12
- joint r_leg_akx: limit lower=-0.8 upper=0.8 effort=90 velocity=12 -> lower=-0.8 upper=0.8 effort=130 velocity=12
- joint r_leg_aky: limit lower=-1 upper=0.7 effort=700 velocity=12 -> lower=-1 upper=0.7 effort=350 velocity=12
- joint r_leg_hpx: limit lower=-0.523599 upper=0.523599 effort=180 velocity=12 -> lower=-0.523599 upper=0.523599 effort=250 velocity=12
- joint r_leg_hpz: limit lower=-1.22173 upper=0.174533 effort=110 velocity=12 -> lower=-1.22173 upper=0.174533 effort=68 velocity=12
- joint r_leg_kny: limit lower=0 upper=2.38569 effort=220 velocity=11 -> lower=0 upper=2.38569 effort=220 velocity=12

File: software/models/mit_gazebo_models/mit_robot_drake/model_minimal_contact_point_hands.urdf (robot description, URDF)
Before this commit: robot atlas, 31 links, 30 joints
Joints:
- joint l_leg_akx: limit lower=-0.8 upper=0.8 effort=90 velocity=12 -> lower=-0.8 upper=0.8 effort=130 velocity=12
- joint l_leg_aky: limit lower=-1 upper=0.7 effort=700 velocity=12 -> lower=-1 upper=0.7 effort=350 velocity=12
- joint l_leg_hpx: limit lower=-0.523599 upper=0.523599 effort=180 velocity=12 -> lower=-0.523599 upper=0.523599 effort=250 velocity=12
- joint l_leg_hpz: limit lower=-0.174533 upper=1.22173 effort=110 velocity=12 -> lower=-0.174533 upper=1.22173 effort=68 velocity=12
- joint r_leg_akx: limit lower=-0.8 upper=0.8 effort=90 velocity=12 -> lower=-0.8 upper=0.8 effort=130 velocity=12
- joint r_leg_aky: limit lower=-1 upper=0.7 effort=700 velocity=12 -> lower=-1 upper=0.7 effort=350 velocity=12
- joint r_leg_hpx: limit lower=-0.523599 upper=0.523599 effort=180 velocity=12 -> lower=-0.523599 upper=0.523599 effort=250 velocity=12
- joint r_leg_hpz: limit lower=-1.22173 upper=0.174533 effort=110 velocity=12 -> lower=-1.22173 upper=0.174533 effort=68 velocity=12
- joint r_leg_kny: limit lower=0 upper=2.38569 effort=220 velocity=11 -> lower=0 upper=2.38569 effort=220 velocity=12

File: software/models/mit_gazebo_models/mit_robot_drake/model_minimal_contact_point_stumps.urdf (robot description, URDF)
Before this commit: robot atlas, 31 links, 30 joints
Joints:
- joint l_leg_akx: limit lower=-0.8 upper=0.8 effort=90 velocity=12 -> lower=-0.8 upper=0.8 effort=130 velocity=12
- joint l_leg_aky: limit lower=-1 upper=0.7 effort=700 velocity=12 -> lower=-1 upper=0.7 effort=350 velocity=12
- joint l_leg_hpx: limit lower=-0.523599 upper=0.523599 effort=180 velocity=12 -> lower=-0.523599 upper=0.523599 effort=250 velocity=12
- joint l_leg_hpz: limit lower=-0.174533 upper=1.22173 effort=110 velocity=12 -> lower=-0.174533 upper=1.22173 effort=68 velocity=12
- joint r_leg_akx: limit lower=-0.8 upper=0.8 effort=90 velocity=12 -> lower=-0.8 upper=0.8 effort=130 velocity=12
- joint r_leg_aky: limit lower=-1 upper=0.7 effort=700 velocity=12 -> lower=-1 upper=0.7 effort=350 velocity=12
- joint r_leg_hpx: limit lower=-0.523599 upper=0.523599 effort=180 velocity=12 -> lower=-0.523599 upper=0.523599 effort=250 velocity=12
- joint r_leg_hpz: limit lower=-1.22173 upper=0.174533 effort=110 velocity=12 -> lower=-1.22173 upper=0.174533 effort=68 velocity=12
- joint r_leg_kny: limit lower=0 upper=2.38569 effort=220 velocity=11 -> lower=0 upper=2.38569 effort=220 velocity=12

File: software/models/mit_gazebo_models/mit_robot_drake/xacro/atlas_skeleton.urdf (robot description, URDF)
Before this commit: robot drc_skeleton, 28 links, 28 joints
Joints:
- joint l_leg_akx: limit lower=-0.8 upper=0.8 effort=90 velocity=12 -> lower=-0.8 upper=0.8 effort=130 velocity=12
- joint l_leg_aky: limit lower=-1 upper=0.7 effort=700 velocity=12 -> lower=-1 upper=0.7 effort=350 velocity=12
- joint l_leg_hpx: limit lower=-0.523599 upper=0.523599 effort=180 velocity=12 -> lower=-0.523599 upper=0.523599 effort=250 velocity=12
- joint l_leg_hpz: limit lower=-0.174533 upper=1.22173 effort=110 velocity=12 -> lower=-0.174533 upper=1.22173 effort=68 velocity=12
- joint r_leg_akx: limit lower=-0.8 upper=0.8 effort=90 velocity=12 -> lower=-0.8 upper=0.8 effort=130 velocity=12
- joint r_leg_aky: limit lower=-1 upper=0.7 effort=700 velocity=12 -> lower=-1 upper=0.7 effort=350 velocity=12
- joint r_leg_hpx: limit lower=-0.523599 upper=0.523599 effort=180 velocity=12 -> lower=-0.523599 upper=0.523599 effort=250 velocity=12
- joint r_leg_hpz: limit lower=-1.22173 upper=0.174533 effort=110 velocity=12 -> lower=-1.22173 upper=0.174533 effort=68 velocity=12
- joint r_leg_kny: limit lower=0 upper=2.38569 effort=220 velocity=11 -> lower=0 upper=2.38569 effort=220 velocity=12

File: software/models/mit_gazebo_models/mit_robot_drake/xacro/atlas_skeleton_minimal_contact.urdf (robot description, URDF)
Before this commit: robot drc_skeleton, 28 links, 28 joints
Joints:
- joint l_leg_akx: limit lower=-0.8 upper=0.8 effort=90 velocity=12 -> lower=-0.8 upper=0.8 effort=130 velocity=12
- joint l_leg_aky: limit lower=-1 upper=0.7 effort=700 velocity=12 -> lower=-1 upper=0.7 effort=350 velocity=12
- joint l_leg_hpx: limit lower=-0.523599 upper=0.523599 effort=180 velocity=12 -> lower=-0.523599 upper=0.523599 effort=250 velocity=12
- joint l_leg_hpz: limit lower=-0.174533 upper=1.22173 effort=110 velocity=12 -> lower=-0.174533 upper=1.22173 effort=68 velocity=12
- joint r_leg_akx: limit lower=-0.8 upper=0.8 effort=90 velocity=12 -> lower=-0.8 upper=0.8 effort=130 velocity=12
- joint r_leg_aky: limit lower=-1 upper=0.7 effort=700 velocity=12 -> lower=-1 upper=0.7 effort=350 velocity=12
- joint r_leg_hpx: limit lower=-0.523599 upper=0.523599 effort=180 velocity=12 -> lower=-0.523599 upper=0.523599 effort=250 velocity=12
- joint r_leg_hpz: limit lower=-1.22173 upper=0.174533 effort=110 velocity=12 -> lower=-1.22173 upper=0.174533 effort=68 velocity=12
- joint r_leg_kny: limit lower=0 upper=2.38569 effort=220 velocity=11 -> lower=0 upper=2.38569 effort=220 velocity=12

Commit message: Decrease number of faces in Atlas chull meshes.
Also remove hands and replace foot boxes with foot meshes in the Atlas chull
urdf (mit_robot_drake/model.urdf)

File: software/models/mit_gazebo_models/mit_robot_drake/model.urdf (robot description, URDF)
Before this commit: robot atlas, 95 links, 94 joints
Links:
- removed link left_f0_0
- removed link left_f0_1
- removed link left_f0_1_accel
- removed link left_f0_2
- removed link left_f0_2_accel
- removed link left_f0_base
- removed link left_f0_fixed_accel
- removed link left_f1_0
- removed link left_f1_1
- removed link left_f1_1_accel
- removed link left_f1_2
- removed link left_f1_2_accel
- removed link left_f1_base
- removed link left_f1_fixed_accel
- removed link left_f2_0
- removed link left_f2_1
- removed link left_f2_1_accel
- removed link left_f2_2
- removed link left_f2_2_accel
- removed link left_f2_base
- removed link left_f2_fixed_accel
- removed link left_f3_0
- removed link left_f3_1
- removed link left_f3_1_accel
- removed link left_f3_2
- removed link left_f3_2_accel
- removed link left_f3_base
- removed link left_f3_fixed_accel
- removed link left_palm
- removed link left_palm_left_camera_frame
- removed link left_palm_left_camera_optical_frame
- removed link left_palm_right_camera_frame
- removed link left_palm_right_camera_optical_frame
- removed link right_f0_0
- removed link right_f0_1
- removed link right_f0_1_accel
- removed link right_f0_2
- removed link right_f0_2_accel
- removed link right_f0_base
- removed link right_f0_fixed_accel
- removed link right_f1_0
- removed link right_f1_1
- removed link right_f1_1_accel
- removed link right_f1_2
- removed link right_f1_2_accel
- removed link right_f1_base
- removed link right_f1_fixed_accel
- removed link right_f2_0
- removed link right_f2_1
- removed link right_f2_1_accel
- removed link right_f2_2
- removed link right_f2_2_accel
- removed link right_f2_base
- removed link right_f2_fixed_accel
- removed link right_f3_0
- removed link right_f3_1
- removed link right_f3_1_accel
- removed link right_f3_2
- removed link right_f3_2_accel
- removed link right_f3_base
- removed link right_f3_fixed_accel
- removed link right_palm
- removed link right_palm_left_camera_frame
- removed link right_palm_left_camera_optical_frame
- removed link right_palm_right_camera_frame
- removed link right_palm_right_camera_optical_frame
- link l_foot: geometry collision mesh filename=package://mit_drcsim_scripts/models/mit_robot/meshes/l_foot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 scale=1 1 1; visual mesh filename=package://mit_drcsim_scripts/models/mit_robot/meshes/l_foot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 scale=1 1 1
- link r_foot: geometry collision mesh filename=package://mit_drcsim_scripts/models/mit_robot/meshes/r_foot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 scale=1 1 1; visual mesh filename=package://mit_drcsim_scripts/models/mit_robot/meshes/r_foot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 scale=1 1 1
Joints:
- removed joint left_f0_1_accel
- removed joint left_f0_2_accel
- removed joint left_f0_base
- removed joint left_f0_fixed_accel
- removed joint left_f0_j0
- removed joint left_f0_j1
- removed joint left_f0_j2
- removed joint left_f1_1_accel
- removed joint left_f1_2_accel
- removed joint left_f1_base
- removed joint left_f1_fixed_accel
- removed joint left_f1_j0
- removed joint left_f1_j1
- removed joint left_f1_j2
- removed joint left_f2_1_accel
- removed joint left_f2_2_accel
- removed joint left_f2_base
- removed joint left_f2_fixed_accel
- removed joint left_f2_j0
- removed joint left_f2_j1
- removed joint left_f2_j2
- removed joint left_f3_1_accel
- removed joint left_f3_2_accel
- removed joint left_f3_base
- removed joint left_f3_fixed_accel
- removed joint left_f3_j0
- removed joint left_f3_j1
- removed joint left_f3_j2
- removed joint left_palm_left_camera_frame_joint
- removed joint left_palm_left_camera_optical_frame_joint
- removed joint left_palm_right_camera_frame_joint
- removed joint left_palm_right_camera_optical_frame_joint
- removed joint left_sandia_hand_joint
- removed joint right_f0_1_accel
- removed joint right_f0_2_accel
- removed joint right_f0_base
- removed joint right_f0_fixed_accel
- removed joint right_f0_j0
- removed joint right_f0_j1
- removed joint right_f0_j2
- removed joint right_f1_1_accel
- removed joint right_f1_2_accel
- removed joint right_f1_base
- removed joint right_f1_fixed_accel
- removed joint right_f1_j0
- removed joint right_f1_j1
- removed joint right_f1_j2
- removed joint right_f2_1_accel
- removed joint right_f2_2_accel
- removed joint right_f2_base
- removed joint right_f2_fixed_accel
- removed joint right_f2_j0
- removed joint right_f2_j1
- removed joint right_f2_j2
- removed joint right_f3_1_accel
- removed joint right_f3_2_accel
- removed joint right_f3_base
- removed joint right_f3_fixed_accel
- removed joint right_f3_j0
- removed joint right_f3_j1
- removed joint right_f3_j2
- removed joint right_palm_left_camera_frame_joint
- removed joint right_palm_left_camera_optical_frame_joint
- removed joint right_palm_right_camera_frame_joint
- removed joint right_palm_right_camera_optical_frame_joint
- removed joint right_sandia_hand_joint

File: software/models/mit_gazebo_models/mit_robot_drake/xacro/atlas_skeleton.urdf (robot description, URDF)
Before this commit: robot drc_skeleton, 28 links, 28 joints
Links:
- link l_foot: geometry collision mesh filename=package://mit_drcsim_scripts/models/mit_robot/meshes/l_foot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 scale=1 1 1; visual mesh filename=package://mit_drcsim_scripts/models/mit_robot/meshes/l_foot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 scale=1 1 1
- link r_foot: geometry collision mesh filename=package://mit_drcsim_scripts/models/mit_robot/meshes/r_foot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 scale=1 1 1; visual mesh filename=package://mit_drcsim_scripts/models/mit_robot/meshes/r_foot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 scale=1 1 1

Commit message: utorso mass retweak

File: software/models/mit_gazebo_models/mit_robot_drake/model.urdf (robot description, URDF)
Before this commit: robot atlas, 29 links, 28 joints
Links:
- link utorso: mass 52.007 -> 52

File: software/models/mit_gazebo_models/mit_robot_drake/xacro/atlas_skeleton.urdf (robot description, URDF)
Before this commit: robot drc_skeleton, 28 links, 28 joints
Links:
- link utorso: mass 52.007 -> 52
