Commit message: Add updated urdfs to mit_robot_drake

File: software/models/mit_gazebo_models/mit_robot_drake/model_convex_hull_no_hands.urdf (robot description, URDF)
Before this commit: robot atlas, 31 links, 30 joints
Links:
- removed link l_hand_point_mass
- removed link r_hand_point_mass
- link l_clav: geometry collision mesh filename=package://mit_drcsim_scripts/models/mit_robot/meshes/l_clav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 scale=1 1 1; visual mesh filename=package://mit_drcsim_scripts/models/mit_robot/meshes/l_clav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 scale=1 1 1
- link l_farm: geometry collision mesh filename=package://mit_drcsim_scripts/models/mit_robot/meshes/l_farm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 scale=1 1 1; visual mesh filename=package://mit_drcsim_scripts/models/mit_robot/meshes/l_farm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 scale=1 1 1
- link l_foot: geometry collision mesh filename=package://mit_drcsim_scripts/models/mit_robot/meshes/l_foot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 scale=1 1 1; collision sphere radius=0
- link l_hand: geometry collision mesh filename=package://mit_drcsim_scripts/models/mit_robot/meshes/l_hand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 scale=1 1 1; visual mesh filename=package://mit_drcsim_scripts/models/mit_robot/meshes/l_hand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 scale=1 1 1
- link l_larm: geometry collision mesh filename=package://mit_drcsim_scripts/models/mit_robot/meshes/l_elbo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 scale=1 1 1; visual mesh filename=package://mit_drcsim_scripts/models/mit_robot/meshes/l_elbo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 scale=1 1 1
- link l_lglut: geometry 
- link l_lleg: geometry collision mesh filename=package://mit_drcsim_scripts/models/mit_robot/meshes/l_lleg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 scale=1 1 1; visual mesh filename=package://mit_drcsim_scripts/models/mit_robot/meshes/l_lleg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 scale=1 1 1
- link l_scap: geometry collision mesh filename=package://mit_drcsim_scripts/models/mit_robot/meshes/l_sh_r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 scale=1 1 1; visual mesh filename=package://mit_drcsim_scripts/models/mit_robot/meshes/l_sh_r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 scale=1 1 1
- link l_talus: geometry 
- link l_uarm: geometry collision mesh filename=package://mit_drcsim_scripts/models/mit_robot/meshes/l_elbo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 scale=1 1 1; visual mesh filename=package://mit_drcsim_scripts/models/mit_robot/meshes/l_elbo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 scale=1 1 1
- link l_uglut: geometry 
- link l_uleg: geometry collision mesh filename=package://mit_drcsim_scripts/models/mit_robot/meshes/l_uleg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 scale=1 1 1; visual mesh filename=package://mit_drcsim_scripts/models/mit_robot/meshes/l_uleg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 scale=1 1 1
- link ltorso: geometry 
- link pelvis: geometry collision mesh filename=package://mit_drcsim_scripts/models/mit_robot/meshes/pelvis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 scale=1 1 1; visual mesh filename=package://mit_drcsim_scripts/models/mit_robot/meshes/pelvis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 scale=1 1 1
- link r_clav: geometry collision mesh filename=package://mit_drcsim_scripts/models/mit_robot/meshes/r_clav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 scale=1 1 1; visual mesh filename=package://mit_drcsim_scripts/models/mit_robot/meshes/r_clav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 scale=1 1 1
- link r_farm: geometry collision mesh filename=package://mit_drcsim_scripts/models/mit_robot/meshes/r_farm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 scale=1 1 1; visual mesh filename=package://mit_drcsim_scripts/models/mit_robot/meshes/r_farm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 scale=1 1 1
- link r_foot: geometry collision mesh filename=package://mit_drcsim_scripts/models/mit_robot/meshes/r_foot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 scale=1 1 1; collision sphere radius=0
- link r_hand: geometry collision mesh filename=package://mit_drcsim_scripts/models/mit_robot/meshes/r_hand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 scale=1 1 1; visual mesh filename=package://mit_drcsim_scripts/models/mit_robot/meshes/r_hand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 scale=1 1 1
- link r_larm: geometry collision mesh filename=package://mit_drcsim_scripts/models/mit_robot/meshes/r_elbo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 scale=1 1 1; visual mesh filename=package://mit_drcsim_scripts/models/mit_robot/meshes/r_elbo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 scale=1 1 1
- link r_lglut: geometry 
- link r_lleg: geometry collision mesh filename=package://mit_drcsim_scripts/models/mit_robot/meshes/r_lleg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 scale=1 1 1; visual mesh filename=package://mit_drcsim_scripts/models/mit_robot/meshes/r_lleg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 scale=1 1 1
- link r_scap: geometry collision mesh filename=package://mit_drcsim_scripts/models/mit_robot/meshes/r_sh_r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 scale=1 1 1; visual mesh filename=package://mit_drcsim_scripts/models/mit_robot/meshes/r_sh_r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 scale=1 1 1
- link r_talus: geometry 
- link r_uarm: geometry collision mesh filename=package://mit_drcsim_scripts/models/mit_robot/meshes/r_elbo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 scale=1 1 1; visual mesh filename=package://mit_drcsim_scripts/models/mit_robot/meshes/r_elbo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 scale=1 1 1
- link r_uglut: geometry 
- link r_uleg: geometry collision mesh filename=package://mit_drcsim_scripts/models/mit_robot/meshes/r_uleg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 scale=1 1 1; visual mesh filename=package://mit_drcsim_scripts/models/mit_robot/meshes/r_uleg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 scale=1 1 1
- link utorso: geometry collision mesh filename=package://mit_drcsim_scripts/models/mit_robot/meshes/utorso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 scale=1 1 1; collision mesh filename=package://mit_drcsim_scripts/models/mit_robot/meshes/utorso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 scale=1 1 1
Joints:
- removed joint l_hand_joint
- removed joint r_hand_joint

File: software/models/mit_gazebo_models/mit_robot_drake/model_convex_hull_robotiq_hands.urdf (robot description, URDF)
Before this commit: robot atlas, 31 links, 30 joints
Links:
- added link l_robotiq_convex_hull; collision mesh filename=package://mit_drcsim_scripts/models/mit_robot/meshes/GRIPPE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 scale=1 1 1; visual mesh filename=package://mit_drcsim_scripts/models/mit_robot/meshes/GRIPPE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 scale=1 1 1
- added link r_robotiq_convex_hull; collision mesh filename=package://mit_drcsim_scripts/models/mit_robot/meshes/GRIPPE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 scale=1 1 1; visual mesh filename=package://mit_drcsim_scripts/models/mit_robot/meshes/GRIPPE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 scale=1 1 1
- link l_clav: geometry collision mesh filename=package://mit_drcsim_scripts/models/mit_robot/meshes/l_clav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 scale=1 1 1; visual mesh filename=package://mit_drcsim_scripts/models/mit_robot/meshes/l_clav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 scale=1 1 1
- link l_farm: geometry collision mesh filename=package://mit_drcsim_scripts/models/mit_robot/meshes/l_farm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 scale=1 1 1; visual mesh filename=package://mit_drcsim_scripts/models/mit_robot/meshes/l_farm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 scale=1 1 1
- link l_foot: geometry collision mesh filename=package://mit_drcsim_scripts/models/mit_robot/meshes/l_foot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 scale=1 1 1; collision sphere radius=0
- link l_hand: geometry collision mesh filename=package://mit_drcsim_scripts/models/mit_robot/meshes/l_hand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 scale=1 1 1; visual mesh filename=package://mit_drcsim_scripts/models/mit_robot/meshes/l_hand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 scale=1 1 1
- link l_hand_point_mass: mass 2.25 -> 5.131
- link l_larm: geometry collision mesh filename=package://mit_drcsim_scripts/models/mit_robot/meshes/l_elbo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 scale=1 1 1; visual mesh filename=package://mit_drcsim_scripts/models/mit_robot/meshes/l_elbo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 scale=1 1 1
- link l_lglut: geometry 
- link l_lleg: geometry collision mesh filename=package://mit_drcsim_scripts/models/mit_robot/meshes/l_lleg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 scale=1 1 1; visual mesh filename=package://mit_drcsim_scripts/models/mit_robot/meshes/l_lleg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 scale=1 1 1
- link l_scap: geometry collision mesh filename=package://mit_drcsim_scripts/models/mit_robot/meshes/l_sh_r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 scale=1 1 1; visual mesh filename=package://mit_drcsim_scripts/models/mit_robot/meshes/l_sh_r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 scale=1 1 1
- link l_talus: geometry 
- link l_uarm: geometry collision mesh filename=package://mit_drcsim_scripts/models/mit_robot/meshes/l_elbo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 scale=1 1 1; visual mesh filename=package://mit_drcsim_scripts/models/mit_robot/meshes/l_elbo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 scale=1 1 1
- link l_uglut: geometry 
- link l_uleg: geometry collision mesh filename=package://mit_drcsim_scripts/models/mit_robot/meshes/l_uleg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 scale=1 1 1; visual mesh filename=package://mit_drcsim_scripts/models/mit_robot/meshes/l_uleg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 scale=1 1 1
- link ltorso: geometry 
- link pelvis: geometry collision mesh filename=package://mit_drcsim_scripts/models/mit_robot/meshes/pelvis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 scale=1 1 1; visual mesh filename=package://mit_drcsim_scripts/models/mit_robot/meshes/pelvis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 scale=1 1 1
- link r_clav: geometry collision mesh filename=package://mit_drcsim_scripts/models/mit_robot/meshes/r_clav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 scale=1 1 1; visual mesh filename=package://mit_drcsim_scripts/models/mit_robot/meshes/r_clav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 scale=1 1 1
- link r_farm: geometry collision mesh filename=package://mit_drcsim_scripts/models/mit_robot/meshes/r_farm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 scale=1 1 1; visual mesh filename=package://mit_drcsim_scripts/models/mit_robot/meshes/r_farm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 scale=1 1 1
- link r_foot: geometry collision mesh filename=package://mit_drcsim_scripts/models/mit_robot/meshes/r_foot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 scale=1 1 1; collision sphere radius=0
- link r_hand: geometry collision mesh filename=package://mit_drcsim_scripts/models/mit_robot/meshes/r_hand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 scale=1 1 1; visual mesh filename=package://mit_drcsim_scripts/models/mit_robot/meshes/r_hand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 scale=1 1 1
- link r_hand_point_mass: mass 2.25 -> 5.131
- link r_larm: geometry collision mesh filename=package://mit_drcsim_scripts/models/mit_robot/meshes/r_elbo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 scale=1 1 1; visual mesh filename=package://mit_drcsim_scripts/models/mit_robot/meshes/r_elbo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 scale=1 1 1
- link r_lglut: geometry 
- link r_lleg: geometry collision mesh filename=package://mit_drcsim_scripts/models/mit_robot/meshes/r_lleg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 scale=1 1 1; visual mesh filename=package://mit_drcsim_scripts/models/mit_robot/meshes/r_lleg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 scale=1 1 1
- link r_scap: geometry collision mesh filename=package://mit_drcsim_scripts/models/mit_robot/meshes/r_sh_r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 scale=1 1 1; visual mesh filename=package://mit_drcsim_scripts/models/mit_robot/meshes/r_sh_r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 scale=1 1 1
- link r_talus: geometry 
- link r_uarm: geometry collision mesh filename=package://mit_drcsim_scripts/models/mit_robot/meshes/r_elbo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 scale=1 1 1; visual mesh filename=package://mit_drcsim_scripts/models/mit_robot/meshes/r_elbo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 scale=1 1 1
- link r_uglut: geometry 
- link r_uleg: geometry collision mesh filename=package://mit_drcsim_scripts/models/mit_robot/meshes/r_uleg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 scale=1 1 1; visual mesh filename=package://mit_drcsim_scripts/models/mit_robot/meshes/r_uleg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 scale=1 1 1
- link utorso: geometry collision mesh filename=package://mit_drcsim_scripts/models/mit_robot/meshes/utorso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 scale=1 1 1; collision mesh filename=package://mit_drcsim_scripts/models/mit_robot/meshes/utorso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 scale=1 1 1
Joints:
- added joint l_robotiq_convex_hull_joint: type fixed, parent l_hand, child l_robotiq_convex_hull
- added joint r_robotiq_convex_hull_joint: type fixed, parent r_hand, child r_robotiq_convex_hull
- joint l_hand_joint: origin xyz=0.0 0.15 0.01 rpy=0 0 0 -> xyz=-0.0037 0.1603 0.0087 rpy=0 0 0
- joint r_hand_joint: origin xyz=0.0 -0.15 0.01 rpy=0 0 0 -> xyz=0.0037 -0.1603 -0.0087 rpy=0 0 0
