Commit message: cleaned up drake models a bit
git-svn-id: https://svn.csail.mit.edu/drc@2792 c7283977-0100-402a-a91a-fa70b306dbfe

File: software/models/mit_gazebo_models/mit_robot_drake/model_minimal_contact_point_hands.urdf (robot description, URDF)
Before this commit: robot atlas, 31 links, 30 joints
Links:
- link l_foot: mass 0.817 -> 0.867
- link l_lglut: mass 0.69 -> 0.803
- link l_talus: mass 0.817 -> 0.867
- link l_uglut: mass 0.5166 -> 1.51622
- link l_uleg: mass 7.34 -> 7.227
- link ltorso: mass 1.92 -> 1.62729
- link mtorso: mass 0.55 -> 3.8068
- link pelvis: mass 14.2529 -> 12.54638
- link r_foot: mass 0.817 -> 0.867
- link r_lglut: mass 0.69 -> 0.803
- link r_talus: mass 0.817 -> 0.867
- link r_uglut: mass 0.5166 -> 1.51622
- link r_uleg: mass 7.34 -> 7.227
- link utorso: mass 18.484 -> 15.2272

File: software/models/mit_gazebo_models/mit_robot_drake/xacro/atlas.urdf.xacro (robot description, xacro)
@@ -1,5 +1,4 @@
 <robot name="atlas" >
   <include filename="$(find mit_drcsim_scripts)/models/mit_robot_drake/xacro/atlas_skeleton_minimal_contact.urdf" />
-<!--  <include filename="$(find mit_drcsim_scripts)/models/mit_robot_drake/xacro/point_mass_hands.urdf" />-->
   <include filename="$(find mit_drcsim_scripts)/models/mit_robot_drake/xacro/atlas.transmission" />
   <include filename="$(find mit_drcsim_scripts)/models/mit_robot_drake/xacro/multisense_sl_no_contact.urdf" />

File: software/models/mit_gazebo_models/mit_robot_drake/xacro/atlas_point_hands.urdf.xacro (robot description, xacro)
@@ -1,5 +1,5 @@
 <robot name="atlas" >
   <include filename="$(find mit_drcsim_scripts)/models/mit_robot_drake/xacro/atlas_skeleton_minimal_contact.urdf" />
-  <include filename="$(find mit_drcsim_scripts)/models/mit_robot_drake/xacro/point_mass_hands_march.urdf" />
+  <include filename="$(find mit_drcsim_scripts)/models/mit_robot_drake/xacro/point_mass_hands.urdf" />
   <include filename="$(find mit_drcsim_scripts)/models/mit_robot_drake/xacro/atlas.transmission" />
   <include filename="$(find mit_drcsim_scripts)/models/mit_robot_drake/xacro/multisense_sl_no_contact.urdf" />

File: software/models/mit_gazebo_models/mit_robot_drake/xacro/point_mass_hands.urdf (robot description, URDF)
Before this commit: robot drc_skeleton, 2 links, 2 joints
Links:
- link l_hand_point_mass: mass 2.9 -> 3.1690
- link r_hand_point_mass: mass 2.9 -> 3.1690
Joints:
- joint l_hand_joint: origin xyz=0.0 0.15 0.0 rpy=0 0 0 -> xyz=0.004 0.1601 -0.0078 rpy=0 0 0
- joint r_hand_joint: origin xyz=0.0 -0.15 0.0 rpy=0 0 0 -> xyz=0.004 -0.1601 -0.0078 rpy=0 0 0

Commit message: modified COM of point hands
git-svn-id: https://svn.csail.mit.edu/drc@3420 c7283977-0100-402a-a91a-fa70b306dbfe

File: software/models/mit_gazebo_models/mit_robot_drake/model_minimal_contact_point_hands.urdf (robot description, URDF)
Before this commit: robot atlas, 31 links, 30 joints
Joints:
- joint l_hand_joint: origin xyz=0.004 0.1601 -0.0078 rpy=0 0 0 -> xyz=-0.0052 -0.0124  0.0972 rpy=0 0 0
- joint r_hand_joint: origin xyz=0.004 -0.1601 -0.0078 rpy=0 0 0 -> xyz=-0.0052 -0.0124  0.0972 rpy=0 0 0

File: software/models/mit_gazebo_models/mit_robot_drake/xacro/point_mass_hands.urdf (robot description, URDF)
Before this commit: robot drc_skeleton, 2 links, 2 joints
Joints:
- joint l_hand_joint: origin xyz=0.004 0.1601 -0.0078 rpy=0 0 0 -> xyz=-0.0052 -0.0124  0.0972 rpy=0 0 0
- joint r_hand_joint: origin xyz=0.004 -0.1601 -0.0078 rpy=0 0 0 -> xyz=-0.0052 -0.0124  0.0972 rpy=0 0 0

Commit message: hand point mass COM is updated
git-svn-id: https://svn.csail.mit.edu/drc@3421 c7283977-0100-402a-a91a-fa70b306dbfe

File: software/models/mit_gazebo_models/mit_robot_drake/model_minimal_contact_point_hands.urdf (robot description, URDF)
Before this commit: robot atlas, 31 links, 30 joints
Joints:
- joint l_hand_joint: origin xyz=-0.0052 -0.0124  0.0972 rpy=0 0 0 -> xyz=0.0037 0.1603 -0.0087 rpy=0 0 0
- joint r_hand_joint: origin xyz=-0.0052 -0.0124  0.0972 rpy=0 0 0 -> xyz=0.0037 -0.1603 -0.0087 rpy=0 0 0

File: software/models/mit_gazebo_models/mit_robot_drake/xacro/point_mass_hands.urdf (robot description, URDF)
Before this commit: robot drc_skeleton, 2 links, 2 joints
Joints:
- joint l_hand_joint: origin xyz=-0.0052 -0.0124  0.0972 rpy=0 0 0 -> xyz=0.0037 0.1603 -0.0087 rpy=0 0 0
- joint r_hand_joint: origin xyz=-0.0052 -0.0124  0.0972 rpy=0 0 0 -> xyz=0.0037 -0.1603 -0.0087 rpy=0 0 0

Commit message: point mass hand values for old and new hand masses. Old ones are checked in.
git-svn-id: https://svn.csail.mit.edu/drc@3432 c7283977-0100-402a-a91a-fa70b306dbfe

File: software/models/mit_gazebo_models/mit_robot_drake/model_minimal_contact_point_hands.urdf (robot description, URDF)
Before this commit: robot atlas, 31 links, 30 joints
Links:
- link l_hand_point_mass: mass 3.111 -> 2.312
- link r_hand_point_mass: mass 3.111 -> 2.312
Joints:
- joint l_hand_joint: origin xyz=0.0037 0.1603 -0.0087 rpy=0 0 0 -> xyz=0.0054 0.1905 -0.0129 rpy=0 0 0
- joint r_hand_joint: origin xyz=0.0037 -0.1603 -0.0087 rpy=0 0 0 -> xyz=0.0054 -0.1905 -0.0129 rpy=0 0 0

File: software/models/mit_gazebo_models/mit_robot_drake/xacro/point_mass_hands.urdf (robot description, URDF)
Before this commit: robot drc_skeleton, 2 links, 2 joints
Links:
- link l_hand_point_mass: mass 3.111 -> 2.312
- link r_hand_point_mass: mass 3.111 -> 2.312
Joints:
- joint l_hand_joint: origin xyz=0.0037 0.1603 -0.0087 rpy=0 0 0 -> xyz=0.0054 0.1905 -0.0129 rpy=0 0 0
- joint r_hand_joint: origin xyz=0.0037 -0.1603 -0.0087 rpy=0 0 0 -> xyz=0.0054 -0.1905 -0.0129 rpy=0 0 0

Commit message: minor changes made during  qual2 logs. The new drcsim version has new hand values.
git-svn-id: https://svn.csail.mit.edu/drc@3458 c7283977-0100-402a-a91a-fa70b306dbfe

File: software/models/mit_gazebo_models/mit_robot_drake/model_minimal_contact_point_hands.urdf (robot description, URDF)
Before this commit: robot atlas, 31 links, 30 joints
Links:
- link l_hand_point_mass: mass 2.312 -> 3.131
- link r_hand_point_mass: mass 2.312 -> 3.131
Joints:
- joint l_hand_joint: origin xyz=0.0054 0.1905 -0.0129 rpy=0 0 0 -> xyz=0.0037 0.1603 -0.0087 rpy=0 0 0
- joint r_hand_joint: origin xyz=0.0054 -0.1905 -0.0129 rpy=0 0 0 -> xyz=0.0037 -0.1603 -0.0087 rpy=0 0 0

File: software/models/mit_gazebo_models/mit_robot_drake/xacro/point_mass_hands.urdf (robot description, URDF)
Before this commit: robot drc_skeleton, 2 links, 2 joints
Links:
- link l_hand_point_mass: mass 2.312 -> 3.131
- link r_hand_point_mass: mass 2.312 -> 3.131
Joints:
- joint l_hand_joint: origin xyz=0.0054 0.1905 -0.0129 rpy=0 0 0 -> xyz=0.0037 0.1603 -0.0087 rpy=0 0 0
- joint r_hand_joint: origin xyz=0.0054 -0.1905 -0.0129 rpy=0 0 0 -> xyz=0.0037 -0.1603 -0.0087 rpy=0 0 0

Commit message: minor changes to drake multisense head urdf
git-svn-id: https://svn.csail.mit.edu/drc@4253 c7283977-0100-402a-a91a-fa70b306dbfe

File: software/models/mit_gazebo_models/mit_robot_drake/model_minimal_contact_point_hands.urdf (robot description, URDF)
Before this commit: robot atlas, 31 links, 30 joints
Links:
- link head: geometry visual mesh filename=package://mit_drcsim_scripts/models/multisense_sl/meshes/he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

File: software/models/mit_gazebo_models/mit_robot_drake/model_minimal_contact_with_hands.urdf (robot description, URDF)
Before this commit: robot atlas, 101 links, 100 joints
Links:
- link head: geometry visual mesh filename=package://mit_drcsim_scripts/models/multisense_sl/meshes/he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

File: software/models/mit_gazebo_models/mit_robot_drake/model_simple_visuals_minimal_contact_point_hands.urdf (robot description, URDF)
Before this commit: robot atlas, 29 links, 28 joints
Links:
- added link l_hand_point_mass, mass 3.131; visual sphere radius=0.03
- added link r_hand_point_mass, mass 3.131; visual sphere radius=0.03
- link head: geometry collision box size=0.0468 0.12 0.1184; collision box size=0.1311 0.12 0.0591
- link l_clav: geometry collision box size=0.13 0.15 0.05; collision cylinder length=0.1525 radius=0.045
- link l_farm: geometry collision box size=0.135 0.1 0.045; collision cylinder length=0.125 radius=0.045
- link l_foot: geometry collision box size=0.26 0.124887 0.05; collision sphere radius=0
- link l_hand: geometry collision box size=0.13 0.09 0.07; collision cylinder length=0.05 radius=0.03
- link l_larm: geometry collision box size=0.135 0.15 0.06; collision cylinder length=0.125 radius=0.045
- link l_lglut: geometry collision cylinder length=0.060306 radius=0.02009687; collision cylinder length=0.12 radius=0.02
- link l_lleg: geometry collision cylinder length=0.40 radius=0.07; collision sphere radius=0
- link l_scap: geometry collision cylinder length=0.125 radius=0.045; visual box size=0.15 0.15 0.06
- link l_talus: geometry collision cylinder length=0.029542 radius=0.010181; visual cylinder length=0.010059 radius=0.010348
- link l_uarm: geometry collision cylinder length=0.125 radius=0.045; visual box size=0.04 0.07 0.13
- link l_uglut: geometry collision cylinder length=0.078396 radius=0.019096; visual cylinder length=0.078396 radius=0.019096
- link l_uleg: geometry collision cylinder length=0.10 radius=0.1; collision cylinder length=0.15 radius=0.07
- link ltorso: geometry 
- link mtorso: geometry collision cylinder length=0.02 radius=0.015; collision cylinder length=0.02 radius=0.015
- link pelvis: mass 12.64638 -> 12.54638; geometry collision box size=0.1 0.15 0.2; collision box size=0.1 0.15 0.2
- link r_clav: geometry collision box size=0.13 0.15 0.05; collision cylinder length=0.1525 radius=0.045
- link r_farm: geometry collision box size=0.135 0.1 0.045; collision cylinder length=0.125 radius=0.045
- link r_foot: geometry collision box size=0.26 0.124887 0.05; collision sphere radius=0
- link r_hand: geometry collision box size=0.13 0.09 0.07; collision cylinder length=0.05 radius=0.03
- link r_larm: geometry collision box size=0.135 0.15 0.06; collision cylinder length=0.125 radius=0.045
- link r_lglut: geometry collision cylinder length=0.060306 radius=0.02009687; collision cylinder length=0.12 radius=0.02
- link r_lleg: geometry collision cylinder length=0.40 radius=0.07; collision sphere radius=0
- link r_scap: geometry collision box size=0.15 0.15 0.06; collision cylinder length=0.125 radius=0.045
- link r_talus: geometry collision cylinder length=0.010059 radius=0.010348; collision cylinder length=0.029542 radius=0.010181
- link r_uarm: geometry collision box size=0.04 0.07 0.13; collision cylinder length=0.125 radius=0.045
- link r_uglut: geometry collision cylinder length=0.078396 radius=0.019096; collision cylinder length=0.080842 radius=0.019841
- link r_uleg: geometry collision cylinder length=0.10 radius=0.1; collision cylinder length=0.15 radius=0.07
- link utorso: geometry collision box size=0.3188 0.24 0.3162; collision cylinder length=0.22375 radius=0.0363
Joints:
- added joint l_hand_joint: type fixed, parent l_hand, child l_hand_point_mass, origin xyz=0.0037 0.1603 -0.0087 rpy=0 0 0
- added joint r_hand_joint: type fixed, parent r_hand, child r_hand_point_mass, origin xyz=0.0037 -0.1603 -0.0087 rpy=0 0 0

File: software/models/mit_gazebo_models/mit_robot_drake/xacro/multisense_sl_no_contact.urdf (robot description, URDF)
Before this commit: robot multisense_sl, 1 links, 0 joints
Links:
- link head: geometry visual mesh filename=package://mit_drcsim_scripts/models/multisense_sl/meshes/he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

Commit message: heavier point hands

File: software/models/mit_gazebo_models/mit_robot_drake/model_minimal_contact_point_hands.urdf (robot description, URDF)
Before this commit: robot atlas, 31 links, 30 joints
Links:
- link l_hand_point_mass: mass 3.131 -> 5.131
- link r_hand_point_mass: mass 3.131 -> 5.131

File: software/models/mit_gazebo_models/mit_robot_drake/xacro/point_mass_sandia_hands.urdf (robot description, URDF)
Before this commit: robot drc_skeleton, 2 links, 2 joints
Links:
- link l_hand_point_mass: mass 3.131 -> 5.131
- link r_hand_point_mass: mass 3.131 -> 5.131

Commit message: adding back nominal friction params for legs

File: software/models/mit_gazebo_models/mit_robot_drake/model_minimal_contact_point_hands.urdf (robot description, URDF)
Before this commit: robot atlas, 31 links, 30 joints
Links:
- link l_hand_point_mass: mass 5.131 -> 6.131
- link r_hand_point_mass: mass 5.131 -> 6.131

Commit message: updating compiled model in repo

File: software/models/mit_gazebo_models/mit_robot_drake/model_minimal_contact_point_hands.urdf (robot description, URDF)
Before this commit: robot atlas, 31 links, 30 joints
Links:
- link l_hand_point_mass: mass 6.131 -> 5.131
- link r_hand_point_mass: mass 6.131 -> 5.131

Commit message: local edits to controller urdf

File: software/models/mit_gazebo_models/mit_robot_drake/model_minimal_contact_point_hands.urdf (robot description, URDF)
Before this commit: robot atlas, 31 links, 30 joints
Joints:
- joint l_leg_aky: limit lower=-1 upper=0.7 effort=350 velocity=12 -> lower=-1 upper=0.7 effort=450 velocity=12
- joint r_leg_aky: limit lower=-1 upper=0.7 effort=350 velocity=12 -> lower=-1 upper=0.7 effort=450 velocity=12

Commit message: knee torque lims and various working edits in controller

File: software/models/mit_gazebo_models/mit_robot_drake/model_minimal_contact_point_hands.urdf (robot description, URDF)
Before this commit: robot atlas, 31 links, 30 joints
Joints:
- joint l_leg_kny: limit lower=0 upper=2.38569 effort=220 velocity=12 -> lower=0 upper=2.38569 effort=320 velocity=12
- joint r_leg_kny: limit lower=0 upper=2.38569 effort=220 velocity=12 -> lower=0 upper=2.38569 effort=320 velocity=12
