Commit message: Shift utorso COM and increase kny/aky torque limit
Resolves #548

File: software/models/mit_gazebo_models/mit_robot_drake/model_convex_hull_closed_robotiq_hands.urdf (robot description, URDF)
Before this commit: robot atlas, 33 links, 32 joints
Joints:
- joint l_leg_aky: limit lower=-1 upper=0.7 effort=350 velocity=12 -> lower=-1 upper=0.7 effort=450 velocity=12
- joint l_leg_kny: limit lower=0 upper=2.38569 effort=220 velocity=12 -> lower=0 upper=2.38569 effort=320 velocity=12
- joint r_leg_aky: limit lower=-1 upper=0.7 effort=350 velocity=12 -> lower=-1 upper=0.7 effort=450 velocity=12
- joint r_leg_kny: limit lower=0 upper=2.38569 effort=220 velocity=12 -> lower=0 upper=2.38569 effort=320 velocity=12

File: software/models/mit_gazebo_models/mit_robot_drake/model_convex_hull_no_hands.urdf (robot description, URDF)
Before this commit: robot atlas, 29 links, 28 joints
Joints:
- joint l_leg_aky: limit lower=-1 upper=0.7 effort=350 velocity=12 -> lower=-1 upper=0.7 effort=450 velocity=12
- joint l_leg_kny: limit lower=0 upper=2.38569 effort=220 velocity=12 -> lower=0 upper=2.38569 effort=320 velocity=12
- joint r_leg_aky: limit lower=-1 upper=0.7 effort=350 velocity=12 -> lower=-1 upper=0.7 effort=450 velocity=12
- joint r_leg_kny: limit lower=0 upper=2.38569 effort=220 velocity=12 -> lower=0 upper=2.38569 effort=320 velocity=12

File: software/models/mit_gazebo_models/mit_robot_drake/model_convex_hull_robotiq_hands.urdf (robot description, URDF)
Before this commit: robot atlas, 33 links, 32 joints
Joints:
- joint l_leg_aky: limit lower=-1 upper=0.7 effort=350 velocity=12 -> lower=-1 upper=0.7 effort=450 velocity=12
- joint l_leg_kny: limit lower=0 upper=2.38569 effort=220 velocity=12 -> lower=0 upper=2.38569 effort=320 velocity=12
- joint r_leg_aky: limit lower=-1 upper=0.7 effort=350 velocity=12 -> lower=-1 upper=0.7 effort=450 velocity=12
- joint r_leg_kny: limit lower=0 upper=2.38569 effort=220 velocity=12 -> lower=0 upper=2.38569 effort=320 velocity=12

File: software/models/mit_gazebo_models/mit_robot_drake/model_minimal_contact.urdf (robot description, URDF)
Before this commit: robot atlas, 29 links, 28 joints
Joints:
- joint l_leg_aky: limit lower=-1 upper=0.7 effort=350 velocity=12 -> lower=-1 upper=0.7 effort=450 velocity=12
- joint l_leg_kny: limit lower=0 upper=2.38569 effort=220 velocity=12 -> lower=0 upper=2.38569 effort=320 velocity=12
- joint r_leg_aky: limit lower=-1 upper=0.7 effort=350 velocity=12 -> lower=-1 upper=0.7 effort=450 velocity=12
- joint r_leg_kny: limit lower=0 upper=2.38569 effort=220 velocity=12 -> lower=0 upper=2.38569 effort=320 velocity=12

File: software/models/mit_gazebo_models/mit_robot_drake/model_minimal_contact_point_hands.urdf (robot description, URDF)
Before this commit: robot atlas, 31 links, 30 joints
Joints:
- joint l_leg_aky: limit lower=-1 upper=0.7 effort=350 velocity=12 -> lower=-1 upper=0.7 effort=450 velocity=12
- joint l_leg_kny: limit lower=0 upper=2.38569 effort=220 velocity=12 -> lower=0 upper=2.38569 effort=320 velocity=12
- joint r_leg_aky: limit lower=-1 upper=0.7 effort=350 velocity=12 -> lower=-1 upper=0.7 effort=450 velocity=12
- joint r_leg_kny: limit lower=0 upper=2.38569 effort=220 velocity=12 -> lower=0 upper=2.38569 effort=320 velocity=12

File: software/models/mit_gazebo_models/mit_robot_drake/model_minimal_contact_point_stumps.urdf (robot description, URDF)
Before this commit: robot atlas, 31 links, 30 joints
Joints:
- joint l_leg_aky: limit lower=-1 upper=0.7 effort=350 velocity=12 -> lower=-1 upper=0.7 effort=450 velocity=12
- joint l_leg_kny: limit lower=0 upper=2.38569 effort=220 velocity=12 -> lower=0 upper=2.38569 effort=320 velocity=12
- joint r_leg_aky: limit lower=-1 upper=0.7 effort=350 velocity=12 -> lower=-1 upper=0.7 effort=450 velocity=12
- joint r_leg_kny: limit lower=0 upper=2.38569 effort=220 velocity=12 -> lower=0 upper=2.38569 effort=320 velocity=12

File: software/models/mit_gazebo_models/mit_robot_drake/xacro/atlas_skeleton.xacro (robot description, xacro)
@@ -770,5 +770,5 @@
         <inertial>
 	        <mass value="52" />
-            <origin xyz="-0.11 0 0.3" rpy="0 -0 0" />
+            <origin xyz="-0.13 0 0.3" rpy="0 -0 0" />
             <inertia ixx="1.466" ixy="0.00362" ixz="0.336" iyy="1.51" iyz="0.001" izz="1.3" />
         </inertial>
@@ -959,5 +959,5 @@
         <child link="l_talus" />
         <dynamics damping="0.5" friction="5.0" coulomb_window="0.175"/>
-        <limit effort="350" velocity="12" lower="-1" upper="0.7" />
+        <limit effort="450" velocity="12" lower="-1" upper="0.7" />
         <safety_controller k_position="100" k_velocity="100" soft_lower_limit="-11" soft_upper_limit="10.7" />
     </joint>
@@ -995,5 +995,5 @@
         <child link="l_lleg" />
         <dynamics damping="0.1" friction="0" />
-        <limit effort="220" effort_max="220" effort_min="-300" velocity="12" lower="0" upper="2.38569" />
+        <limit effort="320" effort_max="320" effort_min="-400" velocity="12" lower="0" upper="2.38569" />
         <safety_controller k_position="100" k_velocity="100" soft_lower_limit="-10" soft_upper_limit="12.3857" />
     </joint>
@@ -1076,5 +1076,5 @@
         <child link="r_talus" />
         <dynamics damping="0.5" friction="5.0" coulomb_window="0.175"/>
-        <limit effort="350" velocity="12" lower="-1" upper="0.7" />
+        <limit effort="450" velocity="12" lower="-1" upper="0.7" />
         <safety_controller k_position="100" k_velocity="100" soft_lower_limit="-11" soft_upper_limit="10.7" />
     </joint>
@@ -1112,5 +1112,5 @@
         <child link="r_lleg" />
         <dynamics damping="0.1" friction="0" />
-        <limit effort="220" effort_max="220" effort_min="-300" velocity="12" lower="0" upper="2.38569" />
+        <limit effort="320" effort_max="320" effort_min="-400" velocity="12" lower="0" upper="2.38569" />
         <safety_controller k_position="100" k_velocity="100" soft_lower_limit="-10" soft_upper_limit="12.3857" />
     </joint>

Commit message: Revert "Shift utorso COM and increase kny/aky torque limit"
This reverts commit 0c9af4bfaaecfa3c6db6fd0b2dfdad258cf317c4.

File: software/models/mit_gazebo_models/mit_robot_drake/model_convex_hull_closed_robotiq_hands.urdf (robot description, URDF)
Before this commit: robot atlas, 33 links, 32 joints
Joints:
- joint l_leg_aky: limit lower=-1 upper=0.7 effort=450 velocity=12 -> lower=-1 upper=0.7 effort=350 velocity=12
- joint l_leg_kny: limit lower=0 upper=2.38569 effort=320 velocity=12 -> lower=0 upper=2.38569 effort=220 velocity=12
- joint r_leg_aky: limit lower=-1 upper=0.7 effort=450 velocity=12 -> lower=-1 upper=0.7 effort=350 velocity=12
- joint r_leg_kny: limit lower=0 upper=2.38569 effort=320 velocity=12 -> lower=0 upper=2.38569 effort=220 velocity=12

File: software/models/mit_gazebo_models/mit_robot_drake/model_convex_hull_no_hands.urdf (robot description, URDF)
Before this commit: robot atlas, 29 links, 28 joints
Joints:
- joint l_leg_aky: limit lower=-1 upper=0.7 effort=450 velocity=12 -> lower=-1 upper=0.7 effort=350 velocity=12
- joint l_leg_kny: limit lower=0 upper=2.38569 effort=320 velocity=12 -> lower=0 upper=2.38569 effort=220 velocity=12
- joint r_leg_aky: limit lower=-1 upper=0.7 effort=450 velocity=12 -> lower=-1 upper=0.7 effort=350 velocity=12
- joint r_leg_kny: limit lower=0 upper=2.38569 effort=320 velocity=12 -> lower=0 upper=2.38569 effort=220 velocity=12

File: software/models/mit_gazebo_models/mit_robot_drake/model_convex_hull_robotiq_hands.urdf (robot description, URDF)
Before this commit: robot atlas, 33 links, 32 joints
Joints:
- joint l_leg_aky: limit lower=-1 upper=0.7 effort=450 velocity=12 -> lower=-1 upper=0.7 effort=350 velocity=12
- joint l_leg_kny: limit lower=0 upper=2.38569 effort=320 velocity=12 -> lower=0 upper=2.38569 effort=220 velocity=12
- joint r_leg_aky: limit lower=-1 upper=0.7 effort=450 velocity=12 -> lower=-1 upper=0.7 effort=350 velocity=12
- joint r_leg_kny: limit lower=0 upper=2.38569 effort=320 velocity=12 -> lower=0 upper=2.38569 effort=220 velocity=12

File: software/models/mit_gazebo_models/mit_robot_drake/model_minimal_contact.urdf (robot description, URDF)
Before this commit: robot atlas, 29 links, 28 joints
Joints:
- joint l_leg_aky: limit lower=-1 upper=0.7 effort=450 velocity=12 -> lower=-1 upper=0.7 effort=350 velocity=12
- joint l_leg_kny: limit lower=0 upper=2.38569 effort=320 velocity=12 -> lower=0 upper=2.38569 effort=220 velocity=12
- joint r_leg_aky: limit lower=-1 upper=0.7 effort=450 velocity=12 -> lower=-1 upper=0.7 effort=350 velocity=12
- joint r_leg_kny: limit lower=0 upper=2.38569 effort=320 velocity=12 -> lower=0 upper=2.38569 effort=220 velocity=12

File: software/models/mit_gazebo_models/mit_robot_drake/model_minimal_contact_point_hands.urdf (robot description, URDF)
Before this commit: robot atlas, 31 links, 30 joints
Joints:
- joint l_leg_aky: limit lower=-1 upper=0.7 effort=450 velocity=12 -> lower=-1 upper=0.7 effort=350 velocity=12
- joint l_leg_kny: limit lower=0 upper=2.38569 effort=320 velocity=12 -> lower=0 upper=2.38569 effort=220 velocity=12
- joint r_leg_aky: limit lower=-1 upper=0.7 effort=450 velocity=12 -> lower=-1 upper=0.7 effort=350 velocity=12
- joint r_leg_kny: limit lower=0 upper=2.38569 effort=320 velocity=12 -> lower=0 upper=2.38569 effort=220 velocity=12

File: software/models/mit_gazebo_models/mit_robot_drake/model_minimal_contact_point_stumps.urdf (robot description, URDF)
Before this commit: robot atlas, 31 links, 30 joints
Joints:
- joint l_leg_aky: limit lower=-1 upper=0.7 effort=450 velocity=12 -> lower=-1 upper=0.7 effort=350 velocity=12
- joint l_leg_kny: limit lower=0 upper=2.38569 effort=320 velocity=12 -> lower=0 upper=2.38569 effort=220 velocity=12
- joint r_leg_aky: limit lower=-1 upper=0.7 effort=450 velocity=12 -> lower=-1 upper=0.7 effort=350 velocity=12
- joint r_leg_kny: limit lower=0 upper=2.38569 effort=320 velocity=12 -> lower=0 upper=2.38569 effort=220 velocity=12

File: software/models/mit_gazebo_models/mit_robot_drake/xacro/atlas_skeleton.xacro (robot description, xacro)
@@ -770,5 +770,5 @@
         <inertial>
 	        <mass value="52" />
-            <origin xyz="-0.13 0 0.3" rpy="0 -0 0" />
+            <origin xyz="-0.11 0 0.3" rpy="0 -0 0" />
             <inertia ixx="1.466" ixy="0.00362" ixz="0.336" iyy="1.51" iyz="0.001" izz="1.3" />
         </inertial>
@@ -959,5 +959,5 @@
         <child link="l_talus" />
         <dynamics damping="0.5" friction="5.0" coulomb_window="0.175"/>
-        <limit effort="450" velocity="12" lower="-1" upper="0.7" />
+        <limit effort="350" velocity="12" lower="-1" upper="0.7" />
         <safety_controller k_position="100" k_velocity="100" soft_lower_limit="-11" soft_upper_limit="10.7" />
     </joint>
@@ -995,5 +995,5 @@
         <child link="l_lleg" />
         <dynamics damping="0.1" friction="0" />
-        <limit effort="320" effort_max="320" effort_min="-400" velocity="12" lower="0" upper="2.38569" />
+        <limit effort="220" effort_max="220" effort_min="-300" velocity="12" lower="0" upper="2.38569" />
         <safety_controller k_position="100" k_velocity="100" soft_lower_limit="-10" soft_upper_limit="12.3857" />
     </joint>
@@ -1076,5 +1076,5 @@
         <child link="r_talus" />
         <dynamics damping="0.5" friction="5.0" coulomb_window="0.175"/>
-        <limit effort="450" velocity="12" lower="-1" upper="0.7" />
+        <limit effort="350" velocity="12" lower="-1" upper="0.7" />
         <safety_controller k_position="100" k_velocity="100" soft_lower_limit="-11" soft_upper_limit="10.7" />
     </joint>
@@ -1112,5 +1112,5 @@
         <child link="r_lleg" />
         <dynamics damping="0.1" friction="0" />
-        <limit effort="320" effort_max="320" effort_min="-400" velocity="12" lower="0" upper="2.38569" />
+        <limit effort="220" effort_max="220" effort_min="-300" velocity="12" lower="0" upper="2.38569" />
         <safety_controller k_position="100" k_velocity="100" soft_lower_limit="-10" soft_upper_limit="12.3857" />
     </joint>

Commit message: Increase kny and aky torque limits.
They were

  aky: +- 350 Nm
  kny: [-300 Nm, 220 Nm]

Now they are

  aky: +- 700 Nm
  kny: [-400 Nm, 320 Nm]

File: software/models/mit_gazebo_models/mit_robot_drake/model_convex_hull_closed_robotiq_hands.urdf (robot description, URDF)
Before this commit: robot atlas, 33 links, 32 joints
Joints:
- joint l_leg_aky: limit lower=-1 upper=0.7 effort=350 velocity=12 -> lower=-1 upper=0.7 effort=700 velocity=12
- joint l_leg_kny: limit lower=0 upper=2.38569 effort=220 velocity=12 -> lower=0 upper=2.38569 effort=320 velocity=12
- joint r_leg_aky: limit lower=-1 upper=0.7 effort=350 velocity=12 -> lower=-1 upper=0.7 effort=700 velocity=12
- joint r_leg_kny: limit lower=0 upper=2.38569 effort=220 velocity=12 -> lower=0 upper=2.38569 effort=320 velocity=12

File: software/models/mit_gazebo_models/mit_robot_drake/model_convex_hull_no_hands.urdf (robot description, URDF)
Before this commit: robot atlas, 29 links, 28 joints
Joints:
- joint l_leg_aky: limit lower=-1 upper=0.7 effort=350 velocity=12 -> lower=-1 upper=0.7 effort=700 velocity=12
- joint l_leg_kny: limit lower=0 upper=2.38569 effort=220 velocity=12 -> lower=0 upper=2.38569 effort=320 velocity=12
- joint r_leg_aky: limit lower=-1 upper=0.7 effort=350 velocity=12 -> lower=-1 upper=0.7 effort=700 velocity=12
- joint r_leg_kny: limit lower=0 upper=2.38569 effort=220 velocity=12 -> lower=0 upper=2.38569 effort=320 velocity=12

File: software/models/mit_gazebo_models/mit_robot_drake/model_convex_hull_robotiq_hands.urdf (robot description, URDF)
Before this commit: robot atlas, 33 links, 32 joints
Joints:
- joint l_leg_aky: limit lower=-1 upper=0.7 effort=350 velocity=12 -> lower=-1 upper=0.7 effort=700 velocity=12
- joint l_leg_kny: limit lower=0 upper=2.38569 effort=220 velocity=12 -> lower=0 upper=2.38569 effort=320 velocity=12
- joint r_leg_aky: limit lower=-1 upper=0.7 effort=350 velocity=12 -> lower=-1 upper=0.7 effort=700 velocity=12
- joint r_leg_kny: limit lower=0 upper=2.38569 effort=220 velocity=12 -> lower=0 upper=2.38569 effort=320 velocity=12

File: software/models/mit_gazebo_models/mit_robot_drake/model_minimal_contact.urdf (robot description, URDF)
Before this commit: robot atlas, 29 links, 28 joints
Joints:
- joint l_leg_aky: limit lower=-1 upper=0.7 effort=350 velocity=12 -> lower=-1 upper=0.7 effort=700 velocity=12
- joint l_leg_kny: limit lower=0 upper=2.38569 effort=220 velocity=12 -> lower=0 upper=2.38569 effort=320 velocity=12
- joint r_leg_aky: limit lower=-1 upper=0.7 effort=350 velocity=12 -> lower=-1 upper=0.7 effort=700 velocity=12
- joint r_leg_kny: limit lower=0 upper=2.38569 effort=220 velocity=12 -> lower=0 upper=2.38569 effort=320 velocity=12

File: software/models/mit_gazebo_models/mit_robot_drake/model_minimal_contact_point_hands.urdf (robot description, URDF)
Before this commit: robot atlas, 31 links, 30 joints
Joints:
- joint l_leg_aky: limit lower=-1 upper=0.7 effort=450 velocity=12 -> lower=-1 upper=0.7 effort=700 velocity=12
- joint r_leg_aky: limit lower=-1 upper=0.7 effort=450 velocity=12 -> lower=-1 upper=0.7 effort=700 velocity=12

File: software/models/mit_gazebo_models/mit_robot_drake/model_minimal_contact_point_stumps.urdf (robot description, URDF)
Before this commit: robot atlas, 31 links, 30 joints
Joints:
- joint l_leg_aky: limit lower=-1 upper=0.7 effort=350 velocity=12 -> lower=-1 upper=0.7 effort=700 velocity=12
- joint l_leg_kny: limit lower=0 upper=2.38569 effort=220 velocity=12 -> lower=0 upper=2.38569 effort=320 velocity=12
- joint r_leg_aky: limit lower=-1 upper=0.7 effort=350 velocity=12 -> lower=-1 upper=0.7 effort=700 velocity=12
- joint r_leg_kny: limit lower=0 upper=2.38569 effort=220 velocity=12 -> lower=0 upper=2.38569 effort=320 velocity=12

File: software/models/mit_gazebo_models/mit_robot_drake/xacro/atlas_skeleton.xacro (robot description, xacro)
@@ -959,5 +959,5 @@
         <child link="l_talus" />
         <dynamics damping="0.5" friction="5.0" coulomb_window="0.175"/>
-        <limit effort="350" velocity="12" lower="-1" upper="0.7" />
+        <limit effort="700" velocity="12" lower="-1" upper="0.7" />
         <safety_controller k_position="100" k_velocity="100" soft_lower_limit="-11" soft_upper_limit="10.7" />
     </joint>
@@ -995,5 +995,5 @@
         <child link="l_lleg" />
         <dynamics damping="0.1" friction="0" />
-        <limit effort="220" effort_max="220" effort_min="-300" velocity="12" lower="0" upper="2.38569" />
+        <limit effort="320" effort_max="320" effort_min="-400" velocity="12" lower="0" upper="2.38569" />
         <safety_controller k_position="100" k_velocity="100" soft_lower_limit="-10" soft_upper_limit="12.3857" />
     </joint>
@@ -1076,5 +1076,5 @@
         <child link="r_talus" />
         <dynamics damping="0.5" friction="5.0" coulomb_window="0.175"/>
-        <limit effort="350" velocity="12" lower="-1" upper="0.7" />
+        <limit effort="700" velocity="12" lower="-1" upper="0.7" />
         <safety_controller k_position="100" k_velocity="100" soft_lower_limit="-11" soft_upper_limit="10.7" />
     </joint>
@@ -1112,5 +1112,5 @@
         <child link="r_lleg" />
         <dynamics damping="0.1" friction="0" />
-        <limit effort="220" effort_max="220" effort_min="-300" velocity="12" lower="0" upper="2.38569" />
+        <limit effort="320" effort_max="320" effort_min="-400" velocity="12" lower="0" upper="2.38569" />
         <safety_controller k_position="100" k_velocity="100" soft_lower_limit="-10" soft_upper_limit="12.3857" />
     </joint>
