Commit message: changes to PnC model and PD gains
git-svn-id: https://svn.csail.mit.edu/drc@936 c7283977-0100-402a-a91a-fa70b306dbfe

File: software/models/mit_gazebo_models/mit_robot_PnC/model.urdf (robot description, URDF)
Before this commit: robot atlas, 35 links, 34 joints
Links:
- added link l_f0_0, mass 0.1; collision mesh filename=package://sandia_hand/meshes/f0.stl; visual mesh filename=package://sandia_hand/meshes/f0.stl
- added link l_f0_1, mass 0.1; collision mesh filename=package://sandia_hand/meshes/f1.stl; visual mesh filename=package://sandia_hand/meshes/f1.stl
- added link l_f0_1_accel, mass 0.1
- added link l_f0_2, mass 0.1; collision mesh filename=package://sandia_hand/meshes/f2.stl; visual mesh filename=package://sandia_hand/meshes/f2.stl
- added link l_f0_2_accel, mass 0.1
- added link l_f0_base, mass 0.1
- added link l_f0_fixed_accel, mass 0.1
- added link l_f1_0, mass 0.1; collision mesh filename=package://sandia_hand/meshes/f0.stl; visual mesh filename=package://sandia_hand/meshes/f0.stl
- added link l_f1_1, mass 0.1; collision mesh filename=package://sandia_hand/meshes/f1.stl; visual mesh filename=package://sandia_hand/meshes/f1.stl
- added link l_f1_1_accel, mass 0.1
- added link l_f1_2, mass 0.1; collision mesh filename=package://sandia_hand/meshes/f2.stl; visual mesh filename=package://sandia_hand/meshes/f2.stl
- added link l_f1_2_accel, mass 0.1
- added link l_f1_base, mass 0.1
- added link l_f1_fixed_accel, mass 0.1
- added link l_f2_0, mass 0.1; collision mesh filename=package://sandia_hand/meshes/f0.stl; visual mesh filename=package://sandia_hand/meshes/f0.stl
- added link l_f2_1, mass 0.1; collision mesh filename=package://sandia_hand/meshes/f1.stl; visual mesh filename=package://sandia_hand/meshes/f1.stl
- added link l_f2_1_accel, mass 0.1
- added link l_f2_2, mass 0.1; collision mesh filename=package://sandia_hand/meshes/f2.stl; visual mesh filename=package://sandia_hand/meshes/f2.stl
- added link l_f2_2_accel, mass 0.1
- added link l_f2_base, mass 0.1
- added link l_f2_fixed_accel, mass 0.1
- added link l_f3_0, mass 0.1; collision mesh filename=package://sandia_hand/meshes/f0.stl; visual mesh filename=package://sandia_hand/meshes/f0.stl
- added link l_f3_1, mass 0.1; collision mesh filename=package://sandia_hand/meshes/f1.stl; visual mesh filename=package://sandia_hand/meshes/f1.stl
- added link l_f3_1_accel, mass 0.1
- added link l_f3_2, mass 0.1; collision mesh filename=package://sandia_hand/meshes/f2.stl; visual mesh filename=package://sandia_hand/meshes/f2.stl
- added link l_f3_2_accel, mass 0.1
- added link l_f3_base, mass 0.1
- added link l_f3_fixed_accel, mass 0.1
- added link l_palm, mass 0.1; collision mesh filename=package://sandia_hand/meshes/palm.stl; visual mesh filename=package://sandia_hand/meshes/palm.stl
- added link r_f0_0, mass 0.1; collision mesh filename=package://sandia_hand/meshes/f0.stl; visual mesh filename=package://sandia_hand/meshes/f0.stl
- added link r_f0_1, mass 0.1; collision mesh filename=package://sandia_hand/meshes/f1.stl; visual mesh filename=package://sandia_hand/meshes/f1.stl
- added link r_f0_1_accel, mass 0.1
- added link r_f0_2, mass 0.1; collision mesh filename=package://sandia_hand/meshes/f2.stl; visual mesh filename=package://sandia_hand/meshes/f2.stl
- added link r_f0_2_accel, mass 0.1
- added link r_f0_base, mass 0.1
- added link r_f0_fixed_accel, mass 0.1
- added link r_f1_0, mass 0.1; collision mesh filename=package://sandia_hand/meshes/f0.stl; visual mesh filename=package://sandia_hand/meshes/f0.stl
- added link r_f1_1, mass 0.1; collision mesh filename=package://sandia_hand/meshes/f1.stl; visual mesh filename=package://sandia_hand/meshes/f1.stl
- added link r_f1_1_accel, mass 0.1
- added link r_f1_2, mass 0.1; collision mesh filename=package://sandia_hand/meshes/f2.stl; visual mesh filename=package://sandia_hand/meshes/f2.stl
- added link r_f1_2_accel, mass 0.1
- added link r_f1_base, mass 0.1
- added link r_f1_fixed_accel, mass 0.1
- added link r_f2_0, mass 0.1; collision mesh filename=package://sandia_hand/meshes/f0.stl; visual mesh filename=package://sandia_hand/meshes/f0.stl
- added link r_f2_1, mass 0.1; collision mesh filename=package://sandia_hand/meshes/f1.stl; visual mesh filename=package://sandia_hand/meshes/f1.stl
- added link r_f2_1_accel, mass 0.1
- added link r_f2_2, mass 0.1; collision mesh filename=package://sandia_hand/meshes/f2.stl; visual mesh filename=package://sandia_hand/meshes/f2.stl
- added link r_f2_2_accel, mass 0.1
- added link r_f2_base, mass 0.1
- added link r_f2_fixed_accel, mass 0.1
- added link r_f3_0, mass 0.1; collision mesh filename=package://sandia_hand/meshes/f0.stl; visual mesh filename=package://sandia_hand/meshes/f0.stl
- added link r_f3_1, mass 0.1; collision mesh filename=package://sandia_hand/meshes/f1.stl; visual mesh filename=package://sandia_hand/meshes/f1.stl
- added link r_f3_1_accel, mass 0.1
- added link r_f3_2, mass 0.1; collision mesh filename=package://sandia_hand/meshes/f2.stl; visual mesh filename=package://sandia_hand/meshes/f2.stl
- added link r_f3_2_accel, mass 0.1
- added link r_f3_base, mass 0.1
- added link r_f3_fixed_accel, mass 0.1
- added link r_palm, mass 0.1; collision mesh filename=package://sandia_hand/meshes/palm.stl; visual mesh filename=package://sandia_hand/meshes/palm.stl
Joints:
- added joint l_f0_1_accel: type fixed, parent l_f0_1, child l_f0_1_accel, origin xyz=0.03 0 0 rpy=-1.5709 0 0
- added joint l_f0_2_accel: type fixed, parent l_f0_2, child l_f0_2_accel, origin xyz=0.04 0 0 rpy=-1.5709 0 0
- added joint l_f0_base: type fixed, parent l_palm, child l_f0_base, origin xyz=0.14 0.0 0 rpy=0 0 0.3
- added joint l_f0_fixed_accel: type fixed, parent l_f0_base, child l_f0_fixed_accel, origin xyz=-0.05 0 0 rpy=0 0 0
- added joint l_f0_j0: type revolute, parent l_f0_base, child l_f0_0, origin xyz=0 0 0 rpy=0 0 0, axis 0 0 1, limit lower=-1.57079 upper=1.57079 effort=1 velocity=1
- added joint l_f0_j1: type revolute, parent l_f0_0, child l_f0_1, origin xyz=0.028 0 0 rpy=1.57079 0 0, axis 0 0 1, limit lower=-1.57079 upper=1.57079 effort=1 velocity=1
- added joint l_f0_j2: type revolute, parent l_f0_1, child l_f0_2, origin xyz=0.05 0 0 rpy=0 0 0, axis 0 0 1, limit lower=-1.57079 upper=1.57079 effort=1 velocity=1
- added joint l_f1_1_accel: type fixed, parent l_f1_1, child l_f1_1_accel, origin xyz=0.03 0 0 rpy=-1.5709 0 0
- added joint l_f1_2_accel: type fixed, parent l_f1_2, child l_f1_2_accel, origin xyz=0.04 0 0 rpy=-1.5709 0 0
- added joint l_f1_base: type fixed, parent l_palm, child l_f1_base, origin xyz=0.115 0.03122 0 rpy=0 0 0.3
- added joint l_f1_fixed_accel: type fixed, parent l_f1_base, child l_f1_fixed_accel, origin xyz=-0.05 0 0 rpy=0 0 0
- added joint l_f1_j0: type revolute, parent l_f1_base, child l_f1_0, origin xyz=0 0 0 rpy=0 0 0, axis 0 0 1, limit lower=-1.57079 upper=1.57079 effort=1 velocity=1
- added joint l_f1_j1: type revolute, parent l_f1_0, child l_f1_1, origin xyz=0.028 0 0 rpy=1.57079 0 0, axis 0 0 1, limit lower=-1.57079 upper=1.57079 effort=1 velocity=1
- added joint l_f1_j2: type revolute, parent l_f1_1, child l_f1_2, origin xyz=0.05 0 0 rpy=0 0 0, axis 0 0 1, limit lower=-1.57079 upper=1.57079 effort=1 velocity=1
- added joint l_f2_1_accel: type fixed, parent l_f2_1, child l_f2_1_accel, origin xyz=0.03 0 0 rpy=-1.5709 0 0
- added joint l_f2_2_accel: type fixed, parent l_f2_2, child l_f2_2_accel, origin xyz=0.04 0 0 rpy=-1.5709 0 0
- added joint l_f2_base: type fixed, parent l_palm, child l_f2_base, origin xyz=0.09 0.06245 0 rpy=0 0 0.3
- added joint l_f2_fixed_accel: type fixed, parent l_f2_base, child l_f2_fixed_accel, origin xyz=-0.05 0 0 rpy=0 0 0
- added joint l_f2_j0: type revolute, parent l_f2_base, child l_f2_0, origin xyz=0 0 0 rpy=0 0 0, axis 0 0 1, limit lower=-1.57079 upper=1.57079 effort=1 velocity=1
- added joint l_f2_j1: type revolute, parent l_f2_0, child l_f2_1, origin xyz=0.028 0 0 rpy=1.57079 0 0, axis 0 0 1, limit lower=-1.57079 upper=1.57079 effort=1 velocity=1
- added joint l_f2_j2: type revolute, parent l_f2_1, child l_f2_2, origin xyz=0.05 0 0 rpy=0 0 0, axis 0 0 1, limit lower=-1.57079 upper=1.57079 effort=1 velocity=1
- added joint l_f3_1_accel: type fixed, parent l_f3_1, child l_f3_1_accel, origin xyz=0.03 0 0 rpy=-1.5709 0 0
- added joint l_f3_2_accel: type fixed, parent l_f3_2, child l_f3_2_accel, origin xyz=0.04 0 0 rpy=-1.5709 0 0
- added joint l_f3_base: type fixed, parent l_palm, child l_f3_base, origin xyz=0.03995 -0.04383 0.014 rpy=0 -1.57079 -2.3562
- added joint l_f3_fixed_accel: type fixed, parent l_f3_base, child l_f3_fixed_accel, origin xyz=-0.05 0 0 rpy=0 0 0
- added joint l_f3_j0: type revolute, parent l_f3_base, child l_f3_0, origin xyz=0 0 0 rpy=0 0 0, axis 0 0 1, limit lower=-1.57079 upper=1.57079 effort=1 velocity=1
- added joint l_f3_j1: type revolute, parent l_f3_0, child l_f3_1, origin xyz=0.028 0 0 rpy=1.57079 0 0, axis 0 0 1, limit lower=-1.57079 upper=1.57079 effort=1 velocity=1
- added joint l_f3_j2: type revolute, parent l_f3_1, child l_f3_2, origin xyz=0.05 0 0 rpy=0 0 0, axis 0 0 1, limit lower=-1.57079 upper=1.57079 effort=1 velocity=1
- added joint l_sandia_hand_joint: type fixed, parent l_hand, child l_palm, origin xyz=0  0.1 -0.03 rpy=0 3.1416 -1.57079
- added joint r_f0_1_accel: type fixed, parent r_f0_1, child r_f0_1_accel, origin xyz=0.03 0 0 rpy=-1.5709 0 0
- added joint r_f0_2_accel: type fixed, parent r_f0_2, child r_f0_2_accel, origin xyz=0.04 0 0 rpy=-1.5709 0 0
- added joint r_f0_base: type fixed, parent r_palm, child r_f0_base, origin xyz=0.14 0.0 0 rpy=0 0 0.3
- added joint r_f0_fixed_accel: type fixed, parent r_f0_base, child r_f0_fixed_accel, origin xyz=-0.05 0 0 rpy=0 0 0
- added joint r_f0_j0: type revolute, parent r_f0_base, child r_f0_0, origin xyz=0 0 0 rpy=0 0 0, axis 0 0 1, limit lower=-1.57079 upper=1.57079 effort=1 velocity=1
- added joint r_f0_j1: type revolute, parent r_f0_0, child r_f0_1, origin xyz=0.028 0 0 rpy=1.57079 0 0, axis 0 0 1, limit lower=-1.57079 upper=1.57079 effort=1 velocity=1
- added joint r_f0_j2: type revolute, parent r_f0_1, child r_f0_2, origin xyz=0.05 0 0 rpy=0 0 0, axis 0 0 1, limit lower=-1.57079 upper=1.57079 effort=1 velocity=1
- added joint r_f1_1_accel: type fixed, parent r_f1_1, child r_f1_1_accel, origin xyz=0.03 0 0 rpy=-1.5709 0 0
- added joint r_f1_2_accel: type fixed, parent r_f1_2, child r_f1_2_accel, origin xyz=0.04 0 0 rpy=-1.5709 0 0
- added joint r_f1_base: type fixed, parent r_palm, child r_f1_base, origin xyz=0.115 0.03122 0 rpy=0 0 0.3
- added joint r_f1_fixed_accel: type fixed, parent r_f1_base, child r_f1_fixed_accel, origin xyz=-0.05 0 0 rpy=0 0 0
- added joint r_f1_j0: type revolute, parent r_f1_base, child r_f1_0, origin xyz=0 0 0 rpy=0 0 0, axis 0 0 1, limit lower=-1.57079 upper=1.57079 effort=1 velocity=1
- added joint r_f1_j1: type revolute, parent r_f1_0, child r_f1_1, origin xyz=0.028 0 0 rpy=1.57079 0 0, axis 0 0 1, limit lower=-1.57079 upper=1.57079 effort=1 velocity=1
- added joint r_f1_j2: type revolute, parent r_f1_1, child r_f1_2, origin xyz=0.05 0 0 rpy=0 0 0, axis 0 0 1, limit lower=-1.57079 upper=1.57079 effort=1 velocity=1
- added joint r_f2_1_accel: type fixed, parent r_f2_1, child r_f2_1_accel, origin xyz=0.03 0 0 rpy=-1.5709 0 0
- added joint r_f2_2_accel: type fixed, parent r_f2_2, child r_f2_2_accel, origin xyz=0.04 0 0 rpy=-1.5709 0 0
- added joint r_f2_base: type fixed, parent r_palm, child r_f2_base, origin xyz=0.09 0.06245 0 rpy=0 0 0.3
- added joint r_f2_fixed_accel: type fixed, parent r_f2_base, child r_f2_fixed_accel, origin xyz=-0.05 0 0 rpy=0 0 0
- added joint r_f2_j0: type revolute, parent r_f2_base, child r_f2_0, origin xyz=0 0 0 rpy=0 0 0, axis 0 0 1, limit lower=-1.57079 upper=1.57079 effort=1 velocity=1
- added joint r_f2_j1: type revolute, parent r_f2_0, child r_f2_1, origin xyz=0.028 0 0 rpy=1.57079 0 0, axis 0 0 1, limit lower=-1.57079 upper=1.57079 effort=1 velocity=1
- added joint r_f2_j2: type revolute, parent r_f2_1, child r_f2_2, origin xyz=0.05 0 0 rpy=0 0 0, axis 0 0 1, limit lower=-1.57079 upper=1.57079 effort=1 velocity=1
- added joint r_f3_1_accel: type fixed, parent r_f3_1, child r_f3_1_accel, origin xyz=0.03 0 0 rpy=-1.5709 0 0
- added joint r_f3_2_accel: type fixed, parent r_f3_2, child r_f3_2_accel, origin xyz=0.04 0 0 rpy=-1.5709 0 0
- added joint r_f3_base: type fixed, parent r_palm, child r_f3_base, origin xyz=0.03995 -0.04383 0.014 rpy=0 -1.57079 -2.3562
- added joint r_f3_fixed_accel: type fixed, parent r_f3_base, child r_f3_fixed_accel, origin xyz=-0.05 0 0 rpy=0 0 0
- added joint r_f3_j0: type revolute, parent r_f3_base, child r_f3_0, origin xyz=0 0 0 rpy=0 0 0, axis 0 0 1, limit lower=-1.57079 upper=1.57079 effort=1 velocity=1
- added joint r_f3_j1: type revolute, parent r_f3_0, child r_f3_1, origin xyz=0.028 0 0 rpy=1.57079 0 0, axis 0 0 1, limit lower=-1.57079 upper=1.57079 effort=1 velocity=1
- added joint r_f3_j2: type revolute, parent r_f3_1, child r_f3_2, origin xyz=0.05 0 0 rpy=0 0 0, axis 0 0 1, limit lower=-1.57079 upper=1.57079 effort=1 velocity=1
- added joint r_sandia_hand_joint: type fixed, parent r_hand, child r_palm, origin xyz=0 -0.1 -0.03 rpy=0 3.1416  1.57079

File: software/models/mit_gazebo_models/mit_robot_PnC/xacro/atlas_sandia_hands.model.xacro (robot description, xacro)
@@ -4,5 +4,5 @@
        xmlns:xacro="http://playerstage.sourceforge.net/gazebo/xmlschema/#interface"
        name="atlas" >
-  <include filename="$(find atlas_utils)/urdf/atlas.urdf" />
+  <include filename="$(find mit_drcsim_scripts)/models/mit_robot_PnC/xacro/atlas_skeleton.urdf" />
   <include filename="$(find sandia_hand_utils)/urdf/sandia_hand.urdf.xacro" />
   <xacro:sandia_hand side="r" parent="r_hand">
@@ -14,4 +14,5 @@
   <include filename="$(find atlas_utils)/urdf/atlas.transmission" />
   <include filename="$(find atlas_utils)/urdf/atlas.sensors" />
-  <include filename="$(find mit_drcsim_scripts)/models/mit_robot_PnC/xacro/mit_atlas.gazebo" />
+<!--  <include filename="$(find mit_drcsim_scripts)/models/mit_robot_PnC/xacro/mit_atlas.gazebo" /> -->
+  <include filename="$(find mit_drcsim_scripts)/models/mit_robot_PnC/xacro/mit_atlas_position_control.gazebo" />
 </robot>

Commit message: updating drake and PnC models for drcsim 2.0
git-svn-id: https://svn.csail.mit.edu/drc@1600 c7283977-0100-402a-a91a-fa70b306dbfe

File: software/models/mit_gazebo_models/mit_robot_PnC/model.urdf (robot description, URDF)
Before this commit: robot atlas, 41 links, 40 joints
Links:
- removed link head_hokuyo
- removed link head_imu_link
- added link head_hokuyo_frame, mass 0.01
- link head: geometry collision box size=0.0468 0.12 0.1184; collision box size=0.1311 0.12 0.0591
- link hokuyo_link: geometry collision box size=0.08 0.06 0.04238; collision cylinder length=0.047 radius=0.024425
- link l_clav: geometry collision cylinder length=0.027 radius=0.04; collision cylinder length=0.1525 radius=0.045
- link l_farm: geometry collision cylinder length=0.035181 radius=0.0458825; collision cylinder length=0.050472 radius=0.0279
- link l_foot: geometry collision box size=0.26 0.124887 0.01; visual mesh filename=package://mit_robot/meshes/l_foot.dae scale=1 1 1
- link l_hand: geometry collision cylinder length=0.019 radius=0.035939; collision cylinder length=0.019 radius=0.035939
- link l_larm: geometry collision cylinder length=0.0161 radius=0.045; collision cylinder length=0.0161 radius=0.045
- link l_lglut: geometry collision cylinder length=0.060306 radius=0.02009687; collision cylinder length=0.12 radius=0.02
- link l_lleg: geometry collision box size=0.1465 0.1205 0.476; visual mesh filename=package://mit_robot/meshes/l_lleg.dae scale=1 1 1
- link l_scap: geometry collision cylinder length=0.013737 radius=0.048709; collision cylinder length=0.013937 radius=0.048709
- link l_talus: geometry collision cylinder length=0.010059 radius=0.010348; collision cylinder length=0.029542 radius=0.010181
- link l_uarm: geometry collision cylinder length=0.088934 radius=0.04504847; collision cylinder length=0.116677 radius=0.0449
- link l_uglut: geometry collision cylinder length=0.078396 radius=0.019096; collision cylinder length=0.080842 radius=0.019841
- link l_uleg: geometry collision box size=0.2 0.1865 0.26; visual mesh filename=package://mit_robot/meshes/l_uleg.dae scale=1 1 1
- link ltorso: geometry visual mesh filename=package://mit_robot/meshes/ltorso.dae scale=1 1 1
- link mtorso: geometry collision cylinder length=0.02 radius=0.015; collision cylinder length=0.02 radius=0.015
- link pelvis: geometry collision cylinder length=0.07 radius=0.130; collision cylinder length=0.07 radius=0.130
- link r_clav: geometry collision cylinder length=0.027 radius=0.04; collision cylinder length=0.1525 radius=0.045
- link r_farm: geometry collision cylinder length=0.035181 radius=0.0458825; collision cylinder length=0.050472 radius=0.0279
- link r_foot: geometry collision box size=0.26 0.124887 0.01; visual mesh filename=package://mit_robot/meshes/r_foot.dae scale=1 1 1
- link r_hand: geometry collision cylinder length=0.019 radius=0.035939; collision cylinder length=0.019 radius=0.035939
- link r_larm: geometry collision cylinder length=0.0161 radius=0.045; collision cylinder length=0.0161 radius=0.045
- link r_lglut: geometry collision cylinder length=0.060306 radius=0.02009687; collision cylinder length=0.12 radius=0.02
- link r_lleg: geometry collision box size=0.1465 0.1205 0.476; visual mesh filename=package://mit_robot/meshes/r_lleg.dae scale=1 1 1
- link r_scap: geometry collision cylinder length=0.013737 radius=0.048709; collision cylinder length=0.013937 radius=0.048709
- link r_talus: geometry collision cylinder length=0.010059 radius=0.010348; collision cylinder length=0.029542 radius=0.010181
- link r_uarm: geometry collision cylinder length=0.088934 radius=0.04504847; collision cylinder length=0.116677 radius=0.0449
- link r_uglut: geometry collision cylinder length=0.078396 radius=0.019096; collision cylinder length=0.080842 radius=0.019841
- link r_uleg: geometry collision box size=0.2 0.1865 0.26; visual mesh filename=package://mit_robot/meshes/r_uleg.dae scale=1 1 1
- link utorso: geometry collision box size=0.3188 0.24 0.3662; collision cylinder length=0.22375 radius=0.0363
Joints:
- removed joint head_imu_joint
- joint head_hokuyo_joint: child head_hokuyo -> head_hokuyo_frame
- joint neck_ay: origin xyz=0.16555 0 0.50823 rpy=0 0 0 -> xyz=0.16555 0 0.50823 rpy=0 -0 0
- joint r_arm_usy: axis 0 -0.5 0.866025 -> 0 0.5 -0.866025

File: software/models/mit_gazebo_models/mit_robot_PnC/xacro/atlas_skeleton.urdf (robot description, URDF)
Before this commit: robot drc_skeleton, 30 links, 29 joints
Links:
- removed link head
- removed link hokuyo_link
- link l_clav: geometry collision cylinder length=0.027 radius=0.04; collision cylinder length=0.1525 radius=0.045
- link l_farm: geometry collision cylinder length=0.035181 radius=0.0458825; collision cylinder length=0.050472 radius=0.0279
- link l_foot: geometry collision box size=0.26 0.124887 0.01; visual mesh filename=package://mit_robot/meshes/l_foot.dae scale=1 1 1
- link l_hand: geometry collision cylinder length=0.019 radius=0.035939; collision cylinder length=0.019 radius=0.035939
- link l_larm: geometry collision cylinder length=0.0161 radius=0.045; collision cylinder length=0.0161 radius=0.045
- link l_lglut: geometry collision cylinder length=0.060306 radius=0.02009687; collision cylinder length=0.12 radius=0.02
- link l_lleg: geometry collision box size=0.1465 0.1205 0.476; visual mesh filename=package://mit_robot/meshes/l_lleg.dae scale=1 1 1
- link l_scap: geometry collision cylinder length=0.013737 radius=0.048709; collision cylinder length=0.013937 radius=0.048709
- link l_talus: geometry collision cylinder length=0.010059 radius=0.010348; collision cylinder length=0.029542 radius=0.010181
- link l_uarm: geometry collision cylinder length=0.088934 radius=0.04504847; collision cylinder length=0.116677 radius=0.0449
- link l_uglut: geometry collision cylinder length=0.078396 radius=0.019096; collision cylinder length=0.080842 radius=0.019841
- link l_uleg: geometry collision box size=0.2 0.1865 0.26; visual mesh filename=package://mit_robot/meshes/l_uleg.dae scale=1 1 1
- link ltorso: geometry visual mesh filename=package://mit_robot/meshes/ltorso.dae scale=1 1 1
- link mtorso: geometry collision cylinder length=0.02 radius=0.015; collision cylinder length=0.02 radius=0.015
- link pelvis: geometry collision cylinder length=0.07 radius=0.130; collision cylinder length=0.07 radius=0.130
- link r_clav: geometry collision cylinder length=0.027 radius=0.04; collision cylinder length=0.1525 radius=0.045
- link r_farm: geometry collision cylinder length=0.035181 radius=0.0458825; collision cylinder length=0.050472 radius=0.0279
- link r_foot: geometry collision box size=0.26 0.124887 0.01; visual mesh filename=package://mit_robot/meshes/r_foot.dae scale=1 1 1
- link r_hand: geometry collision cylinder length=0.019 radius=0.035939; collision cylinder length=0.019 radius=0.035939
- link r_larm: geometry collision cylinder length=0.0161 radius=0.045; collision cylinder length=0.0161 radius=0.045
- link r_lglut: geometry collision cylinder length=0.060306 radius=0.02009687; collision cylinder length=0.12 radius=0.02
- link r_lleg: geometry collision box size=0.1465 0.1205 0.476; visual mesh filename=package://mit_robot/meshes/r_lleg.dae scale=1 1 1
- link r_scap: geometry collision cylinder length=0.013737 radius=0.048709; collision cylinder length=0.013937 radius=0.048709
- link r_talus: geometry collision cylinder length=0.010059 radius=0.010348; collision cylinder length=0.029542 radius=0.010181
- link r_uarm: geometry collision cylinder length=0.088934 radius=0.04504847; collision cylinder length=0.116677 radius=0.0449
- link r_uglut: geometry collision cylinder length=0.078396 radius=0.019096; collision cylinder length=0.080842 radius=0.019841
- link r_uleg: geometry collision box size=0.2 0.1865 0.26; visual mesh filename=package://mit_robot/meshes/r_uleg.dae scale=1 1 1
- link utorso: geometry collision box size=0.3188 0.24 0.3662; collision cylinder length=0.22375 radius=0.0363
Joints:
- removed joint hokuyo_joint
- joint neck_ay: origin xyz=0.16555 0 0.50823 rpy=0 0 0 -> xyz=0.16555 0 0.50823 rpy=0 -0 0
- joint r_arm_usy: axis 0 -0.5 0.866025 -> 0 0.5 -0.866025

File: software/models/mit_gazebo_models/mit_robot_drake/model_minimal_contact.urdf (robot description, URDF)
Before this commit: robot atlas, 31 links, 30 joints
Joints:
- joint l_hand_joint: origin xyz=0.0089 0.1855 0.0047 rpy=0 0 0 -> xyz=0.0 0.15 0.0 rpy=0 0 0
- joint r_hand_joint: origin xyz=0.0089 -0.1855 -0.0047 rpy=0 0 0 -> xyz=0.0 -0.15 0.0 rpy=0 0 0

File: software/models/mit_gazebo_models/mit_robot_drake/xacro/atlas_point_mass_hands.urdf (robot description, URDF)
Before this commit: robot drc_skeleton, 2 links, 2 joints
Joints:
- joint l_hand_joint: origin xyz=0.0089 0.1855 0.0047 rpy=0 0 0 -> xyz=0.0 0.15 0.0 rpy=0 0 0
- joint r_hand_joint: origin xyz=0.0089 -0.1855 -0.0047 rpy=0 0 0 -> xyz=0.0 -0.15 0.0 rpy=0 0 0
