Commit message: PnC model has hands by default
git-svn-id: https://svn.csail.mit.edu/drc@1617 c7283977-0100-402a-a91a-fa70b306dbfe

File: software/models/mit_gazebo_models/mit_robot_PnC/model.urdf (robot description, URDF)
Before this commit: robot atlas, 40 links, 39 joints
Links:
- added link left_f0_0, mass 0.05; collision cylinder length=0.023 radius=0.01; collision cylinder length=0.023 radius=0.015
- added link left_f0_1, mass 0.05; collision cylinder length=0.067 radius=0.01; visual cylinder length=0.067 radius=0.01
- added link left_f0_1_accel, mass 0.001
- added link left_f0_2, mass 0.05; collision cylinder length=0.057 radius=0.009; collision sphere radius=0.009
- added link left_f0_2_accel, mass 0.001
- added link left_f0_base, mass 0.35
- added link left_f0_fixed_accel, mass 0.001
- added link left_f1_0, mass 0.05; collision cylinder length=0.023 radius=0.01; collision cylinder length=0.023 radius=0.015
- added link left_f1_1, mass 0.05; collision cylinder length=0.067 radius=0.01; visual cylinder length=0.067 radius=0.01
- added link left_f1_1_accel, mass 0.001
- added link left_f1_2, mass 0.05; collision cylinder length=0.057 radius=0.009; collision sphere radius=0.009
- added link left_f1_2_accel, mass 0.001
- added link left_f1_base, mass 0.35
- added link left_f1_fixed_accel, mass 0.001
- added link left_f2_0, mass 0.05; collision cylinder length=0.023 radius=0.01; collision cylinder length=0.023 radius=0.015
- added link left_f2_1, mass 0.05; collision cylinder length=0.067 radius=0.01; visual cylinder length=0.067 radius=0.01
- added link left_f2_1_accel, mass 0.001
- added link left_f2_2, mass 0.05; collision cylinder length=0.057 radius=0.009; collision sphere radius=0.009
- added link left_f2_2_accel, mass 0.001
- added link left_f2_base, mass 0.35
- added link left_f2_fixed_accel, mass 0.001
- added link left_f3_0, mass 0.05; collision cylinder length=0.023 radius=0.01; collision cylinder length=0.023 radius=0.015
- added link left_f3_1, mass 0.05; collision cylinder length=0.067 radius=0.01; visual cylinder length=0.067 radius=0.01
- added link left_f3_1_accel, mass 0.001
- added link left_f3_2, mass 0.05; collision cylinder length=0.057 radius=0.009; collision sphere radius=0.009
- added link left_f3_2_accel, mass 0.001
- added link left_f3_base, mass 0.35
- added link left_f3_fixed_accel, mass 0.001
- added link left_palm, mass 0.3; collision box size=0.09 .03 .06; collision box size=0.09 .03 .06
- added link right_f0_0, mass 0.05; collision cylinder length=0.023 radius=0.01; collision cylinder length=0.023 radius=0.015
- added link right_f0_1, mass 0.05; collision cylinder length=0.067 radius=0.01; visual cylinder length=0.067 radius=0.01
- added link right_f0_1_accel, mass 0.001
- added link right_f0_2, mass 0.05; collision cylinder length=0.057 radius=0.009; collision sphere radius=0.009
- added link right_f0_2_accel, mass 0.001
- added link right_f0_base, mass 0.35
- added link right_f0_fixed_accel, mass 0.001
- added link right_f1_0, mass 0.05; collision cylinder length=0.023 radius=0.01; collision cylinder length=0.023 radius=0.015
- added link right_f1_1, mass 0.05; collision cylinder length=0.067 radius=0.01; visual cylinder length=0.067 radius=0.01
- added link right_f1_1_accel, mass 0.001
- added link right_f1_2, mass 0.05; collision cylinder length=0.057 radius=0.009; collision sphere radius=0.009
- added link right_f1_2_accel, mass 0.001
- added link right_f1_base, mass 0.35
- added link right_f1_fixed_accel, mass 0.001
- added link right_f2_0, mass 0.05; collision cylinder length=0.023 radius=0.01; collision cylinder length=0.023 radius=0.015
- added link right_f2_1, mass 0.05; collision cylinder length=0.067 radius=0.01; visual cylinder length=0.067 radius=0.01
- added link right_f2_1_accel, mass 0.001
- added link right_f2_2, mass 0.05; collision cylinder length=0.057 radius=0.009; collision sphere radius=0.009
- added link right_f2_2_accel, mass 0.001
- added link right_f2_base, mass 0.35
- added link right_f2_fixed_accel, mass 0.001
- added link right_f3_0, mass 0.05; collision cylinder length=0.023 radius=0.01; collision cylinder length=0.023 radius=0.015
- added link right_f3_1, mass 0.05; collision cylinder length=0.067 radius=0.01; visual cylinder length=0.067 radius=0.01
- added link right_f3_1_accel, mass 0.001
- added link right_f3_2, mass 0.05; collision cylinder length=0.057 radius=0.009; collision sphere radius=0.009
- added link right_f3_2_accel, mass 0.001
- added link right_f3_base, mass 0.35
- added link right_f3_fixed_accel, mass 0.001
- added link right_palm, mass 0.3; collision box size=0.09 .03 .06; collision box size=0.09 .03 .06
Joints:
- added joint left_f0_1_accel: type fixed, parent left_f0_1, child left_f0_1_accel, origin xyz=0.03 0 0 rpy=-1.57079632679 0 0
- added joint left_f0_2_accel: type fixed, parent left_f0_2, child left_f0_2_accel, origin xyz=0.04 0 0 rpy=-1.57079632679 0 0
- added joint left_f0_base: type fixed, parent left_palm, child left_f0_base, origin xyz=0.14 0.0 0 rpy=0 0 -0.3
- added joint left_f0_fixed_accel: type fixed, parent left_f0_base, child left_f0_fixed_accel, origin xyz=-0.05 0 0 rpy=0 0 0
- added joint left_f0_j0: type revolute, parent left_f0_base, child left_f0_0, origin xyz=0 0 0 rpy=0 0 0, axis 0 0 -1, limit lower=-1.57079632679 upper=1.57079632679 effort=1 velocity=1
- added joint left_f0_j1: type revolute, parent left_f0_0, child left_f0_1, origin xyz=0.028 0 0 rpy=1.57079632679 0 0, axis 0 0 1, limit lower=-1.57079632679 upper=1.57079632679 effort=1 velocity=1
- added joint left_f0_j2: type revolute, parent left_f0_1, child left_f0_2, origin xyz=0.05 0 0 rpy=0 0 0, axis 0 0 1, limit lower=-1.57079632679 upper=1.57079632679 effort=1 velocity=1
- added joint left_f1_1_accel: type fixed, parent left_f1_1, child left_f1_1_accel, origin xyz=0.03 0 0 rpy=-1.57079632679 0 0
- added joint left_f1_2_accel: type fixed, parent left_f1_2, child left_f1_2_accel, origin xyz=0.04 0 0 rpy=-1.57079632679 0 0
- added joint left_f1_base: type fixed, parent left_palm, child left_f1_base, origin xyz=0.115 -0.03122 0 rpy=0 0 -0.3
- added joint left_f1_fixed_accel: type fixed, parent left_f1_base, child left_f1_fixed_accel, origin xyz=-0.05 0 0 rpy=0 0 0
- added joint left_f1_j0: type revolute, parent left_f1_base, child left_f1_0, origin xyz=0 0 0 rpy=0 0 0, axis 0 0 -1, limit lower=-1.57079632679 upper=1.57079632679 effort=1 velocity=1
- added joint left_f1_j1: type revolute, parent left_f1_0, child left_f1_1, origin xyz=0.028 0 0 rpy=1.57079632679 0 0, axis 0 0 1, limit lower=-1.57079632679 upper=1.57079632679 effort=1 velocity=1
- added joint left_f1_j2: type revolute, parent left_f1_1, child left_f1_2, origin xyz=0.05 0 0 rpy=0 0 0, axis 0 0 1, limit lower=-1.57079632679 upper=1.57079632679 effort=1 velocity=1
- added joint left_f2_1_accel: type fixed, parent left_f2_1, child left_f2_1_accel, origin xyz=0.03 0 0 rpy=-1.57079632679 0 0
- added joint left_f2_2_accel: type fixed, parent left_f2_2, child left_f2_2_accel, origin xyz=0.04 0 0 rpy=-1.57079632679 0 0
- added joint left_f2_base: type fixed, parent left_palm, child left_f2_base, origin xyz=0.09 -0.06245 0 rpy=0 0 -0.3
- added joint left_f2_fixed_accel: type fixed, parent left_f2_base, child left_f2_fixed_accel, origin xyz=-0.05 0 0 rpy=0 0 0
- added joint left_f2_j0: type revolute, parent left_f2_base, child left_f2_0, origin xyz=0 0 0 rpy=0 0 0, axis 0 0 -1, limit lower=-1.57079632679 upper=1.57079632679 effort=1 velocity=1
- added joint left_f2_j1: type revolute, parent left_f2_0, child left_f2_1, origin xyz=0.028 0 0 rpy=1.57079632679 0 0, axis 0 0 1, limit lower=-1.57079632679 upper=1.57079632679 effort=1 velocity=1
- added joint left_f2_j2: type revolute, parent left_f2_1, child left_f2_2, origin xyz=0.05 0 0 rpy=0 0 0, axis 0 0 1, limit lower=-1.57079632679 upper=1.57079632679 effort=1 velocity=1
- added joint left_f3_1_accel: type fixed, parent left_f3_1, child left_f3_1_accel, origin xyz=0.03 0 0 rpy=-1.57079632679 0 0
- added joint left_f3_2_accel: type fixed, parent left_f3_2, child left_f3_2_accel, origin xyz=0.04 0 0 rpy=-1.57079632679 0 0
- added joint left_f3_base: type fixed, parent left_palm, child left_f3_base, origin xyz=0.03995 0.04383 0.014 rpy=0 -1.57079632679 2.3562
- added joint left_f3_fixed_accel: type fixed, parent left_f3_base, child left_f3_fixed_accel, origin xyz=-0.05 0 0 rpy=0 0 0
- added joint left_f3_j0: type revolute, parent left_f3_base, child left_f3_0, origin xyz=0 0 0 rpy=0 0 0, axis 0 0 -1, limit lower=-1.57079632679 upper=1.57079632679 effort=1 velocity=1
- added joint left_f3_j1: type revolute, parent left_f3_0, child left_f3_1, origin xyz=0.028 0 0 rpy=1.57079632679 0 0, axis 0 0 1, limit lower=-1.57079632679 upper=1.57079632679 effort=1 velocity=1
- added joint left_f3_j2: type revolute, parent left_f3_1, child left_f3_2, origin xyz=0.05 0 0 rpy=0 0 0, axis 0 0 1, limit lower=-1.57079632679 upper=1.57079632679 effort=1 velocity=1
- added joint left_sandia_hand_joint: type fixed, parent l_hand, child left_palm, origin xyz=0  0.1 0 rpy= 1.57079 0  1.57079
- added joint right_f0_1_accel: type fixed, parent right_f0_1, child right_f0_1_accel, origin xyz=0.03 0 0 rpy=-1.57079632679 0 0
- added joint right_f0_2_accel: type fixed, parent right_f0_2, child right_f0_2_accel, origin xyz=0.04 0 0 rpy=-1.57079632679 0 0
- added joint right_f0_base: type fixed, parent right_palm, child right_f0_base, origin xyz=0.14 0.0 0 rpy=0 0 0.3
- added joint right_f0_fixed_accel: type fixed, parent right_f0_base, child right_f0_fixed_accel, origin xyz=-0.05 0 0 rpy=0 0 0
- added joint right_f0_j0: type revolute, parent right_f0_base, child right_f0_0, origin xyz=0 0 0 rpy=0 0 0, axis 0 0 1, limit lower=-1.57079632679 upper=1.57079632679 effort=1 velocity=1
- added joint right_f0_j1: type revolute, parent right_f0_0, child right_f0_1, origin xyz=0.028 0 0 rpy=1.57079632679 0 0, axis 0 0 1, limit lower=-1.57079632679 upper=1.57079632679 effort=1 velocity=1
- added joint right_f0_j2: type revolute, parent right_f0_1, child right_f0_2, origin xyz=0.05 0 0 rpy=0 0 0, axis 0 0 1, limit lower=-1.57079632679 upper=1.57079632679 effort=1 velocity=1
- added joint right_f1_1_accel: type fixed, parent right_f1_1, child right_f1_1_accel, origin xyz=0.03 0 0 rpy=-1.57079632679 0 0
- added joint right_f1_2_accel: type fixed, parent right_f1_2, child right_f1_2_accel, origin xyz=0.04 0 0 rpy=-1.57079632679 0 0
- added joint right_f1_base: type fixed, parent right_palm, child right_f1_base, origin xyz=0.115 0.03122 0 rpy=0 0 0.3
- added joint right_f1_fixed_accel: type fixed, parent right_f1_base, child right_f1_fixed_accel, origin xyz=-0.05 0 0 rpy=0 0 0
- added joint right_f1_j0: type revolute, parent right_f1_base, child right_f1_0, origin xyz=0 0 0 rpy=0 0 0, axis 0 0 1, limit lower=-1.57079632679 upper=1.57079632679 effort=1 velocity=1
- added joint right_f1_j1: type revolute, parent right_f1_0, child right_f1_1, origin xyz=0.028 0 0 rpy=1.57079632679 0 0, axis 0 0 1, limit lower=-1.57079632679 upper=1.57079632679 effort=1 velocity=1
- added joint right_f1_j2: type revolute, parent right_f1_1, child right_f1_2, origin xyz=0.05 0 0 rpy=0 0 0, axis 0 0 1, limit lower=-1.57079632679 upper=1.57079632679 effort=1 velocity=1
- added joint right_f2_1_accel: type fixed, parent right_f2_1, child right_f2_1_accel, origin xyz=0.03 0 0 rpy=-1.57079632679 0 0
- added joint right_f2_2_accel: type fixed, parent right_f2_2, child right_f2_2_accel, origin xyz=0.04 0 0 rpy=-1.57079632679 0 0
- added joint right_f2_base: type fixed, parent right_palm, child right_f2_base, origin xyz=0.09 0.06245 0 rpy=0 0 0.3
- added joint right_f2_fixed_accel: type fixed, parent right_f2_base, child right_f2_fixed_accel, origin xyz=-0.05 0 0 rpy=0 0 0
- added joint right_f2_j0: type revolute, parent right_f2_base, child right_f2_0, origin xyz=0 0 0 rpy=0 0 0, axis 0 0 1, limit lower=-1.57079632679 upper=1.57079632679 effort=1 velocity=1
- added joint right_f2_j1: type revolute, parent right_f2_0, child right_f2_1, origin xyz=0.028 0 0 rpy=1.57079632679 0 0, axis 0 0 1, limit lower=-1.57079632679 upper=1.57079632679 effort=1 velocity=1
- added joint right_f2_j2: type revolute, parent right_f2_1, child right_f2_2, origin xyz=0.05 0 0 rpy=0 0 0, axis 0 0 1, limit lower=-1.57079632679 upper=1.57079632679 effort=1 velocity=1
- added joint right_f3_1_accel: type fixed, parent right_f3_1, child right_f3_1_accel, origin xyz=0.03 0 0 rpy=-1.57079632679 0 0
- added joint right_f3_2_accel: type fixed, parent right_f3_2, child right_f3_2_accel, origin xyz=0.04 0 0 rpy=-1.57079632679 0 0
- added joint right_f3_base: type fixed, parent right_palm, child right_f3_base, origin xyz=0.03995 -0.04383 0.014 rpy=0 -1.57079632679 -2.3562
- added joint right_f3_fixed_accel: type fixed, parent right_f3_base, child right_f3_fixed_accel, origin xyz=-0.05 0 0 rpy=0 0 0
- added joint right_f3_j0: type revolute, parent right_f3_base, child right_f3_0, origin xyz=0 0 0 rpy=0 0 0, axis 0 0 1, limit lower=-1.57079632679 upper=1.57079632679 effort=1 velocity=1
- added joint right_f3_j1: type revolute, parent right_f3_0, child right_f3_1, origin xyz=0.028 0 0 rpy=1.57079632679 0 0, axis 0 0 1, limit lower=-1.57079632679 upper=1.57079632679 effort=1 velocity=1
- added joint right_f3_j2: type revolute, parent right_f3_1, child right_f3_2, origin xyz=0.05 0 0 rpy=0 0 0, axis 0 0 1, limit lower=-1.57079632679 upper=1.57079632679 effort=1 velocity=1
- added joint right_sandia_hand_joint: type fixed, parent r_hand, child right_palm, origin xyz=0 -0.1 0 rpy=-1.57079 0 -1.57079

File: software/models/mit_gazebo_models/mit_robot_PnC/xacro/atlas.urdf.xacro (robot description, xacro)
@@ -1,6 +1,17 @@
-<robot name="atlas" >
+<robot xmlns:xacro="http://playerstage.sourceforge.net/gazebo/xmlschema/#interface" name="atlas" >
   <include filename="$(find mit_drcsim_scripts)/models/mit_robot_PnC/xacro/atlas_skeleton.urdf" />
+  <include filename="$(find sandia_hand_description)/urdf/sandia_hand_simple_shapes.urdf.xacro" />
+  <xacro:sandia_hand side="right" parent="r_hand" reflect="1">
+    <origin xyz="0 -0.1 0" rpy="-1.57079 0 -1.57079"/>
+  </xacro:sandia_hand>
+  <xacro:sandia_hand side="left" parent="l_hand" reflect="-1">
+    <origin xyz="0  0.1 0" rpy=" 1.57079 0  1.57079"/>
+  </xacro:sandia_hand>
   <include filename="$(find mit_drcsim_scripts)/models/mit_robot_PnC/xacro/mit_atlas.gazebo" />
   <include filename="$(find atlas_description)/urdf/atlas.transmission" />
   <include filename="$(find mit_drcsim_scripts)/models/multisense_sl/multisense_sl.urdf" />
+  <gazebo>
+    <!-- include plugin for snadia hands -->
+    <plugin name="sandia_hand_plugin" filename="libSandiaHandPlugin.so"/>
+  </gazebo>
 </robot>

Commit message: git-svn-id: https://svn.csail.mit.edu/drc@1624 c7283977-0100-402a-a91a-fa70b306dbfe

File: software/models/mit_gazebo_models/mit_robot_PnC/model.urdf (robot description, URDF)
Before this commit: robot atlas, 98 links, 97 joints
Joints:
- joint imu_joint: axis 0 0 1 -> (none); limit lower=0 upper=0 effort=0 velocity=0 -> (none); type revolute -> fixed

Commit message: updating PnC model to atlas 2.2
git-svn-id: https://svn.csail.mit.edu/drc@2279 c7283977-0100-402a-a91a-fa70b306dbfe

File: software/models/mit_gazebo_models/mit_robot_PnC/model.urdf (robot description, URDF)
Before this commit: robot atlas, 98 links, 97 joints
Links:
- removed link left_f0_0
- removed link left_f0_1
- removed link left_f0_1_accel
- removed link left_f0_2
- removed link left_f0_2_accel
- removed link left_f0_base
- removed link left_f0_fixed_accel
- removed link left_f1_0
- removed link left_f1_1
- removed link left_f1_1_accel
- removed link left_f1_2
- removed link left_f1_2_accel
- removed link left_f1_base
- removed link left_f1_fixed_accel
- removed link left_f2_0
- removed link left_f2_1
- removed link left_f2_1_accel
- removed link left_f2_2
- removed link left_f2_2_accel
- removed link left_f2_base
- removed link left_f2_fixed_accel
- removed link left_f3_0
- removed link left_f3_1
- removed link left_f3_1_accel
- removed link left_f3_2
- removed link left_f3_2_accel
- removed link left_f3_base
- removed link left_f3_fixed_accel
- removed link left_palm
- removed link right_f0_0
- removed link right_f0_1
- removed link right_f0_1_accel
- removed link right_f0_2
- removed link right_f0_2_accel
- removed link right_f0_base
- removed link right_f0_fixed_accel
- removed link right_f1_0
- removed link right_f1_1
- removed link right_f1_1_accel
- removed link right_f1_2
- removed link right_f1_2_accel
- removed link right_f1_base
- removed link right_f1_fixed_accel
- removed link right_f2_0
- removed link right_f2_1
- removed link right_f2_1_accel
- removed link right_f2_2
- removed link right_f2_2_accel
- removed link right_f2_base
- removed link right_f2_fixed_accel
- removed link right_f3_0
- removed link right_f3_1
- removed link right_f3_1_accel
- removed link right_f3_2
- removed link right_f3_2_accel
- removed link right_f3_base
- removed link right_f3_fixed_accel
- removed link right_palm
- added link head_imu_link, mass 0.1; visual box size=0.01 0.01 0.01
- link imu_link: geometry visual box size=0.01 0.01 0.01
- link l_foot: mass 1.634 -> 0.817
- link l_larm: geometry collision cylinder length=0.0161 radius=0.045; collision cylinder length=0.0161 radius=0.045
- link l_lleg: geometry collision cylinder length=0.20 radius=0.06; collision cylinder length=0.22 radius=0.06
- link l_talus: mass 0.1 -> 0.817
- link l_uleg: geometry collision cylinder length=0.10 radius=0.1; collision cylinder length=0.15 radius=0.07
- link pelvis: geometry collision cylinder length=0.022 radius=0.130; collision cylinder length=0.022 radius=0.130
- link r_foot: mass 1.634 -> 0.817
- link r_larm: geometry collision cylinder length=0.0161 radius=0.045; collision cylinder length=0.0161 radius=0.045
- link r_lleg: geometry collision cylinder length=0.20 radius=0.06; collision cylinder length=0.22 radius=0.06
- link r_talus: mass 0.1 -> 0.817
- link r_uleg: geometry collision cylinder length=0.10 radius=0.1; collision cylinder length=0.15 radius=0.07
- link utorso: geometry collision box size=0.3188 0.24 0.3162; collision cylinder length=0.22375 radius=0.0363
Joints:
- removed joint left_f0_1_accel
- removed joint left_f0_2_accel
- removed joint left_f0_base
- removed joint left_f0_fixed_accel
- removed joint left_f0_j0
- removed joint left_f0_j1
- removed joint left_f0_j2
- removed joint left_f1_1_accel
- removed joint left_f1_2_accel
- removed joint left_f1_base
- removed joint left_f1_fixed_accel
- removed joint left_f1_j0
- removed joint left_f1_j1
- removed joint left_f1_j2
- removed joint left_f2_1_accel
- removed joint left_f2_2_accel
- removed joint left_f2_base
- removed joint left_f2_fixed_accel
- removed joint left_f2_j0
- removed joint left_f2_j1
- removed joint left_f2_j2
- removed joint left_f3_1_accel
- removed joint left_f3_2_accel
- removed joint left_f3_base
- removed joint left_f3_fixed_accel
- removed joint left_f3_j0
- removed joint left_f3_j1
- removed joint left_f3_j2
- removed joint left_sandia_hand_joint
- removed joint right_f0_1_accel
- removed joint right_f0_2_accel
- removed joint right_f0_base
- removed joint right_f0_fixed_accel
- removed joint right_f0_j0
- removed joint right_f0_j1
- removed joint right_f0_j2
- removed joint right_f1_1_accel
- removed joint right_f1_2_accel
- removed joint right_f1_base
- removed joint right_f1_fixed_accel
- removed joint right_f1_j0
- removed joint right_f1_j1
- removed joint right_f1_j2
- removed joint right_f2_1_accel
- removed joint right_f2_2_accel
- removed joint right_f2_base
- removed joint right_f2_fixed_accel
- removed joint right_f2_j0
- removed joint right_f2_j1
- removed joint right_f2_j2
- removed joint right_f3_1_accel
- removed joint right_f3_2_accel
- removed joint right_f3_base
- removed joint right_f3_fixed_accel
- removed joint right_f3_j0
- removed joint right_f3_j1
- removed joint right_f3_j2
- removed joint right_sandia_hand_joint
- added joint head_imu_joint: type fixed, parent head, child head_imu_link, origin xyz=-0.0475 0.035 0.0 rpy=0 0 0

File: software/models/mit_gazebo_models/mit_robot_PnC/xacro/atlas_skeleton.urdf (robot description, URDF)
Before this commit: robot drc_skeleton, 28 links, 28 joints
Links:
- link l_foot: mass 1.634 -> 0.817
- link l_larm: geometry collision cylinder length=0.0161 radius=0.045; collision cylinder length=0.0161 radius=0.045
- link l_lleg: geometry collision cylinder length=0.20 radius=0.06; collision cylinder length=0.22 radius=0.06
- link l_talus: mass 0.1 -> 0.817
- link l_uleg: geometry collision cylinder length=0.10 radius=0.1; collision cylinder length=0.15 radius=0.07
- link pelvis: geometry collision cylinder length=0.022 radius=0.130; collision cylinder length=0.022 radius=0.130
- link r_foot: mass 1.634 -> 0.817
- link r_larm: geometry collision cylinder length=0.0161 radius=0.045; collision cylinder length=0.0161 radius=0.045
- link r_lleg: geometry collision cylinder length=0.20 radius=0.06; collision cylinder length=0.22 radius=0.06
- link r_talus: mass 0.1 -> 0.817
- link r_uleg: geometry collision cylinder length=0.10 radius=0.1; collision cylinder length=0.15 radius=0.07
- link utorso: geometry collision box size=0.3188 0.24 0.3162; collision cylinder length=0.22375 radius=0.0363
