Commit message: Adds simplified polaris models for use with Drake
git-svn-id: https://svn.csail.mit.edu/drc@3168 c7283977-0100-402a-a91a-fa70b306dbfe

File: software/models/mit_gazebo_objects/mit_polaris_ranger_ev/model_welded.urdf (robot description, URDF)
Before this commit: robot polaris_ranger_ev, 5 links, 4 joints
Links:
- removed link brake_pedal
- removed link gas_pedal
- removed link hand_brake
- removed link steering_wheel
- link chassis: geometry collision box size=0.05 1.2 0.25; collision box size=0.05 1.2 0.25
Joints:
- removed joint brake_joint
- removed joint gas_joint
- removed joint hand_brake_joint
- removed joint steering_joint
