Commit message: minor updates to drake component files. added small mass to pelvis to account for IMU link. added small mass to head to account for deleted hokuyo sensor. updated point hand mass values based on sisir's data from new hand models---COM locations still need to be updated.
git-svn-id: https://svn.csail.mit.edu/drc@3410 c7283977-0100-402a-a91a-fa70b306dbfe

File: software/models/mit_gazebo_models/mit_robot_drake/xacro/atlas_skeleton_minimal_contact.urdf (robot description, URDF)
Before this commit: robot drc_skeleton, 28 links, 28 joints
Links:
- link pelvis: mass 12.54638 -> 12.64638

File: software/models/mit_gazebo_models/mit_robot_drake/xacro/multisense_sl_no_contact.urdf (robot description, URDF)
Before this commit: robot multisense_sl, 1 links, 0 joints
Links:
- link head: mass 1.4199 -> 1.477574

File: software/models/mit_gazebo_models/mit_robot_drake/xacro/point_mass_hands.urdf (robot description, URDF)
Before this commit: robot drc_skeleton, 2 links, 2 joints
Links:
- link l_hand_point_mass: mass 3.1690 -> 3.111
- link r_hand_point_mass: mass 3.1690 -> 3.111
