Commit message: Adds simple_visuals version of atlas model for use in authoring.
git-svn-id: https://svn.csail.mit.edu/drc@3771 c7283977-0100-402a-a91a-fa70b306dbfe

File: software/models/mit_gazebo_models/mit_robot_drake/xacro/atlas_skeleton_simple_visuals_minimal_contact.urdf (robot description, URDF)
Before this commit: robot drc_skeleton, 28 links, 28 joints
Links:
- removed link None
- added link l_uleg, mass 7.227; collision sphere radius=0; collision sphere radius=0
- link pelvis: geometry collision sphere radius=0; collision sphere radius=0
- link r_uleg: geometry collision sphere radius=0; collision sphere radius=0
- link utorso: geometry collision sphere radius=0; collision sphere radius=0
