Commit message: Adds contact points to simple_visuals skeleton
git-svn-id: https://svn.csail.mit.edu/drc@3904 c7283977-0100-402a-a91a-fa70b306dbfe

File: software/models/mit_gazebo_models/mit_robot_drake/xacro/atlas_skeleton_simple_visuals.urdf (robot description, URDF)
Before this commit: robot drc_skeleton, 28 links, 28 joints
Links:
- link l_clav: geometry 
- link l_farm: geometry 
- link l_foot: geometry 
- link l_hand: geometry 
- link l_larm: geometry 
- link l_lglut: geometry 
- link l_scap: geometry collision cylinder length=0.125 radius=0.045; visual box size=0.15 0.15 0.06
- link l_talus: geometry collision cylinder length=0.029542 radius=0.010181; visual cylinder length=0.010059 radius=0.010348
- link l_uarm: geometry collision cylinder length=0.125 radius=0.045; visual box size=0.04 0.07 0.13
- link l_uglut: geometry collision cylinder length=0.078396 radius=0.019096; visual cylinder length=0.078396 radius=0.019096
- link l_uleg: geometry collision cylinder length=0.10 radius=0.1; collision cylinder length=0.15 radius=0.07
- link pelvis: geometry collision box size=0.1 0.15 0.2; collision box size=0.1 0.15 0.2
- link r_foot: geometry collision box size=0.26 0.124887 0.05; visual box size=0.26 0.124887 0.05
