Commit message: Moved point mass sandia left hand to align with stump mesh, mirroring right. Flipped visual object of right hand to face the correct direction.
git-svn-id: https://svn.csail.mit.edu/drc/trunk@6716 c7283977-0100-402a-a91a-fa70b306dbfe

File: software/models/mit_gazebo_models/mit_robot_drake/xacro/point_mass_sandia_hands.urdf (robot description, URDF)
Before this commit: robot drc_skeleton, 2 links, 2 joints
Joints:
- joint l_hand_joint: origin xyz=0.0037 0.1603 -0.0087 rpy=0 0 0 -> xyz=-0.0037 0.1603 0.0087 rpy=0 0 0
