Commit message: Add all 9 types of robot. The irobot hand is still missing in URDF
git-svn-id: https://svn.csail.mit.edu/drc/trunk@7113 c7283977-0100-402a-a91a-fa70b306dbfe

File: software/models/mit_gazebo_models/mit_robot_drake/xacro/atlas_LS_RI.urdf.xacro (robot description, xacro)
@@ -2,7 +2,6 @@
   <include filename="$(find mit_drcsim_scripts)/models/mit_robot_drake/xacro/atlas_skeleton_minimal_contact.urdf" />
   <include filename="$(find sandia_hand_description)/urdf/sandia_hand_simple_shapes.urdf.xacro" />
-  <!-- adding an offset in the urdf to account for the ft sensor and the coupling plate, chaning origin form 0.1 to 0.145 for sandia, and 0.05 to 0.095 for irobot-->
-  <xacro:sandia_hand side="right" parent="r_hand" reflect="1" joint_type="revolute" thumb_angle="0">
-    <origin xyz="0 -0.145 0" rpy="0.0 0 -1.57079"/>
+  <xacro:sandia_hand side="left" parent="l_hand" reflect="-1" joint_type="revolute" thumb_angle="0">
+    <origin xyz="0.00179  0.13516 0.01176" rpy="0 0  1.57079"/>
   </xacro:sandia_hand>
   <include filename="$(find mit_drcsim_scripts)/models/mit_robot_drake/xacro/atlas.transmission" />
