Commit message: Update mit_robot_drake/xacro

File: software/models/mit_gazebo_models/mit_robot_drake/xacro/atlas.urdf.xacro (robot description, xacro)
@@ -1,5 +1,6 @@
-<robot name="atlas" >
-  <include filename="$(find mit_drcsim_scripts)/models/mit_robot_drake/xacro/atlas_skeleton_minimal_contact.urdf" />
-  <include filename="$(find mit_drcsim_scripts)/models/mit_robot_drake/xacro/atlas.transmission" />
-  <include filename="$(find mit_drcsim_scripts)/models/mit_robot_drake/xacro/multisense_sl_no_contact.urdf" />
+<robot name="atlas" xmlns:xacro="http://www.ros.org/wiki/xacro">
+  <xacro:include filename="$(find mit_drcsim_scripts)/models/mit_robot_drake/xacro/atlas_skeleton.xacro" />
+  <xacro:atlas_skeleton minimal_contact="true"/>
+  <xacro:include filename="$(find mit_drcsim_scripts)/models/mit_robot_drake/xacro/atlas.transmission" />
+  <xacro:include filename="$(find mit_drcsim_scripts)/models/mit_robot_drake/xacro/multisense_sl_no_contact.urdf" />
 </robot>

File: software/models/mit_gazebo_models/mit_robot_drake/xacro/atlas_convex_hull_no_hands.urdf.xacro (robot description, xacro)
@@ -1,5 +1,6 @@
-<robot name="atlas" >
-  <include filename="$(find mit_drcsim_scripts)/models/mit_robot_drake/xacro/atlas_skeleton.urdf" />
-  <include filename="$(find mit_drcsim_scripts)/models/mit_robot_drake/xacro/atlas.transmission" />
-  <include filename="$(find mit_drcsim_scripts)/models/mit_robot_drake/xacro/multisense_sl_no_contact.urdf" />
+<robot xmlns:xacro="http://www.ros.org/wiki/xacro" name="atlas" >
+  <xacro:include filename="$(find mit_drcsim_scripts)/models/mit_robot_drake/xacro/atlas_skeleton.xacro" />
+  <xacro:atlas_skeleton minimal_contact="false"/>
+  <xacro:include filename="$(find mit_drcsim_scripts)/models/mit_robot_drake/xacro/atlas.transmission" />
+  <xacro:include filename="$(find mit_drcsim_scripts)/models/mit_robot_drake/xacro/multisense_sl_no_contact.urdf" />
 </robot>

File: software/models/mit_gazebo_models/mit_robot_drake/xacro/atlas_convex_hull_robotiq_hands.urdf.xacro (robot description, xacro)
@@ -1,5 +1,8 @@
 <robot xmlns:xacro="http://www.ros.org/wiki/xacro" name="atlas" >
   <xacro:include filename="$(find mit_drcsim_scripts)/models/mit_robot_drake/xacro/atlas_skeleton.xacro" />
-  <xacro:atlas_skeleton minimal_contact="true"/>
+  <xacro:atlas_skeleton minimal_contact="false"/>
+  <xacro:include filename="$(find mit_drcsim_scripts)/models/mit_robot_drake/xacro/robotiq_convex_hull.xacro" />
+  <xacro:robotiq_convex_hull is_left="true"/>
+  <xacro:robotiq_convex_hull is_left="false"/>
   <xacro:include filename="$(find mit_drcsim_scripts)/models/mit_robot_drake/xacro/point_mass_robotiq_hands.urdf" />
   <xacro:include filename="$(find mit_drcsim_scripts)/models/mit_robot_drake/xacro/atlas.transmission" />

File: software/models/mit_gazebo_models/mit_robot_drake/xacro/atlas_point_stumps.urdf.xacro (robot description, xacro)
@@ -1,6 +1,7 @@
-<robot name="atlas" >
-  <include filename="$(find mit_drcsim_scripts)/models/mit_robot_drake/xacro/atlas_skeleton_minimal_contact.urdf" />
-  <include filename="$(find mit_drcsim_scripts)/models/mit_robot_drake/xacro/point_mass_stumps.urdf" />
-  <include filename="$(find mit_drcsim_scripts)/models/mit_robot_drake/xacro/atlas.transmission" />
-  <include filename="$(find mit_drcsim_scripts)/models/mit_robot_drake/xacro/multisense_sl_no_contact.urdf" />
+<robot xmlns:xacro="http://www.ros.org/wiki/xacro" name="atlas" >
+  <xacro:include filename="$(find mit_drcsim_scripts)/models/mit_robot_drake/xacro/atlas_skeleton.xacro" />
+  <xacro:atlas_skeleton minimal_contact="true"/>
+  <xacro:include filename="$(find mit_drcsim_scripts)/models/mit_robot_drake/xacro/point_mass_stumps.urdf" />
+  <xacro:include filename="$(find mit_drcsim_scripts)/models/mit_robot_drake/xacro/atlas.transmission" />
+  <xacro:include filename="$(find mit_drcsim_scripts)/models/mit_robot_drake/xacro/multisense_sl_no_contact.urdf" />
 </robot>

File: software/models/mit_gazebo_models/mit_robot_drake/xacro/atlas_skeleton.xacro (robot description, xacro)
@@ -1,17 +1,20 @@
 <robot name="drc_skeleton" xmlns:xacro="http://www.ros.org/wiki/xacro">
-  <xacro:macro name="collision_point" params="group xyz visualize">
-    <collision group="${group}">
-      <origin rpy="0 0 0" xyz="${xyz}"/>
-      <geometry>
-        <sphere radius="0"/>
-      </geometry>
-    </collision>
-    <visual>
-      <origin rpy="0 0 0" xyz="${xyz}"/>
-      <geometry>
-        <sphere radius="${visualize*0.01}"/>
-      </geometry>
-    </visual>
+  <xacro:macro name="collision_point" params="group xyz visualize enable">
+    <xacro:if value="${enable}">
+      <collision group="${group}">
+        <origin rpy="0 0 0" xyz="${xyz}"/>
+        <geometry>
+          <sphere radius="0"/>
+        </geometry>
+      </collision>
+      <visual>
+        <origin rpy="0 0 0" xyz="${xyz}"/>
+        <geometry>
+          <sphere radius="${visualize*0.01}"/>
+        </geometry>
+      </visual>
+    </xacro:if>
   </xacro:macro>
+  <xacro:macro name="atlas_skeleton" params="minimal_contact">
     <link name="l_clav">
         <inertial>
@@ -20,10 +23,28 @@
             <inertia ixx="0.011" ixy="0" ixz="0" iyy="0.009" iyz="-0.004" izz="0.004" />
         </inertial>
-        <visual>
-            <origin xyz="0 0 0" rpy="0 -0 0" />
-            <geometry>
-                <mesh filename="package://mit_drcsim_scripts/models/mit_robot/meshes/l_clav.wrl" scale="1 1 1" />
-            </geometry>
-        </visual>
+        <xacro:if value="${minimal_contact}">
+          <visual>
+            <origin xyz="0 0 0" rpy="0 -0 0" />
+            <geometry>
+              <mesh filename="package://mit_drcsim_scripts/models/mit_robot/meshes/l_clav.wrl" scale="1 1 1" />
+            </geometry>
+          </visual>
+        </xacro:if>
+        <xacro:unless value="${minimal_contact}">
+          <visual>
+            <origin xyz="0 0 0" rpy="0 -0 0"/>
+            <geometry>
+              <mesh filename="package://mit_drcsim_scripts/models/mit_robot/meshes/l_clav_chull.wrl"
+                scale="1 1 1"/>
+            </geometry>
+          </visual>
+          <collision>
+            <origin xyz="0 0 0" rpy="0 -0 0"/>
+            <geometry>
+              <mesh filename="package://mit_drcsim_scripts/models/mit_robot/meshes/l_clav_chull.wrl"
+                scale="1 1 1"/>
+            </geometry>
+          </collision>
+        </xacro:unless>
     </link>
     <link name="l_farm">
@@ -33,10 +54,28 @@
             <inertia ixx="0.00656" ixy="0" ixz="0" iyy="0.00358" iyz="0" izz="0.00656" />
         </inertial>
-        <visual>
-            <origin xyz="0 0 0" rpy="0 -0 0" />
-            <geometry>
-                <mesh filename="package://mit_drcsim_scripts/models/mit_robot/meshes/l_farm.wrl" scale="1 1 1" />
-            </geometry>
-        </visual>
+        <xacro:if value="${minimal_contact}">
+          <visual>
+            <origin xyz="0 0 0" rpy="0 -0 0" />
+            <geometry>
+              <mesh filename="package://mit_drcsim_scripts/models/mit_robot/meshes/l_farm.wrl" scale="1 1 1" />
+            </geometry>
+          </visual>
+        </xacro:if>
+        <xacro:unless value="${minimal_contact}">
+          <visual>
+            <origin xyz="0 0 0" rpy="0 -0 0"/>
+            <geometry>
+              <mesh filename="package://mit_drcsim_scripts/models/mit_robot/meshes/l_farm_chull.wrl"
+                scale="1 1 1"/>
+            </geometry>
+          </visual>
+          <collision>
+            <origin xyz="0 0 0" rpy="0 -0 0"/>
+            <geometry>
+              <mesh filename="package://mit_drcsim_scripts/models/mit_robot/meshes/l_farm_chull.wrl"
+                scale="1 1 1"/>
+            </geometry>
+          </collision>
+        </xacro:unless>
     </link>
     <link name="l_foot">
@@ -46,14 +85,32 @@
             <inertia ixx="0.002" ixy="0" ixz="0" iyy="0.007" iyz="0" izz="0.008" />
         </inertial>
-        <visual>
-            <origin xyz="0 0 0" rpy="0 -0 0" />
-            <geometry>
-                <mesh filename="package://mit_drcsim_scripts/models/mit_robot/meshes/l_foot.wrl" scale="1 1 1" />
-            </geometry>
-        </visual>
-        <xacro:collision_point group="heel" xyz="-0.082 0.0624435 -0.081119" visualize="1"/>
-        <xacro:collision_point group="heel" xyz="-0.082 -0.0624435 -0.081119" visualize="1"/>
-        <xacro:collision_point group="toe" xyz="0.178 0.0624435 -0.081119" visualize="1"/>
-        <xacro:collision_point group="toe" xyz="0.178 -0.0624435 -0.081119" visualize="1"/>
+        <xacro:if value="${minimal_contact}">
+          <visual>
+            <origin xyz="0 0 0" rpy="0 -0 0" />
+            <geometry>
+              <mesh filename="package://mit_drcsim_scripts/models/mit_robot/meshes/l_foot.wrl" scale="1 1 1" />
+            </geometry>
+          </visual>
+        </xacro:if>
+        <xacro:unless value="${minimal_contact}">
+          <visual>
+            <origin xyz="0 0 0" rpy="0 -0 0"/>
+            <geometry>
+              <mesh filename="package://mit_drcsim_scripts/models/mit_robot/meshes/l_foot_chull.wrl"
+                scale="1 1 1"/>
+            </geometry>
+          </visual>
+          <collision>
+            <origin xyz="0 0 0" rpy="0 -0 0"/>
+            <geometry>
+              <mesh filename="package://mit_drcsim_scripts/models/mit_robot/meshes/l_foot_chull.wrl"
+                scale="1 1 1"/>
+            </geometry>
+          </collision>
+        </xacro:unless>
+        <xacro:collision_point group="heel" xyz="-0.082 0.0624435 -0.081119" visualize="1" enable="1"/>
+        <xacro:collision_point group="heel" xyz="-0.082 -0.0624435 -0.081119" visualize="1" enable="1"/>
+        <xacro:collision_point group="toe" xyz="0.178 0.0624435 -0.081119" visualize="1" enable="1"/>
+        <xacro:collision_point group="toe" xyz="0.178 -0.0624435 -0.081119" visualize="1" enable="1"/>
         <!--<xacro:collision_point group="heel_mid" xyz="-0.082 0 -0.081119" visualize="1"/>-->
         <!--<xacro:collision_point group="toe_mid" xyz="0.178 0 -0.081119" visualize="1"/>-->
@@ -70,12 +127,30 @@
             <inertia ixx="0.00265" ixy="0" ixz="0" iyy="0.00446" iyz="0" izz="0.00446" />
         </inertial>
-        <visual>
-            <origin xyz="0 0 0" rpy="0 -0 0" />
-            <geometry>
-                <mesh filename="package://mit_drcsim_scripts/models/mit_robot/meshes/l_hand.wrl" scale="1 1 1" />
-            </geometry>
-        </visual>
-        <xacro:collision_point group="default" xyz="0.0 0.115 0.0" visualize="1"/>
-        <xacro:collision_point group="knuckle" xyz="0 0.26 0.0" visualize="1"/>
+        <xacro:if value="${minimal_contact}">
+          <visual>
+            <origin xyz="0 0 0" rpy="0 -0 0" />
+            <geometry>
+              <mesh filename="package://mit_drcsim_scripts/models/mit_robot/meshes/l_hand.wrl" scale="1 1 1" />
+            </geometry>
+          </visual>
+        </xacro:if>
+        <xacro:unless value="${minimal_contact}">
+          <visual>
+            <origin xyz="0 0 0" rpy="0 -0 0"/>
+            <geometry>
+              <mesh filename="package://mit_drcsim_scripts/models/mit_robot/meshes/l_hand_chull.wrl"
+                scale="1 1 1"/>
+            </geometry>
+          </visual>
+          <collision>
+            <origin xyz="0 0 0" rpy="0 -0 0"/>
+            <geometry>
+              <mesh filename="package://mit_drcsim_scripts/models/mit_robot/meshes/l_hand_chull.wrl"
+                scale="1 1 1"/>
+            </geometry>
+          </collision>
+        </xacro:unless>
+        <xacro:collision_point group="default" xyz="0.0 0.115 0.0" visualize="1" enable="${minimal_contact}"/>
+        <xacro:collision_point group="knuckle" xyz="0 0.26 0.0" visualize="1" enable="${minimal_contact}"/>
     </link>
     <link name="l_larm">
@@ -85,10 +160,28 @@
             <inertia ixx="0.00265" ixy="0" ixz="0" iyy="0.00446" iyz="0" izz="0.00446" />
         </inertial>
-        <visual>
+        <xacro:if value="${minimal_contact}">
+          <visual>
             <origin xyz="0 0 0" rpy="0 3.14159 0" />
             <geometry>
-                <mesh filename="package://mit_drcsim_scripts/models/mit_robot/meshes/l_elbow_rx.wrl" scale="1 1 1" />
-            </geometry>
-        </visual>
+              <mesh filename="package://mit_drcsim_scripts/models/mit_robot/meshes/l_elbow_rx.wrl" scale="1 1 1" />
+            </geometry>
+          </visual>
+        </xacro:if>
+        <xacro:unless value="${minimal_contact}">
+          <visual>
+            <origin xyz="0 0 0" rpy="0 -0 0"/>
+            <geometry>
+              <mesh filename="package://mit_drcsim_scripts/models/mit_robot/meshes/l_elbow_rx_chull.wrl"
+                scale="1 1 1"/>
+            </geometry>
+          </visual>
+          <collision>
+            <origin xyz="0 0 0" rpy="0 -0 0"/>
+            <geometry>
+              <mesh filename="package://mit_drcsim_scripts/models/mit_robot/meshes/l_elbow_rx_chull.wrl"
+                scale="1 1 1"/>
+            </geometry>
+          </collision>
+        </xacro:unless>
     </link>
     <link name="l_lglut">
@@ -98,10 +191,12 @@
             <inertia ixx="0.000691326" ixy="-2.24344e-05" ixz="2.50508e-06" iyy="0.00126856" iyz="0.000137862" izz="0.00106487" />
         </inertial>
-        <visual>
-            <origin xyz="0 0 0" rpy="0 -0 0" />
-            <geometry>
-                <mesh filename="package://mit_drcsim_scripts/models/mit_robot/meshes/l_lglut.wrl" scale="1 1 1" />
-            </geometry>
-        </visual>
+        <xacro:if value="${minimal_contact}">
+          <visual>
+            <origin xyz="0 0 0" rpy="0 -0 0" />
+            <geometry>
+              <mesh filename="package://mit_drcsim_scripts/models/mit_robot/meshes/l_lglut.wrl" scale="1 1 1" />
+            </geometry>
+          </visual>
+        </xacro:if>
     </link>
     <link name="l_lleg">
@@ -111,11 +206,29 @@
             <inertia ixx="0.077" ixy="0" ixz="-0.003" iyy="0.076" iyz="0" izz="0.01" />
         </inertial>
-        <visual>
-            <origin xyz="0 0 0" rpy="0 -0 0" />
-            <geometry>
-                <mesh filename="package://mit_drcsim_scripts/models/mit_robot/meshes/l_lleg.wrl" scale="1 1 1" />
-            </geometry>
-        </visual>
-        <xacro:collision_point group="knee" xyz="0.1096 0.0029 0.012" visualize="1"/>
+        <xacro:if value="${minimal_contact}">
+          <visual>
+            <origin xyz="0 0 0" rpy="0 -0 0" />
+            <geometry>
+              <mesh filename="package://mit_drcsim_scripts/models/mit_robot/meshes/l_lleg.wrl" scale="1 1 1" />
+            </geometry>
+          </visual>
+        </xacro:if>
+        <xacro:collision_point group="knee" xyz="0.1096 0.0029 0.012" visualize="1" enable="${minimal_contact}"/>
+        <xacro:unless value="${minimal_contact}">
+          <visual>
+            <origin xyz="0 0 0" rpy="0 -0 0"/>
+            <geometry>
+              <mesh filename="package://mit_drcsim_scripts/models/mit_robot/meshes/l_lleg_chull.wrl"
+                scale="1 1 1"/>
+            </geometry>
+          </visual>
+          <collision>
+            <origin xyz="0 0 0" rpy="0 -0 0"/>
+            <geometry>
+              <mesh filename="package://mit_drcsim_scripts/models/mit_robot/meshes/l_lleg_chull.wrl"
+                scale="1 1 1"/>
+            </geometry>
+          </collision>
+        </xacro:unless>
     </link>
     <link name="l_scap">
@@ -125,10 +238,28 @@
             <inertia ixx="0.00319" ixy="0" ixz="0" iyy="0.00583" iyz="0" izz="0.00583" />
         </inertial>
-        <visual>
-            <origin xyz="0 0 0" rpy="0 -0 0" />
-            <geometry>
-                <mesh filename="package://mit_drcsim_scripts/models/mit_robot/meshes/l_sh_rx.wrl" scale="1 1 1" />
-            </geometry>
-        </visual>
+        <xacro:if value="${minimal_contact}">
+          <visual>
+            <origin xyz="0 0 0" rpy="0 -0 0" />
+            <geometry>
+              <mesh filename="package://mit_drcsim_scripts/models/mit_robot/meshes/l_sh_rx.wrl" scale="1 1 1" />
+            </geometry>
+          </visual>
+        </xacro:if>
+        <xacro:unless value="${minimal_contact}">
+          <visual>
+            <origin xyz="0 0 0" rpy="0 -0 0"/>
+            <geometry>
+              <mesh filename="package://mit_drcsim_scripts/models/mit_robot/meshes/l_sh_rx_chull.wrl"
+                scale="1 1 1"/>
+            </geometry>
+          </visual>
+          <collision>
+            <origin xyz="0 0 0" rpy="0 -0 0"/>
+            <geometry>
+              <mesh filename="package://mit_drcsim_scripts/models/mit_robot/meshes/l_sh_rx_chull.wrl"
+                scale="1 1 1"/>
+            </geometry>
+          </collision>
+        </xacro:unless>
     </link>
     <link name="l_talus">
@@ -138,10 +269,12 @@
             <inertia ixx="1.01674e-05" ixy="0" ixz="0" iyy="8.42775e-06" iyz="0" izz="1.30101e-05" />
         </inertial>
-        <visual>
-            <origin xyz="0 0 0" rpy="0 -0 0" />
-            <geometry>
-                <mesh filename="package://mit_drcsim_scripts/models/mit_robot/meshes/l_talus.wrl" scale="1 1 1" />
-            </geometry>
-        </visual>
+        <xacro:if value="${minimal_contact}">
+          <visual>
+            <origin xyz="0 0 0" rpy="0 -0 0" />
+            <geometry>
+              <mesh filename="package://mit_drcsim_scripts/models/mit_robot/meshes/l_talus.wrl" scale="1 1 1" />
+            </geometry>
+          </visual>
+        </xacro:if>
     </link>
     <link name="l_uarm">
@@ -151,10 +284,28 @@
             <inertia ixx="0.00656" ixy="0" ixz="0" iyy="0.00358" iyz="0" izz="0.00656" />
         </inertial>
-        <visual>
-            <origin xyz="0 0 0" rpy="0 -0 0" />
-            <geometry>
-                <mesh filename="package://mit_drcsim_scripts/models/mit_robot/meshes/l_elbow_ry.wrl" scale="1 1 1" />
-            </geometry>
-        </visual>
+        <xacro:if value="${minimal_contact}">
+          <visual>
+            <origin xyz="0 0 0" rpy="0 -0 0" />
+            <geometry>
+              <mesh filename="package://mit_drcsim_scripts/models/mit_robot/meshes/l_elbow_ry.wrl" scale="1 1 1" />
+            </geometry>
+          </visual>
+        </xacro:if>
+        <xacro:unless value="${minimal_contact}">
+          <visual>
+            <origin xyz="0 0 0" rpy="0 -0 0"/>
+            <geometry>
+              <mesh filename="package://mit_drcsim_scripts/models/mit_robot/meshes/l_elbow_ry_chull.wrl"
+                scale="1 1 1"/>
+            </geometry>
+          </visual>
+          <collision>
+            <origin xyz="0 0 0" rpy="0 -0 0"/>
+            <geometry>
+              <mesh filename="package://mit_drcsim_scripts/models/mit_robot/meshes/l_elbow_ry_chull.wrl"
+                scale="1 1 1"/>
+            </geometry>
+          </collision>
+        </xacro:unless>
     </link>
     <link name="l_uglut">
@@ -164,10 +315,12 @@
             <inertia ixx="0.00074276" ixy="-3.79607e-08" ixz="-2.79549e-05" iyy="0.000688179" iyz="-3.2735e-08" izz="0.00041242" />
         </inertial>
-        <visual>
-            <origin xyz="0 0 0" rpy="0 -0 0" />
-            <geometry>
-                <mesh filename="package://mit_drcsim_scripts/models/mit_robot/meshes/l_uglut.wrl" scale="1 1 1" />
-            </geometry>
-        </visual>
+        <xacro:if value="${minimal_contact}">
+          <visual>
+            <origin xyz="0 0 0" rpy="0 -0 0" />
+            <geometry>
+              <mesh filename="package://mit_drcsim_scripts/models/mit_robot/meshes/l_uglut.wrl" scale="1 1 1" />
+            </geometry>
+          </visual>
+        </xacro:if>
     </link>
     <link name="l_uleg">
@@ -177,12 +330,30 @@
             <inertia ixx="0.09" ixy="0" ixz="0" iyy="0.09" iyz="0" izz="0.02" />
         </inertial>
-        <visual>
-            <origin xyz="0 0 0" rpy="0 -0 0" />
-            <geometry>
-                <mesh filename="package://mit_drcsim_scripts/models/mit_robot/meshes/l_uleg.wrl" scale="1 1 1" />
-            </geometry>
-        </visual>
-        <xacro:collision_point group="hamstring" xyz="-0.1179 0.02085 -0.18" visualize="1"/>
-        <xacro:collision_point group="hamstring" xyz="-0.1179 0.02085 -0.08" visualize="1"/>
+        <xacro:if value="${minimal_contact}">
+          <visual>
+            <origin xyz="0 0 0" rpy="0 -0 0" />
+            <geometry>
+              <mesh filename="package://mit_drcsim_scripts/models/mit_robot/meshes/l_uleg.wrl" scale="1 1 1" />
+            </geometry>
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