Commit message: a stack of changes to tracking for better integration. integrated icp, historgram and color tracker and cascade tracking from planes. also added remote command and control
git-svn-id: https://svn.csail.mit.edu/drc@2558 c7283977-0100-402a-a91a-fa70b306dbfe

File: software/models/mit_gazebo_models/mit_robot_nohands/model.urdf (robot description, URDF)
Before this commit: robot atlas, 41 links, 40 joints
Joints:
- joint neck_ay: limit lower=-0.610865238 upper=1.13446401 effort=5 velocity=12 -> lower=-0.610865238 upper=0 effort=5 velocity=12

File: software/models/mit_gazebo_models/real_multisense_sl/multisense.urdf (robot description, URDF)
Before this commit: robot multisense, 12 links, 11 joints
Links:
- removed link head_root
Joints:
- removed joint head_root_joint

Commit message: Fix false lower limit on neck joint
git-svn-id: https://svn.csail.mit.edu/drc@2674 c7283977-0100-402a-a91a-fa70b306dbfe

File: software/models/mit_gazebo_models/mit_robot_nohands/model.urdf (robot description, URDF)
Before this commit: robot atlas, 41 links, 40 joints
Joints:
- joint neck_ay: limit lower=-0.610865238 upper=0 effort=5 velocity=12 -> lower=-0.610865238 upper=1.13446401 effort=5 velocity=12

Commit message: mesh scaling, friction coeff, matched model.config to drcsim release 2.6
git-svn-id: https://svn.csail.mit.edu/drc@3766 c7283977-0100-402a-a91a-fa70b306dbfe

File: software/models/mit_gazebo_models/mit_robot_nohands/model.urdf (robot description, URDF)
Before this commit: robot atlas, 41 links, 40 joints
Links:
- link l_lleg: geometry collision cylinder length=0.40 radius=0.07; visual mesh filename=package://mit_robot/meshes/l_lleg.dae scale=1 1 1
- link l_uleg: geometry collision cylinder length=0.10 radius=0.1; collision cylinder length=0.15 radius=0.07
- link pelvis: geometry collision box size=0.1 0.15 0.2; collision cylinder length=0.05 radius=0.16
- link r_larm: geometry collision box size=0.135 0.15 0.06; collision cylinder length=0.125 radius=0.045
- link r_lglut: geometry collision cylinder length=0.060306 radius=0.02009687; collision cylinder length=0.12 radius=0.02
- link r_lleg: geometry collision cylinder length=0.40 radius=0.07; visual mesh filename=package://mit_robot/meshes/r_lleg.dae scale=1 1 1
- link r_uarm: geometry collision box size=0.04 0.07 0.13; collision cylinder length=0.125 radius=0.045
- link r_uglut: geometry collision cylinder length=0.078396 radius=0.019096; collision cylinder length=0.080842 radius=0.019841
- link r_uleg: geometry collision cylinder length=0.10 radius=0.1; collision cylinder length=0.15 radius=0.07
