Commit message: Removes mud seat collision element freom model_drake.urdf, since it's not rigid.
git-svn-id: https://svn.csail.mit.edu/drc@3890 c7283977-0100-402a-a91a-fa70b306dbfe

File: software/models/mit_gazebo_objects/mit_vehicle/model_drake.urdf (robot description, URDF)
Before this commit: robot polaris_ranger_ev, 6 links, 5 joints
Links:
- link chassis: geometry collision box size=0.05 1.2 0.25; collision box size=0.05 1.2 0.25

Commit message: Adds ground box. Removes mud seat visual.
git-svn-id: https://svn.csail.mit.edu/drc@4658 c7283977-0100-402a-a91a-fa70b306dbfe

File: software/models/mit_gazebo_objects/mit_vehicle/model_drake.urdf (robot description, URDF)
Before this commit: robot polaris_ranger_ev, 6 links, 5 joints
Links:
- added link box; collision box size=10 10 0.1
- link chassis: geometry collision box size=0.05 1.2 0.25; collision box size=0.05 1.2 0.25
Joints:
- added joint chassis_fixed: type fixed, parent box, child chassis, origin xyz=0 0 0 rpy=0 0 0, axis 0 0 1

Commit message: adding inertial properties to drc_vehicle
git-svn-id: https://svn.csail.mit.edu/drc@4768 c7283977-0100-402a-a91a-fa70b306dbfe

File: software/models/mit_gazebo_objects/mit_vehicle/model_drake.urdf (robot description, URDF)
Before this commit: robot polaris_ranger_ev, 7 links, 6 joints
Links:
- link chassis: mass None -> 720.0
