Commit message: more revisions to driver, close to finished
git-svn-id: https://svn.csail.mit.edu/drc/trunk@5534 c7283977-0100-402a-a91a-fa70b306dbfe

File: ros_workspace/multisense/multisense/multisense_description/urdf/multisense.urdf (robot description, URDF)
Before this commit: robot multisense, 25 links, 24 joints
Links:
- removed link head_root
Joints:
- removed joint head_root_joint

Commit message: integrating v2 of multisense driver with lcm publisher
git-svn-id: https://svn.csail.mit.edu/drc/trunk@5614 c7283977-0100-402a-a91a-fa70b306dbfe

File: ros_workspace/multisense/multisense/multisense_description/urdf/multisense.urdf (robot description, URDF)
Before this commit: robot multisense, 24 links, 23 joints
Links:
- added link head_root
Joints:
- added joint head_root_joint: type fixed, parent head_root, child head
