Commit message: updated to latest atlas models
git-svn-id: https://svn.csail.mit.edu/drc@880 c7283977-0100-402a-a91a-fa70b306dbfe

File: software/models/mit_gazebo_models/mit_robot/model.urdf (robot description, URDF)
Before this commit: robot atlas, 29 links, 28 joints
Links:
- added link head_hokuyo, mass 0.1
- added link imu_link, mass 0.1; collision box size=0.01 0.01 0.01; visual box size=0.01 0.01 0.01
- added link left_camera_frame, mass 0.1
- added link left_camera_optical_frame
- added link right_camera_frame, mass 0.1
- added link right_camera_optical_frame
- link head: geometry collision mesh filename=package://atlas/meshes/head.stl scale=1 1 1; visual mesh filename=package://atlas/meshes/head.dae scale=1 1 1
- link l_clav: geometry collision mesh filename=package://atlas/meshes/l_clav.stl scale=1 1 1; visual mesh filename=package://atlas/meshes/l_clav.dae scale=1 1 1
- link l_farm: geometry collision mesh filename=package://atlas/meshes/l_farm.stl scale=1 1 1; visual mesh filename=package://atlas/meshes/l_farm.dae scale=1 1 1
- link l_foot: geometry collision mesh filename=package://atlas/meshes/l_foot.stl scale=1 1 1; visual mesh filename=package://atlas/meshes/l_foot.dae scale=1 1 1
- link l_hand: geometry collision mesh filename=package://atlas/meshes/l_hand.stl scale=1 1 1; visual mesh filename=package://atlas/meshes/l_hand.dae scale=1 1 1
- link l_larm: geometry collision mesh filename=package://atlas/meshes/l_larm.stl scale=1 1 1; visual mesh filename=package://atlas/meshes/l_larm.dae scale=1 1 1
- link l_lglut: geometry collision mesh filename=package://atlas/meshes/l_lglut.stl scale=1 1 1; visual mesh filename=package://atlas/meshes/l_lglut.dae scale=1 1 1
- link l_lleg: geometry collision mesh filename=package://atlas/meshes/l_lleg.stl scale=1 1 1; visual mesh filename=package://atlas/meshes/l_lleg.dae scale=1 1 1
- link l_scap: geometry collision mesh filename=package://atlas/meshes/l_scap.stl scale=1 1 1; visual mesh filename=package://atlas/meshes/l_scap.dae scale=1 1 1
- link l_talus: geometry collision mesh filename=package://atlas/meshes/l_talus.stl scale=1 1 1; visual mesh filename=package://atlas/meshes/l_talus.dae scale=1 1 1
- link l_uarm: geometry collision mesh filename=package://atlas/meshes/l_uarm.stl scale=1 1 1; visual mesh filename=package://atlas/meshes/l_uarm.dae scale=1 1 1
- link l_uglut: geometry collision mesh filename=package://atlas/meshes/l_uglut.stl scale=1 1 1; visual mesh filename=package://atlas/meshes/l_uglut.dae scale=1 1 1
- link l_uleg: geometry collision mesh filename=package://atlas/meshes/l_uleg.stl scale=1 1 1; visual mesh filename=package://atlas/meshes/l_uleg.dae scale=1 1 1
- link ltorso: geometry collision mesh filename=package://atlas/meshes/ltorso.stl scale=1 1 1; visual mesh filename=package://atlas/meshes/ltorso.dae scale=1 1 1
- link mtorso: geometry collision mesh filename=package://atlas/meshes/mtorso.stl scale=1 1 1; visual mesh filename=package://atlas/meshes/mtorso.dae scale=1 1 1
- link pelvis: geometry collision mesh filename=package://atlas/meshes/pelvis.stl scale=1 1 1; visual mesh filename=package://atlas/meshes/pelvis.dae scale=1 1 1
- link r_clav: geometry collision mesh filename=package://atlas/meshes/r_clav.stl scale=1 1 1; visual mesh filename=package://atlas/meshes/r_clav.dae scale=1 1 1
- link r_farm: geometry collision mesh filename=package://atlas/meshes/r_farm.stl scale=1 1 1; visual mesh filename=package://atlas/meshes/r_farm.dae scale=1 1 1
- link r_foot: geometry collision mesh filename=package://atlas/meshes/r_foot.stl scale=1 1 1; visual mesh filename=package://atlas/meshes/r_foot.dae scale=1 1 1
- link r_hand: geometry collision mesh filename=package://atlas/meshes/r_hand.stl scale=1 1 1; visual mesh filename=package://atlas/meshes/r_hand.dae scale=1 1 1
- link r_larm: geometry collision mesh filename=package://atlas/meshes/r_larm.stl scale=1 1 1; visual mesh filename=package://atlas/meshes/r_larm.dae scale=1 1 1
- link r_lglut: geometry collision mesh filename=package://atlas/meshes/r_lglut.stl scale=1 1 1; visual mesh filename=package://atlas/meshes/r_lglut.dae scale=1 1 1
- link r_lleg: geometry collision mesh filename=package://atlas/meshes/r_lleg.stl scale=1 1 1; visual mesh filename=package://atlas/meshes/r_lleg.dae scale=1 1 1
- link r_scap: geometry collision mesh filename=package://atlas/meshes/r_scap.stl scale=1 1 1; visual mesh filename=package://atlas/meshes/r_scap.dae scale=1 1 1
- link r_talus: geometry collision mesh filename=package://atlas/meshes/r_talus.stl scale=1 1 1; visual mesh filename=package://atlas/meshes/r_talus.dae scale=1 1 1
- link r_uarm: geometry collision mesh filename=package://atlas/meshes/r_uarm.stl scale=1 1 1; visual mesh filename=package://atlas/meshes/r_uarm.dae scale=1 1 1
- link r_uglut: geometry collision mesh filename=package://atlas/meshes/r_uglut.stl scale=1 1 1; visual mesh filename=package://atlas/meshes/r_uglut.dae scale=1 1 1
- link r_uleg: geometry collision mesh filename=package://atlas/meshes/r_uleg.stl scale=1 1 1; visual mesh filename=package://atlas/meshes/r_uleg.dae scale=1 1 1
- link utorso: geometry collision mesh filename=package://atlas/meshes/utorso.stl scale=1 1 1; visual mesh filename=package://atlas/meshes/utorso.dae scale=1 1 1
Joints:
- added joint head_hokuyo_joint: type fixed, parent head, child head_hokuyo, origin xyz=0.03 0 0.13 rpy=0 0 0, axis 0 1 0
- added joint imu_joint: type revolute, parent pelvis, child imu_link, origin xyz=0.05991527603 0 -0.01415 rpy=0 0 0, axis 0 0 1, limit lower=0 upper=0 effort=0 velocity=0
- added joint left_camera_frame_joint: type fixed, parent head, child left_camera_frame, origin xyz=0.03 0.1 0.1
- added joint left_camera_optical_frame_joint: type fixed, parent left_camera_frame, child left_camera_optical_frame, origin xyz=0 0 0 rpy=-1.5708 0.0 -1.5708
- added joint right_camera_frame_joint: type fixed, parent head, child right_camera_frame, origin xyz=0.03 -0.1 0.1
- added joint right_camera_optical_frame_joint: type fixed, parent right_camera_frame, child right_camera_optical_frame, origin xyz=0 0 0 rpy=-1.5708 0.0 -1.5708

File: software/models/mit_gazebo_models/mit_robot_PnC/model.urdf (robot description, URDF)
Before this commit: robot mit_drc_robot, 38 links, 37 joints
Links:
- removed link head_imu_link
- removed link head_rightedhokuyo
- removed link head_statichokuyo
- link head_hokuyo: geometry 
Joints:
- removed joint head_imu_joint
- removed joint head_rightedhokuyo_joint
- removed joint head_statichokuyo_joint
- joint head_hokuyo_joint: axis 1 0 0 -> 0 1 0; limit effort=5 velocity=12 -> (none); origin xyz=0 0 0 rpy=0 0 0 -> xyz=0.03 0 0.13 rpy=0 0 0; type continuous -> fixed
- joint imu_joint: axis (none) -> 0 0 1; limit (none) -> lower=0 upper=0 effort=0 velocity=0; origin xyz=0 0 0 rpy=0 0 0 -> xyz=0.05991527603 0 -0.01415 rpy=0 0 0; parent ltorso -> pelvis; type fixed -> revolute
- joint left_camera_frame_joint: origin xyz=0.03 0.35 0.1 -> xyz=0.03 0.1 0.1
- joint neck_ay: origin xyz=0.021 0 0.44 rpy=0 -0 0 -> xyz=0.011 0 0.44 rpy=0 -0 0
- joint right_camera_frame_joint: origin xyz=0.03 -0.35 0.1 -> xyz=0.03 -0.1 0.1

File: software/models/mit_gazebo_models/mit_robot_PnC/statue.urdf (robot description, URDF)
Before this commit: robot atlas, 29 links, 28 joints
Links:
- added link imu_link, mass 0.1; collision box size=0.01 0.01 0.01; visual box size=0.01 0.01 0.01
- added link l_foot_c1, mass 0.001; collision sphere radius=0.001; visual sphere radius=0.001
- added link l_foot_c2, mass 0.001; collision sphere radius=0.001; visual sphere radius=0.001
- added link l_foot_c3, mass 0.001; collision sphere radius=0.001; visual sphere radius=0.001
- added link l_foot_c4, mass 0.001; collision sphere radius=0.001; visual sphere radius=0.001
- added link r_foot_c1, mass 0.001; collision sphere radius=0.001; visual sphere radius=0.001
- added link r_foot_c2, mass 0.001; collision sphere radius=0.001; visual sphere radius=0.001
- added link r_foot_c3, mass 0.001; collision sphere radius=0.001; visual sphere radius=0.001
- added link r_foot_c4, mass 0.001; collision sphere radius=0.001; visual sphere radius=0.001
- link head: geometry visual mesh filename=package://mit_robot/meshes/head.dae scale=1 1 1
- link l_clav: geometry visual mesh filename=package://mit_robot/meshes/l_clav.dae scale=1 1 1
- link l_farm: geometry visual mesh filename=package://mit_robot/meshes/l_farm.dae scale=1 1 1
- link l_foot: geometry visual mesh filename=package://mit_robot/meshes/l_foot.dae scale=1 1 1
- link l_hand: geometry visual mesh filename=package://mit_robot/meshes/l_hand.dae scale=1 1 1
- link l_larm: geometry visual mesh filename=package://mit_robot/meshes/l_larm.dae scale=1 1 1
- link l_lglut: geometry visual mesh filename=package://mit_robot/meshes/l_lglut.dae scale=1 1 1
- link l_lleg: geometry visual mesh filename=package://mit_robot/meshes/l_lleg.dae scale=1 1 1
- link l_scap: geometry visual mesh filename=package://mit_robot/meshes/l_scap.dae scale=1 1 1
- link l_talus: geometry visual mesh filename=package://mit_robot/meshes/l_talus.dae scale=1 1 1
- link l_uarm: geometry visual mesh filename=package://mit_robot/meshes/l_uarm.dae scale=1 1 1
- link l_uglut: geometry visual mesh filename=package://mit_robot/meshes/l_uglut.dae scale=1 1 1
- link l_uleg: geometry visual mesh filename=package://mit_robot/meshes/l_uleg.dae scale=1 1 1
- link ltorso: geometry visual mesh filename=package://mit_robot/meshes/ltorso.dae scale=1 1 1
- link mtorso: geometry visual mesh filename=package://mit_robot/meshes/mtorso.dae scale=1 1 1
- link pelvis: geometry visual mesh filename=package://mit_robot/meshes/pelvis.dae scale=1 1 1
- link r_clav: geometry visual mesh filename=package://mit_robot/meshes/r_clav.dae scale=1 1 1
- link r_farm: geometry visual mesh filename=package://mit_robot/meshes/r_farm.dae scale=1 1 1
- link r_foot: geometry visual mesh filename=package://mit_robot/meshes/r_foot.dae scale=1 1 1
- link r_hand: geometry visual mesh filename=package://mit_robot/meshes/r_hand.dae scale=1 1 1
- link r_larm: geometry visual mesh filename=package://mit_robot/meshes/r_larm.dae scale=1 1 1
- link r_lglut: geometry visual mesh filename=package://mit_robot/meshes/r_lglut.dae scale=1 1 1
- link r_lleg: geometry visual mesh filename=package://mit_robot/meshes/r_lleg.dae scale=1 1 1
- link r_scap: geometry visual mesh filename=package://mit_robot/meshes/r_scap.dae scale=1 1 1
- link r_talus: geometry visual mesh filename=package://mit_robot/meshes/r_talus.dae scale=1 1 1
- link r_uarm: geometry visual mesh filename=package://mit_robot/meshes/r_uarm.dae scale=1 1 1
- link r_uglut: geometry visual mesh filename=package://mit_robot/meshes/r_uglut.dae scale=1 1 1
- link r_uleg: geometry visual mesh filename=package://mit_robot/meshes/r_uleg.dae scale=1 1 1
- link utorso: geometry visual mesh filename=package://mit_robot/meshes/utorso.dae scale=1 1 1
Joints:
- added joint imu_joint: type revolute, parent pelvis, child imu_link, origin xyz=0.05991527603 0 -0.01415 rpy=0 0 0, axis 0 0 1, limit lower=0 upper=0 effort=0 velocity=0
- added joint l_foot_j1: type fixed, parent l_foot, child l_foot_c1, origin xyz=0.178 0.032 -0.080 rpy=0 0 0
- added joint l_foot_j2: type fixed, parent l_foot, child l_foot_c2, origin xyz=0.178 -0.032 -0.080 rpy=0 0 0
- added joint l_foot_j3: type fixed, parent l_foot, child l_foot_c3, origin xyz=-0.075 -0.047 -0.081 rpy=0 0 0
- added joint l_foot_j4: type fixed, parent l_foot, child l_foot_c4, origin xyz=-0.075 0.048 -0.081 rpy=0 0 0
- added joint r_foot_j1: type fixed, parent r_foot, child r_foot_c1, origin xyz=0.178 0.032 -0.080 rpy=0 0 0
- added joint r_foot_j2: type fixed, parent r_foot, child r_foot_c2, origin xyz=0.178 -0.032 -0.080 rpy=0 0 0
- added joint r_foot_j3: type fixed, parent r_foot, child r_foot_c3, origin xyz=-0.075 -0.047 -0.081 rpy=0 0 0
- added joint r_foot_j4: type fixed, parent r_foot, child r_foot_c4, origin xyz=-0.075 0.048 -0.081 rpy=0 0 0
- joint back_lbz: type revolute -> fixed
- joint back_mby: type revolute -> fixed
- joint back_ubx: type revolute -> fixed
- joint l_arm_elx: type revolute -> fixed
- joint l_arm_ely: type revolute -> fixed
- joint l_arm_mwx: type revolute -> fixed
- joint l_arm_shx: type revolute -> fixed
- joint l_arm_usy: type revolute -> fixed
- joint l_arm_uwy: type revolute -> fixed
- joint l_leg_kny: type revolute -> fixed
- joint l_leg_lax: type revolute -> fixed
- joint l_leg_lhy: type revolute -> fixed
- joint l_leg_mhx: type revolute -> fixed
- joint l_leg_uay: type revolute -> fixed
- joint l_leg_uhz: type revolute -> fixed
- joint neck_ay: type revolute -> fixed
- joint r_arm_elx: type revolute -> fixed
- joint r_arm_ely: type revolute -> fixed
- joint r_arm_mwx: type revolute -> fixed
- joint r_arm_shx: type revolute -> fixed
- joint r_arm_usy: type revolute -> fixed
- joint r_arm_uwy: type revolute -> fixed
- joint r_leg_kny: type revolute -> fixed
- joint r_leg_lax: type revolute -> fixed
- joint r_leg_lhy: type revolute -> fixed
- joint r_leg_mhx: type revolute -> fixed
- joint r_leg_uay: type revolute -> fixed
- joint r_leg_uhz: type revolute -> fixed

File: software/models/mit_gazebo_models/mit_robot_PnC/xacro/atlas_sandia_hands.model.xacro (robot description, xacro)
@@ -3,7 +3,6 @@
        xmlns:interface="http://playerstage.sourceforge.net/gazebo/xmlschema/#interface"
        xmlns:xacro="http://playerstage.sourceforge.net/gazebo/xmlschema/#interface"
-       name="mit_drc_robot" >
-<!--  <include filename="$(find mit_drcsim_scripts)/models/mit_robot_PnC/xacro/drc_skeleton.urdf" /> -->
-  <include filename="$(find mit_drcsim_scripts)/models/mit_robot_PnC/xacro/drc_skeleton_minimal_contact_gazebo.urdf" />
+       name="atlas" >
+  <include filename="$(find atlas_utils)/urdf/atlas.urdf" />
   <include filename="$(find sandia_hand_utils)/urdf/sandia_hand.urdf.xacro" />
   <xacro:sandia_hand side="r" parent="r_hand">
@@ -13,7 +12,6 @@
     <origin xyz="0  0.1 -0.03" rpy="0 3.1416 -1.57079"/>
   </xacro:sandia_hand>
-<!--  <include filename="$(find drc_robot_utils)/urdf/drc_robot.gazebo" /> -->
-  <include filename="$(find drc_robot_utils)/urdf/drc_robot.transmission" />
-  <include filename="$(find drc_robot_utils)/urdf/drc_robot.sensors" />
-  <include filename="$(find mit_drcsim_scripts)/models/mit_robot_PnC/xacro/mit_drc_robot.gazebo" />
+  <include filename="$(find atlas_utils)/urdf/atlas.transmission" />
+  <include filename="$(find atlas_utils)/urdf/atlas.sensors" />
+  <include filename="$(find mit_drcsim_scripts)/models/mit_robot_PnC/xacro/mit_atlas.gazebo" />
 </robot>

File: software/models/mit_gazebo_models/mit_robot_PnC/xacro/atlas_statue_minimal_contact.urdf (robot description, URDF)
Before this commit: robot drc_skeleton, 37 links, 36 joints
Links:
- link l_foot_c1: mass 0.0001 -> 0.001; geometry collision sphere radius=0.001; visual sphere radius=0.001
- link l_foot_c2: mass 0.0001 -> 0.001; geometry collision sphere radius=0.001; visual sphere radius=0.001
- link l_foot_c3: mass 0.0001 -> 0.001; geometry collision sphere radius=0.001; visual sphere radius=0.001
- link l_foot_c4: mass 0.0001 -> 0.001; geometry collision sphere radius=0.001; visual sphere radius=0.001
- link r_foot_c1: mass 0.0001 -> 0.001; geometry collision sphere radius=0.001; visual sphere radius=0.001
- link r_foot_c2: mass 0.0001 -> 0.001; geometry collision sphere radius=0.001; visual sphere radius=0.001
- link r_foot_c3: mass 0.0001 -> 0.001; geometry collision sphere radius=0.001; visual sphere radius=0.001
- link r_foot_c4: mass 0.0001 -> 0.001; geometry collision sphere radius=0.001; visual sphere radius=0.001
Joints:
- joint back_lbz: type revolute -> fixed
- joint back_mby: type revolute -> fixed
- joint back_ubx: type revolute -> fixed
- joint l_arm_elx: type revolute -> fixed
- joint l_arm_ely: type revolute -> fixed
- joint l_arm_mwx: type revolute -> fixed
- joint l_arm_shx: type revolute -> fixed
- joint l_arm_usy: type revolute -> fixed
- joint l_arm_uwy: type revolute -> fixed
- joint l_foot_j1: origin xyz=0.18 -0.03 -0.08 rpy=0 0 0 -> xyz=0.178 0.032 -0.080 rpy=0 0 0
- joint l_foot_j2: origin xyz=0.18 0.03 -0.08 rpy=0 0 0 -> xyz=0.178 -0.032 -0.080 rpy=0 0 0
- joint l_foot_j3: origin xyz=-0.07 0.056 -0.08 rpy=0 0 0 -> xyz=-0.075 -0.047 -0.081 rpy=0 0 0
- joint l_foot_j4: origin xyz=-0.07 -0.056 -0.08 rpy=0 0 0 -> xyz=-0.075 0.048 -0.081 rpy=0 0 0
- joint l_leg_kny: type revolute -> fixed
- joint l_leg_lax: type revolute -> fixed
- joint l_leg_lhy: type revolute -> fixed
- joint l_leg_mhx: type revolute -> fixed
- joint l_leg_uay: type revolute -> fixed
- joint l_leg_uhz: type revolute -> fixed
- joint neck_ay: type revolute -> fixed
- joint r_arm_elx: type revolute -> fixed
- joint r_arm_ely: type revolute -> fixed
- joint r_arm_mwx: type revolute -> fixed
- joint r_arm_shx: type revolute -> fixed
- joint r_arm_usy: type revolute -> fixed
- joint r_arm_uwy: type revolute -> fixed
- joint r_foot_j1: origin xyz=0.18 -0.03 -0.08 rpy=0 0 0 -> xyz=0.178 0.032 -0.080 rpy=0 0 0
- joint r_foot_j2: origin xyz=0.18 0.03 -0.08 rpy=0 0 0 -> xyz=0.178 -0.032 -0.080 rpy=0 0 0
- joint r_foot_j3: origin xyz=-0.07 0.056 -0.08 rpy=0 0 0 -> xyz=-0.075 -0.047 -0.081 rpy=0 0 0
- joint r_foot_j4: origin xyz=-0.07 -0.056 -0.08 rpy=0 0 0 -> xyz=-0.075 0.048 -0.081 rpy=0 0 0
- joint r_leg_kny: type revolute -> fixed
- joint r_leg_lax: type revolute -> fixed
- joint r_leg_lhy: type revolute -> fixed
- joint r_leg_mhx: type revolute -> fixed
- joint r_leg_uay: type revolute -> fixed
- joint r_leg_uhz: type revolute -> fixed
