Commit message: various changes, some in progress for new drc 1.3 sim and for new modules
git-svn-id: https://svn.csail.mit.edu/drc@904 c7283977-0100-402a-a91a-fa70b306dbfe

File: software/models/mit_gazebo_models/mit_robot/model.urdf (robot description, URDF)
Before this commit: robot atlas, 35 links, 34 joints
Links:
- added link center_bottom_led_frame, mass 0.1
- added link center_top_led_frame, mass 0.1
- added link head_imu_link, mass 0.1; collision box size=0.01 0.01 0.01; visual box size=0.01 0.01 0.01
- added link hokuyo_link, mass 0.057664; collision mesh filename=package://multisense_sl/meshes/hokuyo_link.STL; visual mesh filename=package://multisense_sl/meshes/hokuyo_link.STL
- added link left_led_frame, mass 0.1
- added link right_led_frame, mass 0.1
- link head: mass 2.6 -> 1.4199; geometry collision mesh filename=package://multisense_sl/meshes/base_link.STL; visual mesh filename=package://multisense_sl/meshes/base_link.STL
- link head_hokuyo: mass 0.1 -> 0.01
- link l_clav: geometry collision mesh filename=package://mit_robot/meshes/l_clav.stl scale=1 1 1; visual mesh filename=package://mit_robot/meshes/l_clav.dae scale=1 1 1
- link l_farm: geometry collision mesh filename=package://mit_robot/meshes/l_farm.stl scale=1 1 1; visual mesh filename=package://mit_robot/meshes/l_farm.dae scale=1 1 1
- link l_foot: geometry collision mesh filename=package://mit_robot/meshes/l_foot.stl scale=1 1 1; visual mesh filename=package://mit_robot/meshes/l_foot.dae scale=1 1 1
- link l_hand: geometry collision mesh filename=package://mit_robot/meshes/l_hand.stl scale=1 1 1; visual mesh filename=package://mit_robot/meshes/l_hand.dae scale=1 1 1
- link l_larm: geometry collision mesh filename=package://mit_robot/meshes/l_larm.stl scale=1 1 1; visual mesh filename=package://mit_robot/meshes/l_larm.dae scale=1 1 1
- link l_lglut: geometry collision mesh filename=package://mit_robot/meshes/l_lglut.stl scale=1 1 1; visual mesh filename=package://mit_robot/meshes/l_lglut.dae scale=1 1 1
- link l_lleg: geometry collision mesh filename=package://mit_robot/meshes/l_lleg.stl scale=1 1 1; visual mesh filename=package://mit_robot/meshes/l_lleg.dae scale=1 1 1
- link l_scap: geometry collision mesh filename=package://mit_robot/meshes/l_scap.stl scale=1 1 1; visual mesh filename=package://mit_robot/meshes/l_scap.dae scale=1 1 1
- link l_talus: geometry collision mesh filename=package://mit_robot/meshes/l_talus.stl scale=1 1 1; visual mesh filename=package://mit_robot/meshes/l_talus.dae scale=1 1 1
- link l_uarm: geometry collision mesh filename=package://mit_robot/meshes/l_uarm.stl scale=1 1 1; visual mesh filename=package://mit_robot/meshes/l_uarm.dae scale=1 1 1
- link l_uglut: geometry collision mesh filename=package://mit_robot/meshes/l_uglut.stl scale=1 1 1; visual mesh filename=package://mit_robot/meshes/l_uglut.dae scale=1 1 1
- link l_uleg: geometry collision mesh filename=package://mit_robot/meshes/l_uleg.stl scale=1 1 1; visual mesh filename=package://mit_robot/meshes/l_uleg.dae scale=1 1 1
- link ltorso: geometry collision mesh filename=package://mit_robot/meshes/ltorso.stl scale=1 1 1; visual mesh filename=package://mit_robot/meshes/ltorso.dae scale=1 1 1
- link mtorso: geometry collision mesh filename=package://mit_robot/meshes/mtorso.stl scale=1 1 1; visual mesh filename=package://mit_robot/meshes/mtorso.dae scale=1 1 1
- link pelvis: geometry collision mesh filename=package://mit_robot/meshes/pelvis.stl scale=1 1 1; visual mesh filename=package://mit_robot/meshes/pelvis.dae scale=1 1 1
- link r_clav: geometry collision mesh filename=package://mit_robot/meshes/r_clav.stl scale=1 1 1; visual mesh filename=package://mit_robot/meshes/r_clav.dae scale=1 1 1
- link r_farm: geometry collision mesh filename=package://mit_robot/meshes/r_farm.stl scale=1 1 1; visual mesh filename=package://mit_robot/meshes/r_farm.dae scale=1 1 1
- link r_foot: geometry collision mesh filename=package://mit_robot/meshes/r_foot.stl scale=1 1 1; visual mesh filename=package://mit_robot/meshes/r_foot.dae scale=1 1 1
- link r_hand: geometry collision mesh filename=package://mit_robot/meshes/r_hand.stl scale=1 1 1; visual mesh filename=package://mit_robot/meshes/r_hand.dae scale=1 1 1
- link r_larm: geometry collision mesh filename=package://mit_robot/meshes/r_larm.stl scale=1 1 1; visual mesh filename=package://mit_robot/meshes/r_larm.dae scale=1 1 1
- link r_lglut: geometry collision mesh filename=package://mit_robot/meshes/r_lglut.stl scale=1 1 1; visual mesh filename=package://mit_robot/meshes/r_lglut.dae scale=1 1 1
- link r_lleg: geometry collision mesh filename=package://mit_robot/meshes/r_lleg.stl scale=1 1 1; visual mesh filename=package://mit_robot/meshes/r_lleg.dae scale=1 1 1
- link r_scap: geometry collision mesh filename=package://mit_robot/meshes/r_scap.stl scale=1 1 1; visual mesh filename=package://mit_robot/meshes/r_scap.dae scale=1 1 1
- link r_talus: geometry collision mesh filename=package://mit_robot/meshes/r_talus.stl scale=1 1 1; visual mesh filename=package://mit_robot/meshes/r_talus.dae scale=1 1 1
- link r_uarm: geometry collision mesh filename=package://mit_robot/meshes/r_uarm.stl scale=1 1 1; visual mesh filename=package://mit_robot/meshes/r_uarm.dae scale=1 1 1
- link r_uglut: geometry collision mesh filename=package://mit_robot/meshes/r_uglut.stl scale=1 1 1; visual mesh filename=package://mit_robot/meshes/r_uglut.dae scale=1 1 1
- link r_uleg: geometry collision mesh filename=package://mit_robot/meshes/r_uleg.stl scale=1 1 1; visual mesh filename=package://mit_robot/meshes/r_uleg.dae scale=1 1 1
- link utorso: geometry collision mesh filename=package://mit_robot/meshes/utorso.stl scale=1 1 1; visual mesh filename=package://mit_robot/meshes/utorso.dae scale=1 1 1
Joints:
- added joint center_bottom_led_frame_joint: type fixed, parent head, child center_bottom_led_frame, origin xyz=0.01125 0.0 -0.0155
- added joint center_top_led_frame_joint: type fixed, parent head, child center_top_led_frame, origin xyz=0.01125 0.0 0.0105
- added joint head_imu_joint: type fixed, parent head, child head_imu_link, origin xyz=0 0 0 rpy=0 0 0
- added joint hokuyo_joint: type continuous, parent head, child hokuyo_link, origin xyz=-0.0446 0 0.0880 rpy=0 0 0, axis 1 0 0
- added joint left_led_frame_joint: type fixed, parent head, child left_led_frame, origin xyz=-0.01443 0.07452 0.050346 rpy=0 -0.15 0.53
- added joint right_led_frame_joint: type fixed, parent head, child right_led_frame, origin xyz=-0.01443 -0.07452 0.050346 rpy=0 -0.15 -0.53
- joint head_hokuyo_joint: origin xyz=0.03 0 0.13 rpy=0 0 0 -> xyz=0.03 0 0.015 rpy=0 0 0; parent head -> hokuyo_link
- joint left_camera_frame_joint: origin xyz=0.03 0.1 0.1 -> xyz=0.0 0.035 -0.002
- joint neck_ay: limit lower=-0.785398 upper=0.785398 effort=5 velocity=12 -> lower=-0.610865238 upper=1.13446401 effort=5 velocity=12; origin xyz=0.011 0 0.44 rpy=0 -0 0 -> xyz=0.16555 0 0.50823 rpy=0 0 0
- joint right_camera_frame_joint: origin xyz=0.03 -0.1 0.1 -> xyz=0.0 -0.035 -0.002

File: software/models/mit_gazebo_models/mit_robot/xacro/atlas_sandia_hands.model.xacro (robot description, xacro)
@@ -4,5 +4,5 @@
        xmlns:xacro="http://playerstage.sourceforge.net/gazebo/xmlschema/#interface"
        name="atlas" >
-  <include filename="$(find atlas_utils)/urdf/atlas.urdf" />
+  <include filename="$(find mit_drcsim_scripts)/models/mit_robot/xacro/mit_atlas.urdf" />
   <include filename="$(find sandia_hand_utils)/urdf/sandia_hand.urdf.xacro" />
   <xacro:sandia_hand side="r" parent="r_hand">
@@ -12,5 +12,5 @@
     <origin xyz="0  0.1 -0.03" rpy="0 3.1416 -1.57079"/>
   </xacro:sandia_hand>
-  <include filename="$(find atlas_utils)/urdf/atlas.gazebo" />
+  <include filename="$(find mit_drcsim_scripts)/models/mit_robot/xacro/mit_atlas.gazebo" />
   <include filename="$(find atlas_utils)/urdf/atlas.transmission" />
   <include filename="$(find atlas_utils)/urdf/atlas.sensors" />

Commit message: git-svn-id: https://svn.csail.mit.edu/drc@1109 c7283977-0100-402a-a91a-fa70b306dbfe

File: software/models/mit_gazebo_models/mit_robot/model.urdf (robot description, URDF)
Before this commit: robot atlas, 41 links, 40 joints
Joints:
- joint head_imu_joint: axis (none) -> 0 0 1; limit (none) -> lower=0 upper=0 effort=0 velocity=0; type fixed -> revolute

File: software/models/mit_gazebo_models/mit_robot_PnC/model.urdf (robot description, URDF)
Before this commit: robot atlas, 93 links, 92 joints
Links:
- removed link l_f0_0
- removed link l_f0_1
- removed link l_f0_1_accel
- removed link l_f0_2
- removed link l_f0_2_accel
- removed link l_f0_base
- removed link l_f0_fixed_accel
- removed link l_f1_0
- removed link l_f1_1
- removed link l_f1_1_accel
- removed link l_f1_2
- removed link l_f1_2_accel
- removed link l_f1_base
- removed link l_f1_fixed_accel
- removed link l_f2_0
- removed link l_f2_1
- removed link l_f2_1_accel
- removed link l_f2_2
- removed link l_f2_2_accel
- removed link l_f2_base
- removed link l_f2_fixed_accel
- removed link l_f3_0
- removed link l_f3_1
- removed link l_f3_1_accel
- removed link l_f3_2
- removed link l_f3_2_accel
- removed link l_f3_base
- removed link l_f3_fixed_accel
- removed link l_palm
- removed link r_f0_0
- removed link r_f0_1
- removed link r_f0_1_accel
- removed link r_f0_2
- removed link r_f0_2_accel
- removed link r_f0_base
- removed link r_f0_fixed_accel
- removed link r_f1_0
- removed link r_f1_1
- removed link r_f1_1_accel
- removed link r_f1_2
- removed link r_f1_2_accel
- removed link r_f1_base
- removed link r_f1_fixed_accel
- removed link r_f2_0
- removed link r_f2_1
- removed link r_f2_1_accel
- removed link r_f2_2
- removed link r_f2_2_accel
- removed link r_f2_base
- removed link r_f2_fixed_accel
- removed link r_f3_0
- removed link r_f3_1
- removed link r_f3_1_accel
- removed link r_f3_2
- removed link r_f3_2_accel
- removed link r_f3_base
- removed link r_f3_fixed_accel
- removed link r_palm
Joints:
- removed joint l_f0_1_accel
- removed joint l_f0_2_accel
- removed joint l_f0_base
- removed joint l_f0_fixed_accel
- removed joint l_f0_j0
- removed joint l_f0_j1
- removed joint l_f0_j2
- removed joint l_f1_1_accel
- removed joint l_f1_2_accel
- removed joint l_f1_base
- removed joint l_f1_fixed_accel
- removed joint l_f1_j0
- removed joint l_f1_j1
- removed joint l_f1_j2
- removed joint l_f2_1_accel
- removed joint l_f2_2_accel
- removed joint l_f2_base
- removed joint l_f2_fixed_accel
- removed joint l_f2_j0
- removed joint l_f2_j1
- removed joint l_f2_j2
- removed joint l_f3_1_accel
- removed joint l_f3_2_accel
- removed joint l_f3_base
- removed joint l_f3_fixed_accel
- removed joint l_f3_j0
- removed joint l_f3_j1
- removed joint l_f3_j2
- removed joint l_sandia_hand_joint
- removed joint r_f0_1_accel
- removed joint r_f0_2_accel
- removed joint r_f0_base
- removed joint r_f0_fixed_accel
- removed joint r_f0_j0
- removed joint r_f0_j1
- removed joint r_f0_j2
- removed joint r_f1_1_accel
- removed joint r_f1_2_accel
- removed joint r_f1_base
- removed joint r_f1_fixed_accel
- removed joint r_f1_j0
- removed joint r_f1_j1
- removed joint r_f1_j2
- removed joint r_f2_1_accel
- removed joint r_f2_2_accel
- removed joint r_f2_base
- removed joint r_f2_fixed_accel
- removed joint r_f2_j0
- removed joint r_f2_j1
- removed joint r_f2_j2
- removed joint r_f3_1_accel
- removed joint r_f3_2_accel
- removed joint r_f3_base
- removed joint r_f3_fixed_accel
- removed joint r_f3_j0
- removed joint r_f3_j1
- removed joint r_f3_j2
- removed joint r_sandia_hand_joint

File: software/models/mit_gazebo_models/mit_robot_drake/model_minimal_contact.urdf (robot description, URDF)
Before this commit: robot atlas, 29 links, 28 joints
Links:
- link head: geometry visual mesh filename=/home/mfallon/drc/ros_workspace/mit_drcsim_scripts/models/m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 scale=1 1 1
- link l_clav: geometry visual mesh filename=/home/mfallon/drc/ros_workspace/mit_drcsim_scripts/models/m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 scale=1 1 1
- link l_farm: geometry visual mesh filename=/home/mfallon/drc/ros_workspace/mit_drcsim_scripts/models/m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 scale=1 1 1
- link l_foot: geometry collision sphere radius=0; collision sphere radius=0
- link l_hand: geometry visual mesh filename=/home/mfallon/drc/ros_workspace/mit_drcsim_scripts/models/m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 scale=1 1 1
- link l_larm: geometry visual mesh filename=/home/mfallon/drc/ros_workspace/mit_drcsim_scripts/models/m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 scale=1 1 1
- link l_lglut: geometry visual mesh filename=/home/mfallon/drc/ros_workspace/mit_drcsim_scripts/models/m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 scale=1 1 1
- link l_lleg: geometry visual mesh filename=/home/mfallon/drc/ros_workspace/mit_drcsim_scripts/models/m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 scale=1 1 1
- link l_scap: geometry visual mesh filename=/home/mfallon/drc/ros_workspace/mit_drcsim_scripts/models/m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 scale=1 1 1
- link l_talus: geometry visual mesh filename=/home/mfallon/drc/ros_workspace/mit_drcsim_scripts/models/m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 scale=1 1 1
- link l_uarm: geometry visual mesh filename=/home/mfallon/drc/ros_workspace/mit_drcsim_scripts/models/m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 scale=1 1 1
- link l_uglut: geometry visual mesh filename=/home/mfallon/drc/ros_workspace/mit_drcsim_scripts/models/m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 scale=1 1 1
- link l_uleg: geometry visual mesh filename=/home/mfallon/drc/ros_workspace/mit_drcsim_scripts/models/m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 scale=1 1 1
- link ltorso: geometry visual mesh filename=/home/mfallon/drc/ros_workspace/mit_drcsim_scripts/models/m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 scale=1 1 1
- link mtorso: geometry visual mesh filename=/home/mfallon/drc/ros_workspace/mit_drcsim_scripts/models/m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 scale=1 1 1
- link pelvis: geometry visual mesh filename=/home/mfallon/drc/ros_workspace/mit_drcsim_scripts/models/m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 scale=1 1 1
- link r_clav: geometry visual mesh filename=/home/mfallon/drc/ros_workspace/mit_drcsim_scripts/models/m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 scale=1 1 1
- link r_farm: geometry visual mesh filename=/home/mfallon/drc/ros_workspace/mit_drcsim_scripts/models/m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 scale=1 1 1
- link r_foot: geometry collision sphere radius=0; collision sphere radius=0
- link r_hand: geometry visual mesh filename=/home/mfallon/drc/ros_workspace/mit_drcsim_scripts/models/m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 scale=1 1 1
- link r_larm: geometry visual mesh filename=/home/mfallon/drc/ros_workspace/mit_drcsim_scripts/models/m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 scale=1 1 1
- link r_lglut: geometry visual mesh filename=/home/mfallon/drc/ros_workspace/mit_drcsim_scripts/models/m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 scale=1 1 1
- link r_lleg: geometry visual mesh filename=/home/mfallon/drc/ros_workspace/mit_drcsim_scripts/models/m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 scale=1 1 1
- link r_scap: geometry visual mesh filename=/home/mfallon/drc/ros_workspace/mit_drcsim_scripts/models/m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 scale=1 1 1
- link r_talus: geometry visual mesh filename=/home/mfallon/drc/ros_workspace/mit_drcsim_scripts/models/m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 scale=1 1 1
- link r_uarm: geometry visual mesh filename=/home/mfallon/drc/ros_workspace/mit_drcsim_scripts/models/m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 scale=1 1 1
- link r_uglut: geometry visual mesh filename=/home/mfallon/drc/ros_workspace/mit_drcsim_scripts/models/m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 scale=1 1 1
- link r_uleg: geometry visual mesh filename=/home/mfallon/drc/ros_workspace/mit_drcsim_scripts/models/m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 scale=1 1 1
- link utorso: geometry visual mesh filename=/home/mfallon/drc/ros_workspace/mit_drcsim_scripts/models/m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 scale=1 1 1

Commit message: use lowercase extension
git-svn-id: https://svn.csail.mit.edu/drc@1581 c7283977-0100-402a-a91a-fa70b306dbfe

File: software/models/mit_gazebo_models/mit_robot/model.urdf (robot description, URDF)
Before this commit: robot atlas, 41 links, 40 joints
Links:
- link head: geometry collision mesh filename=package://multisense_sl/meshes/base_link.stl; visual mesh filename=package://multisense_sl/meshes/base_link.stl

Commit message: use lowercase extension
git-svn-id: https://svn.csail.mit.edu/drc@1583 c7283977-0100-402a-a91a-fa70b306dbfe

File: software/models/mit_gazebo_models/mit_robot/model.urdf (robot description, URDF)
Before this commit: robot atlas, 41 links, 40 joints
Links:
- link hokuyo_link: geometry collision mesh filename=package://multisense_sl/meshes/hokuyo_link.stl; visual mesh filename=package://multisense_sl/meshes/hokuyo_link.stl

Commit message: merging PnC and original robot
git-svn-id: https://svn.csail.mit.edu/drc@2319 c7283977-0100-402a-a91a-fa70b306dbfe

File: software/models/mit_gazebo_models/mit_robot/model.urdf (robot description, URDF)
Before this commit: robot atlas, 41 links, 40 joints
Links:
- removed link head_hokuyo
- added link head_hokuyo_frame, mass 0.01
- link head: geometry collision box size=0.0468 0.12 0.1184; collision box size=0.1311 0.12 0.0591
- link head_imu_link: geometry visual box size=0.01 0.01 0.01
- link hokuyo_link: geometry collision box size=0.08 0.06 0.04238; collision cylinder length=0.047 radius=0.024425
- link imu_link: geometry visual box size=0.01 0.01 0.01
- link l_clav: geometry collision cylinder length=0.027 radius=0.04; collision cylinder length=0.1525 radius=0.045
- link l_farm: geometry collision cylinder length=0.035181 radius=0.0458825; collision cylinder length=0.050472 radius=0.0279
- link l_foot: mass 1.634 -> 0.817; geometry collision box size=0.26 0.124887 0.01; visual mesh filename=package://mit_robot/meshes/l_foot.dae scale=1 1 1
- link l_hand: geometry collision cylinder length=0.019 radius=0.035939; collision cylinder length=0.019 radius=0.035939
- link l_larm: geometry collision cylinder length=0.0161 radius=0.045; collision cylinder length=0.0161 radius=0.045
- link l_lglut: geometry collision cylinder length=0.060306 radius=0.02009687; collision cylinder length=0.12 radius=0.02
- link l_lleg: geometry collision cylinder length=0.20 radius=0.06; collision cylinder length=0.22 radius=0.06
- link l_scap: geometry collision cylinder length=0.013737 radius=0.048709; collision cylinder length=0.013937 radius=0.048709
- link l_talus: mass 0.1 -> 0.817; geometry collision cylinder length=0.010059 radius=0.010348; collision cylinder length=0.029542 radius=0.010181
- link l_uarm: geometry collision cylinder length=0.088934 radius=0.04504847; collision cylinder length=0.116677 radius=0.0449
- link l_uglut: geometry collision cylinder length=0.078396 radius=0.019096; collision cylinder length=0.080842 radius=0.019841
- link l_uleg: geometry collision cylinder length=0.10 radius=0.1; collision cylinder length=0.15 radius=0.07
- link ltorso: geometry visual mesh filename=package://mit_robot/meshes/ltorso.dae scale=1 1 1
- link mtorso: geometry collision cylinder length=0.02 radius=0.015; collision cylinder length=0.02 radius=0.015
- link pelvis: geometry collision cylinder length=0.022 radius=0.130; collision cylinder length=0.022 radius=0.130
- link r_clav: geometry collision cylinder length=0.027 radius=0.04; collision cylinder length=0.1525 radius=0.045
- link r_farm: geometry collision cylinder length=0.035181 radius=0.0458825; collision cylinder length=0.050472 radius=0.0279
- link r_foot: mass 1.634 -> 0.817; geometry collision box size=0.26 0.124887 0.01; visual mesh filename=package://mit_robot/meshes/r_foot.dae scale=1 1 1
- link r_hand: geometry collision cylinder length=0.019 radius=0.035939; collision cylinder length=0.019 radius=0.035939
- link r_larm: geometry collision cylinder length=0.0161 radius=0.045; collision cylinder length=0.0161 radius=0.045
- link r_lglut: geometry collision cylinder length=0.060306 radius=0.02009687; collision cylinder length=0.12 radius=0.02
- link r_lleg: geometry collision cylinder length=0.20 radius=0.06; collision cylinder length=0.22 radius=0.06
- link r_scap: geometry collision cylinder length=0.013737 radius=0.048709; collision cylinder length=0.013937 radius=0.048709
- link r_talus: mass 0.1 -> 0.817; geometry collision cylinder length=0.010059 radius=0.010348; collision cylinder length=0.029542 radius=0.010181
- link r_uarm: geometry collision cylinder length=0.088934 radius=0.04504847; collision cylinder length=0.116677 radius=0.0449
- link r_uglut: geometry collision cylinder length=0.078396 radius=0.019096; collision cylinder length=0.080842 radius=0.019841
- link r_uleg: geometry collision cylinder length=0.10 radius=0.1; collision cylinder length=0.15 radius=0.07
- link utorso: geometry collision box size=0.3188 0.24 0.3162; collision cylinder length=0.22375 radius=0.0363
Joints:
- joint head_hokuyo_joint: child head_hokuyo -> head_hokuyo_frame
- joint head_imu_joint: axis 0 0 1 -> (none); limit lower=0 upper=0 effort=0 velocity=0 -> (none); origin xyz=0 0 0 rpy=0 0 0 -> xyz=-0.0475 0.035 0.0 rpy=0 0 0; type revolute -> fixed
- joint imu_joint: axis 0 0 1 -> (none); limit lower=0 upper=0 effort=0 velocity=0 -> (none); type revolute -> fixed
- joint neck_ay: origin xyz=0.16555 0 0.50823 rpy=0 0 0 -> xyz=0.16555 0 0.50823 rpy=0 -0 0
- joint r_arm_usy: axis 0 -0.5 0.866025 -> 0 0.5 -0.866025
