Commit message: git-svn-id: https://svn.csail.mit.edu/drc@2328 c7283977-0100-402a-a91a-fa70b306dbfe

File: software/models/mit_gazebo_models/mit_robot/model.urdf (robot description, URDF)
Before this commit: robot atlas, 41 links, 40 joints
Links:
- added link left_f0_0, mass 0.05; collision cylinder length=0.023 radius=0.01; collision cylinder length=0.023 radius=0.015
- added link left_f0_1, mass 0.05; collision cylinder length=0.067 radius=0.01; visual cylinder length=0.067 radius=0.01
- added link left_f0_1_accel, mass 0.001
- added link left_f0_2, mass 0.05; collision cylinder length=0.057 radius=0.009; collision sphere radius=0.009
- added link left_f0_2_accel, mass 0.001
- added link left_f0_base, mass 0.35
- added link left_f0_fixed_accel, mass 0.001
- added link left_f1_0, mass 0.05; collision cylinder length=0.023 radius=0.01; collision cylinder length=0.023 radius=0.015
- added link left_f1_1, mass 0.05; collision cylinder length=0.067 radius=0.01; visual cylinder length=0.067 radius=0.01
- added link left_f1_1_accel, mass 0.001
- added link left_f1_2, mass 0.05; collision cylinder length=0.057 radius=0.009; collision sphere radius=0.009
- added link left_f1_2_accel, mass 0.001
- added link left_f1_base, mass 0.35
- added link left_f1_fixed_accel, mass 0.001
- added link left_f2_0, mass 0.05; collision cylinder length=0.023 radius=0.01; collision cylinder length=0.023 radius=0.015
- added link left_f2_1, mass 0.05; collision cylinder length=0.067 radius=0.01; visual cylinder length=0.067 radius=0.01
- added link left_f2_1_accel, mass 0.001
- added link left_f2_2, mass 0.05; collision cylinder length=0.057 radius=0.009; collision sphere radius=0.009
- added link left_f2_2_accel, mass 0.001
- added link left_f2_base, mass 0.35
- added link left_f2_fixed_accel, mass 0.001
- added link left_f3_0, mass 0.05; collision cylinder length=0.023 radius=0.01; collision cylinder length=0.023 radius=0.015
- added link left_f3_1, mass 0.05; collision cylinder length=0.067 radius=0.01; visual cylinder length=0.067 radius=0.01
- added link left_f3_1_accel, mass 0.001
- added link left_f3_2, mass 0.05; collision cylinder length=0.057 radius=0.009; collision sphere radius=0.009
- added link left_f3_2_accel, mass 0.001
- added link left_f3_base, mass 0.35
- added link left_f3_fixed_accel, mass 0.001
- added link left_palm, mass 0.3; collision box size=0.09 .03 .06; collision box size=0.09 .03 .06
- added link right_f0_0, mass 0.05; collision cylinder length=0.023 radius=0.01; collision cylinder length=0.023 radius=0.015
- added link right_f0_1, mass 0.05; collision cylinder length=0.067 radius=0.01; visual cylinder length=0.067 radius=0.01
- added link right_f0_1_accel, mass 0.001
- added link right_f0_2, mass 0.05; collision cylinder length=0.057 radius=0.009; collision sphere radius=0.009
- added link right_f0_2_accel, mass 0.001
- added link right_f0_base, mass 0.35
- added link right_f0_fixed_accel, mass 0.001
- added link right_f1_0, mass 0.05; collision cylinder length=0.023 radius=0.01; collision cylinder length=0.023 radius=0.015
- added link right_f1_1, mass 0.05; collision cylinder length=0.067 radius=0.01; visual cylinder length=0.067 radius=0.01
- added link right_f1_1_accel, mass 0.001
- added link right_f1_2, mass 0.05; collision cylinder length=0.057 radius=0.009; collision sphere radius=0.009
- added link right_f1_2_accel, mass 0.001
- added link right_f1_base, mass 0.35
- added link right_f1_fixed_accel, mass 0.001
- added link right_f2_0, mass 0.05; collision cylinder length=0.023 radius=0.01; collision cylinder length=0.023 radius=0.015
- added link right_f2_1, mass 0.05; collision cylinder length=0.067 radius=0.01; visual cylinder length=0.067 radius=0.01
- added link right_f2_1_accel, mass 0.001
- added link right_f2_2, mass 0.05; collision cylinder length=0.057 radius=0.009; collision sphere radius=0.009
- added link right_f2_2_accel, mass 0.001
- added link right_f2_base, mass 0.35
- added link right_f2_fixed_accel, mass 0.001
- added link right_f3_0, mass 0.05; collision cylinder length=0.023 radius=0.01; collision cylinder length=0.023 radius=0.015
- added link right_f3_1, mass 0.05; collision cylinder length=0.067 radius=0.01; visual cylinder length=0.067 radius=0.01
- added link right_f3_1_accel, mass 0.001
- added link right_f3_2, mass 0.05; collision cylinder length=0.057 radius=0.009; collision sphere radius=0.009
- added link right_f3_2_accel, mass 0.001
- added link right_f3_base, mass 0.35
- added link right_f3_fixed_accel, mass 0.001
- added link right_palm, mass 0.3; collision box size=0.09 .03 .06; collision box size=0.09 .03 .06
Joints:
- added joint left_f0_1_accel: type fixed, parent left_f0_1, child left_f0_1_accel, origin xyz=0.03 0 0 rpy=-1.57079632679 0 0
- added joint left_f0_2_accel: type fixed, parent left_f0_2, child left_f0_2_accel, origin xyz=0.04 0 0 rpy=-1.57079632679 0 0
- added joint left_f0_base: type fixed, parent left_palm, child left_f0_base, origin xyz=0.14 0.0 0 rpy=0 0 -0.3
- added joint left_f0_fixed_accel: type fixed, parent left_f0_base, child left_f0_fixed_accel, origin xyz=-0.05 0 0 rpy=0 0 0
- added joint left_f0_j0: type revolute, parent left_f0_base, child left_f0_0, origin xyz=0 0 0 rpy=0 0 0, axis 0 0 -1, limit lower=-1.57079632679 upper=1.57079632679 effort=1 velocity=1
- added joint left_f0_j1: type revolute, parent left_f0_0, child left_f0_1, origin xyz=0.028 0 0 rpy=1.57079632679 0 0, axis 0 0 1, limit lower=-1.57079632679 upper=1.57079632679 effort=1 velocity=1
- added joint left_f0_j2: type revolute, parent left_f0_1, child left_f0_2, origin xyz=0.05 0 0 rpy=0 0 0, axis 0 0 1, limit lower=-1.57079632679 upper=1.57079632679 effort=1 velocity=1
- added joint left_f1_1_accel: type fixed, parent left_f1_1, child left_f1_1_accel, origin xyz=0.03 0 0 rpy=-1.57079632679 0 0
- added joint left_f1_2_accel: type fixed, parent left_f1_2, child left_f1_2_accel, origin xyz=0.04 0 0 rpy=-1.57079632679 0 0
- added joint left_f1_base: type fixed, parent left_palm, child left_f1_base, origin xyz=0.115 -0.03122 0 rpy=0 0 -0.3
- added joint left_f1_fixed_accel: type fixed, parent left_f1_base, child left_f1_fixed_accel, origin xyz=-0.05 0 0 rpy=0 0 0
- added joint left_f1_j0: type revolute, parent left_f1_base, child left_f1_0, origin xyz=0 0 0 rpy=0 0 0, axis 0 0 -1, limit lower=-1.57079632679 upper=1.57079632679 effort=1 velocity=1
- added joint left_f1_j1: type revolute, parent left_f1_0, child left_f1_1, origin xyz=0.028 0 0 rpy=1.57079632679 0 0, axis 0 0 1, limit lower=-1.57079632679 upper=1.57079632679 effort=1 velocity=1
- added joint left_f1_j2: type revolute, parent left_f1_1, child left_f1_2, origin xyz=0.05 0 0 rpy=0 0 0, axis 0 0 1, limit lower=-1.57079632679 upper=1.57079632679 effort=1 velocity=1
- added joint left_f2_1_accel: type fixed, parent left_f2_1, child left_f2_1_accel, origin xyz=0.03 0 0 rpy=-1.57079632679 0 0
- added joint left_f2_2_accel: type fixed, parent left_f2_2, child left_f2_2_accel, origin xyz=0.04 0 0 rpy=-1.57079632679 0 0
- added joint left_f2_base: type fixed, parent left_palm, child left_f2_base, origin xyz=0.09 -0.06245 0 rpy=0 0 -0.3
- added joint left_f2_fixed_accel: type fixed, parent left_f2_base, child left_f2_fixed_accel, origin xyz=-0.05 0 0 rpy=0 0 0
- added joint left_f2_j0: type revolute, parent left_f2_base, child left_f2_0, origin xyz=0 0 0 rpy=0 0 0, axis 0 0 -1, limit lower=-1.57079632679 upper=1.57079632679 effort=1 velocity=1
- added joint left_f2_j1: type revolute, parent left_f2_0, child left_f2_1, origin xyz=0.028 0 0 rpy=1.57079632679 0 0, axis 0 0 1, limit lower=-1.57079632679 upper=1.57079632679 effort=1 velocity=1
- added joint left_f2_j2: type revolute, parent left_f2_1, child left_f2_2, origin xyz=0.05 0 0 rpy=0 0 0, axis 0 0 1, limit lower=-1.57079632679 upper=1.57079632679 effort=1 velocity=1
- added joint left_f3_1_accel: type fixed, parent left_f3_1, child left_f3_1_accel, origin xyz=0.03 0 0 rpy=-1.57079632679 0 0
- added joint left_f3_2_accel: type fixed, parent left_f3_2, child left_f3_2_accel, origin xyz=0.04 0 0 rpy=-1.57079632679 0 0
- added joint left_f3_base: type fixed, parent left_palm, child left_f3_base, origin xyz=0.03995 0.04383 0.014 rpy=0 -1.57079632679 2.3562
- added joint left_f3_fixed_accel: type fixed, parent left_f3_base, child left_f3_fixed_accel, origin xyz=-0.05 0 0 rpy=0 0 0
- added joint left_f3_j0: type revolute, parent left_f3_base, child left_f3_0, origin xyz=0 0 0 rpy=0 0 0, axis 0 0 -1, limit lower=-1.57079632679 upper=1.57079632679 effort=1 velocity=1
- added joint left_f3_j1: type revolute, parent left_f3_0, child left_f3_1, origin xyz=0.028 0 0 rpy=1.57079632679 0 0, axis 0 0 1, limit lower=-1.57079632679 upper=1.57079632679 effort=1 velocity=1
- added joint left_f3_j2: type revolute, parent left_f3_1, child left_f3_2, origin xyz=0.05 0 0 rpy=0 0 0, axis 0 0 1, limit lower=-1.57079632679 upper=1.57079632679 effort=1 velocity=1
- added joint left_sandia_hand_joint: type fixed, parent l_hand, child left_palm, origin xyz=0  0.1 0 rpy= 1.57079 0  1.57079
- added joint right_f0_1_accel: type fixed, parent right_f0_1, child right_f0_1_accel, origin xyz=0.03 0 0 rpy=-1.57079632679 0 0
- added joint right_f0_2_accel: type fixed, parent right_f0_2, child right_f0_2_accel, origin xyz=0.04 0 0 rpy=-1.57079632679 0 0
- added joint right_f0_base: type fixed, parent right_palm, child right_f0_base, origin xyz=0.14 0.0 0 rpy=0 0 0.3
- added joint right_f0_fixed_accel: type fixed, parent right_f0_base, child right_f0_fixed_accel, origin xyz=-0.05 0 0 rpy=0 0 0
- added joint right_f0_j0: type revolute, parent right_f0_base, child right_f0_0, origin xyz=0 0 0 rpy=0 0 0, axis 0 0 1, limit lower=-1.57079632679 upper=1.57079632679 effort=1 velocity=1
- added joint right_f0_j1: type revolute, parent right_f0_0, child right_f0_1, origin xyz=0.028 0 0 rpy=1.57079632679 0 0, axis 0 0 1, limit lower=-1.57079632679 upper=1.57079632679 effort=1 velocity=1
- added joint right_f0_j2: type revolute, parent right_f0_1, child right_f0_2, origin xyz=0.05 0 0 rpy=0 0 0, axis 0 0 1, limit lower=-1.57079632679 upper=1.57079632679 effort=1 velocity=1
- added joint right_f1_1_accel: type fixed, parent right_f1_1, child right_f1_1_accel, origin xyz=0.03 0 0 rpy=-1.57079632679 0 0
- added joint right_f1_2_accel: type fixed, parent right_f1_2, child right_f1_2_accel, origin xyz=0.04 0 0 rpy=-1.57079632679 0 0
- added joint right_f1_base: type fixed, parent right_palm, child right_f1_base, origin xyz=0.115 0.03122 0 rpy=0 0 0.3
- added joint right_f1_fixed_accel: type fixed, parent right_f1_base, child right_f1_fixed_accel, origin xyz=-0.05 0 0 rpy=0 0 0
- added joint right_f1_j0: type revolute, parent right_f1_base, child right_f1_0, origin xyz=0 0 0 rpy=0 0 0, axis 0 0 1, limit lower=-1.57079632679 upper=1.57079632679 effort=1 velocity=1
- added joint right_f1_j1: type revolute, parent right_f1_0, child right_f1_1, origin xyz=0.028 0 0 rpy=1.57079632679 0 0, axis 0 0 1, limit lower=-1.57079632679 upper=1.57079632679 effort=1 velocity=1
- added joint right_f1_j2: type revolute, parent right_f1_1, child right_f1_2, origin xyz=0.05 0 0 rpy=0 0 0, axis 0 0 1, limit lower=-1.57079632679 upper=1.57079632679 effort=1 velocity=1
- added joint right_f2_1_accel: type fixed, parent right_f2_1, child right_f2_1_accel, origin xyz=0.03 0 0 rpy=-1.57079632679 0 0
- added joint right_f2_2_accel: type fixed, parent right_f2_2, child right_f2_2_accel, origin xyz=0.04 0 0 rpy=-1.57079632679 0 0
- added joint right_f2_base: type fixed, parent right_palm, child right_f2_base, origin xyz=0.09 0.06245 0 rpy=0 0 0.3
- added joint right_f2_fixed_accel: type fixed, parent right_f2_base, child right_f2_fixed_accel, origin xyz=-0.05 0 0 rpy=0 0 0
- added joint right_f2_j0: type revolute, parent right_f2_base, child right_f2_0, origin xyz=0 0 0 rpy=0 0 0, axis 0 0 1, limit lower=-1.57079632679 upper=1.57079632679 effort=1 velocity=1
- added joint right_f2_j1: type revolute, parent right_f2_0, child right_f2_1, origin xyz=0.028 0 0 rpy=1.57079632679 0 0, axis 0 0 1, limit lower=-1.57079632679 upper=1.57079632679 effort=1 velocity=1
- added joint right_f2_j2: type revolute, parent right_f2_1, child right_f2_2, origin xyz=0.05 0 0 rpy=0 0 0, axis 0 0 1, limit lower=-1.57079632679 upper=1.57079632679 effort=1 velocity=1
- added joint right_f3_1_accel: type fixed, parent right_f3_1, child right_f3_1_accel, origin xyz=0.03 0 0 rpy=-1.57079632679 0 0
- added joint right_f3_2_accel: type fixed, parent right_f3_2, child right_f3_2_accel, origin xyz=0.04 0 0 rpy=-1.57079632679 0 0
- added joint right_f3_base: type fixed, parent right_palm, child right_f3_base, origin xyz=0.03995 -0.04383 0.014 rpy=0 -1.57079632679 -2.3562
- added joint right_f3_fixed_accel: type fixed, parent right_f3_base, child right_f3_fixed_accel, origin xyz=-0.05 0 0 rpy=0 0 0
- added joint right_f3_j0: type revolute, parent right_f3_base, child right_f3_0, origin xyz=0 0 0 rpy=0 0 0, axis 0 0 1, limit lower=-1.57079632679 upper=1.57079632679 effort=1 velocity=1
- added joint right_f3_j1: type revolute, parent right_f3_0, child right_f3_1, origin xyz=0.028 0 0 rpy=1.57079632679 0 0, axis 0 0 1, limit lower=-1.57079632679 upper=1.57079632679 effort=1 velocity=1
- added joint right_f3_j2: type revolute, parent right_f3_1, child right_f3_2, origin xyz=0.05 0 0 rpy=0 0 0, axis 0 0 1, limit lower=-1.57079632679 upper=1.57079632679 effort=1 velocity=1
- added joint right_sandia_hand_joint: type fixed, parent r_hand, child right_palm, origin xyz=0 -0.1 0 rpy=-1.57079 0 -1.57079

Commit message: upated xacro outputs
git-svn-id: https://svn.csail.mit.edu/drc@2785 c7283977-0100-402a-a91a-fa70b306dbfe

File: software/models/mit_gazebo_models/mit_robot/model.urdf (robot description, URDF)
Before this commit: robot atlas, 99 links, 98 joints
Links:
- link l_foot: mass 0.817 -> 0.867
- link l_lglut: mass 0.69 -> 0.803
- link l_talus: mass 0.817 -> 0.867
- link l_uglut: mass 0.5166 -> 1.51622
- link l_uleg: mass 7.34 -> 7.227
- link left_f0_0: mass 0.05 -> 0.106
- link left_f0_1: mass 0.05 -> 0.033
- link left_f0_1_accel: mass 0.001 -> 0.01
- link left_f0_2: mass 0.05 -> 0.033
- link left_f0_2_accel: mass 0.001 -> 0.01
- link left_f0_base: mass 0.35 -> 0.250
- link left_f0_fixed_accel: mass 0.001 -> 0.01
- link left_f1_0: mass 0.05 -> 0.106
- link left_f1_1: mass 0.05 -> 0.033
- link left_f1_1_accel: mass 0.001 -> 0.01
- link left_f1_2: mass 0.05 -> 0.033
- link left_f1_2_accel: mass 0.001 -> 0.01
- link left_f1_base: mass 0.35 -> 0.250
- link left_f1_fixed_accel: mass 0.001 -> 0.01
- link left_f2_0: mass 0.05 -> 0.106
- link left_f2_1: mass 0.05 -> 0.033
- link left_f2_1_accel: mass 0.001 -> 0.01
- link left_f2_2: mass 0.05 -> 0.033
- link left_f2_2_accel: mass 0.001 -> 0.01
- link left_f2_base: mass 0.35 -> 0.250
- link left_f2_fixed_accel: mass 0.001 -> 0.01
- link left_f3_0: mass 0.05 -> 0.106
- link left_f3_1: mass 0.05 -> 0.033
- link left_f3_1_accel: mass 0.001 -> 0.01
- link left_f3_2: mass 0.05 -> 0.033
- link left_f3_2_accel: mass 0.001 -> 0.01
- link left_f3_base: mass 0.35 -> 0.250
- link left_f3_fixed_accel: mass 0.001 -> 0.01
- link left_palm: mass 0.3 -> 1.303
- link ltorso: mass 1.92 -> 1.62729
- link mtorso: mass 0.55 -> 3.8068
- link pelvis: mass 14.2529 -> 12.54638
- link r_foot: mass 0.817 -> 0.867
- link r_lglut: mass 0.69 -> 0.803
- link r_talus: mass 0.817 -> 0.867
- link r_uglut: mass 0.5166 -> 1.51622
- link r_uleg: mass 7.34 -> 7.227
- link right_f0_0: mass 0.05 -> 0.106
- link right_f0_1: mass 0.05 -> 0.033
- link right_f0_1_accel: mass 0.001 -> 0.01
- link right_f0_2: mass 0.05 -> 0.033
- link right_f0_2_accel: mass 0.001 -> 0.01
- link right_f0_base: mass 0.35 -> 0.250
- link right_f0_fixed_accel: mass 0.001 -> 0.01
- link right_f1_0: mass 0.05 -> 0.106
- link right_f1_1: mass 0.05 -> 0.033
- link right_f1_1_accel: mass 0.001 -> 0.01
- link right_f1_2: mass 0.05 -> 0.033
- link right_f1_2_accel: mass 0.001 -> 0.01
- link right_f1_base: mass 0.35 -> 0.250
- link right_f1_fixed_accel: mass 0.001 -> 0.01
- link right_f2_0: mass 0.05 -> 0.106
- link right_f2_1: mass 0.05 -> 0.033
- link right_f2_1_accel: mass 0.001 -> 0.01
- link right_f2_2: mass 0.05 -> 0.033
- link right_f2_2_accel: mass 0.001 -> 0.01
- link right_f2_base: mass 0.35 -> 0.250
- link right_f2_fixed_accel: mass 0.001 -> 0.01
- link right_f3_0: mass 0.05 -> 0.106
- link right_f3_1: mass 0.05 -> 0.033
- link right_f3_1_accel: mass 0.001 -> 0.01
- link right_f3_2: mass 0.05 -> 0.033
- link right_f3_2_accel: mass 0.001 -> 0.01
- link right_f3_base: mass 0.35 -> 0.250
- link right_f3_fixed_accel: mass 0.001 -> 0.01
- link right_palm: mass 0.3 -> 1.303
- link utorso: mass 18.484 -> 15.2272
Joints:
- joint left_f0_j0: limit lower=-1.57079632679 upper=1.57079632679 effort=1 velocity=1 -> lower=-1.57079632679 upper=1.57079632679 effort=11 velocity=1
- joint left_f0_j1: limit lower=-1.57079632679 upper=1.57079632679 effort=1 velocity=1 -> lower=-1.57079632679 upper=1.57079632679 effort=28 velocity=1
- joint left_f0_j2: limit lower=-1.57079632679 upper=1.57079632679 effort=1 velocity=1 -> lower=-1.57079632679 upper=1.57079632679 effort=28 velocity=1
- joint left_f1_j0: limit lower=-1.57079632679 upper=1.57079632679 effort=1 velocity=1 -> lower=-1.57079632679 upper=1.57079632679 effort=11 velocity=1
- joint left_f1_j1: limit lower=-1.57079632679 upper=1.57079632679 effort=1 velocity=1 -> lower=-1.57079632679 upper=1.57079632679 effort=28 velocity=1
- joint left_f1_j2: limit lower=-1.57079632679 upper=1.57079632679 effort=1 velocity=1 -> lower=-1.57079632679 upper=1.57079632679 effort=28 velocity=1
- joint left_f2_j0: limit lower=-1.57079632679 upper=1.57079632679 effort=1 velocity=1 -> lower=-1.57079632679 upper=1.57079632679 effort=11 velocity=1
- joint left_f2_j1: limit lower=-1.57079632679 upper=1.57079632679 effort=1 velocity=1 -> lower=-1.57079632679 upper=1.57079632679 effort=28 velocity=1
- joint left_f2_j2: limit lower=-1.57079632679 upper=1.57079632679 effort=1 velocity=1 -> lower=-1.57079632679 upper=1.57079632679 effort=28 velocity=1
- joint left_f3_j0: limit lower=-1.57079632679 upper=1.57079632679 effort=1 velocity=1 -> lower=-1.57079632679 upper=1.57079632679 effort=11 velocity=1
- joint left_f3_j1: limit lower=-1.57079632679 upper=1.57079632679 effort=1 velocity=1 -> lower=-1.57079632679 upper=1.57079632679 effort=28 velocity=1
- joint left_f3_j2: limit lower=-1.57079632679 upper=1.57079632679 effort=1 velocity=1 -> lower=-1.57079632679 upper=1.57079632679 effort=28 velocity=1
- joint right_f0_j0: limit lower=-1.57079632679 upper=1.57079632679 effort=1 velocity=1 -> lower=-1.57079632679 upper=1.57079632679 effort=11 velocity=1
- joint right_f0_j1: limit lower=-1.57079632679 upper=1.57079632679 effort=1 velocity=1 -> lower=-1.57079632679 upper=1.57079632679 effort=28 velocity=1
- joint right_f0_j2: limit lower=-1.57079632679 upper=1.57079632679 effort=1 velocity=1 -> lower=-1.57079632679 upper=1.57079632679 effort=28 velocity=1
- joint right_f1_j0: limit lower=-1.57079632679 upper=1.57079632679 effort=1 velocity=1 -> lower=-1.57079632679 upper=1.57079632679 effort=11 velocity=1
- joint right_f1_j1: limit lower=-1.57079632679 upper=1.57079632679 effort=1 velocity=1 -> lower=-1.57079632679 upper=1.57079632679 effort=28 velocity=1
- joint right_f1_j2: limit lower=-1.57079632679 upper=1.57079632679 effort=1 velocity=1 -> lower=-1.57079632679 upper=1.57079632679 effort=28 velocity=1
- joint right_f2_j0: limit lower=-1.57079632679 upper=1.57079632679 effort=1 velocity=1 -> lower=-1.57079632679 upper=1.57079632679 effort=11 velocity=1
- joint right_f2_j1: limit lower=-1.57079632679 upper=1.57079632679 effort=1 velocity=1 -> lower=-1.57079632679 upper=1.57079632679 effort=28 velocity=1
- joint right_f2_j2: limit lower=-1.57079632679 upper=1.57079632679 effort=1 velocity=1 -> lower=-1.57079632679 upper=1.57079632679 effort=28 velocity=1
- joint right_f3_j0: limit lower=-1.57079632679 upper=1.57079632679 effort=1 velocity=1 -> lower=-1.57079632679 upper=1.57079632679 effort=11 velocity=1
- joint right_f3_j1: limit lower=-1.57079632679 upper=1.57079632679 effort=1 velocity=1 -> lower=-1.57079632679 upper=1.57079632679 effort=28 velocity=1
- joint right_f3_j2: limit lower=-1.57079632679 upper=1.57079632679 effort=1 velocity=1 -> lower=-1.57079632679 upper=1.57079632679 effort=28 velocity=1

File: software/models/mit_gazebo_models/mit_robot_nohands/model.urdf (robot description, URDF)
Before this commit: robot atlas, 41 links, 40 joints
Links:
- link l_foot: mass 0.817 -> 0.867
- link l_lglut: mass 0.69 -> 0.803
- link l_talus: mass 0.817 -> 0.867
- link l_uglut: mass 0.5166 -> 1.51622
- link l_uleg: mass 7.34 -> 7.227
- link ltorso: mass 2.0 -> 1.62729
- link mtorso: mass 0.55 -> 3.8068
- link pelvis: mass 14.2529 -> 12.54638
- link r_foot: mass 0.817 -> 0.867
- link r_lglut: mass 0.69 -> 0.803
- link r_talus: mass 0.817 -> 0.867
- link r_uglut: mass 0.5166 -> 1.51622
- link r_uleg: mass 7.34 -> 7.227
- link utorso: mass 18.484 -> 15.2272

Commit message: updated atlas models for drcsim 2.5
git-svn-id: https://svn.csail.mit.edu/drc@2938 c7283977-0100-402a-a91a-fa70b306dbfe

File: software/models/mit_gazebo_models/mit_robot/model.urdf (robot description, URDF)
Before this commit: robot atlas, 99 links, 98 joints
Links:
- link center_bottom_led_frame: mass 0.1 -> 1e-5
- link center_top_led_frame: mass 0.1 -> 1e-5
- link head: mass 1.4199 -> 1.41984
- link head_hokuyo_frame: mass 0.01 -> 1e-5
- link head_imu_link: mass 0.1 -> 1e-5
- link hokuyo_link: mass 0.057664 -> 0.057654
- link left_camera_frame: mass 0.1 -> 1e-5
- link left_led_frame: mass 0.1 -> 1e-5
- link right_camera_frame: mass 0.1 -> 1e-5
- link right_led_frame: mass 0.1 -> 1e-5

File: software/models/mit_gazebo_models/mit_robot_nohands/model.urdf (robot description, URDF)
Before this commit: robot atlas, 41 links, 40 joints
Links:
- link center_bottom_led_frame: mass 0.1 -> 1e-5
- link center_top_led_frame: mass 0.1 -> 1e-5
- link head: mass 1.4199 -> 1.41984
- link head_hokuyo_frame: mass 0.01 -> 1e-5
- link head_imu_link: mass 0.1 -> 1e-5
- link hokuyo_link: mass 0.057664 -> 0.057654
- link left_camera_frame: mass 0.1 -> 1e-5
- link left_led_frame: mass 0.1 -> 1e-5
- link right_camera_frame: mass 0.1 -> 1e-5
- link right_led_frame: mass 0.1 -> 1e-5
