Commit message: adding 800x800 cams
git-svn-id: https://svn.csail.mit.edu/drc@3048 c7283977-0100-402a-a91a-fa70b306dbfe

File: software/models/mit_gazebo_models/mit_robot/model.urdf (robot description, URDF)
Before this commit: robot atlas, 99 links, 98 joints
Links:
- added link left_palm_left_camera_frame, mass 0.01; visual box size=0.003 0.010 0.007
- added link left_palm_left_camera_optical_frame
- added link left_palm_right_camera_frame, mass 0.01; visual box size=0.003 0.010 0.007
- added link left_palm_right_camera_optical_frame
- added link right_palm_left_camera_frame, mass 0.01; visual box size=0.003 0.010 0.007
- added link right_palm_left_camera_optical_frame
- added link right_palm_right_camera_frame, mass 0.01; visual box size=0.003 0.010 0.007
- added link right_palm_right_camera_optical_frame
Joints:
- added joint left_palm_left_camera_frame_joint: type fixed, parent left_palm, child left_palm_left_camera_frame, origin xyz=0.0435128991906 -0.0451672761576 0.025 rpy=-0.6708 -1.57079632679 3.14159265359
- added joint left_palm_left_camera_optical_frame_joint: type fixed, parent left_palm_left_camera_frame, child left_palm_left_camera_optical_frame, origin xyz=0 0 0 rpy=-1.57079632679 0.0 -1.57079632679
- added joint left_palm_right_camera_frame_joint: type fixed, parent left_palm, child left_palm_right_camera_frame, origin xyz=0.0683774130138 -0.0138342911048 0.025 rpy=-0.6708 -1.57079632679 3.14159265359
- added joint left_palm_right_camera_optical_frame_joint: type fixed, parent left_palm_right_camera_frame, child left_palm_right_camera_optical_frame, origin xyz=0 0 0 rpy=-1.57079632679 0.0 -1.57079632679
- added joint right_palm_left_camera_frame_joint: type fixed, parent right_palm, child right_palm_left_camera_frame, origin xyz=0.0683774130138 0.0138342911048 0.025 rpy=0.6708 -1.57079632679 3.14159265359
- added joint right_palm_left_camera_optical_frame_joint: type fixed, parent right_palm_left_camera_frame, child right_palm_left_camera_optical_frame, origin xyz=0 0 0 rpy=-1.57079632679 0.0 -1.57079632679
- added joint right_palm_right_camera_frame_joint: type fixed, parent right_palm, child right_palm_right_camera_frame, origin xyz=0.0435128991906 0.0451672761576 0.025 rpy=0.6708 -1.57079632679 3.14159265359
- added joint right_palm_right_camera_optical_frame_joint: type fixed, parent right_palm_right_camera_frame, child right_palm_right_camera_optical_frame, origin xyz=0 0 0 rpy=-1.57079632679 0.0 -1.57079632679

Commit message: upgraded drake/gazebo models to prerelease versions
git-svn-id: https://svn.csail.mit.edu/drc@3737 c7283977-0100-402a-a91a-fa70b306dbfe

File: software/models/mit_gazebo_models/mit_robot/model.urdf (robot description, URDF)
Before this commit: robot atlas, 107 links, 106 joints
Links:
- link head: geometry collision box size=0.0468 0.12 0.1184; collision box size=0.1311 0.12 0.0591
- link hokuyo_link: geometry collision box size=0.08 0.06 0.04238; collision cylinder length=0.047 radius=0.024425
- link l_clav: geometry collision box size=0.13 0.15 0.05; collision cylinder length=0.1525 radius=0.045
- link l_farm: geometry collision box size=0.135 0.1 0.045; collision cylinder length=0.125 radius=0.045
- link l_foot: geometry collision box size=0.26 0.124887 0.05; visual mesh filename=package://mit_robot/meshes/l_foot.dae scale=1 1 1
- link l_hand: geometry collision box size=0.13 0.09 0.07; collision cylinder length=0.05 radius=0.03
- link l_larm: geometry collision box size=0.135 0.15 0.06; collision cylinder length=0.125 radius=0.045
- link l_lleg: geometry collision cylinder length=0.40 radius=0.07; visual mesh filename=package://mit_robot/meshes/l_lleg.dae scale=100. 100. 100.
- link l_scap: geometry collision box size=0.15 0.15 0.06; collision cylinder length=0.125 radius=0.045
- link l_uarm: geometry collision box size=0.04 0.07 0.13; collision cylinder length=0.125 radius=0.045
- link l_uleg: geometry collision cylinder length=0.10 radius=0.1; collision cylinder length=0.15 radius=0.07
- link pelvis: geometry collision box size=0.1 0.15 0.2; collision cylinder length=0.05 radius=0.16
- link r_clav: geometry collision box size=0.13 0.15 0.05; collision cylinder length=0.1525 radius=0.045
- link r_farm: geometry collision box size=0.135 0.1 0.045; collision cylinder length=0.125 radius=0.045
- link r_foot: geometry collision box size=0.26 0.124887 0.05; visual mesh filename=package://mit_robot/meshes/r_foot.dae scale=1 1 1
- link r_hand: geometry collision box size=0.13 0.09 0.07; collision cylinder length=0.05 radius=0.03
- link r_larm: geometry collision box size=0.135 0.15 0.06; collision cylinder length=0.125 radius=0.045
- link r_lglut: geometry collision cylinder length=0.060306 radius=0.02009687; collision cylinder length=0.12 radius=0.02
- link r_lleg: geometry collision cylinder length=0.40 radius=0.07; visual mesh filename=package://mit_robot/meshes/r_lleg.dae scale=100. 100. 100.
- link r_scap: geometry collision box size=0.15 0.15 0.06; collision cylinder length=0.125 radius=0.045
- link r_uarm: geometry collision box size=0.04 0.07 0.13; collision cylinder length=0.125 radius=0.045
- link r_uglut: geometry collision cylinder length=0.078396 radius=0.019096; collision cylinder length=0.080842 radius=0.019841
- link r_uleg: geometry collision cylinder length=0.10 radius=0.1; collision cylinder length=0.15 radius=0.07
Joints:
- joint left_f0_j0: limit lower=-1.57079632679 upper=1.57079632679 effort=11 velocity=1 -> lower=-1.57079632679 upper=1.57079632679 effort=11 velocity=-1
- joint left_f0_j1: limit lower=-1.57079632679 upper=1.57079632679 effort=28 velocity=1 -> lower=-1.57079632679 upper=1.57079632679 effort=28 velocity=-1
- joint left_f0_j2: limit lower=-1.57079632679 upper=1.57079632679 effort=28 velocity=1 -> lower=-1.57079632679 upper=1.57079632679 effort=28 velocity=-1
- joint left_f1_j0: limit lower=-1.57079632679 upper=1.57079632679 effort=11 velocity=1 -> lower=-1.57079632679 upper=1.57079632679 effort=11 velocity=-1
- joint left_f1_j1: limit lower=-1.57079632679 upper=1.57079632679 effort=28 velocity=1 -> lower=-1.57079632679 upper=1.57079632679 effort=28 velocity=-1
- joint left_f1_j2: limit lower=-1.57079632679 upper=1.57079632679 effort=28 velocity=1 -> lower=-1.57079632679 upper=1.57079632679 effort=28 velocity=-1
- joint left_f2_j0: limit lower=-1.57079632679 upper=1.57079632679 effort=11 velocity=1 -> lower=-1.57079632679 upper=1.57079632679 effort=11 velocity=-1
- joint left_f2_j1: limit lower=-1.57079632679 upper=1.57079632679 effort=28 velocity=1 -> lower=-1.57079632679 upper=1.57079632679 effort=28 velocity=-1
- joint left_f2_j2: limit lower=-1.57079632679 upper=1.57079632679 effort=28 velocity=1 -> lower=-1.57079632679 upper=1.57079632679 effort=28 velocity=-1
- joint left_f3_j0: limit lower=-1.57079632679 upper=1.57079632679 effort=11 velocity=1 -> lower=-1.57079632679 upper=1.57079632679 effort=11 velocity=-1
- joint left_f3_j1: limit lower=-1.57079632679 upper=1.57079632679 effort=28 velocity=1 -> lower=-1.57079632679 upper=1.57079632679 effort=28 velocity=-1
- joint left_f3_j2: limit lower=-1.57079632679 upper=1.57079632679 effort=28 velocity=1 -> lower=-1.57079632679 upper=1.57079632679 effort=28 velocity=-1
- joint neck_ay: origin xyz=0.16555 0 0.50823 rpy=0 -0 0 -> xyz=0.21672 0 0.53796 rpy=0 -0 0
- joint right_f0_j0: limit lower=-1.57079632679 upper=1.57079632679 effort=11 velocity=1 -> lower=-1.57079632679 upper=1.57079632679 effort=11 velocity=-1
- joint right_f0_j1: limit lower=-1.57079632679 upper=1.57079632679 effort=28 velocity=1 -> lower=-1.57079632679 upper=1.57079632679 effort=28 velocity=-1
- joint right_f0_j2: limit lower=-1.57079632679 upper=1.57079632679 effort=28 velocity=1 -> lower=-1.57079632679 upper=1.57079632679 effort=28 velocity=-1
- joint right_f1_j0: limit lower=-1.57079632679 upper=1.57079632679 effort=11 velocity=1 -> lower=-1.57079632679 upper=1.57079632679 effort=11 velocity=-1
- joint right_f1_j1: limit lower=-1.57079632679 upper=1.57079632679 effort=28 velocity=1 -> lower=-1.57079632679 upper=1.57079632679 effort=28 velocity=-1
- joint right_f1_j2: limit lower=-1.57079632679 upper=1.57079632679 effort=28 velocity=1 -> lower=-1.57079632679 upper=1.57079632679 effort=28 velocity=-1
- joint right_f2_j0: limit lower=-1.57079632679 upper=1.57079632679 effort=11 velocity=1 -> lower=-1.57079632679 upper=1.57079632679 effort=11 velocity=-1
- joint right_f2_j1: limit lower=-1.57079632679 upper=1.57079632679 effort=28 velocity=1 -> lower=-1.57079632679 upper=1.57079632679 effort=28 velocity=-1
- joint right_f2_j2: limit lower=-1.57079632679 upper=1.57079632679 effort=28 velocity=1 -> lower=-1.57079632679 upper=1.57079632679 effort=28 velocity=-1
- joint right_f3_j0: limit lower=-1.57079632679 upper=1.57079632679 effort=11 velocity=1 -> lower=-1.57079632679 upper=1.57079632679 effort=11 velocity=-1
- joint right_f3_j1: limit lower=-1.57079632679 upper=1.57079632679 effort=28 velocity=1 -> lower=-1.57079632679 upper=1.57079632679 effort=28 velocity=-1
- joint right_f3_j2: limit lower=-1.57079632679 upper=1.57079632679 effort=28 velocity=1 -> lower=-1.57079632679 upper=1.57079632679 effort=28 velocity=-1

File: software/models/mit_gazebo_models/mit_robot/xacro/atlas.urdf.xacro (robot description, xacro)
@@ -1,3 +1,3 @@
-<robot xmlns:xacro="http://playerstage.sourceforge.net/gazebo/xmlschema/#interface" name="atlas" >
+<robot name="atlas" >
   <include filename="$(find mit_drcsim_scripts)/models/mit_robot/xacro/atlas_skeleton.urdf" />
   <include filename="$(find atlas_description)/urdf/atlas.transmission" />

File: software/models/mit_gazebo_models/mit_robot/xacro/atlas_sandia_hands.urdf.xacro (robot description, xacro)
@@ -2,8 +2,8 @@
   <include filename="$(find mit_drcsim_scripts)/models/mit_robot/xacro/atlas_skeleton.urdf" />
   <include filename="$(find sandia_hand_description)/urdf/sandia_hand_simple_shapes.urdf.xacro" />
-  <xacro:sandia_hand side="right" parent="r_hand" reflect="1">
+  <xacro:sandia_hand side="right" parent="r_hand" reflect="1" joint_type="revolute" thumb_angle="0">
     <origin xyz="0 -0.1 0" rpy="-1.57079 0 -1.57079"/>
   </xacro:sandia_hand>
-  <xacro:sandia_hand side="left" parent="l_hand" reflect="-1">
+  <xacro:sandia_hand side="left" parent="l_hand" reflect="-1" joint_type="revolute" thumb_angle="0">
     <origin xyz="0  0.1 0" rpy=" 1.57079 0  1.57079"/>
   </xacro:sandia_hand>
@@ -12,5 +12,5 @@
   <include filename="$(find mit_drcsim_scripts)/models/mit_robot/xacro/mit_atlas.gazebo" />
   <gazebo>
-    <!-- include plugin for snadia hands -->
+    <!-- include plugin for sandia hands -->
     <plugin name="sandia_hand_plugin" filename="libSandiaHandPlugin.so"/>
   </gazebo>

File: software/models/mit_gazebo_models/mit_robot/xacro/atlas_skeleton.urdf (robot description, URDF)
Before this commit: robot drc_skeleton, 28 links, 28 joints
Links:
- link l_clav: geometry collision box size=0.13 0.15 0.05; collision cylinder length=0.1525 radius=0.045
- link l_farm: geometry collision box size=0.135 0.1 0.045; collision cylinder length=0.125 radius=0.045
- link l_foot: geometry collision box size=0.26 0.124887 0.05; visual mesh filename=package://mit_robot/meshes/l_foot.dae scale=1 1 1
- link l_hand: geometry collision box size=0.13 0.09 0.07; collision cylinder length=0.05 radius=0.03
- link l_larm: geometry collision box size=0.135 0.15 0.06; collision cylinder length=0.125 radius=0.045
- link l_lleg: geometry collision cylinder length=0.40 radius=0.07; visual mesh filename=package://mit_robot/meshes/l_lleg.dae scale=100. 100. 100.
- link l_scap: geometry collision box size=0.15 0.15 0.06; collision cylinder length=0.125 radius=0.045
- link l_uarm: geometry collision box size=0.04 0.07 0.13; collision cylinder length=0.125 radius=0.045
- link l_uleg: geometry collision cylinder length=0.10 radius=0.1; collision cylinder length=0.15 radius=0.07
- link pelvis: geometry collision box size=0.1 0.15 0.2; collision cylinder length=0.05 radius=0.16
- link r_clav: geometry collision box size=0.13 0.15 0.05; collision cylinder length=0.1525 radius=0.045
- link r_farm: geometry collision box size=0.135 0.1 0.045; collision cylinder length=0.125 radius=0.045
- link r_foot: geometry collision box size=0.26 0.124887 0.05; visual mesh filename=package://mit_robot/meshes/r_foot.dae scale=1 1 1
- link r_hand: geometry collision box size=0.13 0.09 0.07; collision cylinder length=0.05 radius=0.03
- link r_larm: geometry collision box size=0.135 0.15 0.06; collision cylinder length=0.125 radius=0.045
- link r_lglut: geometry collision cylinder length=0.060306 radius=0.02009687; collision cylinder length=0.12 radius=0.02
- link r_lleg: geometry collision cylinder length=0.40 radius=0.07; visual mesh filename=package://mit_robot/meshes/r_lleg.dae scale=100. 100. 100.
- link r_scap: geometry collision box size=0.15 0.15 0.06; collision cylinder length=0.125 radius=0.045
- link r_uarm: geometry collision box size=0.04 0.07 0.13; collision cylinder length=0.125 radius=0.045
- link r_uglut: geometry collision cylinder length=0.078396 radius=0.019096; collision cylinder length=0.080842 radius=0.019841
- link r_uleg: geometry collision cylinder length=0.10 radius=0.1; collision cylinder length=0.15 radius=0.07
Joints:
- joint neck_ay: origin xyz=0.16555 0 0.50823 rpy=0 -0 0 -> xyz=0.21672 0 0.53796 rpy=0 -0 0

File: software/models/mit_gazebo_models/mit_robot_drake/model_minimal_contact.urdf (robot description, URDF)
Before this commit: robot atlas, 29 links, 28 joints
Links:
- link l_lleg: geometry collision sphere radius=0; visual mesh filename=package://mit_drcsim_scripts/models/mit_robot/meshes/l_lleg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 scale=100. 100. 100.
- link l_uleg: geometry visual mesh filename=package://mit_drcsim_scripts/models/mit_robot/meshes/l_uleg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 scale=100. 100. 100.
- link pelvis: geometry visual mesh filename=package://mit_drcsim_scripts/models/mit_robot/meshes/pelvis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 scale=100. 100. 100.
- link r_larm: geometry visual mesh filename=package://mit_drcsim_scripts/models/mit_robot/meshes/r_larm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 scale=100. 100. 100.
- link r_lglut: geometry visual mesh filename=package://mit_drcsim_scripts/models/mit_robot/meshes/r_lglu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 scale=100. 100. 100.
- link r_lleg: geometry collision sphere radius=0; visual mesh filename=package://mit_drcsim_scripts/models/mit_robot/meshes/r_lleg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 scale=100. 100. 100.
- link r_uarm: geometry visual mesh filename=package://mit_drcsim_scripts/models/mit_robot/meshes/r_uarm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 scale=100. 100. 100.
- link r_uglut: geometry visual mesh filename=package://mit_drcsim_scripts/models/mit_robot/meshes/r_uglu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 scale=100. 100. 100.
- link r_uleg: geometry visual mesh filename=package://mit_drcsim_scripts/models/mit_robot/meshes/r_uleg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 scale=100. 100. 100.
Joints:
- joint neck_ay: origin xyz=0.16555 0 0.50823 rpy=0 -0 0 -> xyz=0.21672 0 0.53796 rpy=0 -0 0

File: software/models/mit_gazebo_models/mit_robot_drake/model_minimal_contact_point_hands.urdf (robot description, URDF)
Before this commit: robot atlas, 31 links, 30 joints
Links:
- link l_lleg: geometry collision sphere radius=0; visual mesh filename=package://mit_drcsim_scripts/models/mit_robot/meshes/l_lleg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 scale=100. 100. 100.
- link l_uleg: geometry visual mesh filename=package://mit_drcsim_scripts/models/mit_robot/meshes/l_uleg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 scale=100. 100. 100.
- link pelvis: geometry visual mesh filename=package://mit_drcsim_scripts/models/mit_robot/meshes/pelvis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 scale=100. 100. 100.
- link r_larm: geometry visual mesh filename=package://mit_drcsim_scripts/models/mit_robot/meshes/r_larm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 scale=100. 100. 100.
- link r_lglut: geometry visual mesh filename=package://mit_drcsim_scripts/models/mit_robot/meshes/r_lglu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 scale=100. 100. 100.
- link r_lleg: geometry collision sphere radius=0; visual mesh filename=package://mit_drcsim_scripts/models/mit_robot/meshes/r_lleg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 scale=100. 100. 100.
- link r_uarm: geometry visual mesh filename=package://mit_drcsim_scripts/models/mit_robot/meshes/r_uarm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 scale=100. 100. 100.
- link r_uglut: geometry visual mesh filename=package://mit_drcsim_scripts/models/mit_robot/meshes/r_uglu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 scale=100. 100. 100.
- link r_uleg: geometry visual mesh filename=package://mit_drcsim_scripts/models/mit_robot/meshes/r_uleg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 scale=100. 100. 100.
Joints:
- joint neck_ay: origin xyz=0.16555 0 0.50823 rpy=0 -0 0 -> xyz=0.21672 0 0.53796 rpy=0 -0 0

File: software/models/mit_gazebo_models/mit_robot_drake/model_minimal_contact_with_hands.urdf (robot description, URDF)
Before this commit: robot atlas, 101 links, 100 joints
Links:
- link l_lleg: geometry collision sphere radius=0; visual mesh filename=package://mit_drcsim_scripts/models/mit_robot/meshes/l_lleg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 scale=100. 100. 100.
- link l_uleg: geometry visual mesh filename=package://mit_drcsim_scripts/models/mit_robot/meshes/l_uleg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 scale=100. 100. 100.
- link pelvis: geometry visual mesh filename=package://mit_drcsim_scripts/models/mit_robot/meshes/pelvis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 scale=100. 100. 100.
- link r_larm: geometry visual mesh filename=package://mit_drcsim_scripts/models/mit_robot/meshes/r_larm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 scale=100. 100. 100.
- link r_lglut: geometry visual mesh filename=package://mit_drcsim_scripts/models/mit_robot/meshes/r_lglu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 scale=100. 100. 100.
- link r_lleg: geometry collision sphere radius=0; visual mesh filename=package://mit_drcsim_scripts/models/mit_robot/meshes/r_lleg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 scale=100. 100. 100.
- link r_uarm: geometry visual mesh filename=package://mit_drcsim_scripts/models/mit_robot/meshes/r_uarm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 scale=100. 100. 100.
- link r_uglut: geometry visual mesh filename=package://mit_drcsim_scripts/models/mit_robot/meshes/r_uglu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 scale=100. 100. 100.
- link r_uleg: geometry visual mesh filename=package://mit_drcsim_scripts/models/mit_robot/meshes/r_uleg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 scale=100. 100. 100.
Joints:
- joint neck_ay: origin xyz=0.16555 0 0.50823 rpy=0 -0 0 -> xyz=0.21672 0 0.53796 rpy=0 -0 0

File: software/models/mit_gazebo_models/mit_robot_drake/xacro/atlas_skeleton_minimal_contact.urdf (robot description, URDF)
Before this commit: robot drc_skeleton, 28 links, 28 joints
Links:
- link l_lleg: geometry collision sphere radius=0; visual mesh filename=package://mit_drcsim_scripts/models/mit_robot/meshes/l_lleg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 scale=100. 100. 100.
- link l_uleg: geometry visual mesh filename=package://mit_drcsim_scripts/models/mit_robot/meshes/l_uleg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 scale=100. 100. 100.
- link pelvis: geometry visual mesh filename=package://mit_drcsim_scripts/models/mit_robot/meshes/pelvis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 scale=100. 100. 100.
- link r_larm: geometry visual mesh filename=package://mit_drcsim_scripts/models/mit_robot/meshes/r_larm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 scale=100. 100. 100.
- link r_lglut: geometry visual mesh filename=package://mit_drcsim_scripts/models/mit_robot/meshes/r_lglu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 scale=100. 100. 100.
- link r_lleg: geometry collision sphere radius=0; visual mesh filename=package://mit_drcsim_scripts/models/mit_robot/meshes/r_lleg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 scale=100. 100. 100.
- link r_uarm: geometry visual mesh filename=package://mit_drcsim_scripts/models/mit_robot/meshes/r_uarm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 scale=100. 100. 100.
- link r_uglut: geometry visual mesh filename=package://mit_drcsim_scripts/models/mit_robot/meshes/r_uglu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 scale=100. 100. 100.
- link r_uleg: geometry visual mesh filename=package://mit_drcsim_scripts/models/mit_robot/meshes/r_uleg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 scale=100. 100. 100.
Joints:
- joint neck_ay: origin xyz=0.16555 0 0.50823 rpy=0 -0 0 -> xyz=0.21672 0 0.53796 rpy=0 -0 0

File: software/models/mit_gazebo_models/mit_robot_nohands/model.urdf (robot description, URDF)
Before this commit: robot atlas, 41 links, 40 joints
Links:
- link head: geometry collision box size=0.0468 0.12 0.1184; collision box size=0.1311 0.12 0.0591
- link hokuyo_link: geometry collision box size=0.08 0.06 0.04238; collision cylinder length=0.047 radius=0.024425
- link l_clav: geometry collision box size=0.13 0.15 0.05; collision cylinder length=0.1525 radius=0.045
- link l_farm: geometry collision box size=0.135 0.1 0.045; collision cylinder length=0.125 radius=0.045
- link l_foot: geometry collision box size=0.26 0.124887 0.05; visual mesh filename=package://mit_robot/meshes/l_foot.dae scale=1 1 1
- link l_hand: geometry collision box size=0.13 0.09 0.07; collision cylinder length=0.05 radius=0.03
- link l_larm: geometry collision box size=0.135 0.15 0.06; collision cylinder length=0.125 radius=0.045
- link l_lleg: geometry collision cylinder length=0.40 radius=0.07; visual mesh filename=package://mit_robot/meshes/l_lleg.dae scale=100. 100. 100.
- link l_scap: geometry collision box size=0.15 0.15 0.06; collision cylinder length=0.125 radius=0.045
- link l_uarm: geometry collision box size=0.04 0.07 0.13; collision cylinder length=0.125 radius=0.045
- link l_uleg: geometry collision cylinder length=0.10 radius=0.1; collision cylinder length=0.15 radius=0.07
- link pelvis: geometry collision box size=0.1 0.15 0.2; collision cylinder length=0.05 radius=0.16
- link r_clav: geometry collision box size=0.13 0.15 0.05; collision cylinder length=0.1525 radius=0.045
- link r_farm: geometry collision box size=0.135 0.1 0.045; collision cylinder length=0.125 radius=0.045
- link r_foot: geometry collision box size=0.26 0.124887 0.05; visual mesh filename=package://mit_robot/meshes/r_foot.dae scale=1 1 1
- link r_hand: geometry collision box size=0.13 0.09 0.07; collision cylinder length=0.05 radius=0.03
- link r_larm: geometry collision box size=0.135 0.15 0.06; collision cylinder length=0.125 radius=0.045
- link r_lglut: geometry collision cylinder length=0.060306 radius=0.02009687; collision cylinder length=0.12 radius=0.02
- link r_lleg: geometry collision cylinder length=0.40 radius=0.07; visual mesh filename=package://mit_robot/meshes/r_lleg.dae scale=100. 100. 100.
- link r_scap: geometry collision box size=0.15 0.15 0.06; collision cylinder length=0.125 radius=0.045
- link r_uarm: geometry collision box size=0.04 0.07 0.13; collision cylinder length=0.125 radius=0.045
- link r_uglut: geometry collision cylinder length=0.078396 radius=0.019096; collision cylinder length=0.080842 radius=0.019841
- link r_uleg: geometry collision cylinder length=0.10 radius=0.1; collision cylinder length=0.15 radius=0.07
Joints:
- joint neck_ay: origin xyz=0.16555 0 0.50823 rpy=0 -0 0 -> xyz=0.21672 0 0.53796 rpy=0 -0 0

File: software/models/mit_gazebo_models/multisense_sl/multisense_sl.urdf (robot description, URDF)
Before this commit: robot multisense_sl, 12 links, 11 joints
Links:
- link head: geometry collision box size=0.0468 0.12 0.1184; collision box size=0.1311 0.12 0.0591
- link hokuyo_link: geometry collision box size=0.08 0.06 0.04238; collision cylinder length=0.047 radius=0.024425
