Commit message: updated mesh scaling and foot friction coeff to match drcsim 2.6 release
git-svn-id: https://svn.csail.mit.edu/drc@3765 c7283977-0100-402a-a91a-fa70b306dbfe

File: software/models/mit_gazebo_models/mit_robot/model.urdf (robot description, URDF)
Before this commit: robot atlas, 107 links, 106 joints
Links:
- link l_lleg: geometry collision cylinder length=0.40 radius=0.07; visual mesh filename=package://mit_robot/meshes/l_lleg.dae scale=1 1 1
- link l_uleg: geometry collision cylinder length=0.10 radius=0.1; collision cylinder length=0.15 radius=0.07
- link pelvis: geometry collision box size=0.1 0.15 0.2; collision cylinder length=0.05 radius=0.16
- link r_larm: geometry collision box size=0.135 0.15 0.06; collision cylinder length=0.125 radius=0.045
- link r_lglut: geometry collision cylinder length=0.060306 radius=0.02009687; collision cylinder length=0.12 radius=0.02
- link r_lleg: geometry collision cylinder length=0.40 radius=0.07; visual mesh filename=package://mit_robot/meshes/r_lleg.dae scale=1 1 1
- link r_uarm: geometry collision box size=0.04 0.07 0.13; collision cylinder length=0.125 radius=0.045
- link r_uglut: geometry collision cylinder length=0.078396 radius=0.019096; collision cylinder length=0.080842 radius=0.019841
- link r_uleg: geometry collision cylinder length=0.10 radius=0.1; collision cylinder length=0.15 radius=0.07

File: software/models/mit_gazebo_models/mit_robot/xacro/atlas_skeleton.urdf (robot description, URDF)
Before this commit: robot drc_skeleton, 28 links, 28 joints
Links:
- link l_lleg: geometry collision cylinder length=0.40 radius=0.07; visual mesh filename=package://mit_robot/meshes/l_lleg.dae scale=1 1 1
- link l_uleg: geometry collision cylinder length=0.10 radius=0.1; collision cylinder length=0.15 radius=0.07
- link pelvis: geometry collision box size=0.1 0.15 0.2; collision cylinder length=0.05 radius=0.16
- link r_larm: geometry collision box size=0.135 0.15 0.06; collision cylinder length=0.125 radius=0.045
- link r_lglut: geometry collision cylinder length=0.060306 radius=0.02009687; collision cylinder length=0.12 radius=0.02
- link r_lleg: geometry collision cylinder length=0.40 radius=0.07; visual mesh filename=package://mit_robot/meshes/r_lleg.dae scale=1 1 1
- link r_uarm: geometry collision box size=0.04 0.07 0.13; collision cylinder length=0.125 radius=0.045
- link r_uglut: geometry collision cylinder length=0.078396 radius=0.019096; collision cylinder length=0.080842 radius=0.019841
- link r_uleg: geometry collision cylinder length=0.10 radius=0.1; collision cylinder length=0.15 radius=0.07

Commit message: cleaing up  a bit: mit models use default gazebo file plus a small one with our rateset plugin
git-svn-id: https://svn.csail.mit.edu/drc@3917 c7283977-0100-402a-a91a-fa70b306dbfe

File: software/models/mit_gazebo_models/mit_robot/model.urdf (robot description, URDF)
Before this commit: robot atlas, 107 links, 106 joints
Links:
- removed link imu_link
Joints:
- removed joint imu_joint

File: software/models/mit_gazebo_models/mit_robot/xacro/atlas.urdf.xacro (robot description, xacro)
@@ -1,4 +1,5 @@
 <robot name="atlas" >
   <include filename="$(find mit_drcsim_scripts)/models/mit_robot/xacro/atlas_skeleton.urdf" />
+  <include filename="$(find atlas_description)/urdf/atlas.gazebo" />
   <include filename="$(find atlas_description)/urdf/atlas.transmission" />
   <include filename="$(find multisense_sl_description)/multisense_sl_description.urdf" />

Commit message: whoops, xacros are now fixed
git-svn-id: https://svn.csail.mit.edu/drc@3950 c7283977-0100-402a-a91a-fa70b306dbfe

File: software/models/mit_gazebo_models/mit_robot/model.urdf (robot description, URDF)
Before this commit: robot atlas, 106 links, 105 joints
Links:
- added link imu_link, mass 0.1; visual box size=0.01 0.01 0.01
Joints:
- added joint imu_joint: type fixed, parent pelvis, child imu_link, origin xyz=0.05991527603 0 -0.01415 rpy=0 0 0

File: software/models/mit_gazebo_models/mit_robot/xacro/atlas_sandia_hands.urdf.xacro (robot description, xacro)
@@ -8,4 +8,5 @@
     <origin xyz="0  0.1 0" rpy=" 1.57079 0  1.57079"/>
   </xacro:sandia_hand>
+  <include filename="$(find atlas_description)/urdf/atlas.gazebo" />
   <include filename="$(find atlas_description)/urdf/atlas.transmission" />
   <include filename="$(find multisense_sl_description)/multisense_sl_description.urdf" />

File: software/models/mit_gazebo_models/mit_robot/xacro/atlas_sandia_hands_stumps.urdf.xacro (robot description, xacro)
@@ -8,4 +8,5 @@
     <origin xyz="0  0.1 0" rpy=" 1.57079 0  1.57079"/>
   </xacro:sandia_hand>
+  <include filename="$(find atlas_description)/urdf/atlas.gazebo" />
   <include filename="$(find atlas_description)/urdf/atlas.transmission" />
   <include filename="$(find multisense_sl_description)/multisense_sl_description.urdf" />

Commit message: updating model ankle joint limits and knee torque limit to match their forthcoming values
git-svn-id: https://svn.csail.mit.edu/drc@4087 c7283977-0100-402a-a91a-fa70b306dbfe

File: software/models/mit_gazebo_models/mit_robot/model.urdf (robot description, URDF)
Before this commit: robot atlas, 107 links, 106 joints
Joints:
- joint l_leg_kny: limit lower=0 upper=2.45 effort=220 velocity=12 -> lower=0 upper=2.45 effort=400 velocity=12
- joint l_leg_uay: limit lower=-0.698 upper=0.698 effort=220 velocity=12 -> lower=-0.9 upper=0.698 effort=220 velocity=12
- joint r_leg_kny: limit lower=0 upper=2.45 effort=220 velocity=12 -> lower=0 upper=2.45 effort=400 velocity=12
- joint r_leg_uay: limit lower=-0.698 upper=0.698 effort=220 velocity=12 -> lower=-0.9 upper=0.698 effort=220 velocity=12

File: software/models/mit_gazebo_models/mit_robot/xacro/atlas_skeleton.urdf (robot description, URDF)
Before this commit: robot drc_skeleton, 28 links, 28 joints
Joints:
- joint l_leg_kny: limit lower=0 upper=2.45 effort=220 velocity=12 -> lower=0 upper=2.45 effort=400 velocity=12
- joint l_leg_uay: limit lower=-0.698 upper=0.698 effort=220 velocity=12 -> lower=-0.9 upper=0.698 effort=220 velocity=12
- joint r_leg_kny: limit lower=0 upper=2.45 effort=220 velocity=12 -> lower=0 upper=2.45 effort=400 velocity=12
- joint r_leg_uay: limit lower=-0.698 upper=0.698 effort=220 velocity=12 -> lower=-0.9 upper=0.698 effort=220 velocity=12

File: software/models/mit_gazebo_models/mit_robot_drake/model_minimal_contact.urdf (robot description, URDF)
Before this commit: robot atlas, 29 links, 28 joints
Joints:
- joint l_leg_kny: limit lower=0 upper=2.45 effort=220 velocity=12 -> lower=0 upper=2.45 effort=400 velocity=12
- joint l_leg_uay: limit lower=-0.698 upper=0.698 effort=220 velocity=12 -> lower=-0.9 upper=0.698 effort=220 velocity=12
- joint r_leg_kny: limit lower=0 upper=2.45 effort=220 velocity=12 -> lower=0 upper=2.45 effort=400 velocity=12
- joint r_leg_uay: limit lower=-0.698 upper=0.698 effort=220 velocity=12 -> lower=-0.9 upper=0.698 effort=220 velocity=12

File: software/models/mit_gazebo_models/mit_robot_drake/model_minimal_contact_point_hands.urdf (robot description, URDF)
Before this commit: robot atlas, 31 links, 30 joints
Joints:
- joint l_leg_kny: limit lower=0 upper=2.45 effort=220 velocity=12 -> lower=0 upper=2.45 effort=400 velocity=12
- joint l_leg_uay: limit lower=-0.698 upper=0.698 effort=220 velocity=12 -> lower=-0.9 upper=0.698 effort=220 velocity=12
- joint r_leg_kny: limit lower=0 upper=2.45 effort=220 velocity=12 -> lower=0 upper=2.45 effort=400 velocity=12
- joint r_leg_uay: limit lower=-0.698 upper=0.698 effort=220 velocity=12 -> lower=-0.9 upper=0.698 effort=220 velocity=12

File: software/models/mit_gazebo_models/mit_robot_drake/model_minimal_contact_with_hands.urdf (robot description, URDF)
Before this commit: robot atlas, 101 links, 100 joints
Joints:
- joint l_leg_kny: limit lower=0 upper=2.45 effort=220 velocity=12 -> lower=0 upper=2.45 effort=400 velocity=12
- joint l_leg_uay: limit lower=-0.698 upper=0.698 effort=220 velocity=12 -> lower=-0.9 upper=0.698 effort=220 velocity=12
- joint r_leg_kny: limit lower=0 upper=2.45 effort=220 velocity=12 -> lower=0 upper=2.45 effort=400 velocity=12
- joint r_leg_uay: limit lower=-0.698 upper=0.698 effort=220 velocity=12 -> lower=-0.9 upper=0.698 effort=220 velocity=12

File: software/models/mit_gazebo_models/mit_robot_drake/xacro/atlas_skeleton_minimal_contact.urdf (robot description, URDF)
Before this commit: robot drc_skeleton, 28 links, 28 joints
Joints:
- joint l_leg_kny: limit lower=0 upper=2.45 effort=220 velocity=12 -> lower=0 upper=2.45 effort=400 velocity=12
- joint l_leg_uay: limit lower=-0.698 upper=0.698 effort=220 velocity=12 -> lower=-0.9 upper=0.698 effort=220 velocity=12
- joint r_leg_kny: limit lower=0 upper=2.45 effort=220 velocity=12 -> lower=0 upper=2.45 effort=400 velocity=12
- joint r_leg_uay: limit lower=-0.698 upper=0.698 effort=220 velocity=12 -> lower=-0.9 upper=0.698 effort=220 velocity=12

File: software/models/mit_gazebo_models/mit_robot_drake/xacro/atlas_skeleton_simple_visuals.urdf (robot description, URDF)
Before this commit: robot drc_skeleton, 28 links, 28 joints
Joints:
- joint l_leg_kny: limit lower=0 upper=2.45 effort=220 velocity=12 -> lower=0 upper=2.45 effort=400 velocity=12
- joint l_leg_uay: limit lower=-0.698 upper=0.698 effort=220 velocity=12 -> lower=-0.9 upper=0.698 effort=220 velocity=12
- joint r_leg_kny: limit lower=0 upper=2.45 effort=220 velocity=12 -> lower=0 upper=2.45 effort=400 velocity=12
- joint r_leg_uay: limit lower=-0.698 upper=0.698 effort=220 velocity=12 -> lower=-0.9 upper=0.698 effort=220 velocity=12

File: software/models/mit_gazebo_models/mit_robot_drake/xacro/atlas_skeleton_simple_visuals_minimal_contact.urdf (robot description, URDF)
Before this commit: robot drc_skeleton, 28 links, 28 joints
Joints:
- joint l_leg_kny: limit lower=0 upper=2.45 effort=220 velocity=12 -> lower=0 upper=2.45 effort=400 velocity=12
- joint l_leg_uay: limit lower=-0.698 upper=0.698 effort=220 velocity=12 -> lower=-0.9 upper=0.698 effort=220 velocity=12
- joint r_leg_kny: limit lower=0 upper=2.45 effort=220 velocity=12 -> lower=0 upper=2.45 effort=400 velocity=12
- joint r_leg_uay: limit lower=-0.698 upper=0.698 effort=220 velocity=12 -> lower=-0.9 upper=0.698 effort=220 velocity=12

File: software/models/mit_gazebo_models/mit_robot_nohands/model.urdf (robot description, URDF)
Before this commit: robot atlas, 41 links, 40 joints
Joints:
- joint l_leg_kny: limit lower=0 upper=2.45 effort=220 velocity=12 -> lower=0 upper=2.45 effort=400 velocity=12
- joint l_leg_uay: limit lower=-0.698 upper=0.698 effort=220 velocity=12 -> lower=-0.9 upper=0.698 effort=220 velocity=12
- joint r_leg_kny: limit lower=0 upper=2.45 effort=220 velocity=12 -> lower=0 upper=2.45 effort=400 velocity=12
- joint r_leg_uay: limit lower=-0.698 upper=0.698 effort=220 velocity=12 -> lower=-0.9 upper=0.698 effort=220 velocity=12

Commit message: updating r_leg_uhz effort to match left leg (fix from todays drcsim release)
git-svn-id: https://svn.csail.mit.edu/drc@4600 c7283977-0100-402a-a91a-fa70b306dbfe

File: software/models/mit_gazebo_models/mit_robot/model.urdf (robot description, URDF)
Before this commit: robot atlas, 107 links, 106 joints
Joints:
- joint r_leg_uhz: limit lower=-1.14 upper=0.32 effort=260 velocity=12 -> lower=-1.14 upper=0.32 effort=110 velocity=12

File: software/models/mit_gazebo_models/mit_robot/xacro/atlas_skeleton.urdf (robot description, URDF)
Before this commit: robot drc_skeleton, 28 links, 28 joints
Joints:
- joint r_leg_uhz: limit lower=-1.14 upper=0.32 effort=260 velocity=12 -> lower=-1.14 upper=0.32 effort=110 velocity=12

File: software/models/mit_gazebo_models/mit_robot_drake/model_minimal_contact.urdf (robot description, URDF)
Before this commit: robot atlas, 29 links, 28 joints
Joints:
- joint r_leg_uhz: limit lower=-1.14 upper=0.32 effort=260 velocity=12 -> lower=-1.14 upper=0.32 effort=110 velocity=12

File: software/models/mit_gazebo_models/mit_robot_drake/model_minimal_contact_point_hands.urdf (robot description, URDF)
Before this commit: robot atlas, 31 links, 30 joints
Joints:
- joint r_leg_uhz: limit lower=-1.14 upper=0.32 effort=260 velocity=12 -> lower=-1.14 upper=0.32 effort=110 velocity=12

File: software/models/mit_gazebo_models/mit_robot_drake/model_minimal_contact_with_hands.urdf (robot description, URDF)
Before this commit: robot atlas, 101 links, 100 joints
Joints:
- joint r_leg_uhz: limit lower=-1.14 upper=0.32 effort=260 velocity=12 -> lower=-1.14 upper=0.32 effort=110 velocity=12

File: software/models/mit_gazebo_models/mit_robot_drake/model_simple_visuals_minimal_contact_point_hands.urdf (robot description, URDF)
Before this commit: robot atlas, 31 links, 30 joints
Joints:
- joint r_leg_uhz: limit lower=-1.14 upper=0.32 effort=260 velocity=12 -> lower=-1.14 upper=0.32 effort=110 velocity=12

File: software/models/mit_gazebo_models/mit_robot_drake/model_simple_visuals_point_hands.urdf (robot description, URDF)
Before this commit: robot atlas, 31 links, 30 joints
Joints:
- joint r_leg_uhz: limit lower=-1.14 upper=0.32 effort=260 velocity=12 -> lower=-1.14 upper=0.32 effort=110 velocity=12

File: software/models/mit_gazebo_models/mit_robot_drake/xacro/atlas_skeleton_minimal_contact.urdf (robot description, URDF)
Before this commit: robot drc_skeleton, 28 links, 28 joints
Joints:
- joint r_leg_uhz: limit lower=-1.14 upper=0.32 effort=260 velocity=12 -> lower=-1.14 upper=0.32 effort=110 velocity=12

File: software/models/mit_gazebo_models/mit_robot_drake/xacro/atlas_skeleton_simple_visuals.urdf (robot description, URDF)
Before this commit: robot drc_skeleton, 28 links, 28 joints
Joints:
- joint r_leg_uhz: limit lower=-1.14 upper=0.32 effort=260 velocity=12 -> lower=-1.14 upper=0.32 effort=110 velocity=12

File: software/models/mit_gazebo_models/mit_robot_drake/xacro/atlas_skeleton_simple_visuals_minimal_contact.urdf (robot description, URDF)
Before this commit: robot drc_skeleton, 28 links, 28 joints
Joints:
- joint r_leg_uhz: limit lower=-1.14 upper=0.32 effort=260 velocity=12 -> lower=-1.14 upper=0.32 effort=110 velocity=12

File: software/models/mit_gazebo_models/mit_robot_nohands/model.urdf (robot description, URDF)
Before this commit: robot atlas, 41 links, 40 joints
Joints:
- joint r_leg_uhz: limit lower=-1.14 upper=0.32 effort=260 velocity=12 -> lower=-1.14 upper=0.32 effort=110 velocity=12
