Commit message: changing to bdi joint naming convention
git-svn-id: https://svn.csail.mit.edu/drc/trunk@5735 c7283977-0100-402a-a91a-fa70b306dbfe

File: software/models/mit_gazebo_models/mit_robot/model.urdf (robot description, URDF)
Before this commit: robot atlas, 107 links, 106 joints
Joints:
- joint back_bky: axis 0 0 1 -> 0 1 0; child ltorso -> mtorso; limit lower=-0.610865 upper=0.610865 effort=124.016 velocity=12 -> lower=-1.2 upper=1.28 effort=206.843 velocity=12; origin xyz=-0.0125 0 0 rpy=0 -0 0 -> xyz=0 0 0.09 rpy=0 -0 0; parent pelvis -> ltorso
- joint back_bkz: axis 0 1 0 -> 0 0 1; child mtorso -> ltorso; limit lower=-1.2 upper=1.28 effort=206.843 velocity=12 -> lower=-0.610865 upper=0.610865 effort=124.016 velocity=12; origin xyz=0 0 0.09 rpy=0 -0 0 -> xyz=-0.0125 0 0 rpy=0 -0 0; parent ltorso -> pelvis

File: software/models/mit_gazebo_models/mit_robot/xacro/atlas_skeleton.urdf (robot description, URDF)
Before this commit: robot drc_skeleton, 28 links, 28 joints
Joints:
- removed joint back_lbz
- removed joint back_mby
- removed joint back_ubx
- removed joint l_leg_lax
- removed joint l_leg_lhy
- removed joint l_leg_mhx
- removed joint l_leg_uay
- removed joint l_leg_uhz
- removed joint r_leg_lax
- removed joint r_leg_lhy
- removed joint r_leg_mhx
- removed joint r_leg_uay
- removed joint r_leg_uhz
- added joint back_bkx: type revolute, parent mtorso, child utorso, origin xyz=0 0 0.05 rpy=0 -0 0, axis 1 0 0, limit lower=-0.790809 upper=0.790809 effort=94.91 velocity=12
- added joint back_bky: type revolute, parent ltorso, child mtorso, origin xyz=0 0 0.09 rpy=0 -0 0, axis 0 1 0, limit lower=-1.2 upper=1.28 effort=206.843 velocity=12
- added joint back_bkz: type revolute, parent pelvis, child ltorso, origin xyz=-0.0125 0 0 rpy=0 -0 0, axis 0 0 1, limit lower=-0.610865 upper=0.610865 effort=124.016 velocity=12
- added joint l_leg_akx: type revolute, parent l_talus, child l_foot, origin xyz=0 0 0 rpy=0 -0 0, axis 1 0 0, limit lower=-0.436 upper=0.436 effort=90 velocity=12
- added joint l_leg_aky: type revolute, parent l_lleg, child l_talus, origin xyz=0 0 -0.422 rpy=0 -0 0, axis 0 1 0, limit lower=-0.9 upper=0.698 effort=220 velocity=12
- added joint l_leg_hpx: type revolute, parent l_uglut, child l_lglut, origin xyz=0 0 0 rpy=0 -0 0, axis 1 0 0, limit lower=-0.47 upper=0.495 effort=180 velocity=12
- added joint l_leg_hpy: type revolute, parent l_lglut, child l_uleg, origin xyz=0.05 0 -0.05 rpy=0 -0 0, axis 0 1 0, limit lower=-1.75 upper=0.524 effort=260 velocity=12
- added joint l_leg_hpz: type revolute, parent pelvis, child l_uglut, origin xyz=0 0.089 0 rpy=0 -0 0, axis 0 0 1, limit lower=-0.32 upper=1.14 effort=110 velocity=12
- added joint r_leg_akx: type revolute, parent r_talus, child r_foot, origin xyz=0 0 0 rpy=0 -0 0, axis 1 0 0, limit lower=-0.436 upper=0.436 effort=90 velocity=12
- added joint r_leg_aky: type revolute, parent r_lleg, child r_talus, origin xyz=0 0 -0.422 rpy=0 -0 0, axis 0 1 0, limit lower=-0.9 upper=0.698 effort=220 velocity=12
- added joint r_leg_hpx: type revolute, parent r_uglut, child r_lglut, origin xyz=0 0 0 rpy=0 -0 0, axis 1 0 0, limit lower=-0.495 upper=0.47 effort=180 velocity=12
- added joint r_leg_hpy: type revolute, parent r_lglut, child r_uleg, origin xyz=0.05 0 -0.05 rpy=0 -0 0, axis 0 1 0, limit lower=-1.745 upper=0.524 effort=260 velocity=12
- added joint r_leg_hpz: type revolute, parent pelvis, child r_uglut, origin xyz=0 -0.089 0 rpy=0 -0 0, axis 0 0 1, limit lower=-1.14 upper=0.32 effort=110 velocity=12

File: software/models/mit_gazebo_models/mit_robot_drake/model_minimal_contact.urdf (robot description, URDF)
Before this commit: robot atlas, 29 links, 28 joints
Joints:
- removed joint back_lbz
- removed joint back_mby
- removed joint back_ubx
- removed joint l_leg_lax
- removed joint l_leg_lhy
- removed joint l_leg_mhx
- removed joint l_leg_uay
- removed joint l_leg_uhz
- removed joint r_leg_lax
- removed joint r_leg_lhy
- removed joint r_leg_mhx
- removed joint r_leg_uay
- removed joint r_leg_uhz
- added joint back_bkx: type revolute, parent mtorso, child utorso, origin xyz=0 0 0.05 rpy=0 -0 0, axis 1 0 0, limit lower=-0.790809 upper=0.790809 effort=94.91 velocity=12
- added joint back_bky: type revolute, parent ltorso, child mtorso, origin xyz=0 0 0.09 rpy=0 -0 0, axis 0 1 0, limit lower=-1.2 upper=1.28 effort=206.843 velocity=12
- added joint back_bkz: type revolute, parent pelvis, child ltorso, origin xyz=-0.0125 0 0 rpy=0 -0 0, axis 0 0 1, limit lower=-0.610865 upper=0.610865 effort=124.016 velocity=12
- added joint l_leg_akx: type revolute, parent l_talus, child l_foot, origin xyz=0 0 0 rpy=0 -0 0, axis 1 0 0, limit lower=-0.436 upper=0.436 effort=90 velocity=12
- added joint l_leg_aky: type revolute, parent l_lleg, child l_talus, origin xyz=0 0 -0.422 rpy=0 -0 0, axis 0 1 0, limit lower=-0.9 upper=0.698 effort=220 velocity=12
- added joint l_leg_hpx: type revolute, parent l_uglut, child l_lglut, origin xyz=0 0 0 rpy=0 -0 0, axis 1 0 0, limit lower=-0.47 upper=0.495 effort=180 velocity=12
- added joint l_leg_hpy: type revolute, parent l_lglut, child l_uleg, origin xyz=0.05 0 -0.05 rpy=0 -0 0, axis 0 1 0, limit lower=-1.75 upper=0.524 effort=260 velocity=12
- added joint l_leg_hpz: type revolute, parent pelvis, child l_uglut, origin xyz=0 0.089 0 rpy=0 -0 0, axis 0 0 1, limit lower=-0.32 upper=1.14 effort=110 velocity=12
- added joint r_leg_akx: type revolute, parent r_talus, child r_foot, origin xyz=0 0 0 rpy=0 -0 0, axis 1 0 0, limit lower=-0.436 upper=0.436 effort=90 velocity=12
- added joint r_leg_aky: type revolute, parent r_lleg, child r_talus, origin xyz=0 0 -0.422 rpy=0 -0 0, axis 0 1 0, limit lower=-0.9 upper=0.698 effort=220 velocity=12
- added joint r_leg_hpx: type revolute, parent r_uglut, child r_lglut, origin xyz=0 0 0 rpy=0 -0 0, axis 1 0 0, limit lower=-0.495 upper=0.47 effort=180 velocity=12
- added joint r_leg_hpy: type revolute, parent r_lglut, child r_uleg, origin xyz=0.05 0 -0.05 rpy=0 -0 0, axis 0 1 0, limit lower=-1.745 upper=0.524 effort=260 velocity=12
- added joint r_leg_hpz: type revolute, parent pelvis, child r_uglut, origin xyz=0 -0.089 0 rpy=0 -0 0, axis 0 0 1, limit lower=-1.14 upper=0.32 effort=110 velocity=12

File: software/models/mit_gazebo_models/mit_robot_drake/model_minimal_contact_fixedjoint_hands.urdf (robot description, URDF)
Before this commit: robot atlas, 95 links, 94 joints
Joints:
- removed joint back_lbz
- removed joint back_mby
- removed joint back_ubx
- removed joint l_leg_lax
- removed joint l_leg_lhy
- removed joint l_leg_mhx
- removed joint l_leg_uay
- removed joint l_leg_uhz
- removed joint r_leg_lax
- removed joint r_leg_lhy
- removed joint r_leg_mhx
- removed joint r_leg_uay
- removed joint r_leg_uhz
- added joint back_bkx: type revolute, parent mtorso, child utorso, origin xyz=0 0 0.05 rpy=0 -0 0, axis 1 0 0, limit lower=-0.790809 upper=0.790809 effort=94.91 velocity=12
- added joint back_bky: type revolute, parent ltorso, child mtorso, origin xyz=0 0 0.09 rpy=0 -0 0, axis 0 1 0, limit lower=-1.2 upper=1.28 effort=206.843 velocity=12
- added joint back_bkz: type revolute, parent pelvis, child ltorso, origin xyz=-0.0125 0 0 rpy=0 -0 0, axis 0 0 1, limit lower=-0.610865 upper=0.610865 effort=124.016 velocity=12
- added joint l_leg_akx: type revolute, parent l_talus, child l_foot, origin xyz=0 0 0 rpy=0 -0 0, axis 1 0 0, limit lower=-0.436 upper=0.436 effort=90 velocity=12
- added joint l_leg_aky: type revolute, parent l_lleg, child l_talus, origin xyz=0 0 -0.422 rpy=0 -0 0, axis 0 1 0, limit lower=-0.9 upper=0.698 effort=220 velocity=12
- added joint l_leg_hpx: type revolute, parent l_uglut, child l_lglut, origin xyz=0 0 0 rpy=0 -0 0, axis 1 0 0, limit lower=-0.47 upper=0.495 effort=180 velocity=12
- added joint l_leg_hpy: type revolute, parent l_lglut, child l_uleg, origin xyz=0.05 0 -0.05 rpy=0 -0 0, axis 0 1 0, limit lower=-1.75 upper=0.524 effort=260 velocity=12
- added joint l_leg_hpz: type revolute, parent pelvis, child l_uglut, origin xyz=0 0.089 0 rpy=0 -0 0, axis 0 0 1, limit lower=-0.32 upper=1.14 effort=110 velocity=12
- added joint r_leg_akx: type revolute, parent r_talus, child r_foot, origin xyz=0 0 0 rpy=0 -0 0, axis 1 0 0, limit lower=-0.436 upper=0.436 effort=90 velocity=12
- added joint r_leg_aky: type revolute, parent r_lleg, child r_talus, origin xyz=0 0 -0.422 rpy=0 -0 0, axis 0 1 0, limit lower=-0.9 upper=0.698 effort=220 velocity=12
- added joint r_leg_hpx: type revolute, parent r_uglut, child r_lglut, origin xyz=0 0 0 rpy=0 -0 0, axis 1 0 0, limit lower=-0.495 upper=0.47 effort=180 velocity=12
- added joint r_leg_hpy: type revolute, parent r_lglut, child r_uleg, origin xyz=0.05 0 -0.05 rpy=0 -0 0, axis 0 1 0, limit lower=-1.745 upper=0.524 effort=260 velocity=12
- added joint r_leg_hpz: type revolute, parent pelvis, child r_uglut, origin xyz=0 -0.089 0 rpy=0 -0 0, axis 0 0 1, limit lower=-1.14 upper=0.32 effort=110 velocity=12

File: software/models/mit_gazebo_models/mit_robot_drake/model_minimal_contact_point_hands.urdf (robot description, URDF)
Before this commit: robot atlas, 31 links, 30 joints
Joints:
- removed joint back_lbz
- removed joint back_mby
- removed joint back_ubx
- removed joint l_leg_lax
- removed joint l_leg_lhy
- removed joint l_leg_mhx
- removed joint l_leg_uay
- removed joint l_leg_uhz
- removed joint r_leg_lax
- removed joint r_leg_lhy
- removed joint r_leg_mhx
- removed joint r_leg_uay
- removed joint r_leg_uhz
- added joint back_bkx: type revolute, parent mtorso, child utorso, origin xyz=0 0 0.05 rpy=0 -0 0, axis 1 0 0, limit lower=-0.790809 upper=0.790809 effort=94.91 velocity=12
- added joint back_bky: type revolute, parent ltorso, child mtorso, origin xyz=0 0 0.09 rpy=0 -0 0, axis 0 1 0, limit lower=-1.2 upper=1.28 effort=206.843 velocity=12
- added joint back_bkz: type revolute, parent pelvis, child ltorso, origin xyz=-0.0125 0 0 rpy=0 -0 0, axis 0 0 1, limit lower=-0.610865 upper=0.610865 effort=124.016 velocity=12
- added joint l_leg_akx: type revolute, parent l_talus, child l_foot, origin xyz=0 0 0 rpy=0 -0 0, axis 1 0 0, limit lower=-0.436 upper=0.436 effort=90 velocity=12
- added joint l_leg_aky: type revolute, parent l_lleg, child l_talus, origin xyz=0 0 -0.422 rpy=0 -0 0, axis 0 1 0, limit lower=-0.9 upper=0.698 effort=220 velocity=12
- added joint l_leg_hpx: type revolute, parent l_uglut, child l_lglut, origin xyz=0 0 0 rpy=0 -0 0, axis 1 0 0, limit lower=-0.47 upper=0.495 effort=180 velocity=12
- added joint l_leg_hpy: type revolute, parent l_lglut, child l_uleg, origin xyz=0.05 0 -0.05 rpy=0 -0 0, axis 0 1 0, limit lower=-1.75 upper=0.524 effort=260 velocity=12
- added joint l_leg_hpz: type revolute, parent pelvis, child l_uglut, origin xyz=0 0.089 0 rpy=0 -0 0, axis 0 0 1, limit lower=-0.32 upper=1.14 effort=110 velocity=12
- added joint r_leg_akx: type revolute, parent r_talus, child r_foot, origin xyz=0 0 0 rpy=0 -0 0, axis 1 0 0, limit lower=-0.436 upper=0.436 effort=90 velocity=12
- added joint r_leg_aky: type revolute, parent r_lleg, child r_talus, origin xyz=0 0 -0.422 rpy=0 -0 0, axis 0 1 0, limit lower=-0.9 upper=0.698 effort=220 velocity=12
- added joint r_leg_hpx: type revolute, parent r_uglut, child r_lglut, origin xyz=0 0 0 rpy=0 -0 0, axis 1 0 0, limit lower=-0.495 upper=0.47 effort=180 velocity=12
- added joint r_leg_hpy: type revolute, parent r_lglut, child r_uleg, origin xyz=0.05 0 -0.05 rpy=0 -0 0, axis 0 1 0, limit lower=-1.745 upper=0.524 effort=260 velocity=12
- added joint r_leg_hpz: type revolute, parent pelvis, child r_uglut, origin xyz=0 -0.089 0 rpy=0 -0 0, axis 0 0 1, limit lower=-1.14 upper=0.32 effort=110 velocity=12

File: software/models/mit_gazebo_models/mit_robot_drake/model_simple_visuals.urdf (robot description, URDF)
Before this commit: robot atlas, 33 links, 32 joints
Joints:
- removed joint back_lbz
- removed joint back_mby
- removed joint back_ubx
- removed joint l_leg_lax
- removed joint l_leg_lhy
- removed joint l_leg_mhx
- removed joint l_leg_uay
- removed joint l_leg_uhz
- removed joint r_leg_lax
- removed joint r_leg_lhy
- removed joint r_leg_mhx
- removed joint r_leg_uay
- removed joint r_leg_uhz
- added joint back_bkx: type revolute, parent mtorso, child utorso, origin xyz=0 0 0.05 rpy=0 -0 0, axis 1 0 0, limit lower=-0.790809 upper=0.790809 effort=94.91 velocity=12
- added joint back_bky: type revolute, parent ltorso, child mtorso, origin xyz=0 0 0.09 rpy=0 -0 0, axis 0 1 0, limit lower=-1.2 upper=1.28 effort=206.843 velocity=12
- added joint back_bkz: type revolute, parent pelvis, child ltorso, origin xyz=-0.0125 0 0 rpy=0 -0 0, axis 0 0 1, limit lower=-0.610865 upper=0.610865 effort=124.016 velocity=12
- added joint l_leg_akx: type revolute, parent l_talus, child l_foot, origin xyz=0 0 0 rpy=0 -0 0, axis 1 0 0, limit lower=-0.436 upper=0.436 effort=90 velocity=12
- added joint l_leg_aky: type revolute, parent l_lleg, child l_talus, origin xyz=0 0 -0.422 rpy=0 -0 0, axis 0 1 0, limit lower=-0.9 upper=0.698 effort=220 velocity=12
- added joint l_leg_hpx: type revolute, parent l_uglut, child l_lglut, origin xyz=0 0 0 rpy=0 -0 0, axis 1 0 0, limit lower=-0.47 upper=0.495 effort=180 velocity=12
- added joint l_leg_hpy: type revolute, parent l_lglut, child l_uleg, origin xyz=0.05 0 -0.05 rpy=0 -0 0, axis 0 1 0, limit lower=-1.75 upper=0.524 effort=260 velocity=12
- added joint l_leg_hpz: type revolute, parent pelvis, child l_uglut, origin xyz=0 0.089 0 rpy=0 -0 0, axis 0 0 1, limit lower=-0.32 upper=1.14 effort=110 velocity=12
- added joint r_leg_akx: type revolute, parent r_talus, child r_foot, origin xyz=0 0 0 rpy=0 -0 0, axis 1 0 0, limit lower=-0.436 upper=0.436 effort=90 velocity=12
- added joint r_leg_aky: type revolute, parent r_lleg, child r_talus, origin xyz=0 0 -0.422 rpy=0 -0 0, axis 0 1 0, limit lower=-0.9 upper=0.698 effort=220 velocity=12
- added joint r_leg_hpx: type revolute, parent r_uglut, child r_lglut, origin xyz=0 0 0 rpy=0 -0 0, axis 1 0 0, limit lower=-0.495 upper=0.47 effort=180 velocity=12
- added joint r_leg_hpy: type revolute, parent r_lglut, child r_uleg, origin xyz=0.05 0 -0.05 rpy=0 -0 0, axis 0 1 0, limit lower=-1.745 upper=0.524 effort=260 velocity=12
- added joint r_leg_hpz: type revolute, parent pelvis, child r_uglut, origin xyz=0 -0.089 0 rpy=0 -0 0, axis 0 0 1, limit lower=-1.14 upper=0.32 effort=110 velocity=12

File: software/models/mit_gazebo_models/mit_robot_drake/xacro/atlas_skeleton_minimal_contact.urdf (robot description, URDF)
Before this commit: robot drc_skeleton, 28 links, 28 joints
Joints:
- removed joint back_lbz
- removed joint back_mby
- removed joint back_ubx
- removed joint l_leg_lax
- removed joint l_leg_lhy
- removed joint l_leg_mhx
- removed joint l_leg_uay
- removed joint l_leg_uhz
- removed joint r_leg_lax
- removed joint r_leg_lhy
- removed joint r_leg_mhx
- removed joint r_leg_uay
- removed joint r_leg_uhz
- added joint back_bkx: type revolute, parent mtorso, child utorso, origin xyz=0 0 0.05 rpy=0 -0 0, axis 1 0 0, limit lower=-0.790809 upper=0.790809 effort=94.91 velocity=12
- added joint back_bky: type revolute, parent ltorso, child mtorso, origin xyz=0 0 0.09 rpy=0 -0 0, axis 0 1 0, limit lower=-1.2 upper=1.28 effort=206.843 velocity=12
- added joint back_bkz: type revolute, parent pelvis, child ltorso, origin xyz=-0.0125 0 0 rpy=0 -0 0, axis 0 0 1, limit lower=-0.610865 upper=0.610865 effort=124.016 velocity=12
- added joint l_leg_akx: type revolute, parent l_talus, child l_foot, origin xyz=0 0 0 rpy=0 -0 0, axis 1 0 0, limit lower=-0.436 upper=0.436 effort=90 velocity=12
- added joint l_leg_aky: type revolute, parent l_lleg, child l_talus, origin xyz=0 0 -0.422 rpy=0 -0 0, axis 0 1 0, limit lower=-0.9 upper=0.698 effort=220 velocity=12
- added joint l_leg_hpx: type revolute, parent l_uglut, child l_lglut, origin xyz=0 0 0 rpy=0 -0 0, axis 1 0 0, limit lower=-0.47 upper=0.495 effort=180 velocity=12
- added joint l_leg_hpy: type revolute, parent l_lglut, child l_uleg, origin xyz=0.05 0 -0.05 rpy=0 -0 0, axis 0 1 0, limit lower=-1.75 upper=0.524 effort=260 velocity=12
- added joint l_leg_hpz: type revolute, parent pelvis, child l_uglut, origin xyz=0 0.089 0 rpy=0 -0 0, axis 0 0 1, limit lower=-0.32 upper=1.14 effort=110 velocity=12
- added joint r_leg_akx: type revolute, parent r_talus, child r_foot, origin xyz=0 0 0 rpy=0 -0 0, axis 1 0 0, limit lower=-0.436 upper=0.436 effort=90 velocity=12
- added joint r_leg_aky: type revolute, parent r_lleg, child r_talus, origin xyz=0 0 -0.422 rpy=0 -0 0, axis 0 1 0, limit lower=-0.9 upper=0.698 effort=220 velocity=12
- added joint r_leg_hpx: type revolute, parent r_uglut, child r_lglut, origin xyz=0 0 0 rpy=0 -0 0, axis 1 0 0, limit lower=-0.495 upper=0.47 effort=180 velocity=12
- added joint r_leg_hpy: type revolute, parent r_lglut, child r_uleg, origin xyz=0.05 0 -0.05 rpy=0 -0 0, axis 0 1 0, limit lower=-1.745 upper=0.524 effort=260 velocity=12
- added joint r_leg_hpz: type revolute, parent pelvis, child r_uglut, origin xyz=0 -0.089 0 rpy=0 -0 0, axis 0 0 1, limit lower=-1.14 upper=0.32 effort=110 velocity=12

File: software/models/mit_gazebo_models/mit_robot_drake/xacro/atlas_skeleton_simple_visuals.urdf (robot description, URDF)
Before this commit: robot drc_skeleton, 28 links, 28 joints
Joints:
- removed joint back_lbz
- removed joint back_mby
- removed joint back_ubx
- removed joint l_leg_lax
- removed joint l_leg_lhy
- removed joint l_leg_mhx
- removed joint l_leg_uay
- removed joint l_leg_uhz
- removed joint r_leg_lax
- removed joint r_leg_lhy
- removed joint r_leg_mhx
- removed joint r_leg_uay
- removed joint r_leg_uhz
- added joint back_bkx: type revolute, parent mtorso, child utorso, origin xyz=0 0 0.05 rpy=0 -0 0, axis 1 0 0, limit lower=-0.790809 upper=0.790809 effort=94.91 velocity=12
- added joint back_bky: type revolute, parent ltorso, child mtorso, origin xyz=0 0 0.09 rpy=0 -0 0, axis 0 1 0, limit lower=-1.2 upper=1.28 effort=206.843 velocity=12
- added joint back_bkz: type revolute, parent pelvis, child ltorso, origin xyz=-0.0125 0 0 rpy=0 -0 0, axis 0 0 1, limit lower=-0.610865 upper=0.610865 effort=124.016 velocity=12
- added joint l_leg_akx: type revolute, parent l_talus, child l_foot, origin xyz=0 0 0 rpy=0 -0 0, axis 1 0 0, limit lower=-0.436 upper=0.436 effort=90 velocity=12
- added joint l_leg_aky: type revolute, parent l_lleg, child l_talus, origin xyz=0 0 -0.422 rpy=0 -0 0, axis 0 1 0, limit lower=-0.9 upper=0.698 effort=220 velocity=12
- added joint l_leg_hpx: type revolute, parent l_uglut, child l_lglut, origin xyz=0 0 0 rpy=0 -0 0, axis 1 0 0, limit lower=-0.47 upper=0.495 effort=180 velocity=12
- added joint l_leg_hpy: type revolute, parent l_lglut, child l_uleg, origin xyz=0.05 0 -0.05 rpy=0 -0 0, axis 0 1 0, limit lower=-1.75 upper=0.524 effort=260 velocity=12
- added joint l_leg_hpz: type revolute, parent pelvis, child l_uglut, origin xyz=0 0.089 0 rpy=0 -0 0, axis 0 0 1, limit lower=-0.32 upper=1.14 effort=110 velocity=12
- added joint r_leg_akx: type revolute, parent r_talus, child r_foot, origin xyz=0 0 0 rpy=0 -0 0, axis 1 0 0, limit lower=-0.436 upper=0.436 effort=90 velocity=12
- added joint r_leg_aky: type revolute, parent r_lleg, child r_talus, origin xyz=0 0 -0.422 rpy=0 -0 0, axis 0 1 0, limit lower=-0.9 upper=0.698 effort=220 velocity=12
- added joint r_leg_hpx: type revolute, parent r_uglut, child r_lglut, origin xyz=0 0 0 rpy=0 -0 0, axis 1 0 0, limit lower=-0.495 upper=0.47 effort=180 velocity=12
- added joint r_leg_hpy: type revolute, parent r_lglut, child r_uleg, origin xyz=0.05 0 -0.05 rpy=0 -0 0, axis 0 1 0, limit lower=-1.745 upper=0.524 effort=260 velocity=12
- added joint r_leg_hpz: type revolute, parent pelvis, child r_uglut, origin xyz=0 -0.089 0 rpy=0 -0 0, axis 0 0 1, limit lower=-1.14 upper=0.32 effort=110 velocity=12

File: software/models/mit_gazebo_models/mit_robot_drake/xacro/atlas_skeleton_simple_visuals_minimal_contact.urdf (robot description, URDF)
Before this commit: robot drc_skeleton, 28 links, 28 joints
Joints:
- removed joint back_lbz
- removed joint back_mby
- removed joint back_ubx
- removed joint l_leg_lax
- removed joint l_leg_lhy
- removed joint l_leg_mhx
- removed joint l_leg_uay
- removed joint l_leg_uhz
- removed joint r_leg_lax
- removed joint r_leg_lhy
- removed joint r_leg_mhx
- removed joint r_leg_uay
- removed joint r_leg_uhz
- added joint back_bkx: type revolute, parent mtorso, child utorso, origin xyz=0 0 0.05 rpy=0 -0 0, axis 1 0 0, limit lower=-0.790809 upper=0.790809 effort=94.91 velocity=12
- added joint back_bky: type revolute, parent ltorso, child mtorso, origin xyz=0 0 0.09 rpy=0 -0 0, axis 0 1 0, limit lower=-1.2 upper=1.28 effort=206.843 velocity=12
- added joint back_bkz: type revolute, parent pelvis, child ltorso, origin xyz=-0.0125 0 0 rpy=0 -0 0, axis 0 0 1, limit lower=-0.610865 upper=0.610865 effort=124.016 velocity=12
- added joint l_leg_akx: type revolute, parent l_talus, child l_foot, origin xyz=0 0 0 rpy=0 -0 0, axis 1 0 0, limit lower=-0.436 upper=0.436 effort=90 velocity=12
- added joint l_leg_aky: type revolute, parent l_lleg, child l_talus, origin xyz=0 0 -0.422 rpy=0 -0 0, axis 0 1 0, limit lower=-0.9 upper=0.698 effort=220 velocity=12
- added joint l_leg_hpx: type revolute, parent l_uglut, child l_lglut, origin xyz=0 0 0 rpy=0 -0 0, axis 1 0 0, limit lower=-0.47 upper=0.495 effort=180 velocity=12
- added joint l_leg_hpy: type revolute, parent l_lglut, child l_uleg, origin xyz=0.05 0 -0.05 rpy=0 -0 0, axis 0 1 0, limit lower=-1.75 upper=0.524 effort=260 velocity=12
- added joint l_leg_hpz: type revolute, parent pelvis, child l_uglut, origin xyz=0 0.089 0 rpy=0 -0 0, axis 0 0 1, limit lower=-0.32 upper=1.14 effort=110 velocity=12
- added joint r_leg_akx: type revolute, parent r_talus, child r_foot, origin xyz=0 0 0 rpy=0 -0 0, axis 1 0 0, limit lower=-0.436 upper=0.436 effort=90 velocity=12
- added joint r_leg_aky: type revolute, parent r_lleg, child r_talus, origin xyz=0 0 -0.422 rpy=0 -0 0, axis 0 1 0, limit lower=-0.9 upper=0.698 effort=220 velocity=12
- added joint r_leg_hpx: type revolute, parent r_uglut, child r_lglut, origin xyz=0 0 0 rpy=0 -0 0, axis 1 0 0, limit lower=-0.495 upper=0.47 effort=180 velocity=12
- added joint r_leg_hpy: type revolute, parent r_lglut, child r_uleg, origin xyz=0.05 0 -0.05 rpy=0 -0 0, axis 0 1 0, limit lower=-1.745 upper=0.524 effort=260 velocity=12
- added joint r_leg_hpz: type revolute, parent pelvis, child r_uglut, origin xyz=0 -0.089 0 rpy=0 -0 0, axis 0 0 1, limit lower=-1.14 upper=0.32 effort=110 velocity=12

File: software/models/mit_gazebo_models/mit_robot_feet/l_foot.urdf (robot description, URDF)
Before this commit: robot left_foot, 3 links, 2 joints
Joints:
- removed joint l_leg_lax
- removed joint l_leg_uay
- added joint l_leg_akx: type revolute, parent l_talus, child l_foot, origin xyz=0 0 0 rpy=0 -0 0, axis 1 0 0, limit lower=-0.436 upper=0.436 effort=90 velocity=12
- added joint l_leg_aky: type revolute, parent base, child l_talus, origin xyz=0 0 0 rpy=0 -0 0, axis 0 1 0, limit lower=-0.9 upper=0.698 effort=220 velocity=12
