Commit message: changing to bdi joint naming convention
git-svn-id: https://svn.csail.mit.edu/drc/trunk@5735 c7283977-0100-402a-a91a-fa70b306dbfe

File: software/models/mit_gazebo_models/mit_robot_feet/r_foot.urdf (robot description, URDF)
Before this commit: robot right_foot, 3 links, 2 joints
Joints:
- removed joint r_leg_lax
- removed joint r_leg_uay
- added joint r_leg_akx: type revolute, parent r_talus, child r_foot, origin xyz=0 0 0 rpy=0 -0 0, axis 1 0 0, limit lower=-0.436 upper=0.436 effort=90 velocity=12
- added joint r_leg_aky: type revolute, parent base, child r_talus, origin xyz=0 0 0 rpy=0 -0 0, axis 0 1 0, limit lower=-0.9 upper=0.698 effort=220 velocity=12

File: software/models/mit_gazebo_models/mit_robot_nohands/model.urdf (robot description, URDF)
Before this commit: robot atlas, 41 links, 40 joints
Joints:
- removed joint back_lbz
- removed joint back_mby
- removed joint back_ubx
- removed joint l_leg_lax
- removed joint l_leg_lhy
- removed joint l_leg_mhx
- removed joint l_leg_uay
- removed joint l_leg_uhz
- removed joint r_leg_lax
- removed joint r_leg_lhy
- removed joint r_leg_mhx
- removed joint r_leg_uay
- removed joint r_leg_uhz
- added joint back_bkx: type revolute, parent mtorso, child utorso, origin xyz=0 0 0.05 rpy=0 -0 0, axis 1 0 0, limit lower=-0.790809 upper=0.790809 effort=94.91 velocity=12
- added joint back_bky: type revolute, parent ltorso, child mtorso, origin xyz=0 0 0.09 rpy=0 -0 0, axis 0 1 0, limit lower=-1.2 upper=1.28 effort=206.843 velocity=12
- added joint back_bkz: type revolute, parent pelvis, child ltorso, origin xyz=-0.0125 0 0 rpy=0 -0 0, axis 0 0 1, limit lower=-0.610865 upper=0.610865 effort=124.016 velocity=12
- added joint l_leg_akx: type revolute, parent l_talus, child l_foot, origin xyz=0 0 0 rpy=0 -0 0, axis 1 0 0, limit lower=-0.436 upper=0.436 effort=90 velocity=12
- added joint l_leg_aky: type revolute, parent l_lleg, child l_talus, origin xyz=0 0 -0.422 rpy=0 -0 0, axis 0 1 0, limit lower=-0.9 upper=0.698 effort=220 velocity=12
- added joint l_leg_hpx: type revolute, parent l_uglut, child l_lglut, origin xyz=0 0 0 rpy=0 -0 0, axis 1 0 0, limit lower=-0.47 upper=0.495 effort=180 velocity=12
- added joint l_leg_hpy: type revolute, parent l_lglut, child l_uleg, origin xyz=0.05 0 -0.05 rpy=0 -0 0, axis 0 1 0, limit lower=-1.75 upper=0.524 effort=260 velocity=12
- added joint l_leg_hpz: type revolute, parent pelvis, child l_uglut, origin xyz=0 0.089 0 rpy=0 -0 0, axis 0 0 1, limit lower=-0.32 upper=1.14 effort=110 velocity=12
- added joint r_leg_akx: type revolute, parent r_talus, child r_foot, origin xyz=0 0 0 rpy=0 -0 0, axis 1 0 0, limit lower=-0.436 upper=0.436 effort=90 velocity=12
- added joint r_leg_aky: type revolute, parent r_lleg, child r_talus, origin xyz=0 0 -0.422 rpy=0 -0 0, axis 0 1 0, limit lower=-0.9 upper=0.698 effort=220 velocity=12
- added joint r_leg_hpx: type revolute, parent r_uglut, child r_lglut, origin xyz=0 0 0 rpy=0 -0 0, axis 1 0 0, limit lower=-0.495 upper=0.47 effort=180 velocity=12
- added joint r_leg_hpy: type revolute, parent r_lglut, child r_uleg, origin xyz=0.05 0 -0.05 rpy=0 -0 0, axis 0 1 0, limit lower=-1.745 upper=0.524 effort=260 velocity=12
- added joint r_leg_hpz: type revolute, parent pelvis, child r_uglut, origin xyz=0 -0.089 0 rpy=0 -0 0, axis 0 0 1, limit lower=-1.14 upper=0.32 effort=110 velocity=12

Commit message: fixing model and sim generate script
git-svn-id: https://svn.csail.mit.edu/drc/trunk@5736 c7283977-0100-402a-a91a-fa70b306dbfe

File: software/models/mit_gazebo_models/mit_robot/model.urdf (robot description, URDF)
Before this commit: robot atlas, 107 links, 106 joints
Joints:
- removed joint l_arm_wrx
- removed joint l_arm_wry
- removed joint neck_ry
- removed joint r_arm_wrx
- removed joint r_arm_wry
- added joint l_arm_mwx: type revolute, parent l_farm, child l_hand, origin xyz=0 0.058 0 rpy=0 -0 0, axis 1 0 0, limit lower=-0.436 upper=1.571 effort=60 velocity=12
- added joint l_arm_uwy: type revolute, parent l_larm, child l_farm, origin xyz=0 0.188 -0.013 rpy=0 -0 0, axis 0 1 0, limit lower=-1.571 upper=1.571 effort=114 velocity=12
- added joint neck_ay: type revolute, parent utorso, child head, origin xyz=0.21672 0 0.53796 rpy=0 -0 0, axis 0 1 0, limit lower=-0.610865238 upper=1.13446401 effort=5 velocity=12
- added joint r_arm_mwx: type revolute, parent r_farm, child r_hand, origin xyz=0 -0.058 0 rpy=0 -0 0, axis 1 0 0, limit lower=-1.571 upper=0.436 effort=60 velocity=12
- added joint r_arm_uwy: type revolute, parent r_larm, child r_farm, origin xyz=0 -0.188 -0.013 rpy=0 -0 0, axis 0 1 0, limit lower=-1.571 upper=1.571 effort=114 velocity=12

Commit message: fixed usy joint in model and updated gen script
git-svn-id: https://svn.csail.mit.edu/drc/trunk@5745 c7283977-0100-402a-a91a-fa70b306dbfe

File: software/models/mit_gazebo_models/mit_robot/model.urdf (robot description, URDF)
Before this commit: robot atlas, 107 links, 106 joints
Joints:
- removed joint l_arm_shy
- removed joint r_arm_shy
- added joint l_arm_usy: type revolute, parent utorso, child l_clav, origin xyz=0.024 0.221 0.289 rpy=0 -0 0, axis 0 0.5 0.866025, limit lower=-1.9635 upper=1.9635 effort=212 velocity=12
- added joint r_arm_usy: type revolute, parent utorso, child r_clav, origin xyz=0.024 -0.221 0.289 rpy=0 -0 0, axis 0 0.5 -0.866025, limit lower=-1.9635 upper=1.9635 effort=212 velocity=12

Commit message: switching ack to laptop
git-svn-id: https://svn.csail.mit.edu/drc/trunk@5848 c7283977-0100-402a-a91a-fa70b306dbfe

File: software/models/mit_gazebo_models/mit_robot/model.urdf (robot description, URDF)
Before this commit: robot atlas, 107 links, 106 joints
Links:
- removed link head_imu_link
- added link head_root
- added link post_spindle
- added link post_spindle_cal_pitch
- added link post_spindle_cal_roll
- added link post_spindle_cal_x
- added link post_spindle_cal_y
- added link post_spindle_cal_z
- added link pre_spindle
- added link pre_spindle_cal_pitch
- added link pre_spindle_cal_roll
- added link pre_spindle_cal_x
- added link pre_spindle_cal_y
- added link pre_spindle_cal_yaw
- added link pre_spindle_cal_z
- link center_bottom_led_frame: mass 1e-5 -> 0.1
- link center_top_led_frame: mass 1e-5 -> 0.1
- link head: mass 1.41984 -> 1.4199; geometry collision box size=0.1311 0.12 0.0591; visual mesh filename=package://multisense_sl/meshes/base_link.STL
- link head_hokuyo_frame: mass 1e-5 -> 0.01
- link hokuyo_link: mass 0.057654 -> 0.057664; geometry collision cylinder length=0.047 radius=0.024425; visual mesh filename=package://multisense_sl/meshes/hokuyo_link.STL
- link left_camera_frame: mass 1e-5 -> 0.1
- link left_led_frame: mass 1e-5 -> 0.1
- link right_camera_frame: mass 1e-5 -> 0.1
- link right_led_frame: mass 1e-5 -> 0.1
Joints:
- removed joint head_imu_joint
- added joint head_root_joint: type fixed, parent head_root, child head
- added joint post_spindle_cal_pitch_joint: type continuous, parent post_spindle_cal_roll, child post_spindle_cal_pitch, axis 0 1 0
- added joint post_spindle_cal_roll_joint: type continuous, parent post_spindle_cal_z, child post_spindle_cal_roll, axis 1 0 0
- added joint post_spindle_cal_x_joint: type prismatic, parent post_spindle, child post_spindle_cal_x, axis 1 0 0, limit lower=-0.5 upper=0.5 effort=0.0 velocity=0.0
- added joint post_spindle_cal_y_joint: type prismatic, parent post_spindle_cal_x, child post_spindle_cal_y, axis 0 1 0, limit lower=-0.5 upper=0.5 effort=0.0 velocity=0.0
- added joint post_spindle_cal_yaw_joint: type continuous, parent post_spindle_cal_pitch, child hokuyo_link, axis 0 0 1
- added joint post_spindle_cal_z_joint: type prismatic, parent post_spindle_cal_y, child post_spindle_cal_z, axis 0 0 1, limit lower=-0.5 upper=0.5 effort=0.0 velocity=0.0
- added joint pre_spindle_cal_pitch_joint: type continuous, parent pre_spindle_cal_roll, child pre_spindle_cal_pitch, axis 0 1 0
- added joint pre_spindle_cal_roll_joint: type continuous, parent pre_spindle_cal_z, child pre_spindle_cal_roll, axis 1 0 0
- added joint pre_spindle_cal_x_joint: type prismatic, parent pre_spindle, child pre_spindle_cal_x, axis 1 0 0, limit lower=-0.5 upper=0.5 effort=0.0 velocity=0.0
- added joint pre_spindle_cal_y_joint: type prismatic, parent pre_spindle_cal_x, child pre_spindle_cal_y, axis 0 1 0, limit lower=-0.5 upper=0.5 effort=0.0 velocity=0.0
- added joint pre_spindle_cal_yaw_joint: type continuous, parent pre_spindle_cal_pitch, child pre_spindle_cal_yaw, axis 0 0 1
- added joint pre_spindle_cal_z_joint: type prismatic, parent pre_spindle_cal_y, child pre_spindle_cal_z, axis 0 0 1, limit lower=-0.5 upper=0.5 effort=0.0 velocity=0.0
- added joint pre_spindle_joint: type fixed, parent head, child pre_spindle, origin xyz=-0.0446 0 0.0880 rpy=0 0 0, axis 0 1 0
- joint hokuyo_joint: child hokuyo_link -> post_spindle; origin xyz=-0.0446 0 0.0880 rpy=0 0 0 -> xyz=0 0 0 rpy=0 0 0; parent head -> pre_spindle_cal_yaw

File: software/models/mit_gazebo_models/mit_robot/model_sim_gazebo.urdf (robot description, URDF)
Before this commit: robot atlas, 107 links, 106 joints
Joints:
- removed joint back_bkx
- removed joint back_bky
- removed joint back_bkz
- removed joint l_leg_akx
- removed joint l_leg_aky
- removed joint l_leg_hpx
- removed joint l_leg_hpy
- removed joint l_leg_hpz
- removed joint r_leg_akx
- removed joint r_leg_aky
- removed joint r_leg_hpx
- removed joint r_leg_hpy
- removed joint r_leg_hpz
- added joint back_lbz: type revolute, parent pelvis, child ltorso, origin xyz=-0.0125 0 0 rpy=0 -0 0, axis 0 0 1, limit lower=-0.610865 upper=0.610865 effort=124.016 velocity=12
- added joint back_mby: type revolute, parent ltorso, child mtorso, origin xyz=0 0 0.09 rpy=0 -0 0, axis 0 1 0, limit lower=-1.2 upper=1.28 effort=206.843 velocity=12
- added joint back_ubx: type revolute, parent mtorso, child utorso, origin xyz=0 0 0.05 rpy=0 -0 0, axis 1 0 0, limit lower=-0.790809 upper=0.790809 effort=94.91 velocity=12
- added joint l_leg_lax: type revolute, parent l_talus, child l_foot, origin xyz=0 0 0 rpy=0 -0 0, axis 1 0 0, limit lower=-0.436 upper=0.436 effort=90 velocity=12
- added joint l_leg_lhy: type revolute, parent l_lglut, child l_uleg, origin xyz=0.05 0 -0.05 rpy=0 -0 0, axis 0 1 0, limit lower=-1.75 upper=0.524 effort=260 velocity=12
- added joint l_leg_mhx: type revolute, parent l_uglut, child l_lglut, origin xyz=0 0 0 rpy=0 -0 0, axis 1 0 0, limit lower=-0.47 upper=0.495 effort=180 velocity=12
- added joint l_leg_uay: type revolute, parent l_lleg, child l_talus, origin xyz=0 0 -0.422 rpy=0 -0 0, axis 0 1 0, limit lower=-0.9 upper=0.698 effort=220 velocity=12
- added joint l_leg_uhz: type revolute, parent pelvis, child l_uglut, origin xyz=0 0.089 0 rpy=0 -0 0, axis 0 0 1, limit lower=-0.32 upper=1.14 effort=110 velocity=12
- added joint r_leg_lax: type revolute, parent r_talus, child r_foot, origin xyz=0 0 0 rpy=0 -0 0, axis 1 0 0, limit lower=-0.436 upper=0.436 effort=90 velocity=12
- added joint r_leg_lhy: type revolute, parent r_lglut, child r_uleg, origin xyz=0.05 0 -0.05 rpy=0 -0 0, axis 0 1 0, limit lower=-1.745 upper=0.524 effort=260 velocity=12
- added joint r_leg_mhx: type revolute, parent r_uglut, child r_lglut, origin xyz=0 0 0 rpy=0 -0 0, axis 1 0 0, limit lower=-0.495 upper=0.47 effort=180 velocity=12
- added joint r_leg_uay: type revolute, parent r_lleg, child r_talus, origin xyz=0 0 -0.422 rpy=0 -0 0, axis 0 1 0, limit lower=-0.9 upper=0.698 effort=220 velocity=12
- added joint r_leg_uhz: type revolute, parent pelvis, child r_uglut, origin xyz=0 -0.089 0 rpy=0 -0 0, axis 0 0 1, limit lower=-1.14 upper=0.32 effort=110 velocity=12
