Commit message: close to completeing xacro systwem
git-svn-id: https://svn.csail.mit.edu/drc/trunk@5858 c7283977-0100-402a-a91a-fa70b306dbfe

File: software/models/mit_gazebo_models/mit_robot/model_LS_RS.urdf (robot description, URDF)
Before this commit: robot atlas, 120 links, 119 joints
Links:
- removed link imu_link
Joints:
- removed joint imu_joint

File: software/models/mit_gazebo_models/mit_robot/model_sim.urdf (robot description, URDF)
Before this commit: robot atlas, 107 links, 106 joints
Links:
- link head: geometry collision box size=0.0468 0.12 0.1184; collision box size=0.1311 0.12 0.0591
- link hokuyo_link: geometry collision box size=0.08 0.06 0.04238; collision cylinder length=0.047 radius=0.024425

File: software/models/mit_gazebo_models/mit_robot/model_sim_gazebo.urdf (robot description, URDF)
Before this commit: robot atlas, 107 links, 106 joints
Links:
- link head: geometry collision box size=0.0468 0.12 0.1184; collision box size=0.1311 0.12 0.0591
- link hokuyo_link: geometry collision box size=0.08 0.06 0.04238; collision cylinder length=0.047 radius=0.024425

File: software/models/mit_gazebo_models/mit_robot/xacro/atlas_irobot_hands.urdf.xacro (robot description, xacro)
@@ -1,4 +1,7 @@
 <robot xmlns:xacro="http://playerstage.sourceforge.net/gazebo/xmlschema/#interface" name="atlas" >
   <include filename="$(find mit_drcsim_scripts)/models/mit_robot/xacro/atlas_skeleton.urdf" />
+  <include filename="$(find mit_drcsim_scripts)/models/mit_robot/xacro/atlas.transmission" />
+  <include filename="$(find mit_drcsim_scripts)/models/multisense_sl/multisense_sl.urdf" />
+  <!-- Hands -->
   <include filename="$(find handle_description)/src/irobot_hand_simple.urdf.xacro" />
   <xacro:irobot_hand side="right" parent="r_hand" reflect="1">
@@ -8,7 +11,3 @@
     <origin rpy="1.57079 0 3.14159" xyz="0 0.05 0"/>
   </xacro:irobot_hand>
-  <include filename="$(find mit_drcsim_scripts)/models/mit_robot/xacro/atlas.gazebo" />
-  <include filename="$(find mit_drcsim_scripts)/models/mit_robot/xacro/atlas.transmission" />
-  <include filename="$(find multisense_sl_description)/multisense_sl_description.urdf" />
-  <include filename="$(find mit_drcsim_scripts)/models/mit_robot/xacro/mit_atlas.gazebo" />
 </robot>

File: software/models/mit_gazebo_models/mit_robot/xacro/atlas_irobot_left_sandia_right.urdf.xacro (robot description, xacro)
@@ -1,4 +1,7 @@
 <robot xmlns:xacro="http://playerstage.sourceforge.net/gazebo/xmlschema/#interface" name="atlas" >
   <include filename="$(find mit_drcsim_scripts)/models/mit_robot/xacro/atlas_skeleton.urdf" />
+  <include filename="$(find mit_drcsim_scripts)/models/mit_robot/xacro/atlas.transmission" />
+  <include filename="$(find mit_drcsim_scripts)/models/multisense_sl/multisense_sl.urdf" />
+  <!-- Hands -->
   <include filename="$(find sandia_hand_description)/urdf/sandia_hand_simple_shapes.urdf.xacro" />
   <include filename="$(find handle_description)/src/irobot_hand_simple.urdf.xacro" />
@@ -15,11 +18,3 @@
     <origin rpy="1.57079 0 3.14159" xyz="0 0.05 0"/>
   </xacro:irobot_hand>
-  <include filename="$(find mit_drcsim_scripts)/models/mit_robot/xacro/atlas.gazebo" />
-  <include filename="$(find mit_drcsim_scripts)/models/mit_robot/xacro/atlas.transmission" />
-  <include filename="$(find multisense_sl_description)/multisense_sl_description.urdf" />
-  <include filename="$(find mit_drcsim_scripts)/models/mit_robot/xacro/mit_atlas.gazebo" />
-  <gazebo>
-    <!-- include plugin for sandia hands -->
-    <plugin name="sandia_hand_plugin" filename="libSandiaHandPlugin.so"/>
-  </gazebo>
 </robot>

File: software/models/mit_gazebo_models/mit_robot/xacro/atlas_sandia_hands.urdf.xacro (robot description, xacro)
@@ -1,4 +1,7 @@
 <robot xmlns:xacro="http://playerstage.sourceforge.net/gazebo/xmlschema/#interface" name="atlas" >
   <include filename="$(find mit_drcsim_scripts)/models/mit_robot/xacro/atlas_skeleton.urdf" />
+  <include filename="$(find mit_drcsim_scripts)/models/mit_robot/xacro/atlas.transmission" />
+  <include filename="$(find mit_drcsim_scripts)/models/multisense_sl/multisense_sl.urdf" />
+  <!-- Hands -->
   <include filename="$(find sandia_hand_description)/urdf/sandia_hand_simple_shapes.urdf.xacro" />
   <xacro:sandia_hand side="right" parent="r_hand" reflect="1" joint_type="revolute" thumb_angle="0">
@@ -8,11 +11,3 @@
     <origin xyz="0  0.1 0" rpy=" 1.57079 0  1.57079"/>
   </xacro:sandia_hand>
-  <include filename="$(find mit_drcsim_scripts)/models/mit_robot/xacro/atlas.gazebo" />
-  <include filename="$(find mit_drcsim_scripts)/models/mit_robot/xacro/atlas.transmission" />
-  <include filename="$(find mit_drcsim_scripts)/models/multisense_sl/multisense_sl.urdf" />
-  <include filename="$(find mit_drcsim_scripts)/models/mit_robot/xacro/mit_atlas.gazebo" />
-  <gazebo>
-    <!-- include plugin for sandia hands -->
-    <plugin name="sandia_hand_plugin" filename="libSandiaHandPlugin.so"/>
-  </gazebo>
 </robot>

File: software/models/mit_gazebo_models/mit_robot/xacro/atlas_sandia_hands_sim.urdf.xacro (robot description, xacro)
@@ -2,12 +2,12 @@
   <include filename="$(find mit_drcsim_scripts)/models/mit_robot/xacro/atlas_skeleton.urdf" />
   <include filename="$(find sandia_hand_description)/urdf/sandia_hand_simple_shapes.urdf.xacro" />
-  <xacro:sandia_hand side="right" parent="r_hand" reflect="1" joint_type="fixed" thumb_angle="1.57">
+  <xacro:sandia_hand side="right" parent="r_hand" reflect="1" joint_type="revolute" thumb_angle="0">
     <origin xyz="0 -0.1 0" rpy="-1.57079 0 -1.57079"/>
   </xacro:sandia_hand>
-  <xacro:sandia_hand side="left" parent="l_hand" reflect="-1" joint_type="fixed" thumb_angle="1.57">
+  <xacro:sandia_hand side="left" parent="l_hand" reflect="-1" joint_type="revolute" thumb_angle="0">
     <origin xyz="0  0.1 0" rpy=" 1.57079 0  1.57079"/>
   </xacro:sandia_hand>
-  <include filename="$(find atlas_description)/urdf/atlas.gazebo" />
-  <include filename="$(find atlas_description)/urdf/atlas.transmission" />
+  <include filename="$(find mit_drcsim_scripts)/models/mit_robot/xacro/atlas.gazebo" />
+  <include filename="$(find mit_drcsim_scripts)/models/mit_robot/xacro/atlas.transmission" />
   <include filename="$(find multisense_sl_description)/multisense_sl_description.urdf" />
   <include filename="$(find mit_drcsim_scripts)/models/mit_robot/xacro/mit_atlas.gazebo" />

File: software/models/mit_gazebo_models/mit_robot/xacro/atlas_sandia_left_irobot_right.urdf.xacro (robot description, xacro)
@@ -1,4 +1,7 @@
 <robot xmlns:xacro="http://playerstage.sourceforge.net/gazebo/xmlschema/#interface" name="atlas" >
   <include filename="$(find mit_drcsim_scripts)/models/mit_robot/xacro/atlas_skeleton.urdf" />
+  <include filename="$(find mit_drcsim_scripts)/models/mit_robot/xacro/atlas.transmission" />
+  <include filename="$(find mit_drcsim_scripts)/models/multisense_sl/multisense_sl.urdf" />
+<!-- Hands -->
   <include filename="$(find sandia_hand_description)/urdf/sandia_hand_simple_shapes.urdf.xacro" />
   <include filename="$(find handle_description)/src/irobot_hand_simple.urdf.xacro" />
@@ -15,11 +18,3 @@
 <!--    <origin rpy="1.57079 0 3.14159" xyz="0 0.05 0"/>-->
 <!--  </xacro:irobot_hand>-->
-  <include filename="$(find mit_drcsim_scripts)/models/mit_robot/xacro/atlas.gazebo" />
-  <include filename="$(find mit_drcsim_scripts)/models/mit_robot/xacro/atlas.transmission" />
-  <include filename="$(find multisense_sl_description)/multisense_sl_description.urdf" />
-  <include filename="$(find mit_drcsim_scripts)/models/mit_robot/xacro/mit_atlas.gazebo" />
-  <gazebo>
-    <!-- include plugin for sandia hands -->
-    <plugin name="sandia_hand_plugin" filename="libSandiaHandPlugin.so"/>
-  </gazebo>
 </robot>

Commit message: sandia hands orientation fix - reality doesnt match simulator by 90d
git-svn-id: https://svn.csail.mit.edu/drc/trunk@5880 c7283977-0100-402a-a91a-fa70b306dbfe

File: software/models/mit_gazebo_models/mit_robot/model_LS_RS.urdf (robot description, URDF)
Before this commit: robot atlas, 118 links, 117 joints
Joints:
- joint left_sandia_hand_joint: origin xyz=0  0.1 0 rpy= 1.57079 0  1.57079 -> xyz=0  0.1 0 rpy= 3.14158 0  1.57079
- joint right_sandia_hand_joint: origin xyz=0 -0.1 0 rpy=-1.57079 0 -1.57079 -> xyz=0 -0.1 0 rpy=-3.14158 0 -1.57079

File: software/models/mit_gazebo_models/mit_robot/xacro/atlas_sandia_hands.urdf.xacro (robot description, xacro)
@@ -4,10 +4,11 @@
   <include filename="$(find mit_drcsim_scripts)/models/multisense_sl/multisense_sl.urdf" />
   <!-- Hands -->
+  <!-- NB: the Roll of the Sandia Hands is not identical in Sim and Reality -->
   <include filename="$(find sandia_hand_description)/urdf/sandia_hand_simple_shapes.urdf.xacro" />
   <xacro:sandia_hand side="right" parent="r_hand" reflect="1" joint_type="revolute" thumb_angle="0">
-    <origin xyz="0 -0.1 0" rpy="-1.57079 0 -1.57079"/>
+    <origin xyz="0 -0.1 0" rpy="-3.14158 0 -1.57079"/>
   </xacro:sandia_hand>
   <xacro:sandia_hand side="left" parent="l_hand" reflect="-1" joint_type="revolute" thumb_angle="0">
-    <origin xyz="0  0.1 0" rpy=" 1.57079 0  1.57079"/>
+    <origin xyz="0  0.1 0" rpy=" 3.14158 0  1.57079"/>
   </xacro:sandia_hand>
 </robot>

File: software/models/mit_gazebo_models/mit_robot/xacro/atlas_sandia_hands_sim.urdf.xacro (robot description, xacro)
@@ -2,4 +2,6 @@
   <include filename="$(find mit_drcsim_scripts)/models/mit_robot/xacro/atlas_skeleton.urdf" />
   <include filename="$(find sandia_hand_description)/urdf/sandia_hand_simple_shapes.urdf.xacro" />
+  <!-- Hands -->
+  <!-- NB: the Roll of the Sandia Hands is not identical in Sim and Reality -->
   <xacro:sandia_hand side="right" parent="r_hand" reflect="1" joint_type="revolute" thumb_angle="0">
     <origin xyz="0 -0.1 0" rpy="-1.57079 0 -1.57079"/>

Commit message: fixed issue with rotation of sandia hands and mounting
git-svn-id: https://svn.csail.mit.edu/drc/trunk@5891 c7283977-0100-402a-a91a-fa70b306dbfe

File: software/models/mit_gazebo_models/mit_robot/model_LS_RS.urdf (robot description, URDF)
Before this commit: robot atlas, 118 links, 117 joints
Joints:
- joint left_sandia_hand_joint: origin xyz=0  0.1 0 rpy= 3.14158 0  1.57079 -> xyz=0  0.1 0 rpy=0 0  1.57079
- joint right_sandia_hand_joint: origin xyz=0 -0.1 0 rpy=-3.14158 0 -1.57079 -> xyz=0 -0.1 0 rpy=0.0 0 -1.57079

File: software/models/mit_gazebo_models/mit_robot/xacro/atlas_sandia_hands.urdf.xacro (robot description, xacro)
@@ -7,8 +7,8 @@
   <include filename="$(find sandia_hand_description)/urdf/sandia_hand_simple_shapes.urdf.xacro" />
   <xacro:sandia_hand side="right" parent="r_hand" reflect="1" joint_type="revolute" thumb_angle="0">
-    <origin xyz="0 -0.1 0" rpy="-3.14158 0 -1.57079"/>
+    <origin xyz="0 -0.1 0" rpy="0.0 0 -1.57079"/>
   </xacro:sandia_hand>
   <xacro:sandia_hand side="left" parent="l_hand" reflect="-1" joint_type="revolute" thumb_angle="0">
-    <origin xyz="0  0.1 0" rpy=" 3.14158 0  1.57079"/>
+    <origin xyz="0  0.1 0" rpy="0 0  1.57079"/>
   </xacro:sandia_hand>
 </robot>
