Commit message: correction
git-svn-id: https://svn.csail.mit.edu/drc/trunk@6535 c7283977-0100-402a-a91a-fa70b306dbfe

File: software/models/mit_gazebo_models/mit_robot/model_LN_RS.urdf (robot description, URDF)
Before this commit: robot atlas, 74 links, 73 joints
Links:
- removed link left_base_link
- removed link left_finger[0]/base_rotation_link
- removed link left_finger[0]/distal_link
- removed link left_finger[0]/proximal_link
- removed link left_finger[1]/base_rotation_link
- removed link left_finger[1]/distal_link
- removed link left_finger[1]/proximal_link
- removed link left_finger[2]/distal_link
- removed link left_finger[2]/proximal_link
- removed link right_base_link
- removed link right_finger[0]/base_rotation_link
- removed link right_finger[0]/distal_link
- removed link right_finger[0]/proximal_link
- removed link right_finger[1]/base_rotation_link
- removed link right_finger[1]/distal_link
- removed link right_finger[1]/proximal_link
- removed link right_finger[2]/distal_link
- removed link right_finger[2]/proximal_link
- added link right_f0_0, mass 0.106; collision cylinder length=0.023 radius=0.01; collision cylinder length=0.023 radius=0.015
- added link right_f0_1, mass 0.033; collision cylinder length=0.067 radius=0.01; visual cylinder length=0.067 radius=0.01
- added link right_f0_1_accel, mass 0.01
- added link right_f0_2, mass 0.033; collision cylinder length=0.057 radius=0.009; collision sphere radius=0.009
- added link right_f0_2_accel, mass 0.01
- added link right_f0_base, mass 0.250
- added link right_f0_fixed_accel, mass 0.01
- added link right_f1_0, mass 0.106; collision cylinder length=0.023 radius=0.01; collision cylinder length=0.023 radius=0.015
- added link right_f1_1, mass 0.033; collision cylinder length=0.067 radius=0.01; visual cylinder length=0.067 radius=0.01
- added link right_f1_1_accel, mass 0.01
- added link right_f1_2, mass 0.033; collision cylinder length=0.057 radius=0.009; collision sphere radius=0.009
- added link right_f1_2_accel, mass 0.01
- added link right_f1_base, mass 0.250
- added link right_f1_fixed_accel, mass 0.01
- added link right_f2_0, mass 0.106; collision cylinder length=0.023 radius=0.01; collision cylinder length=0.023 radius=0.015
- added link right_f2_1, mass 0.033; collision cylinder length=0.067 radius=0.01; visual cylinder length=0.067 radius=0.01
- added link right_f2_1_accel, mass 0.01
- added link right_f2_2, mass 0.033; collision cylinder length=0.057 radius=0.009; collision sphere radius=0.009
- added link right_f2_2_accel, mass 0.01
- added link right_f2_base, mass 0.250
- added link right_f2_fixed_accel, mass 0.01
- added link right_f3_0, mass 0.106; collision cylinder length=0.023 radius=0.01; collision cylinder length=0.023 radius=0.015
- added link right_f3_1, mass 0.033; collision cylinder length=0.067 radius=0.01; visual cylinder length=0.067 radius=0.01
- added link right_f3_1_accel, mass 0.01
- added link right_f3_2, mass 0.033; collision cylinder length=0.057 radius=0.009; collision sphere radius=0.009
- added link right_f3_2_accel, mass 0.01
- added link right_f3_base, mass 0.250
- added link right_f3_fixed_accel, mass 0.01
- added link right_palm, mass 1.303; collision box size=0.09 .03 .06; collision box size=0.09 .03 .06
- added link right_palm_left_camera_frame, mass 0.01; visual box size=0.003 0.010 0.007
- added link right_palm_left_camera_optical_frame
- added link right_palm_right_camera_frame, mass 0.01; visual box size=0.003 0.010 0.007
- added link right_palm_right_camera_optical_frame
Joints:
- removed joint left_finger[0]/joint_base
- removed joint left_finger[0]/joint_base_rotation
- removed joint left_finger[0]/joint_flex
- removed joint left_finger[1]/joint_base
- removed joint left_finger[1]/joint_base_rotation
- removed joint left_finger[1]/joint_flex
- removed joint left_finger[2]/joint_base
- removed joint left_finger[2]/joint_flex
- removed joint left_irobot_hand_joint
- removed joint right_finger[0]/joint_base
- removed joint right_finger[0]/joint_base_rotation
- removed joint right_finger[0]/joint_flex
- removed joint right_finger[1]/joint_base
- removed joint right_finger[1]/joint_base_rotation
- removed joint right_finger[1]/joint_flex
- removed joint right_finger[2]/joint_base
- removed joint right_finger[2]/joint_flex
- removed joint right_irobot_hand_joint
- added joint right_f0_1_accel: type fixed, parent right_f0_1, child right_f0_1_accel, origin xyz=0.03 0 0 rpy=-1.57079632679 0 0
- added joint right_f0_2_accel: type fixed, parent right_f0_2, child right_f0_2_accel, origin xyz=0.04 0 0 rpy=-1.57079632679 0 0
- added joint right_f0_base: type fixed, parent right_palm, child right_f0_base, origin xyz=0.14 0.0 0 rpy=0 0 0.3
- added joint right_f0_fixed_accel: type fixed, parent right_f0_base, child right_f0_fixed_accel, origin xyz=-0.05 0 0 rpy=0 0 0
- added joint right_f0_j0: type revolute, parent right_f0_base, child right_f0_0, origin xyz=0 0 0 rpy=0 0 0, axis 0 0 1, limit lower=-1.57079632679 upper=1.57079632679 effort=11 velocity=-1
- added joint right_f0_j1: type revolute, parent right_f0_0, child right_f0_1, origin xyz=0.028 0 0 rpy=1.57079632679 0 0, axis 0 0 1, limit lower=-1.57079632679 upper=1.57079632679 effort=28 velocity=-1
- added joint right_f0_j2: type revolute, parent right_f0_1, child right_f0_2, origin xyz=0.05 0 0 rpy=0 0 0, axis 0 0 1, limit lower=-1.57079632679 upper=1.57079632679 effort=28 velocity=-1
- added joint right_f1_1_accel: type fixed, parent right_f1_1, child right_f1_1_accel, origin xyz=0.03 0 0 rpy=-1.57079632679 0 0
- added joint right_f1_2_accel: type fixed, parent right_f1_2, child right_f1_2_accel, origin xyz=0.04 0 0 rpy=-1.57079632679 0 0
- added joint right_f1_base: type fixed, parent right_palm, child right_f1_base, origin xyz=0.115 0.03122 0 rpy=0 0 0.3
- added joint right_f1_fixed_accel: type fixed, parent right_f1_base, child right_f1_fixed_accel, origin xyz=-0.05 0 0 rpy=0 0 0
- added joint right_f1_j0: type revolute, parent right_f1_base, child right_f1_0, origin xyz=0 0 0 rpy=0 0 0, axis 0 0 1, limit lower=-1.57079632679 upper=1.57079632679 effort=11 velocity=-1
- added joint right_f1_j1: type revolute, parent right_f1_0, child right_f1_1, origin xyz=0.028 0 0 rpy=1.57079632679 0 0, axis 0 0 1, limit lower=-1.57079632679 upper=1.57079632679 effort=28 velocity=-1
- added joint right_f1_j2: type revolute, parent right_f1_1, child right_f1_2, origin xyz=0.05 0 0 rpy=0 0 0, axis 0 0 1, limit lower=-1.57079632679 upper=1.57079632679 effort=28 velocity=-1
- added joint right_f2_1_accel: type fixed, parent right_f2_1, child right_f2_1_accel, origin xyz=0.03 0 0 rpy=-1.57079632679 0 0
- added joint right_f2_2_accel: type fixed, parent right_f2_2, child right_f2_2_accel, origin xyz=0.04 0 0 rpy=-1.57079632679 0 0
- added joint right_f2_base: type fixed, parent right_palm, child right_f2_base, origin xyz=0.09 0.06245 0 rpy=0 0 0.3
- added joint right_f2_fixed_accel: type fixed, parent right_f2_base, child right_f2_fixed_accel, origin xyz=-0.05 0 0 rpy=0 0 0
- added joint right_f2_j0: type revolute, parent right_f2_base, child right_f2_0, origin xyz=0 0 0 rpy=0 0 0, axis 0 0 1, limit lower=-1.57079632679 upper=1.57079632679 effort=11 velocity=-1
- added joint right_f2_j1: type revolute, parent right_f2_0, child right_f2_1, origin xyz=0.028 0 0 rpy=1.57079632679 0 0, axis 0 0 1, limit lower=-1.57079632679 upper=1.57079632679 effort=28 velocity=-1
- added joint right_f2_j2: type revolute, parent right_f2_1, child right_f2_2, origin xyz=0.05 0 0 rpy=0 0 0, axis 0 0 1, limit lower=-1.57079632679 upper=1.57079632679 effort=28 velocity=-1
- added joint right_f3_1_accel: type fixed, parent right_f3_1, child right_f3_1_accel, origin xyz=0.03 0 0 rpy=-1.57079632679 0 0
- added joint right_f3_2_accel: type fixed, parent right_f3_2, child right_f3_2_accel, origin xyz=0.04 0 0 rpy=-1.57079632679 0 0
- added joint right_f3_base: type fixed, parent right_palm, child right_f3_base, origin xyz=0.03995 -0.04383 0.014 rpy=0 -1.57079632679 -2.3562
- added joint right_f3_fixed_accel: type fixed, parent right_f3_base, child right_f3_fixed_accel, origin xyz=-0.05 0 0 rpy=0 0 0
- added joint right_f3_j0: type revolute, parent right_f3_base, child right_f3_0, origin xyz=0 0 0 rpy=0 0 0, axis 0 0 1, limit lower=-1.57079632679 upper=1.57079632679 effort=11 velocity=-1
- added joint right_f3_j1: type revolute, parent right_f3_0, child right_f3_1, origin xyz=0.028 0 0 rpy=1.57079632679 0 0, axis 0 0 1, limit lower=-1.57079632679 upper=1.57079632679 effort=28 velocity=-1
- added joint right_f3_j2: type revolute, parent right_f3_1, child right_f3_2, origin xyz=0.05 0 0 rpy=0 0 0, axis 0 0 1, limit lower=-1.57079632679 upper=1.57079632679 effort=28 velocity=-1
- added joint right_palm_left_camera_frame_joint: type fixed, parent right_palm, child right_palm_left_camera_frame, origin xyz=0.0683774130138 0.0138342911048 0.025 rpy=0.6708 -1.57079632679 3.14159265359
- added joint right_palm_left_camera_optical_frame_joint: type fixed, parent right_palm_left_camera_frame, child right_palm_left_camera_optical_frame, origin xyz=0 0 0 rpy=-1.57079632679 0.0 -1.57079632679
- added joint right_palm_right_camera_frame_joint: type fixed, parent right_palm, child right_palm_right_camera_frame, origin xyz=0.0435128991906 0.0451672761576 0.025 rpy=0.6708 -1.57079632679 3.14159265359
- added joint right_palm_right_camera_optical_frame_joint: type fixed, parent right_palm_right_camera_frame, child right_palm_right_camera_optical_frame, origin xyz=0 0 0 rpy=-1.57079632679 0.0 -1.57079632679
- added joint right_sandia_hand_joint: type fixed, parent r_hand, child right_palm, origin xyz=-0.00179 -0.13516 0.01176 rpy=0 0 -1.57079

File: software/models/mit_gazebo_models/mit_robot/model_LS_RN.urdf (robot description, URDF)
Before this commit: robot atlas, 122 links, 121 joints
Links:
- removed link right_f0_0
- removed link right_f0_1
- removed link right_f0_1_accel
- removed link right_f0_2
- removed link right_f0_2_accel
- removed link right_f0_base
- removed link right_f0_fixed_accel
- removed link right_f1_0
- removed link right_f1_1
- removed link right_f1_1_accel
- removed link right_f1_2
- removed link right_f1_2_accel
- removed link right_f1_base
- removed link right_f1_fixed_accel
- removed link right_f2_0
- removed link right_f2_1
- removed link right_f2_1_accel
- removed link right_f2_2
- removed link right_f2_2_accel
- removed link right_f2_base
- removed link right_f2_fixed_accel
- removed link right_f3_0
- removed link right_f3_1
- removed link right_f3_1_accel
- removed link right_f3_2
- removed link right_f3_2_accel
- removed link right_f3_base
- removed link right_f3_fixed_accel
- removed link right_palm
- removed link right_palm_left_camera_frame
- removed link right_palm_left_camera_optical_frame
- removed link right_palm_right_camera_frame
- removed link right_palm_right_camera_optical_frame
Joints:
- removed joint right_f0_1_accel
- removed joint right_f0_2_accel
- removed joint right_f0_base
- removed joint right_f0_fixed_accel
- removed joint right_f0_j0
- removed joint right_f0_j1
- removed joint right_f0_j2
- removed joint right_f1_1_accel
- removed joint right_f1_2_accel
- removed joint right_f1_base
- removed joint right_f1_fixed_accel
- removed joint right_f1_j0
- removed joint right_f1_j1
- removed joint right_f1_j2
- removed joint right_f2_1_accel
- removed joint right_f2_2_accel
- removed joint right_f2_base
- removed joint right_f2_fixed_accel
- removed joint right_f2_j0
- removed joint right_f2_j1
- removed joint right_f2_j2
- removed joint right_f3_1_accel
- removed joint right_f3_2_accel
- removed joint right_f3_base
- removed joint right_f3_fixed_accel
- removed joint right_f3_j0
- removed joint right_f3_j1
- removed joint right_f3_j2
- removed joint right_palm_left_camera_frame_joint
- removed joint right_palm_left_camera_optical_frame_joint
- removed joint right_palm_right_camera_frame_joint
- removed joint right_palm_right_camera_optical_frame_joint
- removed joint right_sandia_hand_joint
