Commit message: Changed z-sign of right sandia to correspond with new mesh location (rotated right hand mesh in skeleton)
git-svn-id: https://svn.csail.mit.edu/drc/trunk@6724 c7283977-0100-402a-a91a-fa70b306dbfe

File: software/models/mit_gazebo_models/mit_robot/model_LI_RS.urdf (robot description, URDF)
Before this commit: robot atlas, 98 links, 97 joints
Joints:
- joint right_sandia_hand_joint: origin xyz=-0.00179 -0.13516 0.01176 rpy=0 0 -1.57079 -> xyz=-0.00179 -0.13516 -0.01176 rpy=0 0 -1.57079

File: software/models/mit_gazebo_models/mit_robot/model_LN_RS.urdf (robot description, URDF)
Before this commit: robot atlas, 89 links, 88 joints
Joints:
- joint right_sandia_hand_joint: origin xyz=-0.00179 -0.13516 0.01176 rpy=0 0 -1.57079 -> xyz=-0.00179 -0.13516 -0.01176 rpy=0 0 -1.57079

File: software/models/mit_gazebo_models/mit_robot/model_LS_RS.urdf (robot description, URDF)
Before this commit: robot atlas, 122 links, 121 joints
Joints:
- joint right_sandia_hand_joint: origin xyz=-0.00179 -0.13516 0.01176 rpy=0 0 -1.57079 -> xyz=-0.00179 -0.13516 -0.01176 rpy=0 0 -1.57079

File: software/models/mit_gazebo_models/mit_robot/model_sim.urdf (robot description, URDF)
Before this commit: robot atlas, 111 links, 110 joints
Joints:
- joint right_sandia_hand_joint: origin xyz=-0.00179 -0.13516 0.01176 rpy=0 0 -1.57079 -> xyz=-0.00179 -0.13516 -0.01176 rpy=0 0 -1.57079

File: software/models/mit_gazebo_models/mit_robot/model_sim_gazebo.urdf (robot description, URDF)
Before this commit: robot atlas, 111 links, 110 joints
Joints:
- joint right_sandia_hand_joint: origin xyz=-0.00179 -0.13516 0.01176 rpy=0 0 -1.57079 -> xyz=-0.00179 -0.13516 -0.01176 rpy=0 0 -1.57079

File: software/models/mit_gazebo_models/mit_robot/xacro/atlas_irobot_left_sandia_right.urdf.xacro (robot description, xacro)
@@ -3,5 +3,5 @@
   <xacro:include filename="$(find handle_description)/src/irobot_hand_simple.urdf.xacro" />
   <xacro:sandia_hand side="right" parent="r_hand" reflect="1" joint_type="revolute" thumb_angle="0">
-    <origin xyz="-0.00179 -0.13516 0.01176" rpy="0 0 -1.57079"/>
+    <origin xyz="-0.00179 -0.13516 -0.01176" rpy="0 0 -1.57079"/>
   </xacro:sandia_hand>
   <xacro:irobot_hand side="left" parent="l_hand" reflect="-1">

File: software/models/mit_gazebo_models/mit_robot/xacro/atlas_sandia_hands.urdf.xacro (robot description, xacro)
@@ -2,5 +2,5 @@
   <xacro:include filename="$(find sandia_hand_description)/urdf/sandia_hand_simple_shapes.urdf.xacro" />
   <xacro:sandia_hand side="right" parent="r_hand" reflect="1" joint_type="revolute" thumb_angle="0">
-    <origin xyz="-0.00179 -0.13516 0.01176" rpy="0 0 -1.57079"/>
+    <origin xyz="-0.00179 -0.13516 -0.01176" rpy="0 0 -1.57079"/>
   </xacro:sandia_hand>
   <xacro:sandia_hand side="left" parent="l_hand" reflect="-1" joint_type="revolute" thumb_angle="0">

File: software/models/mit_gazebo_models/mit_robot/xacro/atlas_sandia_hands_sim.urdf.xacro (robot description, xacro)
@@ -2,5 +2,5 @@
   <xacro:include filename="$(find sandia_hand_description)/urdf/sandia_hand_simple_shapes.urdf.xacro" />
   <xacro:sandia_hand side="right" parent="r_hand" reflect="1" joint_type="revolute" thumb_angle="0">
-    <origin xyz="-0.00179 -0.13516 0.01176" rpy="0 0 -1.57079"/>
+    <origin xyz="-0.00179 -0.13516 -0.01176" rpy="0 0 -1.57079"/>
   </xacro:sandia_hand>
   <xacro:sandia_hand side="left" parent="l_hand" reflect="-1" joint_type="revolute" thumb_angle="0">

File: software/models/mit_gazebo_models/mit_robot/xacro/atlas_stump_left_sandia_right.urdf.xacro (robot description, xacro)
@@ -2,5 +2,5 @@
   <xacro:include filename="$(find sandia_hand_description)/urdf/sandia_hand_simple_shapes.urdf.xacro" />
   <xacro:sandia_hand side="right" parent="r_hand" reflect="1" joint_type="revolute" thumb_angle="0">
-    <origin xyz="-0.00179 -0.13516 0.01176" rpy="0 0 -1.57079"/>
+    <origin xyz="-0.00179 -0.13516 -0.01176" rpy="0 0 -1.57079"/>
   </xacro:sandia_hand>
   <include filename="$(find mit_drcsim_scripts)/models/mit_robot/xacro/atlas_skeleton.urdf" />
