Commit message: working models for all robots
git-svn-id: https://svn.csail.mit.edu/drc/trunk@5870 c7283977-0100-402a-a91a-fa70b306dbfe

File: software/models/mit_gazebo_models/mit_robot/model_LI_RI.urdf (robot description, URDF)
Before this commit: robot atlas, 71 links, 70 joints
Links:
- removed link head_root
Joints:
- removed joint head_root_joint

File: software/models/mit_gazebo_models/mit_robot/model_LI_RS.urdf (robot description, URDF)
Before this commit: robot atlas, 95 links, 94 joints
Links:
- removed link head_root
Joints:
- removed joint head_root_joint

File: software/models/mit_gazebo_models/mit_robot/model_LS_RI.urdf (robot description, URDF)
Before this commit: robot atlas, 95 links, 94 joints
Links:
- removed link head_root
Joints:
- removed joint head_root_joint

File: software/models/mit_gazebo_models/mit_robot/model_LS_RS.urdf (robot description, URDF)
Before this commit: robot atlas, 119 links, 118 joints
Links:
- removed link head_root
Joints:
- removed joint head_root_joint

File: software/models/mit_gazebo_models/mit_robot/model_stumps.urdf (robot description, URDF)
Before this commit: robot atlas, 54 links, 53 joints
Links:
- removed link head_root
Joints:
- removed joint head_root_joint

Commit message: updated arm joint limits to sync up with the real robot. this will break some things in control until fixed points have been updated
git-svn-id: https://svn.csail.mit.edu/drc/trunk@5992 c7283977-0100-402a-a91a-fa70b306dbfe

File: software/models/mit_gazebo_models/mit_robot/model_LI_RI.urdf (robot description, URDF)
Before this commit: robot atlas, 70 links, 69 joints
Joints:
- joint back_bkx: limit lower=-0.790809 upper=0.790809 effort=94.91 velocity=12 -> lower=-0.5 upper=0.5 effort=94.91 velocity=12
- joint back_bky: limit lower=-1.2 upper=1.28 effort=206.843 velocity=12 -> lower=-0.62 upper=0.46 effort=206.843 velocity=12
- joint l_arm_mwx: limit lower=-0.436 upper=1.571 effort=60 velocity=12 -> lower=-1.165 upper=1.125 effort=60 velocity=12
- joint l_arm_shx: limit lower=-1.39626 upper=1.74533 effort=170 velocity=12 -> lower=-1.54 upper=1.45 effort=170 velocity=12
- joint l_arm_usy: limit lower=-1.9635 upper=1.9635 effort=212 velocity=12 -> lower=-1.55 upper=0.75 effort=212 velocity=12
- joint l_arm_uwy: limit lower=-1.571 upper=1.571 effort=114 velocity=12 -> lower=0.0 upper=3.07 effort=114 velocity=12
- joint r_arm_mwx: limit lower=-1.571 upper=0.436 effort=60 velocity=12 -> lower=-1.165 upper=1.125 effort=60 velocity=12
- joint r_arm_shx: limit lower=-1.74533 upper=1.39626 effort=170 velocity=12 -> lower=-1.45 upper=1.54 effort=170 velocity=12
- joint r_arm_usy: limit lower=-1.9635 upper=1.9635 effort=212 velocity=12 -> lower=-1.55 upper=0.75 effort=212 velocity=12
- joint r_arm_uwy: limit lower=-1.571 upper=1.571 effort=114 velocity=12 -> lower=0.0 upper=3.07 effort=114 velocity=12

File: software/models/mit_gazebo_models/mit_robot/model_LI_RS.urdf (robot description, URDF)
Before this commit: robot atlas, 94 links, 93 joints
Joints:
- joint back_bkx: limit lower=-0.790809 upper=0.790809 effort=94.91 velocity=12 -> lower=-0.5 upper=0.5 effort=94.91 velocity=12
- joint back_bky: limit lower=-1.2 upper=1.28 effort=206.843 velocity=12 -> lower=-0.62 upper=0.46 effort=206.843 velocity=12
- joint l_arm_mwx: limit lower=-0.436 upper=1.571 effort=60 velocity=12 -> lower=-1.165 upper=1.125 effort=60 velocity=12
- joint l_arm_shx: limit lower=-1.39626 upper=1.74533 effort=170 velocity=12 -> lower=-1.54 upper=1.45 effort=170 velocity=12
- joint l_arm_usy: limit lower=-1.9635 upper=1.9635 effort=212 velocity=12 -> lower=-1.55 upper=0.75 effort=212 velocity=12
- joint l_arm_uwy: limit lower=-1.571 upper=1.571 effort=114 velocity=12 -> lower=0.0 upper=3.07 effort=114 velocity=12
- joint r_arm_mwx: limit lower=-1.571 upper=0.436 effort=60 velocity=12 -> lower=-1.165 upper=1.125 effort=60 velocity=12
- joint r_arm_shx: limit lower=-1.74533 upper=1.39626 effort=170 velocity=12 -> lower=-1.45 upper=1.54 effort=170 velocity=12
- joint r_arm_usy: limit lower=-1.9635 upper=1.9635 effort=212 velocity=12 -> lower=-1.55 upper=0.75 effort=212 velocity=12
- joint r_arm_uwy: limit lower=-1.571 upper=1.571 effort=114 velocity=12 -> lower=0.0 upper=3.07 effort=114 velocity=12

File: software/models/mit_gazebo_models/mit_robot/model_LS_RI.urdf (robot description, URDF)
Before this commit: robot atlas, 94 links, 93 joints
Joints:
- joint back_bkx: limit lower=-0.790809 upper=0.790809 effort=94.91 velocity=12 -> lower=-0.5 upper=0.5 effort=94.91 velocity=12
- joint back_bky: limit lower=-1.2 upper=1.28 effort=206.843 velocity=12 -> lower=-0.62 upper=0.46 effort=206.843 velocity=12
- joint l_arm_mwx: limit lower=-0.436 upper=1.571 effort=60 velocity=12 -> lower=-1.165 upper=1.125 effort=60 velocity=12
- joint l_arm_shx: limit lower=-1.39626 upper=1.74533 effort=170 velocity=12 -> lower=-1.54 upper=1.45 effort=170 velocity=12
- joint l_arm_usy: limit lower=-1.9635 upper=1.9635 effort=212 velocity=12 -> lower=-1.55 upper=0.75 effort=212 velocity=12
- joint l_arm_uwy: limit lower=-1.571 upper=1.571 effort=114 velocity=12 -> lower=0.0 upper=3.07 effort=114 velocity=12
- joint r_arm_mwx: limit lower=-1.571 upper=0.436 effort=60 velocity=12 -> lower=-1.165 upper=1.125 effort=60 velocity=12
- joint r_arm_shx: limit lower=-1.74533 upper=1.39626 effort=170 velocity=12 -> lower=-1.45 upper=1.54 effort=170 velocity=12
- joint r_arm_usy: limit lower=-1.9635 upper=1.9635 effort=212 velocity=12 -> lower=-1.55 upper=0.75 effort=212 velocity=12
- joint r_arm_uwy: limit lower=-1.571 upper=1.571 effort=114 velocity=12 -> lower=0.0 upper=3.07 effort=114 velocity=12

File: software/models/mit_gazebo_models/mit_robot/model_LS_RS.urdf (robot description, URDF)
Before this commit: robot atlas, 118 links, 117 joints
Joints:
- joint back_bkx: limit lower=-0.790809 upper=0.790809 effort=94.91 velocity=12 -> lower=-0.5 upper=0.5 effort=94.91 velocity=12
- joint back_bky: limit lower=-1.2 upper=1.28 effort=206.843 velocity=12 -> lower=-0.62 upper=0.46 effort=206.843 velocity=12
- joint l_arm_mwx: limit lower=-0.436 upper=1.571 effort=60 velocity=12 -> lower=-1.165 upper=1.125 effort=60 velocity=12
- joint l_arm_shx: limit lower=-1.39626 upper=1.74533 effort=170 velocity=12 -> lower=-1.54 upper=1.45 effort=170 velocity=12
- joint l_arm_usy: limit lower=-1.9635 upper=1.9635 effort=212 velocity=12 -> lower=-1.55 upper=0.75 effort=212 velocity=12
- joint l_arm_uwy: limit lower=-1.571 upper=1.571 effort=114 velocity=12 -> lower=0.0 upper=3.07 effort=114 velocity=12
- joint r_arm_mwx: limit lower=-1.571 upper=0.436 effort=60 velocity=12 -> lower=-1.165 upper=1.125 effort=60 velocity=12
- joint r_arm_shx: limit lower=-1.74533 upper=1.39626 effort=170 velocity=12 -> lower=-1.45 upper=1.54 effort=170 velocity=12
- joint r_arm_usy: limit lower=-1.9635 upper=1.9635 effort=212 velocity=12 -> lower=-1.55 upper=0.75 effort=212 velocity=12
- joint r_arm_uwy: limit lower=-1.571 upper=1.571 effort=114 velocity=12 -> lower=0.0 upper=3.07 effort=114 velocity=12

File: software/models/mit_gazebo_models/mit_robot/model_sim.urdf (robot description, URDF)
Before this commit: robot atlas, 107 links, 106 joints
Joints:
- joint back_bkx: limit lower=-0.790809 upper=0.790809 effort=94.91 velocity=12 -> lower=-0.5 upper=0.5 effort=94.91 velocity=12
- joint back_bky: limit lower=-1.2 upper=1.28 effort=206.843 velocity=12 -> lower=-0.62 upper=0.46 effort=206.843 velocity=12
- joint l_arm_mwx: limit lower=-0.436 upper=1.571 effort=60 velocity=12 -> lower=-1.165 upper=1.125 effort=60 velocity=12
- joint l_arm_shx: limit lower=-1.39626 upper=1.74533 effort=170 velocity=12 -> lower=-1.54 upper=1.45 effort=170 velocity=12
- joint l_arm_usy: limit lower=-1.9635 upper=1.9635 effort=212 velocity=12 -> lower=-1.55 upper=0.75 effort=212 velocity=12
- joint l_arm_uwy: limit lower=-1.571 upper=1.571 effort=114 velocity=12 -> lower=0.0 upper=3.07 effort=114 velocity=12
- joint r_arm_mwx: limit lower=-1.571 upper=0.436 effort=60 velocity=12 -> lower=-1.165 upper=1.125 effort=60 velocity=12
- joint r_arm_shx: limit lower=-1.74533 upper=1.39626 effort=170 velocity=12 -> lower=-1.45 upper=1.54 effort=170 velocity=12
- joint r_arm_usy: limit lower=-1.9635 upper=1.9635 effort=212 velocity=12 -> lower=-1.55 upper=0.75 effort=212 velocity=12
- joint r_arm_uwy: limit lower=-1.571 upper=1.571 effort=114 velocity=12 -> lower=0.0 upper=3.07 effort=114 velocity=12

File: software/models/mit_gazebo_models/mit_robot/model_sim_gazebo.urdf (robot description, URDF)
Before this commit: robot atlas, 107 links, 106 joints
Joints:
- joint back_mby: limit lower=-1.2 upper=1.28 effort=206.843 velocity=12 -> lower=-0.62 upper=0.46 effort=206.843 velocity=12
- joint back_ubx: limit lower=-0.790809 upper=0.790809 effort=94.91 velocity=12 -> lower=-0.5 upper=0.5 effort=94.91 velocity=12
- joint l_arm_mwx: limit lower=-0.436 upper=1.571 effort=60 velocity=12 -> lower=-1.165 upper=1.125 effort=60 velocity=12
- joint l_arm_shx: limit lower=-1.39626 upper=1.74533 effort=170 velocity=12 -> lower=-1.54 upper=1.45 effort=170 velocity=12
- joint l_arm_usy: limit lower=-1.9635 upper=1.9635 effort=212 velocity=12 -> lower=-1.55 upper=0.75 effort=212 velocity=12
- joint l_arm_uwy: limit lower=-1.571 upper=1.571 effort=114 velocity=12 -> lower=0.0 upper=3.07 effort=114 velocity=12
- joint r_arm_mwx: limit lower=-1.571 upper=0.436 effort=60 velocity=12 -> lower=-1.165 upper=1.125 effort=60 velocity=12
- joint r_arm_shx: limit lower=-1.74533 upper=1.39626 effort=170 velocity=12 -> lower=-1.45 upper=1.54 effort=170 velocity=12
- joint r_arm_usy: limit lower=-1.9635 upper=1.9635 effort=212 velocity=12 -> lower=-1.55 upper=0.75 effort=212 velocity=12
- joint r_arm_uwy: limit lower=-1.571 upper=1.571 effort=114 velocity=12 -> lower=0.0 upper=3.07 effort=114 velocity=12

File: software/models/mit_gazebo_models/mit_robot/model_stumps.urdf (robot description, URDF)
Before this commit: robot atlas, 53 links, 52 joints
Joints:
- joint back_bkx: limit lower=-0.790809 upper=0.790809 effort=94.91 velocity=12 -> lower=-0.5 upper=0.5 effort=94.91 velocity=12
- joint back_bky: limit lower=-1.2 upper=1.28 effort=206.843 velocity=12 -> lower=-0.62 upper=0.46 effort=206.843 velocity=12
- joint l_arm_mwx: limit lower=-0.436 upper=1.571 effort=60 velocity=12 -> lower=-1.165 upper=1.125 effort=60 velocity=12
- joint l_arm_shx: limit lower=-1.39626 upper=1.74533 effort=170 velocity=12 -> lower=-1.54 upper=1.45 effort=170 velocity=12
- joint l_arm_usy: limit lower=-1.9635 upper=1.9635 effort=212 velocity=12 -> lower=-1.55 upper=0.75 effort=212 velocity=12
- joint l_arm_uwy: limit lower=-1.571 upper=1.571 effort=114 velocity=12 -> lower=0.0 upper=3.07 effort=114 velocity=12
- joint r_arm_mwx: limit lower=-1.571 upper=0.436 effort=60 velocity=12 -> lower=-1.165 upper=1.125 effort=60 velocity=12
- joint r_arm_shx: limit lower=-1.74533 upper=1.39626 effort=170 velocity=12 -> lower=-1.45 upper=1.54 effort=170 velocity=12
- joint r_arm_usy: limit lower=-1.9635 upper=1.9635 effort=212 velocity=12 -> lower=-1.55 upper=0.75 effort=212 velocity=12
- joint r_arm_uwy: limit lower=-1.571 upper=1.571 effort=114 velocity=12 -> lower=0.0 upper=3.07 effort=114 velocity=12

File: software/models/mit_gazebo_models/mit_robot/xacro/atlas_skeleton.urdf (robot description, URDF)
Before this commit: robot drc_skeleton, 28 links, 28 joints
Joints:
- joint back_bkx: limit lower=-0.790809 upper=0.790809 effort=94.91 velocity=12 -> lower=-0.5 upper=0.5 effort=94.91 velocity=12
- joint back_bky: limit lower=-1.2 upper=1.28 effort=206.843 velocity=12 -> lower=-0.62 upper=0.46 effort=206.843 velocity=12
- joint l_arm_mwx: limit lower=-0.436 upper=1.571 effort=60 velocity=12 -> lower=-1.165 upper=1.125 effort=60 velocity=12
- joint l_arm_shx: limit lower=-1.39626 upper=1.74533 effort=170 velocity=12 -> lower=-1.54 upper=1.45 effort=170 velocity=12
- joint l_arm_usy: limit lower=-1.9635 upper=1.9635 effort=212 velocity=12 -> lower=-1.55 upper=0.75 effort=212 velocity=12
- joint l_arm_uwy: limit lower=-1.571 upper=1.571 effort=114 velocity=12 -> lower=0.0 upper=3.07 effort=114 velocity=12
- joint r_arm_mwx: limit lower=-1.571 upper=0.436 effort=60 velocity=12 -> lower=-1.165 upper=1.125 effort=60 velocity=12
- joint r_arm_shx: limit lower=-1.74533 upper=1.39626 effort=170 velocity=12 -> lower=-1.45 upper=1.54 effort=170 velocity=12
- joint r_arm_usy: limit lower=-1.9635 upper=1.9635 effort=212 velocity=12 -> lower=-1.55 upper=0.75 effort=212 velocity=12
- joint r_arm_uwy: limit lower=-1.571 upper=1.571 effort=114 velocity=12 -> lower=0.0 upper=3.07 effort=114 velocity=12

File: software/models/mit_gazebo_models/mit_robot_drake/model_minimal_contact.urdf (robot description, URDF)
Before this commit: robot atlas, 29 links, 28 joints
Joints:
- joint back_bkx: limit lower=-0.790809 upper=0.790809 effort=94.91 velocity=12 -> lower=-0.5 upper=0.5 effort=94.91 velocity=12
- joint back_bky: limit lower=-1.2 upper=1.28 effort=206.843 velocity=12 -> lower=-0.62 upper=0.46 effort=206.843 velocity=12
- joint l_arm_mwx: limit lower=-0.436 upper=1.571 effort=60 velocity=12 -> lower=-1.165 upper=1.125 effort=60 velocity=12
- joint l_arm_shx: limit lower=-1.5 upper=1.74533 effort=170 velocity=12 -> lower=-1.54 upper=1.45 effort=170 velocity=12
- joint l_arm_usy: limit lower=-1.9635 upper=1.9635 effort=212 velocity=12 -> lower=-1.55 upper=0.75 effort=212 velocity=12
- joint l_arm_uwy: limit lower=-1.571 upper=1.571 effort=114 velocity=12 -> lower=0.0 upper=3.07 effort=114 velocity=12
- joint r_arm_mwx: limit lower=-1.571 upper=0.436 effort=60 velocity=12 -> lower=-1.165 upper=1.125 effort=60 velocity=12
- joint r_arm_shx: limit lower=-1.74533 upper=1.5 effort=170 velocity=12 -> lower=-1.45 upper=1.54 effort=170 velocity=12
- joint r_arm_usy: limit lower=-1.9635 upper=1.9635 effort=212 velocity=12 -> lower=-1.55 upper=0.75 effort=212 velocity=12
- joint r_arm_uwy: limit lower=-1.571 upper=1.571 effort=114 velocity=12 -> lower=0.0 upper=3.07 effort=114 velocity=12

File: software/models/mit_gazebo_models/mit_robot_drake/model_minimal_contact_fixedjoint_hands.urdf (robot description, URDF)
Before this commit: robot atlas, 95 links, 94 joints
Joints:
- joint back_bkx: limit lower=-0.790809 upper=0.790809 effort=94.91 velocity=12 -> lower=-0.5 upper=0.5 effort=94.91 velocity=12
- joint back_bky: limit lower=-1.2 upper=1.28 effort=206.843 velocity=12 -> lower=-0.62 upper=0.46 effort=206.843 velocity=12
- joint l_arm_mwx: limit lower=-0.436 upper=1.571 effort=60 velocity=12 -> lower=-1.165 upper=1.125 effort=60 velocity=12
- joint l_arm_shx: limit lower=-1.5 upper=1.74533 effort=170 velocity=12 -> lower=-1.54 upper=1.45 effort=170 velocity=12
- joint l_arm_usy: limit lower=-1.9635 upper=1.9635 effort=212 velocity=12 -> lower=-1.55 upper=0.75 effort=212 velocity=12
- joint l_arm_uwy: limit lower=-1.571 upper=1.571 effort=114 velocity=12 -> lower=0.0 upper=3.07 effort=114 velocity=12
- joint r_arm_mwx: limit lower=-1.571 upper=0.436 effort=60 velocity=12 -> lower=-1.165 upper=1.125 effort=60 velocity=12
- joint r_arm_shx: limit lower=-1.74533 upper=1.5 effort=170 velocity=12 -> lower=-1.45 upper=1.54 effort=170 velocity=12
- joint r_arm_usy: limit lower=-1.9635 upper=1.9635 effort=212 velocity=12 -> lower=-1.55 upper=0.75 effort=212 velocity=12
- joint r_arm_uwy: limit lower=-1.571 upper=1.571 effort=114 velocity=12 -> lower=0.0 upper=3.07 effort=114 velocity=12

File: software/models/mit_gazebo_models/mit_robot_drake/model_minimal_contact_point_hands.urdf (robot description, URDF)
Before this commit: robot atlas, 31 links, 30 joints
Joints:
- joint back_bkx: limit lower=-0.790809 upper=0.790809 effort=94.91 velocity=12 -> lower=-0.5 upper=0.5 effort=94.91 velocity=12
- joint back_bky: limit lower=-1.2 upper=1.28 effort=206.843 velocity=12 -> lower=-0.62 upper=0.46 effort=206.843 velocity=12
- joint l_arm_mwx: limit lower=-0.436 upper=1.571 effort=60 velocity=12 -> lower=-1.165 upper=1.125 effort=60 velocity=12
- joint l_arm_shx: limit lower=-1.5 upper=1.74533 effort=170 velocity=12 -> lower=-1.54 upper=1.45 effort=170 velocity=12
- joint l_arm_usy: limit lower=-1.9635 upper=1.9635 effort=212 velocity=12 -> lower=-1.55 upper=0.75 effort=212 velocity=12
- joint l_arm_uwy: limit lower=-1.571 upper=1.571 effort=114 velocity=12 -> lower=0.0 upper=3.07 effort=114 velocity=12
- joint r_arm_mwx: limit lower=-1.571 upper=0.436 effort=60 velocity=12 -> lower=-1.165 upper=1.125 effort=60 velocity=12
- joint r_arm_shx: limit lower=-1.74533 upper=1.5 effort=170 velocity=12 -> lower=-1.45 upper=1.54 effort=170 velocity=12
- joint r_arm_usy: limit lower=-1.9635 upper=1.9635 effort=212 velocity=12 -> lower=-1.55 upper=0.75 effort=212 velocity=12
- joint r_arm_uwy: limit lower=-1.571 upper=1.571 effort=114 velocity=12 -> lower=0.0 upper=3.07 effort=114 velocity=12

File: software/models/mit_gazebo_models/mit_robot_drake/model_simple_visuals.urdf (robot description, URDF)
Before this commit: robot atlas, 33 links, 32 joints
Joints:
- joint back_bkx: limit lower=-0.790809 upper=0.790809 effort=94.91 velocity=12 -> lower=-0.5 upper=0.5 effort=94.91 velocity=12
- joint back_bky: limit lower=-1.2 upper=1.28 effort=206.843 velocity=12 -> lower=-0.62 upper=0.46 effort=206.843 velocity=12
- joint l_arm_mwx: limit lower=-0.436 upper=1.571 effort=60 velocity=12 -> lower=-1.165 upper=1.125 effort=60 velocity=12
- joint l_arm_shx: limit lower=-1.5 upper=1.74533 effort=170 velocity=12 -> lower=-1.54 upper=1.45 effort=170 velocity=12
- joint l_arm_usy: limit lower=-1.9635 upper=1.9635 effort=212 velocity=12 -> lower=-1.55 upper=0.75 effort=212 velocity=12
- joint l_arm_uwy: limit lower=-1.571 upper=1.571 effort=114 velocity=12 -> lower=0.0 upper=3.07 effort=114 velocity=12
- joint r_arm_mwx: limit lower=-1.571 upper=0.436 effort=60 velocity=12 -> lower=-1.165 upper=1.125 effort=60 velocity=12
- joint r_arm_shx: limit lower=-1.74533 upper=1.5 effort=170 velocity=12 -> lower=-1.45 upper=1.54 effort=170 velocity=12
- joint r_arm_usy: limit lower=-1.9635 upper=1.9635 effort=212 velocity=12 -> lower=-1.55 upper=0.75 effort=212 velocity=12
- joint r_arm_uwy: limit lower=-1.571 upper=1.571 effort=114 velocity=12 -> lower=0.0 upper=3.07 effort=114 velocity=12

File: software/models/mit_gazebo_models/mit_robot_drake/xacro/atlas_skeleton_minimal_contact.urdf (robot description, URDF)
Before this commit: robot drc_skeleton, 28 links, 28 joints
Joints:
- joint back_bkx: limit lower=-0.790809 upper=0.790809 effort=94.91 velocity=12 -> lower=-0.5 upper=0.5 effort=94.91 velocity=12
- joint back_bky: limit lower=-1.2 upper=1.28 effort=206.843 velocity=12 -> lower=-0.62 upper=0.46 effort=206.843 velocity=12
- joint l_arm_mwx: limit lower=-0.436 upper=1.571 effort=60 velocity=12 -> lower=-1.165 upper=1.125 effort=60 velocity=12
- joint l_arm_shx: limit lower=-1.5 upper=1.74533 effort=170 velocity=12 -> lower=-1.54 upper=1.45 effort=170 velocity=12
- joint l_arm_usy: limit lower=-1.9635 upper=1.9635 effort=212 velocity=12 -> lower=-1.55 upper=0.75 effort=212 velocity=12
- joint l_arm_uwy: limit lower=-1.571 upper=1.571 effort=114 velocity=12 -> lower=0.0 upper=3.07 effort=114 velocity=12
- joint r_arm_mwx: limit lower=-1.571 upper=0.436 effort=60 velocity=12 -> lower=-1.165 upper=1.125 effort=60 velocity=12
- joint r_arm_shx: limit lower=-1.74533 upper=1.5 effort=170 velocity=12 -> lower=-1.45 upper=1.54 effort=170 velocity=12
- joint r_arm_usy: limit lower=-1.9635 upper=1.9635 effort=212 velocity=12 -> lower=-1.55 upper=0.75 effort=212 velocity=12
- joint r_arm_uwy: limit lower=-1.571 upper=1.571 effort=114 velocity=12 -> lower=0.0 upper=3.07 effort=114 velocity=12

File: software/models/mit_gazebo_models/mit_robot_drake/xacro/atlas_skeleton_simple_visuals.urdf (robot description, URDF)
Before this commit: robot drc_skeleton, 28 links, 28 joints
Joints:
- joint back_bkx: limit lower=-0.790809 upper=0.790809 effort=94.91 velocity=12 -> lower=-0.5 upper=0.5 effort=94.91 velocity=12
- joint back_bky: limit lower=-1.2 upper=1.28 effort=206.843 velocity=12 -> lower=-0.62 upper=0.46 effort=206.843 velocity=12
- joint l_arm_mwx: limit lower=-0.436 upper=1.571 effort=60 velocity=12 -> lower=-1.165 upper=1.125 effort=60 velocity=12
- joint l_arm_shx: limit lower=-1.5 upper=1.74533 effort=170 velocity=12 -> lower=-1.54 upper=1.45 effort=170 velocity=12
- joint l_arm_usy: limit lower=-1.9635 upper=1.9635 effort=212 velocity=12 -> lower=-1.55 upper=0.75 effort=212 velocity=12
- joint l_arm_uwy: limit lower=-1.571 upper=1.571 effort=114 velocity=12 -> lower=0.0 upper=3.07 effort=114 velocity=12
- joint r_arm_mwx: limit lower=-1.571 upper=0.436 effort=60 velocity=12 -> lower=-1.165 upper=1.125 effort=60 velocity=12
- joint r_arm_shx: limit lower=-1.74533 upper=1.5 effort=170 velocity=12 -> lower=-1.45 upper=1.54 effort=170 velocity=12
- joint r_arm_usy: limit lower=-1.9635 upper=1.9635 effort=212 velocity=12 -> lower=-1.55 upper=0.75 effort=212 velocity=12
- joint r_arm_uwy: limit lower=-1.571 upper=1.571 effort=114 velocity=12 -> lower=0.0 upper=3.07 effort=114 velocity=12

File: software/models/mit_gazebo_models/mit_robot_drake/xacro/atlas_skeleton_simple_visuals_minimal_contact.urdf (robot description, URDF)
Before this commit: robot drc_skeleton, 28 links, 28 joints
Joints:
- joint back_bkx: limit lower=-0.790809 upper=0.790809 effort=94.91 velocity=12 -> lower=-0.5 upper=0.5 effort=94.91 velocity=12
- joint back_bky: limit lower=-1.2 upper=1.28 effort=206.843 velocity=12 -> lower=-0.62 upper=0.46 effort=206.843 velocity=12
- joint l_arm_mwx: limit lower=-0.436 upper=1.571 effort=60 velocity=12 -> lower=-1.165 upper=1.125 effort=60 velocity=12
- joint l_arm_shx: limit lower=-1.5 upper=1.74533 effort=170 velocity=12 -> lower=-1.54 upper=1.45 effort=170 velocity=12
- joint l_arm_usy: limit lower=-1.9635 upper=1.9635 effort=212 velocity=12 -> lower=-1.55 upper=0.75 effort=212 velocity=12
- joint l_arm_uwy: limit lower=-1.571 upper=1.571 effort=114 velocity=12 -> lower=0 upper=3.07 effort=114 velocity=12
- joint r_arm_mwx: limit lower=-1.571 upper=0.436 effort=60 velocity=12 -> lower=-1.165 upper=1.125 effort=60 velocity=12
- joint r_arm_shx: limit lower=-1.74533 upper=1.5 effort=170 velocity=12 -> lower=-1.45 upper=1.54 effort=170 velocity=12
- joint r_arm_usy: limit lower=-1.9635 upper=1.9635 effort=212 velocity=12 -> lower=-1.55 upper=0.75 effort=212 velocity=12
- joint r_arm_uwy: limit lower=-1.571 upper=1.571 effort=114 velocity=12 -> lower=0.0 upper=3.07 effort=114 velocity=12
