Commit message: very slight change to neck joint limits based on measurements taken today
git-svn-id: https://svn.csail.mit.edu/drc/trunk@6019 c7283977-0100-402a-a91a-fa70b306dbfe

File: software/models/mit_gazebo_models/mit_robot/model_LI_RI.urdf (robot description, URDF)
Before this commit: robot atlas, 70 links, 69 joints
Joints:
- joint neck_ay: limit lower=-0.610865238 upper=1.13446401 effort=5 velocity=12 -> lower=-0.594 upper=1.147 effort=10 velocity=12

File: software/models/mit_gazebo_models/mit_robot/model_LI_RS.urdf (robot description, URDF)
Before this commit: robot atlas, 94 links, 93 joints
Joints:
- joint neck_ay: limit lower=-0.610865238 upper=1.13446401 effort=5 velocity=12 -> lower=-0.594 upper=1.147 effort=10 velocity=12

File: software/models/mit_gazebo_models/mit_robot/model_LS_RI.urdf (robot description, URDF)
Before this commit: robot atlas, 94 links, 93 joints
Joints:
- joint neck_ay: limit lower=-0.610865238 upper=1.13446401 effort=5 velocity=12 -> lower=-0.594 upper=1.147 effort=10 velocity=12

File: software/models/mit_gazebo_models/mit_robot/model_LS_RS.urdf (robot description, URDF)
Before this commit: robot atlas, 118 links, 117 joints
Joints:
- joint neck_ay: limit lower=-0.610865238 upper=1.13446401 effort=5 velocity=12 -> lower=-0.594 upper=1.147 effort=10 velocity=12

File: software/models/mit_gazebo_models/mit_robot/model_sim.urdf (robot description, URDF)
Before this commit: robot atlas, 107 links, 106 joints
Joints:
- joint neck_ay: limit lower=-0.610865238 upper=1.13446401 effort=5 velocity=12 -> lower=-0.594 upper=1.147 effort=10 velocity=12

File: software/models/mit_gazebo_models/mit_robot/model_sim_gazebo.urdf (robot description, URDF)
Before this commit: robot atlas, 107 links, 106 joints
Joints:
- joint neck_ay: limit lower=-0.610865238 upper=1.13446401 effort=5 velocity=12 -> lower=-0.594 upper=1.147 effort=10 velocity=12

File: software/models/mit_gazebo_models/mit_robot/model_stumps.urdf (robot description, URDF)
Before this commit: robot atlas, 53 links, 52 joints
Joints:
- joint neck_ay: limit lower=-0.610865238 upper=1.13446401 effort=5 velocity=12 -> lower=-0.594 upper=1.147 effort=10 velocity=12

File: software/models/mit_gazebo_models/mit_robot/xacro/atlas_skeleton.urdf (robot description, URDF)
Before this commit: robot drc_skeleton, 28 links, 28 joints
Joints:
- joint neck_ay: limit lower=-0.610865238 upper=1.13446401 effort=5 velocity=12 -> lower=-0.594 upper=1.147 effort=10 velocity=12

File: software/models/mit_gazebo_models/mit_robot_drake/model_minimal_contact.urdf (robot description, URDF)
Before this commit: robot atlas, 29 links, 28 joints
Joints:
- joint neck_ay: limit lower=-0.610865238 upper=1.13446401 effort=5 velocity=12 -> lower=-0.594 upper=1.147 effort=10 velocity=12

File: software/models/mit_gazebo_models/mit_robot_drake/model_minimal_contact_fixedjoint_hands.urdf (robot description, URDF)
Before this commit: robot atlas, 95 links, 94 joints
Joints:
- joint neck_ay: limit lower=-0.610865238 upper=1.13446401 effort=5 velocity=12 -> lower=-0.594 upper=1.147 effort=10 velocity=12

File: software/models/mit_gazebo_models/mit_robot_drake/model_minimal_contact_point_hands.urdf (robot description, URDF)
Before this commit: robot atlas, 31 links, 30 joints
Joints:
- joint neck_ay: limit lower=-0.610865238 upper=1.13446401 effort=5 velocity=12 -> lower=-0.594 upper=1.147 effort=10 velocity=12

File: software/models/mit_gazebo_models/mit_robot_drake/model_simple_visuals.urdf (robot description, URDF)
Before this commit: robot atlas, 33 links, 32 joints
Joints:
- joint neck_ay: limit lower=-0.610865238 upper=1.13446401 effort=5 velocity=12 -> lower=-0.594 upper=1.147 effort=10 velocity=12

File: software/models/mit_gazebo_models/mit_robot_drake/xacro/atlas_skeleton_minimal_contact.urdf (robot description, URDF)
Before this commit: robot drc_skeleton, 28 links, 28 joints
Joints:
- joint neck_ay: limit lower=-0.610865238 upper=1.13446401 effort=5 velocity=12 -> lower=-0.594 upper=1.147 effort=10 velocity=12

File: software/models/mit_gazebo_models/mit_robot_drake/xacro/atlas_skeleton_simple_visuals.urdf (robot description, URDF)
Before this commit: robot drc_skeleton, 28 links, 28 joints
Joints:
- joint neck_ay: limit lower=-0.610865238 upper=1.13446401 effort=5 velocity=12 -> lower=-0.594 upper=1.147 effort=10 velocity=12

File: software/models/mit_gazebo_models/mit_robot_drake/xacro/atlas_skeleton_simple_visuals_minimal_contact.urdf (robot description, URDF)
Before this commit: robot drc_skeleton, 28 links, 28 joints
Joints:
- joint neck_ay: limit lower=-0.610865238 upper=1.13446401 effort=5 velocity=12 -> lower=-0.594 upper=1.147 effort=10 velocity=12

Commit message: committing new models with lo-fi head
git-svn-id: https://svn.csail.mit.edu/drc/trunk@6049 c7283977-0100-402a-a91a-fa70b306dbfe

File: software/models/mit_gazebo_models/mit_robot/model_LI_RI.urdf (robot description, URDF)
Before this commit: robot atlas, 70 links, 69 joints
Links:
- link head: geometry collision box size=0.1311 0.12 0.0591; visual mesh filename=package://multisense_sl/meshes/head.dae
- link hokuyo_link: geometry collision cylinder length=0.047 radius=0.024425; visual mesh filename=package://multisense_sl/meshes/head_camera.dae

File: software/models/mit_gazebo_models/mit_robot/model_LI_RS.urdf (robot description, URDF)
Before this commit: robot atlas, 94 links, 93 joints
Links:
- link head: geometry collision box size=0.1311 0.12 0.0591; visual mesh filename=package://multisense_sl/meshes/head.dae
- link hokuyo_link: geometry collision cylinder length=0.047 radius=0.024425; visual mesh filename=package://multisense_sl/meshes/head_camera.dae

File: software/models/mit_gazebo_models/mit_robot/model_LS_RI.urdf (robot description, URDF)
Before this commit: robot atlas, 94 links, 93 joints
Links:
- link head: geometry collision box size=0.1311 0.12 0.0591; visual mesh filename=package://multisense_sl/meshes/head.dae
- link hokuyo_link: geometry collision cylinder length=0.047 radius=0.024425; visual mesh filename=package://multisense_sl/meshes/head_camera.dae

File: software/models/mit_gazebo_models/mit_robot/model_LS_RS.urdf (robot description, URDF)
Before this commit: robot atlas, 118 links, 117 joints
Links:
- link head: geometry collision box size=0.1311 0.12 0.0591; visual mesh filename=package://multisense_sl/meshes/head.dae
- link hokuyo_link: geometry collision cylinder length=0.047 radius=0.024425; visual mesh filename=package://multisense_sl/meshes/head_camera.dae

File: software/models/mit_gazebo_models/mit_robot/model_stumps.urdf (robot description, URDF)
Before this commit: robot atlas, 53 links, 52 joints
Links:
- link head: geometry collision box size=0.1311 0.12 0.0591; visual mesh filename=package://multisense_sl/meshes/head.dae
- link hokuyo_link: geometry collision cylinder length=0.047 radius=0.024425; visual mesh filename=package://multisense_sl/meshes/head_camera.dae

File: software/models/mit_gazebo_models/multisense_sl/multisense_sl.urdf (robot description, URDF)
Before this commit: robot multisense, 24 links, 23 joints
Links:
- link head: geometry collision box size=0.1311 0.12 0.0591; visual mesh filename=package://multisense_sl/meshes/head.dae
- link hokuyo_link: geometry collision cylinder length=0.047 radius=0.024425; visual mesh filename=package://multisense_sl/meshes/head_camera.dae

Commit message: adding ft sensor and coupling plate offset into the urdf
git-svn-id: https://svn.csail.mit.edu/drc/trunk@6175 c7283977-0100-402a-a91a-fa70b306dbfe

File: software/models/mit_gazebo_models/mit_robot/model_LI_RI.urdf (robot description, URDF)
Before this commit: robot atlas, 70 links, 69 joints
Joints:
- joint left_irobot_hand_joint: origin xyz=0 0.05 0 rpy=1.57079 0 3.14159 -> xyz=0 0.095 0 rpy=1.57079 0 3.14159
- joint right_irobot_hand_joint: origin xyz=0 -0.05 0 rpy=1.57079 0 0 -> xyz=0 -0.095 0 rpy=1.57079 0 0

File: software/models/mit_gazebo_models/mit_robot/model_LI_RS.urdf (robot description, URDF)
Before this commit: robot atlas, 94 links, 93 joints
Joints:
- joint left_irobot_hand_joint: origin xyz=0 0.05 0 rpy=1.57079 0 3.14159 -> xyz=0 0.095 0 rpy=1.57079 0 3.14159
- joint right_sandia_hand_joint: origin xyz=0 -0.1 0 rpy=-1.57079 0 -1.57079 -> xyz=0 -0.145 0 rpy=-1.57079 0 -1.57079

File: software/models/mit_gazebo_models/mit_robot/model_LS_RI.urdf (robot description, URDF)
Before this commit: robot atlas, 94 links, 93 joints
Joints:
- joint left_sandia_hand_joint: origin xyz=0  0.1 0 rpy= 1.57079 0  1.57079 -> xyz=0  0.145 0 rpy= 1.57079 0  1.57079
- joint right_irobot_hand_joint: origin xyz=0 -0.05 0 rpy=1.57079 0 0 -> xyz=0 -0.095 0 rpy=1.57079 0 0

File: software/models/mit_gazebo_models/mit_robot/model_LS_RS.urdf (robot description, URDF)
Before this commit: robot atlas, 118 links, 117 joints
Joints:
- joint left_sandia_hand_joint: origin xyz=0  0.1 0 rpy=0 0  1.57079 -> xyz=0  0.145 0 rpy=0 0  1.57079
- joint right_sandia_hand_joint: origin xyz=0 -0.1 0 rpy=0.0 0 -1.57079 -> xyz=0 -0.145 0 rpy=0.0 0 -1.57079

File: software/models/mit_gazebo_models/mit_robot/model_sim.urdf (robot description, URDF)
Before this commit: robot atlas, 107 links, 106 joints
Joints:
- joint left_sandia_hand_joint: origin xyz=0  0.1 0 rpy=0.0 0  1.57079 -> xyz=0  0.145 0 rpy=0.0 0  1.57079
- joint right_sandia_hand_joint: origin xyz=0 -0.1 0 rpy=0.0 0 -1.57079 -> xyz=0 -0.145 0 rpy=0.0 0 -1.57079

File: software/models/mit_gazebo_models/mit_robot/model_sim_gazebo.urdf (robot description, URDF)
Before this commit: robot atlas, 107 links, 106 joints
Joints:
- joint left_sandia_hand_joint: origin xyz=0  0.1 0 rpy=0.0 0  1.57079 -> xyz=0  0.145 0 rpy=0.0 0  1.57079
- joint right_sandia_hand_joint: origin xyz=0 -0.1 0 rpy=0.0 0 -1.57079 -> xyz=0 -0.145 0 rpy=0.0 0 -1.57079

File: software/models/mit_gazebo_models/mit_robot/xacro/atlas_irobot_hands.urdf.xacro (robot description, xacro)
@@ -4,10 +4,11 @@
   <include filename="$(find mit_drcsim_scripts)/models/multisense_sl/multisense_sl.urdf" />
   <!-- Hands -->
+  <!-- adding an offset in the urdf to account for the ft sensor and the coupling plate, chaning origin form 0.1 to 0.145 for sandia, and 0.05 to 0.095 for irobot-->
   <include filename="$(find handle_description)/src/irobot_hand_simple.urdf.xacro" />
   <xacro:irobot_hand side="right" parent="r_hand" reflect="1">
-    <origin rpy="1.57079 0 0" xyz="0 -0.05 0"/>
+    <origin rpy="1.57079 0 0" xyz="0 -0.095 0"/>
   </xacro:irobot_hand>
   <xacro:irobot_hand side="left" parent="l_hand" reflect="-1">
-    <origin rpy="1.57079 0 3.14159" xyz="0 0.05 0"/>
+    <origin rpy="1.57079 0 3.14159" xyz="0 0.095 0"/>
   </xacro:irobot_hand>
 </robot>

File: software/models/mit_gazebo_models/mit_robot/xacro/atlas_irobot_left_sandia_right.urdf.xacro (robot description, xacro)
@@ -6,6 +6,7 @@
   <include filename="$(find sandia_hand_description)/urdf/sandia_hand_simple_shapes.urdf.xacro" />
   <include filename="$(find handle_description)/src/irobot_hand_simple.urdf.xacro" />
+  <!-- adding an offset in the urdf to account for the ft sensor and the coupling plate, chaning origin form 0.1 to 0.145 for sandia, and 0.05 to 0.095 for irobot-->
   <xacro:sandia_hand side="right" parent="r_hand" reflect="1" joint_type="revolute" thumb_angle="0">
-    <origin xyz="0 -0.1 0" rpy="-1.57079 0 -1.57079"/>
+    <origin xyz="0 -0.145 0" rpy="-1.57079 0 -1.57079"/>
   </xacro:sandia_hand>
 <!--  <xacro:sandia_hand side="left" parent="l_hand" reflect="-1" joint_type="revolute" thumb_angle="0">-->
@@ -13,8 +14,8 @@
 <!--  </xacro:sandia_hand>-->
 <!--  <xacro:irobot_hand side="right" parent="r_hand" reflect="1">-->
-<!--    <origin rpy="1.57079 0 0" xyz="0 -0.05 0"/>-->
+<!--    <origin rpy="1.57079 0 0" xyz="0 -0.095 0"/>-->
 <!--  </xacro:irobot_hand>-->
   <xacro:irobot_hand side="left" parent="l_hand" reflect="-1">
-    <origin rpy="1.57079 0 3.14159" xyz="0 0.05 0"/>
+    <origin rpy="1.57079 0 3.14159" xyz="0 0.095 0"/>
   </xacro:irobot_hand>
 </robot>

File: software/models/mit_gazebo_models/mit_robot/xacro/atlas_sandia_hands.urdf.xacro (robot description, xacro)
@@ -5,10 +5,11 @@
   <!-- Hands -->
   <!-- NB: the Roll of the Sandia Hands is not identical in Sim and Reality -->
+   <!-- adding an offset in the urdf to account for the ft sensor and the coupling plate, chaning origin form 0.1 to 0.145 for sandia, and 0.05 to 0.095 for irobot-->
   <include filename="$(find sandia_hand_description)/urdf/sandia_hand_simple_shapes.urdf.xacro" />
   <xacro:sandia_hand side="right" parent="r_hand" reflect="1" joint_type="revolute" thumb_angle="0">
-    <origin xyz="0 -0.1 0" rpy="0.0 0 -1.57079"/>
+    <origin xyz="0 -0.145 0" rpy="0.0 0 -1.57079"/>
   </xacro:sandia_hand>
   <xacro:sandia_hand side="left" parent="l_hand" reflect="-1" joint_type="revolute" thumb_angle="0">
-    <origin xyz="0  0.1 0" rpy="0 0  1.57079"/>
+    <origin xyz="0  0.145 0" rpy="0 0  1.57079"/>
   </xacro:sandia_hand>
 </robot>

File: software/models/mit_gazebo_models/mit_robot/xacro/atlas_sandia_hands_sim.urdf.xacro (robot description, xacro)
@@ -4,9 +4,10 @@
   <!-- Hands -->
   <!-- NB: the Roll of the Sandia Hands is not identical in Sim and Reality -->
+   <!-- adding an offset in the urdf to account for the ft sensor and the coupling plate, chaning origin form 0.1 to 0.145 for sandia, and 0.05 to 0.095 for irobot-->
   <xacro:sandia_hand side="right" parent="r_hand" reflect="1" joint_type="revolute" thumb_angle="0">
-    <origin xyz="0 -0.1 0" rpy="0.0 0 -1.57079"/>
+    <origin xyz="0 -0.145 0" rpy="0.0 0 -1.57079"/>
   </xacro:sandia_hand>
   <xacro:sandia_hand side="left" parent="l_hand" reflect="-1" joint_type="revolute" thumb_angle="0">
-    <origin xyz="0  0.1 0" rpy="0.0 0  1.57079"/>
+    <origin xyz="0  0.145 0" rpy="0.0 0  1.57079"/>
   </xacro:sandia_hand>
   <include filename="$(find mit_drcsim_scripts)/models/mit_robot/xacro/atlas.gazebo" />

File: software/models/mit_gazebo_models/mit_robot/xacro/atlas_sandia_left_irobot_right.urdf.xacro (robot description, xacro)
@@ -4,17 +4,18 @@
   <include filename="$(find mit_drcsim_scripts)/models/multisense_sl/multisense_sl.urdf" />
 <!-- Hands -->
+ <!-- adding an offset in the urdf to account for the ft sensor and the coupling plate, chaning origin form 0.1 to 0.145 for sandia, and 0.05 to 0.095 for irobot-->
   <include filename="$(find sandia_hand_description)/urdf/sandia_hand_simple_shapes.urdf.xacro" />
   <include filename="$(find handle_description)/src/irobot_hand_simple.urdf.xacro" />
 <!--  <xacro:sandia_hand side="right" parent="r_hand" reflect="1" joint_type="revolute" thumb_angle="0">-->
-<!--    <origin xyz="0 -0.1 0" rpy="-1.57079 0 -1.57079"/>-->
+<!--    <origin xyz="0 -0.145 0" rpy="-1.57079 0 -1.57079"/>-->
 <!--  </xacro:sandia_hand>-->
   <xacro:sandia_hand side="left" parent="l_hand" reflect="-1" joint_type="revolute" thumb_angle="0">
-    <origin xyz="0  0.1 0" rpy=" 1.57079 0  1.57079"/>
+    <origin xyz="0  0.145 0" rpy=" 1.57079 0  1.57079"/>
   </xacro:sandia_hand>
   <xacro:irobot_hand side="right" parent="r_hand" reflect="1">
-    <origin rpy="1.57079 0 0" xyz="0 -0.05 0"/>
+    <origin rpy="1.57079 0 0" xyz="0 -0.095 0"/>
   </xacro:irobot_hand>
 <!--  <xacro:irobot_hand side="left" parent="l_hand" reflect="-1">-->
-<!--    <origin rpy="1.57079 0 3.14159" xyz="0 0.05 0"/>-->
+<!--    <origin rpy="1.57079 0 3.14159" xyz="0 0.095 0"/>-->
 <!--  </xacro:irobot_hand>-->
 </robot>

File: software/models/mit_gazebo_models/mit_robot_drake/xacro/atlas_sandia_hands.urdf.xacro (robot description, xacro)
@@ -2,9 +2,10 @@
   <include filename="$(find mit_drcsim_scripts)/models/mit_robot_drake/xacro/atlas_skeleton_minimal_contact.urdf" />
   <include filename="$(find sandia_hand_description)/urdf/sandia_hand_simple_shapes.urdf.xacro" />
+  <!-- adding an offset in the urdf to account for the ft sensor and the coupling plate, chaning origin form 0.1 to 0.145 for sandia, and 0.05 to 0.095 for irobot-->
   <xacro:sandia_hand side="right" parent="r_hand" reflect="1" joint_type="revolute" thumb_angle="0">
-	<origin xyz="0 -0.1 0" rpy="-1.57079 0 -1.57079"/>
+	<origin xyz="0 -0.145 0" rpy="-1.57079 0 -1.57079"/>
   </xacro:sandia_hand>
   <xacro:sandia_hand side="left" parent="l_hand" reflect="-1" joint_type="revolute" thumb_angle="0">
-	<origin xyz="0  0.1 0" rpy=" 1.57079 0  1.57079"/>
+	<origin xyz="0  0.145 0" rpy=" 1.57079 0  1.57079"/>
   </xacro:sandia_hand>
   <include filename="$(find mit_drcsim_scripts)/models/mit_robot_drake/xacro/atlas.transmission" />
