Commit message: updating hpz torque limit and sandia hand mount position based on latest from osrf
git-svn-id: https://svn.csail.mit.edu/drc/trunk@6360 c7283977-0100-402a-a91a-fa70b306dbfe

File: software/models/mit_gazebo_models/mit_robot/model_LI_RI.urdf (robot description, URDF)
Before this commit: robot atlas, 70 links, 69 joints
Links:
- added link l_situational_awareness_camera_link, mass 0.1; visual box size=0.01 0.01 0.01
- added link l_situational_awareness_camera_optical_frame
- added link r_situational_awareness_camera_link, mass 0.1; visual box size=0.01 0.01 0.01
- added link r_situational_awareness_camera_optical_frame
Joints:
- added joint l_situational_awareness_camera_joint: type fixed, parent utorso, child l_situational_awareness_camera_link, origin xyz=0.216409 0.121799 0.406759 rpy=-1.57079633 0 1.30899694
- added joint l_situational_awareness_camera_optical_frame_joint: type fixed, parent l_situational_awareness_camera_link, child l_situational_awareness_camera_optical_frame, origin xyz=0 0 0 rpy=-1.5708 0.0 -1.5708
- added joint r_situational_awareness_camera_joint: type fixed, parent utorso, child r_situational_awareness_camera_link, origin xyz=0.216409 -0.121799 0.406759 rpy=1.57079633 0 -1.30899694
- added joint r_situational_awareness_camera_optical_frame_joint: type fixed, parent r_situational_awareness_camera_link, child r_situational_awareness_camera_optical_frame, origin xyz=0 0 0 rpy=-1.5708 0.0 -1.5708
- joint r_leg_hpz: limit lower=-1.22173 upper=0.174533 effort=260 velocity=12 -> lower=-1.22173 upper=0.174533 effort=110 velocity=12

File: software/models/mit_gazebo_models/mit_robot/model_LI_RS.urdf (robot description, URDF)
Before this commit: robot atlas, 94 links, 93 joints
Links:
- removed link left_base_link
- removed link left_finger[0]/base_rotation_link
- removed link left_finger[0]/distal_link
- removed link left_finger[0]/proximal_link
- removed link left_finger[1]/base_rotation_link
- removed link left_finger[1]/distal_link
- removed link left_finger[1]/proximal_link
- removed link left_finger[2]/distal_link
- removed link left_finger[2]/proximal_link
- added link l_situational_awareness_camera_link, mass 0.1; visual box size=0.01 0.01 0.01
- added link l_situational_awareness_camera_optical_frame
- added link r_situational_awareness_camera_link, mass 0.1; visual box size=0.01 0.01 0.01
- added link r_situational_awareness_camera_optical_frame
Joints:
- removed joint left_finger[0]/joint_base
- removed joint left_finger[0]/joint_base_rotation
- removed joint left_finger[0]/joint_flex
- removed joint left_finger[1]/joint_base
- removed joint left_finger[1]/joint_base_rotation
- removed joint left_finger[1]/joint_flex
- removed joint left_finger[2]/joint_base
- removed joint left_finger[2]/joint_flex
- removed joint left_irobot_hand_joint
- added joint l_situational_awareness_camera_joint: type fixed, parent utorso, child l_situational_awareness_camera_link, origin xyz=0.216409 0.121799 0.406759 rpy=-1.57079633 0 1.30899694
- added joint l_situational_awareness_camera_optical_frame_joint: type fixed, parent l_situational_awareness_camera_link, child l_situational_awareness_camera_optical_frame, origin xyz=0 0 0 rpy=-1.5708 0.0 -1.5708
- added joint r_situational_awareness_camera_joint: type fixed, parent utorso, child r_situational_awareness_camera_link, origin xyz=0.216409 -0.121799 0.406759 rpy=1.57079633 0 -1.30899694
- added joint r_situational_awareness_camera_optical_frame_joint: type fixed, parent r_situational_awareness_camera_link, child r_situational_awareness_camera_optical_frame, origin xyz=0 0 0 rpy=-1.5708 0.0 -1.5708
- joint r_leg_hpz: limit lower=-1.22173 upper=0.174533 effort=260 velocity=12 -> lower=-1.22173 upper=0.174533 effort=110 velocity=12
- joint right_sandia_hand_joint: origin xyz=0 -0.145 0 rpy=-1.57079 0 -1.57079 -> xyz=-0.00179 -0.13516 0.01176 rpy=0 0 -1.57079

File: software/models/mit_gazebo_models/mit_robot/model_LS_RI.urdf (robot description, URDF)
Before this commit: robot atlas, 94 links, 93 joints
Links:
- added link l_situational_awareness_camera_link, mass 0.1; visual box size=0.01 0.01 0.01
- added link l_situational_awareness_camera_optical_frame
- added link r_situational_awareness_camera_link, mass 0.1; visual box size=0.01 0.01 0.01
- added link r_situational_awareness_camera_optical_frame
Joints:
- added joint l_situational_awareness_camera_joint: type fixed, parent utorso, child l_situational_awareness_camera_link, origin xyz=0.216409 0.121799 0.406759 rpy=-1.57079633 0 1.30899694
- added joint l_situational_awareness_camera_optical_frame_joint: type fixed, parent l_situational_awareness_camera_link, child l_situational_awareness_camera_optical_frame, origin xyz=0 0 0 rpy=-1.5708 0.0 -1.5708
- added joint r_situational_awareness_camera_joint: type fixed, parent utorso, child r_situational_awareness_camera_link, origin xyz=0.216409 -0.121799 0.406759 rpy=1.57079633 0 -1.30899694
- added joint r_situational_awareness_camera_optical_frame_joint: type fixed, parent r_situational_awareness_camera_link, child r_situational_awareness_camera_optical_frame, origin xyz=0 0 0 rpy=-1.5708 0.0 -1.5708
- joint left_sandia_hand_joint: origin xyz=0  0.145 0 rpy= 1.57079 0  1.57079 -> xyz=0.00179  0.13516 0.01176 rpy=0 0  1.57079
- joint r_leg_hpz: limit lower=-1.22173 upper=0.174533 effort=260 velocity=12 -> lower=-1.22173 upper=0.174533 effort=110 velocity=12

File: software/models/mit_gazebo_models/mit_robot/model_LS_RS.urdf (robot description, URDF)
Before this commit: robot atlas, 118 links, 117 joints
Links:
- added link l_situational_awareness_camera_link, mass 0.1; visual box size=0.01 0.01 0.01
- added link l_situational_awareness_camera_optical_frame
- added link r_situational_awareness_camera_link, mass 0.1; visual box size=0.01 0.01 0.01
- added link r_situational_awareness_camera_optical_frame
Joints:
- added joint l_situational_awareness_camera_joint: type fixed, parent utorso, child l_situational_awareness_camera_link, origin xyz=0.216409 0.121799 0.406759 rpy=-1.57079633 0 1.30899694
- added joint l_situational_awareness_camera_optical_frame_joint: type fixed, parent l_situational_awareness_camera_link, child l_situational_awareness_camera_optical_frame, origin xyz=0 0 0 rpy=-1.5708 0.0 -1.5708
- added joint r_situational_awareness_camera_joint: type fixed, parent utorso, child r_situational_awareness_camera_link, origin xyz=0.216409 -0.121799 0.406759 rpy=1.57079633 0 -1.30899694
- added joint r_situational_awareness_camera_optical_frame_joint: type fixed, parent r_situational_awareness_camera_link, child r_situational_awareness_camera_optical_frame, origin xyz=0 0 0 rpy=-1.5708 0.0 -1.5708
- joint left_sandia_hand_joint: origin xyz=0  0.145 0 rpy=0 0  1.57079 -> xyz=0.00179  0.13516 0.01176 rpy=0 0  1.57079
- joint r_leg_hpz: limit lower=-1.22173 upper=0.174533 effort=260 velocity=12 -> lower=-1.22173 upper=0.174533 effort=110 velocity=12
- joint right_sandia_hand_joint: origin xyz=0 -0.145 0 rpy=0.0 0 -1.57079 -> xyz=-0.00179 -0.13516 0.01176 rpy=0 0 -1.57079

File: software/models/mit_gazebo_models/mit_robot/model_sim.urdf (robot description, URDF)
Before this commit: robot atlas, 107 links, 106 joints
Links:
- added link l_situational_awareness_camera_link, mass 0.1; visual box size=0.01 0.01 0.01
- added link l_situational_awareness_camera_optical_frame
- added link r_situational_awareness_camera_link, mass 0.1; visual box size=0.01 0.01 0.01
- added link r_situational_awareness_camera_optical_frame
Joints:
- added joint l_situational_awareness_camera_joint: type fixed, parent utorso, child l_situational_awareness_camera_link, origin xyz=0.216409 0.121799 0.406759 rpy=-1.57079633 0 1.30899694
- added joint l_situational_awareness_camera_optical_frame_joint: type fixed, parent l_situational_awareness_camera_link, child l_situational_awareness_camera_optical_frame, origin xyz=0 0 0 rpy=-1.5708 0.0 -1.5708
- added joint r_situational_awareness_camera_joint: type fixed, parent utorso, child r_situational_awareness_camera_link, origin xyz=0.216409 -0.121799 0.406759 rpy=1.57079633 0 -1.30899694
- added joint r_situational_awareness_camera_optical_frame_joint: type fixed, parent r_situational_awareness_camera_link, child r_situational_awareness_camera_optical_frame, origin xyz=0 0 0 rpy=-1.5708 0.0 -1.5708
- joint left_sandia_hand_joint: origin xyz=0  0.145 0 rpy=0.0 0  1.57079 -> xyz=0.00179  0.13516 0.01176 rpy=0 0  1.57079
- joint r_leg_hpz: limit lower=-1.22173 upper=0.174533 effort=260 velocity=12 -> lower=-1.22173 upper=0.174533 effort=110 velocity=12
- joint right_sandia_hand_joint: origin xyz=0 -0.145 0 rpy=0.0 0 -1.57079 -> xyz=-0.00179 -0.13516 0.01176 rpy=0 0 -1.57079

File: software/models/mit_gazebo_models/mit_robot/model_sim_gazebo.urdf (robot description, URDF)
Before this commit: robot atlas, 107 links, 106 joints
Links:
- added link l_situational_awareness_camera_link, mass 0.1; visual box size=0.01 0.01 0.01
- added link l_situational_awareness_camera_optical_frame
- added link r_situational_awareness_camera_link, mass 0.1; visual box size=0.01 0.01 0.01
- added link r_situational_awareness_camera_optical_frame
Joints:
- added joint l_situational_awareness_camera_joint: type fixed, parent utorso, child l_situational_awareness_camera_link, origin xyz=0.216409 0.121799 0.406759 rpy=-1.57079633 0 1.30899694
- added joint l_situational_awareness_camera_optical_frame_joint: type fixed, parent l_situational_awareness_camera_link, child l_situational_awareness_camera_optical_frame, origin xyz=0 0 0 rpy=-1.5708 0.0 -1.5708
- added joint r_situational_awareness_camera_joint: type fixed, parent utorso, child r_situational_awareness_camera_link, origin xyz=0.216409 -0.121799 0.406759 rpy=1.57079633 0 -1.30899694
- added joint r_situational_awareness_camera_optical_frame_joint: type fixed, parent r_situational_awareness_camera_link, child r_situational_awareness_camera_optical_frame, origin xyz=0 0 0 rpy=-1.5708 0.0 -1.5708
- joint left_sandia_hand_joint: origin xyz=0  0.145 0 rpy=0.0 0  1.57079 -> xyz=0.00179  0.13516 0.01176 rpy=0 0  1.57079
- joint r_leg_uhz: limit lower=-1.22173 upper=0.174533 effort=260 velocity=12 -> lower=-1.22173 upper=0.174533 effort=110 velocity=12
- joint right_sandia_hand_joint: origin xyz=0 -0.145 0 rpy=0.0 0 -1.57079 -> xyz=-0.00179 -0.13516 0.01176 rpy=0 0 -1.57079

File: software/models/mit_gazebo_models/mit_robot/model_stumps.urdf (robot description, URDF)
Before this commit: robot atlas, 53 links, 52 joints
Links:
- added link l_situational_awareness_camera_link, mass 0.1; visual box size=0.01 0.01 0.01
- added link l_situational_awareness_camera_optical_frame
- added link r_situational_awareness_camera_link, mass 0.1; visual box size=0.01 0.01 0.01
- added link r_situational_awareness_camera_optical_frame
Joints:
- added joint l_situational_awareness_camera_joint: type fixed, parent utorso, child l_situational_awareness_camera_link, origin xyz=0.216409 0.121799 0.406759 rpy=-1.57079633 0 1.30899694
- added joint l_situational_awareness_camera_optical_frame_joint: type fixed, parent l_situational_awareness_camera_link, child l_situational_awareness_camera_optical_frame, origin xyz=0 0 0 rpy=-1.5708 0.0 -1.5708
- added joint r_situational_awareness_camera_joint: type fixed, parent utorso, child r_situational_awareness_camera_link, origin xyz=0.216409 -0.121799 0.406759 rpy=1.57079633 0 -1.30899694
- added joint r_situational_awareness_camera_optical_frame_joint: type fixed, parent r_situational_awareness_camera_link, child r_situational_awareness_camera_optical_frame, origin xyz=0 0 0 rpy=-1.5708 0.0 -1.5708
- joint r_leg_hpz: limit lower=-1.22173 upper=0.174533 effort=260 velocity=12 -> lower=-1.22173 upper=0.174533 effort=110 velocity=12

File: software/models/mit_gazebo_models/mit_robot/xacro/atlas_irobot_left_sandia_right.urdf.xacro (robot description, xacro)
@@ -1,21 +1,12 @@
-<robot xmlns:xacro="http://playerstage.sourceforge.net/gazebo/xmlschema/#interface" name="atlas" >
+<robot xmlns:xacro="http://www.ros.org/wiki/xacro" name="atlas" >
+  <xacro:include filename="$(find sandia_hand_description)/urdf/sandia_hand_simple_shapes.urdf.xacro" />
+  <xacro:sandia_hand side="right" parent="r_hand" reflect="1" joint_type="revolute" thumb_angle="0">
+    <origin xyz="-0.00179 -0.13516 0.01176" rpy="0 0 -1.57079"/>
+  </xacro:sandia_hand>
+  <xacro:irobot_hand side="left" parent="l_hand" reflect="-1">
+    <origin rpy="1.57079 0 3.14159" xyz="0 0.095 0"/>
+  </xacro:irobot_hand>
   <include filename="$(find mit_drcsim_scripts)/models/mit_robot/xacro/atlas_skeleton.urdf" />
   <include filename="$(find mit_drcsim_scripts)/models/mit_robot/xacro/atlas.transmission" />
   <include filename="$(find mit_drcsim_scripts)/models/multisense_sl/multisense_sl.urdf" />
-  <!-- Hands -->
-  <include filename="$(find sandia_hand_description)/urdf/sandia_hand_simple_shapes.urdf.xacro" />
-  <include filename="$(find handle_description)/src/irobot_hand_simple.urdf.xacro" />
-  <!-- adding an offset in the urdf to account for the ft sensor and the coupling plate, chaning origin form 0.1 to 0.145 for sandia, and 0.05 to 0.095 for irobot-->
-  <xacro:sandia_hand side="right" parent="r_hand" reflect="1" joint_type="revolute" thumb_angle="0">
-    <origin xyz="0 -0.145 0" rpy="-1.57079 0 -1.57079"/>
-  </xacro:sandia_hand>
-<!--  <xacro:sandia_hand side="left" parent="l_hand" reflect="-1" joint_type="revolute" thumb_angle="0">-->
-<!--    <origin xyz="0  0.1 0" rpy=" 1.57079 0  1.57079"/>-->
-<!--  </xacro:sandia_hand>-->
-<!--  <xacro:irobot_hand side="right" parent="r_hand" reflect="1">-->
-<!--    <origin rpy="1.57079 0 0" xyz="0 -0.095 0"/>-->
-<!--  </xacro:irobot_hand>-->
-  <xacro:irobot_hand side="left" parent="l_hand" reflect="-1">
-    <origin rpy="1.57079 0 3.14159" xyz="0 0.095 0"/>
-  </xacro:irobot_hand>
 </robot>

File: software/models/mit_gazebo_models/mit_robot/xacro/atlas_sandia_hands.urdf.xacro (robot description, xacro)
@@ -1,15 +1,12 @@
-<robot xmlns:xacro="http://playerstage.sourceforge.net/gazebo/xmlschema/#interface" name="atlas" >
+<robot xmlns:xacro="http://www.ros.org/wiki/xacro" name="atlas" >
+  <xacro:include filename="$(find sandia_hand_description)/urdf/sandia_hand_simple_shapes.urdf.xacro" />
+  <xacro:sandia_hand side="right" parent="r_hand" reflect="1" joint_type="revolute" thumb_angle="0">
+    <origin xyz="-0.00179 -0.13516 0.01176" rpy="0 0 -1.57079"/>
+  </xacro:sandia_hand>
+  <xacro:sandia_hand side="left" parent="l_hand" reflect="-1" joint_type="revolute" thumb_angle="0">
+    <origin xyz="0.00179  0.13516 0.01176" rpy="0 0  1.57079"/>
+  </xacro:sandia_hand>
   <include filename="$(find mit_drcsim_scripts)/models/mit_robot/xacro/atlas_skeleton.urdf" />
   <include filename="$(find mit_drcsim_scripts)/models/mit_robot/xacro/atlas.transmission" />
   <include filename="$(find mit_drcsim_scripts)/models/multisense_sl/multisense_sl.urdf" />
-  <!-- Hands -->
-  <!-- NB: the Roll of the Sandia Hands is not identical in Sim and Reality -->
-   <!-- adding an offset in the urdf to account for the ft sensor and the coupling plate, chaning origin form 0.1 to 0.145 for sandia, and 0.05 to 0.095 for irobot-->
-  <include filename="$(find sandia_hand_description)/urdf/sandia_hand_simple_shapes.urdf.xacro" />
-  <xacro:sandia_hand side="right" parent="r_hand" reflect="1" joint_type="revolute" thumb_angle="0">
-    <origin xyz="0 -0.145 0" rpy="0.0 0 -1.57079"/>
-  </xacro:sandia_hand>
-  <xacro:sandia_hand side="left" parent="l_hand" reflect="-1" joint_type="revolute" thumb_angle="0">
-    <origin xyz="0  0.145 0" rpy="0 0  1.57079"/>
-  </xacro:sandia_hand>
 </robot>

File: software/models/mit_gazebo_models/mit_robot/xacro/atlas_sandia_hands_sim.urdf.xacro (robot description, xacro)
@@ -1,14 +1,11 @@
-<robot xmlns:xacro="http://playerstage.sourceforge.net/gazebo/xmlschema/#interface" name="atlas" >
-  <include filename="$(find mit_drcsim_scripts)/models/mit_robot/xacro/atlas_skeleton.urdf" />
-  <include filename="$(find sandia_hand_description)/urdf/sandia_hand_simple_shapes.urdf.xacro" />
-  <!-- Hands -->
-  <!-- NB: the Roll of the Sandia Hands is not identical in Sim and Reality -->
-   <!-- adding an offset in the urdf to account for the ft sensor and the coupling plate, chaning origin form 0.1 to 0.145 for sandia, and 0.05 to 0.095 for irobot-->
+<robot xmlns:xacro="http://www.ros.org/wiki/xacro" name="atlas" >
+  <xacro:include filename="$(find sandia_hand_description)/urdf/sandia_hand_simple_shapes.urdf.xacro" />
   <xacro:sandia_hand side="right" parent="r_hand" reflect="1" joint_type="revolute" thumb_angle="0">
-    <origin xyz="0 -0.145 0" rpy="0.0 0 -1.57079"/>
+    <origin xyz="-0.00179 -0.13516 0.01176" rpy="0 0 -1.57079"/>
   </xacro:sandia_hand>
   <xacro:sandia_hand side="left" parent="l_hand" reflect="-1" joint_type="revolute" thumb_angle="0">
-    <origin xyz="0  0.145 0" rpy="0.0 0  1.57079"/>
+    <origin xyz="0.00179  0.13516 0.01176" rpy="0 0  1.57079"/>
   </xacro:sandia_hand>
+  <include filename="$(find mit_drcsim_scripts)/models/mit_robot/xacro/atlas_skeleton.urdf" />
   <include filename="$(find mit_drcsim_scripts)/models/mit_robot/xacro/atlas.gazebo" />
   <include filename="$(find mit_drcsim_scripts)/models/mit_robot/xacro/atlas.transmission" />

File: software/models/mit_gazebo_models/mit_robot/xacro/atlas_sandia_left_irobot_right.urdf.xacro (robot description, xacro)
@@ -1,21 +1,13 @@
-<robot xmlns:xacro="http://playerstage.sourceforge.net/gazebo/xmlschema/#interface" name="atlas" >
-  <include filename="$(find mit_drcsim_scripts)/models/mit_robot/xacro/atlas_skeleton.urdf" />
-  <include filename="$(find mit_drcsim_scripts)/models/mit_robot/xacro/atlas.transmission" />
-  <include filename="$(find mit_drcsim_scripts)/models/multisense_sl/multisense_sl.urdf" />
-<!-- Hands -->
- <!-- adding an offset in the urdf to account for the ft sensor and the coupling plate, chaning origin form 0.1 to 0.145 for sandia, and 0.05 to 0.095 for irobot-->
-  <include filename="$(find sandia_hand_description)/urdf/sandia_hand_simple_shapes.urdf.xacro" />
+<robot xmlns:xacro="http://www.ros.org/wiki/xacro" name="atlas" >
+  <xacro:include filename="$(find sandia_hand_description)/urdf/sandia_hand_simple_shapes.urdf.xacro" />
   <include filename="$(find handle_description)/src/irobot_hand_simple.urdf.xacro" />
-<!--  <xacro:sandia_hand side="right" parent="r_hand" reflect="1" joint_type="revolute" thumb_angle="0">-->
-<!--    <origin xyz="0 -0.145 0" rpy="-1.57079 0 -1.57079"/>-->
-<!--  </xacro:sandia_hand>-->
   <xacro:sandia_hand side="left" parent="l_hand" reflect="-1" joint_type="revolute" thumb_angle="0">
-    <origin xyz="0  0.145 0" rpy=" 1.57079 0  1.57079"/>
+    <origin xyz="0.00179  0.13516 0.01176" rpy="0 0  1.57079"/>
   </xacro:sandia_hand>
   <xacro:irobot_hand side="right" parent="r_hand" reflect="1">
     <origin rpy="1.57079 0 0" xyz="0 -0.095 0"/>
   </xacro:irobot_hand>
-<!--  <xacro:irobot_hand side="left" parent="l_hand" reflect="-1">-->
-<!--    <origin rpy="1.57079 0 3.14159" xyz="0 0.095 0"/>-->
-<!--  </xacro:irobot_hand>-->
+  <include filename="$(find mit_drcsim_scripts)/models/mit_robot/xacro/atlas_skeleton.urdf" />
+  <include filename="$(find mit_drcsim_scripts)/models/mit_robot/xacro/atlas.transmission" />
+  <include filename="$(find mit_drcsim_scripts)/models/multisense_sl/multisense_sl.urdf" />
 </robot>

File: software/models/mit_gazebo_models/mit_robot/xacro/atlas_skeleton.urdf (robot description, URDF)
Before this commit: robot drc_skeleton, 28 links, 28 joints
Links:
- added link l_situational_awareness_camera_link, mass 0.1; visual box size=0.01 0.01 0.01
- added link l_situational_awareness_camera_optical_frame
- added link r_situational_awareness_camera_link, mass 0.1; visual box size=0.01 0.01 0.01
- added link r_situational_awareness_camera_optical_frame
Joints:
- added joint l_situational_awareness_camera_joint: type fixed, parent utorso, child l_situational_awareness_camera_link, origin xyz=0.216409 0.121799 0.406759 rpy=-1.57079633 0 1.30899694
- added joint l_situational_awareness_camera_optical_frame_joint: type fixed, parent l_situational_awareness_camera_link, child l_situational_awareness_camera_optical_frame, origin xyz=0 0 0 rpy=-1.5708 0.0 -1.5708
- added joint r_situational_awareness_camera_joint: type fixed, parent utorso, child r_situational_awareness_camera_link, origin xyz=0.216409 -0.121799 0.406759 rpy=1.57079633 0 -1.30899694
- added joint r_situational_awareness_camera_optical_frame_joint: type fixed, parent r_situational_awareness_camera_link, child r_situational_awareness_camera_optical_frame, origin xyz=0 0 0 rpy=-1.5708 0.0 -1.5708
- joint r_leg_hpz: limit lower=-1.22173 upper=0.174533 effort=260 velocity=12 -> lower=-1.22173 upper=0.174533 effort=110 velocity=12

File: software/models/mit_gazebo_models/mit_robot_drake/model.urdf (robot description, URDF)
Before this commit: robot atlas, 95 links, 94 joints
Joints:
- joint r_leg_hpz: limit lower=-1.22173 upper=0.174533 effort=260 velocity=12 -> lower=-1.22173 upper=0.174533 effort=110 velocity=12

File: software/models/mit_gazebo_models/mit_robot_drake/model_minimal_contact.urdf (robot description, URDF)
Before this commit: robot atlas, 29 links, 28 joints
Joints:
- joint r_leg_hpz: limit lower=-1.22173 upper=0.174533 effort=260 velocity=12 -> lower=-1.22173 upper=0.174533 effort=110 velocity=12

File: software/models/mit_gazebo_models/mit_robot_drake/model_minimal_contact_fixedjoint_hands.urdf (robot description, URDF)
Before this commit: robot atlas, 95 links, 94 joints
Joints:
- joint r_leg_hpz: limit lower=-1.22173 upper=0.174533 effort=260 velocity=12 -> lower=-1.22173 upper=0.174533 effort=110 velocity=12

File: software/models/mit_gazebo_models/mit_robot_drake/model_minimal_contact_point_hands.urdf (robot description, URDF)
Before this commit: robot atlas, 31 links, 30 joints
Joints:
- joint r_leg_hpz: limit lower=-1.22173 upper=0.174533 effort=260 velocity=12 -> lower=-1.22173 upper=0.174533 effort=110 velocity=12

File: software/models/mit_gazebo_models/mit_robot_drake/xacro/atlas_skeleton.urdf (robot description, URDF)
Before this commit: robot drc_skeleton, 28 links, 28 joints
Joints:
- joint r_leg_hpz: limit lower=-1.22173 upper=0.174533 effort=260 velocity=12 -> lower=-1.22173 upper=0.174533 effort=110 velocity=12

File: software/models/mit_gazebo_models/mit_robot_drake/xacro/atlas_skeleton_minimal_contact.urdf (robot description, URDF)
Before this commit: robot drc_skeleton, 28 links, 28 joints
Joints:
- joint r_leg_hpz: limit lower=-1.22173 upper=0.174533 effort=260 velocity=12 -> lower=-1.22173 upper=0.174533 effort=110 velocity=12
