Commit message: adjusted irobot hand offset according to updates from OSRF: todo check on real robot
git-svn-id: https://svn.csail.mit.edu/drc/trunk@6369 c7283977-0100-402a-a91a-fa70b306dbfe

File: software/models/mit_gazebo_models/mit_robot/model_LI_RI.urdf (robot description, URDF)
Before this commit: robot atlas, 74 links, 73 joints
Joints:
- joint left_irobot_hand_joint: origin xyz=0 0.095 0 rpy=1.57079 0 3.14159 -> xyz=0 0.08516 0 rpy=1.57079 0 3.14159
- joint right_irobot_hand_joint: origin xyz=0 -0.095 0 rpy=1.57079 0 0 -> xyz=0 -0.08516 0 rpy=1.57079 0 0

File: software/models/mit_gazebo_models/mit_robot/model_LS_RI.urdf (robot description, URDF)
Before this commit: robot atlas, 98 links, 97 joints
Joints:
- joint right_irobot_hand_joint: origin xyz=0 -0.095 0 rpy=1.57079 0 0 -> xyz=0 -0.08516 0 rpy=1.57079 0 0

File: software/models/mit_gazebo_models/mit_robot/xacro/atlas_irobot_hands.urdf.xacro (robot description, xacro)
@@ -3,12 +3,19 @@
   <include filename="$(find mit_drcsim_scripts)/models/mit_robot/xacro/atlas.transmission" />
   <include filename="$(find mit_drcsim_scripts)/models/multisense_sl/multisense_sl.urdf" />
-  <!-- Hands -->
-  <!-- adding an offset in the urdf to account for the ft sensor and the coupling plate, chaning origin form 0.1 to 0.145 for sandia, and 0.05 to 0.095 for irobot-->
+<!--
+05 sept: Sisir added an offset of 0.045 in the urdf to account
+for the force sensor and the coupling plate, changing
+origin from 0.1 to 0.145 for sandia, and 0.05 to 0.095 for irobot
+26 sept: instead OSRF added an offset of 0.03516.
+mfallon made this adjustment:
+0.05 + 0.03516 = 0.08516
+0.1  + 0.03516 = 0.13516
+-->
   <include filename="$(find handle_description)/src/irobot_hand_simple.urdf.xacro" />
   <xacro:irobot_hand side="right" parent="r_hand" reflect="1">
-    <origin rpy="1.57079 0 0" xyz="0 -0.095 0"/>
+    <origin rpy="1.57079 0 0" xyz="0 -0.08516 0"/>
   </xacro:irobot_hand>
   <xacro:irobot_hand side="left" parent="l_hand" reflect="-1">
-    <origin rpy="1.57079 0 3.14159" xyz="0 0.095 0"/>
+    <origin rpy="1.57079 0 3.14159" xyz="0 0.08516 0"/>
   </xacro:irobot_hand>
 </robot>

File: software/models/mit_gazebo_models/mit_robot/xacro/atlas_irobot_left_sandia_right.urdf.xacro (robot description, xacro)
@@ -5,5 +5,5 @@
   </xacro:sandia_hand>
   <xacro:irobot_hand side="left" parent="l_hand" reflect="-1">
-    <origin rpy="1.57079 0 3.14159" xyz="0 0.095 0"/>
+    <origin rpy="1.57079 0 3.14159" xyz="0 0.08516 0"/>
   </xacro:irobot_hand>
   <include filename="$(find mit_drcsim_scripts)/models/mit_robot/xacro/atlas_skeleton.urdf" />

File: software/models/mit_gazebo_models/mit_robot/xacro/atlas_sandia_left_irobot_right.urdf.xacro (robot description, xacro)
@@ -6,5 +6,5 @@
   </xacro:sandia_hand>
   <xacro:irobot_hand side="right" parent="r_hand" reflect="1">
-    <origin rpy="1.57079 0 0" xyz="0 -0.095 0"/>
+    <origin rpy="1.57079 0 0" xyz="0 -0.08516 0"/>
   </xacro:irobot_hand>
   <include filename="$(find mit_drcsim_scripts)/models/mit_robot/xacro/atlas_skeleton.urdf" />

Commit message: adding stump and sandia combos
git-svn-id: https://svn.csail.mit.edu/drc/trunk@6720 c7283977-0100-402a-a91a-fa70b306dbfe

File: software/models/mit_gazebo_models/mit_robot/model_LI_RI.urdf (robot description, URDF)
Before this commit: robot atlas, 74 links, 73 joints
Joints:
- joint left_irobot_hand_joint: origin xyz=0 0.08516 0 rpy=1.57079 0 3.14159 -> xyz=0 0.11516 0 rpy=1.57079 3.14159 3.14159

File: software/models/mit_gazebo_models/mit_robot/model_LI_RS.urdf (robot description, URDF)
Before this commit: robot atlas, 89 links, 88 joints
Links:
- added link left_base_link, mass 0.1; collision mesh filename=package://handle_description/meshes/palm.stl; visual mesh filename=package://handle_description/meshes/palm.stl
- added link left_finger[0]/base_rotation_link, mass 0.1; collision mesh filename=package://handle_description/meshes/finger_base.stl; visual mesh filename=package://handle_description/meshes/finger_base.stl
- added link left_finger[0]/distal_link, mass 0.1; collision mesh filename=package://handle_description/meshes/finger_distal.stl; visual mesh filename=package://handle_description/meshes/finger_distal.stl
- added link left_finger[0]/proximal_link, mass 0.1; collision mesh filename=package://handle_description/meshes/finger_proximal.stl; visual mesh filename=package://handle_description/meshes/finger_proximal.stl
- added link left_finger[1]/base_rotation_link, mass 0.1; collision mesh filename=package://handle_description/meshes/finger_base.stl; visual mesh filename=package://handle_description/meshes/finger_base.stl
- added link left_finger[1]/distal_link, mass 0.1; collision mesh filename=package://handle_description/meshes/finger_distal.stl; visual mesh filename=package://handle_description/meshes/finger_distal.stl
- added link left_finger[1]/proximal_link, mass 0.1; collision mesh filename=package://handle_description/meshes/finger_proximal.stl; visual mesh filename=package://handle_description/meshes/finger_proximal.stl
- added link left_finger[2]/distal_link, mass 0.1; collision mesh filename=package://handle_description/meshes/finger_distal.stl; visual mesh filename=package://handle_description/meshes/finger_distal.stl
- added link left_finger[2]/proximal_link, mass 0.1; collision mesh filename=package://handle_description/meshes/finger_proximal.stl; visual mesh filename=package://handle_description/meshes/finger_proximal.stl
Joints:
- added joint left_finger[0]/joint_base: type revolute, parent left_finger[0]/base_rotation_link, child left_finger[0]/proximal_link, origin xyz=0 0 0.0135 rpy=1.57 0 -3.14, axis -1 0 0, limit lower=0.0 upper=1.57 effort=1000.0 velocity=0.5
- added joint left_finger[0]/joint_base_rotation: type revolute, parent left_base_link, child left_finger[0]/base_rotation_link, origin xyz=0.03075 0.038 0.069477 rpy=0 0 0, axis 0 0 -1, limit lower=0.0 upper=1.57 effort=1000.0 velocity=0.5
- added joint left_finger[0]/joint_flex: type revolute, parent left_finger[0]/proximal_link, child left_finger[0]/distal_link, origin xyz=0 0 0.078, axis -1 0 0, limit lower=0.0 upper=1.57 effort=1000.0 velocity=0.5
- added joint left_finger[1]/joint_base: type revolute, parent left_finger[1]/base_rotation_link, child left_finger[1]/proximal_link, origin xyz=0 0 0.0135 rpy=1.57 0 -3.14, axis -1 0 0, limit lower=0.0 upper=1.57 effort=1000.0 velocity=0.5
- added joint left_finger[1]/joint_base_rotation: type revolute, parent left_base_link, child left_finger[1]/base_rotation_link, origin xyz=-0.03075 0.038 0.069477 rpy=0 0 0, axis 0 0 1, limit lower=0.0 upper=1.57 effort=1000.0 velocity=0.5
- added joint left_finger[1]/joint_flex: type revolute, parent left_finger[1]/proximal_link, child left_finger[1]/distal_link, origin xyz=0 0 0.078, axis -1 0 0, limit lower=0.0 upper=1.57 effort=1000.0 velocity=0.5
- added joint left_finger[2]/joint_base: type revolute, parent left_base_link, child left_finger[2]/proximal_link, origin xyz=0 -0.038 0.082755 rpy=1.57 0 0, axis -1 0 0, limit lower=0.0 upper=1.57 effort=1000.0 velocity=0.5
- added joint left_finger[2]/joint_flex: type revolute, parent left_finger[2]/proximal_link, child left_finger[2]/distal_link, origin xyz=0 0 0.078, axis -1 0 0, limit lower=0.0 upper=1.57 effort=1000.0 velocity=0.5
- added joint left_irobot_hand_joint: type fixed, parent l_hand, child left_base_link, origin xyz=0 0.11516 0 rpy=1.57079 3.14159 3.14159

Commit message: correcting irobot offset
git-svn-id: https://svn.csail.mit.edu/drc/trunk@6738 c7283977-0100-402a-a91a-fa70b306dbfe

File: software/models/mit_gazebo_models/mit_robot/model_LI_RI.urdf (robot description, URDF)
Before this commit: robot atlas, 74 links, 73 joints
Joints:
- joint right_irobot_hand_joint: origin xyz=0 -0.08516 0 rpy=1.57079 0 0 -> xyz=0 -0.11516 0 rpy=1.57079 0 0

File: software/models/mit_gazebo_models/mit_robot/model_LS_RI.urdf (robot description, URDF)
Before this commit: robot atlas, 98 links, 97 joints
Joints:
- joint right_irobot_hand_joint: origin xyz=0 -0.08516 0 rpy=1.57079 0 0 -> xyz=0 -0.11516 0 rpy=1.57079 0 0

File: software/models/mit_gazebo_models/mit_robot/xacro/atlas_irobot_hands.urdf.xacro (robot description, xacro)
@@ -5,5 +5,5 @@
   <xacro:include filename="$(find handle_description)/src/irobot_hand_simple.urdf.xacro" />
   <xacro:irobot_hand side="right" parent="r_hand" reflect="1">
-    <origin rpy="1.57079 0 0" xyz="0 -0.08516 0"/>
+    <origin rpy="1.57079 0 0" xyz="0 -0.11516 0"/>
   </xacro:irobot_hand>
   <xacro:irobot_hand side="left" parent="l_hand" reflect="-1">
@@ -20,5 +20,6 @@
 27 sept: mfallon tested with the left irobot hand on the robot and found
 significant errors in yaw and y. fixed them as best as I could (3-4cm)
-needs to be improved further
+needs to be improved further.
+New y seperation: 0 0.11516
 -->
 </robot>

File: software/models/mit_gazebo_models/mit_robot/xacro/atlas_sandia_left_irobot_right.urdf.xacro (robot description, xacro)
@@ -6,5 +6,5 @@
   </xacro:sandia_hand>
   <xacro:irobot_hand side="right" parent="r_hand" reflect="1">
-    <origin rpy="1.57079 0 0" xyz="0 -0.08516 0"/>
+    <origin rpy="1.57079 0 0" xyz="0 -0.11516 0"/>
   </xacro:irobot_hand>
   <include filename="$(find mit_drcsim_scripts)/models/mit_robot/xacro/atlas_skeleton.urdf" />
