Commit message: updating arm joint torque limits from BDI's spec. these are asymmetric, but I've just taken the smaller value for each joint
git-svn-id: https://svn.csail.mit.edu/drc/trunk@6741 c7283977-0100-402a-a91a-fa70b306dbfe

File: software/models/mit_gazebo_models/mit_robot_drake/model_minimal_contact_point_hands.urdf (robot description, URDF)
Before this commit: robot atlas, 31 links, 30 joints
Joints:
- joint l_arm_elx: limit lower=0 upper=2.35619 effort=114 velocity=12 -> lower=0 upper=2.35619 effort=55 velocity=12
- joint l_arm_ely: limit lower=0 upper=3.14159 effort=114 velocity=12 -> lower=0 upper=3.14159 effort=55 velocity=12
- joint l_arm_mwx: limit lower=-1.1781 upper=1.1781 effort=60 velocity=12 -> lower=-1.1781 upper=1.1781 effort=55 velocity=12
- joint l_arm_shx: limit lower=-1.5708 upper=1.5708 effort=170 velocity=12 -> lower=-1.5708 upper=1.5708 effort=107 velocity=12
- joint l_arm_usy: limit lower=-1.5708 upper=0.785398 effort=212 velocity=12 -> lower=-1.5708 upper=0.785398 effort=75 velocity=12
- joint l_arm_uwy: limit lower=0 upper=3.14159 effort=114 velocity=12 -> lower=0 upper=3.14159 effort=55 velocity=12
- joint r_arm_elx: limit lower=-2.35619 upper=0 effort=114 velocity=12 -> lower=-2.35619 upper=0 effort=55 velocity=12
- joint r_arm_ely: limit lower=0 upper=3.14159 effort=114 velocity=12 -> lower=0 upper=3.14159 effort=55 velocity=12
- joint r_arm_mwx: limit lower=-1.1781 upper=1.1781 effort=60 velocity=12 -> lower=-1.1781 upper=1.1781 effort=55 velocity=12
- joint r_arm_shx: limit lower=-1.5708 upper=1.5708 effort=170 velocity=12 -> lower=-1.5708 upper=1.5708 effort=107 velocity=12
- joint r_arm_usy: limit lower=-1.5708 upper=0.785398 effort=212 velocity=12 -> lower=-1.5708 upper=0.785398 effort=75 velocity=12
- joint r_arm_uwy: limit lower=0 upper=3.14159 effort=114 velocity=12 -> lower=0 upper=3.14159 effort=55 velocity=12

File: software/models/mit_gazebo_models/mit_robot_drake/model_minimal_contact_point_stumps.urdf (robot description, URDF)
Before this commit: robot atlas, 31 links, 30 joints
Joints:
- joint l_arm_elx: limit lower=0 upper=2.35619 effort=114 velocity=12 -> lower=0 upper=2.35619 effort=55 velocity=12
- joint l_arm_ely: limit lower=0 upper=3.14159 effort=114 velocity=12 -> lower=0 upper=3.14159 effort=55 velocity=12
- joint l_arm_mwx: limit lower=-1.1781 upper=1.1781 effort=60 velocity=12 -> lower=-1.1781 upper=1.1781 effort=55 velocity=12
- joint l_arm_shx: limit lower=-1.5708 upper=1.5708 effort=170 velocity=12 -> lower=-1.5708 upper=1.5708 effort=107 velocity=12
- joint l_arm_usy: limit lower=-1.5708 upper=0.785398 effort=212 velocity=12 -> lower=-1.5708 upper=0.785398 effort=75 velocity=12
- joint l_arm_uwy: limit lower=0 upper=3.14159 effort=114 velocity=12 -> lower=0 upper=3.14159 effort=55 velocity=12
- joint r_arm_elx: limit lower=-2.35619 upper=0 effort=114 velocity=12 -> lower=-2.35619 upper=0 effort=55 velocity=12
- joint r_arm_ely: limit lower=0 upper=3.14159 effort=114 velocity=12 -> lower=0 upper=3.14159 effort=55 velocity=12
- joint r_arm_mwx: limit lower=-1.1781 upper=1.1781 effort=60 velocity=12 -> lower=-1.1781 upper=1.1781 effort=55 velocity=12
- joint r_arm_shx: limit lower=-1.5708 upper=1.5708 effort=170 velocity=12 -> lower=-1.5708 upper=1.5708 effort=107 velocity=12
- joint r_arm_usy: limit lower=-1.5708 upper=0.785398 effort=212 velocity=12 -> lower=-1.5708 upper=0.785398 effort=75 velocity=12
- joint r_arm_uwy: limit lower=0 upper=3.14159 effort=114 velocity=12 -> lower=0 upper=3.14159 effort=55 velocity=12

File: software/models/mit_gazebo_models/mit_robot_drake/model_right_sandia_hand.urdf (robot description, URDF)
Before this commit: robot atlas, 62 links, 61 joints
Joints:
- joint l_arm_elx: limit lower=0 upper=2.35619 effort=114 velocity=12 -> lower=0 upper=2.35619 effort=55 velocity=12
- joint l_arm_ely: limit lower=0 upper=3.14159 effort=114 velocity=12 -> lower=0 upper=3.14159 effort=55 velocity=12
- joint l_arm_mwx: limit lower=-1.1781 upper=1.1781 effort=60 velocity=12 -> lower=-1.1781 upper=1.1781 effort=55 velocity=12
- joint l_arm_shx: limit lower=-1.5708 upper=1.5708 effort=170 velocity=12 -> lower=-1.5708 upper=1.5708 effort=107 velocity=12
- joint l_arm_usy: limit lower=-1.5708 upper=0.785398 effort=212 velocity=12 -> lower=-1.5708 upper=0.785398 effort=75 velocity=12
- joint l_arm_uwy: limit lower=0 upper=3.14159 effort=114 velocity=12 -> lower=0 upper=3.14159 effort=55 velocity=12
- joint r_arm_elx: limit lower=-2.35619 upper=0 effort=114 velocity=12 -> lower=-2.35619 upper=0 effort=55 velocity=12
- joint r_arm_ely: limit lower=0 upper=3.14159 effort=114 velocity=12 -> lower=0 upper=3.14159 effort=55 velocity=12
- joint r_arm_mwx: limit lower=-1.1781 upper=1.1781 effort=60 velocity=12 -> lower=-1.1781 upper=1.1781 effort=55 velocity=12
- joint r_arm_shx: limit lower=-1.5708 upper=1.5708 effort=170 velocity=12 -> lower=-1.5708 upper=1.5708 effort=107 velocity=12
- joint r_arm_usy: limit lower=-1.5708 upper=0.785398 effort=212 velocity=12 -> lower=-1.5708 upper=0.785398 effort=75 velocity=12
- joint r_arm_uwy: limit lower=0 upper=3.14159 effort=114 velocity=12 -> lower=0 upper=3.14159 effort=55 velocity=12

File: software/models/mit_gazebo_models/mit_robot_drake/xacro/atlas_skeleton.urdf (robot description, URDF)
Before this commit: robot drc_skeleton, 28 links, 28 joints
Joints:
- joint l_arm_elx: limit lower=0 upper=2.35619 effort=114 velocity=12 -> lower=0 upper=2.35619 effort=55 velocity=12
- joint l_arm_ely: limit lower=0 upper=3.14159 effort=114 velocity=12 -> lower=0 upper=3.14159 effort=55 velocity=12
- joint l_arm_mwx: limit lower=-1.1781 upper=1.1781 effort=60 velocity=12 -> lower=-1.1781 upper=1.1781 effort=55 velocity=12
- joint l_arm_shx: limit lower=-1.5708 upper=1.5708 effort=170 velocity=12 -> lower=-1.5708 upper=1.5708 effort=107 velocity=12
- joint l_arm_usy: limit lower=-1.5708 upper=0.785398 effort=212 velocity=12 -> lower=-1.5708 upper=0.785398 effort=75 velocity=12
- joint l_arm_uwy: limit lower=0 upper=3.14159 effort=114 velocity=12 -> lower=0 upper=3.14159 effort=55 velocity=12
- joint r_arm_elx: limit lower=-2.35619 upper=0 effort=114 velocity=12 -> lower=-2.35619 upper=0 effort=55 velocity=12
- joint r_arm_ely: limit lower=0 upper=3.14159 effort=114 velocity=12 -> lower=0 upper=3.14159 effort=55 velocity=12
- joint r_arm_mwx: limit lower=-1.1781 upper=1.1781 effort=60 velocity=12 -> lower=-1.1781 upper=1.1781 effort=55 velocity=12
- joint r_arm_shx: limit lower=-1.5708 upper=1.5708 effort=170 velocity=12 -> lower=-1.5708 upper=1.5708 effort=107 velocity=12
- joint r_arm_usy: limit lower=-1.5708 upper=0.785398 effort=212 velocity=12 -> lower=-1.5708 upper=0.785398 effort=75 velocity=12
- joint r_arm_uwy: limit lower=0 upper=3.14159 effort=114 velocity=12 -> lower=0 upper=3.14159 effort=55 velocity=12

File: software/models/mit_gazebo_models/mit_robot_drake/xacro/atlas_skeleton_minimal_contact.urdf (robot description, URDF)
Before this commit: robot drc_skeleton, 28 links, 28 joints
Joints:
- joint l_arm_elx: limit lower=0 upper=2.35619 effort=114 velocity=12 -> lower=0 upper=2.35619 effort=55 velocity=12
- joint l_arm_ely: limit lower=0 upper=3.14159 effort=114 velocity=12 -> lower=0 upper=3.14159 effort=55 velocity=12
- joint l_arm_mwx: limit lower=-1.1781 upper=1.1781 effort=60 velocity=12 -> lower=-1.1781 upper=1.1781 effort=55 velocity=12
- joint l_arm_shx: limit lower=-1.5708 upper=1.5708 effort=170 velocity=12 -> lower=-1.5708 upper=1.5708 effort=107 velocity=12
- joint l_arm_usy: limit lower=-1.5708 upper=0.785398 effort=212 velocity=12 -> lower=-1.5708 upper=0.785398 effort=75 velocity=12
- joint l_arm_uwy: limit lower=0 upper=3.14159 effort=114 velocity=12 -> lower=0 upper=3.14159 effort=55 velocity=12
- joint r_arm_elx: limit lower=-2.35619 upper=0 effort=114 velocity=12 -> lower=-2.35619 upper=0 effort=55 velocity=12
- joint r_arm_ely: limit lower=0 upper=3.14159 effort=114 velocity=12 -> lower=0 upper=3.14159 effort=55 velocity=12
- joint r_arm_mwx: limit lower=-1.1781 upper=1.1781 effort=60 velocity=12 -> lower=-1.1781 upper=1.1781 effort=55 velocity=12
- joint r_arm_shx: limit lower=-1.5708 upper=1.5708 effort=170 velocity=12 -> lower=-1.5708 upper=1.5708 effort=107 velocity=12
- joint r_arm_usy: limit lower=-1.5708 upper=0.785398 effort=212 velocity=12 -> lower=-1.5708 upper=0.785398 effort=75 velocity=12
- joint r_arm_uwy: limit lower=0 upper=3.14159 effort=114 velocity=12 -> lower=0 upper=3.14159 effort=55 velocity=12

Commit message: corrected irobot hand positions, now happy that they are correct - except possibly the extension dimension of the palm to hand
git-svn-id: https://svn.csail.mit.edu/drc/trunk@6743 c7283977-0100-402a-a91a-fa70b306dbfe

File: software/models/mit_gazebo_models/mit_robot/model_LI_RI.urdf (robot description, URDF)
Before this commit: robot atlas, 74 links, 73 joints
Joints:
- joint left_irobot_hand_joint: origin xyz=0 0.11516 0 rpy=1.57079 3.14159 3.14159 -> xyz=0 0.11516 0.015 rpy=1.57079 3.14159 3.14159
- joint right_irobot_hand_joint: origin xyz=0 -0.11516 0 rpy=1.57079 0 0 -> xyz=0 -0.11516 -0.015 rpy=1.57079 0 0

File: software/models/mit_gazebo_models/mit_robot/model_LI_RS.urdf (robot description, URDF)
Before this commit: robot atlas, 98 links, 97 joints
Joints:
- joint left_irobot_hand_joint: origin xyz=0 0.11516 0 rpy=1.57079 3.14159 3.14159 -> xyz=0 0.11516 0.015 rpy=1.57079 3.14159 3.14159

File: software/models/mit_gazebo_models/mit_robot/model_LS_RI.urdf (robot description, URDF)
Before this commit: robot atlas, 98 links, 97 joints
Joints:
- joint right_irobot_hand_joint: origin xyz=0 -0.11516 0 rpy=1.57079 0 0 -> xyz=0 -0.11516 -0.015 rpy=1.57079 0 0

File: software/models/mit_gazebo_models/mit_robot/xacro/atlas_irobot_hands.urdf.xacro (robot description, xacro)
@@ -5,8 +5,8 @@
   <xacro:include filename="$(find handle_description)/src/irobot_hand_simple.urdf.xacro" />
   <xacro:irobot_hand side="right" parent="r_hand" reflect="1">
-    <origin rpy="1.57079 0 0" xyz="0 -0.11516 0"/>
+    <origin rpy="1.57079 0 0" xyz="0 -0.11516 -0.015"/>
   </xacro:irobot_hand>
   <xacro:irobot_hand side="left" parent="l_hand" reflect="-1">
-    <origin rpy="1.57079 3.14159 3.14159" xyz="0 0.11516 0"/>
+    <origin rpy="1.57079 3.14159 3.14159" xyz="0 0.11516 0.015"/>
   </xacro:irobot_hand>
 <!--
@@ -22,4 +22,7 @@
 needs to be improved further.
 New y seperation: 0 0.11516
+24 oct: mfallon:
+set z=0.015 as the irobot hand center is clearly aligned with the force torque
+still think that y seperaton could be improved
 -->
 </robot>

File: software/models/mit_gazebo_models/mit_robot/xacro/atlas_irobot_left_sandia_right.urdf.xacro (robot description, xacro)
@@ -6,5 +6,5 @@
   </xacro:sandia_hand>
   <xacro:irobot_hand side="left" parent="l_hand" reflect="-1">
-    <origin rpy="1.57079 3.14159 3.14159" xyz="0 0.11516 0"/>
+    <origin rpy="1.57079 3.14159 3.14159" xyz="0 0.11516 0.015"/>
   </xacro:irobot_hand>
   <include filename="$(find mit_drcsim_scripts)/models/mit_robot/xacro/atlas_skeleton.urdf" />

File: software/models/mit_gazebo_models/mit_robot/xacro/atlas_sandia_left_irobot_right.urdf.xacro (robot description, xacro)
@@ -6,5 +6,5 @@
   </xacro:sandia_hand>
   <xacro:irobot_hand side="right" parent="r_hand" reflect="1">
-    <origin rpy="1.57079 0 0" xyz="0 -0.11516 0"/>
+    <origin rpy="1.57079 0 0" xyz="0 -0.11516 -0.015"/>
   </xacro:irobot_hand>
   <include filename="$(find mit_drcsim_scripts)/models/mit_robot/xacro/atlas_skeleton.urdf" />

Commit message: removed friction from gazebo model to make simulation stable again
git-svn-id: https://svn.csail.mit.edu/drc/trunk@6782 c7283977-0100-402a-a91a-fa70b306dbfe

File: software/models/mit_gazebo_models/mit_robot/model_LI_RI.urdf (robot description, URDF)
Before this commit: robot atlas, 74 links, 73 joints
Joints:
- joint back_bkz: limit lower=-0.663225 upper=0.663225 effort=124.016 velocity=12 -> lower=-0.663225 upper=0.663225 effort=114 velocity=12
- joint r_leg_kny: limit lower=0 upper=2.38569 effort=220 velocity=11 -> lower=0 upper=2.38569 effort=220 velocity=12

File: software/models/mit_gazebo_models/mit_robot/model_LI_RS.urdf (robot description, URDF)
Before this commit: robot atlas, 98 links, 97 joints
Joints:
- joint back_bkz: limit lower=-0.663225 upper=0.663225 effort=124.016 velocity=12 -> lower=-0.663225 upper=0.663225 effort=114 velocity=12
- joint r_leg_kny: limit lower=0 upper=2.38569 effort=220 velocity=11 -> lower=0 upper=2.38569 effort=220 velocity=12

File: software/models/mit_gazebo_models/mit_robot/model_LN_RS.urdf (robot description, URDF)
Before this commit: robot atlas, 89 links, 88 joints
Joints:
- joint back_bkz: limit lower=-0.663225 upper=0.663225 effort=124.016 velocity=12 -> lower=-0.663225 upper=0.663225 effort=114 velocity=12
- joint r_leg_kny: limit lower=0 upper=2.38569 effort=220 velocity=11 -> lower=0 upper=2.38569 effort=220 velocity=12

File: software/models/mit_gazebo_models/mit_robot/model_LS_RI.urdf (robot description, URDF)
Before this commit: robot atlas, 98 links, 97 joints
Joints:
- joint back_bkz: limit lower=-0.663225 upper=0.663225 effort=124.016 velocity=12 -> lower=-0.663225 upper=0.663225 effort=114 velocity=12
- joint r_leg_kny: limit lower=0 upper=2.38569 effort=220 velocity=11 -> lower=0 upper=2.38569 effort=220 velocity=12

File: software/models/mit_gazebo_models/mit_robot/model_LS_RN.urdf (robot description, URDF)
Before this commit: robot atlas, 89 links, 88 joints
Joints:
- joint back_bkz: limit lower=-0.663225 upper=0.663225 effort=124.016 velocity=12 -> lower=-0.663225 upper=0.663225 effort=114 velocity=12
- joint r_leg_kny: limit lower=0 upper=2.38569 effort=220 velocity=11 -> lower=0 upper=2.38569 effort=220 velocity=12

File: software/models/mit_gazebo_models/mit_robot/model_LS_RS.urdf (robot description, URDF)
Before this commit: robot atlas, 122 links, 121 joints
Joints:
- joint back_bkz: limit lower=-0.663225 upper=0.663225 effort=124.016 velocity=12 -> lower=-0.663225 upper=0.663225 effort=114 velocity=12
- joint r_leg_kny: limit lower=0 upper=2.38569 effort=220 velocity=11 -> lower=0 upper=2.38569 effort=220 velocity=12

File: software/models/mit_gazebo_models/mit_robot/model_sim.urdf (robot description, URDF)
Before this commit: robot atlas, 111 links, 110 joints
Joints:
- joint back_bkz: limit lower=-0.663225 upper=0.663225 effort=124.016 velocity=12 -> lower=-0.663225 upper=0.663225 effort=114 velocity=12
- joint r_leg_kny: limit lower=0 upper=2.38569 effort=220 velocity=11 -> lower=0 upper=2.38569 effort=220 velocity=12

File: software/models/mit_gazebo_models/mit_robot/model_sim_gazebo.urdf (robot description, URDF)
Before this commit: robot atlas, 111 links, 110 joints
Joints:
- joint back_lbz: limit lower=-0.663225 upper=0.663225 effort=124.016 velocity=12 -> lower=-0.663225 upper=0.663225 effort=114 velocity=12
- joint r_leg_kny: limit lower=0 upper=2.38569 effort=220 velocity=11 -> lower=0 upper=2.38569 effort=220 velocity=12

File: software/models/mit_gazebo_models/mit_robot/model_stumps.urdf (robot description, URDF)
Before this commit: robot atlas, 57 links, 56 joints
Joints:
- joint back_bkz: limit lower=-0.663225 upper=0.663225 effort=124.016 velocity=12 -> lower=-0.663225 upper=0.663225 effort=114 velocity=12
- joint r_leg_kny: limit lower=0 upper=2.38569 effort=220 velocity=11 -> lower=0 upper=2.38569 effort=220 velocity=12

File: software/models/mit_gazebo_models/mit_robot/xacro/atlas_skeleton.urdf (robot description, URDF)
Before this commit: robot drc_skeleton, 32 links, 32 joints
Joints:
- joint back_bkz: limit lower=-0.663225 upper=0.663225 effort=124.016 velocity=12 -> lower=-0.663225 upper=0.663225 effort=114 velocity=12
- joint r_leg_kny: limit lower=0 upper=2.38569 effort=220 velocity=11 -> lower=0 upper=2.38569 effort=220 velocity=12

File: software/models/mit_gazebo_models/mit_robot_drake/model.urdf (robot description, URDF)
Before this commit: robot atlas, 95 links, 94 joints
Joints:
- joint back_bkz: limit lower=-0.663225 upper=0.663225 effort=124.016 velocity=12 -> lower=-0.663225 upper=0.663225 effort=114 velocity=12

File: software/models/mit_gazebo_models/mit_robot_drake/model_minimal_contact.urdf (robot description, URDF)
Before this commit: robot atlas, 29 links, 28 joints
Joints:
- joint back_bkz: limit lower=-0.663225 upper=0.663225 effort=124.016 velocity=12 -> lower=-0.663225 upper=0.663225 effort=114 velocity=12

File: software/models/mit_gazebo_models/mit_robot_drake/model_minimal_contact_fixedjoint_hands.urdf (robot description, URDF)
Before this commit: robot atlas, 95 links, 94 joints
Joints:
- joint back_bkz: limit lower=-0.663225 upper=0.663225 effort=124.016 velocity=12 -> lower=-0.663225 upper=0.663225 effort=114 velocity=12

File: software/models/mit_gazebo_models/mit_robot_drake/model_minimal_contact_point_hands.urdf (robot description, URDF)
Before this commit: robot atlas, 31 links, 30 joints
Joints:
- joint back_bkz: limit lower=-0.663225 upper=0.663225 effort=124.016 velocity=12 -> lower=-0.663225 upper=0.663225 effort=114 velocity=12

File: software/models/mit_gazebo_models/mit_robot_drake/model_minimal_contact_point_stumps.urdf (robot description, URDF)
Before this commit: robot atlas, 31 links, 30 joints
Joints:
- joint back_bkz: limit lower=-0.663225 upper=0.663225 effort=124.016 velocity=12 -> lower=-0.663225 upper=0.663225 effort=114 velocity=12

File: software/models/mit_gazebo_models/mit_robot_drake/model_right_sandia_hand.urdf (robot description, URDF)
Before this commit: robot atlas, 62 links, 61 joints
Joints:
- joint back_bkz: limit lower=-0.663225 upper=0.663225 effort=124.016 velocity=12 -> lower=-0.663225 upper=0.663225 effort=114 velocity=12

File: software/models/mit_gazebo_models/mit_robot_drake/xacro/atlas_skeleton.urdf (robot description, URDF)
Before this commit: robot drc_skeleton, 28 links, 28 joints
Joints:
- joint back_bkz: limit lower=-0.663225 upper=0.663225 effort=124.016 velocity=12 -> lower=-0.663225 upper=0.663225 effort=114 velocity=12

File: software/models/mit_gazebo_models/mit_robot_drake/xacro/atlas_skeleton_minimal_contact.urdf (robot description, URDF)
Before this commit: robot drc_skeleton, 28 links, 28 joints
Joints:
- joint back_bkz: limit lower=-0.663225 upper=0.663225 effort=124.016 velocity=12 -> lower=-0.663225 upper=0.663225 effort=114 velocity=12
