Commit message: git-svn-id: https://svn.csail.mit.edu/drc/trunk@6893 c7283977-0100-402a-a91a-fa70b306dbfe

File: software/models/mit_gazebo_models/mit_robot/model_LI_RN.urdf (robot description, URDF)
Before this commit: robot atlas, 57 links, 56 joints
Links:
- removed link imu_link
- added link left_base_link, mass 0.1; collision mesh filename=package://handle_description/meshes/palm.stl; visual mesh filename=package://handle_description/meshes/palm.stl
- added link left_finger[0]/base_rotation_link, mass 0.1; collision mesh filename=package://handle_description/meshes/finger_base.stl; visual mesh filename=package://handle_description/meshes/finger_base.stl
- added link left_finger[0]/distal_link, mass 0.1; collision mesh filename=package://handle_description/meshes/finger_distal.stl; visual mesh filename=package://handle_description/meshes/finger_distal.stl
- added link left_finger[0]/proximal_link, mass 0.1; collision mesh filename=package://handle_description/meshes/finger_proximal.stl; visual mesh filename=package://handle_description/meshes/finger_proximal.stl
- added link left_finger[1]/base_rotation_link, mass 0.1; collision mesh filename=package://handle_description/meshes/finger_base.stl; visual mesh filename=package://handle_description/meshes/finger_base.stl
- added link left_finger[1]/distal_link, mass 0.1; collision mesh filename=package://handle_description/meshes/finger_distal.stl; visual mesh filename=package://handle_description/meshes/finger_distal.stl
- added link left_finger[1]/proximal_link, mass 0.1; collision mesh filename=package://handle_description/meshes/finger_proximal.stl; visual mesh filename=package://handle_description/meshes/finger_proximal.stl
- added link left_finger[2]/distal_link, mass 0.1; collision mesh filename=package://handle_description/meshes/finger_distal.stl; visual mesh filename=package://handle_description/meshes/finger_distal.stl
- added link left_finger[2]/proximal_link, mass 0.1; collision mesh filename=package://handle_description/meshes/finger_proximal.stl; visual mesh filename=package://handle_description/meshes/finger_proximal.stl
Joints:
- removed joint imu_joint
- added joint left_finger[0]/joint_base: type revolute, parent left_finger[0]/base_rotation_link, child left_finger[0]/proximal_link, origin xyz=0 0 0.0135 rpy=1.57 0 -3.14, axis -1 0 0, limit lower=0.0 upper=1.57 effort=1000.0 velocity=0.5
- added joint left_finger[0]/joint_base_rotation: type revolute, parent left_base_link, child left_finger[0]/base_rotation_link, origin xyz=0.03075 0.038 0.069477 rpy=0 0 0, axis 0 0 -1, limit lower=0.0 upper=1.57 effort=1000.0 velocity=0.5
- added joint left_finger[0]/joint_flex: type revolute, parent left_finger[0]/proximal_link, child left_finger[0]/distal_link, origin xyz=0 0 0.078, axis -1 0 0, limit lower=0.0 upper=1.57 effort=1000.0 velocity=0.5
- added joint left_finger[1]/joint_base: type revolute, parent left_finger[1]/base_rotation_link, child left_finger[1]/proximal_link, origin xyz=0 0 0.0135 rpy=1.57 0 -3.14, axis -1 0 0, limit lower=0.0 upper=1.57 effort=1000.0 velocity=0.5
- added joint left_finger[1]/joint_base_rotation: type revolute, parent left_base_link, child left_finger[1]/base_rotation_link, origin xyz=-0.03075 0.038 0.069477 rpy=0 0 0, axis 0 0 1, limit lower=0.0 upper=1.57 effort=1000.0 velocity=0.5
- added joint left_finger[1]/joint_flex: type revolute, parent left_finger[1]/proximal_link, child left_finger[1]/distal_link, origin xyz=0 0 0.078, axis -1 0 0, limit lower=0.0 upper=1.57 effort=1000.0 velocity=0.5
- added joint left_finger[2]/joint_base: type revolute, parent left_base_link, child left_finger[2]/proximal_link, origin xyz=0 -0.038 0.082755 rpy=1.57 0 0, axis -1 0 0, limit lower=0.0 upper=1.57 effort=1000.0 velocity=0.5
- added joint left_finger[2]/joint_flex: type revolute, parent left_finger[2]/proximal_link, child left_finger[2]/distal_link, origin xyz=0 0 0.078, axis -1 0 0, limit lower=0.0 upper=1.57 effort=1000.0 velocity=0.5
- added joint left_irobot_hand_joint: type fixed, parent l_hand, child left_base_link, origin xyz=0 0.11516 0.015 rpy=1.57079 3.14159 3.14159

File: software/models/mit_gazebo_models/mit_robot/model_LN_RI.urdf (robot description, URDF)
Before this commit: robot atlas, 74 links, 73 joints
Links:
- removed link left_base_link
- removed link left_finger[0]/base_rotation_link
- removed link left_finger[0]/distal_link
- removed link left_finger[0]/proximal_link
- removed link left_finger[1]/base_rotation_link
- removed link left_finger[1]/distal_link
- removed link left_finger[1]/proximal_link
- removed link left_finger[2]/distal_link
- removed link left_finger[2]/proximal_link
Joints:
- removed joint left_finger[0]/joint_base
- removed joint left_finger[0]/joint_base_rotation
- removed joint left_finger[0]/joint_flex
- removed joint left_finger[1]/joint_base
- removed joint left_finger[1]/joint_base_rotation
- removed joint left_finger[1]/joint_flex
- removed joint left_finger[2]/joint_base
- removed joint left_finger[2]/joint_flex
- removed joint left_irobot_hand_joint

File: software/models/mit_gazebo_models/mit_robot/model_LN_RN.urdf (robot description, URDF)
Before this commit: robot atlas, 74 links, 73 joints
Links:
- removed link left_base_link
- removed link left_finger[0]/base_rotation_link
- removed link left_finger[0]/distal_link
- removed link left_finger[0]/proximal_link
- removed link left_finger[1]/base_rotation_link
- removed link left_finger[1]/distal_link
- removed link left_finger[1]/proximal_link
- removed link left_finger[2]/distal_link
- removed link left_finger[2]/proximal_link
- removed link right_base_link
- removed link right_finger[0]/base_rotation_link
- removed link right_finger[0]/distal_link
- removed link right_finger[0]/proximal_link
- removed link right_finger[1]/base_rotation_link
- removed link right_finger[1]/distal_link
- removed link right_finger[1]/proximal_link
- removed link right_finger[2]/distal_link
- removed link right_finger[2]/proximal_link
- added link imu_link, mass 0.1; visual box size=0.01 0.01 0.01
Joints:
- removed joint left_finger[0]/joint_base
- removed joint left_finger[0]/joint_base_rotation
- removed joint left_finger[0]/joint_flex
- removed joint left_finger[1]/joint_base
- removed joint left_finger[1]/joint_base_rotation
- removed joint left_finger[1]/joint_flex
- removed joint left_finger[2]/joint_base
- removed joint left_finger[2]/joint_flex
- removed joint left_irobot_hand_joint
- removed joint right_finger[0]/joint_base
- removed joint right_finger[0]/joint_base_rotation
- removed joint right_finger[0]/joint_flex
- removed joint right_finger[1]/joint_base
- removed joint right_finger[1]/joint_base_rotation
- removed joint right_finger[1]/joint_flex
- removed joint right_finger[2]/joint_base
- removed joint right_finger[2]/joint_flex
- removed joint right_irobot_hand_joint
- added joint imu_joint: type fixed, parent pelvis, child imu_link, origin xyz=0.05991527603 0 -0.01415 rpy=0 0 0
