Commit message: git-svn-id: https://svn.csail.mit.edu/drc/trunk@7418 c7283977-0100-402a-a91a-fa70b306dbfe

File: software/models/mit_gazebo_models/mit_robot/model_LH_RI.urdf (robot description, URDF)
Before this commit: robot atlas, 68 links, 67 joints
Links:
- removed link left_finger[0]/base_rotation_link
- removed link left_finger[0]/distal_link
- removed link left_finger[0]/proximal_link
- removed link left_finger[1]/base_rotation_link
- removed link left_finger[1]/distal_link
- removed link left_finger[1]/proximal_link
- removed link left_finger[2]/distal_link
- removed link left_finger[2]/proximal_link
- removed link right_pipe_hand
- removed link right_pipe_hook
- added link right_finger[0]/base_rotation_link, mass 0.1; collision mesh filename=package://handle_description/meshes/finger_base.stl; visual mesh filename=package://handle_description/meshes/finger_base.stl
- added link right_finger[0]/distal_link, mass 0.1; collision mesh filename=package://handle_description/meshes/finger_distal.stl; visual mesh filename=package://handle_description/meshes/finger_distal.stl
- added link right_finger[0]/proximal_link, mass 0.1; collision mesh filename=package://handle_description/meshes/finger_proximal.stl; visual mesh filename=package://handle_description/meshes/finger_proximal.stl
- added link right_finger[1]/base_rotation_link, mass 0.1; collision mesh filename=package://handle_description/meshes/finger_base.stl; visual mesh filename=package://handle_description/meshes/finger_base.stl
- added link right_finger[1]/distal_link, mass 0.1; collision mesh filename=package://handle_description/meshes/finger_distal.stl; visual mesh filename=package://handle_description/meshes/finger_distal.stl
- added link right_finger[1]/proximal_link, mass 0.1; collision mesh filename=package://handle_description/meshes/finger_proximal.stl; visual mesh filename=package://handle_description/meshes/finger_proximal.stl
- added link right_finger[2]/distal_link, mass 0.1; collision mesh filename=package://handle_description/meshes/finger_distal.stl; visual mesh filename=package://handle_description/meshes/finger_distal.stl
- added link right_finger[2]/proximal_link, mass 0.1; collision mesh filename=package://handle_description/meshes/finger_proximal.stl; visual mesh filename=package://handle_description/meshes/finger_proximal.stl
- link left_base_link: geometry collision cylinder length=0.01 radius=0.045; collision cylinder length=0.04 radius=0.006
- link right_base_link: geometry collision mesh filename=package://handle_description/meshes/palm.stl; visual mesh filename=package://handle_description/meshes/palm.stl
Joints:
- removed joint left_finger[0]/joint_base
- removed joint left_finger[0]/joint_base_rotation
- removed joint left_finger[0]/joint_flex
- removed joint left_finger[1]/joint_base
- removed joint left_finger[1]/joint_base_rotation
- removed joint left_finger[1]/joint_flex
- removed joint left_finger[2]/joint_base
- removed joint left_finger[2]/joint_flex
- removed joint right_hook_hand_hook_joint
- removed joint right_hook_hand_joint
- removed joint right_hook_hand_pipe_joint
- added joint right_finger[0]/joint_base: type revolute, parent right_finger[0]/base_rotation_link, child right_finger[0]/proximal_link, origin xyz=0 0 0.0135 rpy=1.57 0 -3.14, axis -1 0 0, limit lower=0.0 upper=1.57 effort=1000.0 velocity=0.5
- added joint right_finger[0]/joint_base_rotation: type revolute, parent right_base_link, child right_finger[0]/base_rotation_link, origin xyz=0.03075 0.038 0.069477 rpy=0 0 0, axis 0 0 -1, limit lower=0.0 upper=1.57 effort=1000.0 velocity=0.5
- added joint right_finger[0]/joint_flex: type revolute, parent right_finger[0]/proximal_link, child right_finger[0]/distal_link, origin xyz=0 0 0.078, axis -1 0 0, limit lower=0.0 upper=1.57 effort=1000.0 velocity=0.5
- added joint right_finger[1]/joint_base: type revolute, parent right_finger[1]/base_rotation_link, child right_finger[1]/proximal_link, origin xyz=0 0 0.0135 rpy=1.57 0 -3.14, axis -1 0 0, limit lower=0.0 upper=1.57 effort=1000.0 velocity=0.5
- added joint right_finger[1]/joint_base_rotation: type revolute, parent right_base_link, child right_finger[1]/base_rotation_link, origin xyz=-0.03075 0.038 0.069477 rpy=0 0 0, axis 0 0 1, limit lower=0.0 upper=1.57 effort=1000.0 velocity=0.5
- added joint right_finger[1]/joint_flex: type revolute, parent right_finger[1]/proximal_link, child right_finger[1]/distal_link, origin xyz=0 0 0.078, axis -1 0 0, limit lower=0.0 upper=1.57 effort=1000.0 velocity=0.5
- added joint right_finger[2]/joint_base: type revolute, parent right_base_link, child right_finger[2]/proximal_link, origin xyz=0 -0.038 0.082755 rpy=1.57 0 0, axis -1 0 0, limit lower=0.0 upper=1.57 effort=1000.0 velocity=0.5
- added joint right_finger[2]/joint_flex: type revolute, parent right_finger[2]/proximal_link, child right_finger[2]/distal_link, origin xyz=0 0 0.078, axis -1 0 0, limit lower=0.0 upper=1.57 effort=1000.0 velocity=0.5
- added joint right_irobot_hand_joint: type fixed, parent r_hand, child right_base_link, origin xyz=0 -0.11516 -0.015 rpy=1.57079 0 0

Commit message: tobuidl
git-svn-id: https://svn.csail.mit.edu/drc/trunk@7458 c7283977-0100-402a-a91a-fa70b306dbfe

File: software/models/mit_gazebo_models/mit_robot/model_LH_RI.urdf (robot description, URDF)
Before this commit: robot atlas, 66 links, 65 joints
Links:
- link left_base_link: geometry collision cylinder length=0.02 radius=0.045; collision cylinder length=0.04 radius=0.006

Commit message: Updated hook description
git-svn-id: https://svn.csail.mit.edu/drc/trunk@7516 c7283977-0100-402a-a91a-fa70b306dbfe

File: software/models/mit_gazebo_models/mit_robot/model_LH_RI.urdf (robot description, URDF)
Before this commit: robot atlas, 66 links, 65 joints
Links:
- link left_base_link: geometry collision cylinder length=0.01 radius=0.045; collision cylinder length=0.15 radius=0.006
