Commit message: adding stickyhand urdfs for hook and robotiq hand. And atlas models with robotiq hands
git-svn-id: https://svn.csail.mit.edu/drc/trunk@7676 c7283977-0100-402a-a91a-fa70b306dbfe

File: software/models/mit_gazebo_models/mit_robot/model_LN_RR.urdf (robot description, URDF)
Before this commit: robot atlas, 66 links, 65 joints
Links:
- removed link left_base_link
- removed link right_base_link
- removed link right_finger[0]/base_rotation_link
- removed link right_finger[0]/distal_link
- removed link right_finger[0]/proximal_link
- removed link right_finger[1]/base_rotation_link
- removed link right_finger[1]/distal_link
- removed link right_finger[1]/proximal_link
- removed link right_finger[2]/distal_link
- removed link right_finger[2]/proximal_link
- added link right_finger_1_link_0; collision mesh filename=package://robotiq_hand_description/meshes/s-model_articulat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; visual mesh filename=package://robotiq_hand_description/meshes/s-model_articulat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
- added link right_finger_1_link_1; collision mesh filename=package://robotiq_hand_description/meshes/s-model_articulat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; visual mesh filename=package://robotiq_hand_description/meshes/s-model_articulat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
- added link right_finger_1_link_2; collision mesh filename=package://robotiq_hand_description/meshes/s-model_articulat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; visual mesh filename=package://robotiq_hand_description/meshes/s-model_articulat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
- added link right_finger_1_link_3; collision mesh filename=package://robotiq_hand_description/meshes/s-model_articulat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; visual mesh filename=package://robotiq_hand_description/meshes/s-model_articulat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
- added link right_finger_2_link_0; collision mesh filename=package://robotiq_hand_description/meshes/s-model_articulat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; visual mesh filename=package://robotiq_hand_description/meshes/s-model_articulat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
- added link right_finger_2_link_1; collision mesh filename=package://robotiq_hand_description/meshes/s-model_articulat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; visual mesh filename=package://robotiq_hand_description/meshes/s-model_articulat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
- added link right_finger_2_link_2; collision mesh filename=package://robotiq_hand_description/meshes/s-model_articulat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; visual mesh filename=package://robotiq_hand_description/meshes/s-model_articulat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
- added link right_finger_2_link_3; collision mesh filename=package://robotiq_hand_description/meshes/s-model_articulat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; visual mesh filename=package://robotiq_hand_description/meshes/s-model_articulat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
- added link right_finger_middle_link_0; collision mesh filename=package://robotiq_hand_description/meshes/s-model_articulat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; visual mesh filename=package://robotiq_hand_description/meshes/s-model_articulat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
- added link right_finger_middle_link_1; collision mesh filename=package://robotiq_hand_description/meshes/s-model_articulat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; visual mesh filename=package://robotiq_hand_description/meshes/s-model_articulat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
- added link right_finger_middle_link_2; collision mesh filename=package://robotiq_hand_description/meshes/s-model_articulat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; visual mesh filename=package://robotiq_hand_description/meshes/s-model_articulat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
- added link right_finger_middle_link_3; collision mesh filename=package://robotiq_hand_description/meshes/s-model_articulat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; visual mesh filename=package://robotiq_hand_description/meshes/s-model_articulat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
- added link right_palm; collision mesh filename=package://robotiq_hand_description/meshes/s-model_articulat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; visual mesh filename=package://robotiq_hand_description/meshes/s-model_articulat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
Joints:
- removed joint left_hook_hand_joint
- removed joint right_finger[0]/joint_base
- removed joint right_finger[0]/joint_base_rotation
- removed joint right_finger[0]/joint_flex
- removed joint right_finger[1]/joint_base
- removed joint right_finger[1]/joint_base_rotation
- removed joint right_finger[1]/joint_flex
- removed joint right_finger[2]/joint_base
- removed joint right_finger[2]/joint_flex
- removed joint right_irobot_hand_joint
- added joint right_finger_1_joint_1: type revolute, parent right_finger_1_link_0, child right_finger_1_link_1, origin xyz=0.020 0 0 rpy=0 0 0, axis 0 0 1, limit lower=0 upper=3.1416 effort=100 velocity=100
- added joint right_finger_1_joint_2: type revolute, parent right_finger_1_link_1, child right_finger_1_link_2, origin xyz=0.050 -.028 0 rpy=0 0 -0.52, axis 0 0 1, limit lower=0 upper=3.1416 effort=100 velocity=100
- added joint right_finger_1_joint_3: type revolute, parent right_finger_1_link_2, child right_finger_1_link_3, origin xyz=0.039 0 0 rpy=0 0 0, axis 0 0 1, limit lower=0 upper=3.1416 effort=100 velocity=100
- added joint right_finger_2_joint_1: type revolute, parent right_finger_2_link_0, child right_finger_2_link_1, origin xyz=0.020 0 0 rpy=0 0 0, axis 0 0 1, limit lower=0 upper=3.1416 effort=100 velocity=100
- added joint right_finger_2_joint_2: type revolute, parent right_finger_2_link_1, child right_finger_2_link_2, origin xyz=0.050 -.028 0 rpy=0 0 -0.52, axis 0 0 1, limit lower=0 upper=3.1416 effort=100 velocity=100
- added joint right_finger_2_joint_3: type revolute, parent right_finger_2_link_2, child right_finger_2_link_3, origin xyz=0.039 0 0 rpy=0 0 0, axis 0 0 1, limit lower=0 upper=3.1416 effort=100 velocity=100
- added joint right_finger_middle_joint_1: type revolute, parent right_finger_middle_link_0, child right_finger_middle_link_1, origin xyz=0.020 0 0 rpy=0 0 0, axis 0 0 1, limit lower=0 upper=3.1416 effort=100 velocity=100
- added joint right_finger_middle_joint_2: type revolute, parent right_finger_middle_link_1, child right_finger_middle_link_2, origin xyz=0.050 -.028 0 rpy=0 0 -0.52, axis 0 0 1, limit lower=0 upper=3.1416 effort=100 velocity=100
- added joint right_finger_middle_joint_3: type revolute, parent right_finger_middle_link_2, child right_finger_middle_link_3, origin xyz=0.039 0 0 rpy=0 0 0, axis 0 0 1, limit lower=0 upper=3.1416 effort=100 velocity=100
- added joint right_palm_finger_1_joint: type revolute, parent right_palm, child right_finger_1_link_0, origin xyz=-0.0455 0.0214 0.036 rpy=0 3.1416 -1.57, axis 0 1 0, limit lower=-0.16 upper=0.25 effort=100 velocity=100
- added joint right_palm_finger_2_joint: type revolute, parent right_palm, child right_finger_2_link_0, origin xyz=-0.0455 0.0214 -0.036 rpy=0 3.1416 -1.57, axis 0 1 0, limit lower=-0.25 upper=0.16 effort=100 velocity=100
- added joint right_palm_finger_middle_joint: type fixed, parent right_palm, child right_finger_middle_link_0, origin xyz=0.0455 0.0214 0 rpy=0 0 1.57, axis 0 0 1
- added joint right_robotiq_hand_joint: type fixed, parent r_hand, child right_palm, origin xyz=0 -0.11516 -0.015 rpy=0 3.141 3.141

File: software/models/mit_gazebo_models/mit_robot/model_LR_RN.urdf (robot description, URDF)
Before this commit: robot atlas, 66 links, 65 joints
Links:
- removed link left_base_link
- removed link right_base_link
- removed link right_finger[0]/base_rotation_link
- removed link right_finger[0]/distal_link
- removed link right_finger[0]/proximal_link
- removed link right_finger[1]/base_rotation_link
- removed link right_finger[1]/distal_link
- removed link right_finger[1]/proximal_link
- removed link right_finger[2]/distal_link
- removed link right_finger[2]/proximal_link
- added link left_finger_1_link_0; collision mesh filename=package://robotiq_hand_description/meshes/s-model_articulat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; visual mesh filename=package://robotiq_hand_description/meshes/s-model_articulat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
- added link left_finger_1_link_1; collision mesh filename=package://robotiq_hand_description/meshes/s-model_articulat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; visual mesh filename=package://robotiq_hand_description/meshes/s-model_articulat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
- added link left_finger_1_link_2; collision mesh filename=package://robotiq_hand_description/meshes/s-model_articulat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; visual mesh filename=package://robotiq_hand_description/meshes/s-model_articulat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
- added link left_finger_1_link_3; collision mesh filename=package://robotiq_hand_description/meshes/s-model_articulat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; visual mesh filename=package://robotiq_hand_description/meshes/s-model_articulat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
- added link left_finger_2_link_0; collision mesh filename=package://robotiq_hand_description/meshes/s-model_articulat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; visual mesh filename=package://robotiq_hand_description/meshes/s-model_articulat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
- added link left_finger_2_link_1; collision mesh filename=package://robotiq_hand_description/meshes/s-model_articulat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; visual mesh filename=package://robotiq_hand_description/meshes/s-model_articulat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
- added link left_finger_2_link_2; collision mesh filename=package://robotiq_hand_description/meshes/s-model_articulat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; visual mesh filename=package://robotiq_hand_description/meshes/s-model_articulat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
- added link left_finger_2_link_3; collision mesh filename=package://robotiq_hand_description/meshes/s-model_articulat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; visual mesh filename=package://robotiq_hand_description/meshes/s-model_articulat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
- added link left_finger_middle_link_0; collision mesh filename=package://robotiq_hand_description/meshes/s-model_articulat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; visual mesh filename=package://robotiq_hand_description/meshes/s-model_articulat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
- added link left_finger_middle_link_1; collision mesh filename=package://robotiq_hand_description/meshes/s-model_articulat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; visual mesh filename=package://robotiq_hand_description/meshes/s-model_articulat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
- added link left_finger_middle_link_2; collision mesh filename=package://robotiq_hand_description/meshes/s-model_articulat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; visual mesh filename=package://robotiq_hand_description/meshes/s-model_articulat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
- added link left_finger_middle_link_3; collision mesh filename=package://robotiq_hand_description/meshes/s-model_articulat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; visual mesh filename=package://robotiq_hand_description/meshes/s-model_articulat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
- added link left_palm; collision mesh filename=package://robotiq_hand_description/meshes/s-model_articulat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; visual mesh filename=package://robotiq_hand_description/meshes/s-model_articulat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
Joints:
- removed joint left_hook_hand_joint
- removed joint right_finger[0]/joint_base
- removed joint right_finger[0]/joint_base_rotation
- removed joint right_finger[0]/joint_flex
- removed joint right_finger[1]/joint_base
- removed joint right_finger[1]/joint_base_rotation
- removed joint right_finger[1]/joint_flex
- removed joint right_finger[2]/joint_base
- removed joint right_finger[2]/joint_flex
- removed joint right_irobot_hand_joint
- added joint left_finger_1_joint_1: type revolute, parent left_finger_1_link_0, child left_finger_1_link_1, origin xyz=0.020 0 0 rpy=0 0 0, axis 0 0 1, limit lower=0 upper=3.1416 effort=100 velocity=100
- added joint left_finger_1_joint_2: type revolute, parent left_finger_1_link_1, child left_finger_1_link_2, origin xyz=0.050 -.028 0 rpy=0 0 -0.52, axis 0 0 1, limit lower=0 upper=3.1416 effort=100 velocity=100
- added joint left_finger_1_joint_3: type revolute, parent left_finger_1_link_2, child left_finger_1_link_3, origin xyz=0.039 0 0 rpy=0 0 0, axis 0 0 1, limit lower=0 upper=3.1416 effort=100 velocity=100
- added joint left_finger_2_joint_1: type revolute, parent left_finger_2_link_0, child left_finger_2_link_1, origin xyz=0.020 0 0 rpy=0 0 0, axis 0 0 1, limit lower=0 upper=3.1416 effort=100 velocity=100
- added joint left_finger_2_joint_2: type revolute, parent left_finger_2_link_1, child left_finger_2_link_2, origin xyz=0.050 -.028 0 rpy=0 0 -0.52, axis 0 0 1, limit lower=0 upper=3.1416 effort=100 velocity=100
- added joint left_finger_2_joint_3: type revolute, parent left_finger_2_link_2, child left_finger_2_link_3, origin xyz=0.039 0 0 rpy=0 0 0, axis 0 0 1, limit lower=0 upper=3.1416 effort=100 velocity=100
- added joint left_finger_middle_joint_1: type revolute, parent left_finger_middle_link_0, child left_finger_middle_link_1, origin xyz=0.020 0 0 rpy=0 0 0, axis 0 0 1, limit lower=0 upper=3.1416 effort=100 velocity=100
- added joint left_finger_middle_joint_2: type revolute, parent left_finger_middle_link_1, child left_finger_middle_link_2, origin xyz=0.050 -.028 0 rpy=0 0 -0.52, axis 0 0 1, limit lower=0 upper=3.1416 effort=100 velocity=100
- added joint left_finger_middle_joint_3: type revolute, parent left_finger_middle_link_2, child left_finger_middle_link_3, origin xyz=0.039 0 0 rpy=0 0 0, axis 0 0 1, limit lower=0 upper=3.1416 effort=100 velocity=100
- added joint left_palm_finger_1_joint: type revolute, parent left_palm, child left_finger_1_link_0, origin xyz=-0.0455 0.0214 0.036 rpy=0 3.1416 -1.57, axis 0 1 0, limit lower=-0.16 upper=0.25 effort=100 velocity=100
- added joint left_palm_finger_2_joint: type revolute, parent left_palm, child left_finger_2_link_0, origin xyz=-0.0455 0.0214 -0.036 rpy=0 3.1416 -1.57, axis 0 1 0, limit lower=-0.25 upper=0.16 effort=100 velocity=100
- added joint left_palm_finger_middle_joint: type fixed, parent left_palm, child left_finger_middle_link_0, origin xyz=0.0455 0.0214 0 rpy=0 0 1.57, axis 0 0 1
- added joint left_robotiq_hand_joint: type fixed, parent l_hand, child left_palm, origin xyz=0 0.11516 0.015 rpy=0 0 0
