Commit message: modifying models for bdi hooks
git-svn-id: https://svn.csail.mit.edu/drc/trunk@7736 c7283977-0100-402a-a91a-fa70b306dbfe

File: software/models/mit_gazebo_models/mit_robot/model_LH_RN.urdf (robot description, URDF)
Before this commit: robot atlas, 57 links, 56 joints
Links:
- link left_base_link: geometry collision mesh filename=package://hook_description/meshes/bdi_hook.stl scale=0.001 0.001 0.001; visual mesh filename=package://hook_description/meshes/bdi_hook.stl scale=0.001 0.001 0.001

File: software/models/mit_gazebo_models/mit_robot/model_LH_RR.urdf (robot description, URDF)
Before this commit: robot atlas, 66 links, 65 joints
Joints:
- removed joint left_irobot_hand_joint
- added joint left_hook_hand_joint: type fixed, parent l_hand, child left_base_link, origin xyz=0 0.11516 0.015 rpy=1.57079 3.14159 3.14159

File: software/models/mit_gazebo_models/mit_robot/xacro/atlas_LH_RI.urdf.xacro (robot description, xacro)
@@ -4,6 +4,6 @@
   <include filename="$(find mit_drcsim_scripts)/models/multisense_sl/multisense_sl.urdf" />
   <xacro:include filename="$(find handle_description)/src/irobot_hand_simple.urdf.xacro" />
- <xacro:include filename="$(find hook_description)/src/hook_hand_simple.urdf.xacro" />
-<!--    <xacro:include filename="$(find hook_description)/src/bdihook_hand.urdf.xacro" />-->
+ <!-- <xacro:include filename="$(find hook_description)/src/hook_hand_simple.urdf.xacro" />-->
+  <xacro:include filename="$(find hook_description)/src/bdihook_hand.urdf.xacro" />
   <xacro:irobot_hand side="right" parent="r_hand" reflect="1">
     <origin rpy="1.57079 0 0" xyz="0 -0.11516 -0.015"/>

File: software/models/mit_gazebo_models/mit_robot/xacro/atlas_LH_RN.urdf.xacro (robot description, xacro)
@@ -3,6 +3,6 @@
   <include filename="$(find mit_drcsim_scripts)/models/mit_robot/xacro/atlas.transmission" />
   <include filename="$(find mit_drcsim_scripts)/models/multisense_sl/multisense_sl.urdf" />
- <xacro:include filename="$(find hook_description)/src/hook_hand_simple.urdf.xacro" />
-<!--    <xacro:include filename="$(find hook_description)/src/bdihook_hand.urdf.xacro" />-->
+<!-- <xacro:include filename="$(find hook_description)/src/hook_hand_simple.urdf.xacro" />-->
+    <xacro:include filename="$(find hook_description)/src/bdihook_hand.urdf.xacro" />
   <xacro:hook_hand side="left" parent="l_hand" reflect="-1" hookflip="1">
     <origin rpy="1.57079 3.14159 3.14159" xyz="0 0.11516 0.015"/>

File: software/models/mit_gazebo_models/mit_robot_hands/inert_hand_left.urdf (robot description, URDF)
Before this commit: robot inert_hand_left, 2 links, 1 joints
Links:
- link left_base_link: geometry collision mesh filename=package://hook_description/meshes/bdi_hook.stl scale=0.001 0.001 0.001; visual mesh filename=package://hook_description/meshes/bdi_hook.stl scale=0.001 0.001 0.001

File: software/models/mit_gazebo_models/mit_robot_hands/inert_hand_right.urdf (robot description, URDF)
Before this commit: robot inert_hand_right, 2 links, 1 joints
Links:
- link right_base_link: geometry collision mesh filename=package://hook_description/meshes/bdi_hook.stl scale=0.001 0.001 0.001; visual mesh filename=package://hook_description/meshes/bdi_hook.stl scale=0.001 0.001 0.001
Joints:
- joint right_hook_hand_joint: origin xyz=0 0 0 rpy=1.57 0.0 -1.57 -> xyz=0 0 0 rpy=1.57 3.14 -1.57

File: software/models/mit_gazebo_models/mit_robot_hands/xacro/inert_hand_left.urdf.xacro (robot description, xacro)
@@ -11,11 +11,11 @@
     </inertial>
   </link>
- <xacro:include filename="$(find hook_description)/src/hook_hand_simple.urdf.xacro" />
+<!-- <xacro:include filename="$(find hook_description)/src/hook_hand_simple.urdf.xacro" />-->
+<!--  <xacro:hook_hand side="left" parent="plane::xy::base" reflect="-1" hookflip="1">-->
+<!--    <origin rpy="1.57 0.0 -1.57" xyz="0.0 0.0 0.0"/>-->
+<!--  </xacro:hook_hand>-->
+ <xacro:include filename="$(find hook_description)/src/bdihook_hand.urdf.xacro" />
   <xacro:hook_hand side="left" parent="plane::xy::base" reflect="-1" hookflip="1">
     <origin rpy="1.57 0.0 -1.57" xyz="0.0 0.0 0.0"/>
   </xacro:hook_hand>
-<!-- <xacro:include filename="$(find hook_description)/src/bdihook_hand.urdf.xacro" />-->
-<!--  <xacro:hook_hand side="left" parent="plane::xy::base" reflect="-1" hookflip="1">-->
-<!--    <origin rpy="1.57 0.0 -1.57" xyz="0.0 0.0 0.0"/>-->
-<!--  </xacro:hook_hand>-->
 </robot>

File: software/models/mit_gazebo_models/mit_robot_hands/xacro/inert_hand_right.urdf.xacro (robot description, xacro)
@@ -11,11 +11,11 @@
     </inertial>
   </link>
- <xacro:include filename="$(find hook_description)/src/hook_hand_simple.urdf.xacro" />
+<!-- <xacro:include filename="$(find hook_description)/src/hook_hand_simple.urdf.xacro" />-->
+<!--  <xacro:hook_hand side="right" parent="plane::xy::base" reflect="1" hookflip="1">-->
+<!--    <origin rpy="1.57 0.0 -1.57" xyz="0 0 0"/>   -->
+<!--  </xacro:hook_hand>  -->
+  <xacro:include filename="$(find hook_description)/src/bdihook_hand.urdf.xacro" />
   <xacro:hook_hand side="right" parent="plane::xy::base" reflect="1" hookflip="1">
-    <origin rpy="1.57 0.0 -1.57" xyz="0 0 0"/>
+    <origin rpy="1.57 3.14 -1.57" xyz="0 0 0"/>
   </xacro:hook_hand>
-<!--  <xacro:include filename="$(find hook_description)/src/bdihook_hand.urdf.xacro" />-->
-<!--  <xacro:hook_hand side="right" parent="plane::xy::base" reflect="1" hookflip="1">-->
-<!--    <origin rpy="1.57 3.14 -1.57" xyz="0 0 0"/>   -->
-<!--  </xacro:hook_hand>  -->
 </robot>

Commit message: reverting atlas_LH_RN and atlas_LH_RI
git-svn-id: https://svn.csail.mit.edu/drc/trunk@7738 c7283977-0100-402a-a91a-fa70b306dbfe

File: software/models/mit_gazebo_models/mit_robot/model_LH_RN.urdf (robot description, URDF)
Before this commit: robot atlas, 57 links, 56 joints
Links:
- link left_base_link: geometry collision cylinder length=0.01 radius=0.045; collision cylinder length=0.04 radius=0.006

File: software/models/mit_gazebo_models/mit_robot/xacro/atlas_LH_RI.urdf.xacro (robot description, xacro)
@@ -4,6 +4,6 @@
   <include filename="$(find mit_drcsim_scripts)/models/multisense_sl/multisense_sl.urdf" />
   <xacro:include filename="$(find handle_description)/src/irobot_hand_simple.urdf.xacro" />
- <!-- <xacro:include filename="$(find hook_description)/src/hook_hand_simple.urdf.xacro" />-->
-  <xacro:include filename="$(find hook_description)/src/bdihook_hand.urdf.xacro" />
+ <xacro:include filename="$(find hook_description)/src/hook_hand_simple.urdf.xacro" />
+ <!-- <xacro:include filename="$(find hook_description)/src/bdihook_hand.urdf.xacro" />-->
   <xacro:irobot_hand side="right" parent="r_hand" reflect="1">
     <origin rpy="1.57079 0 0" xyz="0 -0.11516 -0.015"/>

File: software/models/mit_gazebo_models/mit_robot/xacro/atlas_LH_RN.urdf.xacro (robot description, xacro)
@@ -3,6 +3,6 @@
   <include filename="$(find mit_drcsim_scripts)/models/mit_robot/xacro/atlas.transmission" />
   <include filename="$(find mit_drcsim_scripts)/models/multisense_sl/multisense_sl.urdf" />
-<!-- <xacro:include filename="$(find hook_description)/src/hook_hand_simple.urdf.xacro" />-->
-    <xacro:include filename="$(find hook_description)/src/bdihook_hand.urdf.xacro" />
+  <xacro:include filename="$(find hook_description)/src/hook_hand_simple.urdf.xacro" />
+<!-- <xacro:include filename="$(find hook_description)/src/bdihook_hand.urdf.xacro" />-->
   <xacro:hook_hand side="left" parent="l_hand" reflect="-1" hookflip="1">
     <origin rpy="1.57079 3.14159 3.14159" xyz="0 0.11516 0.015"/>

File: software/models/mit_gazebo_models/mit_robot_hands/inert_hand_left.urdf (robot description, URDF)
Before this commit: robot inert_hand_left, 2 links, 1 joints
Links:
- link left_base_link: geometry collision cylinder length=0.01 radius=0.045; collision cylinder length=0.04 radius=0.006

File: software/models/mit_gazebo_models/mit_robot_hands/inert_hand_right.urdf (robot description, URDF)
Before this commit: robot inert_hand_right, 2 links, 1 joints
Links:
- link right_base_link: geometry collision cylinder length=0.01 radius=0.045; collision cylinder length=0.04 radius=0.006
Joints:
- joint right_hook_hand_joint: origin xyz=0 0 0 rpy=1.57 3.14 -1.57 -> xyz=0 0 0 rpy=1.57 0.0 -1.57

File: software/models/mit_gazebo_models/mit_robot_hands/xacro/inert_hand_left.urdf.xacro (robot description, xacro)
@@ -11,11 +11,11 @@
     </inertial>
   </link>
-<!-- <xacro:include filename="$(find hook_description)/src/hook_hand_simple.urdf.xacro" />-->
+ <xacro:include filename="$(find hook_description)/src/hook_hand_simple.urdf.xacro" />
+  <xacro:hook_hand side="left" parent="plane::xy::base" reflect="-1" hookflip="1">
+    <origin rpy="1.57 0.0 -1.57" xyz="0.0 0.0 0.0"/>
+  </xacro:hook_hand>
+<!-- <xacro:include filename="$(find hook_description)/src/bdihook_hand.urdf.xacro" />-->
 <!--  <xacro:hook_hand side="left" parent="plane::xy::base" reflect="-1" hookflip="1">-->
 <!--    <origin rpy="1.57 0.0 -1.57" xyz="0.0 0.0 0.0"/>-->
 <!--  </xacro:hook_hand>-->
- <xacro:include filename="$(find hook_description)/src/bdihook_hand.urdf.xacro" />
-  <xacro:hook_hand side="left" parent="plane::xy::base" reflect="-1" hookflip="1">
-    <origin rpy="1.57 0.0 -1.57" xyz="0.0 0.0 0.0"/>
-  </xacro:hook_hand>
 </robot>

File: software/models/mit_gazebo_models/mit_robot_hands/xacro/inert_hand_right.urdf.xacro (robot description, xacro)
@@ -11,11 +11,11 @@
     </inertial>
   </link>
-<!-- <xacro:include filename="$(find hook_description)/src/hook_hand_simple.urdf.xacro" />-->
+ <xacro:include filename="$(find hook_description)/src/hook_hand_simple.urdf.xacro" />
+  <xacro:hook_hand side="right" parent="plane::xy::base" reflect="1" hookflip="1">
+    <origin rpy="1.57 0.0 -1.57" xyz="0 0 0"/>
+  </xacro:hook_hand>
+<!--  <xacro:include filename="$(find hook_description)/src/bdihook_hand.urdf.xacro" />-->
 <!--  <xacro:hook_hand side="right" parent="plane::xy::base" reflect="1" hookflip="1">-->
-<!--    <origin rpy="1.57 0.0 -1.57" xyz="0 0 0"/>   -->
+<!--    <origin rpy="1.57 3.14 -1.57" xyz="0 0 0"/>   -->
 <!--  </xacro:hook_hand>  -->
-  <xacro:include filename="$(find hook_description)/src/bdihook_hand.urdf.xacro" />
-  <xacro:hook_hand side="right" parent="plane::xy::base" reflect="1" hookflip="1">
-    <origin rpy="1.57 3.14 -1.57" xyz="0 0 0"/>
-  </xacro:hook_hand>
 </robot>
