Commit message: Modified LH_RR to use simple hook hand
git-svn-id: https://svn.csail.mit.edu/drc/trunk@7778 c7283977-0100-402a-a91a-fa70b306dbfe

File: software/models/mit_gazebo_models/mit_robot/model_LH_RR.urdf (robot description, URDF)
Before this commit: robot atlas, 66 links, 65 joints
Links:
- link left_base_link: geometry collision cylinder length=0.01 radius=0.045; collision cylinder length=0.04 radius=0.006

File: software/models/mit_gazebo_models/mit_robot/xacro/atlas_LH_RR.urdf.xacro (robot description, xacro)
@@ -4,5 +4,5 @@
   <include filename="$(find mit_drcsim_scripts)/models/multisense_sl/multisense_sl.urdf" />
   <xacro:include filename="$(find handle_description)/src/irobot_hand_simple.urdf.xacro" />
-  <xacro:include filename="$(find hook_description)/src/bdihook_hand.urdf.xacro" />
+  <xacro:include filename="$(find hook_description)/src/hook_hand_simple.urdf.xacro" />
   <xacro:irobot_hand side="right" parent="r_hand" reflect="1">
     <origin rpy="1.57079 2.0944 0" xyz="0 -0.11516 -0.015"/>
