Commit message: Updated position of robotiq hand on body (for drill task)
git-svn-id: https://svn.csail.mit.edu/drc/trunk@7812 c7283977-0100-402a-a91a-fa70b306dbfe

File: software/models/mit_gazebo_models/mit_robot/model_LH_RQ.urdf (robot description, URDF)
Before this commit: robot atlas, 70 links, 69 joints
Joints:
- joint right_robotiq_hand_joint: origin xyz=0 -0.11516 -0.015 rpy=0 -.5236 3.141 -> xyz=0 -.19016 -0.015 rpy=0 -.5236 3.141

File: software/models/mit_gazebo_models/mit_robot/xacro/atlas_LH_RQ.urdf.xacro (robot description, xacro)
@@ -7,5 +7,5 @@
   <xacro:robotiq_hand side="right" parent="r_hand" reflect="1">
 <!--    <origin rpy="1.57079 2.0944 0" xyz="0 -0.11516 -0.015"/> -->
-    <origin rpy="0 -.5236 3.141" xyz="0 -0.11516 -0.015"/>
+    <origin rpy="0 -.5236 3.141" xyz="0 -.19016 -0.015"/>
   </xacro:robotiq_hand>
   <xacro:hook_hand side="left" parent="l_hand" reflect="-1"  hookflip="1">

Commit message: Added a right_base_link to robotiq description, drill model only
git-svn-id: https://svn.csail.mit.edu/drc/trunk@7815 c7283977-0100-402a-a91a-fa70b306dbfe

File: software/models/mit_gazebo_models/mit_robot/model_LH_RQ.urdf (robot description, URDF)
Before this commit: robot atlas, 70 links, 69 joints
Links:
- added link right_base_link
Joints:
- added joint right_base_link_fix: type fixed, parent r_hand, child right_base_link, origin xyz=0 -.19016 -0.015 rpy=0 -.5236 3.141
- joint right_robotiq_hand_joint: origin xyz=0 -.19016 -0.015 rpy=0 -.5236 3.141 -> xyz=0 0 0 rpy=0 0 0; parent r_hand -> right_base_link

File: software/models/mit_gazebo_models/mit_robot/xacro/atlas_LH_RQ.urdf.xacro (robot description, xacro)
@@ -5,7 +5,13 @@
   <xacro:include filename="$(find robotiq_hand_description)/cfg/robotiq_hand.urdf.xacro" />
   <xacro:include filename="$(find hook_description)/src/hook_hand_simple.urdf.xacro" />
-  <xacro:robotiq_hand side="right" parent="r_hand" reflect="1">
-<!--    <origin rpy="1.57079 2.0944 0" xyz="0 -0.11516 -0.015"/> -->
+  <link name="right_base_link"/>
+  <joint name="right_base_link_fix" type="fixed">
+    <parent link="r_hand"/>
+    <child link="right_base_link"/>
     <origin rpy="0 -.5236 3.141" xyz="0 -.19016 -0.015"/>
+  </joint>
+  <xacro:robotiq_hand side="right" parent="right_base_link" reflect="1">
+<!--    <origin rpy="0 -.5236 3.141" xyz="0 -.19016 -0.015"/>-->
+    <origin rpy="0 0 0" xyz="0 0 0"/>
   </xacro:robotiq_hand>
   <xacro:hook_hand side="left" parent="l_hand" reflect="-1"  hookflip="1">
