Commit message: Fixed LQ_RH orientation
git-svn-id: https://svn.csail.mit.edu/drc/trunk@7912 c7283977-0100-402a-a91a-fa70b306dbfe

File: software/models/mit_gazebo_models/mit_robot/model_LQ_RH.urdf (robot description, URDF)
Before this commit: robot atlas, 71 links, 70 joints
Joints:
- joint left_base_link_fix: origin xyz=0 .19016 0.015 rpy=0 -.5236 0 -> xyz=0 .19016 0.015 rpy=0 .5236 0

File: software/models/mit_gazebo_models/mit_robot/xacro/atlas_LQ_RH.urdf.xacro (robot description, xacro)
@@ -9,5 +9,5 @@
     <parent link="l_hand"/>
     <child link="left_base_link"/>
-    <origin rpy="0 -.5236 0" xyz="0 .19016 0.015"/>
+    <origin rpy="0 .5236 0" xyz="0 .19016 0.015"/>
   </joint>
   <xacro:robotiq_hand side="left" parent="left_base_link" reflect="-1">
