Commit message: fixed the hook orientation
git-svn-id: https://svn.csail.mit.edu/drc/trunk@8013 c7283977-0100-402a-a91a-fa70b306dbfe

File: software/models/mit_gazebo_models/mit_robot/model_LP_RP.urdf (robot description, URDF)
Before this commit: robot atlas, 58 links, 57 joints
Links:
- link left_base_link: geometry collision cylinder length=0.01 radius=0.045; collision cylinder length=0.044 radius=0.006
- link right_base_link: geometry collision cylinder length=0.01 radius=0.045; collision cylinder length=0.044 radius=0.006

File: software/models/mit_gazebo_models/mit_robot/model_LP_RR.urdf (robot description, URDF)
Before this commit: robot atlas, 70 links, 69 joints
Links:
- link left_base_link: geometry collision cylinder length=0.01 radius=0.045; collision cylinder length=0.044 radius=0.006

File: software/models/mit_gazebo_models/mit_robot/model_LQ_RP.urdf (robot description, URDF)
Before this commit: robot atlas, 71 links, 70 joints
Links:
- link right_base_link: geometry collision cylinder length=0.01 radius=0.045; collision cylinder length=0.044 radius=0.006

File: software/models/mit_gazebo_models/mit_robot_hands/xacro/inert_hand_left.urdf.xacro (robot description, xacro)
@@ -12,5 +12,5 @@
   </link>
  <xacro:include filename="$(find hook_description)/src/bdihook_hand.urdf.xacro" />
-<!-- <xacro:include filename="$(find mit_drcsim_scripts)/models/mit_robot_hands/xacro/bdihook_hand.urdf.xacro" />-->
+<!--  <xacro:include filename="$(find hook_description)/src/hook_hand_simple.urdf.xacro" /> -->
   <xacro:hook_hand side="left" parent="plane::xy::base" reflect="-1" hookflip="-1" noof30degoffset="0">
     <origin rpy="1.57 0.0 -1.57" xyz="0.243 0.0 -0.127"/>

File: software/models/mit_gazebo_models/mit_robot_hands/xacro/inert_hand_right.urdf.xacro (robot description, xacro)
@@ -12,4 +12,5 @@
   </link>
   <xacro:include filename="$(find hook_description)/src/bdihook_hand.urdf.xacro" />
+<!--  <xacro:include filename="$(find hook_description)/src/hook_hand_simple.urdf.xacro" />  -->
    <xacro:hook_hand side="right" parent="plane::xy::base" reflect="1" hookflip="-1" noof30degoffset="0">
      <origin rpy="1.57 3.14 -1.57" xyz="0.243 0.0 -0.127"/>
