Commit message: Rotated LQ_RP hand 180 degrees so thumb is on button side
git-svn-id: https://svn.csail.mit.edu/drc/trunk@8003 c7283977-0100-402a-a91a-fa70b306dbfe

File: software/models/mit_gazebo_models/mit_robot/model_LI_RR_extender.urdf (robot description, URDF)
Before this commit: robot atlas, 78 links, 77 joints
Joints:
- joint right_robotiq_hand_joint: origin xyz=0 -0.322 -0.015 rpy=0 3.141 3.141 -> xyz=0 -0.397 -0.015 rpy=0 3.141 3.141

File: software/models/mit_gazebo_models/mit_robot/model_LQ_RP.urdf (robot description, URDF)
Before this commit: robot atlas, 71 links, 70 joints
Joints:
- joint left_base_link_fix: origin xyz=0 .19016 0.015 rpy=0 .5236 0 -> xyz=0 .19016 0.015 rpy=0 -2.618 0

File: software/models/mit_gazebo_models/mit_robot/xacro/atlas_LQ_RP.urdf.xacro (robot description, xacro)
@@ -9,5 +9,6 @@
     <parent link="l_hand"/>
     <child link="left_base_link"/>
-    <origin rpy="0 .5236 0" xyz="0 .19016 0.015"/>
+<!--    <origin rpy="0 .5236 0" xyz="0 .19016 0.015"/>-->
+    <origin rpy="0 -2.618 0" xyz="0 .19016 0.015"/>
   </joint>
   <xacro:robotiq_hand side="left" parent="left_base_link" reflect="-1">

Commit message: extender lenguth fix for 6 inch extender
git-svn-id: https://svn.csail.mit.edu/drc/trunk@8028 c7283977-0100-402a-a91a-fa70b306dbfe

File: software/models/mit_gazebo_models/mit_robot/model_LI_RR_extender.urdf (robot description, URDF)
Before this commit: robot atlas, 78 links, 77 joints
Joints:
- joint left_irobot_hand_joint: origin xyz=0 0.322 0.015 rpy=1.57079 3.14159 3.14159 -> xyz=0 0.26756 0.015 rpy=1.57079 3.14159 3.14159
- joint right_robotiq_hand_joint: origin xyz=0 -0.397 -0.015 rpy=0 3.141 3.141 -> xyz=0 -0.34256 -0.015 rpy=0 3.141 3.141

File: software/models/mit_gazebo_models/mit_robot/xacro/atlas_LI_RR_extender.urdf.xacro (robot description, xacro)
@@ -18,13 +18,18 @@
 set z=0.015 as the irobot hand center is clearly aligned with the force torque
 still think that y seperaton could be improved
+1 dec:
 Extender is 8" - 0.2047m long
+6 dec:
+Newer extender is 6" - 0.1524m
+robotiq = 0.19016 +  0.1524 = 0.39486
+irobot  = 0.11516 +  0.1524 = 0.26756
 -->
   <xacro:include filename="$(find handle_description)/src/irobot_hand_simple.urdf.xacro" />
   <xacro:include filename="$(find robotiq_hand_description)/cfg/robotiq_hand.urdf.xacro" />
   <xacro:irobot_hand side="left" parent="l_hand" reflect="-1">
-    <origin rpy="1.57079 3.14159 3.14159" xyz="0 0.322 0.015"/>
+    <origin rpy="1.57079 3.14159 3.14159" xyz="0 0.26756 0.015"/>
   </xacro:irobot_hand>
   <xacro:robotiq_hand side="right" parent="r_hand" reflect="1">
-    <origin rpy="0 3.141 3.141" xyz="0 -0.397 -0.015"/>
+    <origin rpy="0 3.141 3.141" xyz="0 -0.34256 -0.015"/>
   </xacro:robotiq_hand>
 </robot>

Commit message: stuff for extended reach
git-svn-id: https://svn.csail.mit.edu/drc/trunk@8037 c7283977-0100-402a-a91a-fa70b306dbfe

File: software/models/mit_gazebo_models/mit_robot/model_LI_RR_extender.urdf (robot description, URDF)
Before this commit: robot atlas, 78 links, 77 joints
Joints:
- joint left_irobot_hand_joint: origin xyz=0 0.26756 0.015 rpy=1.57079 3.14159 3.14159 -> xyz=0 0.26756 0.015 rpy=1.57079 0 -3.14159

File: software/models/mit_gazebo_models/mit_robot/xacro/atlas_LI_RR_extender.urdf.xacro (robot description, xacro)
@@ -28,8 +28,13 @@
   <xacro:include filename="$(find robotiq_hand_description)/cfg/robotiq_hand.urdf.xacro" />
   <xacro:irobot_hand side="left" parent="l_hand" reflect="-1">
-    <origin rpy="1.57079 3.14159 3.14159" xyz="0 0.26756 0.015"/>
+    <origin rpy="1.57079 0 -3.14159" xyz="0 0.26756 0.015"/>
   </xacro:irobot_hand>
   <xacro:robotiq_hand side="right" parent="r_hand" reflect="1">
     <origin rpy="0 3.141 3.141" xyz="0 -0.34256 -0.015"/>
   </xacro:robotiq_hand>
+<!-- if using other combo
+  <xacro:irobot_hand side="right" parent="r_hand" reflect="1">
+    <origin rpy="1.57079 0 3.141" xyz="0 -0.26756 -0.015"/>
+  </xacro:irobot_hand>
+-->
 </robot>

Commit message: added 90 degrees rot
git-svn-id: https://svn.csail.mit.edu/drc/trunk@8064 c7283977-0100-402a-a91a-fa70b306dbfe

File: software/models/mit_gazebo_models/mit_robot/model_LI_RR_extender.urdf (robot description, URDF)
Before this commit: robot atlas, 78 links, 77 joints
Joints:
- joint right_robotiq_hand_joint: origin xyz=0 -0.34256 -0.015 rpy=0 3.141 3.141 -> xyz=0 -0.34256 -0.015 rpy=0 1.57079 3.141

File: software/models/mit_gazebo_models/mit_robot/xacro/atlas_LI_RR_extender.urdf.xacro (robot description, xacro)
@@ -24,4 +24,6 @@
 robotiq = 0.19016 +  0.1524 = 0.39486
 irobot  = 0.11516 +  0.1524 = 0.26756
+8 dec:
+rotated robotiq to match an irobot orientation on the right
 -->
   <xacro:include filename="$(find handle_description)/src/irobot_hand_simple.urdf.xacro" />
@@ -31,5 +33,5 @@
   </xacro:irobot_hand>
   <xacro:robotiq_hand side="right" parent="r_hand" reflect="1">
-    <origin rpy="0 3.141 3.141" xyz="0 -0.34256 -0.015"/>
+    <origin rpy="0 1.57079 3.141" xyz="0 -0.34256 -0.015"/>
   </xacro:robotiq_hand>
 <!-- if using other combo
@@ -37,4 +39,5 @@
     <origin rpy="1.57079 0 3.141" xyz="0 -0.26756 -0.015"/>
   </xacro:irobot_hand>
+robotiq not done
 -->
 </robot>

Commit message: added cylinders to extender model
git-svn-id: https://svn.csail.mit.edu/drc/trunk@8251 c7283977-0100-402a-a91a-fa70b306dbfe

File: software/models/mit_gazebo_models/mit_robot/model_LI_RR_extender.urdf (robot description, URDF)
Before this commit: robot atlas, 78 links, 77 joints
Links:
- added link left_extender; visual cylinder length=0.184 radius=0.03
- added link right_extender; visual cylinder length=0.184 radius=0.03
Joints:
- added joint left_extender_fixed_joint: type fixed, parent l_hand, child left_extender, origin xyz=0 0.11516 0.015 rpy=1.57079 1.57079 3.141
- added joint right_extender_fixed_joint: type fixed, parent r_hand, child right_extender, origin xyz=0 -0.11516 -0.015 rpy=1.57079 1.57079 3.141

File: software/models/mit_gazebo_models/mit_robot/xacro/atlas_LI_RR_extender.urdf.xacro (robot description, xacro)
@@ -26,4 +26,6 @@
 8 dec:
 rotated robotiq to match an irobot orientation on the right
+12 dec:
+added visual element for cylinder
 -->
   <xacro:include filename="$(find handle_description)/src/irobot_hand_simple.urdf.xacro" />
@@ -35,4 +37,36 @@
     <origin rpy="0 1.57079 3.141" xyz="0 -0.34256 -0.015"/>
   </xacro:robotiq_hand>
+  <link name="left_extender">
+    <visual>
+      <origin rpy="0 0 0" xyz = "0 0 .0862"/>
+      <geometry>
+        <cylinder length="0.184" radius="0.03"/>
+      </geometry>
+      <material name="left_extender">
+        <color rgba="0.835 0.655 0.345 1.0"/>
+      </material>
+    </visual>
+  </link>
+  <joint name="left_extender_fixed_joint" type="fixed">
+    <parent link="l_hand"/>
+    <child link="left_extender"/>
+    <origin rpy="1.57079 1.57079 3.141" xyz="0 0.11516 0.015"/>
+  </joint>
+  <link name="right_extender">
+    <visual>
+      <origin rpy="0 0 0" xyz = "0 0 -.0862"/>
+      <geometry>
+        <cylinder length="0.184" radius="0.03"/>
+      </geometry>
+      <material name="right_extender">
+        <color rgba="0.835 0.655 0.345 1.0"/>
+      </material>
+    </visual>
+  </link>
+  <joint name="right_extender_fixed_joint" type="fixed">
+    <parent link="r_hand"/>
+    <child link="right_extender"/>
+    <origin rpy="1.57079 1.57079 3.141" xyz="0 -0.11516 -0.015"/>
+  </joint>
 <!-- if using other combo
   <xacro:irobot_hand side="right" parent="r_hand" reflect="1">
