Commit message: added robotiq extension to hands other than michaels
git-svn-id: https://svn.csail.mit.edu/drc/trunk@7997 c7283977-0100-402a-a91a-fa70b306dbfe

File: software/models/mit_gazebo_models/mit_robot/model_LI_RR.urdf (robot description, URDF)
Before this commit: robot atlas, 78 links, 77 joints
Joints:
- joint right_robotiq_hand_joint: origin xyz=0 -0.11516 -0.015 rpy=0 3.141 3.141 -> xyz=0 -0.19016 -0.015 rpy=0 3.141 3.141

File: software/models/mit_gazebo_models/mit_robot/model_LI_RR_extender.urdf (robot description, URDF)
Before this commit: robot atlas, 87 links, 86 joints
Links:
- removed link right_base_link
- removed link right_finger[0]/base_rotation_link
- removed link right_finger[0]/distal_link
- removed link right_finger[0]/proximal_link
- removed link right_finger[1]/base_rotation_link
- removed link right_finger[1]/distal_link
- removed link right_finger[1]/proximal_link
- removed link right_finger[2]/distal_link
- removed link right_finger[2]/proximal_link
Joints:
- removed joint right_finger[0]/joint_base
- removed joint right_finger[0]/joint_base_rotation
- removed joint right_finger[0]/joint_flex
- removed joint right_finger[1]/joint_base
- removed joint right_finger[1]/joint_base_rotation
- removed joint right_finger[1]/joint_flex
- removed joint right_finger[2]/joint_base
- removed joint right_finger[2]/joint_flex
- removed joint right_irobot_hand_joint

File: software/models/mit_gazebo_models/mit_robot/model_LP_RR.urdf (robot description, URDF)
Before this commit: robot atlas, 70 links, 69 joints
Joints:
- joint right_robotiq_hand_joint: origin xyz=0 -0.11516 -0.015 rpy=0 3.141 3.141 -> xyz=0 -0.19016 -0.015 rpy=0 3.141 3.141

File: software/models/mit_gazebo_models/mit_robot/xacro/atlas_LI_RR.urdf.xacro (robot description, xacro)
@@ -9,5 +9,5 @@
   </xacro:irobot_hand>
   <xacro:robotiq_hand side="right" parent="r_hand" reflect="1">
-    <origin rpy="0 3.141 3.141" xyz="0 -0.11516 -0.015"/>
+    <origin rpy="0 3.141 3.141" xyz="0 -0.19016 -0.015"/>
   </xacro:robotiq_hand>
 </robot>

File: software/models/mit_gazebo_models/mit_robot/xacro/atlas_LI_RR_extender.urdf.xacro (robot description, xacro)
@@ -3,11 +3,4 @@
   <include filename="$(find mit_drcsim_scripts)/models/mit_robot/xacro/atlas.transmission" />
   <include filename="$(find mit_drcsim_scripts)/models/multisense_sl/multisense_sl.urdf" />
-  <xacro:include filename="$(find handle_description)/src/irobot_hand_simple.urdf.xacro" />
-  <xacro:irobot_hand side="right" parent="r_hand" reflect="1">
-    <origin rpy="1.57079 0 0" xyz="0 -0.322 -0.015"/>
-  </xacro:irobot_hand>
-  <xacro:irobot_hand side="left" parent="l_hand" reflect="-1">
-    <origin rpy="1.57079 3.14159 3.14159" xyz="0 0.322 0.015"/>
-  </xacro:irobot_hand>
 <!--
 05 sept: Sisir added an offset of 0.045 in the urdf to account
@@ -25,5 +18,5 @@
 set z=0.015 as the irobot hand center is clearly aligned with the force torque
 still think that y seperaton could be improved
-Extender is 0.2047m long
+Extender is 8" - 0.2047m long
 -->
   <xacro:include filename="$(find handle_description)/src/irobot_hand_simple.urdf.xacro" />
@@ -33,5 +26,5 @@
   </xacro:irobot_hand>
   <xacro:robotiq_hand side="right" parent="r_hand" reflect="1">
-    <origin rpy="0 3.141 3.141" xyz="0 -0.322 -0.015"/>
+    <origin rpy="0 3.141 3.141" xyz="0 -0.397 -0.015"/>
   </xacro:robotiq_hand>
 </robot>

File: software/models/mit_gazebo_models/mit_robot/xacro/atlas_LP_RR.urdf.xacro (robot description, xacro)
@@ -9,5 +9,5 @@
   </xacro:hook_hand>
   <xacro:robotiq_hand side="right" parent="r_hand" reflect="1">
-    <origin rpy="0 3.141 3.141" xyz="0 -0.11516 -0.015"/>
+    <origin rpy="0 3.141 3.141" xyz="0 -0.19016 -0.015"/>
   </xacro:robotiq_hand>
 </robot>

Commit message: rbotoiq right orinetation change in urdf and planner. code reviewed by scott
git-svn-id: https://svn.csail.mit.edu/drc/trunk@8266 c7283977-0100-402a-a91a-fa70b306dbfe

File: software/models/mit_gazebo_models/mit_robot/model_LI_RR.urdf (robot description, URDF)
Before this commit: robot atlas, 78 links, 77 joints
Joints:
- joint right_robotiq_hand_joint: origin xyz=0 -0.19016 -0.015 rpy=0 3.141 3.141 -> xyz=0 -0.19016 -0.015 rpy=0 1.57079 3.141

File: software/models/mit_gazebo_models/mit_robot/xacro/atlas_LI_RR.urdf.xacro (robot description, xacro)
@@ -9,5 +9,5 @@
   </xacro:irobot_hand>
   <xacro:robotiq_hand side="right" parent="r_hand" reflect="1">
-    <origin rpy="0 3.141 3.141" xyz="0 -0.19016 -0.015"/>
+    <origin rpy="0 1.57079 3.141" xyz="0 -0.19016 -0.015"/>
   </xacro:robotiq_hand>
 </robot>
