Commit message: adding urdf for bdi joint names and another for simulator joint names
git-svn-id: https://svn.csail.mit.edu/drc/trunk@5698 c7283977-0100-402a-a91a-fa70b306dbfe

File: software/models/mit_gazebo_models/mit_robot/model_sim.urdf (robot description, URDF)
Before this commit: robot atlas, 107 links, 106 joints
Joints:
- removed joint back_bkx
- removed joint back_bky
- removed joint back_bkz
- removed joint l_arm_shy
- removed joint l_arm_wrx
- removed joint l_arm_wry
- removed joint l_leg_akx
- removed joint l_leg_aky
- removed joint l_leg_hpx
- removed joint l_leg_hpy
- removed joint l_leg_hpz
- removed joint neck_ry
- removed joint r_arm_shy
- removed joint r_arm_wrx
- removed joint r_arm_wry
- removed joint r_leg_akx
- removed joint r_leg_aky
- removed joint r_leg_hpx
- removed joint r_leg_hpy
- removed joint r_leg_hpz
- added joint back_lbz: type revolute, parent pelvis, child ltorso, origin xyz=-0.0125 0 0 rpy=0 -0 0, axis 0 0 1, limit lower=-0.610865 upper=0.610865 effort=124.016 velocity=12
- added joint back_mby: type revolute, parent ltorso, child mtorso, origin xyz=0 0 0.09 rpy=0 -0 0, axis 0 1 0, limit lower=-1.2 upper=1.28 effort=206.843 velocity=12
- added joint back_ubx: type revolute, parent mtorso, child utorso, origin xyz=0 0 0.05 rpy=0 -0 0, axis 1 0 0, limit lower=-0.790809 upper=0.790809 effort=94.91 velocity=12
- added joint l_arm_mwx: type revolute, parent l_farm, child l_hand, origin xyz=0 0.058 0 rpy=0 -0 0, axis 1 0 0, limit lower=-0.436 upper=1.571 effort=60 velocity=12
- added joint l_arm_usy: type revolute, parent utorso, child l_clav, origin xyz=0.024 0.221 0.289 rpy=0 -0 0, axis 0 0.5 0.866025, limit lower=-1.9635 upper=1.9635 effort=212 velocity=12
- added joint l_arm_uwy: type revolute, parent l_larm, child l_farm, origin xyz=0 0.188 -0.013 rpy=0 -0 0, axis 0 1 0, limit lower=-1.571 upper=1.571 effort=114 velocity=12
- added joint l_leg_lax: type revolute, parent l_talus, child l_foot, origin xyz=0 0 0 rpy=0 -0 0, axis 1 0 0, limit lower=-0.436 upper=0.436 effort=90 velocity=12
- added joint l_leg_lhy: type revolute, parent l_lglut, child l_uleg, origin xyz=0.05 0 -0.05 rpy=0 -0 0, axis 0 1 0, limit lower=-1.75 upper=0.524 effort=260 velocity=12
- added joint l_leg_mhx: type revolute, parent l_uglut, child l_lglut, origin xyz=0 0 0 rpy=0 -0 0, axis 1 0 0, limit lower=-0.47 upper=0.495 effort=180 velocity=12
- added joint l_leg_uay: type revolute, parent l_lleg, child l_talus, origin xyz=0 0 -0.422 rpy=0 -0 0, axis 0 1 0, limit lower=-0.9 upper=0.698 effort=220 velocity=12
- added joint l_leg_uhz: type revolute, parent pelvis, child l_uglut, origin xyz=0 0.089 0 rpy=0 -0 0, axis 0 0 1, limit lower=-0.32 upper=1.14 effort=110 velocity=12
- added joint neck_ay: type revolute, parent utorso, child head, origin xyz=0.21672 0 0.53796 rpy=0 -0 0, axis 0 1 0, limit lower=-0.610865238 upper=1.13446401 effort=5 velocity=12
- added joint r_arm_mwx: type revolute, parent r_farm, child r_hand, origin xyz=0 -0.058 0 rpy=0 -0 0, axis 1 0 0, limit lower=-1.571 upper=0.436 effort=60 velocity=12
- added joint r_arm_usy: type revolute, parent utorso, child r_clav, origin xyz=0.024 -0.221 0.289 rpy=0 -0 0, axis 0 0.5 -0.866025, limit lower=-1.9635 upper=1.9635 effort=212 velocity=12
- added joint r_arm_uwy: type revolute, parent r_larm, child r_farm, origin xyz=0 -0.188 -0.013 rpy=0 -0 0, axis 0 1 0, limit lower=-1.571 upper=1.571 effort=114 velocity=12
- added joint r_leg_lax: type revolute, parent r_talus, child r_foot, origin xyz=0 0 0 rpy=0 -0 0, axis 1 0 0, limit lower=-0.436 upper=0.436 effort=90 velocity=12
- added joint r_leg_lhy: type revolute, parent r_lglut, child r_uleg, origin xyz=0.05 0 -0.05 rpy=0 -0 0, axis 0 1 0, limit lower=-1.745 upper=0.524 effort=260 velocity=12
- added joint r_leg_mhx: type revolute, parent r_uglut, child r_lglut, origin xyz=0 0 0 rpy=0 -0 0, axis 1 0 0, limit lower=-0.495 upper=0.47 effort=180 velocity=12
- added joint r_leg_uay: type revolute, parent r_lleg, child r_talus, origin xyz=0 0 -0.422 rpy=0 -0 0, axis 0 1 0, limit lower=-0.9 upper=0.698 effort=220 velocity=12
- added joint r_leg_uhz: type revolute, parent pelvis, child r_uglut, origin xyz=0 -0.089 0 rpy=0 -0 0, axis 0 0 1, limit lower=-1.14 upper=0.32 effort=110 velocity=12

Commit message: completing xacro scripts, seems to be finished
git-svn-id: https://svn.csail.mit.edu/drc/trunk@5859 c7283977-0100-402a-a91a-fa70b306dbfe

File: software/models/mit_gazebo_models/mit_robot/model_sim.urdf (robot description, URDF)
Before this commit: robot atlas, 107 links, 106 joints
Links:
- link head: geometry collision box size=0.0468 0.12 0.1184; collision box size=0.1311 0.12 0.0591
- link hokuyo_link: geometry collision box size=0.08 0.06 0.04238; collision cylinder length=0.047 radius=0.024425

File: software/models/mit_gazebo_models/mit_robot/model_sim_gazebo.urdf (robot description, URDF)
Before this commit: robot atlas, 107 links, 106 joints
Links:
- link head: geometry collision box size=0.0468 0.12 0.1184; collision box size=0.1311 0.12 0.0591
- link hokuyo_link: geometry collision box size=0.08 0.06 0.04238; collision cylinder length=0.047 radius=0.024425

File: software/models/mit_gazebo_models/mit_robot/xacro/atlas_sandia_hands_sim.urdf.xacro (robot description, xacro)
@@ -10,5 +10,5 @@
   <include filename="$(find mit_drcsim_scripts)/models/mit_robot/xacro/atlas.gazebo" />
   <include filename="$(find mit_drcsim_scripts)/models/mit_robot/xacro/atlas.transmission" />
-  <include filename="$(find multisense_sl_description)/multisense_sl_description.urdf" />
+  <include filename="$(find mit_drcsim_scripts)/models/multisense_sl/multisense_sl_sim.urdf" />
   <include filename="$(find mit_drcsim_scripts)/models/mit_robot/xacro/mit_atlas.gazebo" />
   <gazebo>

Commit message: making sim version hand orientation conform to the real hardware
git-svn-id: https://svn.csail.mit.edu/drc/trunk@6002 c7283977-0100-402a-a91a-fa70b306dbfe

File: software/models/mit_gazebo_models/mit_robot/model_sim.urdf (robot description, URDF)
Before this commit: robot atlas, 107 links, 106 joints
Joints:
- joint left_sandia_hand_joint: origin xyz=0  0.1 0 rpy= 1.57079 0  1.57079 -> xyz=0  0.1 0 rpy=0.0 0  1.57079
- joint right_sandia_hand_joint: origin xyz=0 -0.1 0 rpy=-1.57079 0 -1.57079 -> xyz=0 -0.1 0 rpy=0.0 0 -1.57079

File: software/models/mit_gazebo_models/mit_robot/model_sim_gazebo.urdf (robot description, URDF)
Before this commit: robot atlas, 107 links, 106 joints
Joints:
- joint left_sandia_hand_joint: origin xyz=0  0.1 0 rpy= 1.57079 0  1.57079 -> xyz=0  0.1 0 rpy=0.0 0  1.57079
- joint right_sandia_hand_joint: origin xyz=0 -0.1 0 rpy=-1.57079 0 -1.57079 -> xyz=0 -0.1 0 rpy=0.0 0 -1.57079

File: software/models/mit_gazebo_models/mit_robot/xacro/atlas_sandia_hands_sim.urdf.xacro (robot description, xacro)
@@ -5,8 +5,8 @@
   <!-- NB: the Roll of the Sandia Hands is not identical in Sim and Reality -->
   <xacro:sandia_hand side="right" parent="r_hand" reflect="1" joint_type="revolute" thumb_angle="0">
-    <origin xyz="0 -0.1 0" rpy="-1.57079 0 -1.57079"/>
+    <origin xyz="0 -0.1 0" rpy="0.0 0 -1.57079"/>
   </xacro:sandia_hand>
   <xacro:sandia_hand side="left" parent="l_hand" reflect="-1" joint_type="revolute" thumb_angle="0">
-    <origin xyz="0  0.1 0" rpy=" 1.57079 0  1.57079"/>
+    <origin xyz="0  0.1 0" rpy="0.0 0  1.57079"/>
   </xacro:sandia_hand>
   <include filename="$(find mit_drcsim_scripts)/models/mit_robot/xacro/atlas.gazebo" />

Commit message: minor updates to sim model

File: software/models/mit_gazebo_models/mit_robot/model_sim.urdf (robot description, URDF)
Before this commit: robot atlas, 111 links, 110 joints
Joints:
- joint right_sandia_hand_joint: origin xyz=-0.00179 -0.13516 -0.01176 rpy=0 0 -1.57079 -> xyz=-0.00179 -0.13516 0.01176 rpy=0 0 -1.57079

File: software/models/mit_gazebo_models/mit_robot/model_sim_gazebo.urdf (robot description, URDF)
Before this commit: robot atlas, 111 links, 110 joints
Joints:
- joint right_sandia_hand_joint: origin xyz=-0.00179 -0.13516 -0.01176 rpy=0 0 -1.57079 -> xyz=-0.00179 -0.13516 0.01176 rpy=0 0 -1.57079

File: software/models/mit_gazebo_models/mit_robot/xacro/atlas_sandia_hands_sim.urdf.xacro (robot description, xacro)
@@ -2,5 +2,5 @@
   <xacro:include filename="$(find sandia_hand_description)/urdf/sandia_hand_simple_shapes.urdf.xacro" />
   <xacro:sandia_hand side="right" parent="r_hand" reflect="1" joint_type="revolute" thumb_angle="0">
-    <origin xyz="-0.00179 -0.13516 -0.01176" rpy="0 0 -1.57079"/>
+    <origin xyz="-0.00179 -0.13516 0.01176" rpy="0 0 -1.57079"/>
   </xacro:sandia_hand>
   <xacro:sandia_hand side="left" parent="l_hand" reflect="-1" joint_type="revolute" thumb_angle="0">
