Commit message: adding hand camera xacro
generates hand cameras for left and right located at the center of the palm
added an april tag box

File: software/models/mit_gazebo_models/mit_robot/model_sim_v3_v1_inertia.urdf (robot description, URDF)
Before this commit: robot atlas, 74 links, 73 joints
Links:
- removed link left_finger_1_link_0
- removed link left_finger_1_link_1
- removed link left_finger_1_link_2
- removed link left_finger_1_link_3
- removed link left_finger_2_link_0
- removed link left_finger_2_link_1
- removed link left_finger_2_link_2
- removed link left_finger_2_link_3
- removed link left_finger_middle_link_0
- removed link left_finger_middle_link_1
- removed link left_finger_middle_link_2
- removed link left_finger_middle_link_3
- removed link left_palm
- removed link right_finger_1_link_0
- removed link right_finger_1_link_1
- removed link right_finger_1_link_2
- removed link right_finger_1_link_3
- removed link right_finger_2_link_0
- removed link right_finger_2_link_1
- removed link right_finger_2_link_2
- removed link right_finger_2_link_3
- removed link right_finger_middle_link_0
- removed link right_finger_middle_link_1
- removed link right_finger_middle_link_2
- removed link right_finger_middle_link_3
- removed link right_palm
- added link imu_link, mass 0.1; visual box size=0.01 0.01 0.01
- link head: geometry collision box size=0.0468 0.12 0.1184; collision box size=0.1311 0.12 0.0591
- link hokuyo_link: geometry collision box size=0.08 0.06 0.04238; collision cylinder length=0.047 radius=0.024425
- link l_clav: mass 3.45 -> 2.369; geometry collision mesh filename=package://atlas_description/meshes_v3/l_clav.stl scale=1 1 1; visual mesh filename=package://atlas_description/meshes_v3/l_clav.DAE scale=1 1 1
- link l_farm: mass 3.388 -> 0.981; geometry collision mesh filename=package://atlas_description/meshes_v3/l_farm.stl scale=1 1 1; visual mesh filename=package://atlas_description/meshes_v3/l_farm.DAE scale=1 1 1
- link l_foot: mass 2.05 -> 1.634; geometry collision mesh filename=package://atlas_description/meshes_v3/l_foot.stl scale=1 1 1; visual mesh filename=package://atlas_description/meshes_v3/l_foot.DAE scale=1 1 1
- link l_hand: mass 2.509 -> 2.263; geometry collision mesh filename=package://atlas_description/meshes_v3/l_hand.stl scale=1 1 1; visual mesh filename=package://atlas_description/meshes_v3/l_hand.DAE scale=1 1 1
- link l_larm: mass 2.509 -> 2.148; geometry collision mesh filename=package://atlas_description/meshes_v3/l_elbow_rx.stl scale=1 1 1; visual mesh filename=package://atlas_description/meshes_v3/l_elbow_rx.DAE scale=1 1 1
- link l_lglut: mass 0.866 -> 0.69; geometry collision mesh filename=package://atlas_description/meshes_v3/l_lglut.stl scale=1 1 1; visual mesh filename=package://atlas_description/meshes_v3/l_lglut.DAE scale=1 1 1
- link l_lleg: mass 5.479 -> 4.367; geometry collision mesh filename=package://atlas_description/meshes_v3/l_lleg.stl scale=1 1 1; visual mesh filename=package://atlas_description/meshes_v3/l_lleg.DAE scale=1 1 1
- link l_scap: mass 3.012 -> 2.707; geometry collision mesh filename=package://atlas_description/meshes_v3/l_sh_rx.stl scale=1 1 1; visual mesh filename=package://atlas_description/meshes_v3/l_sh_rx.DAE scale=1 1 1
- link l_talus: mass 0.125 -> 0.1; geometry collision mesh filename=package://atlas_description/meshes_v3/l_talus.stl scale=1 1 1; visual mesh filename=package://atlas_description/meshes_v3/l_talus.DAE scale=1 1 1
- link l_uarm: mass 3.388 -> 1.881; geometry collision mesh filename=package://atlas_description/meshes_v3/l_elbow_ry.stl scale=1 1 1; visual mesh filename=package://atlas_description/meshes_v3/l_elbow_ry.DAE scale=1 1 1
- link l_uglut: mass 0.648 -> 0.5166; geometry collision mesh filename=package://atlas_description/meshes_v3/l_uglut.stl scale=1 1 1; visual mesh filename=package://atlas_description/meshes_v3/l_uglut.DAE scale=1 1 1
- link l_uleg: mass 9.209 -> 7.34; geometry collision mesh filename=package://atlas_description/meshes_v3/l_uleg.stl scale=1 1 1; visual mesh filename=package://atlas_description/meshes_v3/l_uleg.DAE scale=1 1 1
- link ltorso: mass 2.409 -> 1.92; geometry collision mesh filename=package://atlas_description/meshes_v3/ltorso.stl scale=1 1 1; visual mesh filename=package://atlas_description/meshes_v3/ltorso.DAE scale=1 1 1
- link mtorso: mass 0.69 -> 0.55; geometry collision mesh filename=package://atlas_description/meshes_v3/mtorso.stl scale=1 1 1; visual mesh filename=package://atlas_description/meshes_v3/mtorso.DAE scale=1 1 1
- link pelvis: mass 17.882 -> 14.2529; geometry collision mesh filename=package://atlas_description/meshes_v3/pelvis.stl scale=1 1 1; visual mesh filename=package://atlas_description/meshes_v3/pelvis.DAE scale=1 1 1
- link r_clav: mass 3.45 -> 2.369; geometry collision mesh filename=package://atlas_description/meshes_v3/r_clav.stl scale=1 1 1; visual mesh filename=package://atlas_description/meshes_v3/r_clav.DAE scale=1 1 1
- link r_farm: mass 3.388 -> 0.981; geometry collision mesh filename=package://atlas_description/meshes_v3/r_farm.stl scale=1 1 1; visual mesh filename=package://atlas_description/meshes_v3/r_farm.DAE scale=1 1 1
- link r_foot: mass 2.05 -> 1.634; geometry collision mesh filename=package://atlas_description/meshes_v3/r_foot.stl scale=1 1 1; visual mesh filename=package://atlas_description/meshes_v3/r_foot.DAE scale=1 1 1
- link r_hand: mass 2.509 -> 2.263; geometry collision mesh filename=package://atlas_description/meshes_v3/r_hand.stl scale=1 1 1; visual mesh filename=package://atlas_description/meshes_v3/r_hand.DAE scale=1 1 1
- link r_larm: mass 2.509 -> 2.148; geometry collision mesh filename=package://atlas_description/meshes_v3/r_elbow_rx.stl scale=1 1 1; visual mesh filename=package://atlas_description/meshes_v3/r_elbow_rx.DAE scale=1 1 1
- link r_lglut: mass 0.866 -> 0.69; geometry collision mesh filename=package://atlas_description/meshes_v3/r_lglut.stl scale=1 1 1; visual mesh filename=package://atlas_description/meshes_v3/r_lglut.DAE scale=1 1 1
- link r_lleg: mass 5.479 -> 4.367; geometry collision mesh filename=package://atlas_description/meshes_v3/r_lleg.stl scale=1 1 1; visual mesh filename=package://atlas_description/meshes_v3/r_lleg.DAE scale=1 1 1
- link r_scap: mass 3.012 -> 2.707; geometry collision mesh filename=package://atlas_description/meshes_v3/r_sh_rx.stl scale=1 1 1; visual mesh filename=package://atlas_description/meshes_v3/r_sh_rx.DAE scale=1 1 1
- link r_talus: mass 0.125 -> 0.1; geometry collision mesh filename=package://atlas_description/meshes_v3/r_talus.stl scale=1 1 1; visual mesh filename=package://atlas_description/meshes_v3/r_talus.DAE scale=1 1 1
- link r_uarm: mass 3.388 -> 1.881; geometry collision mesh filename=package://atlas_description/meshes_v3/r_elbow_ry.stl scale=1 1 1; visual mesh filename=package://atlas_description/meshes_v3/r_elbow_ry.DAE scale=1 1 1
- link r_uglut: mass 0.648 -> 0.5166; geometry collision mesh filename=package://atlas_description/meshes_v3/r_uglut.stl scale=1 1 1; visual mesh filename=package://atlas_description/meshes_v3/r_uglut.DAE scale=1 1 1
- link r_uleg: mass 9.209 -> 7.34; geometry collision mesh filename=package://atlas_description/meshes_v3/r_uleg.stl scale=1 1 1; visual mesh filename=package://atlas_description/meshes_v3/r_uleg.DAE scale=1 1 1
- link utorso: mass 52.007 -> 18.484; geometry collision mesh filename=package://atlas_description/meshes_v3/utorso.stl scale=1 1 1; collision mesh filename=package://atlas_description/meshes_v3/utorso_pack.stl scale=1 1 1
Joints:
- removed joint l_arm_mwx
- removed joint l_arm_usy
- removed joint l_arm_uwy
- removed joint left_finger_1_joint_1
- removed joint left_finger_1_joint_2
- removed joint left_finger_1_joint_3
- removed joint left_finger_2_joint_1
- removed joint left_finger_2_joint_2
- removed joint left_finger_2_joint_3
- removed joint left_finger_middle_joint_1
- removed joint left_finger_middle_joint_2
- removed joint left_finger_middle_joint_3
- removed joint left_palm_finger_1_joint
- removed joint left_palm_finger_2_joint
- removed joint left_palm_finger_middle_joint
- removed joint left_robotiq_hand_joint
- removed joint neck_ay
- removed joint r_arm_mwx
- removed joint r_arm_usy
- removed joint r_arm_uwy
- removed joint right_finger_1_joint_1
- removed joint right_finger_1_joint_2
- removed joint right_finger_1_joint_3
- removed joint right_finger_2_joint_1
- removed joint right_finger_2_joint_2
- removed joint right_finger_2_joint_3
- removed joint right_finger_middle_joint_1
- removed joint right_finger_middle_joint_2
- removed joint right_finger_middle_joint_3
- removed joint right_palm_finger_1_joint
- removed joint right_palm_finger_2_joint
- removed joint right_palm_finger_middle_joint
- removed joint right_robotiq_hand_joint
- added joint imu_joint: type fixed, parent pelvis, child imu_link, origin xyz=0.05991527603 0 -0.01415 rpy=0 0 0
- added joint l_arm_shy: type revolute, parent utorso, child l_clav, origin xyz=0.06441 0.13866 0.10718 rpy=0 -0 0, axis 0 0.5 0.866025, limit lower=-1.5708 upper=0.785398 effort=212 velocity=12
- added joint l_arm_wrx: type revolute, parent l_farm, child l_hand, origin xyz=0 0.119 0.00921 rpy=0 -0 0, axis 1 0 0, limit lower=-1.1781 upper=1.1781 effort=60 velocity=12
- added joint l_arm_wry: type revolute, parent l_larm, child l_farm, origin xyz=0 0.187 -0.00921 rpy=0 -0 0, axis 0 1 0, limit lower=0 upper=3.14159 effort=114 velocity=12
- added joint neck_ry: type revolute, parent utorso, child head, origin xyz=0.21672 0 0.53796 rpy=0 -0 0, axis 0 1 0, limit lower=-0.602139 upper=1.14494 effort=5 velocity=12
- added joint r_arm_shy: type revolute, parent utorso, child r_clav, origin xyz=0.06441 -0.13866 0.10718 rpy=0 -0 0, axis 0 0.5 -0.866025, limit lower=-1.5708 upper=0.785398 effort=212 velocity=12
- added joint r_arm_wrx: type revolute, parent r_farm, child r_hand, origin xyz=0 -0.119 0.00921 rpy=0 -0 0, axis 1 0 0, limit lower=-1.1781 upper=1.1781 effort=60 velocity=12
- added joint r_arm_wry: type revolute, parent r_larm, child r_farm, origin xyz=0 -0.187 -0.00921 rpy=0 -0 0, axis 0 1 0, limit lower=0 upper=3.14159 effort=114 velocity=12
- joint back_bky: limit lower=-0.610691 upper=0.49 effort=206.843 velocity=12 -> lower=-0.610691 upper=0.438427 effort=206.843 velocity=12
- joint back_bkz: limit lower=-0.663225 upper=0.663225 effort=114 velocity=12 -> lower=-0.663225 upper=0.663225 effort=124.016 velocity=12
- joint l_arm_elx: limit lower=0 upper=2.35619 effort=55 velocity=12 -> lower=0 upper=2.35619 effort=114 velocity=12
- joint l_arm_ely: limit lower=0 upper=3.14159 effort=55 velocity=12 -> lower=0 upper=3.14159 effort=114 velocity=12
- joint l_arm_shx: limit lower=-1.5708 upper=1.5708 effort=107 velocity=12 -> lower=-1.5708 upper=1.5708 effort=170 velocity=12
- joint r_arm_elx: limit lower=-2.35619 upper=0 effort=55 velocity=12 -> lower=-2.35619 upper=0 effort=114 velocity=12
- joint r_arm_ely: limit lower=0 upper=3.14159 effort=55 velocity=12 -> lower=0 upper=3.14159 effort=114 velocity=12
- joint r_arm_shx: limit lower=-1.5708 upper=1.5708 effort=107 velocity=12 -> lower=-1.5708 upper=1.5708 effort=170 velocity=12

File: software/models/mit_gazebo_models/mit_robot/xacro/atlas_LR_RR.urdf.xacro (robot description, xacro)
@@ -10,3 +10,10 @@
     <origin rpy="0 1.57079 3.141" xyz="0 -0.19016 -0.015"/>
   </xacro:robotiq_hand>
+  <xacro:include filename="$(find robotiq_camera)/urdf/robotiq_camera.urdf.xacro" />
+  <xacro:robotiq_camera side="left" parent="l_hand" >
+    <origin xyz="0.0  0.25 0.0" rpy="-1.57079 0  1.57079"/>
+  </xacro:robotiq_camera>
+  <xacro:robotiq_camera side="right" parent="r_hand" >
+    <origin xyz="0.0  -0.25 0.0" rpy="-1.57079 3.14158 1.57079"/>
+  </xacro:robotiq_camera>
 </robot>
