Commit message: remaining changes from experiment 2014-02-24-camera-rhand-tabletop

File: software/models/mit_gazebo_models/mit_robot/model_LR_RR.urdf (robot description, URDF)
Before this commit: robot atlas, 74 links, 73 joints
Links:
- removed link head_imu_link
- added link post_spindle
- added link post_spindle_cal_pitch
- added link post_spindle_cal_roll
- added link post_spindle_cal_x
- added link post_spindle_cal_y
- added link post_spindle_cal_z
- added link pre_spindle
- added link pre_spindle_cal_pitch
- added link pre_spindle_cal_roll
- added link pre_spindle_cal_x
- added link pre_spindle_cal_y
- added link pre_spindle_cal_yaw
- added link pre_spindle_cal_z
- link center_bottom_led_frame: mass 1e-5 -> 0.1
- link center_top_led_frame: mass 1e-5 -> 0.1
- link head: mass 1.41984 -> 1.4199; geometry collision box size=0.1311 0.12 0.0591; visual mesh filename=package://multisense_sl/meshes/head.dae
- link head_hokuyo_frame: mass 1e-5 -> 0.01
- link hokuyo_link: mass 0.057654 -> 0.057664; geometry collision cylinder length=0.047 radius=0.024425; visual mesh filename=package://multisense_sl/meshes/head_camera.dae
- link left_camera_frame: mass 1e-5 -> 0.1
- link left_led_frame: mass 1e-5 -> 0.1
- link right_camera_frame: mass 1e-5 -> 0.1
- link right_led_frame: mass 1e-5 -> 0.1
Joints:
- removed joint head_imu_joint
- added joint post_spindle_cal_pitch_joint: type continuous, parent post_spindle_cal_roll, child post_spindle_cal_pitch, axis 0 1 0
- added joint post_spindle_cal_roll_joint: type continuous, parent post_spindle_cal_z, child post_spindle_cal_roll, axis 1 0 0
- added joint post_spindle_cal_x_joint: type prismatic, parent post_spindle, child post_spindle_cal_x, axis 1 0 0, limit lower=-0.5 upper=0.5 effort=0.0 velocity=0.0
- added joint post_spindle_cal_y_joint: type prismatic, parent post_spindle_cal_x, child post_spindle_cal_y, axis 0 1 0, limit lower=-0.5 upper=0.5 effort=0.0 velocity=0.0
- added joint post_spindle_cal_yaw_joint: type continuous, parent post_spindle_cal_pitch, child hokuyo_link, axis 0 0 1
- added joint post_spindle_cal_z_joint: type prismatic, parent post_spindle_cal_y, child post_spindle_cal_z, axis 0 0 1, limit lower=-0.5 upper=0.5 effort=0.0 velocity=0.0
- added joint pre_spindle_cal_pitch_joint: type continuous, parent pre_spindle_cal_roll, child pre_spindle_cal_pitch, axis 0 1 0
- added joint pre_spindle_cal_roll_joint: type continuous, parent pre_spindle_cal_z, child pre_spindle_cal_roll, axis 1 0 0
- added joint pre_spindle_cal_x_joint: type prismatic, parent pre_spindle, child pre_spindle_cal_x, axis 1 0 0, limit lower=-0.5 upper=0.5 effort=0.0 velocity=0.0
- added joint pre_spindle_cal_y_joint: type prismatic, parent pre_spindle_cal_x, child pre_spindle_cal_y, axis 0 1 0, limit lower=-0.5 upper=0.5 effort=0.0 velocity=0.0
- added joint pre_spindle_cal_yaw_joint: type continuous, parent pre_spindle_cal_pitch, child pre_spindle_cal_yaw, axis 0 0 1
- added joint pre_spindle_cal_z_joint: type prismatic, parent pre_spindle_cal_y, child pre_spindle_cal_z, axis 0 0 1, limit lower=-0.5 upper=0.5 effort=0.0 velocity=0.0
- added joint pre_spindle_joint: type fixed, parent head, child pre_spindle, origin xyz=-0.0446 0 0.0880 rpy=0 0 0, axis 0 1 0
- joint hokuyo_joint: child hokuyo_link -> post_spindle; origin xyz=-0.0446 0 0.0880 rpy=0 0 0 -> xyz=0 0 0 rpy=0 0 0; parent head -> pre_spindle_cal_yaw

File: software/models/mit_gazebo_models/mit_robot/xacro/atlas_LR_RR.urdf.xacro (robot description, xacro)
@@ -2,5 +2,5 @@
   <include filename="$(find mit_drcsim_scripts)/models/mit_robot/xacro/atlas_skeleton.urdf" />
   <include filename="$(find mit_drcsim_scripts)/models/mit_robot/xacro/atlas.transmission" />
-  <include filename="$(find mit_drcsim_scripts)/models/multisense_sl/multisense_sl_sim.urdf" />
+  <include filename="$(find mit_drcsim_scripts)/models/multisense_sl/multisense_sl.urdf" />
 <!--  left was  0 1.57079 0 -->
 <!-- right was  0 1.57079 3.141 -->

Commit message: remove multisense sim from atlas_LR_RR.urdf.xacro

File: software/models/mit_gazebo_models/mit_robot/model_LR_RR.urdf (robot description, URDF)
Before this commit: robot atlas, 80 links, 79 joints
Links:
- removed link head_imu_link
- added link post_spindle
- added link post_spindle_cal_pitch
- added link post_spindle_cal_roll
- added link post_spindle_cal_x
- added link post_spindle_cal_y
- added link post_spindle_cal_z
- added link pre_spindle
- added link pre_spindle_cal_pitch
- added link pre_spindle_cal_roll
- added link pre_spindle_cal_x
- added link pre_spindle_cal_y
- added link pre_spindle_cal_yaw
- added link pre_spindle_cal_z
- link center_bottom_led_frame: mass 1e-5 -> 0.1
- link center_top_led_frame: mass 1e-5 -> 0.1
- link head: mass 1.41984 -> 1.4199; geometry collision box size=0.1311 0.12 0.0591; visual mesh filename=package://multisense_sl/meshes/head.dae
- link head_hokuyo_frame: mass 1e-5 -> 0.01
- link hokuyo_link: mass 0.057654 -> 0.057664; geometry collision cylinder length=0.047 radius=0.024425; visual mesh filename=package://multisense_sl/meshes/head_camera.dae
- link left_camera_frame: mass 1e-5 -> 0.1
- link left_led_frame: mass 1e-5 -> 0.1
- link right_camera_frame: mass 1e-5 -> 0.1
- link right_led_frame: mass 1e-5 -> 0.1
Joints:
- removed joint head_imu_joint
- added joint post_spindle_cal_pitch_joint: type continuous, parent post_spindle_cal_roll, child post_spindle_cal_pitch, axis 0 1 0
- added joint post_spindle_cal_roll_joint: type continuous, parent post_spindle_cal_z, child post_spindle_cal_roll, axis 1 0 0
- added joint post_spindle_cal_x_joint: type prismatic, parent post_spindle, child post_spindle_cal_x, axis 1 0 0, limit lower=-0.5 upper=0.5 effort=0.0 velocity=0.0
- added joint post_spindle_cal_y_joint: type prismatic, parent post_spindle_cal_x, child post_spindle_cal_y, axis 0 1 0, limit lower=-0.5 upper=0.5 effort=0.0 velocity=0.0
- added joint post_spindle_cal_yaw_joint: type continuous, parent post_spindle_cal_pitch, child hokuyo_link, axis 0 0 1
- added joint post_spindle_cal_z_joint: type prismatic, parent post_spindle_cal_y, child post_spindle_cal_z, axis 0 0 1, limit lower=-0.5 upper=0.5 effort=0.0 velocity=0.0
- added joint pre_spindle_cal_pitch_joint: type continuous, parent pre_spindle_cal_roll, child pre_spindle_cal_pitch, axis 0 1 0
- added joint pre_spindle_cal_roll_joint: type continuous, parent pre_spindle_cal_z, child pre_spindle_cal_roll, axis 1 0 0
- added joint pre_spindle_cal_x_joint: type prismatic, parent pre_spindle, child pre_spindle_cal_x, axis 1 0 0, limit lower=-0.5 upper=0.5 effort=0.0 velocity=0.0
- added joint pre_spindle_cal_y_joint: type prismatic, parent pre_spindle_cal_x, child pre_spindle_cal_y, axis 0 1 0, limit lower=-0.5 upper=0.5 effort=0.0 velocity=0.0
- added joint pre_spindle_cal_yaw_joint: type continuous, parent pre_spindle_cal_pitch, child pre_spindle_cal_yaw, axis 0 0 1
- added joint pre_spindle_cal_z_joint: type prismatic, parent pre_spindle_cal_y, child pre_spindle_cal_z, axis 0 0 1, limit lower=-0.5 upper=0.5 effort=0.0 velocity=0.0
- added joint pre_spindle_joint: type fixed, parent head, child pre_spindle, origin xyz=-0.0446 0 0.0880 rpy=0 0 0, axis 0 1 0
- joint hokuyo_joint: child hokuyo_link -> post_spindle; origin xyz=-0.0446 0 0.0880 rpy=0 0 0 -> xyz=0 0 0 rpy=0 0 0; parent head -> pre_spindle_cal_yaw

File: software/models/mit_gazebo_models/mit_robot/xacro/atlas_LR_RR.urdf.xacro (robot description, xacro)
@@ -2,6 +2,5 @@
   <include filename="$(find mit_drcsim_scripts)/models/mit_robot/xacro/atlas_skeleton.urdf" />
   <include filename="$(find mit_drcsim_scripts)/models/mit_robot/xacro/atlas.transmission" />
-<!--  <include filename="$(find mit_drcsim_scripts)/models/multisense_sl/multisense_sl.urdf" /> -->
-  <include filename="$(find mit_drcsim_scripts)/models/multisense_sl/multisense_sl_sim.urdf" />
+  <include filename="$(find mit_drcsim_scripts)/models/multisense_sl/multisense_sl.urdf" />
   <include filename="$(find mit_drcsim_scripts)/models/mit_robot/xacro/hand_force_torque.urdf" />
   <xacro:include filename="$(find robotiq_hand_description)/cfg/robotiq_hand.urdf.xacro" />
