Commit message: adding support for bdi hooks
git-svn-id: https://svn.csail.mit.edu/drc/trunk@7722 c7283977-0100-402a-a91a-fa70b306dbfe

File: software/models/mit_gazebo_models/mit_robot/model_LH_RH.urdf (robot description, URDF)
Before this commit: robot atlas, 66 links, 65 joints
Links:
- removed link right_finger[0]/base_rotation_link
- removed link right_finger[0]/distal_link
- removed link right_finger[0]/proximal_link
- removed link right_finger[1]/base_rotation_link
- removed link right_finger[1]/distal_link
- removed link right_finger[1]/proximal_link
- removed link right_finger[2]/distal_link
- removed link right_finger[2]/proximal_link
- link right_base_link: geometry collision cylinder length=0.01 radius=0.045; collision cylinder length=0.04 radius=0.006
Joints:
- removed joint right_finger[0]/joint_base
- removed joint right_finger[0]/joint_base_rotation
- removed joint right_finger[0]/joint_flex
- removed joint right_finger[1]/joint_base
- removed joint right_finger[1]/joint_base_rotation
- removed joint right_finger[1]/joint_flex
- removed joint right_finger[2]/joint_base
- removed joint right_finger[2]/joint_flex
- removed joint right_irobot_hand_joint
- added joint right_hook_hand_joint: type fixed, parent r_hand, child right_base_link, origin xyz=0 -0.11516 -0.015 rpy=1.57079 0 0

File: software/models/mit_gazebo_models/mit_robot/model_LH_RN.urdf (robot description, URDF)
Before this commit: robot atlas, 66 links, 65 joints
Links:
- removed link right_base_link
- removed link right_finger[0]/base_rotation_link
- removed link right_finger[0]/distal_link
- removed link right_finger[0]/proximal_link
- removed link right_finger[1]/base_rotation_link
- removed link right_finger[1]/distal_link
- removed link right_finger[1]/proximal_link
- removed link right_finger[2]/distal_link
- removed link right_finger[2]/proximal_link
Joints:
- removed joint right_finger[0]/joint_base
- removed joint right_finger[0]/joint_base_rotation
- removed joint right_finger[0]/joint_flex
- removed joint right_finger[1]/joint_base
- removed joint right_finger[1]/joint_base_rotation
- removed joint right_finger[1]/joint_flex
- removed joint right_finger[2]/joint_base
- removed joint right_finger[2]/joint_flex
- removed joint right_irobot_hand_joint

File: software/models/mit_gazebo_models/mit_robot/model_LN_RH.urdf (robot description, URDF)
Before this commit: robot atlas, 66 links, 65 joints
Links:
- removed link left_base_link
- removed link right_finger[0]/base_rotation_link
- removed link right_finger[0]/distal_link
- removed link right_finger[0]/proximal_link
- removed link right_finger[1]/base_rotation_link
- removed link right_finger[1]/distal_link
- removed link right_finger[1]/proximal_link
- removed link right_finger[2]/distal_link
- removed link right_finger[2]/proximal_link
- link right_base_link: geometry collision cylinder length=0.01 radius=0.045; collision cylinder length=0.04 radius=0.006
Joints:
- removed joint left_hook_hand_joint
- removed joint right_finger[0]/joint_base
- removed joint right_finger[0]/joint_base_rotation
- removed joint right_finger[0]/joint_flex
- removed joint right_finger[1]/joint_base
- removed joint right_finger[1]/joint_base_rotation
- removed joint right_finger[1]/joint_flex
- removed joint right_finger[2]/joint_base
- removed joint right_finger[2]/joint_flex
- removed joint right_irobot_hand_joint
- added joint right_hook_hand_joint: type fixed, parent r_hand, child right_base_link, origin xyz=0 -0.11516 -0.015 rpy=1.57079 0 0

File: software/models/mit_gazebo_models/mit_robot/xacro/atlas_LH_RH.urdf.xacro (robot description, xacro)
@@ -3,10 +3,9 @@
   <include filename="$(find mit_drcsim_scripts)/models/mit_robot/xacro/atlas.transmission" />
   <include filename="$(find mit_drcsim_scripts)/models/multisense_sl/multisense_sl.urdf" />
-  <xacro:include filename="$(find handle_description)/src/irobot_hand_simple.urdf.xacro" />
  <xacro:include filename="$(find hook_description)/src/hook_hand_simple.urdf.xacro" />
 <!--    <xacro:include filename="$(find hook_description)/src/bdihook_hand.urdf.xacro" />-->
-  <xacro:irobot_hand side="right" parent="r_hand" reflect="1">
+  <xacro:hook_hand side="right" parent="r_hand" reflect="1" hookflip="1">
     <origin rpy="1.57079 0 0" xyz="0 -0.11516 -0.015"/>
-  </xacro:irobot_hand>
+  </xacro:hook_hand>
   <xacro:hook_hand side="left" parent="l_hand" reflect="-1" hookflip="1">
     <origin rpy="1.57079 3.14159 3.14159" xyz="0 0.11516 0.015"/>

File: software/models/mit_gazebo_models/mit_robot/xacro/atlas_LH_RN.urdf.xacro (robot description, xacro)
@@ -3,10 +3,6 @@
   <include filename="$(find mit_drcsim_scripts)/models/mit_robot/xacro/atlas.transmission" />
   <include filename="$(find mit_drcsim_scripts)/models/multisense_sl/multisense_sl.urdf" />
-  <xacro:include filename="$(find handle_description)/src/irobot_hand_simple.urdf.xacro" />
  <xacro:include filename="$(find hook_description)/src/hook_hand_simple.urdf.xacro" />
 <!--    <xacro:include filename="$(find hook_description)/src/bdihook_hand.urdf.xacro" />-->
-  <xacro:irobot_hand side="right" parent="r_hand" reflect="1">
-    <origin rpy="1.57079 0 0" xyz="0 -0.11516 -0.015"/>
-  </xacro:irobot_hand>
   <xacro:hook_hand side="left" parent="l_hand" reflect="-1" hookflip="1">
     <origin rpy="1.57079 3.14159 3.14159" xyz="0 0.11516 0.015"/>

File: software/models/mit_gazebo_models/mit_robot/xacro/atlas_LN_RH.urdf.xacro (robot description, xacro)
@@ -3,12 +3,8 @@
   <include filename="$(find mit_drcsim_scripts)/models/mit_robot/xacro/atlas.transmission" />
   <include filename="$(find mit_drcsim_scripts)/models/multisense_sl/multisense_sl.urdf" />
-  <xacro:include filename="$(find handle_description)/src/irobot_hand_simple.urdf.xacro" />
  <xacro:include filename="$(find hook_description)/src/hook_hand_simple.urdf.xacro" />
 <!--    <xacro:include filename="$(find hook_description)/src/bdihook_hand.urdf.xacro" />-->
-  <xacro:irobot_hand side="right" parent="r_hand" reflect="1">
+  <xacro:hook_hand side="right" parent="r_hand" reflect="1" hookflip="1">
     <origin rpy="1.57079 0 0" xyz="0 -0.11516 -0.015"/>
-  </xacro:irobot_hand>
-  <xacro:hook_hand side="left" parent="l_hand" reflect="-1" hookflip="1">
-    <origin rpy="1.57079 3.14159 3.14159" xyz="0 0.11516 0.015"/>
   </xacro:hook_hand>
 </robot>

Commit message: increasing back-y upper joint limit
git-svn-id: https://svn.csail.mit.edu/drc/trunk@7751 c7283977-0100-402a-a91a-fa70b306dbfe

File: software/models/mit_gazebo_models/mit_robot/model_LH_RH.urdf (robot description, URDF)
Before this commit: robot atlas, 58 links, 57 joints
Joints:
- joint back_bky: limit lower=-0.610691 upper=0.438427 effort=206.843 velocity=12 -> lower=-0.610691 upper=0.49 effort=206.843 velocity=12

File: software/models/mit_gazebo_models/mit_robot/model_LH_RI.urdf (robot description, URDF)
Before this commit: robot atlas, 66 links, 65 joints
Joints:
- joint back_bky: limit lower=-0.610691 upper=0.438427 effort=206.843 velocity=12 -> lower=-0.610691 upper=0.49 effort=206.843 velocity=12

File: software/models/mit_gazebo_models/mit_robot/model_LH_RN.urdf (robot description, URDF)
Before this commit: robot atlas, 57 links, 56 joints
Joints:
- joint back_bky: limit lower=-0.610691 upper=0.438427 effort=206.843 velocity=12 -> lower=-0.610691 upper=0.49 effort=206.843 velocity=12

File: software/models/mit_gazebo_models/mit_robot/model_LH_RR.urdf (robot description, URDF)
Before this commit: robot atlas, 66 links, 65 joints
Joints:
- joint back_bky: limit lower=-0.610691 upper=0.438427 effort=206.843 velocity=12 -> lower=-0.610691 upper=0.49 effort=206.843 velocity=12

File: software/models/mit_gazebo_models/mit_robot/model_LN_RH.urdf (robot description, URDF)
Before this commit: robot atlas, 57 links, 56 joints
Joints:
- joint back_bky: limit lower=-0.610691 upper=0.438427 effort=206.843 velocity=12 -> lower=-0.610691 upper=0.49 effort=206.843 velocity=12

File: software/models/mit_gazebo_models/mit_robot/model_LN_RR.urdf (robot description, URDF)
Before this commit: robot atlas, 69 links, 68 joints
Joints:
- joint back_bky: limit lower=-0.610691 upper=0.438427 effort=206.843 velocity=12 -> lower=-0.610691 upper=0.49 effort=206.843 velocity=12

File: software/models/mit_gazebo_models/mit_robot/model_LR_RN.urdf (robot description, URDF)
Before this commit: robot atlas, 69 links, 68 joints
Joints:
- joint back_bky: limit lower=-0.610691 upper=0.438427 effort=206.843 velocity=12 -> lower=-0.610691 upper=0.49 effort=206.843 velocity=12

File: software/models/mit_gazebo_models/mit_robot/model_sim.urdf (robot description, URDF)
Before this commit: robot atlas, 111 links, 110 joints
Joints:
- joint back_bky: limit lower=-0.610691 upper=0.438427 effort=206.843 velocity=12 -> lower=-0.610691 upper=0.49 effort=206.843 velocity=12

File: software/models/mit_gazebo_models/mit_robot/model_sim_gazebo.urdf (robot description, URDF)
Before this commit: robot atlas, 111 links, 110 joints
Joints:
- joint back_mby: limit lower=-0.610691 upper=0.438427 effort=206.843 velocity=12 -> lower=-0.610691 upper=0.49 effort=206.843 velocity=12

File: software/models/mit_gazebo_models/mit_robot/xacro/atlas_skeleton.urdf (robot description, URDF)
Before this commit: robot drc_skeleton, 32 links, 32 joints
Joints:
- joint back_bky: limit lower=-0.610691 upper=0.438427 effort=206.843 velocity=12 -> lower=-0.610691 upper=0.49 effort=206.843 velocity=12

File: software/models/mit_gazebo_models/mit_robot_drake/model.urdf (robot description, URDF)
Before this commit: robot atlas, 95 links, 94 joints
Joints:
- joint back_bky: limit lower=-0.610691 upper=0.438427 effort=206.843 velocity=12 -> lower=-0.610691 upper=0.49 effort=206.843 velocity=12

File: software/models/mit_gazebo_models/mit_robot_drake/model_minimal_contact.urdf (robot description, URDF)
Before this commit: robot atlas, 29 links, 28 joints
Joints:
- joint back_bky: limit lower=-0.610691 upper=0.438427 effort=206.843 velocity=12 -> lower=-0.610691 upper=0.49 effort=206.843 velocity=12

File: software/models/mit_gazebo_models/mit_robot_drake/model_minimal_contact_fixedjoint_hands.urdf (robot description, URDF)
Before this commit: robot atlas, 95 links, 94 joints
Joints:
- joint back_bky: limit lower=-0.610691 upper=0.438427 effort=206.843 velocity=12 -> lower=-0.610691 upper=0.49 effort=206.843 velocity=12

File: software/models/mit_gazebo_models/mit_robot_drake/model_minimal_contact_point_hands.urdf (robot description, URDF)
Before this commit: robot atlas, 31 links, 30 joints
Joints:
- joint back_bky: limit lower=-0.610691 upper=0.438427 effort=206.843 velocity=12 -> lower=-0.610691 upper=0.49 effort=206.843 velocity=12

File: software/models/mit_gazebo_models/mit_robot_drake/model_minimal_contact_point_stumps.urdf (robot description, URDF)
Before this commit: robot atlas, 31 links, 30 joints
Joints:
- joint back_bky: limit lower=-0.610691 upper=0.438427 effort=206.843 velocity=12 -> lower=-0.610691 upper=0.49 effort=206.843 velocity=12

File: software/models/mit_gazebo_models/mit_robot_drake/xacro/atlas_skeleton.urdf (robot description, URDF)
Before this commit: robot drc_skeleton, 28 links, 28 joints
Joints:
- joint back_bky: limit lower=-0.610691 upper=0.438427 effort=206.843 velocity=12 -> lower=-0.610691 upper=0.49 effort=206.843 velocity=12

File: software/models/mit_gazebo_models/mit_robot_drake/xacro/atlas_skeleton_minimal_contact.urdf (robot description, URDF)
Before this commit: robot drc_skeleton, 28 links, 28 joints
Joints:
- joint back_bky: limit lower=-0.610691 upper=0.438427 effort=206.843 velocity=12 -> lower=-0.610691 upper=0.49 effort=206.843 velocity=12

Commit message: adding new config for robotiq and hooks
git-svn-id: https://svn.csail.mit.edu/drc/trunk@7773 c7283977-0100-402a-a91a-fa70b306dbfe

File: software/models/mit_gazebo_models/mit_robot/model_LH_RH.urdf (robot description, URDF)
Before this commit: robot atlas, 58 links, 57 joints
Links:
- link left_base_link: geometry collision mesh filename=package://hook_description/meshes/bdi_hook.stl scale=0.001 0.001 0.001; visual mesh filename=package://hook_description/meshes/bdi_hook.stl scale=1 1 1
- link right_base_link: geometry collision mesh filename=package://hook_description/meshes/bdi_hook.stl scale=0.001 0.001 0.001; visual mesh filename=package://hook_description/meshes/bdi_hook.stl scale=1 1 1

File: software/models/mit_gazebo_models/mit_robot/model_LH_RI.urdf (robot description, URDF)
Before this commit: robot atlas, 66 links, 65 joints
Links:
- link left_base_link: geometry collision mesh filename=package://hook_description/meshes/bdi_hook.stl scale=0.001 0.001 0.001; visual mesh filename=package://hook_description/meshes/bdi_hook.stl scale=1 1 1

File: software/models/mit_gazebo_models/mit_robot/model_LH_RN.urdf (robot description, URDF)
Before this commit: robot atlas, 57 links, 56 joints
Links:
- link left_base_link: geometry collision mesh filename=package://hook_description/meshes/bdi_hook.stl scale=0.001 0.001 0.001; visual mesh filename=package://hook_description/meshes/bdi_hook.stl scale=1 1 1

File: software/models/mit_gazebo_models/mit_robot/model_LH_RR.urdf (robot description, URDF)
Before this commit: robot atlas, 66 links, 65 joints
Links:
- link left_base_link: geometry collision mesh filename=package://hook_description/meshes/bdi_hook.stl scale=0.001 0.001 0.001; visual mesh filename=package://hook_description/meshes/bdi_hook.stl scale=1 1 1

File: software/models/mit_gazebo_models/mit_robot/model_LI_RI.urdf (robot description, URDF)
Before this commit: robot atlas, 74 links, 73 joints
Joints:
- joint back_bky: limit lower=-0.610691 upper=0.438427 effort=206.843 velocity=12 -> lower=-0.610691 upper=0.49 effort=206.843 velocity=12

File: software/models/mit_gazebo_models/mit_robot/model_LI_RN.urdf (robot description, URDF)
Before this commit: robot atlas, 65 links, 64 joints
Joints:
- joint back_bky: limit lower=-0.610691 upper=0.438427 effort=206.843 velocity=12 -> lower=-0.610691 upper=0.49 effort=206.843 velocity=12

File: software/models/mit_gazebo_models/mit_robot/model_LI_RS.urdf (robot description, URDF)
Before this commit: robot atlas, 98 links, 97 joints
Joints:
- joint back_bky: limit lower=-0.610691 upper=0.438427 effort=206.843 velocity=12 -> lower=-0.610691 upper=0.49 effort=206.843 velocity=12

File: software/models/mit_gazebo_models/mit_robot/model_LN_RH.urdf (robot description, URDF)
Before this commit: robot atlas, 57 links, 56 joints
Links:
- link right_base_link: geometry collision mesh filename=package://hook_description/meshes/bdi_hook.stl scale=0.001 0.001 0.001; visual mesh filename=package://hook_description/meshes/bdi_hook.stl scale=1 1 1

File: software/models/mit_gazebo_models/mit_robot/model_LN_RI.urdf (robot description, URDF)
Before this commit: robot atlas, 65 links, 64 joints
Joints:
- joint back_bky: limit lower=-0.610691 upper=0.438427 effort=206.843 velocity=12 -> lower=-0.610691 upper=0.49 effort=206.843 velocity=12

File: software/models/mit_gazebo_models/mit_robot/model_LN_RN.urdf (robot description, URDF)
Before this commit: robot atlas, 57 links, 56 joints
Joints:
- joint back_bky: limit lower=-0.610691 upper=0.438427 effort=206.843 velocity=12 -> lower=-0.610691 upper=0.49 effort=206.843 velocity=12

File: software/models/mit_gazebo_models/mit_robot/model_LN_RS.urdf (robot description, URDF)
Before this commit: robot atlas, 89 links, 88 joints
Joints:
- joint back_bky: limit lower=-0.610691 upper=0.438427 effort=206.843 velocity=12 -> lower=-0.610691 upper=0.49 effort=206.843 velocity=12

File: software/models/mit_gazebo_models/mit_robot/model_LS_RI.urdf (robot description, URDF)
Before this commit: robot atlas, 98 links, 97 joints
Joints:
- joint back_bky: limit lower=-0.610691 upper=0.438427 effort=206.843 velocity=12 -> lower=-0.610691 upper=0.49 effort=206.843 velocity=12

File: software/models/mit_gazebo_models/mit_robot/model_LS_RN.urdf (robot description, URDF)
Before this commit: robot atlas, 89 links, 88 joints
Joints:
- joint back_bky: limit lower=-0.610691 upper=0.438427 effort=206.843 velocity=12 -> lower=-0.610691 upper=0.49 effort=206.843 velocity=12

File: software/models/mit_gazebo_models/mit_robot/model_LS_RS.urdf (robot description, URDF)
Before this commit: robot atlas, 122 links, 121 joints
Joints:
- joint back_bky: limit lower=-0.610691 upper=0.438427 effort=206.843 velocity=12 -> lower=-0.610691 upper=0.49 effort=206.843 velocity=12

File: software/models/mit_gazebo_models/mit_robot/xacro/atlas_LH_RH.urdf.xacro (robot description, xacro)
@@ -3,6 +3,5 @@
   <include filename="$(find mit_drcsim_scripts)/models/mit_robot/xacro/atlas.transmission" />
   <include filename="$(find mit_drcsim_scripts)/models/multisense_sl/multisense_sl.urdf" />
- <xacro:include filename="$(find hook_description)/src/hook_hand_simple.urdf.xacro" />
- <!--<xacro:include filename="$(find hook_description)/src/bdihook_hand.urdf.xacro" />-->
+ <xacro:include filename="$(find hook_description)/src/bdihook_hand.urdf.xacro" />
   <xacro:hook_hand side="right" parent="r_hand" reflect="1" hookflip="1">
     <origin rpy="1.57079 0 0" xyz="0 -0.11516 -0.015"/>

File: software/models/mit_gazebo_models/mit_robot/xacro/atlas_LH_RI.urdf.xacro (robot description, xacro)
@@ -4,6 +4,5 @@
   <include filename="$(find mit_drcsim_scripts)/models/multisense_sl/multisense_sl.urdf" />
   <xacro:include filename="$(find handle_description)/src/irobot_hand_simple.urdf.xacro" />
- <xacro:include filename="$(find hook_description)/src/hook_hand_simple.urdf.xacro" />
- <!-- <xacro:include filename="$(find hook_description)/src/bdihook_hand.urdf.xacro" />-->
+ <xacro:include filename="$(find hook_description)/src/bdihook_hand.urdf.xacro" />
   <xacro:irobot_hand side="right" parent="r_hand" reflect="1">
     <origin rpy="1.57079 0 0" xyz="0 -0.11516 -0.015"/>

File: software/models/mit_gazebo_models/mit_robot/xacro/atlas_LH_RN.urdf.xacro (robot description, xacro)
@@ -3,6 +3,5 @@
   <include filename="$(find mit_drcsim_scripts)/models/mit_robot/xacro/atlas.transmission" />
   <include filename="$(find mit_drcsim_scripts)/models/multisense_sl/multisense_sl.urdf" />
-  <xacro:include filename="$(find hook_description)/src/hook_hand_simple.urdf.xacro" />
-<!-- <xacro:include filename="$(find hook_description)/src/bdihook_hand.urdf.xacro" />-->
+  <xacro:include filename="$(find hook_description)/src/bdihook_hand.urdf.xacro" />
   <xacro:hook_hand side="left" parent="l_hand" reflect="-1" hookflip="1">
     <origin rpy="1.57079 3.14159 3.14159" xyz="0 0.11516 0.015"/>

File: software/models/mit_gazebo_models/mit_robot/xacro/atlas_LH_RR.urdf.xacro (robot description, xacro)
@@ -4,6 +4,5 @@
   <include filename="$(find mit_drcsim_scripts)/models/multisense_sl/multisense_sl.urdf" />
   <xacro:include filename="$(find handle_description)/src/irobot_hand_simple.urdf.xacro" />
- <xacro:include filename="$(find hook_description)/src/hook_hand_simple.urdf.xacro" />
-<!--    <xacro:include filename="$(find hook_description)/src/bdihook_hand.urdf.xacro" />-->
+  <xacro:include filename="$(find hook_description)/src/bdihook_hand.urdf.xacro" />
   <xacro:irobot_hand side="right" parent="r_hand" reflect="1">
     <origin rpy="1.57079 2.0944 0" xyz="0 -0.11516 -0.015"/>

File: software/models/mit_gazebo_models/mit_robot/xacro/atlas_LN_RH.urdf.xacro (robot description, xacro)
@@ -4,5 +4,5 @@
   <include filename="$(find mit_drcsim_scripts)/models/multisense_sl/multisense_sl.urdf" />
  <xacro:include filename="$(find hook_description)/src/hook_hand_simple.urdf.xacro" />
-<!--    <xacro:include filename="$(find hook_description)/src/bdihook_hand.urdf.xacro" />-->
+ <xacro:include filename="$(find hook_description)/src/bdihook_hand.urdf.xacro" />
   <xacro:hook_hand side="right" parent="r_hand" reflect="1" hookflip="1">
     <origin rpy="1.57079 0 0" xyz="0 -0.11516 -0.015"/>

File: software/models/mit_gazebo_models/mit_robot_hands/inert_hand_left.urdf (robot description, URDF)
Before this commit: robot inert_hand_left, 2 links, 1 joints
Links:
- link left_base_link: geometry collision mesh filename=package://hook_description/meshes/bdi_hook.stl scale=0.001 0.001 0.001; visual mesh filename=package://hook_description/meshes/bdi_hook.stl scale=1 1 1
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
Commit message: collision element of bdi hook had wrong scaling
git-svn-id: https://svn.csail.mit.edu/drc/trunk@7828 c7283977-0100-402a-a91a-fa70b306dbfe

File: software/models/mit_gazebo_models/mit_robot/model_LH_RH.urdf (robot description, URDF)
Before this commit: robot atlas, 58 links, 57 joints
Links:
- link left_base_link: geometry collision mesh filename=package://hook_description/meshes/bdi_hook.stl scale=1 1 1; visual mesh filename=package://hook_description/meshes/bdi_hook.stl scale=1 1 1
- link right_base_link: geometry collision mesh filename=package://hook_description/meshes/bdi_hook.stl scale=1 1 1; visual mesh filename=package://hook_description/meshes/bdi_hook.stl scale=1 1 1

File: software/models/mit_gazebo_models/mit_robot/model_LH_RI.urdf (robot description, URDF)
Before this commit: robot atlas, 66 links, 65 joints
Links:
- link left_base_link: geometry collision mesh filename=package://hook_description/meshes/bdi_hook.stl scale=1 1 1; visual mesh filename=package://hook_description/meshes/bdi_hook.stl scale=1 1 1

File: software/models/mit_gazebo_models/mit_robot/model_LH_RN.urdf (robot description, URDF)
Before this commit: robot atlas, 57 links, 56 joints
Links:
- link left_base_link: geometry collision mesh filename=package://hook_description/meshes/bdi_hook.stl scale=1 1 1; visual mesh filename=package://hook_description/meshes/bdi_hook.stl scale=1 1 1

File: software/models/mit_gazebo_models/mit_robot/model_LN_RH.urdf (robot description, URDF)
Before this commit: robot atlas, 57 links, 56 joints
Links:
- link right_base_link: geometry collision mesh filename=package://hook_description/meshes/bdi_hook.stl scale=1 1 1; visual mesh filename=package://hook_description/meshes/bdi_hook.stl scale=1 1 1

File: software/models/mit_gazebo_models/mit_robot/xacro/atlas_LH_RH.urdf.xacro (robot description, xacro)
@@ -4,8 +4,8 @@
   <include filename="$(find mit_drcsim_scripts)/models/multisense_sl/multisense_sl.urdf" />
  <xacro:include filename="$(find hook_description)/src/bdihook_hand.urdf.xacro" />
-  <xacro:hook_hand side="right" parent="r_hand" reflect="1" hookflip="1">
+  <xacro:hook_hand side="right" parent="r_hand" reflect="1" hookflip="-1">
     <origin rpy="1.57079 0 0" xyz="0 -0.11516 -0.015"/>
   </xacro:hook_hand>
-  <xacro:hook_hand side="left" parent="l_hand" reflect="-1" hookflip="1">
+  <xacro:hook_hand side="left" parent="l_hand" reflect="-1" hookflip="-1">
     <origin rpy="1.57079 3.14159 3.14159" xyz="0 0.11516 0.015"/>
   </xacro:hook_hand>
