Commit message: updating joint limits for new back-y actuator

File: software/models/mit_gazebo_models/mit_robot/model_LH_RH.urdf (robot description, URDF)
Before this commit: robot atlas, 58 links, 57 joints
Joints:
- joint back_bky: limit lower=-0.610691 upper=0.49 effort=206.843 velocity=12 -> lower=-0.262 upper=0.524 effort=206.843 velocity=12

File: software/models/mit_gazebo_models/mit_robot/model_LI_RI.urdf (robot description, URDF)
Before this commit: robot atlas, 74 links, 73 joints
Joints:
- joint back_bky: limit lower=-0.610691 upper=0.49 effort=206.843 velocity=12 -> lower=-0.262 upper=0.524 effort=206.843 velocity=12

File: software/models/mit_gazebo_models/mit_robot/model_LI_RR.urdf (robot description, URDF)
Before this commit: robot atlas, 78 links, 77 joints
Joints:
- joint back_bky: limit lower=-0.610691 upper=0.49 effort=206.843 velocity=12 -> lower=-0.262 upper=0.524 effort=206.843 velocity=12

File: software/models/mit_gazebo_models/mit_robot/model_LI_RR_extender.urdf (robot description, URDF)
Before this commit: robot atlas, 80 links, 79 joints
Joints:
- joint back_bky: limit lower=-0.610691 upper=0.49 effort=206.843 velocity=12 -> lower=-0.262 upper=0.524 effort=206.843 velocity=12

File: software/models/mit_gazebo_models/mit_robot/model_LP_RP.urdf (robot description, URDF)
Before this commit: robot atlas, 58 links, 57 joints
Joints:
- joint back_bky: limit lower=-0.610691 upper=0.49 effort=206.843 velocity=12 -> lower=-0.262 upper=0.524 effort=206.843 velocity=12

File: software/models/mit_gazebo_models/mit_robot/model_LP_RR.urdf (robot description, URDF)
Before this commit: robot atlas, 70 links, 69 joints
Joints:
- joint back_bky: limit lower=-0.610691 upper=0.49 effort=206.843 velocity=12 -> lower=-0.262 upper=0.524 effort=206.843 velocity=12

File: software/models/mit_gazebo_models/mit_robot/model_LQ_RP.urdf (robot description, URDF)
Before this commit: robot atlas, 71 links, 70 joints
Joints:
- joint back_bky: limit lower=-0.610691 upper=0.49 effort=206.843 velocity=12 -> lower=-0.262 upper=0.524 effort=206.843 velocity=12

File: software/models/mit_gazebo_models/mit_robot/model_LR_RR.urdf (robot description, URDF)
Before this commit: robot atlas, 70 links, 69 joints
Joints:
- joint back_bky: limit lower=-0.610691 upper=0.49 effort=206.843 velocity=12 -> lower=-0.262 upper=0.524 effort=206.843 velocity=12

File: software/models/mit_gazebo_models/mit_robot/model_sim.urdf (robot description, URDF)
Before this commit: robot atlas, 111 links, 110 joints
Joints:
- joint back_bky: limit lower=-0.610691 upper=0.49 effort=206.843 velocity=12 -> lower=-0.262 upper=0.524 effort=206.843 velocity=12

File: software/models/mit_gazebo_models/mit_robot/model_sim_gazebo.urdf (robot description, URDF)
Before this commit: robot atlas, 111 links, 110 joints
Joints:
- joint back_mby: limit lower=-0.610691 upper=0.49 effort=206.843 velocity=12 -> lower=-0.262 upper=0.524 effort=206.843 velocity=12

File: software/models/mit_gazebo_models/mit_robot/xacro/atlas_skeleton.urdf (robot description, URDF)
Before this commit: robot drc_skeleton, 32 links, 32 joints
Joints:
- joint back_bky: limit lower=-0.610691 upper=0.49 effort=206.843 velocity=12 -> lower=-0.262 upper=0.524 effort=206.843 velocity=12

File: software/models/mit_gazebo_models/mit_robot_drake/model.urdf (robot description, URDF)
Before this commit: robot atlas, 95 links, 94 joints
Joints:
- joint back_bky: limit lower=-0.610691 upper=0.49 effort=206.843 velocity=12 -> lower=-0.262 upper=0.524 effort=206.843 velocity=12

File: software/models/mit_gazebo_models/mit_robot_drake/model_minimal_contact.urdf (robot description, URDF)
Before this commit: robot atlas, 29 links, 28 joints
Joints:
- joint back_bky: limit lower=-0.610691 upper=0.49 effort=206.843 velocity=12 -> lower=-0.262 upper=0.524 effort=206.843 velocity=12

File: software/models/mit_gazebo_models/mit_robot_drake/model_minimal_contact_fixedjoint_hands.urdf (robot description, URDF)
Before this commit: robot atlas, 95 links, 94 joints
Joints:
- joint back_bky: limit lower=-0.610691 upper=0.49 effort=206.843 velocity=12 -> lower=-0.262 upper=0.524 effort=206.843 velocity=12

File: software/models/mit_gazebo_models/mit_robot_drake/model_minimal_contact_point_hands.urdf (robot description, URDF)
Before this commit: robot atlas, 31 links, 30 joints
Joints:
- joint back_bky: limit lower=-0.610691 upper=0.49 effort=206.843 velocity=12 -> lower=-0.262 upper=0.524 effort=206.843 velocity=12

File: software/models/mit_gazebo_models/mit_robot_drake/model_minimal_contact_point_stumps.urdf (robot description, URDF)
Before this commit: robot atlas, 31 links, 30 joints
Joints:
- joint back_bky: limit lower=-0.610691 upper=0.49 effort=206.843 velocity=12 -> lower=-0.262 upper=0.524 effort=206.843 velocity=12

File: software/models/mit_gazebo_models/mit_robot_drake/xacro/atlas_skeleton.urdf (robot description, URDF)
Before this commit: robot drc_skeleton, 28 links, 28 joints
Joints:
- joint back_bky: limit lower=-0.610691 upper=0.49 effort=206.843 velocity=12 -> lower=-0.262 upper=0.524 effort=206.843 velocity=12

File: software/models/mit_gazebo_models/mit_robot_drake/xacro/atlas_skeleton_minimal_contact.urdf (robot description, URDF)
Before this commit: robot drc_skeleton, 28 links, 28 joints
Joints:
- joint back_bky: limit lower=-0.610691 upper=0.49 effort=206.843 velocity=12 -> lower=-0.262 upper=0.524 effort=206.843 velocity=12

Commit message: Resulting urdf files from running xacro

File: software/models/mit_gazebo_models/mit_robot/model_LH_RH.urdf (robot description, URDF)
Before this commit: robot atlas, 60 links, 59 joints
Joints:
- joint l_hand_force_torque_joint: origin xyz=0 0.1245 0.0112 rpy=0 0 0 -> xyz=0 0.2773 0.0112 rpy=0 0 0

File: software/models/mit_gazebo_models/mit_robot/model_LI_RI.urdf (robot description, URDF)
Before this commit: robot atlas, 76 links, 75 joints
Joints:
- joint l_hand_force_torque_joint: origin xyz=0 0.1245 0.0112 rpy=0 0 0 -> xyz=0 0.2773 0.0112 rpy=0 0 0

File: software/models/mit_gazebo_models/mit_robot/model_LP_RP.urdf (robot description, URDF)
Before this commit: robot atlas, 60 links, 59 joints
Joints:
- joint l_hand_force_torque_joint: origin xyz=0 0.1245 0.0112 rpy=0 0 0 -> xyz=0 0.2773 0.0112 rpy=0 0 0

File: software/models/mit_gazebo_models/mit_robot/model_LR_RR.urdf (robot description, URDF)
Before this commit: robot atlas, 92 links, 91 joints
Joints:
- joint l_hand_camera_joint: origin xyz=-0.09  0.12 0.0 rpy= -1.57079 0  1.41372 -> xyz=-0.096  0.06 0.0 rpy= -1.57079 0  1.5708
- joint l_hand_force_torque_joint: origin xyz=0 0.1245 0.0112 rpy=0 0 0 -> xyz=0 0.2773 0.0112 rpy=0 0 0
- joint r_hand_camera_joint: origin xyz=0.09  0.12 0.0 rpy= 1.57079 0  1.72788 -> xyz=0.096  0.06 0.0 rpy= 1.57079 0  1.5708

File: software/models/mit_gazebo_models/mit_robot/model_sim.urdf (robot description, URDF)
Before this commit: robot atlas, 113 links, 112 joints
Joints:
- joint l_hand_force_torque_joint: origin xyz=0 0.1245 0.0112 rpy=0 0 0 -> xyz=0 0.2773 0.0112 rpy=0 0 0

File: software/models/mit_gazebo_models/mit_robot/model_sim_gazebo.urdf (robot description, URDF)
Before this commit: robot atlas, 113 links, 112 joints
Joints:
- joint l_hand_force_torque_joint: origin xyz=0 0.1245 0.0112 rpy=0 0 0 -> xyz=0 0.2773 0.0112 rpy=0 0 0

Commit message: Revert "Resulting urdf files from running xacro"
This reverts commit a0112a8c274069073f74aaa5ce275b1507a7b7bc.

File: software/models/mit_gazebo_models/mit_robot/model_LH_RH.urdf (robot description, URDF)
Before this commit: robot atlas, 60 links, 59 joints
Joints:
- joint l_hand_force_torque_joint: origin xyz=0 0.2773 0.0112 rpy=0 0 0 -> xyz=0 0.1245 0.0112 rpy=0 0 0

File: software/models/mit_gazebo_models/mit_robot/model_LI_RI.urdf (robot description, URDF)
Before this commit: robot atlas, 76 links, 75 joints
Joints:
- joint l_hand_force_torque_joint: origin xyz=0 0.2773 0.0112 rpy=0 0 0 -> xyz=0 0.1245 0.0112 rpy=0 0 0

File: software/models/mit_gazebo_models/mit_robot/model_LP_RP.urdf (robot description, URDF)
Before this commit: robot atlas, 60 links, 59 joints
Joints:
- joint l_hand_force_torque_joint: origin xyz=0 0.2773 0.0112 rpy=0 0 0 -> xyz=0 0.1245 0.0112 rpy=0 0 0

File: software/models/mit_gazebo_models/mit_robot/model_LR_RR.urdf (robot description, URDF)
Before this commit: robot atlas, 92 links, 91 joints
Joints:
- joint l_hand_camera_joint: origin xyz=-0.096  0.06 0.0 rpy= -1.57079 0  1.5708 -> xyz=-0.09  0.12 0.0 rpy= -1.57079 0  1.41372
- joint l_hand_force_torque_joint: origin xyz=0 0.2773 0.0112 rpy=0 0 0 -> xyz=0 0.1245 0.0112 rpy=0 0 0
- joint r_hand_camera_joint: origin xyz=0.096  0.06 0.0 rpy= 1.57079 0  1.5708 -> xyz=0.09  0.12 0.0 rpy= 1.57079 0  1.72788

File: software/models/mit_gazebo_models/mit_robot/model_sim.urdf (robot description, URDF)
Before this commit: robot atlas, 113 links, 112 joints
Joints:
- joint l_hand_force_torque_joint: origin xyz=0 0.2773 0.0112 rpy=0 0 0 -> xyz=0 0.1245 0.0112 rpy=0 0 0

File: software/models/mit_gazebo_models/mit_robot/model_sim_gazebo.urdf (robot description, URDF)
Before this commit: robot atlas, 113 links, 112 joints
Joints:
- joint l_hand_force_torque_joint: origin xyz=0 0.2773 0.0112 rpy=0 0 0 -> xyz=0 0.1245 0.0112 rpy=0 0 0
