Commit message: touching up urdf to mirror robotic

File: software/models/mit_gazebo_models/mit_robot/model_LN_RN.urdf (robot description, URDF)
Before this commit: robot atlas, 57 links, 56 joints
Links:
- removed link imu_link
- added link l_hand_force_torque, mass 0.1; visual box size=0.01 0.01 0.01
- added link r_hand_force_torque, mass 0.1; visual box size=0.01 0.01 0.01
Joints:
- removed joint imu_joint
- added joint l_hand_force_torque_joint: type fixed, parent l_hand, child l_hand_force_torque, origin xyz=0 0.1245 0.0112 rpy=0 0 0
- added joint r_hand_force_torque_joint: type fixed, parent r_hand, child r_hand_force_torque, origin xyz=0 -0.1245 -0.0112 rpy=0 0 3.142

File: software/models/mit_gazebo_models/mit_robot/xacro/atlas_LN_RN.urdf.xacro (robot description, xacro)
@@ -1,7 +1,7 @@
-<robot name="atlas" >
+<robot xmlns:xacro="http://playerstage.sourceforge.net/gazebo/xmlschema/#interface" name="atlas" >
   <include filename="$(find mit_drcsim_scripts)/models/mit_robot/xacro/atlas_skeleton.urdf" />
-  <include filename="$(find mit_drcsim_scripts)/models/mit_robot/xacro/atlas.gazebo" />
   <include filename="$(find mit_drcsim_scripts)/models/mit_robot/xacro/atlas.transmission" />
   <include filename="$(find mit_drcsim_scripts)/models/multisense_sl/multisense_sl.urdf" />
-  <include filename="$(find mit_drcsim_scripts)/models/mit_robot/xacro/mit_atlas.gazebo" />
+<!--  <include filename="$(find mit_drcsim_scripts)/models/multisense_sl/multisense_sl_sim.urdf" /> -->
+  <include filename="$(find mit_drcsim_scripts)/models/mit_robot/xacro/hand_force_torque.urdf" />
 </robot>
