Commit message: update the LP_RR urdf xacro

File: software/models/mit_gazebo_models/mit_robot/model_LP_RR.urdf (robot description, URDF)
Before this commit: robot atlas, 72 links, 71 joints
Links:
- added link left_pointer_tip
- added link r_hand_camera_link
- added link r_hand_camera_optical_frame
- added link r_hand_face
- added link r_hand_gripper
Joints:
- added joint left_pointer_tip_joint: type fixed, parent l_hand_force_torque, child left_pointer_tip, origin xyz=0 0.12 0 rpy=0.0 0.0 0.0
- added joint r_hand_camera_joint: type fixed, parent r_hand_force_torque, child r_hand_camera_link, origin xyz=0.09892  0.01431 0.0 rpy= 1.57079 0  1.5708
- added joint r_hand_camera_optical_frame_joint: type fixed, parent r_hand_camera_link, child r_hand_camera_optical_frame, origin xyz=0 0 0 rpy=-1.57079 0.0 -1.57079
- added joint r_hand_face_joint: type fixed, parent r_hand_force_torque, child r_hand_face, origin xyz=0 0.12 0 rpy=0.0 0.0 0.0
- added joint r_hand_gripper_joint: type fixed, parent r_hand_force_torque, child r_hand_gripper, origin xyz=0 0.18 0 rpy=0.0 0.0 0.0
- joint left_hook_hand_joint: origin xyz=0 0.11516 0.015 rpy=1.57079 3.14159 3.14159 -> xyz=0 0.0 0.0 rpy=1.57079 3.14159 3.14159; parent l_hand -> l_hand_force_torque
- joint right_robotiq_hand_joint: origin xyz=0 -0.19016 -0.015 rpy=0 3.141 3.141 -> xyz=0 0.06566 0.0 rpy=0 -1.57079 0; parent r_hand -> r_hand_force_torque

File: software/models/mit_gazebo_models/mit_robot/xacro/atlas_LP_RR.urdf.xacro (robot description, xacro)
@@ -5,6 +5,6 @@
   <xacro:include filename="$(find mit_drcsim_scripts)/models/mit_robot/xacro/hand_force_torque.urdf" />
   <xacro:include filename="$(find hook_description)/src/hook_hand_simple.urdf.xacro" />
-  <xacro:hook_hand side="left" parent="l_hand" reflect="-1"  hookflip="1"  noof30degoffset="0">
-    <origin rpy="1.57079 3.14159 3.14159" xyz="0 0.11516 0.015"/>
+  <xacro:hook_hand side="left" parent="l_hand_force_torque">
+    <origin rpy="1.57079 3.14159 3.14159" xyz="0 0.0 0.0"/>
   </xacro:hook_hand>
   <xacro:include filename="$(find robotiq_hand_description)/cfg/robotiq_hand.urdf.xacro" />
@@ -12,3 +12,7 @@
     <origin rpy="0 -1.57079 0" xyz="0 0.06566 0.0"/>
   </xacro:robotiq_hand>
+  <xacro:include filename="$(find robotiq_camera)/urdf/robotiq_camera.urdf.xacro" />
+  <xacro:robotiq_camera  side_letter="r" reflect="-1" parent="r_hand_force_torque" >
+    <origin xyz="0.0  0.0 0.0" rpy="0.0 0  0.0"/>
+  </xacro:robotiq_camera>
 </robot>
