Commit message: modifications to sticky hand urdfs
git-svn-id: https://svn.csail.mit.edu/drc/trunk@5953 c7283977-0100-402a-a91a-fa70b306dbfe

File: software/models/mit_gazebo_models/mit_robot_hands/drake_urdfs/debug/xacro/irobot_hand_drake_left.urdf.xacro (robot description, xacro)
@@ -14,5 +14,6 @@
   </link>
   <xacro:irobot_hand side="left" parent="base" reflect="-1">
-    <origin rpy="0 0 3.14159" xyz="0 0.05 0"/>
+     <!--  <origin rpy="0 0 3.14159" xyz="0 0.05 0"/>-->
+    <origin rpy="1.57 0 -1.57" xyz="0 0 0"/>
   </xacro:irobot_hand>
 </robot>

File: software/models/mit_gazebo_models/mit_robot_hands/drake_urdfs/debug/xacro/irobot_hand_drake_right.urdf.xacro (robot description, xacro)
@@ -14,5 +14,6 @@
   </link>
   <xacro:irobot_hand side="right" parent="base" reflect="1">
-    <origin rpy="0 0 0" xyz="0 -0.05 0"/>
+ <!--  <origin rpy="0 0 0" xyz="0 -0.05 0"/>-->
+    <origin rpy="1.57 0 -1.57" xyz="0 0 0"/>
   </xacro:irobot_hand>
 </robot>

File: software/models/mit_gazebo_models/mit_robot_hands/drake_urdfs/xacro/irobot_hand_drake_left.urdf.xacro (robot description, xacro)
@@ -14,5 +14,6 @@
   </link>
   <xacro:irobot_hand side="left" parent="base" reflect="-1">
-    <origin rpy="0 0 3.14159" xyz="0 0.05 0"/>
+<!--    <origin rpy="0 0 3.14159" xyz="0 0.05 0"/>-->
+    <origin rpy="1.57 0 -1.57" xyz="0 0 0"/>
   </xacro:irobot_hand>
 </robot>

File: software/models/mit_gazebo_models/mit_robot_hands/drake_urdfs/xacro/irobot_hand_drake_right.urdf.xacro (robot description, xacro)
@@ -14,5 +14,6 @@
   </link>
   <xacro:irobot_hand side="right" parent="base" reflect="1">
-    <origin rpy="0 0 0" xyz="0 -0.05 0"/>
+ <!--  <origin rpy="0 0 0" xyz="0 -0.05 0"/>-->
+    <origin rpy="1.57 0 -1.57" xyz="0 0 0"/>
   </xacro:irobot_hand>
 </robot>

File: software/models/mit_gazebo_models/mit_robot_hands/irobot_hand_left.urdf (robot description, URDF)
Before this commit: robot irobot_hand_left, 10 links, 9 joints
Links:
- link left_base_link: geometry collision mesh filename=package://irobot_hand/meshes/palm.stl; visual mesh filename=package://irobot_hand/meshes/palm.stl
- link left_finger[0]/base_rotation_link: geometry collision mesh filename=package://irobot_hand/meshes/finger_base.stl; visual mesh filename=package://irobot_hand/meshes/finger_base.stl
- link left_finger[0]/distal_link: geometry collision mesh filename=package://irobot_hand/meshes/finger_distal.stl; visual mesh filename=package://irobot_hand/meshes/finger_distal.stl
- link left_finger[0]/proximal_link: geometry collision mesh filename=package://irobot_hand/meshes/finger_proximal.stl; visual mesh filename=package://irobot_hand/meshes/finger_proximal.stl
- link left_finger[1]/base_rotation_link: geometry collision mesh filename=package://irobot_hand/meshes/finger_base.stl; visual mesh filename=package://irobot_hand/meshes/finger_base.stl
- link left_finger[1]/distal_link: geometry collision mesh filename=package://irobot_hand/meshes/finger_distal.stl; visual mesh filename=package://irobot_hand/meshes/finger_distal.stl
- link left_finger[1]/proximal_link: geometry collision mesh filename=package://irobot_hand/meshes/finger_proximal.stl; visual mesh filename=package://irobot_hand/meshes/finger_proximal.stl
- link left_finger[2]/distal_link: geometry collision mesh filename=package://irobot_hand/meshes/finger_distal.stl; visual mesh filename=package://irobot_hand/meshes/finger_distal.stl
- link left_finger[2]/proximal_link: geometry collision mesh filename=package://irobot_hand/meshes/finger_proximal.stl; visual mesh filename=package://irobot_hand/meshes/finger_proximal.stl

File: software/models/mit_gazebo_models/mit_robot_hands/irobot_hand_right.urdf (robot description, URDF)
Before this commit: robot irobot_hand_right, 10 links, 9 joints
Links:
- link right_base_link: geometry collision mesh filename=package://irobot_hand/meshes/palm.stl; visual mesh filename=package://irobot_hand/meshes/palm.stl
- link right_finger[0]/base_rotation_link: geometry collision mesh filename=package://irobot_hand/meshes/finger_base.stl; visual mesh filename=package://irobot_hand/meshes/finger_base.stl
- link right_finger[0]/distal_link: geometry collision mesh filename=package://irobot_hand/meshes/finger_distal.stl; visual mesh filename=package://irobot_hand/meshes/finger_distal.stl
- link right_finger[0]/proximal_link: geometry collision mesh filename=package://irobot_hand/meshes/finger_proximal.stl; visual mesh filename=package://irobot_hand/meshes/finger_proximal.stl
- link right_finger[1]/base_rotation_link: geometry collision mesh filename=package://irobot_hand/meshes/finger_base.stl; visual mesh filename=package://irobot_hand/meshes/finger_base.stl
- link right_finger[1]/distal_link: geometry collision mesh filename=package://irobot_hand/meshes/finger_distal.stl; visual mesh filename=package://irobot_hand/meshes/finger_distal.stl
- link right_finger[1]/proximal_link: geometry collision mesh filename=package://irobot_hand/meshes/finger_proximal.stl; visual mesh filename=package://irobot_hand/meshes/finger_proximal.stl
- link right_finger[2]/distal_link: geometry collision mesh filename=package://irobot_hand/meshes/finger_distal.stl; visual mesh filename=package://irobot_hand/meshes/finger_distal.stl
- link right_finger[2]/proximal_link: geometry collision mesh filename=package://irobot_hand/meshes/finger_proximal.stl; visual mesh filename=package://irobot_hand/meshes/finger_proximal.stl

File: software/models/mit_gazebo_models/mit_robot_hands/sandia_hand_left.urdf (robot description, URDF)
Before this commit: robot sandia_hand_left, 30 links, 29 joints
Links:
- added link left_palm_left_camera_frame, mass 0.01; visual box size=0.003 0.010 0.007
- added link left_palm_left_camera_optical_frame
- added link left_palm_right_camera_frame, mass 0.01; visual box size=0.003 0.010 0.007
- added link left_palm_right_camera_optical_frame
- link left_f0_0: mass 0.05 -> 0.106
- link left_f0_1: mass 0.05 -> 0.033
- link left_f0_1_accel: mass 0.001 -> 0.01
- link left_f0_2: mass 0.05 -> 0.033
- link left_f0_2_accel: mass 0.001 -> 0.01
- link left_f0_base: mass 0.35 -> 0.250
- link left_f0_fixed_accel: mass 0.001 -> 0.01
- link left_f1_0: mass 0.05 -> 0.106
- link left_f1_1: mass 0.05 -> 0.033
- link left_f1_1_accel: mass 0.001 -> 0.01
- link left_f1_2: mass 0.05 -> 0.033
- link left_f1_2_accel: mass 0.001 -> 0.01
- link left_f1_base: mass 0.35 -> 0.250
- link left_f1_fixed_accel: mass 0.001 -> 0.01
- link left_f2_0: mass 0.05 -> 0.106
- link left_f2_1: mass 0.05 -> 0.033
- link left_f2_1_accel: mass 0.001 -> 0.01
- link left_f2_2: mass 0.05 -> 0.033
- link left_f2_2_accel: mass 0.001 -> 0.01
- link left_f2_base: mass 0.35 -> 0.250
- link left_f2_fixed_accel: mass 0.001 -> 0.01
- link left_f3_0: mass 0.05 -> 0.106
- link left_f3_1: mass 0.05 -> 0.033
- link left_f3_1_accel: mass 0.001 -> 0.01
- link left_f3_2: mass 0.05 -> 0.033
- link left_f3_2_accel: mass 0.001 -> 0.01
- link left_f3_base: mass 0.35 -> 0.250
- link left_f3_fixed_accel: mass 0.001 -> 0.01
- link left_palm: mass 0.3 -> 1.303
Joints:
- added joint left_palm_left_camera_frame_joint: type fixed, parent left_palm, child left_palm_left_camera_frame, origin xyz=0.0435128991906 -0.0451672761576 0.025 rpy=-0.6708 -1.57079632679 3.14159265359
- added joint left_palm_left_camera_optical_frame_joint: type fixed, parent left_palm_left_camera_frame, child left_palm_left_camera_optical_frame, origin xyz=0 0 0 rpy=-1.57079632679 0.0 -1.57079632679
- added joint left_palm_right_camera_frame_joint: type fixed, parent left_palm, child left_palm_right_camera_frame, origin xyz=0.0683774130138 -0.0138342911048 0.025 rpy=-0.6708 -1.57079632679 3.14159265359
- added joint left_palm_right_camera_optical_frame_joint: type fixed, parent left_palm_right_camera_frame, child left_palm_right_camera_optical_frame, origin xyz=0 0 0 rpy=-1.57079632679 0.0 -1.57079632679
- joint left_f0_j0: limit lower=-1.57079632679 upper=1.57079632679 effort=1 velocity=1 -> lower=-1.57079632679 upper=1.57079632679 effort=11 velocity=-1
- joint left_f0_j1: limit lower=-1.57079632679 upper=1.57079632679 effort=1 velocity=1 -> lower=-1.57079632679 upper=1.57079632679 effort=28 velocity=-1
- joint left_f0_j2: limit lower=-1.57079632679 upper=1.57079632679 effort=1 velocity=1 -> lower=-1.57079632679 upper=1.57079632679 effort=28 velocity=-1
- joint left_f1_j0: limit lower=-1.57079632679 upper=1.57079632679 effort=1 velocity=1 -> lower=-1.57079632679 upper=1.57079632679 effort=11 velocity=-1
- joint left_f1_j1: limit lower=-1.57079632679 upper=1.57079632679 effort=1 velocity=1 -> lower=-1.57079632679 upper=1.57079632679 effort=28 velocity=-1
- joint left_f1_j2: limit lower=-1.57079632679 upper=1.57079632679 effort=1 velocity=1 -> lower=-1.57079632679 upper=1.57079632679 effort=28 velocity=-1
- joint left_f2_j0: limit lower=-1.57079632679 upper=1.57079632679 effort=1 velocity=1 -> lower=-1.57079632679 upper=1.57079632679 effort=11 velocity=-1
- joint left_f2_j1: limit lower=-1.57079632679 upper=1.57079632679 effort=1 velocity=1 -> lower=-1.57079632679 upper=1.57079632679 effort=28 velocity=-1
- joint left_f2_j2: limit lower=-1.57079632679 upper=1.57079632679 effort=1 velocity=1 -> lower=-1.57079632679 upper=1.57079632679 effort=28 velocity=-1
- joint left_f3_j0: limit lower=-1.57079632679 upper=1.57079632679 effort=1 velocity=1 -> lower=-1.57079632679 upper=1.57079632679 effort=11 velocity=-1
- joint left_f3_j1: limit lower=-1.57079632679 upper=1.57079632679 effort=1 velocity=1 -> lower=-1.57079632679 upper=1.57079632679 effort=28 velocity=-1
- joint left_f3_j2: limit lower=-1.57079632679 upper=1.57079632679 effort=1 velocity=1 -> lower=-1.57079632679 upper=1.57079632679 effort=28 velocity=-1

File: software/models/mit_gazebo_models/mit_robot_hands/sandia_hand_right.urdf (robot description, URDF)
Before this commit: robot sandia_hand_right, 30 links, 29 joints
Links:
- added link right_palm_left_camera_frame, mass 0.01; visual box size=0.003 0.010 0.007
- added link right_palm_left_camera_optical_frame
- added link right_palm_right_camera_frame, mass 0.01; visual box size=0.003 0.010 0.007
- added link right_palm_right_camera_optical_frame
- link right_f0_0: mass 0.05 -> 0.106
- link right_f0_1: mass 0.05 -> 0.033
- link right_f0_1_accel: mass 0.001 -> 0.01
- link right_f0_2: mass 0.05 -> 0.033
- link right_f0_2_accel: mass 0.001 -> 0.01
- link right_f0_base: mass 0.35 -> 0.250
- link right_f0_fixed_accel: mass 0.001 -> 0.01
- link right_f1_0: mass 0.05 -> 0.106
- link right_f1_1: mass 0.05 -> 0.033
- link right_f1_1_accel: mass 0.001 -> 0.01
- link right_f1_2: mass 0.05 -> 0.033
- link right_f1_2_accel: mass 0.001 -> 0.01
- link right_f1_base: mass 0.35 -> 0.250
- link right_f1_fixed_accel: mass 0.001 -> 0.01
- link right_f2_0: mass 0.05 -> 0.106
- link right_f2_1: mass 0.05 -> 0.033
- link right_f2_1_accel: mass 0.001 -> 0.01
- link right_f2_2: mass 0.05 -> 0.033
- link right_f2_2_accel: mass 0.001 -> 0.01
- link right_f2_base: mass 0.35 -> 0.250
- link right_f2_fixed_accel: mass 0.001 -> 0.01
- link right_f3_0: mass 0.05 -> 0.106
- link right_f3_1: mass 0.05 -> 0.033
- link right_f3_1_accel: mass 0.001 -> 0.01
- link right_f3_2: mass 0.05 -> 0.033
- link right_f3_2_accel: mass 0.001 -> 0.01
- link right_f3_base: mass 0.35 -> 0.250
- link right_f3_fixed_accel: mass 0.001 -> 0.01
- link right_palm: mass 0.3 -> 1.303
Joints:
- added joint right_palm_left_camera_frame_joint: type fixed, parent right_palm, child right_palm_left_camera_frame, origin xyz=0.0683774130138 0.0138342911048 0.025 rpy=0.6708 -1.57079632679 3.14159265359
- added joint right_palm_left_camera_optical_frame_joint: type fixed, parent right_palm_left_camera_frame, child right_palm_left_camera_optical_frame, origin xyz=0 0 0 rpy=-1.57079632679 0.0 -1.57079632679
- added joint right_palm_right_camera_frame_joint: type fixed, parent right_palm, child right_palm_right_camera_frame, origin xyz=0.0435128991906 0.0451672761576 0.025 rpy=0.6708 -1.57079632679 3.14159265359
- added joint right_palm_right_camera_optical_frame_joint: type fixed, parent right_palm_right_camera_frame, child right_palm_right_camera_optical_frame, origin xyz=0 0 0 rpy=-1.57079632679 0.0 -1.57079632679
- joint right_f0_j0: limit lower=-1.57079632679 upper=1.57079632679 effort=1 velocity=1 -> lower=-1.57079632679 upper=1.57079632679 effort=11 velocity=-1
- joint right_f0_j1: limit lower=-1.57079632679 upper=1.57079632679 effort=1 velocity=1 -> lower=-1.57079632679 upper=1.57079632679 effort=28 velocity=-1
- joint right_f0_j2: limit lower=-1.57079632679 upper=1.57079632679 effort=1 velocity=1 -> lower=-1.57079632679 upper=1.57079632679 effort=28 velocity=-1
- joint right_f1_j0: limit lower=-1.57079632679 upper=1.57079632679 effort=1 velocity=1 -> lower=-1.57079632679 upper=1.57079632679 effort=11 velocity=-1
- joint right_f1_j1: limit lower=-1.57079632679 upper=1.57079632679 effort=1 velocity=1 -> lower=-1.57079632679 upper=1.57079632679 effort=28 velocity=-1
- joint right_f1_j2: limit lower=-1.57079632679 upper=1.57079632679 effort=1 velocity=1 -> lower=-1.57079632679 upper=1.57079632679 effort=28 velocity=-1
- joint right_f2_j0: limit lower=-1.57079632679 upper=1.57079632679 effort=1 velocity=1 -> lower=-1.57079632679 upper=1.57079632679 effort=11 velocity=-1
- joint right_f2_j1: limit lower=-1.57079632679 upper=1.57079632679 effort=1 velocity=1 -> lower=-1.57079632679 upper=1.57079632679 effort=28 velocity=-1
- joint right_f2_j2: limit lower=-1.57079632679 upper=1.57079632679 effort=1 velocity=1 -> lower=-1.57079632679 upper=1.57079632679 effort=28 velocity=-1
- joint right_f3_j0: limit lower=-1.57079632679 upper=1.57079632679 effort=1 velocity=1 -> lower=-1.57079632679 upper=1.57079632679 effort=11 velocity=-1
- joint right_f3_j1: limit lower=-1.57079632679 upper=1.57079632679 effort=1 velocity=1 -> lower=-1.57079632679 upper=1.57079632679 effort=28 velocity=-1
- joint right_f3_j2: limit lower=-1.57079632679 upper=1.57079632679 effort=1 velocity=1 -> lower=-1.57079632679 upper=1.57079632679 effort=28 velocity=-1

File: software/models/mit_gazebo_models/mit_robot_hands/xacro/irobot_hand_left.urdf.xacro (robot description, xacro)
@@ -4,5 +4,5 @@
        xmlns:xacro="http://playerstage.sourceforge.net/gazebo/xmlschema/#interface"
        name="irobot_hand_left" >
-  <include filename="$(find handle_description)/src/irobot_hand_simple.urdf.xacro" />
+  <include filename="$(find mit_drcsim_scripts)/models/mit_robot_hands/xacro/irobot_hand_simple.urdf.xacro" />
   <link name="base">
     <inertial>
@@ -13,5 +13,6 @@
   </link>
   <xacro:irobot_hand side="left" parent="base" reflect="-1">
-    <origin rpy="0 0 3.14159" xyz="0 0.05 0"/>
+<!--    <origin rpy="0 0 3.14159" xyz="0 0.05 0"/>-->
+    <origin rpy="1.57 0 -1.57" xyz="0 0 0"/>
   </xacro:irobot_hand>
 </robot>

File: software/models/mit_gazebo_models/mit_robot_hands/xacro/irobot_hand_right.urdf.xacro (robot description, xacro)
@@ -4,5 +4,5 @@
        xmlns:xacro="http://playerstage.sourceforge.net/gazebo/xmlschema/#interface"
        name="irobot_hand_right" >
-  <include filename="$(find handle_description)/src/irobot_hand_simple.urdf.xacro" />
+  <include filename="$(find mit_drcsim_scripts)/models/mit_robot_hands/xacro/irobot_hand_simple.urdf.xacro" />
   <link name="base">
     <inertial>
@@ -13,5 +13,6 @@
   </link>
   <xacro:irobot_hand side="right" parent="base" reflect="1">
-    <origin rpy="0 0 0" xyz="0 -0.05 0"/>
+ <!--  <origin rpy="0 0 0" xyz="0 -0.05 0"/>-->
+    <origin rpy="1.57 0 -1.57" xyz="0 0 0"/>
   </xacro:irobot_hand>
 </robot>
