Commit message: adding more contact points for better grasp optimization
git-svn-id: https://svn.csail.mit.edu/drc/trunk@5972 c7283977-0100-402a-a91a-fa70b306dbfe

File: software/models/mit_gazebo_models/mit_robot_hands/drake_urdfs/debug/xacro/irobot_hand_drake_left.urdf.xacro (robot description, xacro)
@@ -5,5 +5,5 @@
        name="irobot_hand_left" >
 <!--  <include filename="$(find handle_description)/src/irobot_hand_simple.urdf.xacro" />-->
-  <include filename="$(find mit_drcsim_scripts)/models/mit_robot_hands/visual_contact_spheres/xacro/irobot_hand_simple_drake_w_contact_sphere_visuals.urdf.xacro" />
+  <include filename="$(find mit_drcsim_scripts)/models/mit_robot_hands/drake_urdfs/debug/xacro/irobot_hand_simple_drake_w_contact_sphere_visuals.urdf.xacro" />
   <link name="base">
     <inertial>

File: software/models/mit_gazebo_models/mit_robot_hands/drake_urdfs/debug/xacro/irobot_hand_drake_right.urdf.xacro (robot description, xacro)
@@ -5,5 +5,5 @@
        name="irobot_hand_right" >
 <!--  <include filename="$(find handle_description)/src/irobot_hand_simple.urdf.xacro" />-->
-  <include filename="$(find mit_drcsim_scripts)/models/mit_robot_hands/visual_contact_spheres/xacro/irobot_hand_simple_drake_w_contact_sphere_visuals.urdf.xacro" />
+  <include filename="$(find mit_drcsim_scripts)/models/mit_robot_hands/drake_urdfs/debug/xacro/irobot_hand_simple_drake_w_contact_sphere_visuals.urdf.xacro" />
   <link name="base">
     <inertial>

File: software/models/mit_gazebo_models/mit_robot_hands/drake_urdfs/debug/xacro/irobot_hand_simple_drake_w_contact_sphere_visuals.urdf.xacro (robot description, xacro)
@@ -17,4 +17,7 @@
 <xacro:property name="base_contact2y" value="-0.005" />
 <xacro:property name="base_contact2z" value="0.083" />
+<xacro:property name="base_contact3x" value="0.012" />
+<xacro:property name="base_contact3y" value="0.0" />
+<xacro:property name="base_contact3z" value="0.083" />
 <xacro:property name="proximal_contactx" value="0.00" />
 <xacro:property name="proximal_contacty" value="0.01" />
@@ -249,4 +252,16 @@
         </geometry>
       </collision>
+      <collision>
+        <origin rpy="0 0 0" xyz="${base_contact3x} ${base_contact3y} ${base_contact3z}"/>
+        <geometry>
+          <sphere radius="0"/>
+        </geometry>
+      </collision>
+       <collision>
+        <origin rpy="0 0 0" xyz="${-base_contact3x} ${base_contact3y} ${base_contact3z}"/>
+        <geometry>
+          <sphere radius="0"/>
+        </geometry>
+      </collision>
     <visual>
       <geometry>
@@ -333,4 +348,10 @@
         </geometry>
       </collision>
+        <collision>
+        <origin rpy="0 0 0" xyz="${distal_contactx} ${-distal_contacty} ${distal_contactz}"/>
+        <geometry>
+          <sphere radius="0"/>
+        </geometry>
+      </collision>
     <visual>
       <geometry>
@@ -417,4 +438,10 @@
         </geometry>
       </collision>
+        <collision>
+        <origin rpy="0 0 0" xyz="${distal_contactx} ${-distal_contacty} ${distal_contactz}"/>
+        <geometry>
+          <sphere radius="0"/>
+        </geometry>
+      </collision>
     <visual>
       <geometry>
@@ -479,4 +506,10 @@
         </geometry>
       </collision>
+        <collision>
+        <origin rpy="0 0 0" xyz="${distal_contactx} ${-distal_contacty} ${distal_contactz}"/>
+        <geometry>
+          <sphere radius="0"/>
+        </geometry>
+      </collision>
     <visual>
       <geometry>
@@ -563,4 +596,40 @@
       </visual>
   </link>
+  <joint name="${side}_base_link_dummy3_joint" type="fixed">
+    <origin xyz="0 0 0"/>
+    <parent link="${side}_base_link"/>
+    <child link="${side}_base_link_dummy3"/>
+  </joint>
+  <link name="${side}_base_link_dummy3">
+      <inertial>
+        <mass value="0.1"/>
+        <origin xyz="0 0 0"/>
+        <inertia ixx="0.001" ixy="0.0" ixz="0.0" iyy="0.001" iyz="0.0" izz="0.001"/>
+      </inertial>
+      <visual>
+        <origin rpy="0 0 0" xyz="${base_contact3x} ${base_contact3y} ${base_contact3z}"/>
+        <geometry>
+          <sphere radius="0.005"/>
+        </geometry>
+      </visual>
+  </link>
+  <joint name="${side}_base_link_dummy4_joint" type="fixed">
+    <origin xyz="0 0 0"/>
+    <parent link="${side}_base_link"/>
+    <child link="${side}_base_link_dummy4"/>
+  </joint>
+  <link name="${side}_base_link_dummy4">
+      <inertial>
+        <mass value="0.1"/>
+        <origin xyz="0 0 0"/>
+        <inertia ixx="0.001" ixy="0.0" ixz="0.0" iyy="0.001" iyz="0.0" izz="0.001"/>
+      </inertial>
+      <visual>
+        <origin rpy="0 0 0" xyz="${-base_contact3x} ${base_contact3y} ${base_contact3z}"/>
+        <geometry>
+          <sphere radius="0.005"/>
+        </geometry>
+      </visual>
+  </link>
   <joint name="${side}_finger[0]/proximal_link_dummy_joint" type="fixed">
     <origin xyz="0 0 0"/>
@@ -617,4 +686,22 @@
       </visual>
   </link>
+   <joint name="${side}_finger[0]/distal_link_dummy2_joint" type="fixed">
+    <origin xyz="0 0 0"/>
+    <parent link="${side}_finger[0]/distal_link"/>
+    <child link="${side}_finger[0]/distal_link_dummy2"/>
+  </joint>
+  <link name="${side}_finger[0]/distal_link_dummy2">
+      <inertial>
+        <mass value="0.1"/>
+        <origin xyz="0 0 0"/>
+        <inertia ixx="0.001" ixy="0.0" ixz="0.0" iyy="0.001" iyz="0.0" izz="0.001"/>
+      </inertial>
+      <visual>
+        <origin rpy="0 0 0" xyz="${distal_contactx} ${-distal_contacty} ${distal_contactz}"/>
+        <geometry>
+          <sphere radius="0.005"/>
+        </geometry>
+      </visual>
+  </link>
   <joint name="${side}_finger[1]/proximal_link_dummy_joint" type="fixed">
     <origin xyz="0 0 0"/>
@@ -671,4 +758,22 @@
       </visual>
   </link>
+   <joint name="${side}_finger[1]/distal_link_dummy1_joint" type="fixed">
+    <origin xyz="0 0 0"/>
+    <parent link="${side}_finger[1]/distal_link"/>
+    <child link="${side}_finger[1]/distal_link_dummy1"/>
+  </joint>
+  <link name="${side}_finger[1]/distal_link_dummy1">
+      <inertial>
+        <mass value="0.1"/>
+        <origin xyz="0 0 0"/>
+        <inertia ixx="0.001" ixy="0.0" ixz="0.0" iyy="0.001" iyz="0.0" izz="0.001"/>
+      </inertial>
+      <visual>
+        <origin rpy="0 0 0" xyz="${distal_contactx} ${-distal_contacty} ${distal_contactz}"/>
+        <geometry>
+          <sphere radius="0.005"/>
+        </geometry>
+      </visual>
+  </link>
   <joint name="${side}_finger[2]/proximal_link_dummy_joint" type="fixed">
     <origin xyz="0 0 0"/>
@@ -720,4 +825,22 @@
       <visual>
         <origin rpy="0 0 0" xyz="${distal_contactx} ${distal_contacty} ${distal_contactz}"/>
+        <geometry>
+          <sphere radius="0.005"/>
+        </geometry>
+      </visual>
+  </link>
+  <joint name="${side}_finger[2]/distal_link_dummy1_joint" type="fixed">
+    <origin xyz="0 0 0"/>
+    <parent link="${side}_finger[2]/distal_link"/>
+    <child link="${side}_finger[2]/distal_link_dummy1"/>
+  </joint>
+  <link name="${side}_finger[2]/distal_link_dummy1">
+      <inertial>
+        <mass value="0.1"/>
+        <origin xyz="0 0 0"/>
+        <inertia ixx="0.001" ixy="0.0" ixz="0.0" iyy="0.001" iyz="0.0" izz="0.001"/>
+      </inertial>
+      <visual>
+        <origin rpy="0 0 0" xyz="${distal_contactx} ${-distal_contacty} ${distal_contactz}"/>
         <geometry>
           <sphere radius="0.005"/>

File: software/models/mit_gazebo_models/mit_robot_hands/drake_urdfs/debug/xacro/sandia_hand_drake_left.urdf.xacro (robot description, xacro)
@@ -7,5 +7,5 @@
   <!-- Commenting out urdf with meshes, using simple collision shapes instead -->
   <!--<include filename="$(find mit_drcsim_scripts)/models/mit_robot_hands/visual_contact_spheres/xacro/sandia_hand_drake_w_contact_sphere_visuals.urdf.xacro" />-->
-  <include filename="$(find mit_drcsim_scripts)/models/mit_robot_hands/visual_contact_spheres/xacro/sandia_hand_simplified_shapes_drake_w_contact_sphere_visuals.urdf.xacro" />
+  <include filename="$(find mit_drcsim_scripts)/models/mit_robot_hands/drake_urdfs/debug/xacro/sandia_hand_simplified_shapes_drake_w_contact_sphere_visuals.urdf.xacro" />
   <link name="base">
     <inertial>

File: software/models/mit_gazebo_models/mit_robot_hands/drake_urdfs/debug/xacro/sandia_hand_drake_right.urdf.xacro (robot description, xacro)
@@ -7,5 +7,5 @@
   <!-- Commenting out urdf with meshes, using simple collision shapes instead -->
   <!--<include filename="$(find mit_drcsim_scripts)/models/mit_robot_hands/visual_contact_spheres/xacro/sandia_hand_drake_w_contact_sphere_visuals.urdf.xacro" />-->
-  <include filename="$(find mit_drcsim_scripts)/models/mit_robot_hands/visual_contact_spheres/xacro/sandia_hand_simplified_shapes_drake_w_contact_sphere_visuals.urdf.xacro" />
+  <include filename="$(find mit_drcsim_scripts)/models/mit_robot_hands/drake_urdfs/debug/xacro/sandia_hand_simplified_shapes_drake_w_contact_sphere_visuals.urdf.xacro" />
   <link name="base">
     <inertial>

File: software/models/mit_gazebo_models/mit_robot_hands/drake_urdfs/debug/xacro/sandia_hand_simplified_shapes_drake_w_contact_sphere_visuals.urdf.xacro (robot description, xacro)
@@ -281,4 +281,29 @@
       <parent link="${side}_f${idx}_2"/>
       <child link="${side}_f${idx}_2_accel_dummy1"/>
+      <origin xyz="0.04 0 0" rpy="-${M_pi/2} 0 0"/>
+    </joint>
+    <link name="${side}_f${idx}_2_accel_dummy2">
+      <origin xyz="0 0 0" rpy="0 0 0"/>
+      <inertial>
+        <mass value="0.001"/>
+        <origin xyz="0 0 0"/>
+        <inertia ixx="0.01" ixy="0" ixz="0" iyy="0.01" iyz="0" izz="0.01"/>
+      </inertial>
+      <visual>
+        <origin rpy="0 0 0" xyz="0.0 0.0 -0.01"/>
+        <geometry>
+          <sphere radius="0.005"/>
+        </geometry>
+      </visual>
+      <collision>
+        <origin rpy="0 0 0" xyz="0.0 0.0 -0.01"/>
+        <geometry>
+          <sphere radius="0"/>
+        </geometry>
+      </collision>
+    </link>
+     <joint name="${side}_f${idx}_2_accel_dummy2" type="fixed">
+      <parent link="${side}_f${idx}_2"/>
+      <child link="${side}_f${idx}_2_accel_dummy2"/>
       <origin xyz="0.04 0 0" rpy="-${M_pi/2} 0 0"/>
     </joint>
@@ -600,4 +625,29 @@
       <parent link="${side}_f${idx}_2"/>
       <child link="${side}_f${idx}_2_accel_dummy1"/>
+      <origin xyz="0.04 0 0" rpy="-${M_pi/2} 0 0"/>
+    </joint>
+    <link name="${side}_f${idx}_2_accel_dummy2">
+      <origin xyz="0 0 0" rpy="0 0 0"/>
+      <inertial>
+        <mass value="0.001"/>
+        <origin xyz="0 0 0"/>
+        <inertia ixx="0.01" ixy="0" ixz="0" iyy="0.01" iyz="0" izz="0.01"/>
+      </inertial>
+      <visual>
+        <origin rpy="0 0 0" xyz="0.0 0.0 -0.01"/>
+        <geometry>
+          <sphere radius="0.005"/>
+        </geometry>
+      </visual>
+      <collision>
+        <origin rpy="0 0 0" xyz="0.0 0.0 -0.01"/>
+        <geometry>
+          <sphere radius="0"/>
+        </geometry>
+      </collision>
+    </link>
+     <joint name="${side}_f${idx}_2_accel_dummy2" type="fixed">
+      <parent link="${side}_f${idx}_2"/>
+      <child link="${side}_f${idx}_2_accel_dummy2"/>
       <origin xyz="0.04 0 0" rpy="-${M_pi/2} 0 0"/>
     </joint>

File: software/models/mit_gazebo_models/mit_robot_hands/drake_urdfs/irobot_hand_drake_left.urdf (robot description, URDF)
Before this commit: robot irobot_hand_left, 10 links, 9 joints
Links:
- link left_base_link: geometry collision sphere radius=0; collision sphere radius=0
- link left_finger[0]/distal_link: geometry collision sphere radius=0; collision sphere radius=0
- link left_finger[1]/distal_link: geometry collision sphere radius=0; collision sphere radius=0
- link left_finger[2]/distal_link: geometry collision sphere radius=0; collision sphere radius=0

File: software/models/mit_gazebo_models/mit_robot_hands/drake_urdfs/irobot_hand_drake_right.urdf (robot description, URDF)
Before this commit: robot irobot_hand_right, 10 links, 9 joints
Links:
- link right_base_link: geometry collision sphere radius=0; collision sphere radius=0
- link right_finger[0]/distal_link: geometry collision sphere radius=0; collision sphere radius=0
- link right_finger[1]/distal_link: geometry collision sphere radius=0; collision sphere radius=0
- link right_finger[2]/distal_link: geometry collision sphere radius=0; collision sphere radius=0

File: software/models/mit_gazebo_models/mit_robot_hands/drake_urdfs/sandia_hand_drake_left.urdf (robot description, URDF)
Before this commit: robot sandia_hand_left, 37 links, 36 joints
Links:
- added link left_f0_2_accel_dummy2, mass 0.001; collision sphere radius=0
- added link left_f1_2_accel_dummy2, mass 0.001; collision sphere radius=0
- added link left_f2_2_accel_dummy2, mass 0.001; collision sphere radius=0
- added link left_f3_2_accel_dummy2, mass 0.001; collision sphere radius=0
Joints:
- added joint left_f0_2_accel_dummy2: type fixed, parent left_f0_2, child left_f0_2_accel_dummy2, origin xyz=0.04 0 0 rpy=-1.57079632679 0 0
- added joint left_f1_2_accel_dummy2: type fixed, parent left_f1_2, child left_f1_2_accel_dummy2, origin xyz=0.04 0 0 rpy=-1.57079632679 0 0
- added joint left_f2_2_accel_dummy2: type fixed, parent left_f2_2, child left_f2_2_accel_dummy2, origin xyz=0.04 0 0 rpy=-1.57079632679 0 0
- added joint left_f3_2_accel_dummy2: type fixed, parent left_f3_2, child left_f3_2_accel_dummy2, origin xyz=0.04 0 0 rpy=-1.57079632679 0 0

File: software/models/mit_gazebo_models/mit_robot_hands/drake_urdfs/sandia_hand_drake_right.urdf (robot description, URDF)
Before this commit: robot sandia_hand_right, 37 links, 36 joints
Links:
- added link right_f0_2_accel_dummy2, mass 0.001; collision sphere radius=0
- added link right_f1_2_accel_dummy2, mass 0.001; collision sphere radius=0
- added link right_f2_2_accel_dummy2, mass 0.001; collision sphere radius=0
- added link right_f3_2_accel_dummy2, mass 0.001; collision sphere radius=0
Joints:
- added joint right_f0_2_accel_dummy2: type fixed, parent right_f0_2, child right_f0_2_accel_dummy2, origin xyz=0.04 0 0 rpy=-1.57079632679 0 0
- added joint right_f1_2_accel_dummy2: type fixed, parent right_f1_2, child right_f1_2_accel_dummy2, origin xyz=0.04 0 0 rpy=-1.57079632679 0 0
- added joint right_f2_2_accel_dummy2: type fixed, parent right_f2_2, child right_f2_2_accel_dummy2, origin xyz=0.04 0 0 rpy=-1.57079632679 0 0
- added joint right_f3_2_accel_dummy2: type fixed, parent right_f3_2, child right_f3_2_accel_dummy2, origin xyz=0.04 0 0 rpy=-1.57079632679 0 0

File: software/models/mit_gazebo_models/mit_robot_hands/drake_urdfs/xacro/irobot_hand_simple_drake.urdf.xacro (robot description, xacro)
@@ -17,4 +17,7 @@
 <xacro:property name="base_contact2y" value="-0.005" />
 <xacro:property name="base_contact2z" value="0.083" />
+<xacro:property name="base_contact3x" value="0.012" />
+<xacro:property name="base_contact3y" value="0.0" />
+<xacro:property name="base_contact3z" value="0.083" />
 <xacro:property name="proximal_contactx" value="0.00" />
 <xacro:property name="proximal_contacty" value="0.01" />
@@ -249,4 +252,16 @@
         </geometry>
       </collision>
+      <collision>
+        <origin rpy="0 0 0" xyz="${base_contact3x} ${base_contact3y} ${base_contact3z}"/>
+        <geometry>
+          <sphere radius="0"/>
+        </geometry>
+      </collision>
+       <collision>
+        <origin rpy="0 0 0" xyz="${-base_contact3x} ${base_contact3y} ${base_contact3z}"/>
+        <geometry>
+          <sphere radius="0"/>
+        </geometry>
+      </collision>
     <visual>
       <geometry>
@@ -333,4 +348,10 @@
         </geometry>
       </collision>
+       <collision>
+        <origin rpy="0 0 0" xyz="${distal_contactx} ${-distal_contacty} ${distal_contactz}"/>
+        <geometry>
+          <sphere radius="0"/>
+        </geometry>
+      </collision>
     <visual>
       <geometry>
@@ -417,4 +438,10 @@
         </geometry>
       </collision>
+       <collision>
+        <origin rpy="0 0 0" xyz="${distal_contactx} ${-distal_contacty} ${distal_contactz}"/>
+        <geometry>
+          <sphere radius="0"/>
+        </geometry>
+      </collision>
     <visual>
       <geometry>
@@ -475,4 +502,10 @@
        <collision>
         <origin rpy="0 0 0" xyz="${distal_contactx} ${distal_contacty} ${distal_contactz}"/>
+        <geometry>
+          <sphere radius="0"/>
+        </geometry>
+      </collision>
+       <collision>
+        <origin rpy="0 0 0" xyz="${distal_contactx} ${-distal_contacty} ${distal_contactz}"/>
         <geometry>
           <sphere radius="0"/>

File: software/models/mit_gazebo_models/mit_robot_hands/drake_urdfs/xacro/sandia_hand_simple_shapes_drake.urdf.xacro (robot description, xacro)
@@ -257,4 +257,23 @@
       <parent link="${side}_f${idx}_2"/>
       <child link="${side}_f${idx}_2_accel_dummy1"/>
+      <origin xyz="0.04 0 0" rpy="-${M_pi/2} 0 0"/>
+    </joint>
+     <link name="${side}_f${idx}_2_accel_dummy2">
+      <origin xyz="0 0 0" rpy="0 0 0"/>
+      <inertial>
+        <mass value="0.001"/>
+        <origin xyz="0 0 0"/>
+        <inertia ixx="0.01" ixy="0" ixz="0" iyy="0.01" iyz="0" izz="0.01"/>
+      </inertial>
+      <collision>
+        <origin rpy="0 0 0" xyz="0.0 0.0 -0.01"/>
+        <geometry>
+          <sphere radius="0"/>
+        </geometry>
+      </collision>
+    </link>
+     <joint name="${side}_f${idx}_2_accel_dummy2" type="fixed">
+      <parent link="${side}_f${idx}_2"/>
+      <child link="${side}_f${idx}_2_accel_dummy2"/>
       <origin xyz="0.04 0 0" rpy="-${M_pi/2} 0 0"/>
     </joint>
@@ -558,4 +577,23 @@
       <parent link="${side}_f${idx}_2"/>
       <child link="${side}_f${idx}_2_accel_dummy1"/>
+      <origin xyz="0.04 0 0" rpy="-${M_pi/2} 0 0"/>
+    </joint>
+     <link name="${side}_f${idx}_2_accel_dummy2">
+      <origin xyz="0 0 0" rpy="0 0 0"/>
+      <inertial>
+        <mass value="0.001"/>
+        <origin xyz="0 0 0"/>
+        <inertia ixx="0.01" ixy="0" ixz="0" iyy="0.01" iyz="0" izz="0.01"/>
+      </inertial>
+      <collision>
+        <origin rpy="0 0 0" xyz="0.0 0.0 -0.01"/>
+        <geometry>
+          <sphere radius="0"/>
+        </geometry>
+      </collision>
+    </link>
+     <joint name="${side}_f${idx}_2_accel_dummy2" type="fixed">
+      <parent link="${side}_f${idx}_2"/>
+      <child link="${side}_f${idx}_2_accel_dummy2"/>
       <origin xyz="0.04 0 0" rpy="-${M_pi/2} 0 0"/>
     </joint>
