Commit message: reverting changes to sandia_hand_drake_left.urdf related to hook contact points. Was breaking sticky hands, Andres will make a separate URDF and xacro for his purposes.
git-svn-id: https://svn.csail.mit.edu/drc@4845 c7283977-0100-402a-a91a-fa70b306dbfe

File: software/models/mit_gazebo_models/mit_robot_hands/drake_urdfs/sandia_hand_drake_left.urdf (robot description, URDF)
Before this commit: robot sandia_hand_left, 38 links, 37 joints
Links:
- removed link left_hook
Joints:
- removed joint left_hook_joint

File: software/models/mit_gazebo_models/mit_robot_hands/drake_urdfs/sandia_hand_drake_right.urdf (robot description, URDF)
Before this commit: robot sandia_hand_right, 38 links, 37 joints
Links:
- removed link right_hook
Joints:
- removed joint right_hook_joint

File: software/models/mit_gazebo_models/mit_robot_hands/drake_urdfs/xacro/sandia_hand_simple_shapes_drake.urdf.xacro (robot description, xacro)
@@ -15,18 +15,4 @@
   <include filename="$(find sandia_hand_description)/urdf/sandia_hand.transmission.xacro" />
   <xacro:property name="M_pi" value="3.1415926535897931" />
-  <xacro:macro name="collision_point" params="group xyz visualize">
-    <collision group="${group}">
-      <origin rpy="0 0 0" xyz="${xyz}"/>
-      <geometry>
-        <sphere radius="0"/>
-      </geometry>
-    </collision>
-    <visual>
-      <origin rpy="0 0 0" xyz="${xyz}"/>
-      <geometry>
-        <sphere radius="${visualize*0.01}"/>
-      </geometry>
-    </visual>
-  </xacro:macro>
   <xacro:macro name="finger" params="idx x y z r p yaw side reflect">
     <link name="${side}_f${idx}_base">
@@ -246,5 +232,5 @@
       <!-- ############ MIT ADDITION ############ -->
       <collision>
-        <origin rpy="0 0 0" xyz="0 0 0.001"/>
+        <origin rpy="0 0 0" xyz="0 0 0.01"/>
         <geometry>
           <sphere radius="0"/>
@@ -332,5 +318,5 @@
     </inertial>
     <collision>
-      <origin rpy="0 0 0" xyz="0.058 0 0.034"/>
+      <origin rpy="0 0 0" xyz="0.058 0 0.034"/> <!--TODO: THERE IS A ERROR HERE: xyz needs to be "0.058 0 0.034" instead of "0.1 0 0.05"-->
       <geometry>
         <sphere radius="0"/>
@@ -547,5 +533,5 @@
       <!-- ############ MIT ADDITION ############ -->
       <collision>
-        <origin rpy="0 0 0" xyz="0 0 0.001"/>
+        <origin rpy="0 0 0" xyz="0 0 0.01"/>
         <geometry>
           <sphere radius="0"/>
@@ -765,13 +751,4 @@
       <child link="${side}_palm"/>
       <insert_block name="origin" />
-    </joint>
-    <link name="${side}_hook">
-      <xacro:collision_point group="default" xyz="-0.045 ${reflect*0.015} -0.03" visualize="1"/>
-      <xacro:collision_point group="default" xyz="-0.045 ${reflect*0.015} 0.03" visualize="1"/>
-    </link>
-    <joint name="${side}_hook_joint" type="fixed">
-      <origin xyz="0.044 ${-0.04*reflect} -0.005" rpy="0 0 ${0.79*reflect}"/>
-      <parent link="${side}_palm"/>
-      <child link="${side}_hook"/>
     </joint>
     <xacro:finger side="${side}" idx="0" x="0.140" y="0.00000" z="0" r="0" p="0" yaw="${0.3*reflect}" reflect="${reflect}" />

Commit message: changing the sticky hand urdfs for better seeds
git-svn-id: https://svn.csail.mit.edu/drc/trunk@6165 c7283977-0100-402a-a91a-fa70b306dbfe

File: software/models/mit_gazebo_models/mit_robot_hands/drake_urdfs/sandia_hand_drake_left.urdf (robot description, URDF)
Before this commit: robot sandia_hand_left, 41 links, 40 joints
Joints:
- joint left_f3_j0: limit lower=-1.57079632679 upper=1.57079632679 effort=1 velocity=1 -> lower=-1.1780972451 upper=0 effort=1 velocity=1

File: software/models/mit_gazebo_models/mit_robot_hands/drake_urdfs/sandia_hand_drake_right.urdf (robot description, URDF)
Before this commit: robot sandia_hand_right, 41 links, 40 joints
Joints:
- joint right_f3_j0: limit lower=-1.57079632679 upper=1.57079632679 effort=1 velocity=1 -> lower=-1.1780972451 upper=0 effort=1 velocity=1

File: software/models/mit_gazebo_models/mit_robot_hands/drake_urdfs/xacro/sandia_hand_simple_shapes_drake.urdf.xacro (robot description, xacro)
@@ -608,5 +608,5 @@
       <parent link="${side}_f${idx}_base"/>
       <child link="${side}_f${idx}_0"/>
-      <limit lower="-${M_pi/2}" upper="${M_pi/2}" effort="1" velocity="1"/>
+      <limit lower="-${M_pi/2-M_pi/8}" upper="0" effort="1" velocity="1"/>
       <safety_controller soft_lower_limit="${-1.57079-10.0}" soft_upper_limit="${1.57079+10.0}" k_position="1000.0" k_velocity="1000.0"/>
       <dynamics damping="0.2"/>

Commit message: updating urdf for conservative limits on thumb
git-svn-id: https://svn.csail.mit.edu/drc/trunk@6303 c7283977-0100-402a-a91a-fa70b306dbfe

File: software/models/mit_gazebo_models/mit_robot_hands/drake_urdfs/sandia_hand_drake_left.urdf (robot description, URDF)
Before this commit: robot sandia_hand_left, 41 links, 40 joints
Joints:
- joint left_f3_j0: limit lower=-1.1780972451 upper=0 effort=1 velocity=1 -> lower=-0.785398163397 upper=0.785398163397 effort=1 velocity=1

File: software/models/mit_gazebo_models/mit_robot_hands/drake_urdfs/sandia_hand_drake_right.urdf (robot description, URDF)
Before this commit: robot sandia_hand_right, 41 links, 40 joints
Joints:
- joint right_f3_j0: limit lower=-1.1780972451 upper=0 effort=1 velocity=1 -> lower=-0.785398163397 upper=0.785398163397 effort=1 velocity=1

File: software/models/mit_gazebo_models/mit_robot_hands/drake_urdfs/xacro/sandia_hand_simple_shapes_drake.urdf.xacro (robot description, xacro)
@@ -608,5 +608,5 @@
       <parent link="${side}_f${idx}_base"/>
       <child link="${side}_f${idx}_0"/>
-      <limit lower="-${M_pi/2-M_pi/8}" upper="0" effort="1" velocity="1"/>
+      <limit lower="-${M_pi/2-M_pi/4}" upper="${M_pi/4}" effort="1" velocity="1"/>
       <safety_controller soft_lower_limit="${-1.57079-10.0}" soft_upper_limit="${1.57079+10.0}" k_position="1000.0" k_velocity="1000.0"/>
       <dynamics damping="0.2"/>
