Commit message: updating inertial values of hands
git-svn-id: https://svn.csail.mit.edu/drc/trunk@6348 c7283977-0100-402a-a91a-fa70b306dbfe

File: software/models/mit_gazebo_models/mit_robot_hands/drake_urdfs/irobot_hand_drake_left.urdf (robot description, URDF)
Before this commit: robot irobot_hand_left, 10 links, 9 joints
Links:
- link base: mass 0.1 -> 0.001

File: software/models/mit_gazebo_models/mit_robot_hands/drake_urdfs/irobot_hand_drake_right.urdf (robot description, URDF)
Before this commit: robot irobot_hand_right, 10 links, 9 joints
Links:
- link base: mass 0.1 -> 0.001

File: software/models/mit_gazebo_models/mit_robot_hands/drake_urdfs/sandia_hand_drake_left.urdf (robot description, URDF)
Before this commit: robot sandia_hand_left, 41 links, 40 joints
Links:
- link base: mass 0.1 -> 0.001
- link left_f0_0: mass 0.05 -> 0.106
- link left_f0_1: mass 0.05 -> 0.033
- link left_f0_1_accel: mass 0.001 -> 0.01
- link left_f0_2: mass 0.05 -> 0.033
- link left_f0_2_accel: mass 0.001 -> 0.01
- link left_f0_base: mass 0.35 -> 0.250
- link left_f0_fixed_accel: mass 0.001 -> 0.01
- link left_f1_0: mass 0.05 -> 0.106
- link left_f1_1: mass 0.05 -> 0.033
- link left_f1_1_accel: mass 0.001 -> 0.01
- link left_f1_2: mass 0.05 -> 0.033
- link left_f1_2_accel: mass 0.001 -> 0.01
- link left_f1_base: mass 0.35 -> 0.250
- link left_f1_fixed_accel: mass 0.001 -> 0.01
- link left_f2_0: mass 0.05 -> 0.106
- link left_f2_1: mass 0.05 -> 0.033
- link left_f2_1_accel: mass 0.001 -> 0.01
- link left_f2_2: mass 0.05 -> 0.033
- link left_f2_2_accel: mass 0.001 -> 0.01
- link left_f2_base: mass 0.35 -> 0.250
- link left_f2_fixed_accel: mass 0.001 -> 0.01
- link left_palm: mass 0.3 -> 1.303

File: software/models/mit_gazebo_models/mit_robot_hands/drake_urdfs/sandia_hand_drake_right.urdf (robot description, URDF)
Before this commit: robot sandia_hand_right, 41 links, 40 joints
Links:
- link base: mass 0.1 -> 0.001
- link right_f0_0: mass 0.05 -> 0.106
- link right_f0_1: mass 0.05 -> 0.033
- link right_f0_1_accel: mass 0.001 -> 0.01
- link right_f0_2: mass 0.05 -> 0.033
- link right_f0_2_accel: mass 0.001 -> 0.01
- link right_f0_base: mass 0.35 -> 0.250
- link right_f0_fixed_accel: mass 0.001 -> 0.01
- link right_f1_0: mass 0.05 -> 0.106
- link right_f1_1: mass 0.05 -> 0.033
- link right_f1_1_accel: mass 0.001 -> 0.01
- link right_f1_2: mass 0.05 -> 0.033
- link right_f1_2_accel: mass 0.001 -> 0.01
- link right_f1_base: mass 0.35 -> 0.250
- link right_f1_fixed_accel: mass 0.001 -> 0.01
- link right_f2_0: mass 0.05 -> 0.106
- link right_f2_1: mass 0.05 -> 0.033
- link right_f2_1_accel: mass 0.001 -> 0.01
- link right_f2_2: mass 0.05 -> 0.033
- link right_f2_2_accel: mass 0.001 -> 0.01
- link right_f2_base: mass 0.35 -> 0.250
- link right_f2_fixed_accel: mass 0.001 -> 0.01
- link right_palm: mass 0.3 -> 1.303

File: software/models/mit_gazebo_models/mit_robot_hands/drake_urdfs/xacro/irobot_hand_drake_left.urdf.xacro (robot description, xacro)
@@ -8,7 +8,7 @@
   <link name="base">
     <inertial>
-        <mass value="0.1" />
+        <mass value="0.001"/>
         <origin xyz="0 0 0.25" rpy="0 0 0" />
-        <inertia ixx="0.01" ixy="0" ixz="0" iyy="0.01" iyz="0" izz="0.01" />
+        <inertia ixx="0.000001" ixy="0" ixz="0" iyy="0.000001" iyz="0" izz="0.000001"/>
     </inertial>
   </link>

File: software/models/mit_gazebo_models/mit_robot_hands/drake_urdfs/xacro/irobot_hand_drake_right.urdf.xacro (robot description, xacro)
@@ -8,7 +8,7 @@
   <link name="base">
     <inertial>
-        <mass value="0.1" />
+        <mass value="0.001"/>
         <origin xyz="0 0 0.25" rpy="0 0 0" />
-        <inertia ixx="0.01" ixy="0" ixz="0" iyy="0.01" iyz="0" izz="0.01" />
+        <inertia ixx="0.000001" ixy="0" ixz="0" iyy="0.000001" iyz="0" izz="0.000001"/>
     </inertial>
   </link>

File: software/models/mit_gazebo_models/mit_robot_hands/drake_urdfs/xacro/sandia_hand_drake_left.urdf.xacro (robot description, xacro)
@@ -10,7 +10,7 @@
   <link name="base">
     <inertial>
-        <mass value="0.1" />
+        <mass value="0.001"/>
         <origin xyz="0 0 0.25" rpy="0 0 0" />
-        <inertia ixx="0.01" ixy="0" ixz="0" iyy="0.01" iyz="0" izz="0.01" />
+        <inertia ixx="0.000001" ixy="0" ixz="0" iyy="0.000001" iyz="0" izz="0.000001"/>
     </inertial>
    <!-- <visual>

File: software/models/mit_gazebo_models/mit_robot_hands/drake_urdfs/xacro/sandia_hand_drake_right.urdf.xacro (robot description, xacro)
@@ -10,7 +10,7 @@
   <link name="base">
     <inertial>
-        <mass value="0.1" />
+        <mass value="0.001"/>
         <origin xyz="0 0 0.25" rpy="0 0 0" />
-        <inertia ixx="0.01" ixy="0" ixz="0" iyy="0.01" iyz="0" izz="0.01" />
+        <inertia ixx="0.000001" ixy="0" ixz="0" iyy="0.000001" iyz="0" izz="0.000001"/>
     </inertial>
  <!--   <visual>

File: software/models/mit_gazebo_models/mit_robot_hands/drake_urdfs/xacro/sandia_hand_simple_shapes_drake.urdf.xacro (robot description, xacro)
@@ -19,7 +19,9 @@
       <origin xyz="0 0 0" rpy="0 0 0"/>
       <inertial>
-        <mass value="0.35"/>
-        <origin xyz="0 0 0"/>
-        <inertia ixx="0.01" ixy="0" ixz="0" iyy="0.01" iyz="0" izz="0.01"/>
+        <!-- total mass is 2.303 kg, palm is about 1.303 kg, distribute the rest into _base -->
+        <mass value="0.250"/> <!-- (2.303 - 1.303) / 4 -->
+        <origin xyz="0 0 0"/>
+        <!-- model as sphere with radius of 1cm -->
+        <inertia ixx="0.00001" ixy="0" ixz="0" iyy="0.00001" iyz="0" izz="0.00001"/>
       </inertial>
     </link>
@@ -27,7 +29,7 @@
       <origin xyz="0 0 0" rpy="0 0 0"/>
       <inertial>
-        <mass value="0.001"/>
-        <origin xyz="0 0 0"/>
-        <inertia ixx="0.01" ixy="0" ixz="0" iyy="0.01" iyz="0" izz="0.01"/>
+        <mass value="0.01"/>
+        <origin xyz="0 0 0"/>
+        <inertia ixx="0.000001" ixy="0" ixz="0" iyy="0.000001" iyz="0" izz="0.000001"/>
       </inertial>
       <!-- ############ MIT ADDITION ############ -->
@@ -43,7 +45,8 @@
       <origin xyz="0 0 0" rpy="0 0 0"/>
       <inertial>
-        <mass value="0.05"/>
-        <origin xyz="0 0 0"/>
-        <inertia ixx="0.01" ixy="0" ixz="0" iyy="0.01" iyz="0" izz="0.01"/>
+		<mass value="0.106"/> <!-- F1 -->
+        <origin xyz="0 0 0"/>
+        <!-- solid cylinder -->
+        <inertia ixx="0.000011925" ixy="0" ixz="0" iyy="0.00011505" iyz="0" izz="0.00011505"/>
       </inertial>
       <!-- begin simple shape approximation of f0 -->
@@ -104,7 +107,8 @@
       <origin xyz="0 0 0" rpy="0 0 0"/>
       <inertial>
-        <mass value="0.05"/>
-        <origin xyz="0 0 0"/>
-        <inertia ixx="0.01" ixy="0" ixz="0" iyy="0.01" iyz="0" izz="0.01"/>
+        <mass value="0.033"/> <!-- F2 -->
+        <origin xyz="0 0 0"/>
+        <!-- solid cylinder -->
+        <inertia ixx="0.00000165" ixy="0" ixz="0" iyy="0.00001316975" iyz="0" izz="0.00001316975"/>
       </inertial>
       <!-- begin simple shape approximation of f1 -->
@@ -150,7 +154,7 @@
       <origin xyz="0 0 0" rpy="0 0 0"/>
       <inertial>
-        <mass value="0.001"/>
-        <origin xyz="0 0 0"/>
-        <inertia ixx="0.01" ixy="0" ixz="0" iyy="0.01" iyz="0" izz="0.01"/>
+        <mass value="0.01"/>
+        <origin xyz="0 0 0"/>
+        <inertia ixx="0.000001" ixy="0" ixz="0" iyy="0.000001" iyz="0" izz="0.000001"/>
       </inertial>
       <!-- ############ MIT ADDITION ############ -->
@@ -166,7 +170,8 @@
       <origin xyz="0 0 0" rpy="0 0 0"/>
       <inertial>
-        <mass value="0.05"/>
-        <origin xyz="0 0 0"/>
-        <inertia ixx="0.01" ixy="0" ixz="0" iyy="0.01" iyz="0" izz="0.01"/>
+        <mass value="0.033"/>  <!-- F3 -->
+        <origin xyz="0 0 0"/>
+        <!-- solid cylinder -->
+        <inertia ixx="0.0000013365" ixy="0" ixz="0" iyy="0.000009603" iyz="0" izz="0.000009603"/>
       </inertial>
       <!-- begin simple shape approximation of f2 -->
@@ -226,7 +231,7 @@
       <origin xyz="0 0 0" rpy="0 0 0"/>
       <inertial>
-        <mass value="0.001"/>
-        <origin xyz="0 0 0"/>
-        <inertia ixx="0.01" ixy="0" ixz="0" iyy="0.01" iyz="0" izz="0.01"/>
+        <mass value="0.01"/>
+        <origin xyz="0 0 0"/>
+        <inertia ixx="0.000001" ixy="0" ixz="0" iyy="0.000001" iyz="0" izz="0.000001"/>
       </inertial>
       <!-- ############ MIT ADDITION ############ -->
@@ -652,7 +657,8 @@
       <origin xyz="0 0 0" rpy="0 0 0"/>
       <inertial>
-        <mass value="0.3"/>
-        <origin xyz="0 0 0"/>
-        <inertia ixx="0.01" ixy="0" ixz="0" iyy="0.01" iyz="0" izz="0.01"/>
+        <mass value="1.303"/>
+        <origin xyz="0 0 0"/>
+        <!-- solid sphere with 5cm radius -->
+        <inertia ixx="0.001303" ixy="0" ixz="0" iyy="0.001303" iyz="0" izz="0.001303"/>
       </inertial>
       <!-- begin simple shape approximation of palm -->
