Commit message: updated the dof ranges for the feets
git-svn-id: https://svn.csail.mit.edu/drc@4685 c7283977-0100-402a-a91a-fa70b306dbfe

File: software/models/mit_gazebo_models/mit_robot_feet/l_foot.urdf (robot description, URDF)
Before this commit: robot left_foot, 3 links, 2 joints
Joints:
- joint l_leg_uay: limit lower=-0.698 upper=0.698 effort=220 velocity=12 -> lower=-0.9 upper=0.698 effort=220 velocity=12

File: software/models/mit_gazebo_models/mit_robot_feet/r_foot.urdf (robot description, URDF)
Before this commit: robot right_foot, 3 links, 2 joints
Joints:
- joint r_leg_uay: limit lower=-0.698 upper=0.698 effort=220 velocity=12 -> lower=-0.9 upper=0.698 effort=220 velocity=12

Commit message: plane markers for feet and urdf for pelvis and com markers
git-svn-id: https://svn.csail.mit.edu/drc/trunk@6454 c7283977-0100-402a-a91a-fa70b306dbfe

File: software/models/mit_gazebo_models/mit_robot_feet/l_foot.urdf (robot description, URDF)
Before this commit: robot left_foot, 3 links, 2 joints
Links:
- removed link base
- added link plane::xy::base, mass 0.1
Joints:
- joint l_leg_aky: parent base -> plane::xy::base

File: software/models/mit_gazebo_models/mit_robot_feet/r_foot.urdf (robot description, URDF)
Before this commit: robot right_foot, 3 links, 2 joints
Links:
- removed link base
- added link plane::xy::base, mass 0.1
Joints:
- joint r_leg_aky: parent base -> plane::xy::base
