Commit message: plananr markers enabled for sticky hand based keyframe adjustment
git-svn-id: https://svn.csail.mit.edu/drc/trunk@6455 c7283977-0100-402a-a91a-fa70b306dbfe

File: software/models/mit_gazebo_models/mit_robot_hands/irobot_hand_left.urdf (robot description, URDF)
Before this commit: robot irobot_hand_left, 10 links, 9 joints
Links:
- removed link base
- added link plane::xy::base, mass 0.1
Joints:
- joint left_irobot_hand_joint: parent base -> plane::xy::base

File: software/models/mit_gazebo_models/mit_robot_hands/irobot_hand_right.urdf (robot description, URDF)
Before this commit: robot irobot_hand_right, 10 links, 9 joints
Links:
- removed link base
- added link plane::xy::base, mass 0.1
Joints:
- joint right_irobot_hand_joint: parent base -> plane::xy::base

File: software/models/mit_gazebo_models/mit_robot_hands/sandia_hand_left.urdf (robot description, URDF)
Before this commit: robot sandia_hand_left, 34 links, 33 joints
Links:
- removed link base
- added link plane::xy::base, mass 0.1
Joints:
- joint left_sandia_hand_joint: parent base -> plane::xy::base

File: software/models/mit_gazebo_models/mit_robot_hands/sandia_hand_right.urdf (robot description, URDF)
Before this commit: robot sandia_hand_right, 34 links, 33 joints
Links:
- removed link base
- added link plane::xy::base, mass 0.1
Joints:
- joint right_sandia_hand_joint: parent base -> plane::xy::base

File: software/models/mit_gazebo_models/mit_robot_hands/xacro/irobot_hand_left.urdf.xacro (robot description, xacro)
@@ -5,5 +5,5 @@
        name="irobot_hand_left" >
   <include filename="$(find mit_drcsim_scripts)/models/mit_robot_hands/xacro/irobot_hand_simple.urdf.xacro" />
-  <link name="base">
+  <link name="plane::xy::base">
     <inertial>
         <mass value="0.1" />
@@ -12,5 +12,5 @@
     </inertial>
   </link>
-  <xacro:irobot_hand side="left" parent="base" reflect="-1">
+  <xacro:irobot_hand side="left" parent="plane::xy::base" reflect="-1">
 <!--    <origin rpy="0 0 3.14159" xyz="0 0.05 0"/>-->
     <origin rpy="1.57 0 -1.57" xyz="0 0 0"/>

File: software/models/mit_gazebo_models/mit_robot_hands/xacro/irobot_hand_right.urdf.xacro (robot description, xacro)
@@ -5,5 +5,5 @@
        name="irobot_hand_right" >
   <include filename="$(find mit_drcsim_scripts)/models/mit_robot_hands/xacro/irobot_hand_simple.urdf.xacro" />
-  <link name="base">
+  <link name="plane::xy::base">
     <inertial>
         <mass value="0.1" />
@@ -12,5 +12,5 @@
     </inertial>
   </link>
-  <xacro:irobot_hand side="right" parent="base" reflect="1">
+  <xacro:irobot_hand side="right" parent="plane::xy::base" reflect="1">
  <!--  <origin rpy="0 0 0" xyz="0 -0.05 0"/>-->
     <origin rpy="1.57 0 -1.57" xyz="0 0 0"/>

File: software/models/mit_gazebo_models/mit_robot_hands/xacro/sandia_hand_left.urdf.xacro (robot description, xacro)
@@ -8,5 +8,5 @@
   <!--<include filename="$(find sandia_hand_description)/urdf/sandia_hand.urdf.xacro" />-->
   <include filename="$(find sandia_hand_description)/urdf/sandia_hand_simple_shapes.urdf.xacro" />
-  <link name="base">
+  <link name="plane::xy::base">
     <inertial>
         <mass value="0.1" />
@@ -27,5 +27,5 @@
     </collision> -->
   </link>
-   <xacro:sandia_hand side="left" parent="base" reflect="-1" joint_type="revolute" thumb_angle="0">
+   <xacro:sandia_hand side="left" parent="plane::xy::base" reflect="-1" joint_type="revolute" thumb_angle="0">
     <origin xyz="0 0 0.0" rpy="0 -1.57079 0"/>
   </xacro:sandia_hand>

File: software/models/mit_gazebo_models/mit_robot_hands/xacro/sandia_hand_right.urdf.xacro (robot description, xacro)
@@ -8,5 +8,5 @@
   <!--<include filename="$(find sandia_hand_description)/urdf/sandia_hand.urdf.xacro" />-->
   <include filename="$(find sandia_hand_description)/urdf/sandia_hand_simple_shapes.urdf.xacro" />
-  <link name="base">
+  <link name="plane::xy::base">
     <inertial>
         <mass value="0.1" />
@@ -27,5 +27,5 @@
     </collision> -->
   </link>
-  <xacro:sandia_hand side="right" parent="base" reflect="1" joint_type="revolute" thumb_angle="0">
+  <xacro:sandia_hand side="right" parent="plane::xy::base" reflect="1" joint_type="revolute" thumb_angle="0">
     <origin xyz="0 0 0.0" rpy="0 -1.57079 0"/>
   </xacro:sandia_hand>
