Commit message: adding priliinary support for bdi hook hands
git-svn-id: https://svn.csail.mit.edu/drc/trunk@7721 c7283977-0100-402a-a91a-fa70b306dbfe

File: software/models/mit_gazebo_models/mit_robot_hands/inert_hand_left.urdf (robot description, URDF)
Before this commit: robot inert_hand_left, 2 links, 1 joints
Joints:
- joint left_hook_hand_joint: origin xyz=0 0 0 rpy=1.57 0.0 -1.57 -> xyz=0.0 0.0 0.0 rpy=1.57 -1.57 -1.57

File: software/models/mit_gazebo_models/mit_robot_hands/xacro/inert_hand_left.urdf.xacro (robot description, xacro)
@@ -4,5 +4,4 @@
        xmlns:xacro="http://playerstage.sourceforge.net/gazebo/xmlschema/#interface"
        name="inert_hand_left" >
-  <xacro:include filename="$(find hook_description)/src/hook_hand_simple.urdf.xacro" />
   <link name="plane::xy::base">
     <inertial>
@@ -12,7 +11,11 @@
     </inertial>
   </link>
-  <xacro:hook_hand side="left" parent="plane::xy::base" reflect="-1">
-<!--    <origin rpy="0 0 3.14159" xyz="0 0.05 0"/>-->
-    <origin rpy="1.57 0.0 -1.57" xyz="0 0 0"/>
+ <xacro:include filename="$(find hook_description)/src/hook_hand_simple.urdf.xacro" />
+  <xacro:hook_hand side="left" parent="plane::xy::base" reflect="-1" hookflip="1">
+    <origin rpy="1.57 -1.57 -1.57" xyz="0.0 0.0 0.0"/>
   </xacro:hook_hand>
+<!--  <xacro:include filename="$(find hook_description)/src/bdihook_hand.urdf.xacro" />-->
+<!--  <xacro:hook_hand side="left" parent="plane::xy::base" reflect="-1" hookflip="1">-->
+<!--    <origin rpy="1.57 -1.57 -1.57" xyz="0 0 0"/>   -->
+<!--  </xacro:hook_hand>    -->
 </robot>

File: software/models/mit_gazebo_models/mit_robot_hands/xacro/inert_hand_right.urdf.xacro (robot description, xacro)
@@ -4,5 +4,4 @@
        xmlns:xacro="http://playerstage.sourceforge.net/gazebo/xmlschema/#interface"
        name="inert_hand_right" >
-  <xacro:include filename="$(find hook_description)/src/hook_hand_simple.urdf.xacro" />
   <link name="plane::xy::base">
     <inertial>
@@ -12,7 +11,11 @@
     </inertial>
   </link>
-  <xacro:hook_hand side="right" parent="plane::xy::base" reflect="1">
- <!--  <origin rpy="0 0 0" xyz="0 -0.05 0"/>-->
+ <xacro:include filename="$(find hook_description)/src/hook_hand_simple.urdf.xacro" />
+  <xacro:hook_hand side="right" parent="plane::xy::base" reflect="1" hookflip="1">
     <origin rpy="1.57 0.0 -1.57" xyz="0 0 0"/>
   </xacro:hook_hand>
+<!--  <xacro:include filename="$(find hook_description)/src/bdihook_hand.urdf.xacro" />-->
+<!--  <xacro:hook_hand side="right" parent="plane::xy::base" reflect="1" hookflip="1">-->
+<!--    <origin rpy="1.57 -1.57 -1.57" xyz="0 0 0"/>   -->
+<!--  </xacro:hook_hand>  -->
 </robot>

Commit message: modifications to bdi hooks. By default its mit hooks
git-svn-id: https://svn.csail.mit.edu/drc/trunk@7728 c7283977-0100-402a-a91a-fa70b306dbfe

File: software/models/mit_gazebo_models/mit_robot_hands/inert_hand_left.urdf (robot description, URDF)
Before this commit: robot inert_hand_left, 2 links, 1 joints
Joints:
- joint left_hook_hand_joint: origin xyz=0.0 0.0 0.0 rpy=1.57 -1.57 -1.57 -> xyz=0.0 0.0 0.0 rpy=1.57 0.0 -1.57

File: software/models/mit_gazebo_models/mit_robot_hands/xacro/inert_hand_left.urdf.xacro (robot description, xacro)
@@ -13,9 +13,9 @@
  <xacro:include filename="$(find hook_description)/src/hook_hand_simple.urdf.xacro" />
   <xacro:hook_hand side="left" parent="plane::xy::base" reflect="-1" hookflip="1">
-    <origin rpy="1.57 -1.57 -1.57" xyz="0.0 0.0 0.0"/>
+    <origin rpy="1.57 0.0 -1.57" xyz="0.0 0.0 0.0"/>
   </xacro:hook_hand>
-<!--  <xacro:include filename="$(find hook_description)/src/bdihook_hand.urdf.xacro" />-->
+<!-- <xacro:include filename="$(find hook_description)/src/bdihook_hand.urdf.xacro" />-->
 <!--  <xacro:hook_hand side="left" parent="plane::xy::base" reflect="-1" hookflip="1">-->
-<!--    <origin rpy="1.57 -1.57 -1.57" xyz="0 0 0"/>   -->
-<!--  </xacro:hook_hand>    -->
+<!--    <origin rpy="1.57 0.0 -1.57" xyz="0.0 0.0 0.0"/>-->
+<!--  </xacro:hook_hand>-->
 </robot>

File: software/models/mit_gazebo_models/mit_robot_hands/xacro/inert_hand_right.urdf.xacro (robot description, xacro)
@@ -17,5 +17,5 @@
 <!--  <xacro:include filename="$(find hook_description)/src/bdihook_hand.urdf.xacro" />-->
 <!--  <xacro:hook_hand side="right" parent="plane::xy::base" reflect="1" hookflip="1">-->
-<!--    <origin rpy="1.57 -1.57 -1.57" xyz="0 0 0"/>   -->
+<!--    <origin rpy="1.57 3.14 -1.57" xyz="0 0 0"/>   -->
 <!--  </xacro:hook_hand>  -->
 </robot>

Commit message: collision element of bdi hook had wrong scaling
git-svn-id: https://svn.csail.mit.edu/drc/trunk@7829 c7283977-0100-402a-a91a-fa70b306dbfe

File: software/models/mit_gazebo_models/mit_robot_hands/inert_hand_left.urdf (robot description, URDF)
Before this commit: robot inert_hand_left, 2 links, 1 joints
Links:
- link left_base_link: geometry collision mesh filename=package://hook_description/meshes/bdi_hook.stl scale=1 1 1; visual mesh filename=package://hook_description/meshes/bdi_hook.stl scale=1 1 1

File: software/models/mit_gazebo_models/mit_robot_hands/inert_hand_right.urdf (robot description, URDF)
Before this commit: robot inert_hand_right, 2 links, 1 joints
Links:
- link right_base_link: geometry collision mesh filename=package://hook_description/meshes/bdi_hook.stl scale=1 1 1; visual mesh filename=package://hook_description/meshes/bdi_hook.stl scale=1 1 1

File: software/models/mit_gazebo_models/mit_robot_hands/xacro/inert_hand_left.urdf.xacro (robot description, xacro)
@@ -12,5 +12,5 @@
   </link>
  <xacro:include filename="$(find hook_description)/src/bdihook_hand.urdf.xacro" />
-  <xacro:hook_hand side="left" parent="plane::xy::base" reflect="-1" hookflip="1">
+  <xacro:hook_hand side="left" parent="plane::xy::base" reflect="-1" hookflip="-1">
     <origin rpy="1.57 0.0 -1.57" xyz="0.0 0.0 0.0"/>
  </xacro:hook_hand>

File: software/models/mit_gazebo_models/mit_robot_hands/xacro/inert_hand_right.urdf.xacro (robot description, xacro)
@@ -12,5 +12,5 @@
   </link>
   <xacro:include filename="$(find hook_description)/src/bdihook_hand.urdf.xacro" />
-   <xacro:hook_hand side="right" parent="plane::xy::base" reflect="1" hookflip="1">
+   <xacro:hook_hand side="right" parent="plane::xy::base" reflect="1" hookflip="-1">
      <origin rpy="1.57 3.14 -1.57" xyz="0 0 0"/>
   </xacro:hook_hand>

Commit message: ability to add 30 deg offsets to hook hands
git-svn-id: https://svn.csail.mit.edu/drc/trunk@7859 c7283977-0100-402a-a91a-fa70b306dbfe

File: software/models/mit_gazebo_models/mit_robot_hands/inert_hand_left.urdf (robot description, URDF)
Before this commit: robot inert_hand_left, 2 links, 1 joints
Joints:
- joint left_hook_hand_joint: origin xyz=0.0 0.0 0.0 rpy=1.57 0.0 -1.57 -> xyz=0.243 0.0 -0.127 rpy=1.57 0.0 -1.57

File: software/models/mit_gazebo_models/mit_robot_hands/inert_hand_right.urdf (robot description, URDF)
Before this commit: robot inert_hand_right, 2 links, 1 joints
Joints:
- joint right_hook_hand_joint: origin xyz=0 0 0 rpy=1.57 3.14 -1.57 -> xyz=0.243 0.0 -0.127 rpy=1.57 3.14 -1.57

File: software/models/mit_gazebo_models/mit_robot_hands/xacro/inert_hand_left.urdf.xacro (robot description, xacro)
@@ -12,6 +12,7 @@
   </link>
  <xacro:include filename="$(find hook_description)/src/bdihook_hand.urdf.xacro" />
-  <xacro:hook_hand side="left" parent="plane::xy::base" reflect="-1" hookflip="-1">
-    <origin rpy="1.57 0.0 -1.57" xyz="0.0 0.0 0.0"/>
+<!-- <xacro:include filename="$(find mit_drcsim_scripts)/models/mit_robot_hands/xacro/bdihook_hand.urdf.xacro" />-->
+  <xacro:hook_hand side="left" parent="plane::xy::base" reflect="-1" hookflip="-1" noof30degoffset="0">
+    <origin rpy="1.57 0.0 -1.57" xyz="0.243 0.0 -0.127"/>
  </xacro:hook_hand>
 </robot>

File: software/models/mit_gazebo_models/mit_robot_hands/xacro/inert_hand_right.urdf.xacro (robot description, xacro)
@@ -12,6 +12,6 @@
   </link>
   <xacro:include filename="$(find hook_description)/src/bdihook_hand.urdf.xacro" />
-   <xacro:hook_hand side="right" parent="plane::xy::base" reflect="1" hookflip="-1">
-     <origin rpy="1.57 3.14 -1.57" xyz="0 0 0"/>
+   <xacro:hook_hand side="right" parent="plane::xy::base" reflect="1" hookflip="-1" noof30degoffset="0">
+     <origin rpy="1.57 3.14 -1.57" xyz="0.243 0.0 -0.127"/>
   </xacro:hook_hand>
 </robot>

Commit message: fixing stand alone inert hands

File: software/models/mit_gazebo_models/mit_robot_hands/inert_hand_left.urdf (robot description, URDF)
Before this commit: robot inert_hand_left, 2 links, 1 joints
Links:
- added link left_pointer_tip
Joints:
- added joint left_pointer_tip_joint: type fixed, parent plane::xy::base, child left_pointer_tip, origin xyz=0 0.12 0 rpy=0.0 0.0 0.0

File: software/models/mit_gazebo_models/mit_robot_hands/inert_hand_right.urdf (robot description, URDF)
Before this commit: robot inert_hand_right, 2 links, 1 joints
Links:
- added link right_pointer_tip
Joints:
- added joint right_pointer_tip_joint: type fixed, parent plane::xy::base, child right_pointer_tip, origin xyz=0 0.12 0 rpy=0.0 0.0 0.0

File: software/models/mit_gazebo_models/mit_robot_hands/xacro/inert_hand_left.urdf.xacro (robot description, xacro)
@@ -13,5 +13,5 @@
 <!-- <xacro:include filename="$(find hook_description)/src/bdihook_hand.urdf.xacro" />  -->
  <xacro:include filename="$(find hook_description)/src/hook_hand_simple.urdf.xacro" />
-  <xacro:hook_hand side="left" parent="plane::xy::base" reflect="-1" hookflip="-1" noof30degoffset="0">
+  <xacro:hook_hand side="left" parent="plane::xy::base" >
     <origin rpy="1.57 0.0 -1.57" xyz="0.243 0.0 -0.127"/>
  </xacro:hook_hand>

File: software/models/mit_gazebo_models/mit_robot_hands/xacro/inert_hand_right.urdf.xacro (robot description, xacro)
@@ -13,5 +13,5 @@
 <!--  <xacro:include filename="$(find hook_description)/src/bdihook_hand.urdf.xacro" />  -->
   <xacro:include filename="$(find hook_description)/src/hook_hand_simple.urdf.xacro" />
-   <xacro:hook_hand side="right" parent="plane::xy::base" reflect="1" hookflip="-1" noof30degoffset="0">
+   <xacro:hook_hand side="right" parent="plane::xy::base">
      <origin rpy="1.57 3.14 -1.57" xyz="0.243 0.0 -0.127"/>
   </xacro:hook_hand>
