Commit message: renaming val hand meshes to be found by designer

File: software/models/mit_gazebo_models/mit_robot_hands/valkyrie_hand_left.urdf (robot description, URDF)
Before this commit: robot valkyrie_hand_left, 17 links, 16 joints
Links:
- link /v1/LeftLittleDistalPhalanx: geometry collision mesh filename=package://valkyrie/meshes/sf3_ssf4.stl; visual mesh filename=package://valkyrie/meshes/sf3_ssf4.stl
- link /v1/LeftLittleMedialPhalanx: geometry collision mesh filename=package://valkyrie/meshes/sf2_ssf3.stl; visual mesh filename=package://valkyrie/meshes/sf2_ssf3.stl
- link /v1/LeftLittleProximalPhalanx: geometry collision mesh filename=package://valkyrie/meshes/ssf2_Left.stl; visual mesh filename=package://valkyrie/meshes/ssf2_Left.stl
- link /v1/LeftMedialMetacarpal: geometry collision mesh filename=package://valkyrie/meshes/ssf1_Left.stl; visual mesh filename=package://valkyrie/meshes/ssf1_Left.stl
- link /v1/LeftMiddleDistalPhalanx: geometry collision mesh filename=package://valkyrie/meshes/sf3_ssf4.stl; visual mesh filename=package://valkyrie/meshes/sf3_ssf4.stl
- link /v1/LeftMiddleMedialPhalanx: geometry collision mesh filename=package://valkyrie/meshes/sf2_ssf3.stl; visual mesh filename=package://valkyrie/meshes/sf2_ssf3.stl
- link /v1/LeftMiddleProximalPhalanx: geometry collision mesh filename=package://valkyrie/meshes/sf1.stl; visual mesh filename=package://valkyrie/meshes/sf1.stl
- link /v1/LeftPrimaryDistalPhalanx: geometry collision mesh filename=package://valkyrie/meshes/pf4.stl; visual mesh filename=package://valkyrie/meshes/pf4.stl
- link /v1/LeftPrimaryMedialPhalanx: geometry collision mesh filename=package://valkyrie/meshes/pf3.stl; visual mesh filename=package://valkyrie/meshes/pf3.stl
- link /v1/LeftPrimaryMetacarpal: geometry collision mesh filename=package://valkyrie/meshes/pf1.stl; visual mesh filename=package://valkyrie/meshes/pf1.stl
- link /v1/LeftPrimaryProximalPhalanx: geometry collision mesh filename=package://valkyrie/meshes/pf2.stl; visual mesh filename=package://valkyrie/meshes/pf2.stl
- link /v1/LeftThumbDistalPhalanx: geometry collision mesh filename=package://valkyrie/meshes/tf4.stl; visual mesh filename=package://valkyrie/meshes/tf4.stl
- link /v1/LeftThumbMedialPhalanx: geometry collision mesh filename=package://valkyrie/meshes/tf3.stl; visual mesh filename=package://valkyrie/meshes/tf3.stl
- link /v1/LeftThumbMetacarpal: geometry collision mesh filename=package://valkyrie/meshes/tf1_Left.stl; visual mesh filename=package://valkyrie/meshes/tf1_Left.stl
- link /v1/LeftThumbProximalPhalanx: geometry collision mesh filename=package://valkyrie/meshes/tf2.stl; visual mesh filename=package://valkyrie/meshes/tf2.stl
- link left_palm: geometry collision mesh filename=package://valkyrie/meshes/palm_Left.stl; visual mesh filename=package://valkyrie/meshes/palm_Left.stl

File: software/models/mit_gazebo_models/mit_robot_hands/valkyrie_hand_right.urdf (robot description, URDF)
Before this commit: robot valkyrie_hand_right, 17 links, 16 joints
Links:
- link /v1/RightLittleDistalPhalanx: geometry collision mesh filename=package://valkyrie/meshes/sf3_ssf4.stl; visual mesh filename=package://valkyrie/meshes/sf3_ssf4.stl
- link /v1/RightLittleMedialPhalanx: geometry collision mesh filename=package://valkyrie/meshes/sf2_ssf3.stl; visual mesh filename=package://valkyrie/meshes/sf2_ssf3.stl
- link /v1/RightLittleProximalPhalanx: geometry collision mesh filename=package://valkyrie/meshes/ssf2_Right.stl; visual mesh filename=package://valkyrie/meshes/ssf2_Right.stl
- link /v1/RightMedialMetacarpal: geometry collision mesh filename=package://valkyrie/meshes/ssf1_Right.stl; visual mesh filename=package://valkyrie/meshes/ssf1_Right.stl
- link /v1/RightMiddleDistalPhalanx: geometry collision mesh filename=package://valkyrie/meshes/sf3_ssf4.stl; visual mesh filename=package://valkyrie/meshes/sf3_ssf4.stl
- link /v1/RightMiddleMedialPhalanx: geometry collision mesh filename=package://valkyrie/meshes/sf2_ssf3.stl; visual mesh filename=package://valkyrie/meshes/sf2_ssf3.stl
- link /v1/RightMiddleProximalPhalanx: geometry collision mesh filename=package://valkyrie/meshes/sf1.stl; visual mesh filename=package://valkyrie/meshes/sf1.stl
- link /v1/RightPrimaryDistalPhalanx: geometry collision mesh filename=package://valkyrie/meshes/pf4.stl; visual mesh filename=package://valkyrie/meshes/pf4.stl
- link /v1/RightPrimaryMedialPhalanx: geometry collision mesh filename=package://valkyrie/meshes/pf3.stl; visual mesh filename=package://valkyrie/meshes/pf3.stl
- link /v1/RightPrimaryMetacarpal: geometry collision mesh filename=package://valkyrie/meshes/pf1.stl; visual mesh filename=package://valkyrie/meshes/pf1.stl
- link /v1/RightPrimaryProximalPhalanx: geometry collision mesh filename=package://valkyrie/meshes/pf2.stl; visual mesh filename=package://valkyrie/meshes/pf2.stl
- link /v1/RightThumbDistalPhalanx: geometry collision mesh filename=package://valkyrie/meshes/tf4.stl; visual mesh filename=package://valkyrie/meshes/tf4.stl
- link /v1/RightThumbMedialPhalanx: geometry collision mesh filename=package://valkyrie/meshes/tf3.stl; visual mesh filename=package://valkyrie/meshes/tf3.stl
- link /v1/RightThumbMetacarpal: geometry collision mesh filename=package://valkyrie/meshes/tf1_Right.stl; visual mesh filename=package://valkyrie/meshes/tf1_Right.stl
- link /v1/RightThumbProximalPhalanx: geometry collision mesh filename=package://valkyrie/meshes/tf2.stl; visual mesh filename=package://valkyrie/meshes/tf2.stl
- link right_palm: geometry collision mesh filename=package://valkyrie/meshes/palm_Right.stl; visual mesh filename=package://valkyrie/meshes/palm_Right.stl
