Commit message: updating bdi hook xacro
git-svn-id: https://svn.csail.mit.edu/drc/trunk@7724 c7283977-0100-402a-a91a-fa70b306dbfe

File: ros_workspace/hook_description/src/bdihook_hand.urdf.xacro (robot description, xacro)
@@ -19,5 +19,5 @@
         <mesh filename="package://hook_description/meshes/bdi_hook.stl" scale="0.001 0.001 0.001"/>
       </geometry>
-      <origin rpy="0 0 ${hookflip*-1.571}" xyz="0.00 0.0 0.0"/>
+      <origin rpy="0 0 ${reflect*1.57+hookflip*1.57}" xyz="0.00 0.0 0.0"/>
     </collision>
     <visual>
@@ -25,5 +25,5 @@
         <mesh filename="package://hook_description/meshes/bdi_hook.stl" scale="0.001 0.001 0.001"/>
       </geometry>
-      <origin rpy="0 0 ${hookflip*-1.571}" xyz="0.00 0.0 0.0"/>
+      <origin rpy="0 0 ${reflect*1.57+hookflip*1.57}" xyz="0.00 0.0 0.0"/>
     </visual>
   </link>

Commit message: Fixed scaling of bdi_hook meshes. They're now in meters
git-svn-id: https://svn.csail.mit.edu/drc/trunk@7740 c7283977-0100-402a-a91a-fa70b306dbfe

File: ros_workspace/hook_description/src/bdihook_hand.urdf.xacro (robot description, xacro)
@@ -23,5 +23,5 @@
     <visual>
       <geometry>
-        <mesh filename="package://hook_description/meshes/bdi_hook.stl" scale="0.001 0.001 0.001"/>
+        <mesh filename="package://hook_description/meshes/bdi_hook.stl" scale="1 1 1"/>
       </geometry>
       <origin rpy="0 0 ${reflect*1.57+hookflip*1.57}" xyz="0.00 0.0 0.0"/>

Commit message: collision element had wrong scaling
git-svn-id: https://svn.csail.mit.edu/drc/trunk@7827 c7283977-0100-402a-a91a-fa70b306dbfe

File: ros_workspace/hook_description/src/bdihook_hand.urdf.xacro (robot description, xacro)
@@ -17,5 +17,5 @@
     <collision>
       <geometry>
-        <mesh filename="package://hook_description/meshes/bdi_hook.stl" scale="0.001 0.001 0.001"/>
+        <mesh filename="package://hook_description/meshes/bdi_hook.stl" scale="1 1 1"/>
       </geometry>
       <origin rpy="0 0 ${reflect*1.57+hookflip*1.57}" xyz="0.00 0.0 0.0"/>

Commit message: ability to add 30deg offsets to hook hands
git-svn-id: https://svn.csail.mit.edu/drc/trunk@7858 c7283977-0100-402a-a91a-fa70b306dbfe

File: ros_workspace/hook_description/src/bdihook_hand.urdf.xacro (robot description, xacro)
@@ -2,5 +2,5 @@
 <robot xmlns:xacro="http://www.ros.org/wiki/xacro" name="hook_hand">
 <xacro:property name="pi" value="3.14" />
-<xacro:macro name="hook_hand" params="side parent reflect hookflip *origin">
+<xacro:macro name="hook_hand" params="side parent reflect hookflip noof30degoffset *origin">
 <!-- joint to irobot hand -->
   <joint name="${side}_hook_hand_joint" type="fixed">
@@ -19,5 +19,5 @@
         <mesh filename="package://hook_description/meshes/bdi_hook.stl" scale="1 1 1"/>
       </geometry>
-      <origin rpy="0 0 ${reflect*1.57+hookflip*1.57}" xyz="0.00 0.0 0.0"/>
+      <origin rpy="0 0 ${reflect*(pi/2+noof30degoffset*(pi/6))+hookflip*(pi/2)}" xyz="0.00 0.0 0.0"/>
     </collision>
     <visual>
@@ -25,5 +25,5 @@
         <mesh filename="package://hook_description/meshes/bdi_hook.stl" scale="1 1 1"/>
       </geometry>
-      <origin rpy="0 0 ${reflect*1.57+hookflip*1.57}" xyz="0.00 0.0 0.0"/>
+      <origin rpy="0 0 ${reflect*(pi/2+noof30degoffset*(pi/6))+hookflip*(pi/2)}" xyz="0.00 0.0 0.0"/>
     </visual>
   </link>

File: ros_workspace/hook_description/src/hook_hand_simple.urdf.xacro (robot description, xacro)
@@ -7,5 +7,5 @@
 <!-- MIT changes (8th August 2013) -->
 <!-- ########################################### -->
-<xacro:macro name="hook_hand" params="side parent reflect hookflip *origin">
+<xacro:macro name="hook_hand" params="side parent reflect hookflip noof30degoffset *origin">
 <!--<xacro:flex_link side="${side}" finger_id="0" link_id="1"/>-->
 <!--<xacro:flex_link side="${side}" finger_id="0" link_id="2"/>-->
