Commit message: Updated hook urdf
git-svn-id: https://svn.csail.mit.edu/drc/trunk@7515 c7283977-0100-402a-a91a-fa70b306dbfe

File: ros_workspace/hook_description/src/hook_hand_simple.urdf.xacro (robot description, xacro)
@@ -80,5 +80,5 @@
         <cylinder length="0.01" radius="0.045"/>
       </geometry>
-      <origin rpy="0 0 0" xyz="0 0 0"/>
+      <origin rpy="0 0 0" xyz="0 0 0.025"/>
     </collision>
     <visual>
@@ -89,5 +89,5 @@
         <color rgba="0.2 0.2 0.2 1"/>
       </material>
-      <origin rpy="0 0 0" xyz="0 0 0.0"/>
+      <origin rpy="0 0 0" xyz="0 0 0.025"/>
     </visual>
 <!-- MIT's pointer rod -->
@@ -96,5 +96,5 @@
         <cylinder length="0.15" radius="0.006"/>
       </geometry>
-      <origin rpy="0 0 0" xyz="0 0 0.08"/>
+      <origin rpy="0 0 0" xyz="0 0 0.1"/>
     </collision>
     <visual>
@@ -105,12 +105,13 @@
         <color rgba="0.2 0.2 0.2 1"/>
       </material>
-      <origin rpy="0 0 0" xyz="0 0 0.08"/>
+      <origin rpy="0 0 0" xyz="0 0 0.1"/>
     </visual>
-<!-- MIT's pointer rod -->
+<!-- MIT's hook -->
+<!--
     <collision>
       <geometry>
         <cylinder length="0.04" radius="0.006"/>
       </geometry>
-      <origin rpy="0 1.571 1.571" xyz="0.00 -0.02 0.15"/>
+      <origin rpy="0 1.571 1.571" xyz="0.00 -0.02 0.16"/>
     </collision>
     <visual>
@@ -121,6 +122,7 @@
         <color rgba="0.2 0.2 0.2 1"/>
       </material>
-      <origin rpy="0 1.571 1.571" xyz="0.00 -0.02 0.15"/>
+      <origin rpy="0 1.571 1.571" xyz="0.00 -0.02 0.16"/>
     </visual>
+-->
   </link>
 </xacro:macro>

Commit message: minor corrections to get the orientation of the hook in the desired location
git-svn-id: https://svn.csail.mit.edu/drc/trunk@7674 c7283977-0100-402a-a91a-fa70b306dbfe

File: ros_workspace/hook_description/src/hook_hand_simple.urdf.xacro (robot description, xacro)
@@ -64,5 +64,5 @@
 <!-- ########################################### -->
 <!-- joint to irobot hand -->
-  <joint name="${side}_irobot_hand_joint" type="fixed">
+  <joint name="${side}_hook_hand_joint" type="fixed">
     <insert_block name="origin"/>
     <parent link="${parent}"/>
@@ -108,10 +108,9 @@
     </visual>
 <!-- MIT's hook -->
-<!--
     <collision>
       <geometry>
         <cylinder length="0.04" radius="0.006"/>
       </geometry>
-      <origin rpy="0 1.571 1.571" xyz="0.00 -0.02 0.16"/>
+      <origin rpy="0 1.571 1.571" xyz="0.00 0.02 0.16"/>
     </collision>
     <visual>
@@ -122,7 +121,6 @@
         <color rgba="0.2 0.2 0.2 1"/>
       </material>
-      <origin rpy="0 1.571 1.571" xyz="0.00 -0.02 0.16"/>
+      <origin rpy="0 1.571 1.571" xyz="0.00 0.02 0.16"/>
     </visual>
--->
   </link>
 </xacro:macro>

Commit message: adding bdi hook hands
git-svn-id: https://svn.csail.mit.edu/drc/trunk@7719 c7283977-0100-402a-a91a-fa70b306dbfe

File: ros_workspace/hook_description/src/hook_hand_simple.urdf.xacro (robot description, xacro)
@@ -7,5 +7,5 @@
 <!-- MIT changes (8th August 2013) -->
 <!-- ########################################### -->
-<xacro:macro name="hook_hand" params="side parent reflect *origin">
+<xacro:macro name="hook_hand" params="side parent reflect hookflip *origin">
 <!--<xacro:flex_link side="${side}" finger_id="0" link_id="1"/>-->
 <!--<xacro:flex_link side="${side}" finger_id="0" link_id="2"/>-->
@@ -112,5 +112,5 @@
         <cylinder length="0.04" radius="0.006"/>
       </geometry>
-      <origin rpy="0 1.571 1.571" xyz="0.00 0.02 0.16"/>
+      <origin rpy="0 1.571 1.571" xyz="0.00 ${-0.02 * reflect} 0.16"/>
     </collision>
     <visual>
@@ -121,5 +121,5 @@
         <color rgba="0.2 0.2 0.2 1"/>
       </material>
-      <origin rpy="0 1.571 1.571" xyz="0.00 0.02 0.16"/>
+      <origin rpy="0 1.571 1.571" xyz="0.00 ${-0.02 * reflect} 0.16"/>
     </visual>
   </link>

Commit message: fliped the hook
git-svn-id: https://svn.csail.mit.edu/drc/trunk@8012 c7283977-0100-402a-a91a-fa70b306dbfe

File: ros_workspace/hook_description/src/hook_hand_simple.urdf.xacro (robot description, xacro)
@@ -110,16 +110,16 @@
     <collision>
       <geometry>
-        <cylinder length="0.04" radius="0.006"/>
+        <cylinder length="0.044" radius="0.006"/>
       </geometry>
-      <origin rpy="0 1.571 1.571" xyz="0.00 ${-0.02 * reflect} 0.16"/>
+      <origin rpy="0 1.571 1.571" xyz="0.00 ${0.018 * reflect} 0.16"/>
     </collision>
     <visual>
       <geometry>
-        <cylinder length="0.04" radius="0.006"/>
+        <cylinder length="0.044" radius="0.006"/>
       </geometry>
       <material name="darkgray">
         <color rgba="0.2 0.2 0.2 1"/>
       </material>
-      <origin rpy="0 1.571 1.571" xyz="0.00 ${-0.02 * reflect} 0.16"/>
+      <origin rpy="0 1.571 1.571" xyz="0.00 ${0.018 * reflect} 0.16"/>
     </visual>
   </link>

Commit message: final refinements to pointers all looks finishes
git-svn-id: https://svn.csail.mit.edu/drc/trunk@8025 c7283977-0100-402a-a91a-fa70b306dbfe

File: ros_workspace/hook_description/src/hook_hand_simple.urdf.xacro (robot description, xacro)
@@ -94,5 +94,5 @@
     <collision>
       <geometry>
-        <cylinder length="0.15" radius="0.006"/>
+        <cylinder length="0.16" radius="0.006"/>
       </geometry>
       <origin rpy="0 0 0" xyz="0 0 0.1"/>
@@ -100,5 +100,5 @@
     <visual>
       <geometry>
-        <cylinder length="0.15" radius="0.006"/>
+        <cylinder length="0.16" radius="0.006"/>
       </geometry>
       <material name="darkgray">
@@ -112,5 +112,5 @@
         <cylinder length="0.044" radius="0.006"/>
       </geometry>
-      <origin rpy="0 1.571 1.571" xyz="0.00 ${0.018 * reflect} 0.16"/>
+      <origin rpy="0 1.571 1.571" xyz="0.00 ${0.018 * reflect} 0.185"/>
     </collision>
     <visual>
@@ -121,5 +121,5 @@
         <color rgba="0.2 0.2 0.2 1"/>
       </material>
-      <origin rpy="0 1.571 1.571" xyz="0.00 ${0.018 * reflect} 0.16"/>
+      <origin rpy="0 1.571 1.571" xyz="0.00 ${0.018 * reflect} 0.185"/>
     </visual>
   </link>

File: software/models/mit_gazebo_models/mit_robot/model_LP_RP.urdf (robot description, URDF)
Before this commit: robot atlas, 58 links, 57 joints
Links:
- link left_base_link: geometry collision cylinder length=0.01 radius=0.045; collision cylinder length=0.044 radius=0.006
- link right_base_link: geometry collision cylinder length=0.01 radius=0.045; collision cylinder length=0.044 radius=0.006

File: software/models/mit_gazebo_models/mit_robot/model_LP_RR.urdf (robot description, URDF)
Before this commit: robot atlas, 70 links, 69 joints
Links:
- link left_base_link: geometry collision cylinder length=0.01 radius=0.045; collision cylinder length=0.044 radius=0.006

File: software/models/mit_gazebo_models/mit_robot/model_LQ_RP.urdf (robot description, URDF)
Before this commit: robot atlas, 71 links, 70 joints
Links:
- link right_base_link: geometry collision cylinder length=0.01 radius=0.045; collision cylinder length=0.044 radius=0.006

File: software/models/mit_gazebo_models/mit_robot_hands/inert_hand_left.urdf (robot description, URDF)
Before this commit: robot inert_hand_left, 2 links, 1 joints
Links:
- link left_base_link: geometry collision cylinder length=0.01 radius=0.045; collision cylinder length=0.044 radius=0.006

File: software/models/mit_gazebo_models/mit_robot_hands/inert_hand_right.urdf (robot description, URDF)
Before this commit: robot inert_hand_right, 2 links, 1 joints
Links:
- link right_base_link: geometry collision cylinder length=0.01 radius=0.045; collision cylinder length=0.044 radius=0.006

File: software/models/mit_gazebo_models/mit_robot_hands/xacro/inert_hand_left.urdf.xacro (robot description, xacro)
@@ -11,6 +11,6 @@
     </inertial>
   </link>
- <xacro:include filename="$(find hook_description)/src/bdihook_hand.urdf.xacro" />
-<!--  <xacro:include filename="$(find hook_description)/src/hook_hand_simple.urdf.xacro" /> -->
+<!-- <xacro:include filename="$(find hook_description)/src/bdihook_hand.urdf.xacro" />  -->
+ <xacro:include filename="$(find hook_description)/src/hook_hand_simple.urdf.xacro" />
   <xacro:hook_hand side="left" parent="plane::xy::base" reflect="-1" hookflip="-1" noof30degoffset="0">
     <origin rpy="1.57 0.0 -1.57" xyz="0.243 0.0 -0.127"/>

File: software/models/mit_gazebo_models/mit_robot_hands/xacro/inert_hand_right.urdf.xacro (robot description, xacro)
@@ -11,6 +11,6 @@
     </inertial>
   </link>
-  <xacro:include filename="$(find hook_description)/src/bdihook_hand.urdf.xacro" />
-<!--  <xacro:include filename="$(find hook_description)/src/hook_hand_simple.urdf.xacro" />  -->
+<!--  <xacro:include filename="$(find hook_description)/src/bdihook_hand.urdf.xacro" />  -->
+  <xacro:include filename="$(find hook_description)/src/hook_hand_simple.urdf.xacro" />
    <xacro:hook_hand side="right" parent="plane::xy::base" reflect="1" hookflip="-1" noof30degoffset="0">
      <origin rpy="1.57 3.14 -1.57" xyz="0.243 0.0 -0.127"/>

Commit message: revising the pointer urdf to match new conventions

File: ros_workspace/hook_description/src/hook_hand_simple.urdf.xacro (robot description, xacro)
@@ -7,5 +7,5 @@
 <!-- MIT changes (8th August 2013) -->
 <!-- ########################################### -->
-<xacro:macro name="hook_hand" params="side parent reflect hookflip noof30degoffset *origin">
+<xacro:macro name="hook_hand" params="side parent *origin">
 <!--<xacro:flex_link side="${side}" finger_id="0" link_id="1"/>-->
 <!--<xacro:flex_link side="${side}" finger_id="0" link_id="2"/>-->
@@ -80,5 +80,5 @@
         <cylinder length="0.01" radius="0.045"/>
       </geometry>
-      <origin rpy="0 0 0" xyz="0 0 0.025"/>
+      <origin rpy="0 0 0" xyz="0 0 0.005"/>
     </collision>
     <visual>
@@ -89,5 +89,5 @@
         <color rgba="0.2 0.2 0.2 1"/>
       </material>
-      <origin rpy="0 0 0" xyz="0 0 0.025"/>
+      <origin rpy="0 0 0" xyz="0 0 0.005"/>
     </visual>
 <!-- MIT's pointer rod -->
@@ -96,5 +96,5 @@
         <cylinder length="0.16" radius="0.006"/>
       </geometry>
-      <origin rpy="0 0 0" xyz="0 0 0.1"/>
+      <origin rpy="0 0 0" xyz="0 0 0.08"/>
     </collision>
     <visual>
@@ -105,12 +105,13 @@
         <color rgba="0.2 0.2 0.2 1"/>
       </material>
-      <origin rpy="0 0 0" xyz="0 0 0.1"/>
+      <origin rpy="0 0 0" xyz="0 0 0.08"/>
     </visual>
-<!-- MIT's hook -->
+<!-- MIT's hook tip -->
+<!--
     <collision>
       <geometry>
         <cylinder length="0.044" radius="0.006"/>
       </geometry>
-      <origin rpy="0 1.571 1.571" xyz="0.00 ${0.018 * reflect} 0.185"/>
+      <origin rpy="0 1.571 1.571" xyz="0.00 0.018 0.16"/>
     </collision>
     <visual>
@@ -121,7 +122,31 @@
         <color rgba="0.2 0.2 0.2 1"/>
       </material>
-      <origin rpy="0 1.571 1.571" xyz="0.00 ${0.018 * reflect} 0.185"/>
+      <origin rpy="0 1.571 1.571" xyz="0.00 0.018 0.16"/>
+    </visual>
+-->
+<!-- optional off center nub at base (to illustrate rotation) -->
+    <collision>
+      <geometry>
+        <cylinder length="0.044" radius="0.006"/>
+      </geometry>
+      <origin rpy="0 1.571 1.571" xyz="0.00 0.018 0.02"/>
+    </collision>
+    <visual>
+      <geometry>
+        <cylinder length="0.044" radius="0.006"/>
+      </geometry>
+      <material name="darkgray">
+        <color rgba="0.2 0.2 0.2 1"/>
+      </material>
+      <origin rpy="0 1.571 1.571" xyz="0.00 0.018 0.02"/>
     </visual>
   </link>
+<!-- Contact Point near the tip of the pointer -->
+  <joint name="${side}_pointer_tip_joint" type="fixed">
+    <origin rpy="0.0 0.0 0.0" xyz="0 0.12 0"/>
+    <parent link="${parent}"/>
+    <child link="${side}_pointer_tip"/>
+  </joint>
+  <link name="${side}_pointer_tip"/>
 </xacro:macro>
 </robot>

File: software/models/mit_gazebo_models/mit_robot/model_LP_RP.urdf (robot description, URDF)
Before this commit: robot atlas, 60 links, 59 joints
Links:
- added link left_pointer_tip
- added link right_pointer_tip
Joints:
- added joint left_pointer_tip_joint: type fixed, parent l_hand_force_torque, child left_pointer_tip, origin xyz=0 0.12 0 rpy=0.0 0.0 0.0
- added joint right_pointer_tip_joint: type fixed, parent r_hand_force_torque, child right_pointer_tip, origin xyz=0 0.12 0 rpy=0.0 0.0 0.0
- joint left_hook_hand_joint: origin xyz=0 0.11516 0.015 rpy=1.57079 3.14159 3.14159 -> xyz=0 0.0 0.0 rpy=1.57079 3.14159 3.14159; parent l_hand -> l_hand_force_torque
- joint right_hook_hand_joint: origin xyz=0 -0.11516 -0.015 rpy=1.57079 0 0 -> xyz=0 0.0 0.0 rpy=1.57079 3.14159 3.14159; parent r_hand -> r_hand_force_torque

File: software/models/mit_gazebo_models/mit_robot/xacro/atlas_LP_RP.urdf.xacro (robot description, xacro)
@@ -5,9 +5,9 @@
   <xacro:include filename="$(find mit_drcsim_scripts)/models/mit_robot/xacro/hand_force_torque.urdf" />
   <xacro:include filename="$(find hook_description)/src/hook_hand_simple.urdf.xacro" />
-  <xacro:hook_hand side="right" parent="r_hand" reflect="1" hookflip="-1" noof30degoffset="0">
-    <origin rpy="1.57079 0 0" xyz="0 -0.11516 -0.015"/>
+  <xacro:hook_hand side="left" parent="l_hand_force_torque">
+    <origin rpy="1.57079 3.14159 3.14159" xyz="0 0.0 0.0"/>
   </xacro:hook_hand>
-  <xacro:hook_hand side="left" parent="l_hand" reflect="-1" hookflip="-1" noof30degoffset="0">
-    <origin rpy="1.57079 3.14159 3.14159" xyz="0 0.11516 0.015"/>
+  <xacro:hook_hand side="right" parent="r_hand_force_torque">
+    <origin rpy="1.57079 3.14159 3.14159" xyz="0 0.0 0.0"/>
   </xacro:hook_hand>
 </robot>

Commit message: adding a pointer end to the models

File: ros_workspace/hook_description/src/hook_hand_simple.urdf.xacro (robot description, xacro)
@@ -149,4 +149,11 @@
   </joint>
   <link name="${side}_pointer_tip"/>
+<!-- Contact Point AT the tip of the pointer. these were poorly named -->
+  <joint name="${side}_pointer_end_joint" type="fixed">
+    <origin rpy="0.0 0.0 0.0" xyz="0 0.16 0"/>
+    <parent link="${parent}"/>
+    <child link="${side}_pointer_end"/>
+  </joint>
+  <link name="${side}_pointer_end"/>
 </xacro:macro>
 </robot>

File: software/models/mit_gazebo_models/mit_robot/model_LP_RP.urdf (robot description, URDF)
Before this commit: robot atlas, 62 links, 61 joints
Links:
- added link left_pointer_end
- added link right_pointer_end
Joints:
- added joint left_pointer_end_joint: type fixed, parent l_hand_force_torque, child left_pointer_end, origin xyz=0 0.16 0 rpy=0.0 0.0 0.0
- added joint right_pointer_end_joint: type fixed, parent r_hand_force_torque, child right_pointer_end, origin xyz=0 0.16 0 rpy=0.0 0.0 0.0

File: software/models/mit_gazebo_models/mit_robot/model_LP_RR.urdf (robot description, URDF)
Before this commit: robot atlas, 77 links, 76 joints
Links:
- added link left_pointer_end
Joints:
- added joint left_pointer_end_joint: type fixed, parent l_hand_force_torque, child left_pointer_end, origin xyz=0 0.16 0 rpy=0.0 0.0 0.0

File: software/models/mit_gazebo_models/mit_robot/model_LR_RP.urdf (robot description, URDF)
Before this commit: robot atlas, 77 links, 76 joints
Links:
- added link right_pointer_end
Joints:
- added joint right_pointer_end_joint: type fixed, parent r_hand_force_torque, child right_pointer_end, origin xyz=0 0.16 0 rpy=0.0 0.0 0.0

File: software/models/mit_gazebo_models/mit_robot_hands/pointer_hand_left.urdf (robot description, URDF)
Before this commit: robot pointer_hand_left, 3 links, 2 joints
Links:
- added link left_pointer_end
Joints:
- added joint left_pointer_end_joint: type fixed, parent plane::xy::base, child left_pointer_end, origin xyz=0 0.16 0 rpy=0.0 0.0 0.0

File: software/models/mit_gazebo_models/mit_robot_hands/pointer_hand_right.urdf (robot description, URDF)
Before this commit: robot pointer_hand_right, 3 links, 2 joints
Links:
- added link right_pointer_end
Joints:
- added joint right_pointer_end_joint: type fixed, parent plane::xy::base, child right_pointer_end, origin xyz=0 0.16 0 rpy=0.0 0.0 0.0
