Commit message: made robotiq hand camera xacro reflective. added force torque frame
made robotiq and hand camera relative to FT frame for easy use
removed reference to palm and sandia camera in viewer
added hand_face and hand_gripper

File: ros_workspace/robotiq-hand/robotiq_hand_description/cfg/robotiq_hand.urdf.xacro (robot description, xacro)
@@ -1,5 +1,5 @@
 <?xml version="1.0"?>
 <robot xmlns:xacro="http://www.ros.org/wiki/xacro" name="robotiq_hand">
-<xacro:property name="pi" value="3.14" />
+<xacro:property name="pi" value="3.1416" />
 <!-- ########################################### -->
 <!-- Custom MIT XACRO For Robotiq Hand -->

File: ros_workspace/robotiq_camera/urdf/robotiq_camera.urdf.xacro (robot description, xacro)
@@ -1,6 +1,11 @@
 <?xml version="1.0" ?>
 <robot name="robotiq_camera" xmlns:xacro="http://www.ros.org/wiki/xacro">
-  <xacro:macro name="robotiq_camera" params="side parent *origin">
-  <link name="${side}_hand_camera_link">
+  <xacro:macro name="robotiq_camera" params="side_letter reflect parent *origin">
+  <joint name="${side_letter}_hand_face_joint" type="fixed">
+    <origin rpy="0.0 0.0 0.0" xyz="0 0.12 0"/>
+    <parent link="${parent}"/>
+    <child link="${side_letter}_hand_face"/>
+  </joint>
+  <link name="${side_letter}_hand_face">
     <inertial>
       <mass value="0.1"/>
@@ -15,19 +20,51 @@
     </visual>
   </link>
-  <joint name="${side}_hand_camera_joint" type="fixed">
+  <joint name="${side_letter}_hand_gripper_joint" type="fixed">
+    <origin rpy="0.0 0.0 0.0" xyz="0 0.18 0"/>
     <parent link="${parent}"/>
-    <child link="${side}_hand_camera_link"/>
-    <insert_block name="origin" />
+    <child link="${side_letter}_hand_gripper"/>
   </joint>
-  <joint name="${side}_hand_camera_optical_frame_joint" type="fixed">
+  <link name="${side_letter}_hand_gripper">
+    <inertial>
+      <mass value="0.1"/>
+      <origin xyz="0 0 0"/>
+      <inertia ixx="0.00001" ixy="0" ixz="0" iyy="0.00001" iyz="0" izz="0.00001"/>
+    </inertial>
+    <visual>
+      <origin rpy="0 0 0" xyz="0 0 0"/>
+      <geometry>
+        <box size="0.01 0.01 0.01"/>
+      </geometry>
+    </visual>
+  </link>
+  <link name="${side_letter}_hand_camera_link">
+    <inertial>
+      <mass value="0.1"/>
+      <origin xyz="0 0 0"/>
+      <inertia ixx="0.00001" ixy="0" ixz="0" iyy="0.00001" iyz="0" izz="0.00001"/>
+    </inertial>
+    <visual>
+      <origin rpy="0 0 0" xyz="0 0 0"/>
+      <geometry>
+        <box size="0.01 0.01 0.01"/>
+      </geometry>
+    </visual>
+  </link>
+  <joint name="${side_letter}_hand_camera_joint" type="fixed">
+    <parent link="${parent}"/>
+    <child link="${side_letter}_hand_camera_link"/>
+    <!-- 9 degree inward angle-->
+    <origin xyz="${-0.09*reflect}  0.12 0.0" rpy="-1.57079 0  ${1.5708-reflect*0.15708}"/>
+  </joint>
+  <joint name="${side_letter}_hand_camera_optical_frame_joint" type="fixed">
     <origin rpy="-1.5708 0.0 -1.5708" xyz="0 0 0"/>
-    <parent link="${side}_hand_camera_link"/>
-    <child link="${side}_hand_camera_optical_frame"/>
+    <parent link="${side_letter}_hand_camera_link"/>
+    <child link="${side_letter}_hand_camera_optical_frame"/>
   </joint>
-  <link name="${side}_hand_camera_optical_frame"/>
-  <gazebo reference="${side}_hand_camera_link">
-    <sensor name="${side}_hand_camera_sensor" type="camera">
+  <link name="${side_letter}_hand_camera_optical_frame"/>
+  <gazebo reference="${side_letter}_hand_camera_link">
+    <sensor name="${side_letter}_hand_camera_sensor" type="camera">
       <update_rate>10.0</update_rate>
-      <camera name="${side}_hand_camera">
+      <camera name="${side_letter}_hand_camera">
         <pose>0 0 0 0 0 0</pose>
         <!-- m.antone estimate of 2.8mm tamron lense fov -->
@@ -54,11 +91,11 @@
         </noise>
       </camera>
-      <plugin filename="libgazebo_ros_camera.so" name="${side}_hand_camera_controller">
+      <plugin filename="libgazebo_ros_camera.so" name="${side_letter}_hand_camera_controller">
         <alwaysOn>true</alwaysOn>
         <updateRate>0.0</updateRate>
-        <cameraName>robotiq_hands/${side}_hand_camera</cameraName>
+        <cameraName>robotiq_hands/${side_letter}_hand_camera</cameraName>
         <imageTopicName>image_raw</imageTopicName>
         <cameraInfoTopicName>camera_info</cameraInfoTopicName>
-        <frameName>${side}_hand_camera_optical_frame</frameName>
+        <frameName>${side_letter}_hand_camera_optical_frame</frameName>
         <hackBaseline>0.07</hackBaseline>
         <distortionK1>0.0</distortionK1>

File: software/models/mit_gazebo_models/mit_robot/model_LH_RH.urdf (robot description, URDF)
Before this commit: robot atlas, 58 links, 57 joints
Links:
- added link l_hand_force_torque, mass 0.1; visual box size=0.01 0.01 0.01
- added link r_hand_force_torque, mass 0.1; visual box size=0.01 0.01 0.01
Joints:
- added joint l_hand_force_torque_joint: type fixed, parent l_hand, child l_hand_force_torque, origin xyz=0 0.1245 0.0112 rpy=0 0 0
- added joint r_hand_force_torque_joint: type fixed, parent r_hand, child r_hand_force_torque, origin xyz=0 -0.1245 0.0112 rpy=0 0 3.142

File: software/models/mit_gazebo_models/mit_robot/model_LI_RI.urdf (robot description, URDF)
Before this commit: robot atlas, 74 links, 73 joints
Links:
- added link l_hand_force_torque, mass 0.1; visual box size=0.01 0.01 0.01
- added link r_hand_force_torque, mass 0.1; visual box size=0.01 0.01 0.01
Joints:
- added joint l_hand_force_torque_joint: type fixed, parent l_hand, child l_hand_force_torque, origin xyz=0 0.1245 0.0112 rpy=0 0 0
- added joint r_hand_force_torque_joint: type fixed, parent r_hand, child r_hand_force_torque, origin xyz=0 -0.1245 0.0112 rpy=0 0 3.142

File: software/models/mit_gazebo_models/mit_robot/model_LI_RR.urdf (robot description, URDF)
Before this commit: robot atlas, 78 links, 77 joints
Links:
- added link l_hand_force_torque, mass 0.1; visual box size=0.01 0.01 0.01
- added link r_hand_force_torque, mass 0.1; visual box size=0.01 0.01 0.01
Joints:
- added joint l_hand_force_torque_joint: type fixed, parent l_hand, child l_hand_force_torque, origin xyz=0 0.1245 0.0112 rpy=0 0 0
- added joint r_hand_force_torque_joint: type fixed, parent r_hand, child r_hand_force_torque, origin xyz=0 -0.1245 0.0112 rpy=0 0 3.142
- joint left_finger[0]/joint_base: limit lower=0.0 upper=1.57 effort=1000.0 velocity=0.5 -> lower=0.0 upper=1.5708 effort=1000.0 velocity=0.5; origin xyz=0 0 0.0135 rpy=1.57 0 -3.14 -> xyz=0 0 0.0135 rpy=1.5708 0 -3.1416
- joint left_finger[0]/joint_base_rotation: limit lower=0.0 upper=1.57 effort=1000.0 velocity=0.5 -> lower=0.0 upper=1.5708 effort=1000.0 velocity=0.5
- joint left_finger[0]/joint_flex: limit lower=0.0 upper=1.57 effort=1000.0 velocity=0.5 -> lower=0.0 upper=1.5708 effort=1000.0 velocity=0.5
- joint left_finger[1]/joint_base: limit lower=0.0 upper=1.57 effort=1000.0 velocity=0.5 -> lower=0.0 upper=1.5708 effort=1000.0 velocity=0.5; origin xyz=0 0 0.0135 rpy=1.57 0 -3.14 -> xyz=0 0 0.0135 rpy=1.5708 0 -3.1416
- joint left_finger[1]/joint_base_rotation: limit lower=0.0 upper=1.57 effort=1000.0 velocity=0.5 -> lower=0.0 upper=1.5708 effort=1000.0 velocity=0.5
- joint left_finger[1]/joint_flex: limit lower=0.0 upper=1.57 effort=1000.0 velocity=0.5 -> lower=0.0 upper=1.5708 effort=1000.0 velocity=0.5
- joint left_finger[2]/joint_base: limit lower=0.0 upper=1.57 effort=1000.0 velocity=0.5 -> lower=0.0 upper=1.5708 effort=1000.0 velocity=0.5; origin xyz=0 -0.038 0.082755 rpy=1.57 0 0 -> xyz=0 -0.038 0.082755 rpy=1.5708 0 0
- joint left_finger[2]/joint_flex: limit lower=0.0 upper=1.57 effort=1000.0 velocity=0.5 -> lower=0.0 upper=1.5708 effort=1000.0 velocity=0.5

File: software/models/mit_gazebo_models/mit_robot/model_LI_RR_extender.urdf (robot description, URDF)
Before this commit: robot atlas, 80 links, 79 joints
Links:
- added link l_hand_force_torque, mass 0.1; visual box size=0.01 0.01 0.01
- added link r_hand_force_torque, mass 0.1; visual box size=0.01 0.01 0.01
Joints:
- added joint l_hand_force_torque_joint: type fixed, parent l_hand, child l_hand_force_torque, origin xyz=0 0.1245 0.0112 rpy=0 0 0
- added joint r_hand_force_torque_joint: type fixed, parent r_hand, child r_hand_force_torque, origin xyz=0 -0.1245 0.0112 rpy=0 0 3.142
- joint left_finger[0]/joint_base: limit lower=0.0 upper=1.57 effort=1000.0 velocity=0.5 -> lower=0.0 upper=1.5708 effort=1000.0 velocity=0.5; origin xyz=0 0 0.0135 rpy=1.57 0 -3.14 -> xyz=0 0 0.0135 rpy=1.5708 0 -3.1416
- joint left_finger[0]/joint_base_rotation: limit lower=0.0 upper=1.57 effort=1000.0 velocity=0.5 -> lower=0.0 upper=1.5708 effort=1000.0 velocity=0.5
- joint left_finger[0]/joint_flex: limit lower=0.0 upper=1.57 effort=1000.0 velocity=0.5 -> lower=0.0 upper=1.5708 effort=1000.0 velocity=0.5
- joint left_finger[1]/joint_base: limit lower=0.0 upper=1.57 effort=1000.0 velocity=0.5 -> lower=0.0 upper=1.5708 effort=1000.0 velocity=0.5; origin xyz=0 0 0.0135 rpy=1.57 0 -3.14 -> xyz=0 0 0.0135 rpy=1.5708 0 -3.1416
- joint left_finger[1]/joint_base_rotation: limit lower=0.0 upper=1.57 effort=1000.0 velocity=0.5 -> lower=0.0 upper=1.5708 effort=1000.0 velocity=0.5
- joint left_finger[1]/joint_flex: limit lower=0.0 upper=1.57 effort=1000.0 velocity=0.5 -> lower=0.0 upper=1.5708 effort=1000.0 velocity=0.5
- joint left_finger[2]/joint_base: limit lower=0.0 upper=1.57 effort=1000.0 velocity=0.5 -> lower=0.0 upper=1.5708 effort=1000.0 velocity=0.5; origin xyz=0 -0.038 0.082755 rpy=1.57 0 0 -> xyz=0 -0.038 0.082755 rpy=1.5708 0 0
- joint left_finger[2]/joint_flex: limit lower=0.0 upper=1.57 effort=1000.0 velocity=0.5 -> lower=0.0 upper=1.5708 effort=1000.0 velocity=0.5

File: software/models/mit_gazebo_models/mit_robot/model_LP_RP.urdf (robot description, URDF)
Before this commit: robot atlas, 58 links, 57 joints
Links:
- added link l_hand_force_torque, mass 0.1; visual box size=0.01 0.01 0.01
- added link r_hand_force_torque, mass 0.1; visual box size=0.01 0.01 0.01
Joints:
- added joint l_hand_force_torque_joint: type fixed, parent l_hand, child l_hand_force_torque, origin xyz=0 0.1245 0.0112 rpy=0 0 0
- added joint r_hand_force_torque_joint: type fixed, parent r_hand, child r_hand_force_torque, origin xyz=0 -0.1245 0.0112 rpy=0 0 3.142

File: software/models/mit_gazebo_models/mit_robot/model_LP_RR.urdf (robot description, URDF)
Before this commit: robot atlas, 70 links, 69 joints
Links:
- added link l_hand_force_torque, mass 0.1; visual box size=0.01 0.01 0.01
- added link r_hand_force_torque, mass 0.1; visual box size=0.01 0.01 0.01
Joints:
- added joint l_hand_force_torque_joint: type fixed, parent l_hand, child l_hand_force_torque, origin xyz=0 0.1245 0.0112 rpy=0 0 0
- added joint r_hand_force_torque_joint: type fixed, parent r_hand, child r_hand_force_torque, origin xyz=0 -0.1245 0.0112 rpy=0 0 3.142

File: software/models/mit_gazebo_models/mit_robot/model_LQ_RP.urdf (robot description, URDF)
Before this commit: robot atlas, 71 links, 70 joints
Links:
- added link l_hand_force_torque, mass 0.1; visual box size=0.01 0.01 0.01
- added link r_hand_force_torque, mass 0.1; visual box size=0.01 0.01 0.01
Joints:
- added joint l_hand_force_torque_joint: type fixed, parent l_hand, child l_hand_force_torque, origin xyz=0 0.1245 0.0112 rpy=0 0 0
- added joint r_hand_force_torque_joint: type fixed, parent r_hand, child r_hand_force_torque, origin xyz=0 -0.1245 0.0112 rpy=0 0 3.142

File: software/models/mit_gazebo_models/mit_robot/model_LR_RR.urdf (robot description, URDF)
Before this commit: robot atlas, 86 links, 85 joints
Links:
- removed link left_hand_camera_link
- removed link left_hand_camera_optical_frame
- removed link post_spindle
- removed link post_spindle_cal_pitch
- removed link post_spindle_cal_roll
- removed link post_spindle_cal_x
- removed link post_spindle_cal_y
- removed link post_spindle_cal_z
- removed link pre_spindle
- removed link pre_spindle_cal_pitch
- removed link pre_spindle_cal_roll
- removed link pre_spindle_cal_x
- removed link pre_spindle_cal_y
- removed link pre_spindle_cal_yaw
- removed link pre_spindle_cal_z
- removed link right_hand_camera_link
- removed link right_hand_camera_optical_frame
- added link head_imu_link, mass 1e-5; visual box size=0.01 0.01 0.01
- added link l_hand_camera_link, mass 0.1; visual box size=0.01 0.01 0.01
- added link l_hand_camera_optical_frame
- added link l_hand_face, mass 0.1; visual box size=0.01 0.01 0.01
- added link l_hand_force_torque, mass 0.1; visual box size=0.01 0.01 0.01
- added link l_hand_gripper, mass 0.1; visual box size=0.01 0.01 0.01
- added link r_hand_camera_link, mass 0.1; visual box size=0.01 0.01 0.01
- added link r_hand_camera_optical_frame
- added link r_hand_face, mass 0.1; visual box size=0.01 0.01 0.01
- added link r_hand_force_torque, mass 0.1; visual box size=0.01 0.01 0.01
- added link r_hand_gripper, mass 0.1; visual box size=0.01 0.01 0.01
- link center_bottom_led_frame: mass 0.1 -> 1e-5
- link center_top_led_frame: mass 0.1 -> 1e-5
- link head: mass 1.4199 -> 1.41984; geometry collision box size=0.0468 0.12 0.1184; collision box size=0.1311 0.12 0.0591
- link head_hokuyo_frame: mass 0.01 -> 1e-5
- link hokuyo_link: mass 0.057664 -> 0.057654; geometry collision box size=0.08 0.06 0.04238; collision cylinder length=0.047 radius=0.024425
- link left_camera_frame: mass 0.1 -> 1e-5
- link left_led_frame: mass 0.1 -> 1e-5
- link right_camera_frame: mass 0.1 -> 1e-5
- link right_led_frame: mass 0.1 -> 1e-5
Joints:
- removed joint left_hand_camera_joint
- removed joint left_hand_camera_optical_frame_joint
- removed joint post_spindle_cal_pitch_joint
- removed joint post_spindle_cal_roll_joint
- removed joint post_spindle_cal_x_joint
- removed joint post_spindle_cal_y_joint
- removed joint post_spindle_cal_yaw_joint
- removed joint post_spindle_cal_z_joint
- removed joint pre_spindle_cal_pitch_joint
- removed joint pre_spindle_cal_roll_joint
- removed joint pre_spindle_cal_x_joint
- removed joint pre_spindle_cal_y_joint
- removed joint pre_spindle_cal_yaw_joint
- removed joint pre_spindle_cal_z_joint
- removed joint pre_spindle_joint
- removed joint right_hand_camera_joint
- removed joint right_hand_camera_optical_frame_joint
- added joint head_imu_joint: type fixed, parent head, child head_imu_link, origin xyz=-0.0475 0.035 0.0 rpy=0 0 0
- added joint l_hand_camera_joint: type fixed, parent l_hand_force_torque, child l_hand_camera_link, origin xyz=-0.09  0.12 0.0 rpy=-1.57079 0  1.41372
- added joint l_hand_camera_optical_frame_joint: type fixed, parent l_hand_camera_link, child l_hand_camera_optical_frame, origin xyz=0 0 0 rpy=-1.5708 0.0 -1.5708
- added joint l_hand_face_joint: type fixed, parent l_hand_force_torque, child l_hand_face, origin xyz=0 0.12 0 rpy=0.0 0.0 0.0
- added joint l_hand_force_torque_joint: type fixed, parent l_hand, child l_hand_force_torque, origin xyz=0 0.1245 0.0112 rpy=0 0 0
- added joint l_hand_gripper_joint: type fixed, parent l_hand_force_torque, child l_hand_gripper, origin xyz=0 0.18 0 rpy=0.0 0.0 0.0
- added joint r_hand_camera_joint: type fixed, parent r_hand_force_torque, child r_hand_camera_link, origin xyz=0.09  0.12 0.0 rpy=-1.57079 0  1.72788
- added joint r_hand_camera_optical_frame_joint: type fixed, parent r_hand_camera_link, child r_hand_camera_optical_frame, origin xyz=0 0 0 rpy=-1.5708 0.0 -1.5708
- added joint r_hand_face_joint: type fixed, parent r_hand_force_torque, child r_hand_face, origin xyz=0 0.12 0 rpy=0.0 0.0 0.0
- added joint r_hand_force_torque_joint: type fixed, parent r_hand, child r_hand_force_torque, origin xyz=0 -0.1245 0.0112 rpy=0 0 3.142
- added joint r_hand_gripper_joint: type fixed, parent r_hand_force_torque, child r_hand_gripper, origin xyz=0 0.18 0 rpy=0.0 0.0 0.0
- joint hokuyo_joint: child post_spindle -> hokuyo_link; origin xyz=0 0 0 rpy=0 0 0 -> xyz=-0.0446 0 0.0880 rpy=0 0 0; parent pre_spindle_cal_yaw -> head
- joint left_robotiq_hand_joint: origin xyz=0 0.19016 0.015 rpy=0 -1.57079 0 -> xyz=0 0.06566 0.0 rpy=0 -1.57079 0; parent l_hand -> l_hand_force_torque
- joint right_robotiq_hand_joint: origin xyz=0 -0.19016 -0.015 rpy=0 -1.57079 3.141 -> xyz=0 0.06566 0.0 rpy=0 -1.57079 0; parent r_hand -> r_hand_force_torque

File: software/models/mit_gazebo_models/mit_robot/model_sim.urdf (robot description, URDF)
Before this commit: robot atlas, 111 links, 110 joints
Links:
- added link l_hand_force_torque, mass 0.1; visual box size=0.01 0.01 0.01
- added link r_hand_force_torque, mass 0.1; visual box size=0.01 0.01 0.01
Joints:
- added joint l_hand_force_torque_joint: type fixed, parent l_hand, child l_hand_force_torque, origin xyz=0 0.1245 0.0112 rpy=0 0 0
- added joint r_hand_force_torque_joint: type fixed, parent r_hand, child r_hand_force_torque, origin xyz=0 -0.1245 0.0112 rpy=0 0 3.142

File: software/models/mit_gazebo_models/mit_robot/model_sim_gazebo.urdf (robot description, URDF)
Before this commit: robot atlas, 111 links, 110 joints
Links:
- added link l_hand_force_torque, mass 0.1; visual box size=0.01 0.01 0.01
- added link r_hand_force_torque, mass 0.1; visual box size=0.01 0.01 0.01
Joints:
- added joint l_hand_force_torque_joint: type fixed, parent l_hand, child l_hand_force_torque, origin xyz=0 0.1245 0.0112 rpy=0 0 0
- added joint r_hand_force_torque_joint: type fixed, parent r_hand, child r_hand_force_torque, origin xyz=0 -0.1245 0.0112 rpy=0 0 3.142

File: software/models/mit_gazebo_models/mit_robot/model_sim_v3_v1_inertia.urdf (robot description, URDF)
Before this commit: robot atlas, 75 links, 74 joints
Links:
- removed link left_finger_1_link_0
- removed link left_finger_1_link_1
- removed link left_finger_1_link_2
- removed link left_finger_1_link_3
- removed link left_finger_2_link_0
- removed link left_finger_2_link_1
- removed link left_finger_2_link_2
- removed link left_finger_2_link_3
- removed link left_finger_middle_link_0
- removed link left_finger_middle_link_1
- removed link left_finger_middle_link_2
- removed link left_finger_middle_link_3
- removed link left_hand_camera_link
- removed link left_hand_camera_optical_frame
- removed link left_palm
- removed link right_finger_1_link_0
- removed link right_finger_1_link_1
- removed link right_finger_1_link_2
- removed link right_finger_1_link_3
- removed link right_finger_2_link_0
- removed link right_finger_2_link_1
- removed link right_finger_2_link_2
- removed link right_finger_2_link_3
- removed link right_finger_middle_link_0
- removed link right_finger_middle_link_1
- removed link right_finger_middle_link_2
- removed link right_finger_middle_link_3
- removed link right_hand_camera_link
- removed link right_hand_camera_optical_frame
- removed link right_palm
- added link l_hand_camera_link, mass 0.1; visual box size=0.01 0.01 0.01
- added link l_hand_camera_optical_frame
- added link l_hand_face, mass 0.1; visual box size=0.01 0.01 0.01
- added link l_hand_force_torque, mass 0.1; visual box size=0.01 0.01 0.01
- added link l_hand_gripper, mass 0.1; visual box size=0.01 0.01 0.01
- added link r_hand_camera_link, mass 0.1; visual box size=0.01 0.01 0.01
- added link r_hand_camera_optical_frame
- added link r_hand_face, mass 0.1; visual box size=0.01 0.01 0.01
- added link r_hand_force_torque, mass 0.1; visual box size=0.01 0.01 0.01
- added link r_hand_gripper, mass 0.1; visual box size=0.01 0.01 0.01
Joints:
- removed joint left_finger_1_joint_1
- removed joint left_finger_1_joint_2
- removed joint left_finger_1_joint_3
- removed joint left_finger_2_joint_1
- removed joint left_finger_2_joint_2
- removed joint left_finger_2_joint_3
- removed joint left_finger_middle_joint_1
- removed joint left_finger_middle_joint_2
- removed joint left_finger_middle_joint_3
- removed joint left_hand_camera_joint
- removed joint left_hand_camera_optical_frame_joint
- removed joint left_palm_finger_1_joint
- removed joint left_palm_finger_2_joint
- removed joint left_palm_finger_middle_joint
- removed joint left_robotiq_hand_joint
- removed joint right_finger_1_joint_1
- removed joint right_finger_1_joint_2
- removed joint right_finger_1_joint_3
- removed joint right_finger_2_joint_1
- removed joint right_finger_2_joint_2
- removed joint right_finger_2_joint_3
- removed joint right_finger_middle_joint_1
- removed joint right_finger_middle_joint_2
- removed joint right_finger_middle_joint_3
- removed joint right_hand_camera_joint
- removed joint right_hand_camera_optical_frame_joint
- removed joint right_palm_finger_1_joint
- removed joint right_palm_finger_2_joint
- removed joint right_palm_finger_middle_joint
- removed joint right_robotiq_hand_joint
- added joint l_hand_camera_joint: type fixed, parent l_hand_force_torque, child l_hand_camera_link, origin xyz=-0.09  0.12 0.0 rpy=-1.57079 0  1.41372
- added joint l_hand_camera_optical_frame_joint: type fixed, parent l_hand_camera_link, child l_hand_camera_optical_frame, origin xyz=0 0 0 rpy=-1.5708 0.0 -1.5708
- added joint l_hand_face_joint: type fixed, parent l_hand_force_torque, child l_hand_face, origin xyz=0 0.12 0 rpy=0.0 0.0 0.0
- added joint l_hand_force_torque_joint: type fixed, parent l_hand, child l_hand_force_torque, origin xyz=0 0.1245 0.0112 rpy=0 0 0
- added joint l_hand_gripper_joint: type fixed, parent l_hand_force_torque, child l_hand_gripper, origin xyz=0 0.18 0 rpy=0.0 0.0 0.0
- added joint r_hand_camera_joint: type fixed, parent r_hand_force_torque, child r_hand_camera_link, origin xyz=0.09  0.12 0.0 rpy=-1.57079 0  1.72788
- added joint r_hand_camera_optical_frame_joint: type fixed, parent r_hand_camera_link, child r_hand_camera_optical_frame, origin xyz=0 0 0 rpy=-1.5708 0.0 -1.5708
- added joint r_hand_face_joint: type fixed, parent r_hand_force_torque, child r_hand_face, origin xyz=0 0.12 0 rpy=0.0 0.0 0.0
- added joint r_hand_force_torque_joint: type fixed, parent r_hand, child r_hand_force_torque, origin xyz=0 -0.1245 0.0112 rpy=0 0 3.142
- added joint r_hand_gripper_joint: type fixed, parent r_hand_force_torque, child r_hand_gripper, origin xyz=0 0.18 0 rpy=0.0 0.0 0.0

File: software/models/mit_gazebo_models/mit_robot/xacro/atlas_LH_RH.urdf.xacro (robot description, xacro)
@@ -3,5 +3,6 @@
   <include filename="$(find mit_drcsim_scripts)/models/mit_robot/xacro/atlas.transmission" />
   <include filename="$(find mit_drcsim_scripts)/models/multisense_sl/multisense_sl.urdf" />
- <xacro:include filename="$(find hook_description)/src/bdihook_hand.urdf.xacro" />
+  <include filename="$(find mit_drcsim_scripts)/models/mit_robot/xacro/hand_force_torque.urdf" />
+  <xacro:include filename="$(find hook_description)/src/bdihook_hand.urdf.xacro" />
   <xacro:hook_hand side="right" parent="r_hand" reflect="1" hookflip="-1" noof30degoffset="0">
     <origin rpy="1.57079 0 0" xyz="0 -0.11516 -0.015"/>
