Commit message: made robotiq hand camera xacro reflective. added force torque frame
made robotiq and hand camera relative to FT frame for easy use
removed reference to palm and sandia camera in viewer
added hand_face and hand_gripper

File: software/models/mit_gazebo_models/mit_robot/xacro/atlas_LI_RI.urdf.xacro (robot description, xacro)
@@ -3,4 +3,5 @@
   <include filename="$(find mit_drcsim_scripts)/models/mit_robot/xacro/atlas.transmission" />
   <include filename="$(find mit_drcsim_scripts)/models/multisense_sl/multisense_sl.urdf" />
+  <include filename="$(find mit_drcsim_scripts)/models/mit_robot/xacro/hand_force_torque.urdf" />
   <xacro:include filename="$(find handle_description)/src/irobot_hand_simple.urdf.xacro" />
   <xacro:irobot_hand side="right" parent="r_hand" reflect="1">

File: software/models/mit_gazebo_models/mit_robot/xacro/atlas_LI_RR.urdf.xacro (robot description, xacro)
@@ -3,4 +3,5 @@
   <include filename="$(find mit_drcsim_scripts)/models/mit_robot/xacro/atlas.transmission" />
   <include filename="$(find mit_drcsim_scripts)/models/multisense_sl/multisense_sl.urdf" />
+  <include filename="$(find mit_drcsim_scripts)/models/mit_robot/xacro/hand_force_torque.urdf" />
   <xacro:include filename="$(find handle_description)/src/irobot_hand_simple.urdf.xacro" />
   <xacro:include filename="$(find robotiq_hand_description)/cfg/robotiq_hand.urdf.xacro" />

File: software/models/mit_gazebo_models/mit_robot/xacro/atlas_LI_RR_extender.urdf.xacro (robot description, xacro)
@@ -3,4 +3,5 @@
   <include filename="$(find mit_drcsim_scripts)/models/mit_robot/xacro/atlas.transmission" />
   <include filename="$(find mit_drcsim_scripts)/models/multisense_sl/multisense_sl.urdf" />
+  <include filename="$(find mit_drcsim_scripts)/models/mit_robot/xacro/hand_force_torque.urdf" />
 <!--
 05 sept: Sisir added an offset of 0.045 in the urdf to account

File: software/models/mit_gazebo_models/mit_robot/xacro/atlas_LN_RR.urdf.xacro (robot description, xacro)
@@ -3,4 +3,5 @@
   <include filename="$(find mit_drcsim_scripts)/models/mit_robot/xacro/atlas.transmission" />
   <include filename="$(find mit_drcsim_scripts)/models/multisense_sl/multisense_sl.urdf" />
+  <include filename="$(find mit_drcsim_scripts)/models/mit_robot/xacro/hand_force_torque.urdf" />
   <xacro:include filename="$(find robotiq_hand_description)/cfg/robotiq_hand.urdf.xacro" />
   <xacro:robotiq_hand side="right" parent="r_hand" reflect="1">

File: software/models/mit_gazebo_models/mit_robot/xacro/atlas_LP_RP.urdf.xacro (robot description, xacro)
@@ -3,4 +3,5 @@
   <include filename="$(find mit_drcsim_scripts)/models/mit_robot/xacro/atlas.transmission" />
   <include filename="$(find mit_drcsim_scripts)/models/multisense_sl/multisense_sl.urdf" />
+  <include filename="$(find mit_drcsim_scripts)/models/mit_robot/xacro/hand_force_torque.urdf" />
   <xacro:include filename="$(find hook_description)/src/hook_hand_simple.urdf.xacro" />
   <xacro:hook_hand side="right" parent="r_hand" reflect="1" hookflip="-1" noof30degoffset="0">

File: software/models/mit_gazebo_models/mit_robot/xacro/atlas_LP_RR.urdf.xacro (robot description, xacro)
@@ -3,4 +3,5 @@
   <include filename="$(find mit_drcsim_scripts)/models/mit_robot/xacro/atlas.transmission" />
   <include filename="$(find mit_drcsim_scripts)/models/multisense_sl/multisense_sl.urdf" />
+  <include filename="$(find mit_drcsim_scripts)/models/mit_robot/xacro/hand_force_torque.urdf" />
   <xacro:include filename="$(find hook_description)/src/hook_hand_simple.urdf.xacro" />
   <xacro:include filename="$(find robotiq_hand_description)/cfg/robotiq_hand.urdf.xacro" />
