Commit message: changed orientation of hands by 180 degrees to match human reaching
also have the camera outward facing

File: ros_workspace/robotiq_camera/urdf/robotiq_camera.urdf.xacro (robot description, xacro)
@@ -31,17 +31,13 @@
       <camera name="${side}_hand_camera">
         <pose>0 0 0 0 0 0</pose>
-        <!-- Spec sheet says 185deg HFOV @ 1280x1024pi @ 60 hz.
-             Don't think most GPU's can achieve this at real-time right now.
-        <horizontal_fov>3.22885912</horizontal_fov>
-        -->
-        <horizontal_fov>2.0</horizontal_fov>
+        <horizontal_fov>1.25663706144</horizontal_fov>
         <image>
-          <width>1280</width>
-          <height>1024</height>
+          <width>752</width>
+          <height>480</height>
           <format>R8G8B8</format>
         </image>
         <clip>
           <near>0.02</near>
-          <far>300</far>
+          <far>100</far>
         </clip>
         <noise>

File: software/models/mit_gazebo_models/mit_robot/model_LR_RR.urdf (robot description, URDF)
Before this commit: robot atlas, 74 links, 73 joints
Joints:
- joint left_robotiq_hand_joint: origin xyz=0 0.19016 0.015 rpy=0 1.57079 0 -> xyz=0 0.19016 0.015 rpy=0 -1.57079 0
- joint right_robotiq_hand_joint: origin xyz=0 -0.19016 -0.015 rpy=0 1.57079 3.141 -> xyz=0 -0.19016 -0.015 rpy=0 -1.57079 3.141

File: software/models/mit_gazebo_models/mit_robot/xacro/atlas_LR_RR.urdf.xacro (robot description, xacro)
@@ -3,10 +3,13 @@
   <include filename="$(find mit_drcsim_scripts)/models/mit_robot/xacro/atlas.transmission" />
   <include filename="$(find mit_drcsim_scripts)/models/multisense_sl/multisense_sl_sim.urdf" />
+<!--  left was  0 1.57079 0 -->
+<!-- right was  0 1.57079 3.141 -->
+<!-- both were orientated for connectors back and camera outside -->
   <xacro:include filename="$(find robotiq_hand_description)/cfg/robotiq_hand.urdf.xacro" />
   <xacro:robotiq_hand side="left" parent="l_hand" reflect="1">
-    <origin rpy="0 1.57079 0" xyz="0 0.19016 0.015"/>
+    <origin rpy="0 -1.57079 0" xyz="0 0.19016 0.015"/>
   </xacro:robotiq_hand>
   <xacro:robotiq_hand side="right" parent="r_hand" reflect="1">
-    <origin rpy="0 1.57079 3.141" xyz="0 -0.19016 -0.015"/>
+    <origin rpy="0 -1.57079 3.141" xyz="0 -0.19016 -0.015"/>
   </xacro:robotiq_hand>
   <xacro:include filename="$(find robotiq_camera)/urdf/robotiq_camera.urdf.xacro" />

Commit message: approximate configuration of hand cameras
changed to sa fov
added camera[]hand for robotiq
added 9degree rotation and estimated positon transform
planning to depreciate sandia hands support

File: ros_workspace/robotiq_camera/urdf/robotiq_camera.urdf.xacro (robot description, xacro)
@@ -31,8 +31,9 @@
       <camera name="${side}_hand_camera">
         <pose>0 0 0 0 0 0</pose>
-        <horizontal_fov>1.25663706144</horizontal_fov>
+        <!-- m.antone estimate of 2.8mm tamron lense fov -->
+        <horizontal_fov>2.0</horizontal_fov>
         <image>
-          <width>752</width>
-          <height>480</height>
+          <width>1280</width>
+          <height>1024</height>
           <format>R8G8B8</format>
         </image>

File: software/models/mit_gazebo_models/mit_robot/model_LR_RR.urdf (robot description, URDF)
Before this commit: robot atlas, 74 links, 73 joints
Joints:
- joint left_hand_camera_joint: origin xyz=0.0  0.25 0.0 rpy=-1.57079 0  1.57079 -> xyz=-0.09  0.24 0.0 rpy=-1.57079 0  1.41369
- joint right_hand_camera_joint: origin xyz=0.0  -0.25 0.0 rpy=-1.57079 3.14158 1.57079 -> xyz=-0.09  -0.24 0.0 rpy=-1.57079 3.14158 1.72789

File: software/models/mit_gazebo_models/mit_robot/model_sim_v3_v1_inertia.urdf (robot description, URDF)
Before this commit: robot atlas, 49 links, 48 joints
Links:
- added link left_finger_1_link_0; collision mesh filename=package://robotiq_hand_description/meshes/s-model_articulat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; visual mesh filename=package://robotiq_hand_description/meshes/s-model_articulat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
- added link left_finger_1_link_1; collision mesh filename=package://robotiq_hand_description/meshes/s-model_articulat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; visual mesh filename=package://robotiq_hand_description/meshes/s-model_articulat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
- added link left_finger_1_link_2; collision mesh filename=package://robotiq_hand_description/meshes/s-model_articulat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; visual mesh filename=package://robotiq_hand_description/meshes/s-model_articulat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
- added link left_finger_1_link_3; collision mesh filename=package://robotiq_hand_description/meshes/s-model_articulat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; visual mesh filename=package://robotiq_hand_description/meshes/s-model_articulat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
- added link left_finger_2_link_0; collision mesh filename=package://robotiq_hand_description/meshes/s-model_articulat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; visual mesh filename=package://robotiq_hand_description/meshes/s-model_articulat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
- added link left_finger_2_link_1; collision mesh filename=package://robotiq_hand_description/meshes/s-model_articulat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; visual mesh filename=package://robotiq_hand_description/meshes/s-model_articulat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
- added link left_finger_2_link_2; collision mesh filename=package://robotiq_hand_description/meshes/s-model_articulat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; visual mesh filename=package://robotiq_hand_description/meshes/s-model_articulat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
- added link left_finger_2_link_3; collision mesh filename=package://robotiq_hand_description/meshes/s-model_articulat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; visual mesh filename=package://robotiq_hand_description/meshes/s-model_articulat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
- added link left_finger_middle_link_0; collision mesh filename=package://robotiq_hand_description/meshes/s-model_articulat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; visual mesh filename=package://robotiq_hand_description/meshes/s-model_articulat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
- added link left_finger_middle_link_1; collision mesh filename=package://robotiq_hand_description/meshes/s-model_articulat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; visual mesh filename=package://robotiq_hand_description/meshes/s-model_articulat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
- added link left_finger_middle_link_2; collision mesh filename=package://robotiq_hand_description/meshes/s-model_articulat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; visual mesh filename=package://robotiq_hand_description/meshes/s-model_articulat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
- added link left_finger_middle_link_3; collision mesh filename=package://robotiq_hand_description/meshes/s-model_articulat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; visual mesh filename=package://robotiq_hand_description/meshes/s-model_articulat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
- added link left_palm; collision mesh filename=package://robotiq_hand_description/meshes/s-model_articulat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; visual mesh filename=package://robotiq_hand_description/meshes/s-model_articulat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
- added link right_finger_1_link_0; collision mesh filename=package://robotiq_hand_description/meshes/s-model_articulat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; visual mesh filename=package://robotiq_hand_description/meshes/s-model_articulat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
- added link right_finger_1_link_1; collision mesh filename=package://robotiq_hand_description/meshes/s-model_articulat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; visual mesh filename=package://robotiq_hand_description/meshes/s-model_articulat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
- added link right_finger_1_link_2; collision mesh filename=package://robotiq_hand_description/meshes/s-model_articulat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; visual mesh filename=package://robotiq_hand_description/meshes/s-model_articulat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
- added link right_finger_1_link_3; collision mesh filename=package://robotiq_hand_description/meshes/s-model_articulat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; visual mesh filename=package://robotiq_hand_description/meshes/s-model_articulat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
- added link right_finger_2_link_0; collision mesh filename=package://robotiq_hand_description/meshes/s-model_articulat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; visual mesh filename=package://robotiq_hand_description/meshes/s-model_articulat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
- added link right_finger_2_link_1; collision mesh filename=package://robotiq_hand_description/meshes/s-model_articulat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; visual mesh filename=package://robotiq_hand_description/meshes/s-model_articulat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
- added link right_finger_2_link_2; collision mesh filename=package://robotiq_hand_description/meshes/s-model_articulat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; visual mesh filename=package://robotiq_hand_description/meshes/s-model_articulat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
- added link right_finger_2_link_3; collision mesh filename=package://robotiq_hand_description/meshes/s-model_articulat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; visual mesh filename=package://robotiq_hand_description/meshes/s-model_articulat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
- added link right_finger_middle_link_0; collision mesh filename=package://robotiq_hand_description/meshes/s-model_articulat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; visual mesh filename=package://robotiq_hand_description/meshes/s-model_articulat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
- added link right_finger_middle_link_1; collision mesh filename=package://robotiq_hand_description/meshes/s-model_articulat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; visual mesh filename=package://robotiq_hand_description/meshes/s-model_articulat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
- added link right_finger_middle_link_2; collision mesh filename=package://robotiq_hand_description/meshes/s-model_articulat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; visual mesh filename=package://robotiq_hand_description/meshes/s-model_articulat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
- added link right_finger_middle_link_3; collision mesh filename=package://robotiq_hand_description/meshes/s-model_articulat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; visual mesh filename=package://robotiq_hand_description/meshes/s-model_articulat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
- added link right_palm; collision mesh filename=package://robotiq_hand_description/meshes/s-model_articulat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; visual mesh filename=package://robotiq_hand_description/meshes/s-model_articulat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
Joints:
- added joint left_finger_1_joint_1: type revolute, parent left_finger_1_link_0, child left_finger_1_link_1, origin xyz=0.020 0 0 rpy=0 0 0, axis 0 0 1, limit lower=0 upper=3.1416 effort=100 velocity=100
- added joint left_finger_1_joint_2: type revolute, parent left_finger_1_link_1, child left_finger_1_link_2, origin xyz=0.050 -.028 0 rpy=0 0 -0.52, axis 0 0 1, limit lower=0 upper=3.1416 effort=100 velocity=100
- added joint left_finger_1_joint_3: type revolute, parent left_finger_1_link_2, child left_finger_1_link_3, origin xyz=0.039 0 0 rpy=0 0 0, axis 0 0 1, limit lower=0 upper=3.1416 effort=100 velocity=100
- added joint left_finger_2_joint_1: type revolute, parent left_finger_2_link_0, child left_finger_2_link_1, origin xyz=0.020 0 0 rpy=0 0 0, axis 0 0 1, limit lower=0 upper=3.1416 effort=100 velocity=100
- added joint left_finger_2_joint_2: type revolute, parent left_finger_2_link_1, child left_finger_2_link_2, origin xyz=0.050 -.028 0 rpy=0 0 -0.52, axis 0 0 1, limit lower=0 upper=3.1416 effort=100 velocity=100
- added joint left_finger_2_joint_3: type revolute, parent left_finger_2_link_2, child left_finger_2_link_3, origin xyz=0.039 0 0 rpy=0 0 0, axis 0 0 1, limit lower=0 upper=3.1416 effort=100 velocity=100
- added joint left_finger_middle_joint_1: type revolute, parent left_finger_middle_link_0, child left_finger_middle_link_1, origin xyz=0.020 0 0 rpy=0 0 0, axis 0 0 1, limit lower=0 upper=3.1416 effort=100 velocity=100
- added joint left_finger_middle_joint_2: type revolute, parent left_finger_middle_link_1, child left_finger_middle_link_2, origin xyz=0.050 -.028 0 rpy=0 0 -0.52, axis 0 0 1, limit lower=0 upper=3.1416 effort=100 velocity=100
- added joint left_finger_middle_joint_3: type revolute, parent left_finger_middle_link_2, child left_finger_middle_link_3, origin xyz=0.039 0 0 rpy=0 0 0, axis 0 0 1, limit lower=0 upper=3.1416 effort=100 velocity=100
- added joint left_palm_finger_1_joint: type revolute, parent left_palm, child left_finger_1_link_0, origin xyz=-0.0455 0.0214 0.036 rpy=0 3.1416 -1.57, axis 0 1 0, limit lower=-0.16 upper=0.25 effort=100 velocity=100
- added joint left_palm_finger_2_joint: type revolute, parent left_palm, child left_finger_2_link_0, origin xyz=-0.0455 0.0214 -0.036 rpy=0 3.1416 -1.57, axis 0 1 0, limit lower=-0.25 upper=0.16 effort=100 velocity=100
- added joint left_palm_finger_middle_joint: type fixed, parent left_palm, child left_finger_middle_link_0, origin xyz=0.0455 0.0214 0 rpy=0 0 1.57, axis 0 0 1
- added joint left_robotiq_hand_joint: type fixed, parent l_hand, child left_palm, origin xyz=0 0.19016 0.015 rpy=0 -1.57079 0
- added joint right_finger_1_joint_1: type revolute, parent right_finger_1_link_0, child right_finger_1_link_1, origin xyz=0.020 0 0 rpy=0 0 0, axis 0 0 1, limit lower=0 upper=3.1416 effort=100 velocity=100
- added joint right_finger_1_joint_2: type revolute, parent right_finger_1_link_1, child right_finger_1_link_2, origin xyz=0.050 -.028 0 rpy=0 0 -0.52, axis 0 0 1, limit lower=0 upper=3.1416 effort=100 velocity=100
- added joint right_finger_1_joint_3: type revolute, parent right_finger_1_link_2, child right_finger_1_link_3, origin xyz=0.039 0 0 rpy=0 0 0, axis 0 0 1, limit lower=0 upper=3.1416 effort=100 velocity=100
- added joint right_finger_2_joint_1: type revolute, parent right_finger_2_link_0, child right_finger_2_link_1, origin xyz=0.020 0 0 rpy=0 0 0, axis 0 0 1, limit lower=0 upper=3.1416 effort=100 velocity=100
- added joint right_finger_2_joint_2: type revolute, parent right_finger_2_link_1, child right_finger_2_link_2, origin xyz=0.050 -.028 0 rpy=0 0 -0.52, axis 0 0 1, limit lower=0 upper=3.1416 effort=100 velocity=100
- added joint right_finger_2_joint_3: type revolute, parent right_finger_2_link_2, child right_finger_2_link_3, origin xyz=0.039 0 0 rpy=0 0 0, axis 0 0 1, limit lower=0 upper=3.1416 effort=100 velocity=100
- added joint right_finger_middle_joint_1: type revolute, parent right_finger_middle_link_0, child right_finger_middle_link_1, origin xyz=0.020 0 0 rpy=0 0 0, axis 0 0 1, limit lower=0 upper=3.1416 effort=100 velocity=100
- added joint right_finger_middle_joint_2: type revolute, parent right_finger_middle_link_1, child right_finger_middle_link_2, origin xyz=0.050 -.028 0 rpy=0 0 -0.52, axis 0 0 1, limit lower=0 upper=3.1416 effort=100 velocity=100
- added joint right_finger_middle_joint_3: type revolute, parent right_finger_middle_link_2, child right_finger_middle_link_3, origin xyz=0.039 0 0 rpy=0 0 0, axis 0 0 1, limit lower=0 upper=3.1416 effort=100 velocity=100
- added joint right_palm_finger_1_joint: type revolute, parent right_palm, child right_finger_1_link_0, origin xyz=-0.0455 0.0214 0.036 rpy=0 3.1416 -1.57, axis 0 1 0, limit lower=-0.16 upper=0.25 effort=100 velocity=100
- added joint right_palm_finger_2_joint: type revolute, parent right_palm, child right_finger_2_link_0, origin xyz=-0.0455 0.0214 -0.036 rpy=0 3.1416 -1.57, axis 0 1 0, limit lower=-0.25 upper=0.16 effort=100 velocity=100
- added joint right_palm_finger_middle_joint: type fixed, parent right_palm, child right_finger_middle_link_0, origin xyz=0.0455 0.0214 0 rpy=0 0 1.57, axis 0 0 1
- added joint right_robotiq_hand_joint: type fixed, parent r_hand, child right_palm, origin xyz=0 -0.19016 -0.015 rpy=0 -1.57079 3.141
- joint left_hand_camera_joint: origin xyz=0.0  0.25 0.0 rpy=-1.57079 0  1.57079 -> xyz=-0.09  0.24 0.0 rpy=-1.57079 0  1.41369
- joint right_hand_camera_joint: origin xyz=0.0  -0.25 0.0 rpy=-1.57079 3.14158 1.57079 -> xyz=-0.09  -0.24 0.0 rpy=-1.57079 3.14158 1.72789

File: software/models/mit_gazebo_models/mit_robot/xacro/atlas_LR_RR.urdf.xacro (robot description, xacro)
@@ -13,10 +13,13 @@
     <origin rpy="0 -1.57079 3.141" xyz="0 -0.19016 -0.015"/>
   </xacro:robotiq_hand>
+<!-- right was 0  0.25 0    -1.57079 0  1.57079      -->
+<!-- right was 0 -0.25 0    -1.57079 3.14158 1.57079 -->
+<!-- 9d = 0.1571 rad -->
   <xacro:include filename="$(find robotiq_camera)/urdf/robotiq_camera.urdf.xacro" />
   <xacro:robotiq_camera side="left" parent="l_hand" >
-    <origin xyz="0.0  0.25 0.0" rpy="-1.57079 0  1.57079"/>
+    <origin xyz="-0.09  0.24 0.0" rpy="-1.57079 0  1.41369"/>
   </xacro:robotiq_camera>
   <xacro:robotiq_camera side="right" parent="r_hand" >
-    <origin xyz="0.0  -0.25 0.0" rpy="-1.57079 3.14158 1.57079"/>
+    <origin xyz="-0.09  -0.24 0.0" rpy="-1.57079 3.14158 1.72789"/>
   </xacro:robotiq_camera>
 </robot>

File: software/models/mit_gazebo_models/mit_robot/xacro/atlas_sandia_hands_sim_v3_v1_inertia.urdf.xacro (robot description, xacro)
@@ -6,10 +6,19 @@
   <xacro:include filename="$(find multisense_sl_description)/urdf/multisense_sl_v3.urdf" />
   <include filename="$(find mit_drcsim_scripts)/models/mit_robot/xacro/mit_atlas.gazebo" />
+  <xacro:include filename="$(find robotiq_hand_description)/cfg/robotiq_hand.urdf.xacro" />
+  <xacro:robotiq_hand side="left" parent="l_hand" reflect="1">
+    <origin rpy="0 -1.57079 0" xyz="0 0.19016 0.015"/>
+  </xacro:robotiq_hand>
+  <xacro:robotiq_hand side="right" parent="r_hand" reflect="1">
+    <origin rpy="0 -1.57079 3.141" xyz="0 -0.19016 -0.015"/>
+  </xacro:robotiq_hand>
+<!-- left was 0  0.25 0    -1.57079 0  1.57079 -->
+<!-- right was 0 -0.25 0   -1.57079 3.14158 1.57079 -->
   <xacro:include filename="$(find robotiq_camera)/urdf/robotiq_camera.urdf.xacro" />
   <xacro:robotiq_camera side="left" parent="l_hand" >
-    <origin xyz="0.0  0.25 0.0" rpy="-1.57079 0  1.57079"/>
+    <origin xyz="-0.09  0.24 0.0" rpy="-1.57079 0  1.41369"/>
   </xacro:robotiq_camera>
   <xacro:robotiq_camera side="right" parent="r_hand" >
-    <origin xyz="0.0  -0.25 0.0" rpy="-1.57079 3.14158 1.57079"/>
+    <origin xyz="-0.09  -0.24 0.0" rpy="-1.57079 3.14158 1.72789"/>
   </xacro:robotiq_camera>
 </robot>

Commit message: adding angualr poly configuration to camera rhand
corrected rbotiq off line
corrected camera rotation in robotiq
clean up tool for gilwoo and peter

File: ros_workspace/robotiq_camera/urdf/robotiq_camera.urdf.xacro (robot description, xacro)
@@ -55,5 +55,5 @@
     <child link="${side_letter}_hand_camera_link"/>
     <!-- 9 degree inward angle-->
-    <origin xyz="${-0.09*reflect}  0.12 0.0" rpy="-1.57079 0  ${1.5708-reflect*0.15708}"/>
+    <origin xyz="${-0.09*reflect}  0.12 0.0" rpy=" ${-reflect*1.57079} 0  ${1.5708-reflect*0.15708}"/>
   </joint>
   <joint name="${side_letter}_hand_camera_optical_frame_joint" type="fixed">
@@ -69,5 +69,5 @@
         <pose>0 0 0 0 0 0</pose>
         <!-- m.antone estimate of 2.8mm tamron lense fov -->
-        <horizontal_fov>2.0</horizontal_fov>
+        <horizontal_fov>1.7281</horizontal_fov>
         <image>
           <width>1280</width>

File: software/models/mit_gazebo_models/mit_robot/model_LH_RH.urdf (robot description, URDF)
Before this commit: robot atlas, 60 links, 59 joints
Joints:
- joint r_hand_force_torque_joint: origin xyz=0 -0.1245 0.0112 rpy=0 0 3.142 -> xyz=0 -0.1245 -0.0112 rpy=0 0 3.142

File: software/models/mit_gazebo_models/mit_robot/model_LI_RI.urdf (robot description, URDF)
Before this commit: robot atlas, 76 links, 75 joints
Joints:
- joint r_hand_force_torque_joint: origin xyz=0 -0.1245 0.0112 rpy=0 0 3.142 -> xyz=0 -0.1245 -0.0112 rpy=0 0 3.142

File: software/models/mit_gazebo_models/mit_robot/model_LI_RR.urdf (robot description, URDF)
Before this commit: robot atlas, 80 links, 79 joints
Joints:
- joint r_hand_force_torque_joint: origin xyz=0 -0.1245 0.0112 rpy=0 0 3.142 -> xyz=0 -0.1245 -0.0112 rpy=0 0 3.142

File: software/models/mit_gazebo_models/mit_robot/model_LI_RR_extender.urdf (robot description, URDF)
Before this commit: robot atlas, 82 links, 81 joints
Joints:
- joint r_hand_force_torque_joint: origin xyz=0 -0.1245 0.0112 rpy=0 0 3.142 -> xyz=0 -0.1245 -0.0112 rpy=0 0 3.142

File: software/models/mit_gazebo_models/mit_robot/model_LP_RP.urdf (robot description, URDF)
Before this commit: robot atlas, 60 links, 59 joints
Joints:
- joint r_hand_force_torque_joint: origin xyz=0 -0.1245 0.0112 rpy=0 0 3.142 -> xyz=0 -0.1245 -0.0112 rpy=0 0 3.142

File: software/models/mit_gazebo_models/mit_robot/model_LP_RR.urdf (robot description, URDF)
Before this commit: robot atlas, 72 links, 71 joints
Joints:
- joint r_hand_force_torque_joint: origin xyz=0 -0.1245 0.0112 rpy=0 0 3.142 -> xyz=0 -0.1245 -0.0112 rpy=0 0 3.142

File: software/models/mit_gazebo_models/mit_robot/model_LQ_RP.urdf (robot description, URDF)
Before this commit: robot atlas, 73 links, 72 joints
Joints:
- joint r_hand_force_torque_joint: origin xyz=0 -0.1245 0.0112 rpy=0 0 3.142 -> xyz=0 -0.1245 -0.0112 rpy=0 0 3.142

File: software/models/mit_gazebo_models/mit_robot/model_LR_RR.urdf (robot description, URDF)
Before this commit: robot atlas, 80 links, 79 joints
Joints:
- joint l_hand_camera_joint: origin xyz=-0.09  0.12 0.0 rpy=-1.57079 0  1.41372 -> xyz=-0.09  0.12 0.0 rpy= -1.57079 0  1.41372
- joint r_hand_camera_joint: origin xyz=0.09  0.12 0.0 rpy=-1.57079 0  1.72788 -> xyz=0.09  0.12 0.0 rpy= 1.57079 0  1.72788
- joint r_hand_force_torque_joint: origin xyz=0 -0.1245 0.0112 rpy=0 0 3.142 -> xyz=0 -0.1245 -0.0112 rpy=0 0 3.142

File: software/models/mit_gazebo_models/mit_robot/model_sim.urdf (robot description, URDF)
Before this commit: robot atlas, 113 links, 112 joints
Joints:
- joint r_hand_force_torque_joint: origin xyz=0 -0.1245 0.0112 rpy=0 0 3.142 -> xyz=0 -0.1245 -0.0112 rpy=0 0 3.142

File: software/models/mit_gazebo_models/mit_robot/model_sim_gazebo.urdf (robot description, URDF)
Before this commit: robot atlas, 113 links, 112 joints
Joints:
- joint r_hand_force_torque_joint: origin xyz=0 -0.1245 0.0112 rpy=0 0 3.142 -> xyz=0 -0.1245 -0.0112 rpy=0 0 3.142

File: software/models/mit_gazebo_models/mit_robot/model_sim_v3_v1_inertia.urdf (robot description, URDF)
Before this commit: robot atlas, 55 links, 54 joints
Joints:
- joint l_hand_camera_joint: origin xyz=-0.09  0.12 0.0 rpy=-1.57079 0  1.41372 -> xyz=-0.09  0.12 0.0 rpy= -1.57079 0  1.41372
- joint r_hand_camera_joint: origin xyz=0.09  0.12 0.0 rpy=-1.57079 0  1.72788 -> xyz=0.09  0.12 0.0 rpy= 1.57079 0  1.72788
- joint r_hand_force_torque_joint: origin xyz=0 -0.1245 0.0112 rpy=0 0 3.142 -> xyz=0 -0.1245 -0.0112 rpy=0 0 3.142

File: software/models/mit_gazebo_models/mit_robot/xacro/hand_force_torque.urdf (robot description, URDF)
Before this commit: robot hand_force_torque, 2 links, 2 joints
Joints:
- joint r_hand_force_torque_joint: origin xyz=0 -0.1245 0.0112 rpy=0 0 3.142 -> xyz=0 -0.1245 -0.0112 rpy=0 0 3.142
