Commit message: remove link visualization for robotiq fixed frames

File: ros_workspace/robotiq_camera/urdf/robotiq_camera.urdf.xacro (robot description, xacro)
@@ -7,17 +7,5 @@
     <child link="${side_letter}_hand_face"/>
   </joint>
-  <link name="${side_letter}_hand_face">
-    <inertial>
-      <mass value="0.1"/>
-      <origin xyz="0 0 0"/>
-      <inertia ixx="0.00001" ixy="0" ixz="0" iyy="0.00001" iyz="0" izz="0.00001"/>
-    </inertial>
-    <visual>
-      <origin rpy="0 0 0" xyz="0 0 0"/>
-      <geometry>
-        <box size="0.01 0.01 0.01"/>
-      </geometry>
-    </visual>
-  </link>
+  <link name="${side_letter}_hand_face"/>
   <joint name="${side_letter}_hand_gripper_joint" type="fixed">
     <origin rpy="0.0 0.0 0.0" xyz="0 0.18 0"/>
@@ -25,30 +13,6 @@
     <child link="${side_letter}_hand_gripper"/>
   </joint>
-  <link name="${side_letter}_hand_gripper">
-    <inertial>
-      <mass value="0.1"/>
-      <origin xyz="0 0 0"/>
-      <inertia ixx="0.00001" ixy="0" ixz="0" iyy="0.00001" iyz="0" izz="0.00001"/>
-    </inertial>
-    <visual>
-      <origin rpy="0 0 0" xyz="0 0 0"/>
-      <geometry>
-        <box size="0.01 0.01 0.01"/>
-      </geometry>
-    </visual>
-  </link>
-  <link name="${side_letter}_hand_camera_link">
-    <inertial>
-      <mass value="0.1"/>
-      <origin xyz="0 0 0"/>
-      <inertia ixx="0.00001" ixy="0" ixz="0" iyy="0.00001" iyz="0" izz="0.00001"/>
-    </inertial>
-    <visual>
-      <origin rpy="0 0 0" xyz="0 0 0"/>
-      <geometry>
-        <box size="0.01 0.01 0.01"/>
-      </geometry>
-    </visual>
-  </link>
+  <link name="${side_letter}_hand_gripper"/>
+  <link name="${side_letter}_hand_camera_link"/>
   <joint name="${side_letter}_hand_camera_joint" type="fixed">
     <parent link="${parent}"/>

File: software/models/mit_gazebo_models/mit_robot/model_LR_RR.urdf (robot description, URDF)
Before this commit: robot atlas, 92 links, 91 joints
Links:
- link l_hand_camera_link: mass 0.1 -> None; geometry 
- link l_hand_face: mass 0.1 -> None; geometry 
- link l_hand_gripper: mass 0.1 -> None; geometry 
- link r_hand_camera_link: mass 0.1 -> None; geometry 
- link r_hand_face: mass 0.1 -> None; geometry 
- link r_hand_gripper: mass 0.1 -> None; geometry 

File: software/models/mit_gazebo_models/mit_robot/model_LR_RR_sim_v1_inertia.urdf (robot description, URDF)
Before this commit: robot atlas, 55 links, 54 joints
Links:
- link l_hand_camera_link: mass 0.1 -> None; geometry 
- link l_hand_face: mass 0.1 -> None; geometry 
- link l_hand_gripper: mass 0.1 -> None; geometry 
- link r_hand_camera_link: mass 0.1 -> None; geometry 
- link r_hand_face: mass 0.1 -> None; geometry 
- link r_hand_gripper: mass 0.1 -> None; geometry 

Commit message: Modifications to robotiq hands and camera location just for testing.

File: ros_workspace/robotiq_camera/urdf/robotiq_camera.urdf.xacro (robot description, xacro)
@@ -19,5 +19,5 @@
     <child link="${side_letter}_hand_camera_link"/>
     <!-- 9 degree inward angle-->
-    <origin xyz="${-0.09*reflect}  0.12 0.0" rpy=" ${-reflect*1.57079} 0  ${1.5708-reflect*0.15708}"/>
+    <origin xyz="${-0.096*reflect}  0.06 0.0" rpy=" ${-reflect*1.57079} 0  ${1.5708-reflect*0.0}"/>
   </joint>
   <joint name="${side_letter}_hand_camera_optical_frame_joint" type="fixed">

File: software/models/mit_gazebo_models/mit_robot/xacro/atlas_LR_RR.urdf.xacro (robot description, xacro)
@@ -7,5 +7,6 @@
   <xacro:include filename="$(find robotiq_hand_description)/cfg/robotiq_hand.urdf.xacro" />
   <xacro:robotiq_hand side="left" parent="l_hand_force_torque" reflect="1">
-    <origin rpy="0 -1.57079 0" xyz="0 0.06566 0.0"/>
+    <!--origin rpy="0 -1.57079 0" xyz="0 0.06566 0.0"/-->
+    <origin rpy="0 -1.57079 0" xyz="0 0.21846 0.0"/>
   </xacro:robotiq_hand>
   <xacro:robotiq_hand side="right" parent="r_hand_force_torque" reflect="1">

Commit message: Updates to robotiq URDFs after we moved the camera back slightly. This was to give clearance for the drill.

File: ros_workspace/robotiq_camera/urdf/robotiq_camera.urdf.xacro (robot description, xacro)
@@ -18,9 +18,9 @@
     <parent link="${parent}"/>
     <child link="${side_letter}_hand_camera_link"/>
-    <!-- 9 degree inward angle-->
-    <origin xyz="${-0.096*reflect}  0.06 0.0" rpy=" ${-reflect*1.57079} 0  ${1.5708-reflect*0.0}"/>
+    <!-- new camera has no inward angle, placeholder is still here in case it is later tilted-->
+    <origin xyz="${-0.09892*reflect}  0.01431 0.0" rpy=" ${-reflect*1.57079} 0  ${1.5708-reflect*0.0}"/>
   </joint>
   <joint name="${side_letter}_hand_camera_optical_frame_joint" type="fixed">
-    <origin rpy="-1.5708 0.0 -1.5708" xyz="0 0 0"/>
+    <origin rpy="-1.57079 0.0 -1.57079" xyz="0 0 0"/>
     <parent link="${side_letter}_hand_camera_link"/>
     <child link="${side_letter}_hand_camera_optical_frame"/>

File: software/models/mit_gazebo_models/mit_robot/model_LR_RR.urdf (robot description, URDF)
Before this commit: robot atlas, 92 links, 91 joints
Joints:
- joint l_hand_camera_joint: origin xyz=-0.09  0.12 0.0 rpy= -1.57079 0  1.41372 -> xyz=-0.09892  0.01431 0.0 rpy= -1.57079 0  1.5708
- joint l_hand_camera_optical_frame_joint: origin xyz=0 0 0 rpy=-1.5708 0.0 -1.5708 -> xyz=0 0 0 rpy=-1.57079 0.0 -1.57079
- joint r_hand_camera_joint: origin xyz=0.09  0.12 0.0 rpy= 1.57079 0  1.72788 -> xyz=0.09892  0.01431 0.0 rpy= 1.57079 0  1.5708
- joint r_hand_camera_optical_frame_joint: origin xyz=0 0 0 rpy=-1.5708 0.0 -1.5708 -> xyz=0 0 0 rpy=-1.57079 0.0 -1.57079
