Commit message: reorg of hand joint names to use 7th dof

File: software/models/mit_gazebo_models/V1/models/V1/urdf/V1_sim_mit.urdf (robot description, URDF)
Before this commit: robot V1, 92 links, 91 joints
Links:
- added link /v1/LeftMedialMetacarpal, mass 0.047; collision mesh filename=package://V1/models/V1/meshes/2013_05_16/ssf1_Left.stl; visual mesh filename=package://V1/models/V1/meshes/2013_05_16/ssf1_Left.stl
- added link /v1/LeftMiddleProximalPhalanx, mass 0.02; collision mesh filename=package://V1/models/V1/meshes/2013_05_16/sf1.stl; visual mesh filename=package://V1/models/V1/meshes/2013_05_16/sf1.stl
- added link /v1/RightMedialMetacarpal, mass 0.047; collision mesh filename=package://V1/models/V1/meshes/2013_05_16/ssf1_Right.stl; visual mesh filename=package://V1/models/V1/meshes/2013_05_16/ssf1_Right.stl
- added link /v1/RightMiddleProximalPhalanx, mass 0.02; collision mesh filename=package://V1/models/V1/meshes/2013_05_16/sf1.stl; visual mesh filename=package://V1/models/V1/meshes/2013_05_16/sf1.stl
- added link l_uhand, mass 0.1; collision box size=0.03 0.01 0.051; visual box size=0.03 0.01 0.051
- added link r_uhand, mass 0.1; collision box size=0.03 0.01 0.051; visual box size=0.03 0.01 0.051
- link l_hand: mass 0.1 -> 0.712; geometry collision mesh filename=package://V1/models/V1/meshes/2013_05_16/palm_Left.stl; visual mesh filename=package://V1/models/V1/meshes/2013_05_16/palm_Left.stl
- link l_hand_face: mass 0.02 -> 0.001; geometry visual box size=0.01 0.01 0.01
- link l_hand_force_torque: mass 0.047 -> 0.001; geometry visual box size=0.01 0.01 0.01
- link left_palm: mass 0.712 -> 0.001; geometry visual box size=0.01 0.01 0.01
- link r_hand: mass 0.1 -> 0.712; geometry collision mesh filename=package://V1/models/V1/meshes/2013_05_16/palm_Right.stl; visual mesh filename=package://V1/models/V1/meshes/2013_05_16/palm_Right.stl
- link r_hand_face: mass 0.02 -> 0.001; geometry visual box size=0.01 0.01 0.01
- link r_hand_force_torque: mass 0.047 -> 0.001; geometry visual box size=0.01 0.01 0.01
- link right_palm: mass 0.712 -> 0.001; geometry visual box size=0.01 0.01 0.01
Joints:
- added joint l_hand_face_joint: type fixed, parent l_hand_force_torque, child l_hand_face, origin xyz=0 0 0 rpy=0 0 0
- added joint l_hand_force_torque_joint: type fixed, parent l_hand, child l_hand_force_torque, origin xyz=0 0 0 rpy=0 0 0
- added joint left_valkyrie_hand_joint: type fixed, parent l_hand_force_torque, child left_palm, origin xyz=0 0 0 rpy=0 0 0
- added joint r_hand_face_joint: type fixed, parent r_hand_force_torque, child r_hand_face, origin xyz=0 0 0 rpy=0 0 0
- added joint r_hand_force_torque_joint: type fixed, parent r_hand, child r_hand_force_torque, origin xyz=0 0 0 rpy=0 0 0
- added joint right_valkyrie_hand_joint: type fixed, parent r_hand_force_torque, child right_palm, origin xyz=0 0 0 rpy=0 0 0
- joint LeftLittleMPExtensor: parent l_hand_force_torque -> /v1/LeftMedialMetacarpal
- joint LeftLittleMPYaw: child l_hand_force_torque -> /v1/LeftMedialMetacarpal
- joint LeftMiddleMPExtensor: child l_hand_face -> /v1/LeftMiddleProximalPhalanx
- joint LeftMiddlePIPExtensor: parent l_hand_face -> /v1/LeftMiddleProximalPhalanx
- joint RightLittleMPExtensor: parent r_hand_force_torque -> /v1/RightMedialMetacarpal
- joint RightLittleMPYaw: child r_hand_force_torque -> /v1/RightMedialMetacarpal
- joint RightMiddleMPExtensor: child r_hand_face -> /v1/RightMiddleProximalPhalanx
- joint RightMiddlePIPExtensor: parent r_hand_face -> /v1/RightMiddleProximalPhalanx
- joint l_arm_lwz: child left_palm -> l_hand; parent l_hand -> l_uhand
- joint l_arm_mwx: child l_hand -> l_uhand
- joint r_arm_lwz: child right_palm -> r_hand; parent r_hand -> r_uhand
- joint r_arm_mwx: child r_hand -> r_uhand

File: software/models/mit_gazebo_models/V1/models/V1/urdf/V1_sim_mit_drake.urdf (robot description, URDF)
Before this commit: robot V1, 92 links, 91 joints
Links:
- added link /v1/LeftMedialMetacarpal, mass 0.047; collision mesh filename=package://V1/models/V1/meshes/2013_05_16/ssf1_Left.wrl; visual mesh filename=package://V1/models/V1/meshes/2013_05_16/ssf1_Left.wrl
- added link /v1/LeftMiddleProximalPhalanx, mass 0.02; collision mesh filename=package://V1/models/V1/meshes/2013_05_16/sf1.wrl; visual mesh filename=package://V1/models/V1/meshes/2013_05_16/sf1.wrl
- added link /v1/RightMedialMetacarpal, mass 0.047; collision mesh filename=package://V1/models/V1/meshes/2013_05_16/ssf1_Right.wrl; visual mesh filename=package://V1/models/V1/meshes/2013_05_16/ssf1_Right.wrl
- added link /v1/RightMiddleProximalPhalanx, mass 0.02; collision mesh filename=package://V1/models/V1/meshes/2013_05_16/sf1.wrl; visual mesh filename=package://V1/models/V1/meshes/2013_05_16/sf1.wrl
- added link l_uhand, mass 0.1; collision box size=0.03 0.01 0.051; visual box size=0.03 0.01 0.051
- added link r_uhand, mass 0.1; collision box size=0.03 0.01 0.051; visual box size=0.03 0.01 0.051
- link l_hand: mass 0.1 -> 0.712; geometry collision mesh filename=package://V1/models/V1/meshes/2013_05_16/palm_Left.wrl; visual mesh filename=package://V1/models/V1/meshes/2013_05_16/palm_Left.wrl
- link l_hand_face: mass 0.02 -> 0.001; geometry visual box size=0.01 0.01 0.01
- link l_hand_force_torque: mass 0.047 -> 0.001; geometry visual box size=0.01 0.01 0.01
- link left_palm: mass 0.712 -> 0.001; geometry visual box size=0.01 0.01 0.01
- link r_hand: mass 0.1 -> 0.712; geometry collision mesh filename=package://V1/models/V1/meshes/2013_05_16/palm_Right.wrl; visual mesh filename=package://V1/models/V1/meshes/2013_05_16/palm_Right.wrl
- link r_hand_face: mass 0.02 -> 0.001; geometry visual box size=0.01 0.01 0.01
- link r_hand_force_torque: mass 0.047 -> 0.001; geometry visual box size=0.01 0.01 0.01
- link right_palm: mass 0.712 -> 0.001; geometry visual box size=0.01 0.01 0.01
Joints:
- added joint l_hand_face_joint: type fixed, parent l_hand_force_torque, child l_hand_face, origin xyz=0 0 0 rpy=0 0 0
- added joint l_hand_force_torque_joint: type fixed, parent l_hand, child l_hand_force_torque, origin xyz=0 0 0 rpy=0 0 0
- added joint left_valkyrie_hand_joint: type fixed, parent l_hand_force_torque, child left_palm, origin xyz=0 0 0 rpy=0 0 0
- added joint r_hand_face_joint: type fixed, parent r_hand_force_torque, child r_hand_face, origin xyz=0 0 0 rpy=0 0 0
- added joint r_hand_force_torque_joint: type fixed, parent r_hand, child r_hand_force_torque, origin xyz=0 0 0 rpy=0 0 0
- added joint right_valkyrie_hand_joint: type fixed, parent r_hand_force_torque, child right_palm, origin xyz=0 0 0 rpy=0 0 0
- joint LeftLittleMPExtensor: parent l_hand_force_torque -> /v1/LeftMedialMetacarpal
- joint LeftLittleMPYaw: child l_hand_force_torque -> /v1/LeftMedialMetacarpal
- joint LeftMiddleMPExtensor: child l_hand_face -> /v1/LeftMiddleProximalPhalanx
- joint LeftMiddlePIPExtensor: parent l_hand_face -> /v1/LeftMiddleProximalPhalanx
- joint RightLittleMPExtensor: parent r_hand_force_torque -> /v1/RightMedialMetacarpal
- joint RightLittleMPYaw: child r_hand_force_torque -> /v1/RightMedialMetacarpal
- joint RightMiddleMPExtensor: child r_hand_face -> /v1/RightMiddleProximalPhalanx
- joint RightMiddlePIPExtensor: parent r_hand_face -> /v1/RightMiddleProximalPhalanx
- joint l_arm_lwz: child left_palm -> l_hand; parent l_hand -> l_uhand
- joint l_arm_mwx: child l_hand -> l_uhand
- joint r_arm_lwz: child right_palm -> r_hand; parent r_hand -> r_uhand
- joint r_arm_mwx: child r_hand -> r_uhand

File: software/models/mit_gazebo_models/mit_robot_hands/valkyrie_hand_left.urdf (robot description, URDF)
Before this commit: robot valkyrie_hand_left, 17 links, 16 joints
Links:
- removed link l_hand_face
- removed link l_hand_force_torque
- added link /v1/LeftMedialMetacarpal, mass 0.047; collision mesh filename=package://V1/models/V1/meshes/2013_05_16/ssf1_Left.stl; visual mesh filename=package://V1/models/V1/meshes/2013_05_16/ssf1_Left.stl
- added link /v1/LeftMiddleProximalPhalanx, mass 0.02; collision mesh filename=package://V1/models/V1/meshes/2013_05_16/sf1.stl; visual mesh filename=package://V1/models/V1/meshes/2013_05_16/sf1.stl
Joints:
- joint LeftLittleMPExtensor: parent l_hand_force_torque -> /v1/LeftMedialMetacarpal
- joint LeftLittleMPYaw: child l_hand_force_torque -> /v1/LeftMedialMetacarpal
- joint LeftMiddleMPExtensor: child l_hand_face -> /v1/LeftMiddleProximalPhalanx
- joint LeftMiddlePIPExtensor: parent l_hand_face -> /v1/LeftMiddleProximalPhalanx

File: software/models/mit_gazebo_models/mit_robot_hands/valkyrie_hand_right.urdf (robot description, URDF)
Before this commit: robot valkyrie_hand_right, 17 links, 16 joints
Links:
- removed link r_hand_face
- removed link r_hand_force_torque
- added link /v1/RightMedialMetacarpal, mass 0.047; collision mesh filename=package://V1/models/V1/meshes/2013_05_16/ssf1_Right.stl; visual mesh filename=package://V1/models/V1/meshes/2013_05_16/ssf1_Right.stl
- added link /v1/RightMiddleProximalPhalanx, mass 0.02; collision mesh filename=package://V1/models/V1/meshes/2013_05_16/sf1.stl; visual mesh filename=package://V1/models/V1/meshes/2013_05_16/sf1.stl
Joints:
- joint RightLittleMPExtensor: parent r_hand_force_torque -> /v1/RightMedialMetacarpal
- joint RightLittleMPYaw: child r_hand_force_torque -> /v1/RightMedialMetacarpal
- joint RightMiddleMPExtensor: child r_hand_face -> /v1/RightMiddleProximalPhalanx
- joint RightMiddlePIPExtensor: parent r_hand_face -> /v1/RightMiddleProximalPhalanx

Commit message: making hand face match convention for robotic

File: software/models/mit_gazebo_models/V1/models/V1/urdf/V1_sim_mit.urdf (robot description, URDF)
Before this commit: robot V1, 98 links, 97 joints
Links:
- link l_hand_face: geometry 
- link r_hand_face: geometry 
Joints:
- joint l_hand_face_joint: origin xyz=0 0 0 rpy=0 0 0 -> xyz=0.08 0.0 -0.04 rpy=3.14159265359 0 1.57079632679
- joint r_hand_face_joint: origin xyz=0 0 0 rpy=0 0 0 -> xyz=0.08 0 0.04 rpy=0 0 -1.57079632679

File: software/models/mit_gazebo_models/V1/models/V1/urdf/V1_sim_mit_drake.urdf (robot description, URDF)
Before this commit: robot V1, 98 links, 97 joints
Links:
- link l_hand_face: geometry 
- link r_hand_face: geometry 
Joints:
- joint l_hand_face_joint: origin xyz=0 0 0 rpy=0 0 0 -> xyz=0.08 0.0 -0.04 rpy=3.14159265359 0 1.57079632679
- joint r_hand_face_joint: origin xyz=0 0 0 rpy=0 0 0 -> xyz=0.08 0 0.04 rpy=0 0 -1.57079632679
