Commit message: moving heel toe contact points to correct physical locations

File: software/models/mit_gazebo_models/V1/models/V1/urdf/V1_sim_mit_drake.urdf (robot description, URDF)
Before this commit: robot V1, 92 links, 91 joints
Links:
- link r_foot: geometry collision sphere radius=0; collision sphere radius=0

Commit message: fixing drake  contact points for left foot

File: software/models/mit_gazebo_models/V1/models/V1/urdf/V1_sim_mit_drake.urdf (robot description, URDF)
Before this commit: robot V1, 92 links, 91 joints
Links:
- link l_foot: geometry collision sphere radius=0; collision sphere radius=0

Commit message: Add necessary Drake frames to valkyrie URDF

File: software/models/mit_gazebo_models/V1/models/V1/urdf/V1_sim_mit_drake.urdf (robot description, URDF)
Before this commit: robot V1, 98 links, 97 joints
Links:
- link /v1/LeftLittleDistalPhalanx: geometry collision mesh filename=package://mit_drcsim_scripts/models/V1/models/V1/meshes/201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; visual mesh filename=package://mit_drcsim_scripts/models/V1/models/V1/meshes/201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
- link /v1/LeftLittleMedialPhalanx: geometry collision mesh filename=package://mit_drcsim_scripts/models/V1/models/V1/meshes/201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; visual mesh filename=package://mit_drcsim_scripts/models/V1/models/V1/meshes/201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
- link /v1/LeftLittleProximalPhalanx: geometry collision mesh filename=package://mit_drcsim_scripts/models/V1/models/V1/meshes/201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; visual mesh filename=package://mit_drcsim_scripts/models/V1/models/V1/meshes/201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
- link /v1/LeftMedialMetacarpal: geometry collision mesh filename=package://mit_drcsim_scripts/models/V1/models/V1/meshes/201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; visual mesh filename=package://mit_drcsim_scripts/models/V1/models/V1/meshes/201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
- link /v1/LeftMiddleDistalPhalanx: geometry collision mesh filename=package://mit_drcsim_scripts/models/V1/models/V1/meshes/201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; visual mesh filename=package://mit_drcsim_scripts/models/V1/models/V1/meshes/201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
- link /v1/LeftMiddleMedialPhalanx: geometry collision mesh filename=package://mit_drcsim_scripts/models/V1/models/V1/meshes/201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; visual mesh filename=package://mit_drcsim_scripts/models/V1/models/V1/meshes/201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
- link /v1/LeftMiddleProximalPhalanx: geometry collision mesh filename=package://mit_drcsim_scripts/models/V1/models/V1/meshes/201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; visual mesh filename=package://mit_drcsim_scripts/models/V1/models/V1/meshes/201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
- link /v1/LeftPrimaryDistalPhalanx: geometry collision mesh filename=package://mit_drcsim_scripts/models/V1/models/V1/meshes/201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; visual mesh filename=package://mit_drcsim_scripts/models/V1/models/V1/meshes/201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
- link /v1/LeftPrimaryMedialPhalanx: geometry collision mesh filename=package://mit_drcsim_scripts/models/V1/models/V1/meshes/201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; visual mesh filename=package://mit_drcsim_scripts/models/V1/models/V1/meshes/201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
- link /v1/LeftPrimaryMetacarpal: geometry collision mesh filename=package://mit_drcsim_scripts/models/V1/models/V1/meshes/201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; visual mesh filename=package://mit_drcsim_scripts/models/V1/models/V1/meshes/201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
- link /v1/LeftPrimaryProximalPhalanx: geometry collision mesh filename=package://mit_drcsim_scripts/models/V1/models/V1/meshes/201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; visual mesh filename=package://mit_drcsim_scripts/models/V1/models/V1/meshes/201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
- link /v1/LeftThumbDistalPhalanx: geometry collision mesh filename=package://mit_drcsim_scripts/models/V1/models/V1/meshes/201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; visual mesh filename=package://mit_drcsim_scripts/models/V1/models/V1/meshes/201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
- link /v1/LeftThumbMedialPhalanx: geometry collision mesh filename=package://mit_drcsim_scripts/models/V1/models/V1/meshes/201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; visual mesh filename=package://mit_drcsim_scripts/models/V1/models/V1/meshes/201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
- link /v1/LeftThumbMetacarpal: geometry collision mesh filename=package://mit_drcsim_scripts/models/V1/models/V1/meshes/201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; visual mesh filename=package://mit_drcsim_scripts/models/V1/models/V1/meshes/201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
- link /v1/LeftThumbProximalPhalanx: geometry collision mesh filename=package://mit_drcsim_scripts/models/V1/models/V1/meshes/201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; visual mesh filename=package://mit_drcsim_scripts/models/V1/models/V1/meshes/201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
- link /v1/RightLittleDistalPhalanx: geometry collision mesh filename=package://mit_drcsim_scripts/models/V1/models/V1/meshes/201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; visual mesh filename=package://mit_drcsim_scripts/models/V1/models/V1/meshes/201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
- link /v1/RightLittleMedialPhalanx: geometry collision mesh filename=package://mit_drcsim_scripts/models/V1/models/V1/meshes/201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; visual mesh filename=package://mit_drcsim_scripts/models/V1/models/V1/meshes/201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
- link /v1/RightLittleProximalPhalanx: geometry collision mesh filename=package://mit_drcsim_scripts/models/V1/models/V1/meshes/201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; visual mesh filename=package://mit_drcsim_scripts/models/V1/models/V1/meshes/201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
- link /v1/RightMedialMetacarpal: geometry collision mesh filename=package://mit_drcsim_scripts/models/V1/models/V1/meshes/201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; visual mesh filename=package://mit_drcsim_scripts/models/V1/models/V1/meshes/201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
- link /v1/RightMiddleDistalPhalanx: geometry collision mesh filename=package://mit_drcsim_scripts/models/V1/models/V1/meshes/201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; visual mesh filename=package://mit_drcsim_scripts/models/V1/models/V1/meshes/201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
- link /v1/RightMiddleMedialPhalanx: geometry collision mesh filename=package://mit_drcsim_scripts/models/V1/models/V1/meshes/201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; visual mesh filename=package://mit_drcsim_scripts/models/V1/models/V1/meshes/201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
- link /v1/RightMiddleProximalPhalanx: geometry collision mesh filename=package://mit_drcsim_scripts/models/V1/models/V1/meshes/201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; visual mesh filename=package://mit_drcsim_scripts/models/V1/models/V1/meshes/201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
- link /v1/RightPrimaryDistalPhalanx: geometry collision mesh filename=package://mit_drcsim_scripts/models/V1/models/V1/meshes/201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; visual mesh filename=package://mit_drcsim_scripts/models/V1/models/V1/meshes/201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
- link /v1/RightPrimaryMedialPhalanx: geometry collision mesh filename=package://mit_drcsim_scripts/models/V1/models/V1/meshes/201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; visual mesh filename=package://mit_drcsim_scripts/models/V1/models/V1/meshes/201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
- link /v1/RightPrimaryMetacarpal: geometry collision mesh filename=package://mit_drcsim_scripts/models/V1/models/V1/meshes/201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; visual mesh filename=package://mit_drcsim_scripts/models/V1/models/V1/meshes/201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
- link /v1/RightPrimaryProximalPhalanx: geometry collision mesh filename=package://mit_drcsim_scripts/models/V1/models/V1/meshes/201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; visual mesh filename=package://mit_drcsim_scripts/models/V1/models/V1/meshes/201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
- link /v1/RightThumbDistalPhalanx: geometry collision mesh filename=package://mit_drcsim_scripts/models/V1/models/V1/meshes/201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; visual mesh filename=package://mit_drcsim_scripts/models/V1/models/V1/meshes/201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
- link /v1/RightThumbMedialPhalanx: geometry collision mesh filename=package://mit_drcsim_scripts/models/V1/models/V1/meshes/201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; visual mesh filename=package://mit_drcsim_scripts/models/V1/models/V1/meshes/201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
- link /v1/RightThumbMetacarpal: geometry collision mesh filename=package://mit_drcsim_scripts/models/V1/models/V1/meshes/201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; visual mesh filename=package://mit_drcsim_scripts/models/V1/models/V1/meshes/201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
- link /v1/RightThumbProximalPhalanx: geometry collision mesh filename=package://mit_drcsim_scripts/models/V1/models/V1/meshes/201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; visual mesh filename=package://mit_drcsim_scripts/models/V1/models/V1/meshes/201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
- link head: geometry collision mesh filename=package://mit_drcsim_scripts/models/V1/models/V1/meshes/201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; visual mesh filename=package://mit_drcsim_scripts/models/V1/models/V1/meshes/201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
- link l_clav: geometry collision mesh filename=package://mit_drcsim_scripts/models/V1/models/V1/meshes/201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; visual mesh filename=package://mit_drcsim_scripts/models/V1/models/V1/meshes/201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
- link l_farm: geometry collision mesh filename=package://mit_drcsim_scripts/models/V1/models/V1/meshes/201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; visual mesh filename=package://mit_drcsim_scripts/models/V1/models/V1/meshes/201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
- link l_foot: geometry collision sphere radius=0; collision sphere radius=0
- link l_hand: geometry collision mesh filename=package://mit_drcsim_scripts/models/V1/models/V1/meshes/201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; visual mesh filename=package://mit_drcsim_scripts/models/V1/models/V1/meshes/201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
- link l_larm: geometry collision mesh filename=package://mit_drcsim_scripts/models/V1/models/V1/meshes/201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; visual mesh filename=package://mit_drcsim_scripts/models/V1/models/V1/meshes/201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
- link l_lglut: geometry collision mesh filename=package://mit_drcsim_scripts/models/V1/models/V1/meshes/201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; visual mesh filename=package://mit_drcsim_scripts/models/V1/models/V1/meshes/201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
- link l_lleg: geometry collision mesh filename=package://mit_drcsim_scripts/models/V1/models/V1/meshes/201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; visual mesh filename=package://mit_drcsim_scripts/models/V1/models/V1/meshes/201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
- link l_scap: geometry collision mesh filename=package://mit_drcsim_scripts/models/V1/models/V1/meshes/201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; visual mesh filename=package://mit_drcsim_scripts/models/V1/models/V1/meshes/201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
- link l_uarm: geometry collision mesh filename=package://mit_drcsim_scripts/models/V1/models/V1/meshes/201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; visual mesh filename=package://mit_drcsim_scripts/models/V1/models/V1/meshes/201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
- link l_uglut: geometry collision mesh filename=package://mit_drcsim_scripts/models/V1/models/V1/meshes/201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; visual mesh filename=package://mit_drcsim_scripts/models/V1/models/V1/meshes/201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
- link l_uleg: geometry collision mesh filename=package://mit_drcsim_scripts/models/V1/models/V1/meshes/201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; visual mesh filename=package://mit_drcsim_scripts/models/V1/models/V1/meshes/201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
- link mhead: geometry collision mesh filename=package://mit_drcsim_scripts/models/V1/models/V1/meshes/201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; visual mesh filename=package://mit_drcsim_scripts/models/V1/models/V1/meshes/201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
- link pelvis: geometry collision mesh filename=package://mit_drcsim_scripts/models/V1/models/V1/meshes/201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; visual mesh filename=package://mit_drcsim_scripts/models/V1/models/V1/meshes/201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
- link r_clav: geometry collision mesh filename=package://mit_drcsim_scripts/models/V1/models/V1/meshes/201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; visual mesh filename=package://mit_drcsim_scripts/models/V1/models/V1/meshes/201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
- link r_farm: geometry collision mesh filename=package://mit_drcsim_scripts/models/V1/models/V1/meshes/201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; visual mesh filename=package://mit_drcsim_scripts/models/V1/models/V1/meshes/201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
- link r_foot: geometry collision sphere radius=0; collision sphere radius=0
- link r_hand: geometry collision mesh filename=package://mit_drcsim_scripts/models/V1/models/V1/meshes/201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; visual mesh filename=package://mit_drcsim_scripts/models/V1/models/V1/meshes/201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
- link r_larm: geometry collision mesh filename=package://mit_drcsim_scripts/models/V1/models/V1/meshes/201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; visual mesh filename=package://mit_drcsim_scripts/models/V1/models/V1/meshes/201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
- link r_lglut: geometry collision mesh filename=package://mit_drcsim_scripts/models/V1/models/V1/meshes/201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; visual mesh filename=package://mit_drcsim_scripts/models/V1/models/V1/meshes/201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
- link r_lleg: geometry collision mesh filename=package://mit_drcsim_scripts/models/V1/models/V1/meshes/201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; visual mesh filename=package://mit_drcsim_scripts/models/V1/models/V1/meshes/201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
- link r_scap: geometry collision mesh filename=package://mit_drcsim_scripts/models/V1/models/V1/meshes/201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; visual mesh filename=package://mit_drcsim_scripts/models/V1/models/V1/meshes/201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
- link r_uarm: geometry collision mesh filename=package://mit_drcsim_scripts/models/V1/models/V1/meshes/201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; visual mesh filename=package://mit_drcsim_scripts/models/V1/models/V1/meshes/201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
- link r_uglut: geometry collision mesh filename=package://mit_drcsim_scripts/models/V1/models/V1/meshes/201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; visual mesh filename=package://mit_drcsim_scripts/models/V1/models/V1/meshes/201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
- link r_uleg: geometry collision mesh filename=package://mit_drcsim_scripts/models/V1/models/V1/meshes/201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; visual mesh filename=package://mit_drcsim_scripts/models/V1/models/V1/meshes/201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
- link uhead: geometry collision mesh filename=package://mit_drcsim_scripts/models/V1/models/V1/meshes/201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; visual mesh filename=package://mit_drcsim_scripts/models/V1/models/V1/meshes/201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
- link utorso: geometry collision mesh filename=package://mit_drcsim_scripts/models/V1/models/V1/meshes/201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; visual mesh filename=package://mit_drcsim_scripts/models/V1/models/V1/meshes/201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
