Commit message: Revert to package:// syntax for meshes.
This makes publishing the urdf over LCM work again.

File: software/models/common_components/multisense_sl/multisense_sl.urdf (robot description, URDF)
Before this commit: robot multisense, 24 links, 23 joints
Links:
- link head: geometry collision box size=0.1311 0.12 0.0591; visual mesh filename=package://multisense_sl/meshes/head.obj
- link hokuyo_link: geometry collision cylinder length=0.047 radius=0.024425; visual mesh filename=package://multisense_sl/meshes/head_camera.obj

File: software/models/common_components/multisense_sl/multisense_sl_convex_hull.urdf (robot description, URDF)
Before this commit: robot multisense, 24 links, 23 joints
Links:
- link head: geometry collision mesh filename=package://multisense_sl/meshes/head_chull.obj; visual mesh filename=package://multisense_sl/meshes/head_chull.obj
- link hokuyo_link: geometry collision mesh filename=package://multisense_sl/meshes/head_camera_chull.obj; visual mesh filename=package://multisense_sl/meshes/head_camera_chull.obj

File: software/models/common_components/multisense_sl/multisense_sl_no_collision.urdf (robot description, URDF)
Before this commit: robot multisense, 24 links, 23 joints
Links:
- link head: geometry visual mesh filename=package://multisense_sl/meshes/head.obj
- link hokuyo_link: geometry visual mesh filename=package://multisense_sl/meshes/head_camera.obj

File: software/models/common_components/multisense_sl/multisense_sl_no_joint.urdf (robot description, URDF)
Before this commit: robot multisense, 24 links, 23 joints
Links:
- link head: geometry collision box size=0.1311 0.12 0.0591; visual mesh filename=package://multisense_sl/meshes/head.obj
- link hokuyo_link: geometry collision cylinder length=0.047 radius=0.024425; visual mesh filename=package://multisense_sl/meshes/head_camera.obj

File: software/models/common_components/robotiq_hand_description/robotiq_hand.xacro (robot description, xacro)
@@ -10,5 +10,5 @@
         <origin rpy="0 0 0" xyz="0.020 0 0"/>
         <geometry>
-          <mesh filename="../common_components/robotiq_hand_description/meshes/s-model_articulated/visual/link_0.obj"/>
+          <mesh filename="package://robotiq_hand_description/meshes/s-model_articulated/visual/link_0.obj"/>
         </geometry>
         <material name="green">
@@ -19,5 +19,5 @@
         <origin rpy="0 3.1416 -1.57" xyz="-0.0455 0.0414 0.036"/>
         <geometry>
-          <mesh filename="../common_components/robotiq_hand_description/meshes/s-model_articulated/collision/link_0.obj"/>
+          <mesh filename="package://robotiq_hand_description/meshes/s-model_articulated/collision/link_0.obj"/>
         </geometry>
         <material name="yellow">
@@ -30,5 +30,5 @@
         <origin rpy="0 0 -0.52" xyz="0.050 -.028 0"/>
         <geometry>
-          <mesh filename="../common_components/robotiq_hand_description/meshes/s-model_articulated/visual/link_1.obj"/>
+          <mesh filename="package://robotiq_hand_description/meshes/s-model_articulated/visual/link_1.obj"/>
         </geometry>
         <material name="green"/>
@@ -37,5 +37,5 @@
         <origin rpy="0 0 -0.52" xyz="0.050 -.028 0"/>
         <geometry>
-          <mesh filename="../common_components/robotiq_hand_description/meshes/s-model_articulated/collision/link_1.obj"/>
+          <mesh filename="package://robotiq_hand_description/meshes/s-model_articulated/collision/link_1.obj"/>
         </geometry>
         <material name="yellow"/>
@@ -51,5 +51,5 @@
         <origin rpy="0 0 0" xyz="0.039 0 0.0075"/>
         <geometry>
-          <mesh filename="../common_components/robotiq_hand_description/meshes/s-model_articulated/visual/link_2.obj"/>
+          <mesh filename="package://robotiq_hand_description/meshes/s-model_articulated/visual/link_2.obj"/>
         </geometry>
         <material name="green"/>
@@ -58,5 +58,5 @@
         <origin rpy="0 0 0" xyz="0.039 0 0.0075"/>
         <geometry>
-          <mesh filename="../common_components/robotiq_hand_description/meshes/s-model_articulated/collision/link_2.obj"/>
+          <mesh filename="package://robotiq_hand_description/meshes/s-model_articulated/collision/link_2.obj"/>
         </geometry>
         <material name="yellow"/>
@@ -67,5 +67,5 @@
         <origin rpy="0 0 0.52" xyz="0 0 0"/>
         <geometry>
-          <mesh filename="../common_components/robotiq_hand_description/meshes/s-model_articulated/visual/link_3.obj"/>
+          <mesh filename="package://robotiq_hand_description/meshes/s-model_articulated/visual/link_3.obj"/>
         </geometry>
         <material name="green"/>
@@ -74,5 +74,5 @@
         <origin rpy="0 0 0.52" xyz="0 0 0"/>
         <geometry>
-          <mesh filename="../common_components/robotiq_hand_description/meshes/s-model_articulated/collision/link_3.obj"/>
+          <mesh filename="package://robotiq_hand_description/meshes/s-model_articulated/collision/link_3.obj"/>
         </geometry>
         <material name="yellow"/>
@@ -115,5 +115,5 @@
       <visual>
         <geometry>
-          <mesh filename="../common_components/robotiq_hand_description/meshes/s-model_articulated/visual/palm.obj"/>
+          <mesh filename="package://robotiq_hand_description/meshes/s-model_articulated/visual/palm.obj"/>
         </geometry>
         <material name="green">
@@ -123,5 +123,5 @@
       <collision>
         <geometry>
-          <mesh filename="../common_components/robotiq_hand_description/meshes/s-model_articulated/collision/palm.obj"/>
+          <mesh filename="package://robotiq_hand_description/meshes/s-model_articulated/collision/palm.obj"/>
         </geometry>
         <material name="yellow">

File: software/models/common_components/robotiq_hand_description/robotiq_hand_no_collision.xacro (robot description, xacro)
@@ -10,5 +10,5 @@
         <origin rpy="0 0 0" xyz="0.020 0 0"/>
         <geometry>
-          <mesh filename="../common_components/robotiq_hand_description/meshes/s-model_articulated/visual/link_0.obj"/>
+          <mesh filename="package://robotiq_hand_description/meshes/s-model_articulated/visual/link_0.obj"/>
         </geometry>
         <material name="green">
@@ -21,5 +21,5 @@
         <origin rpy="0 0 -0.52" xyz="0.050 -.028 0"/>
         <geometry>
-          <mesh filename="../common_components/robotiq_hand_description/meshes/s-model_articulated/visual/link_1.obj"/>
+          <mesh filename="package://robotiq_hand_description/meshes/s-model_articulated/visual/link_1.obj"/>
         </geometry>
         <material name="green"/>
@@ -35,5 +35,5 @@
         <origin rpy="0 0 0" xyz="0.039 0 0.0075"/>
         <geometry>
-          <mesh filename="../common_components/robotiq_hand_description/meshes/s-model_articulated/visual/link_2.obj"/>
+          <mesh filename="package://robotiq_hand_description/meshes/s-model_articulated/visual/link_2.obj"/>
         </geometry>
         <material name="green"/>
@@ -44,5 +44,5 @@
         <origin rpy="0 0 0.52" xyz="0 0 0"/>
         <geometry>
-          <mesh filename="../common_components/robotiq_hand_description/meshes/s-model_articulated/visual/link_3.obj"/>
+          <mesh filename="package://robotiq_hand_description/meshes/s-model_articulated/visual/link_3.obj"/>
         </geometry>
         <material name="green"/>
@@ -85,5 +85,5 @@
       <visual>
         <geometry>
-          <mesh filename="../common_components/robotiq_hand_description/meshes/s-model_articulated/visual/palm.obj"/>
+          <mesh filename="package://robotiq_hand_description/meshes/s-model_articulated/visual/palm.obj"/>
         </geometry>
         <material name="green">

File: software/models/common_components/robotiq_hand_description/robotiq_hand_no_joint.xacro (robot description, xacro)
@@ -10,5 +10,5 @@
         <origin rpy="0 0 0" xyz="0.020 0 0"/>
         <geometry>
-          <mesh filename="../common_components/robotiq_hand_description/meshes/s-model_articulated/visual/link_0.obj"/>
+          <mesh filename="package://robotiq_hand_description/meshes/s-model_articulated/visual/link_0.obj"/>
         </geometry>
         <material name="green">
@@ -19,5 +19,5 @@
         <origin rpy="0 3.1416 -1.57" xyz="-0.0455 0.0414 0.036"/>
         <geometry>
-          <mesh filename="../common_components/robotiq_hand_description/meshes/s-model_articulated/collision/link_0.obj"/>
+          <mesh filename="package://robotiq_hand_description/meshes/s-model_articulated/collision/link_0.obj"/>
         </geometry>
         <material name="yellow">
@@ -30,5 +30,5 @@
         <origin rpy="0 0 -0.52" xyz="0.050 -.028 0"/>
         <geometry>
-          <mesh filename="../common_components/robotiq_hand_description/meshes/s-model_articulated/visual/link_1.obj"/>
+          <mesh filename="package://robotiq_hand_description/meshes/s-model_articulated/visual/link_1.obj"/>
         </geometry>
         <material name="green"/>
@@ -37,5 +37,5 @@
         <origin rpy="0 0 -0.52" xyz="0.050 -.028 0"/>
         <geometry>
-          <mesh filename="../common_components/robotiq_hand_description/meshes/s-model_articulated/collision/link_1.obj"/>
+          <mesh filename="package://robotiq_hand_description/meshes/s-model_articulated/collision/link_1.obj"/>
         </geometry>
         <material name="yellow"/>
@@ -51,5 +51,5 @@
         <origin rpy="0 0 0" xyz="0.039 0 0.0075"/>
         <geometry>
-          <mesh filename="../common_components/robotiq_hand_description/meshes/s-model_articulated/visual/link_2.obj"/>
+          <mesh filename="package://robotiq_hand_description/meshes/s-model_articulated/visual/link_2.obj"/>
         </geometry>
         <material name="green"/>
@@ -58,5 +58,5 @@
         <origin rpy="0 0 0" xyz="0.039 0 0.0075"/>
         <geometry>
-          <mesh filename="../common_components/robotiq_hand_description/meshes/s-model_articulated/collision/link_2.obj"/>
+          <mesh filename="package://robotiq_hand_description/meshes/s-model_articulated/collision/link_2.obj"/>
         </geometry>
         <material name="yellow"/>
@@ -67,5 +67,5 @@
         <origin rpy="0 0 0.52" xyz="0 0 0"/>
         <geometry>
-          <mesh filename="../common_components/robotiq_hand_description/meshes/s-model_articulated/visual/link_3.obj"/>
+          <mesh filename="package://robotiq_hand_description/meshes/s-model_articulated/visual/link_3.obj"/>
         </geometry>
         <material name="green"/>
@@ -74,5 +74,5 @@
         <origin rpy="0 0 0.52" xyz="0 0 0"/>
         <geometry>
-          <mesh filename="../common_components/robotiq_hand_description/meshes/s-model_articulated/collision/link_3.obj"/>
+          <mesh filename="package://robotiq_hand_description/meshes/s-model_articulated/collision/link_3.obj"/>
         </geometry>
         <material name="yellow"/>
@@ -115,5 +115,5 @@
       <visual>
         <geometry>
-          <mesh filename="../common_components/robotiq_hand_description/meshes/s-model_articulated/visual/palm.obj"/>
+          <mesh filename="package://robotiq_hand_description/meshes/s-model_articulated/visual/palm.obj"/>
         </geometry>
         <material name="green">
@@ -123,5 +123,5 @@
       <collision>
         <geometry>
-          <mesh filename="../common_components/robotiq_hand_description/meshes/s-model_articulated/collision/palm.obj"/>
+          <mesh filename="package://robotiq_hand_description/meshes/s-model_articulated/collision/palm.obj"/>
         </geometry>
         <material name="yellow">
