Commit message: find and replace of meshes

File: software/models/atlas_v3/model_LR_RR.urdf (robot description, URDF)
Before this commit: robot atlas, 92 links, 91 joints
Links:
- link l_clav: geometry collision mesh filename=package://atlas_v3/meshes/l_clav.dae scale=1 1 1; visual mesh filename=package://atlas_v3/meshes/l_clav.dae scale=1 1 1
- link l_farm: geometry collision mesh filename=package://atlas_v3/meshes/l_farm.dae scale=1 1 1; visual mesh filename=package://atlas_v3/meshes/l_farm.dae scale=1 1 1
- link l_foot: geometry collision mesh filename=package://atlas_v3/meshes/l_foot.dae scale=1 1 1; visual mesh filename=package://atlas_v3/meshes/l_foot.dae scale=1 1 1
- link l_hand: geometry collision mesh filename=package://atlas_v3/meshes/l_hand.dae scale=1 1 1; visual mesh filename=package://atlas_v3/meshes/l_hand.dae scale=1 1 1
- link l_larm: geometry collision mesh filename=package://atlas_v3/meshes/l_elbow_rx.dae scale=1 1 1; visual mesh filename=package://atlas_v3/meshes/l_elbow_rx.dae scale=1 1 1
- link l_lglut: geometry collision mesh filename=package://atlas_v3/meshes/l_lglut.dae scale=1 1 1; visual mesh filename=package://atlas_v3/meshes/l_lglut.dae scale=1 1 1
- link l_lleg: geometry collision mesh filename=package://atlas_v3/meshes/l_lleg.dae scale=1 1 1; visual mesh filename=package://atlas_v3/meshes/l_lleg.dae scale=1 1 1
- link l_scap: geometry collision mesh filename=package://atlas_v3/meshes/l_sh_rx.dae scale=1 1 1; visual mesh filename=package://atlas_v3/meshes/l_sh_rx.dae scale=1 1 1
- link l_talus: geometry collision mesh filename=package://atlas_v3/meshes/l_talus.dae scale=1 1 1; visual mesh filename=package://atlas_v3/meshes/l_talus.dae scale=1 1 1
- link l_uarm: geometry collision mesh filename=package://atlas_v3/meshes/l_elbow_ry.dae scale=1 1 1; visual mesh filename=package://atlas_v3/meshes/l_elbow_ry.dae scale=1 1 1
- link l_uglut: geometry collision mesh filename=package://atlas_v3/meshes/l_uglut.dae scale=1 1 1; visual mesh filename=package://atlas_v3/meshes/l_uglut.dae scale=1 1 1
- link l_uleg: geometry collision mesh filename=package://atlas_v3/meshes/l_uleg.dae scale=1 1 1; visual mesh filename=package://atlas_v3/meshes/l_uleg.dae scale=1 1 1
- link ltorso: geometry collision mesh filename=package://atlas_v3/meshes/ltorso.dae scale=1 1 1; visual mesh filename=package://atlas_v3/meshes/ltorso.dae scale=1 1 1
- link mtorso: geometry collision mesh filename=package://atlas_v3/meshes/mtorso.dae scale=1 1 1; visual mesh filename=package://atlas_v3/meshes/mtorso.dae scale=1 1 1
- link pelvis: geometry collision mesh filename=package://atlas_v3/meshes/pelvis.dae scale=1 1 1; visual mesh filename=package://atlas_v3/meshes/pelvis.dae scale=1 1 1
- link r_clav: geometry collision mesh filename=package://atlas_v3/meshes/r_clav.dae scale=1 1 1; visual mesh filename=package://atlas_v3/meshes/r_clav.dae scale=1 1 1
- link r_farm: geometry collision mesh filename=package://atlas_v3/meshes/r_farm.dae scale=1 1 1; visual mesh filename=package://atlas_v3/meshes/r_farm.dae scale=1 1 1
- link r_foot: geometry collision mesh filename=package://atlas_v3/meshes/r_foot.dae scale=1 1 1; visual mesh filename=package://atlas_v3/meshes/r_foot.dae scale=1 1 1
- link r_hand: geometry collision mesh filename=package://atlas_v3/meshes/r_hand.dae scale=1 1 1; visual mesh filename=package://atlas_v3/meshes/r_hand.dae scale=1 1 1
- link r_larm: geometry collision mesh filename=package://atlas_v3/meshes/r_elbow_rx.dae scale=1 1 1; visual mesh filename=package://atlas_v3/meshes/r_elbow_rx.dae scale=1 1 1
- link r_lglut: geometry collision mesh filename=package://atlas_v3/meshes/r_lglut.dae scale=1 1 1; visual mesh filename=package://atlas_v3/meshes/r_lglut.dae scale=1 1 1
- link r_lleg: geometry collision mesh filename=package://atlas_v3/meshes/r_lleg.dae scale=1 1 1; visual mesh filename=package://atlas_v3/meshes/r_lleg.dae scale=1 1 1
- link r_scap: geometry collision mesh filename=package://atlas_v3/meshes/r_sh_rx.dae scale=1 1 1; visual mesh filename=package://atlas_v3/meshes/r_sh_rx.dae scale=1 1 1
- link r_talus: geometry collision mesh filename=package://atlas_v3/meshes/r_talus.dae scale=1 1 1; visual mesh filename=package://atlas_v3/meshes/r_talus.dae scale=1 1 1
- link r_uarm: geometry collision mesh filename=package://atlas_v3/meshes/r_elbow_ry.dae scale=1 1 1; visual mesh filename=package://atlas_v3/meshes/r_elbow_ry.dae scale=1 1 1
- link r_uglut: geometry collision mesh filename=package://atlas_v3/meshes/r_uglut.dae scale=1 1 1; visual mesh filename=package://atlas_v3/meshes/r_uglut.dae scale=1 1 1
- link r_uleg: geometry collision mesh filename=package://atlas_v3/meshes/r_uleg.dae scale=1 1 1; visual mesh filename=package://atlas_v3/meshes/r_uleg.dae scale=1 1 1
- link utorso: geometry collision mesh filename=package://atlas_v3/meshes/utorso.dae scale=1 1 1; collision mesh filename=package://atlas_v3/meshes/utorso_pack.dae scale=1 1 1

File: software/models/atlas_v3/model_convex_hull_robotiq_hands.urdf (robot description, URDF)
Before this commit: robot atlas, 33 links, 32 joints
Links:
- link l_clav: geometry collision mesh filename=package://atlas_v3/meshes/l_clav_chull.wrl scale=1 1 1; visual mesh filename=package://atlas_v3/meshes/l_clav_chull.wrl scale=1 1 1
- link l_farm: geometry collision mesh filename=package://atlas_v3/meshes/l_farm_chull.wrl scale=1 1 1; visual mesh filename=package://atlas_v3/meshes/l_farm_chull.wrl scale=1 1 1
- link l_foot: geometry collision mesh filename=package://atlas_v3/meshes/l_foot_chull.wrl scale=1 1 1; collision sphere radius=0
- link l_hand: geometry collision mesh filename=package://atlas_v3/meshes/l_hand_chull.wrl scale=1 1 1; visual mesh filename=package://atlas_v3/meshes/l_hand_chull.wrl scale=1 1 1
- link l_larm: geometry collision mesh filename=package://atlas_v3/meshes/l_elbow_rx_chull.wrl scale=1 1 1; visual mesh filename=package://atlas_v3/meshes/l_elbow_rx_chull.wrl scale=1 1 1
- link l_lleg: geometry collision mesh filename=package://atlas_v3/meshes/l_lleg_chull.wrl scale=1 1 1; visual mesh filename=package://atlas_v3/meshes/l_lleg_chull.wrl scale=1 1 1
- link l_robotiq_convex_hull: geometry collision mesh filename=package://atlas_v3/meshes/GRIPPER_OPEN_chull.wrl scale=1 1 1; visual mesh filename=package://atlas_v3/meshes/GRIPPER_OPEN_chull.wrl scale=1 1 1
- link l_scap: geometry collision mesh filename=package://atlas_v3/meshes/l_sh_rx_chull.wrl scale=1 1 1; visual mesh filename=package://atlas_v3/meshes/l_sh_rx_chull.wrl scale=1 1 1
- link l_uarm: geometry collision mesh filename=package://atlas_v3/meshes/l_elbow_ry_chull.wrl scale=1 1 1; visual mesh filename=package://atlas_v3/meshes/l_elbow_ry_chull.wrl scale=1 1 1
- link l_uleg: geometry collision mesh filename=package://atlas_v3/meshes/l_uleg_chull.wrl scale=1 1 1; visual mesh filename=package://atlas_v3/meshes/l_uleg_chull.wrl scale=1 1 1
- link mtorso: geometry visual mesh filename=package://atlas_v3/meshes/mtorso.wrl scale=1 1 1
- link pelvis: geometry collision mesh filename=package://atlas_v3/meshes/pelvis_chull.wrl scale=1 1 1; visual mesh filename=package://atlas_v3/meshes/pelvis_chull.wrl scale=1 1 1
- link r_clav: geometry collision mesh filename=package://atlas_v3/meshes/r_clav_chull.wrl scale=1 1 1; visual mesh filename=package://atlas_v3/meshes/r_clav_chull.wrl scale=1 1 1
- link r_farm: geometry collision mesh filename=package://atlas_v3/meshes/r_farm_chull.wrl scale=1 1 1; visual mesh filename=package://atlas_v3/meshes/r_farm_chull.wrl scale=1 1 1
- link r_foot: geometry collision mesh filename=package://atlas_v3/meshes/r_foot_chull.wrl scale=1 1 1; collision sphere radius=0
- link r_hand: geometry collision mesh filename=package://atlas_v3/meshes/r_hand_chull.wrl scale=1 1 1; visual mesh filename=package://atlas_v3/meshes/r_hand_chull.wrl scale=1 1 1
- link r_larm: geometry collision mesh filename=package://atlas_v3/meshes/r_elbow_rx_chull.wrl scale=1 1 1; visual mesh filename=package://atlas_v3/meshes/r_elbow_rx_chull.wrl scale=1 1 1
- link r_lleg: geometry collision mesh filename=package://atlas_v3/meshes/r_lleg_chull.wrl scale=1 1 1; visual mesh filename=package://atlas_v3/meshes/r_lleg_chull.wrl scale=1 1 1
- link r_robotiq_convex_hull: geometry collision mesh filename=package://atlas_v3/meshes/GRIPPER_OPEN_chull.wrl scale=1 1 1; visual mesh filename=package://atlas_v3/meshes/GRIPPER_OPEN_chull.wrl scale=1 1 1
- link r_scap: geometry collision mesh filename=package://atlas_v3/meshes/r_sh_rx_chull.wrl scale=1 1 1; visual mesh filename=package://atlas_v3/meshes/r_sh_rx_chull.wrl scale=1 1 1
- link r_uarm: geometry collision mesh filename=package://atlas_v3/meshes/r_elbow_ry_chull.wrl scale=1 1 1; visual mesh filename=package://atlas_v3/meshes/r_elbow_ry_chull.wrl scale=1 1 1
- link r_uleg: geometry collision mesh filename=package://atlas_v3/meshes/r_uleg_chull.wrl scale=1 1 1; visual mesh filename=package://atlas_v3/meshes/r_uleg_chull.wrl scale=1 1 1
- link utorso: geometry collision mesh filename=package://atlas_v3/meshes/utorso_chull.wrl scale=1 1 1; collision mesh filename=package://atlas_v3/meshes/utorso_pack_chull.wrl scale=1 1 1
