Commit message: clean up urdf and regenerate scripts for v3
- break all simlinks to ros_workspace
- remove hook description
- move irobot hand to common location
- remove sandia hand. at the least there are duplicates of it
- regenerate all v3 robots

File: software/models/atlas_v3/model_minimal_contact.urdf (robot description, URDF)
Before this commit: robot atlas, 29 links, 28 joints
Links:
- link head: geometry visual mesh filename=package://multisense_sl/meshes/head.wrl
- link l_clav: geometry visual mesh filename=package://atlas_v3/meshes/l_clav.wrl scale=1 1 1
- link l_farm: geometry visual mesh filename=package://atlas_v3/meshes/l_farm.wrl scale=1 1 1
- link l_foot: geometry collision sphere radius=0; collision sphere radius=0
- link l_hand: geometry collision sphere radius=0; collision sphere radius=0
- link l_larm: geometry visual mesh filename=package://atlas_v3/meshes/l_elbow_rx.wrl scale=1 1 1
- link l_lglut: geometry visual mesh filename=package://atlas_v3/meshes/l_lglut.wrl scale=1 1 1
- link l_lleg: geometry collision sphere radius=0; visual mesh filename=package://atlas_v3/meshes/l_lleg.wrl scale=1 1 1
- link l_scap: geometry visual mesh filename=package://atlas_v3/meshes/l_sh_rx.wrl scale=1 1 1
- link l_talus: geometry visual mesh filename=package://atlas_v3/meshes/l_talus.wrl scale=1 1 1
- link l_uarm: geometry visual mesh filename=package://atlas_v3/meshes/l_elbow_ry.wrl scale=1 1 1
- link l_uglut: geometry visual mesh filename=package://atlas_v3/meshes/l_uglut.wrl scale=1 1 1
- link l_uleg: geometry collision sphere radius=0; collision sphere radius=0
- link ltorso: geometry visual mesh filename=package://atlas_v3/meshes/ltorso.wrl scale=1 1 1
- link mtorso: geometry visual mesh filename=package://atlas_v3/meshes/mtorso.wrl scale=1 1 1
- link pelvis: geometry collision sphere radius=0; collision sphere radius=0
- link r_clav: geometry visual mesh filename=package://atlas_v3/meshes/r_clav.wrl scale=1 1 1
- link r_farm: geometry visual mesh filename=package://atlas_v3/meshes/r_farm.wrl scale=1 1 1
- link r_foot: geometry collision sphere radius=0; collision sphere radius=0
- link r_hand: geometry collision sphere radius=0; collision sphere radius=0
- link r_larm: geometry visual mesh filename=package://atlas_v3/meshes/r_elbow_rx.wrl scale=1 1 1
- link r_lglut: geometry visual mesh filename=package://atlas_v3/meshes/r_lglut.wrl scale=1 1 1
- link r_lleg: geometry collision sphere radius=0; visual mesh filename=package://atlas_v3/meshes/r_lleg.wrl scale=1 1 1
- link r_scap: geometry visual mesh filename=package://atlas_v3/meshes/r_sh_rx.wrl scale=1 1 1
- link r_talus: geometry visual mesh filename=package://atlas_v3/meshes/r_talus.wrl scale=1 1 1
- link r_uarm: geometry visual mesh filename=package://atlas_v3/meshes/r_elbow_ry.wrl scale=1 1 1
- link r_uglut: geometry visual mesh filename=package://atlas_v3/meshes/r_uglut.wrl scale=1 1 1
- link r_uleg: geometry collision sphere radius=0; collision sphere radius=0
- link utorso: geometry collision sphere radius=0; collision sphere radius=0
