Commit message: add toe frame to v3 to make simul_v3 work again

File: software/models/atlas_v3/model_LH_RH.urdf (robot description, URDF)
Before this commit: robot atlas, 52 links, 51 joints
Joints:
- joint left_camera_optical_joint: type continuous -> fixed
- joint spindle_joint: type continuous -> fixed

File: software/models/atlas_v3/model_LI_RI.urdf (robot description, URDF)
Before this commit: robot atlas, 68 links, 67 joints
Joints:
- joint left_camera_optical_joint: type continuous -> fixed
- joint spindle_joint: type continuous -> fixed

File: software/models/atlas_v3/model_LN_RN.urdf (robot description, URDF)
Before this commit: robot atlas, 50 links, 49 joints
Joints:
- joint left_camera_optical_joint: type continuous -> fixed
- joint spindle_joint: type continuous -> fixed

File: software/models/atlas_v3/model_LP_RP.urdf (robot description, URDF)
Before this commit: robot atlas, 56 links, 55 joints
Joints:
- joint left_camera_optical_joint: type continuous -> fixed
- joint spindle_joint: type continuous -> fixed

File: software/models/atlas_v3/model_LP_RR.urdf (robot description, URDF)
Before this commit: robot atlas, 70 links, 69 joints
Joints:
- joint left_camera_optical_joint: type continuous -> fixed
- joint spindle_joint: type continuous -> fixed

File: software/models/atlas_v3/model_LR_RP.urdf (robot description, URDF)
Before this commit: robot atlas, 70 links, 69 joints
Joints:
- joint left_camera_optical_joint: type continuous -> fixed
- joint spindle_joint: type continuous -> fixed

File: software/models/atlas_v3/model_LR_RR.urdf (robot description, URDF)
Before this commit: robot atlas, 84 links, 83 joints
Joints:
- joint left_camera_optical_joint: type continuous -> fixed
- joint spindle_joint: type continuous -> fixed

Commit message: reverted model_L*_R* changes

File: software/models/atlas_v3/model_LH_RH.urdf (robot description, URDF)
Before this commit: robot atlas, 52 links, 51 joints
Joints:
- joint left_camera_optical_joint: type fixed -> continuous
- joint spindle_joint: type fixed -> continuous

File: software/models/atlas_v3/model_LI_RI.urdf (robot description, URDF)
Before this commit: robot atlas, 68 links, 67 joints
Joints:
- joint left_camera_optical_joint: type fixed -> continuous
- joint spindle_joint: type fixed -> continuous

File: software/models/atlas_v3/model_LN_RN.urdf (robot description, URDF)
Before this commit: robot atlas, 50 links, 49 joints
Joints:
- joint left_camera_optical_joint: type fixed -> continuous
- joint spindle_joint: type fixed -> continuous

File: software/models/atlas_v3/model_LP_RP.urdf (robot description, URDF)
Before this commit: robot atlas, 56 links, 55 joints
Joints:
- joint left_camera_optical_joint: type fixed -> continuous
- joint spindle_joint: type fixed -> continuous

File: software/models/atlas_v3/model_LP_RR.urdf (robot description, URDF)
Before this commit: robot atlas, 70 links, 69 joints
Joints:
- joint left_camera_optical_joint: type fixed -> continuous
- joint spindle_joint: type fixed -> continuous

File: software/models/atlas_v3/model_LR_RP.urdf (robot description, URDF)
Before this commit: robot atlas, 70 links, 69 joints
Joints:
- joint left_camera_optical_joint: type fixed -> continuous
- joint spindle_joint: type fixed -> continuous

File: software/models/atlas_v3/model_LR_RR.urdf (robot description, URDF)
Before this commit: robot atlas, 84 links, 83 joints
Joints:
- joint left_camera_optical_joint: type fixed -> continuous
- joint spindle_joint: type fixed -> continuous
