Commit message: move meshes and rename urdf packages accordingly

File: software/models/valkyrie/V1_sim_mit.urdf (robot description, URDF)
Before this commit: robot V1, 98 links, 97 joints
Links:
- link head: geometry collision mesh filename=package://valkyrie/meshes/nj1.stl; visual mesh filename=package://valkyrie/meshes/nj1.stl
- link l_clav: geometry collision mesh filename=package://valkyrie/meshes/aj1_Left.stl; visual mesh filename=package://valkyrie/meshes/aj1_Left.stl
- link l_foot: geometry collision box size=0.082 0.128 0.3; visual mesh filename=package://valkyrie/meshes/lj6_Left.stl
- link l_hand: geometry collision mesh filename=package://valkyrie/meshes/palm_Left.stl; visual mesh filename=package://valkyrie/meshes/palm_Left.stl
- link l_larm: geometry collision mesh filename=package://valkyrie/meshes/aj4.stl; visual mesh filename=package://valkyrie/meshes/aj4.stl
- link l_lglut: geometry collision mesh filename=package://valkyrie/meshes/lj2.stl; visual mesh filename=package://valkyrie/meshes/lj2.stl
- link l_lleg: geometry collision mesh filename=package://valkyrie/meshes/lj4_Left.stl; visual mesh filename=package://valkyrie/meshes/lj4_Left.stl
- link l_scap: geometry collision mesh filename=package://valkyrie/meshes/aj2.stl; visual mesh filename=package://valkyrie/meshes/aj2.stl
- link l_uarm: geometry collision mesh filename=package://valkyrie/meshes/aj3_Left.stl; visual mesh filename=package://valkyrie/meshes/aj3_Left.stl
- link l_ufarm: geometry collision mesh filename=package://valkyrie/meshes/aj5_Left.stl; visual mesh filename=package://valkyrie/meshes/aj5_Left.stl
- link l_uglut: geometry collision mesh filename=package://valkyrie/meshes/lj1_Left.stl; visual mesh filename=package://valkyrie/meshes/lj1_Left.stl
- link l_uleg: geometry collision mesh filename=package://valkyrie/meshes/lj3_Left.stl; visual mesh filename=package://valkyrie/meshes/lj3_Left.stl
- link mhead: geometry collision mesh filename=package://valkyrie/meshes/nj2.stl; visual mesh filename=package://valkyrie/meshes/nj2.stl
- link pelvis: geometry collision mesh filename=package://valkyrie/meshes/pelvis.stl; visual mesh filename=package://valkyrie/meshes/pelvis.stl
- link r_clav: geometry collision mesh filename=package://valkyrie/meshes/aj1_Right.stl; visual mesh filename=package://valkyrie/meshes/aj1_Right.stl
- link r_foot: geometry collision box size=0.082 0.128 0.3; visual mesh filename=package://valkyrie/meshes/lj6_Right.stl
- link r_hand: geometry collision mesh filename=package://valkyrie/meshes/palm_Right.stl; visual mesh filename=package://valkyrie/meshes/palm_Right.stl
- link r_larm: geometry collision mesh filename=package://valkyrie/meshes/aj4.stl; visual mesh filename=package://valkyrie/meshes/aj4.stl
- link r_lglut: geometry collision mesh filename=package://valkyrie/meshes/lj2.stl; visual mesh filename=package://valkyrie/meshes/lj2.stl
- link r_lleg: geometry collision mesh filename=package://valkyrie/meshes/lj4_Right.stl; visual mesh filename=package://valkyrie/meshes/lj4_Right.stl
- link r_scap: geometry collision mesh filename=package://valkyrie/meshes/aj2.stl; visual mesh filename=package://valkyrie/meshes/aj2.stl
- link r_uarm: geometry collision mesh filename=package://valkyrie/meshes/aj3_Right.stl; visual mesh filename=package://valkyrie/meshes/aj3_Right.stl
- link r_ufarm: geometry collision mesh filename=package://valkyrie/meshes/aj5_Right.stl; visual mesh filename=package://valkyrie/meshes/aj5_Right.stl
- link r_uglut: geometry collision mesh filename=package://valkyrie/meshes/lj1_Right.stl; visual mesh filename=package://valkyrie/meshes/lj1_Right.stl
- link r_uleg: geometry collision mesh filename=package://valkyrie/meshes/lj3_Right.stl; visual mesh filename=package://valkyrie/meshes/lj3_Right.stl
- link uhead: geometry collision mesh filename=package://valkyrie/meshes/head.stl; visual mesh filename=package://valkyrie/meshes/head.stl
- link utorso: geometry collision mesh filename=package://valkyrie/meshes/wj3.stl; visual mesh filename=package://valkyrie/meshes/wj3.stl
- link v1/LeftLittleDistalPhalanx: geometry collision mesh filename=package://valkyrie/meshes/sf3_ssf4.stl; visual mesh filename=package://valkyrie/meshes/sf3_ssf4.stl
- link v1/LeftLittleMedialPhalanx: geometry collision mesh filename=package://valkyrie/meshes/sf2_ssf3.stl; visual mesh filename=package://valkyrie/meshes/sf2_ssf3.stl
- link v1/LeftLittleProximalPhalanx: geometry collision mesh filename=package://valkyrie/meshes/ssf2_Left.stl; visual mesh filename=package://valkyrie/meshes/ssf2_Left.stl
- link v1/LeftMedialMetacarpal: geometry collision mesh filename=package://valkyrie/meshes/ssf1_Left.stl; visual mesh filename=package://valkyrie/meshes/ssf1_Left.stl
- link v1/LeftMiddleDistalPhalanx: geometry collision mesh filename=package://valkyrie/meshes/sf3_ssf4.stl; visual mesh filename=package://valkyrie/meshes/sf3_ssf4.stl
- link v1/LeftMiddleMedialPhalanx: geometry collision mesh filename=package://valkyrie/meshes/sf2_ssf3.stl; visual mesh filename=package://valkyrie/meshes/sf2_ssf3.stl
- link v1/LeftMiddleProximalPhalanx: geometry collision mesh filename=package://valkyrie/meshes/sf1.stl; visual mesh filename=package://valkyrie/meshes/sf1.stl
- link v1/LeftPrimaryDistalPhalanx: geometry collision mesh filename=package://valkyrie/meshes/pf4.stl; visual mesh filename=package://valkyrie/meshes/pf4.stl
- link v1/LeftPrimaryMedialPhalanx: geometry collision mesh filename=package://valkyrie/meshes/pf3.stl; visual mesh filename=package://valkyrie/meshes/pf3.stl
- link v1/LeftPrimaryMetacarpal: geometry collision mesh filename=package://valkyrie/meshes/pf1.stl; visual mesh filename=package://valkyrie/meshes/pf1.stl
- link v1/LeftPrimaryProximalPhalanx: geometry collision mesh filename=package://valkyrie/meshes/pf2.stl; visual mesh filename=package://valkyrie/meshes/pf2.stl
- link v1/LeftThumbDistalPhalanx: geometry collision mesh filename=package://valkyrie/meshes/tf4.stl; visual mesh filename=package://valkyrie/meshes/tf4.stl
- link v1/LeftThumbMedialPhalanx: geometry collision mesh filename=package://valkyrie/meshes/tf3.stl; visual mesh filename=package://valkyrie/meshes/tf3.stl
- link v1/LeftThumbMetacarpal: geometry collision mesh filename=package://valkyrie/meshes/tf1_Left.stl; visual mesh filename=package://valkyrie/meshes/tf1_Left.stl
- link v1/LeftThumbProximalPhalanx: geometry collision mesh filename=package://valkyrie/meshes/tf2.stl; visual mesh filename=package://valkyrie/meshes/tf2.stl
- link v1/RightLittleDistalPhalanx: geometry collision mesh filename=package://valkyrie/meshes/sf3_ssf4.stl; visual mesh filename=package://valkyrie/meshes/sf3_ssf4.stl
- link v1/RightLittleMedialPhalanx: geometry collision mesh filename=package://valkyrie/meshes/sf2_ssf3.stl; visual mesh filename=package://valkyrie/meshes/sf2_ssf3.stl
- link v1/RightLittleProximalPhalanx: geometry collision mesh filename=package://valkyrie/meshes/ssf2_Right.stl; visual mesh filename=package://valkyrie/meshes/ssf2_Right.stl
- link v1/RightMedialMetacarpal: geometry collision mesh filename=package://valkyrie/meshes/ssf1_Right.stl; visual mesh filename=package://valkyrie/meshes/ssf1_Right.stl
- link v1/RightMiddleDistalPhalanx: geometry collision mesh filename=package://valkyrie/meshes/sf3_ssf4.stl; visual mesh filename=package://valkyrie/meshes/sf3_ssf4.stl
- link v1/RightMiddleMedialPhalanx: geometry collision mesh filename=package://valkyrie/meshes/sf2_ssf3.stl; visual mesh filename=package://valkyrie/meshes/sf2_ssf3.stl
- link v1/RightMiddleProximalPhalanx: geometry collision mesh filename=package://valkyrie/meshes/sf1.stl; visual mesh filename=package://valkyrie/meshes/sf1.stl
- link v1/RightPrimaryDistalPhalanx: geometry collision mesh filename=package://valkyrie/meshes/pf4.stl; visual mesh filename=package://valkyrie/meshes/pf4.stl
- link v1/RightPrimaryMedialPhalanx: geometry collision mesh filename=package://valkyrie/meshes/pf3.stl; visual mesh filename=package://valkyrie/meshes/pf3.stl
- link v1/RightPrimaryMetacarpal: geometry collision mesh filename=package://valkyrie/meshes/pf1.stl; visual mesh filename=package://valkyrie/meshes/pf1.stl
- link v1/RightPrimaryProximalPhalanx: geometry collision mesh filename=package://valkyrie/meshes/pf2.stl; visual mesh filename=package://valkyrie/meshes/pf2.stl
- link v1/RightThumbDistalPhalanx: geometry collision mesh filename=package://valkyrie/meshes/tf4.stl; visual mesh filename=package://valkyrie/meshes/tf4.stl
- link v1/RightThumbMedialPhalanx: geometry collision mesh filename=package://valkyrie/meshes/tf3.stl; visual mesh filename=package://valkyrie/meshes/tf3.stl
- link v1/RightThumbMetacarpal: geometry collision mesh filename=package://valkyrie/meshes/tf1_Right.stl; visual mesh filename=package://valkyrie/meshes/tf1_Right.stl
- link v1/RightThumbProximalPhalanx: geometry collision mesh filename=package://valkyrie/meshes/tf2.stl; visual mesh filename=package://valkyrie/meshes/tf2.stl

File: software/models/valkyrie/V1_sim_mit_drake.urdf (robot description, URDF)
Before this commit: robot V1, 98 links, 97 joints
Links:
- link head: geometry collision mesh filename=package://valkyrie/meshes/nj1.wrl; visual mesh filename=package://valkyrie/meshes/nj1.wrl
- link l_clav: geometry collision mesh filename=package://valkyrie/meshes/aj1_Left.wrl; visual mesh filename=package://valkyrie/meshes/aj1_Left.wrl
- link l_foot: geometry collision sphere radius=0; collision sphere radius=0
- link l_hand: geometry collision mesh filename=package://valkyrie/meshes/palm_Left.wrl; visual mesh filename=package://valkyrie/meshes/palm_Left.wrl
- link l_larm: geometry collision mesh filename=package://valkyrie/meshes/aj4.wrl; visual mesh filename=package://valkyrie/meshes/aj4.wrl
- link l_lglut: geometry collision mesh filename=package://valkyrie/meshes/lj2.wrl; visual mesh filename=package://valkyrie/meshes/lj2.wrl
- link l_lleg: geometry collision mesh filename=package://valkyrie/meshes/lj4_Left.wrl; visual mesh filename=package://valkyrie/meshes/lj4_Left.wrl
- link l_scap: geometry collision mesh filename=package://valkyrie/meshes/aj2.wrl; visual mesh filename=package://valkyrie/meshes/aj2.wrl
- link l_uarm: geometry collision mesh filename=package://valkyrie/meshes/aj3_Left.wrl; visual mesh filename=package://valkyrie/meshes/aj3_Left.wrl
- link l_ufarm: geometry collision mesh filename=package://valkyrie/meshes/aj5_Left.wrl; visual mesh filename=package://valkyrie/meshes/aj5_Left.wrl
- link l_uglut: geometry collision mesh filename=package://valkyrie/meshes/lj1_Left.wrl; visual mesh filename=package://valkyrie/meshes/lj1_Left.wrl
- link l_uleg: geometry collision mesh filename=package://valkyrie/meshes/lj3_Left.wrl; visual mesh filename=package://valkyrie/meshes/lj3_Left.wrl
- link mhead: geometry collision mesh filename=package://valkyrie/meshes/nj2.wrl; visual mesh filename=package://valkyrie/meshes/nj2.wrl
- link pelvis: geometry collision mesh filename=package://valkyrie/meshes/pelvis.wrl; visual mesh filename=package://valkyrie/meshes/pelvis.wrl
- link r_clav: geometry collision mesh filename=package://valkyrie/meshes/aj1_Right.wrl; visual mesh filename=package://valkyrie/meshes/aj1_Right.wrl
- link r_foot: geometry collision sphere radius=0; collision sphere radius=0
- link r_hand: geometry collision mesh filename=package://valkyrie/meshes/palm_Right.wrl; visual mesh filename=package://valkyrie/meshes/palm_Right.wrl
- link r_larm: geometry collision mesh filename=package://valkyrie/meshes/aj4.wrl; visual mesh filename=package://valkyrie/meshes/aj4.wrl
- link r_lglut: geometry collision mesh filename=package://valkyrie/meshes/lj2.wrl; visual mesh filename=package://valkyrie/meshes/lj2.wrl
- link r_lleg: geometry collision mesh filename=package://valkyrie/meshes/lj4_Right.wrl; visual mesh filename=package://valkyrie/meshes/lj4_Right.wrl
- link r_scap: geometry collision mesh filename=package://valkyrie/meshes/aj2.wrl; visual mesh filename=package://valkyrie/meshes/aj2.wrl
- link r_uarm: geometry collision mesh filename=package://valkyrie/meshes/aj3_Right.wrl; visual mesh filename=package://valkyrie/meshes/aj3_Right.wrl
- link r_ufarm: geometry collision mesh filename=package://valkyrie/meshes/aj5_Right.wrl; visual mesh filename=package://valkyrie/meshes/aj5_Right.wrl
- link r_uglut: geometry collision mesh filename=package://valkyrie/meshes/lj1_Right.wrl; visual mesh filename=package://valkyrie/meshes/lj1_Right.wrl
- link r_uleg: geometry collision mesh filename=package://valkyrie/meshes/lj3_Right.wrl; visual mesh filename=package://valkyrie/meshes/lj3_Right.wrl
- link uhead: geometry collision mesh filename=package://valkyrie/meshes/head.wrl; visual mesh filename=package://valkyrie/meshes/head.wrl
- link utorso: geometry collision mesh filename=package://valkyrie/meshes/wj3.wrl; visual mesh filename=package://valkyrie/meshes/wj3.wrl
- link v1/LeftLittleDistalPhalanx: geometry collision mesh filename=package://valkyrie/meshes/sf3_ssf4.wrl; visual mesh filename=package://valkyrie/meshes/sf3_ssf4.wrl
- link v1/LeftLittleMedialPhalanx: geometry collision mesh filename=package://valkyrie/meshes/sf2_ssf3.wrl; visual mesh filename=package://valkyrie/meshes/sf2_ssf3.wrl
- link v1/LeftLittleProximalPhalanx: geometry collision mesh filename=package://valkyrie/meshes/ssf2_Left.wrl; visual mesh filename=package://valkyrie/meshes/ssf2_Left.wrl
- link v1/LeftMedialMetacarpal: geometry collision mesh filename=package://valkyrie/meshes/ssf1_Left.wrl; visual mesh filename=package://valkyrie/meshes/ssf1_Left.wrl
- link v1/LeftMiddleDistalPhalanx: geometry collision mesh filename=package://valkyrie/meshes/sf3_ssf4.wrl; visual mesh filename=package://valkyrie/meshes/sf3_ssf4.wrl
- link v1/LeftMiddleMedialPhalanx: geometry collision mesh filename=package://valkyrie/meshes/sf2_ssf3.wrl; visual mesh filename=package://valkyrie/meshes/sf2_ssf3.wrl
- link v1/LeftMiddleProximalPhalanx: geometry collision mesh filename=package://valkyrie/meshes/sf1.wrl; visual mesh filename=package://valkyrie/meshes/sf1.wrl
- link v1/LeftPrimaryDistalPhalanx: geometry collision mesh filename=package://valkyrie/meshes/pf4.wrl; visual mesh filename=package://valkyrie/meshes/pf4.wrl
- link v1/LeftPrimaryMedialPhalanx: geometry collision mesh filename=package://valkyrie/meshes/pf3.wrl; visual mesh filename=package://valkyrie/meshes/pf3.wrl
- link v1/LeftPrimaryMetacarpal: geometry collision mesh filename=package://valkyrie/meshes/pf1.wrl; visual mesh filename=package://valkyrie/meshes/pf1.wrl
- link v1/LeftPrimaryProximalPhalanx: geometry collision mesh filename=package://valkyrie/meshes/pf2.wrl; visual mesh filename=package://valkyrie/meshes/pf2.wrl
- link v1/LeftThumbDistalPhalanx: geometry collision mesh filename=package://valkyrie/meshes/tf4.wrl; visual mesh filename=package://valkyrie/meshes/tf4.wrl
- link v1/LeftThumbMedialPhalanx: geometry collision mesh filename=package://valkyrie/meshes/tf3.wrl; visual mesh filename=package://valkyrie/meshes/tf3.wrl
- link v1/LeftThumbMetacarpal: geometry collision mesh filename=package://valkyrie/meshes/tf1_Left.wrl; visual mesh filename=package://valkyrie/meshes/tf1_Left.wrl
- link v1/LeftThumbProximalPhalanx: geometry collision mesh filename=package://valkyrie/meshes/tf2.wrl; visual mesh filename=package://valkyrie/meshes/tf2.wrl
- link v1/RightLittleDistalPhalanx: geometry collision mesh filename=package://valkyrie/meshes/sf3_ssf4.wrl; visual mesh filename=package://valkyrie/meshes/sf3_ssf4.wrl
- link v1/RightLittleMedialPhalanx: geometry collision mesh filename=package://valkyrie/meshes/sf2_ssf3.wrl; visual mesh filename=package://valkyrie/meshes/sf2_ssf3.wrl
- link v1/RightLittleProximalPhalanx: geometry collision mesh filename=package://valkyrie/meshes/ssf2_Right.wrl; visual mesh filename=package://valkyrie/meshes/ssf2_Right.wrl
- link v1/RightMedialMetacarpal: geometry collision mesh filename=package://valkyrie/meshes/ssf1_Right.wrl; visual mesh filename=package://valkyrie/meshes/ssf1_Right.wrl
- link v1/RightMiddleDistalPhalanx: geometry collision mesh filename=package://valkyrie/meshes/sf3_ssf4.wrl; visual mesh filename=package://valkyrie/meshes/sf3_ssf4.wrl
- link v1/RightMiddleMedialPhalanx: geometry collision mesh filename=package://valkyrie/meshes/sf2_ssf3.wrl; visual mesh filename=package://valkyrie/meshes/sf2_ssf3.wrl
- link v1/RightMiddleProximalPhalanx: geometry collision mesh filename=package://valkyrie/meshes/sf1.wrl; visual mesh filename=package://valkyrie/meshes/sf1.wrl
- link v1/RightPrimaryDistalPhalanx: geometry collision mesh filename=package://valkyrie/meshes/pf4.wrl; visual mesh filename=package://valkyrie/meshes/pf4.wrl
- link v1/RightPrimaryMedialPhalanx: geometry collision mesh filename=package://valkyrie/meshes/pf3.wrl; visual mesh filename=package://valkyrie/meshes/pf3.wrl
- link v1/RightPrimaryMetacarpal: geometry collision mesh filename=package://valkyrie/meshes/pf1.wrl; visual mesh filename=package://valkyrie/meshes/pf1.wrl
- link v1/RightPrimaryProximalPhalanx: geometry collision mesh filename=package://valkyrie/meshes/pf2.wrl; visual mesh filename=package://valkyrie/meshes/pf2.wrl
- link v1/RightThumbDistalPhalanx: geometry collision mesh filename=package://valkyrie/meshes/tf4.wrl; visual mesh filename=package://valkyrie/meshes/tf4.wrl
- link v1/RightThumbMedialPhalanx: geometry collision mesh filename=package://valkyrie/meshes/tf3.wrl; visual mesh filename=package://valkyrie/meshes/tf3.wrl
- link v1/RightThumbMetacarpal: geometry collision mesh filename=package://valkyrie/meshes/tf1_Right.wrl; visual mesh filename=package://valkyrie/meshes/tf1_Right.wrl
- link v1/RightThumbProximalPhalanx: geometry collision mesh filename=package://valkyrie/meshes/tf2.wrl; visual mesh filename=package://valkyrie/meshes/tf2.wrl
