Commit message: Extend joint limit as IHMC's neck is outside this range

File: software/models/valkyrie/V1_sim_shells_reduced_polygon_count_mit.urdf (robot description, URDF)
Before this commit: robot V1, 101 links, 100 joints
Joints:
- joint UpperNeckExtensor: limit lower=-0.08726646255 upper=0.78539816295 effort=26 velocity=5 -> lower=-0.15 upper=0.78539816295 effort=26 velocity=5

Commit message: fix up palm frames orientations in urdf

File: software/models/valkyrie/V1_sim_shells_reduced_polygon_count_mit.urdf (robot description, URDF)
Before this commit: robot V1, 101 links, 100 joints
Joints:
- joint left_valkyrie_hand_joint: origin xyz=0 0 0 rpy=0 0 0 -> xyz=0.08 0 0 rpy=1.57079632679 1.57079632679 0
- joint right_valkyrie_hand_joint: origin xyz=0 0 0 rpy=0 0 0 -> xyz=0.08 0 0 rpy=0 -1.57079632679 -1.57079632679

Commit message: revert to original foot link names
note that l_foot_sole and r_foot_sole remain and are needed

File: software/models/valkyrie/V1_sim_shells_reduced_polygon_count_mit.urdf (robot description, URDF)
Before this commit: robot V1, 101 links, 100 joints
Links:
- removed link l_foot
- removed link r_foot
- added link LeftUpperFoot, mass 1.888; collision box size=0.082 0.128 0.3; collision sphere radius=0.0
- added link RightUpperFoot, mass 1.888; collision box size=0.082 0.128 0.3; collision sphere radius=0.0
Joints:
- joint LeftAnkle: child l_foot -> LeftUpperFoot
- joint LeftCOP_Offset: parent l_foot -> LeftUpperFoot
- joint LeftLeg6Axis_Offset: parent l_foot -> LeftUpperFoot
- joint LeftLegHermes_Offset: parent l_foot -> LeftUpperFoot
- joint LeftMPU6000_Offset: parent l_foot -> LeftUpperFoot
- joint RightAnkle: child r_foot -> RightUpperFoot
- joint RightCOP_Offset: parent r_foot -> RightUpperFoot
- joint RightLeg6Axis_Offset: parent r_foot -> RightUpperFoot
- joint RightLegHermes_Offset: parent r_foot -> RightUpperFoot
- joint RightMPU6000_Offset: parent r_foot -> RightUpperFoot
