Commit message: Update single_valve_wall.urdf - now a generated file

File: software/control/matlab/test/single_valve_wall.urdf (robot description, URDF)
Before this commit: robot valve_wall, 2 links, 1 joints
Links:
- added link Valve_18_torus
- added link Valve_18_torus_segment_0; collision cylinder length=0.131664456 radius=0.01905; visual cylinder length=0.131664456 radius=0.01905
- added link Valve_18_torus_segment_1; collision cylinder length=0.131664456 radius=0.01905; visual cylinder length=0.131664456 radius=0.01905
- added link Valve_18_torus_segment_2; collision cylinder length=0.131664456 radius=0.01905; visual cylinder length=0.131664456 radius=0.01905
- added link Valve_18_torus_segment_3; collision cylinder length=0.131664456 radius=0.01905; visual cylinder length=0.131664456 radius=0.01905
- added link Valve_18_torus_segment_4; collision cylinder length=0.131664456 radius=0.01905; visual cylinder length=0.131664456 radius=0.01905
- added link Valve_18_torus_segment_5; collision cylinder length=0.131664456 radius=0.01905; visual cylinder length=0.131664456 radius=0.01905
- added link Valve_18_torus_segment_6; collision cylinder length=0.131664456 radius=0.01905; visual cylinder length=0.131664456 radius=0.01905
- added link Valve_18_torus_segment_7; collision cylinder length=0.131664456 radius=0.01905; visual cylinder length=0.131664456 radius=0.01905
- added link Valve_18_torus_segment_8; collision cylinder length=0.131664456 radius=0.01905; visual cylinder length=0.131664456 radius=0.01905
- added link Valve_18_torus_segment_9; collision cylinder length=0.131664456 radius=0.01905; visual cylinder length=0.131664456 radius=0.01905
- link Valve_18: geometry visual box size=.0254 .0254 .1778; visual box size=.0254 .0254 .1778
Joints:
- added joint Valve_18_torus_fixed_joint: type fixed, parent Valve_18, child Valve_18_torus, origin xyz=0 0 0 rpy=0 1.5708 0
- added joint Valve_18_torus_segment_0_joint: type fixed, parent Valve_18_torus, child Valve_18_torus_segment_0, origin xyz=0 0 0 rpy=0 0 0.0
- added joint Valve_18_torus_segment_1_joint: type fixed, parent Valve_18_torus, child Valve_18_torus_segment_1, origin xyz=0 0 0 rpy=0 0 0.62832
- added joint Valve_18_torus_segment_2_joint: type fixed, parent Valve_18_torus, child Valve_18_torus_segment_2, origin xyz=0 0 0 rpy=0 0 1.25664
- added joint Valve_18_torus_segment_3_joint: type fixed, parent Valve_18_torus, child Valve_18_torus_segment_3, origin xyz=0 0 0 rpy=0 0 1.88496
- added joint Valve_18_torus_segment_4_joint: type fixed, parent Valve_18_torus, child Valve_18_torus_segment_4, origin xyz=0 0 0 rpy=0 0 2.51328
- added joint Valve_18_torus_segment_5_joint: type fixed, parent Valve_18_torus, child Valve_18_torus_segment_5, origin xyz=0 0 0 rpy=0 0 3.1416
- added joint Valve_18_torus_segment_6_joint: type fixed, parent Valve_18_torus, child Valve_18_torus_segment_6, origin xyz=0 0 0 rpy=0 0 3.76992
- added joint Valve_18_torus_segment_7_joint: type fixed, parent Valve_18_torus, child Valve_18_torus_segment_7, origin xyz=0 0 0 rpy=0 0 4.39824
- added joint Valve_18_torus_segment_8_joint: type fixed, parent Valve_18_torus, child Valve_18_torus_segment_8, origin xyz=0 0 0 rpy=0 0 5.02656
- added joint Valve_18_torus_segment_9_joint: type fixed, parent Valve_18_torus, child Valve_18_torus_segment_9, origin xyz=0 0 0 rpy=0 0 5.65488
