Commit message: add in fixed links into lwr_pen hand

File: software/models/lwr_defs/robots/lwr_pen.urdf (robot description, URDF)
Before this commit: robot lwr, 12 links, 11 joints
Links:
- removed link lwr_arm_7_link
- added link l_hand, mass 0.2; collision cylinder length=0.05 radius=0.04; visual mesh filename=package://lwr_defs/meshes/lwr/link_7.stl
- added link l_hand_face
- added link l_hand_force_torque
- added link left_palm
Joints:
- added joint l_hand_face_joint: type fixed, parent l_hand, child l_hand_face, origin xyz=0 0 0 rpy=1.57 0 0
- added joint l_hand_force_torque_joint: type fixed, parent l_hand, child l_hand_force_torque, origin xyz=0 0 0 rpy=0 0 0
- added joint left_palm_joint: type fixed, parent l_hand, child left_palm, origin xyz=0 0 0 rpy=0 0 0
- joint lwr_arm_6_joint: child lwr_arm_7_link -> l_hand
- joint pen_base_joint: parent lwr_arm_7_link -> l_hand
- joint pen_ori_joint: parent lwr_arm_7_link -> l_hand

File: software/models/lwr_defs/robots/lwr_pen_drake.urdf (robot description, URDF)
Before this commit: robot lwr, 12 links, 11 joints
Links:
- removed link lwr_arm_7_link
- added link l_hand, mass 0.2; collision cylinder length=0.05 radius=0.04; visual mesh filename=package://lwr_defs/meshes/lwr/link_7.wrl
- added link l_hand_face
- added link l_hand_force_torque
- added link left_palm
Joints:
- added joint l_hand_face_joint: type fixed, parent l_hand, child l_hand_face, origin xyz=0 0 0 rpy=1.57 0 0
- added joint l_hand_force_torque_joint: type fixed, parent l_hand, child l_hand_force_torque, origin xyz=0 0 0 rpy=0 0 0
- added joint left_palm_joint: type fixed, parent l_hand, child left_palm, origin xyz=0 0 0 rpy=0 0 0
- joint lwr_arm_6_joint: child lwr_arm_7_link -> l_hand
- joint pen_base_joint: parent lwr_arm_7_link -> l_hand
- joint pen_ori_joint: parent lwr_arm_7_link -> l_hand

Commit message: revert the original changes to the urdf

File: software/models/lwr_defs/robots/lwr_pen.urdf (robot description, URDF)
Before this commit: robot lwr, 15 links, 14 joints
Links:
- removed link l_hand
- added link lwr_arm_7_link, mass 0.2; collision cylinder length=0.05 radius=0.04; visual mesh filename=package://lwr_defs/meshes/lwr/link_7.stl
Joints:
- joint l_hand_face_joint: parent l_hand -> lwr_arm_7_link
- joint l_hand_force_torque_joint: parent l_hand -> lwr_arm_7_link
- joint left_palm_joint: parent l_hand -> lwr_arm_7_link
- joint lwr_arm_6_joint: child l_hand -> lwr_arm_7_link
- joint pen_base_joint: parent l_hand -> lwr_arm_7_link
- joint pen_ori_joint: parent l_hand -> lwr_arm_7_link

File: software/models/lwr_defs/robots/lwr_pen_drake.urdf (robot description, URDF)
Before this commit: robot lwr, 15 links, 14 joints
Links:
- removed link l_hand
- added link lwr_arm_7_link, mass 0.2; collision cylinder length=0.05 radius=0.04; visual mesh filename=package://lwr_defs/meshes/lwr/link_7.wrl
Joints:
- joint l_hand_face_joint: parent l_hand -> lwr_arm_7_link
- joint l_hand_force_torque_joint: parent l_hand -> lwr_arm_7_link
- joint left_palm_joint: parent l_hand -> lwr_arm_7_link
- joint lwr_arm_6_joint: child l_hand -> lwr_arm_7_link
- joint pen_base_joint: parent l_hand -> lwr_arm_7_link
- joint pen_ori_joint: parent l_hand -> lwr_arm_7_link
