Commit message: removing cruft and clean ingup drake urdf

File: software/models/lwr_defs/robots/lwr_pen_robotiq.urdf (robot description, URDF)
Before this commit: robot lwr, 9 links, 8 joints
Links:
- added link l_hand_face
- added link l_hand_force_torque, mass 0.1; visual box size=0.01 0.01 0.01
- added link l_hand_gripper
- added link left_finger_1_link_0; collision mesh filename=package://robotiq_hand_description/meshes/s-model_articulat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; visual mesh filename=package://robotiq_hand_description/meshes/s-model_articulat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
- added link left_finger_1_link_1; collision mesh filename=package://robotiq_hand_description/meshes/s-model_articulat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; visual mesh filename=package://robotiq_hand_description/meshes/s-model_articulat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
- added link left_finger_1_link_2; collision mesh filename=package://robotiq_hand_description/meshes/s-model_articulat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; visual mesh filename=package://robotiq_hand_description/meshes/s-model_articulat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
- added link left_finger_1_link_3; collision mesh filename=package://robotiq_hand_description/meshes/s-model_articulat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; visual mesh filename=package://robotiq_hand_description/meshes/s-model_articulat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
- added link left_finger_2_link_0; collision mesh filename=package://robotiq_hand_description/meshes/s-model_articulat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; visual mesh filename=package://robotiq_hand_description/meshes/s-model_articulat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
- added link left_finger_2_link_1; collision mesh filename=package://robotiq_hand_description/meshes/s-model_articulat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; visual mesh filename=package://robotiq_hand_description/meshes/s-model_articulat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
- added link left_finger_2_link_2; collision mesh filename=package://robotiq_hand_description/meshes/s-model_articulat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; visual mesh filename=package://robotiq_hand_description/meshes/s-model_articulat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
- added link left_finger_2_link_3; collision mesh filename=package://robotiq_hand_description/meshes/s-model_articulat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; visual mesh filename=package://robotiq_hand_description/meshes/s-model_articulat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
- added link left_finger_middle_link_0; collision mesh filename=package://robotiq_hand_description/meshes/s-model_articulat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; visual mesh filename=package://robotiq_hand_description/meshes/s-model_articulat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
- added link left_finger_middle_link_1; collision mesh filename=package://robotiq_hand_description/meshes/s-model_articulat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; visual mesh filename=package://robotiq_hand_description/meshes/s-model_articulat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
- added link left_finger_middle_link_2; collision mesh filename=package://robotiq_hand_description/meshes/s-model_articulat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; visual mesh filename=package://robotiq_hand_description/meshes/s-model_articulat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
- added link left_finger_middle_link_3; collision mesh filename=package://robotiq_hand_description/meshes/s-model_articulat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; visual mesh filename=package://robotiq_hand_description/meshes/s-model_articulat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
- added link left_palm; collision mesh filename=package://robotiq_hand_description/meshes/s-model_articulat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; visual mesh filename=package://robotiq_hand_description/meshes/s-model_articulat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
- link lwr_arm_0_link: geometry collision mesh filename=package://lwr_defs/meshes/lwr/convex/arm_base_convex.stl; visual mesh filename=package://lwr_defs/meshes/lwr/base.stl
- link lwr_arm_1_link: geometry collision mesh filename=package://lwr_defs/meshes/lwr/convex/arm_segment_a_convex.s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; visual mesh filename=package://lwr_defs/meshes/lwr/link_1.stl
- link lwr_arm_2_link: geometry collision mesh filename=package://lwr_defs/meshes/lwr/convex/arm_segment_b_convex.s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; visual mesh filename=package://lwr_defs/meshes/lwr/link_2.stl
- link lwr_arm_3_link: geometry collision mesh filename=package://lwr_defs/meshes/lwr/convex/arm_segment_a_convex.s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; visual mesh filename=package://lwr_defs/meshes/lwr/link_3.stl
- link lwr_arm_4_link: geometry collision mesh filename=package://lwr_defs/meshes/lwr/convex/arm_segment_b_convex.s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; visual mesh filename=package://lwr_defs/meshes/lwr/link_4.stl
- link lwr_arm_5_link: geometry collision mesh filename=package://lwr_defs/meshes/lwr/convex/arm_segment_last_conve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; visual mesh filename=package://lwr_defs/meshes/lwr/link_5.stl
- link lwr_arm_6_link: geometry collision mesh filename=package://lwr_defs/meshes/lwr/convex/arm_wrist_convex.stl; visual mesh filename=package://lwr_defs/meshes/lwr/link_6.stl
- link lwr_arm_7_link: geometry collision cylinder length=0.05 radius=0.04; visual mesh filename=package://lwr_defs/meshes/lwr/link_7.stl
Joints:
- added joint l_hand_face_joint: type fixed, parent l_hand_force_torque, child l_hand_face, origin xyz=0 0.12 0 rpy=0.0 0.0 0.0
- added joint l_hand_force_torque_joint: type fixed, parent lwr_arm_7_link, child l_hand_force_torque, origin xyz=0 0 -0.015 rpy=1.57079 0 3.1416
- added joint l_hand_gripper_joint: type fixed, parent l_hand_force_torque, child l_hand_gripper, origin xyz=0 0.18 0 rpy=0.0 0.0 0.0
- added joint left_finger_1_joint_1: type revolute, parent left_finger_1_link_0, child left_finger_1_link_1, origin xyz=0.020 0 0 rpy=0 0 0, axis 0 0 1, limit lower=0 upper=3.1416 effort=100 velocity=100
- added joint left_finger_1_joint_2: type revolute, parent left_finger_1_link_1, child left_finger_1_link_2, origin xyz=0.050 -.028 0 rpy=0 0 -0.52, axis 0 0 1, limit lower=0 upper=3.1416 effort=100 velocity=100
- added joint left_finger_1_joint_3: type revolute, parent left_finger_1_link_2, child left_finger_1_link_3, origin xyz=0.039 0 0 rpy=0 0 0, axis 0 0 1, limit lower=0 upper=3.1416 effort=100 velocity=100
- added joint left_finger_2_joint_1: type revolute, parent left_finger_2_link_0, child left_finger_2_link_1, origin xyz=0.020 0 0 rpy=0 0 0, axis 0 0 1, limit lower=0 upper=3.1416 effort=100 velocity=100
- added joint left_finger_2_joint_2: type revolute, parent left_finger_2_link_1, child left_finger_2_link_2, origin xyz=0.050 -.028 0 rpy=0 0 -0.52, axis 0 0 1, limit lower=0 upper=3.1416 effort=100 velocity=100
- added joint left_finger_2_joint_3: type revolute, parent left_finger_2_link_2, child left_finger_2_link_3, origin xyz=0.039 0 0 rpy=0 0 0, axis 0 0 1, limit lower=0 upper=3.1416 effort=100 velocity=100
- added joint left_finger_middle_joint_1: type revolute, parent left_finger_middle_link_0, child left_finger_middle_link_1, origin xyz=0.020 0 0 rpy=0 0 0, axis 0 0 1, limit lower=0 upper=3.1416 effort=100 velocity=100
- added joint left_finger_middle_joint_2: type revolute, parent left_finger_middle_link_1, child left_finger_middle_link_2, origin xyz=0.050 -.028 0 rpy=0 0 -0.52, axis 0 0 1, limit lower=0 upper=3.1416 effort=100 velocity=100
- added joint left_finger_middle_joint_3: type revolute, parent left_finger_middle_link_2, child left_finger_middle_link_3, origin xyz=0.039 0 0 rpy=0 0 0, axis 0 0 1, limit lower=0 upper=3.1416 effort=100 velocity=100
- added joint left_palm_finger_1_joint: type revolute, parent left_palm, child left_finger_1_link_0, origin xyz=-0.0455 0.0214 0.036 rpy=0 3.1416 -1.57, axis 0 1 0, limit lower=-0.16 upper=0.25 effort=100 velocity=100
- added joint left_palm_finger_2_joint: type revolute, parent left_palm, child left_finger_2_link_0, origin xyz=-0.0455 0.0214 -0.036 rpy=0 3.1416 -1.57, axis 0 1 0, limit lower=-0.25 upper=0.16 effort=100 velocity=100
- added joint left_palm_finger_middle_joint: type fixed, parent left_palm, child left_finger_middle_link_0, origin xyz=0.0455 0.0214 0 rpy=0 0 1.57, axis 0 0 1
- added joint left_robotiq_hand_joint: type fixed, parent l_hand_force_torque, child left_palm, origin xyz=0 0.06566 0.0 rpy=0 -1.57079 0
