Commit message: robotiq and schunk hands are now supported on lwr
remaining todo is to resolve a teleop and floating hand issue

File: software/models/lwr_defs/robots/lwr_hand.urdf (robot description, URDF)
Before this commit: robot lwr, 21 links, 20 joints
Links:
- added link l_hand_face
- added link l_hand_force_torque, mass 0.1; visual box size=0.01 0.01 0.01
- added link l_hand_gripper
- link lwr_arm_0_link: geometry collision mesh filename=package://lwr_defs/meshes/lwr/convex/arm_base_convex.stl; visual mesh filename=package://lwr_defs/meshes/lwr/base.stl
- link lwr_arm_1_link: geometry collision mesh filename=package://lwr_defs/meshes/lwr/convex/arm_segment_a_convex.s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; visual mesh filename=package://lwr_defs/meshes/lwr/link_1.stl
- link lwr_arm_2_link: geometry collision mesh filename=package://lwr_defs/meshes/lwr/convex/arm_segment_b_convex.s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; visual mesh filename=package://lwr_defs/meshes/lwr/link_2.stl
- link lwr_arm_3_link: geometry collision mesh filename=package://lwr_defs/meshes/lwr/convex/arm_segment_a_convex.s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; visual mesh filename=package://lwr_defs/meshes/lwr/link_3.stl
- link lwr_arm_4_link: geometry collision mesh filename=package://lwr_defs/meshes/lwr/convex/arm_segment_b_convex.s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; visual mesh filename=package://lwr_defs/meshes/lwr/link_4.stl
- link lwr_arm_5_link: geometry collision mesh filename=package://lwr_defs/meshes/lwr/convex/arm_segment_last_conve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; visual mesh filename=package://lwr_defs/meshes/lwr/link_5.stl
- link lwr_arm_6_link: geometry collision mesh filename=package://lwr_defs/meshes/lwr/convex/arm_wrist_convex.stl; visual mesh filename=package://lwr_defs/meshes/lwr/link_6.stl
- link lwr_arm_7_link: geometry collision cylinder length=0.05 radius=0.04; visual mesh filename=package://lwr_defs/meshes/lwr/link_7.stl
Joints:
- added joint l_hand_face_joint: type fixed, parent l_hand_force_torque, child l_hand_face, origin xyz=0 0.12 0 rpy=0.0 0.0 0.0
- added joint l_hand_force_torque_joint: type fixed, parent lwr_arm_7_link, child l_hand_force_torque, origin xyz=0 0 -0.015 rpy=1.57079 0 -1.57079
- added joint l_hand_gripper_joint: type fixed, parent l_hand_force_torque, child l_hand_gripper, origin xyz=0 0.18 0 rpy=0.0 0.0 0.0

File: software/models/lwr_defs/robots/lwr_robotiq.urdf (robot description, URDF)
Before this commit: robot lwr, 25 links, 24 joints
Joints:
- joint l_hand_force_torque_joint: origin xyz=0 0 -0.015 rpy=1.57079 0 3.1416 -> xyz=0 0 -0.015 rpy=1.57079 0 -1.57079

Commit message: minor improvement of shunk hand reach

File: software/models/lwr_defs/robots/lwr_hand.urdf (robot description, URDF)
Before this commit: robot lwr, 24 links, 23 joints
Links:
- removed link l_hand_face
- removed link l_hand_force_torque
- removed link l_hand_gripper
- added link sdh_hand_face
- added link sdh_hand_force_torque, mass 0.1; visual box size=0.01 0.01 0.01
- added link sdh_hand_gripper
Joints:
- removed joint l_hand_face_joint
- removed joint l_hand_force_torque_joint
- removed joint l_hand_gripper_joint
- added joint sdh_hand_face_joint: type fixed, parent sdh_hand_force_torque, child sdh_hand_face, origin xyz=0 0.095 0.01 rpy=0.0 0.0 0.0
- added joint sdh_hand_force_torque_joint: type fixed, parent lwr_arm_7_link, child sdh_hand_force_torque, origin xyz=0 0 -0.015 rpy=1.57079 0 -1.57079
- added joint sdh_hand_gripper_joint: type fixed, parent sdh_hand_force_torque, child sdh_hand_gripper, origin xyz=0 0.225 0.01 rpy=0.0 0.0 0.0

Commit message: fix hand orientation

File: software/models/lwr_defs/robots/lwr_hand.urdf (robot description, URDF)
Before this commit: robot lwr, 24 links, 23 joints
Joints:
- joint sdh_palm_joint: origin (none) -> xyz=0 0 0 rpy=0.0 0.0 -1.57079

Commit message: correcting the sdh_hand_face orientations
also correcting the reachDist to match teleop panel

File: software/models/lwr_defs/robots/lwr_hand.urdf (robot description, URDF)
Before this commit: robot lwr, 24 links, 23 joints
Joints:
- joint sdh_hand_force_torque_joint: origin xyz=0 0 -0.015 rpy=1.57079 0 -1.57079 -> xyz=0 0 -0.015 rpy=1.57079 0 3.14159265
