Commit message: lwr: updated urdf table size to match real table

File: software/models/lwr_defs/robots/lwr_drake.urdf (robot description, URDF)
Before this commit: robot lwr, 9 links, 8 joints
Links:
- link base: geometry collision box size=.8 .85 0.04; visual box size=.7 .75 0.04

File: software/models/lwr_defs/robots/lwr_hand.urdf (robot description, URDF)
Before this commit: robot lwr, 24 links, 23 joints
Links:
- link base: geometry collision box size=.8 .85 0.04; visual box size=.7 .75 0.04
