Commit message: Update generated files for previous commit

File: software/models/common_components/robotiq_hand_description/robotiq_hand.xacro (robot description, xacro)
@@ -19,5 +19,5 @@
         <origin rpy="0 3.1416 -1.57" xyz="-0.0455 0.0414 0.036"/>
         <geometry>
-          <mesh filename="package://robotiq_hand_description/meshes/s-model_articulated/collision/link_0.obj"/>
+          <mesh filename="package://robotiq_hand_description/meshes/s-model_articulated/collision/link_0_chull.obj"/>
         </geometry>
         <material name="yellow">
@@ -37,5 +37,5 @@
         <origin rpy="0 0 -0.52" xyz="0.050 -.028 0"/>
         <geometry>
-          <mesh filename="package://robotiq_hand_description/meshes/s-model_articulated/collision/link_1.obj"/>
+          <mesh filename="package://robotiq_hand_description/meshes/s-model_articulated/collision/link_1_chull.obj"/>
         </geometry>
         <material name="yellow"/>
@@ -58,5 +58,5 @@
         <origin rpy="0 0 0" xyz="0.039 0 0.0075"/>
         <geometry>
-          <mesh filename="package://robotiq_hand_description/meshes/s-model_articulated/collision/link_2.obj"/>
+          <mesh filename="package://robotiq_hand_description/meshes/s-model_articulated/collision/link_2_chull.obj"/>
         </geometry>
         <material name="yellow"/>
@@ -74,5 +74,5 @@
         <origin rpy="0 0 0.52" xyz="0 0 0"/>
         <geometry>
-          <mesh filename="package://robotiq_hand_description/meshes/s-model_articulated/collision/link_3.obj"/>
+          <mesh filename="package://robotiq_hand_description/meshes/s-model_articulated/collision/link_3_chull.obj"/>
         </geometry>
         <material name="yellow"/>
@@ -123,5 +123,5 @@
       <collision>
         <geometry>
-          <mesh filename="package://robotiq_hand_description/meshes/s-model_articulated/collision/palm.obj"/>
+          <mesh filename="package://robotiq_hand_description/meshes/s-model_articulated/collision/palm_chull.obj"/>
         </geometry>
         <material name="yellow">
