Commit message: Update generated files for v4 and v5 models

File: software/models/atlas_v4/model_convex_hull.urdf (robot description, URDF)
Before this commit: robot atlas, 70 links, 69 joints
Links:
- removed link l_robotiq_convex_hull
- removed link r_robotiq_convex_hull
- added link left_palm; collision mesh filename=package://robotiq_hand_description/meshes/s-model/collision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 scale=1 1 1; visual mesh filename=package://robotiq_hand_description/meshes/s-model/visual/GR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 scale=1 1 1
- added link right_palm; collision mesh filename=package://robotiq_hand_description/meshes/s-model/collision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 scale=1 1 1; visual mesh filename=package://robotiq_hand_description/meshes/s-model/visual/GR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 scale=1 1 1
Joints:
- removed joint l_robotiq_convex_hull_joint
- removed joint r_robotiq_convex_hull_joint
- added joint left_palm_joint: type fixed, parent l_hand_force_torque, child left_palm
- added joint right_palm_joint: type fixed, parent r_hand_force_torque, child right_palm

File: software/models/atlas_v4/model_convex_hull_closed_hands.urdf (robot description, URDF)
Before this commit: robot atlas, 70 links, 69 joints
Links:
- removed link l_robotiq_convex_hull
- removed link r_robotiq_convex_hull
- added link left_palm; collision mesh filename=package://robotiq_hand_description/meshes/s-model/collision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 scale=1 1 1; visual mesh filename=package://robotiq_hand_description/meshes/s-model/visual/GR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 scale=1 1 1
- added link right_palm; collision mesh filename=package://robotiq_hand_description/meshes/s-model/collision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 scale=1 1 1; visual mesh filename=package://robotiq_hand_description/meshes/s-model/visual/GR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 scale=1 1 1
Joints:
- removed joint l_robotiq_convex_hull_joint
- removed joint r_robotiq_convex_hull_joint
- added joint left_palm_joint: type fixed, parent l_hand_force_torque, child left_palm
- added joint right_palm_joint: type fixed, parent l_hand_force_torque, child right_palm

File: software/models/atlas_v4/xacro/atlas_v4_convex_hull_closed_hands.xacro (robot description, xacro)
@@ -6,6 +6,6 @@
   <!-- Set the initial hand position and orientation by changing 'rpy' and 'xyz'
   to mach the values in your actual robot. -->
-  <xacro:robotiq_convex_hull is_left="true" is_open="0"/>
-  <xacro:robotiq_convex_hull is_left="false" is_open="0"/>
+  <xacro:robotiq_convex_hull is_left="true" is_open="0" parent="l_hand_force_torque"/>
+  <xacro:robotiq_convex_hull is_left="false" is_open="0" parent="l_hand_force_torque"/>
   <xacro:robotiq_camera  side_letter="l" reflect="1" parent="l_hand_force_torque" >
     <origin xyz="0.0  0.0 0.0" rpy="0.0 0  0.0"/>

File: software/models/atlas_v4/xacro/atlas_v4_convex_hull_open_hands.xacro (robot description, xacro)
@@ -6,6 +6,6 @@
   <!-- Set the initial hand position and orientation by changing 'rpy' and 'xyz'
   to mach the values in your actual robot. -->
-  <xacro:robotiq_convex_hull is_left="1" is_open="1"/>
-  <xacro:robotiq_convex_hull is_left="0" is_open="1"/>
+  <xacro:robotiq_convex_hull is_left="1" is_open="1" parent="l_hand_force_torque"/>
+  <xacro:robotiq_convex_hull is_left="0" is_open="1" parent="r_hand_force_torque"/>
   <xacro:robotiq_camera  side_letter="l" reflect="1" parent="l_hand_force_torque" >
     <origin xyz="0.0  0.0 0.0" rpy="0.0 0  0.0"/>

File: software/models/atlas_v5/model_LR_RR.urdf (robot description, URDF)
Before this commit: robot atlas, 86 links, 85 joints
Joints:
- joint l_hand_force_torque_joint: origin xyz=0 -0.1245 0.0112 rpy=0 0 3.141592 -> xyz=0 -0.1245 0 rpy=0 0 3.141592
- joint r_hand_force_torque_joint: origin xyz=0 -0.1245 -0.0112 rpy=0 0 3.141592 -> xyz=0 -0.1245 0 rpy=0 0 3.141592

File: software/models/atlas_v5/model_convex_hull.urdf (robot description, URDF)
Before this commit: robot atlas, 70 links, 69 joints
Links:
- removed link l_robotiq_convex_hull
- removed link r_robotiq_convex_hull
- added link left_palm; collision mesh filename=package://robotiq_hand_description/meshes/s-model/collision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 scale=1 1 1; visual mesh filename=package://robotiq_hand_description/meshes/s-model/visual/GR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 scale=1 1 1
- added link right_palm; collision mesh filename=package://robotiq_hand_description/meshes/s-model/collision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 scale=1 1 1; visual mesh filename=package://robotiq_hand_description/meshes/s-model/visual/GR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 scale=1 1 1
Joints:
- removed joint l_robotiq_convex_hull_joint
- removed joint r_robotiq_convex_hull_joint
- added joint left_palm_joint: type fixed, parent l_hand_force_torque, child left_palm
- added joint right_palm_joint: type fixed, parent r_hand_force_torque, child right_palm
- joint l_hand_force_torque_joint: origin xyz=0 -0.1245 0.0112 rpy=0 0 3.141592 -> xyz=0 -0.1245 0 rpy=0 0 3.141592
- joint r_hand_force_torque_joint: origin xyz=0 -0.1245 -0.0112 rpy=0 0 3.141592 -> xyz=0 -0.1245 0 rpy=0 0 3.141592

File: software/models/atlas_v5/model_convex_hull_closed_hands.urdf (robot description, URDF)
Before this commit: robot atlas, 70 links, 69 joints
Links:
- removed link l_robotiq_convex_hull
- removed link r_robotiq_convex_hull
- added link left_palm; collision mesh filename=package://robotiq_hand_description/meshes/s-model/collision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 scale=1 1 1; visual mesh filename=package://robotiq_hand_description/meshes/s-model/visual/GR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 scale=1 1 1
- added link right_palm; collision mesh filename=package://robotiq_hand_description/meshes/s-model/collision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 scale=1 1 1; visual mesh filename=package://robotiq_hand_description/meshes/s-model/visual/GR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 scale=1 1 1
Joints:
- removed joint l_robotiq_convex_hull_joint
- removed joint r_robotiq_convex_hull_joint
- added joint left_palm_joint: type fixed, parent l_hand_force_torque, child left_palm
- added joint right_palm_joint: type fixed, parent l_hand_force_torque, child right_palm
- joint l_hand_force_torque_joint: origin xyz=0 -0.1245 0.0112 rpy=0 0 3.141592 -> xyz=0 -0.1245 0 rpy=0 0 3.141592
- joint r_hand_force_torque_joint: origin xyz=0 -0.1245 -0.0112 rpy=0 0 3.141592 -> xyz=0 -0.1245 0 rpy=0 0 3.141592

File: software/models/atlas_v5/model_convex_hull_fingers.urdf (robot description, URDF)
Before this commit: robot atlas, 94 links, 93 joints
Joints:
- joint l_hand_force_torque_joint: origin xyz=0 -0.1245 0.0112 rpy=0 0 3.141592 -> xyz=0 -0.1245 0 rpy=0 0 3.141592
- joint r_hand_force_torque_joint: origin xyz=0 -0.1245 -0.0112 rpy=0 0 3.141592 -> xyz=0 -0.1245 0 rpy=0 0 3.141592

File: software/models/atlas_v5/model_minimal_contact.urdf (robot description, URDF)
Before this commit: robot atlas, 94 links, 93 joints
Joints:
- joint l_hand_force_torque_joint: origin xyz=0 -0.1245 0.0112 rpy=0 0 3.141592 -> xyz=0 -0.1245 0 rpy=0 0 3.141592
- joint r_hand_force_torque_joint: origin xyz=0 -0.1245 -0.0112 rpy=0 0 3.141592 -> xyz=0 -0.1245 0 rpy=0 0 3.141592

File: software/models/atlas_v5/xacro/atlas_v5_common.xacro (robot description, xacro)
@@ -1,5 +1,5 @@
 <robot xmlns:xacro="http://www.ros.org/wiki/xacro" name="atlas" >
   <xacro:include filename="../components/atlas_transmission_v5.urdf" />
-  <xacro:include filename="../../common_components/hand_force_torque.urdf" />
+  <xacro:include filename="../../common_components/hand_force_torque_v5.urdf" />
   <xacro:include filename="../../common_components/robotiq_camera/robotiq_camera.urdf.xacro" />
 </robot>

File: software/models/atlas_v5/xacro/atlas_v5_convex_hull_closed_hands.xacro (robot description, xacro)
@@ -6,6 +6,6 @@
   <!-- Set the initial hand position and orientation by changing 'rpy' and 'xyz'
   to mach the values in your actual robot. -->
-  <xacro:robotiq_convex_hull is_left="true" is_open="0"/>
-  <xacro:robotiq_convex_hull is_left="false" is_open="0"/>
+  <xacro:robotiq_convex_hull is_left="true" is_open="0" parent="l_hand_force_torque"/>
+  <xacro:robotiq_convex_hull is_left="false" is_open="0" parent="l_hand_force_torque"/>
   <xacro:robotiq_camera  side_letter="l" reflect="1" parent="l_hand_force_torque" >
     <origin xyz="0.0  0.0 0.0" rpy="0.0 0  0.0"/>

File: software/models/atlas_v5/xacro/atlas_v5_convex_hull_open_hands.xacro (robot description, xacro)
@@ -6,6 +6,6 @@
   <!-- Set the initial hand position and orientation by changing 'rpy' and 'xyz'
   to mach the values in your actual robot. -->
-  <xacro:robotiq_convex_hull is_left="1" is_open="1"/>
-  <xacro:robotiq_convex_hull is_left="0" is_open="1"/>
+  <xacro:robotiq_convex_hull is_left="1" is_open="1" parent="l_hand_force_torque"/>
+  <xacro:robotiq_convex_hull is_left="0" is_open="1" parent="r_hand_force_torque"/>
   <xacro:robotiq_camera  side_letter="l" reflect="1" parent="l_hand_force_torque" >
     <origin xyz="0.0  0.0 0.0" rpy="0.0 0  0.0"/>
