Commit message: Update atlas_v4 generated files

File: software/models/atlas_v4/model_LR_RR.urdf (robot description, URDF)
Before this commit: robot atlas, 94 links, 93 joints
Joints:
- joint left_robotiq_hand_joint: origin xyz=-0.00125 0.17 0.01 rpy=3.14159 3.14159 3.14159 -> xyz=0 0.06566 0.0 rpy=0 -1.57079 0; parent l_hand -> l_hand_force_torque
- joint right_robotiq_hand_joint: origin xyz=-0.00125 -0.17 0.01 rpy=3.14159 0 0 -> xyz=0 0.06566 0.0 rpy=0 -1.57079 0; parent r_hand -> r_hand_force_torque

File: software/models/atlas_v4/model_minimal_contact.urdf (robot description, URDF)
Before this commit: robot atlas, 94 links, 93 joints
Joints:
- joint left_robotiq_hand_joint: origin xyz=-0.00125 0.17 0.01 rpy=3.14159 3.14159 3.14159 -> xyz=0 0.06566 0.0 rpy=0 -1.57079 0; parent l_hand -> l_hand_force_torque
- joint right_robotiq_hand_joint: origin xyz=-0.00125 -0.17 0.01 rpy=3.14159 0 0 -> xyz=0 0.06566 0.0 rpy=0 -1.57079 0; parent r_hand -> r_hand_force_torque

Commit message: make the urdf and libbot cfg match
also resolved integration of the new driver

File: software/models/atlas_v4/model_LR_RR.urdf (robot description, URDF)
Before this commit: robot atlas, 96 links, 95 joints
Links:
- removed link post_spindle
- removed link post_spindle_cal_pitch
- removed link post_spindle_cal_roll
- removed link post_spindle_cal_x
- removed link post_spindle_cal_y
- removed link post_spindle_cal_z
- removed link pre_spindle
- removed link pre_spindle_cal_pitch
- removed link pre_spindle_cal_roll
- removed link pre_spindle_cal_x
- removed link pre_spindle_cal_y
- removed link pre_spindle_cal_yaw
- removed link pre_spindle_cal_z
- added link accel
- added link gyro
- added link mag
- added link motor
- added link spindle
- link hokuyo_link: geometry collision cylinder length=0.047 radius=0.024425; visual mesh filename=package://multisense_sl/meshes/head_camera.dae
Joints:
- removed joint post_spindle_cal_pitch_joint
- removed joint post_spindle_cal_roll_joint
- removed joint post_spindle_cal_x_joint
- removed joint post_spindle_cal_y_joint
- removed joint post_spindle_cal_yaw_joint
- removed joint post_spindle_cal_z_joint
- removed joint pre_spindle_cal_pitch_joint
- removed joint pre_spindle_cal_roll_joint
- removed joint pre_spindle_cal_x_joint
- removed joint pre_spindle_cal_y_joint
- removed joint pre_spindle_cal_yaw_joint
- removed joint pre_spindle_cal_z_joint
- removed joint pre_spindle_joint
- added joint accel_joint: type fixed, parent head, child accel, origin xyz=-.0475 .0302 -.00275 rpy=0 1.5707 0
- added joint gyro_joint: type fixed, parent head, child gyro, origin xyz=-.0476 .0388 -.00075 rpy=1.5707 3.14159 1.5707 
- added joint left_camera_optical_joint: type continuous, parent left_camera_optical_frame, child motor, origin xyz=0.037817599268810 -0.091862694985753 -0.008823379197658 rpy=-0.00903666 -0.00460568 -0.00953286
- added joint mag_joint: type fixed, parent head, child mag, origin xyz=-.0475 .0302 -.00275 rpy=0 1.5707 0
- added joint spindle_joint: type continuous, parent spindle, child hokuyo_link
- joint head_hokuyo_fixed_joint: origin xyz=0.03 0 0.015 rpy=0 0 0 -> xyz=-0.000160855024446 0.024008705700733 -0.000009006827089 rpy=1.57935 -1.5462 3.13304
- joint hokuyo_joint: axis 1 0 0 -> 0 0 1; child post_spindle -> spindle; origin xyz=0 0 0 rpy=0 0 0 -> xyz=0 0 0 rpy=0 0 3.14159265; parent pre_spindle_cal_yaw -> motor
- joint left_camera_optical_frame_joint: origin xyz=0 0 0 rpy=-1.5708 0.0 -1.5708 -> xyz=0 0 0 rpy=-1.57079632679 0.0 -1.57079632679

File: software/models/atlas_v5/model_LR_RR.urdf (robot description, URDF)
Before this commit: robot atlas, 96 links, 95 joints
Links:
- removed link post_spindle
- removed link post_spindle_cal_pitch
- removed link post_spindle_cal_roll
- removed link post_spindle_cal_x
- removed link post_spindle_cal_y
- removed link post_spindle_cal_z
- removed link pre_spindle
- removed link pre_spindle_cal_pitch
- removed link pre_spindle_cal_roll
- removed link pre_spindle_cal_x
- removed link pre_spindle_cal_y
- removed link pre_spindle_cal_yaw
- removed link pre_spindle_cal_z
- added link accel
- added link gyro
- added link mag
- added link motor
- added link spindle
- link hokuyo_link: geometry collision cylinder length=0.047 radius=0.024425; visual mesh filename=package://multisense_sl/meshes/head_camera.dae
Joints:
- removed joint post_spindle_cal_pitch_joint
- removed joint post_spindle_cal_roll_joint
- removed joint post_spindle_cal_x_joint
- removed joint post_spindle_cal_y_joint
- removed joint post_spindle_cal_yaw_joint
- removed joint post_spindle_cal_z_joint
- removed joint pre_spindle_cal_pitch_joint
- removed joint pre_spindle_cal_roll_joint
- removed joint pre_spindle_cal_x_joint
- removed joint pre_spindle_cal_y_joint
- removed joint pre_spindle_cal_yaw_joint
- removed joint pre_spindle_cal_z_joint
- removed joint pre_spindle_joint
- added joint accel_joint: type fixed, parent head, child accel, origin xyz=-.0475 .0302 -.00275 rpy=0 1.5707 0
- added joint gyro_joint: type fixed, parent head, child gyro, origin xyz=-.0476 .0388 -.00075 rpy=1.5707 3.14159 1.5707 
- added joint left_camera_optical_joint: type continuous, parent left_camera_optical_frame, child motor, origin xyz=0.037817599268810 -0.091862694985753 -0.008823379197658 rpy=-0.00903666 -0.00460568 -0.00953286
- added joint mag_joint: type fixed, parent head, child mag, origin xyz=-.0475 .0302 -.00275 rpy=0 1.5707 0
- added joint spindle_joint: type continuous, parent spindle, child hokuyo_link
- joint head_hokuyo_fixed_joint: origin xyz=0.03 0 0.015 rpy=0 0 0 -> xyz=-0.000160855024446 0.024008705700733 -0.000009006827089 rpy=1.57935 -1.5462 3.13304
- joint hokuyo_joint: axis 1 0 0 -> 0 0 1; child post_spindle -> spindle; origin xyz=0 0 0 rpy=0 0 0 -> xyz=0 0 0 rpy=0 0 3.14159265; parent pre_spindle_cal_yaw -> motor
- joint left_camera_optical_frame_joint: origin xyz=0 0 0 rpy=-1.5708 0.0 -1.5708 -> xyz=0 0 0 rpy=-1.57079632679 0.0 -1.57079632679

Commit message: making all files be obj

File: software/models/atlas_v4/model_LR_RR.urdf (robot description, URDF)
Before this commit: robot atlas, 88 links, 87 joints
Links:
- link hokuyo_link: geometry collision cylinder length=0.047 radius=0.024425; visual mesh filename=package://multisense_sl/meshes/head_camera.obj

File: software/models/atlas_v5/model_LR_RR.urdf (robot description, URDF)
Before this commit: robot atlas, 88 links, 87 joints
Links:
- link hokuyo_link: geometry collision cylinder length=0.047 radius=0.024425; visual mesh filename=package://multisense_sl/meshes/head_camera.obj

File: software/models/common_components/multisense_sl/multisense_sl.urdf (robot description, URDF)
Before this commit: robot multisense, 16 links, 15 joints
Links:
- link hokuyo_link: geometry collision cylinder length=0.047 radius=0.024425; visual mesh filename=package://multisense_sl/meshes/head_camera.obj

Commit message: Revert "make the urdf and libbot cfg match"

File: software/models/atlas_v4/model_LR_RR.urdf (robot description, URDF)
Before this commit: robot atlas, 88 links, 87 joints
Links:
- removed link accel
- removed link gyro
- removed link mag
- removed link motor
- removed link spindle
- added link post_spindle
- added link post_spindle_cal_pitch
- added link post_spindle_cal_roll
- added link post_spindle_cal_x
- added link post_spindle_cal_y
- added link post_spindle_cal_z
- added link pre_spindle
- added link pre_spindle_cal_pitch
- added link pre_spindle_cal_roll
- added link pre_spindle_cal_x
- added link pre_spindle_cal_y
- added link pre_spindle_cal_yaw
- added link pre_spindle_cal_z
Joints:
- removed joint accel_joint
- removed joint gyro_joint
- removed joint left_camera_optical_joint
- removed joint mag_joint
- removed joint spindle_joint
- added joint post_spindle_cal_pitch_joint: type continuous, parent post_spindle_cal_roll, child post_spindle_cal_pitch, axis 0 1 0
- added joint post_spindle_cal_roll_joint: type continuous, parent post_spindle_cal_z, child post_spindle_cal_roll, axis 1 0 0
- added joint post_spindle_cal_x_joint: type prismatic, parent post_spindle, child post_spindle_cal_x, axis 1 0 0, limit lower=-0.5 upper=0.5 effort=0.0 velocity=0.0
- added joint post_spindle_cal_y_joint: type prismatic, parent post_spindle_cal_x, child post_spindle_cal_y, axis 0 1 0, limit lower=-0.5 upper=0.5 effort=0.0 velocity=0.0
- added joint post_spindle_cal_yaw_joint: type continuous, parent post_spindle_cal_pitch, child hokuyo_link, axis 0 0 1
- added joint post_spindle_cal_z_joint: type prismatic, parent post_spindle_cal_y, child post_spindle_cal_z, axis 0 0 1, limit lower=-0.5 upper=0.5 effort=0.0 velocity=0.0
- added joint pre_spindle_cal_pitch_joint: type continuous, parent pre_spindle_cal_roll, child pre_spindle_cal_pitch, axis 0 1 0
- added joint pre_spindle_cal_roll_joint: type continuous, parent pre_spindle_cal_z, child pre_spindle_cal_roll, axis 1 0 0
- added joint pre_spindle_cal_x_joint: type prismatic, parent pre_spindle, child pre_spindle_cal_x, axis 1 0 0, limit lower=-0.5 upper=0.5 effort=0.0 velocity=0.0
- added joint pre_spindle_cal_y_joint: type prismatic, parent pre_spindle_cal_x, child pre_spindle_cal_y, axis 0 1 0, limit lower=-0.5 upper=0.5 effort=0.0 velocity=0.0
- added joint pre_spindle_cal_yaw_joint: type continuous, parent pre_spindle_cal_pitch, child pre_spindle_cal_yaw, axis 0 0 1
- added joint pre_spindle_cal_z_joint: type prismatic, parent pre_spindle_cal_y, child pre_spindle_cal_z, axis 0 0 1, limit lower=-0.5 upper=0.5 effort=0.0 velocity=0.0
- added joint pre_spindle_joint: type fixed, parent head, child pre_spindle, origin xyz=-0.0446 0 0.0880 rpy=0 0 0, axis 0 1 0
- joint head_hokuyo_fixed_joint: origin xyz=-0.000160855024446 0.024008705700733 -0.000009006827089 rpy=1.57935 -1.5462 3.13304 -> xyz=0.03 0 0.015 rpy=0 0 0
- joint hokuyo_joint: axis 0 0 1 -> 1 0 0; child spindle -> post_spindle; origin xyz=0 0 0 rpy=0 0 3.14159265 -> xyz=0 0 0 rpy=0 0 0; parent motor -> pre_spindle_cal_yaw
- joint left_camera_optical_frame_joint: origin xyz=0 0 0 rpy=-1.57079632679 0.0 -1.57079632679 -> xyz=0 0 0 rpy=-1.5708 0.0 -1.5708

File: software/models/atlas_v5/model_LR_RR.urdf (robot description, URDF)
Before this commit: robot atlas, 88 links, 87 joints
Links:
- removed link accel
- removed link gyro
- removed link mag
- removed link motor
- removed link spindle
- added link post_spindle
- added link post_spindle_cal_pitch
- added link post_spindle_cal_roll
- added link post_spindle_cal_x
- added link post_spindle_cal_y
- added link post_spindle_cal_z
- added link pre_spindle
- added link pre_spindle_cal_pitch
- added link pre_spindle_cal_roll
- added link pre_spindle_cal_x
- added link pre_spindle_cal_y
- added link pre_spindle_cal_yaw
- added link pre_spindle_cal_z
Joints:
- removed joint accel_joint
- removed joint gyro_joint
- removed joint left_camera_optical_joint
- removed joint mag_joint
- removed joint spindle_joint
- added joint post_spindle_cal_pitch_joint: type continuous, parent post_spindle_cal_roll, child post_spindle_cal_pitch, axis 0 1 0
- added joint post_spindle_cal_roll_joint: type continuous, parent post_spindle_cal_z, child post_spindle_cal_roll, axis 1 0 0
- added joint post_spindle_cal_x_joint: type prismatic, parent post_spindle, child post_spindle_cal_x, axis 1 0 0, limit lower=-0.5 upper=0.5 effort=0.0 velocity=0.0
- added joint post_spindle_cal_y_joint: type prismatic, parent post_spindle_cal_x, child post_spindle_cal_y, axis 0 1 0, limit lower=-0.5 upper=0.5 effort=0.0 velocity=0.0
- added joint post_spindle_cal_yaw_joint: type continuous, parent post_spindle_cal_pitch, child hokuyo_link, axis 0 0 1
- added joint post_spindle_cal_z_joint: type prismatic, parent post_spindle_cal_y, child post_spindle_cal_z, axis 0 0 1, limit lower=-0.5 upper=0.5 effort=0.0 velocity=0.0
- added joint pre_spindle_cal_pitch_joint: type continuous, parent pre_spindle_cal_roll, child pre_spindle_cal_pitch, axis 0 1 0
- added joint pre_spindle_cal_roll_joint: type continuous, parent pre_spindle_cal_z, child pre_spindle_cal_roll, axis 1 0 0
- added joint pre_spindle_cal_x_joint: type prismatic, parent pre_spindle, child pre_spindle_cal_x, axis 1 0 0, limit lower=-0.5 upper=0.5 effort=0.0 velocity=0.0
- added joint pre_spindle_cal_y_joint: type prismatic, parent pre_spindle_cal_x, child pre_spindle_cal_y, axis 0 1 0, limit lower=-0.5 upper=0.5 effort=0.0 velocity=0.0
- added joint pre_spindle_cal_yaw_joint: type continuous, parent pre_spindle_cal_pitch, child pre_spindle_cal_yaw, axis 0 0 1
- added joint pre_spindle_cal_z_joint: type prismatic, parent pre_spindle_cal_y, child pre_spindle_cal_z, axis 0 0 1, limit lower=-0.5 upper=0.5 effort=0.0 velocity=0.0
- added joint pre_spindle_joint: type fixed, parent head, child pre_spindle, origin xyz=-0.0446 0 0.0880 rpy=0 0 0, axis 0 1 0
- joint head_hokuyo_fixed_joint: origin xyz=-0.000160855024446 0.024008705700733 -0.000009006827089 rpy=1.57935 -1.5462 3.13304 -> xyz=0.03 0 0.015 rpy=0 0 0
- joint hokuyo_joint: axis 0 0 1 -> 1 0 0; child spindle -> post_spindle; origin xyz=0 0 0 rpy=0 0 3.14159265 -> xyz=0 0 0 rpy=0 0 0; parent motor -> pre_spindle_cal_yaw
- joint left_camera_optical_frame_joint: origin xyz=0 0 0 rpy=-1.57079632679 0.0 -1.57079632679 -> xyz=0 0 0 rpy=-1.5708 0.0 -1.5708

File: software/models/common_components/multisense_sl/multisense_sl.urdf (robot description, URDF)
Before this commit: robot multisense, 16 links, 15 joints
Links:
- removed link accel
- removed link gyro
- removed link mag
- removed link motor
- removed link spindle
- added link post_spindle
- added link post_spindle_cal_pitch
- added link post_spindle_cal_roll
- added link post_spindle_cal_x
- added link post_spindle_cal_y
- added link post_spindle_cal_z
- added link pre_spindle
- added link pre_spindle_cal_pitch
- added link pre_spindle_cal_roll
- added link pre_spindle_cal_x
- added link pre_spindle_cal_y
- added link pre_spindle_cal_yaw
- added link pre_spindle_cal_z
Joints:
- removed joint accel_joint
- removed joint gyro_joint
- removed joint left_camera_optical_joint
- removed joint mag_joint
- removed joint spindle_joint
- added joint post_spindle_cal_pitch_joint: type continuous, parent post_spindle_cal_roll, child post_spindle_cal_pitch, axis 0 1 0
- added joint post_spindle_cal_roll_joint: type continuous, parent post_spindle_cal_z, child post_spindle_cal_roll, axis 1 0 0
- added joint post_spindle_cal_x_joint: type prismatic, parent post_spindle, child post_spindle_cal_x, axis 1 0 0, limit lower=-0.5 upper=0.5 effort=0.0 velocity=0.0
- added joint post_spindle_cal_y_joint: type prismatic, parent post_spindle_cal_x, child post_spindle_cal_y, axis 0 1 0, limit lower=-0.5 upper=0.5 effort=0.0 velocity=0.0
- added joint post_spindle_cal_yaw_joint: type continuous, parent post_spindle_cal_pitch, child hokuyo_link, axis 0 0 1
- added joint post_spindle_cal_z_joint: type prismatic, parent post_spindle_cal_y, child post_spindle_cal_z, axis 0 0 1, limit lower=-0.5 upper=0.5 effort=0.0 velocity=0.0
- added joint pre_spindle_cal_pitch_joint: type continuous, parent pre_spindle_cal_roll, child pre_spindle_cal_pitch, axis 0 1 0
- added joint pre_spindle_cal_roll_joint: type continuous, parent pre_spindle_cal_z, child pre_spindle_cal_roll, axis 1 0 0
- added joint pre_spindle_cal_x_joint: type prismatic, parent pre_spindle, child pre_spindle_cal_x, axis 1 0 0, limit lower=-0.5 upper=0.5 effort=0.0 velocity=0.0
- added joint pre_spindle_cal_y_joint: type prismatic, parent pre_spindle_cal_x, child pre_spindle_cal_y, axis 0 1 0, limit lower=-0.5 upper=0.5 effort=0.0 velocity=0.0
- added joint pre_spindle_cal_yaw_joint: type continuous, parent pre_spindle_cal_pitch, child pre_spindle_cal_yaw, axis 0 0 1
- added joint pre_spindle_cal_z_joint: type prismatic, parent pre_spindle_cal_y, child pre_spindle_cal_z, axis 0 0 1, limit lower=-0.5 upper=0.5 effort=0.0 velocity=0.0
- added joint pre_spindle_joint: type fixed, parent head, child pre_spindle, origin xyz=-0.0446 0 0.0880 rpy=0 0 0, axis 0 1 0
- joint head_hokuyo_fixed_joint: origin xyz=-0.000160855024446 0.024008705700733 -0.000009006827089 rpy=1.57935 -1.5462 3.13304 -> xyz=0.03 0 0.015 rpy=0 0 0
- joint hokuyo_joint: axis 0 0 1 -> 1 0 0; child spindle -> post_spindle; origin xyz=0 0 0 rpy=0 0 3.14159265 -> xyz=0 0 0 rpy=0 0 0; parent motor -> pre_spindle_cal_yaw
- joint left_camera_optical_frame_joint: origin xyz=0 0 0 rpy=-1.57079632679 0.0 -1.57079632679 -> xyz=0 0 0 rpy=-1.5708 0.0 -1.5708

Commit message: made spindle_joint and left_camera_optical_joint fixed rather than continuous

File: software/models/atlas_v4/model_LR_RR.urdf (robot description, URDF)
Before this commit: robot atlas, 86 links, 85 joints
Joints:
- joint left_camera_optical_joint: type continuous -> fixed
- joint spindle_joint: type continuous -> fixed

File: software/models/atlas_v5/model_LR_RR.urdf (robot description, URDF)
Before this commit: robot atlas, 86 links, 85 joints
Joints:
- joint left_camera_optical_joint: type continuous -> fixed
- joint spindle_joint: type continuous -> fixed

File: software/models/common_components/multisense_sl/multisense_sl.urdf (robot description, URDF)
Before this commit: robot multisense, 16 links, 15 joints
Joints:
- joint left_camera_optical_joint: type continuous -> fixed
- joint spindle_joint: type continuous -> fixed
