Commit message: Update generated files.
Resolves #1331

File: software/models/atlas_v4/model_LR_RR.urdf (robot description, URDF)
Before this commit: robot atlas, 86 links, 85 joints
Links:
- added link left_convex_palm; collision mesh filename=package://robotiq_hand_description/meshes/s-model/collision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 scale=1 1 1
- added link right_convex_palm; collision mesh filename=package://robotiq_hand_description/meshes/s-model/collision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 scale=1 1 1
Joints:
- added joint left_convex_palm_joint: type fixed, parent l_hand_force_torque, child left_convex_palm
- added joint right_convex_palm_joint: type fixed, parent r_hand_force_torque, child right_convex_palm

File: software/models/atlas_v5/model_LR_RR.urdf (robot description, URDF)
Before this commit: robot atlas, 86 links, 85 joints
Links:
- added link left_convex_palm; collision mesh filename=package://robotiq_hand_description/meshes/s-model/collision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 scale=1 1 1
- added link right_convex_palm; collision mesh filename=package://robotiq_hand_description/meshes/s-model/collision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 scale=1 1 1
- link left_finger_1_link_0: geometry visual mesh filename=package://robotiq_hand_description/meshes/s-model_articulat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
- link left_finger_1_link_1: geometry visual mesh filename=package://robotiq_hand_description/meshes/s-model_articulat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
- link left_finger_1_link_2: geometry visual mesh filename=package://robotiq_hand_description/meshes/s-model_articulat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
- link left_finger_1_link_3: geometry visual mesh filename=package://robotiq_hand_description/meshes/s-model_articulat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
- link left_finger_2_link_0: geometry visual mesh filename=package://robotiq_hand_description/meshes/s-model_articulat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
- link left_finger_2_link_1: geometry visual mesh filename=package://robotiq_hand_description/meshes/s-model_articulat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
- link left_finger_2_link_2: geometry visual mesh filename=package://robotiq_hand_description/meshes/s-model_articulat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
- link left_finger_2_link_3: geometry visual mesh filename=package://robotiq_hand_description/meshes/s-model_articulat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
- link left_finger_middle_link_0: geometry visual mesh filename=package://robotiq_hand_description/meshes/s-model_articulat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
- link left_finger_middle_link_1: geometry visual mesh filename=package://robotiq_hand_description/meshes/s-model_articulat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
- link left_finger_middle_link_2: geometry visual mesh filename=package://robotiq_hand_description/meshes/s-model_articulat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
- link left_finger_middle_link_3: geometry visual mesh filename=package://robotiq_hand_description/meshes/s-model_articulat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
- link left_palm: geometry visual mesh filename=package://robotiq_hand_description/meshes/s-model_articulat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
- link right_finger_1_link_0: geometry visual mesh filename=package://robotiq_hand_description/meshes/s-model_articulat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
- link right_finger_1_link_1: geometry visual mesh filename=package://robotiq_hand_description/meshes/s-model_articulat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
- link right_finger_1_link_2: geometry visual mesh filename=package://robotiq_hand_description/meshes/s-model_articulat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
- link right_finger_1_link_3: geometry visual mesh filename=package://robotiq_hand_description/meshes/s-model_articulat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
- link right_finger_2_link_0: geometry visual mesh filename=package://robotiq_hand_description/meshes/s-model_articulat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
- link right_finger_2_link_1: geometry visual mesh filename=package://robotiq_hand_description/meshes/s-model_articulat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
- link right_finger_2_link_2: geometry visual mesh filename=package://robotiq_hand_description/meshes/s-model_articulat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
- link right_finger_2_link_3: geometry visual mesh filename=package://robotiq_hand_description/meshes/s-model_articulat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
- link right_finger_middle_link_0: geometry visual mesh filename=package://robotiq_hand_description/meshes/s-model_articulat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
- link right_finger_middle_link_1: geometry visual mesh filename=package://robotiq_hand_description/meshes/s-model_articulat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
- link right_finger_middle_link_2: geometry visual mesh filename=package://robotiq_hand_description/meshes/s-model_articulat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
- link right_finger_middle_link_3: geometry visual mesh filename=package://robotiq_hand_description/meshes/s-model_articulat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
- link right_palm: geometry visual mesh filename=package://robotiq_hand_description/meshes/s-model_articulat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
Joints:
- added joint left_convex_palm_joint: type fixed, parent l_hand_force_torque, child left_convex_palm
- added joint right_convex_palm_joint: type fixed, parent r_hand_force_torque, child right_convex_palm

File: software/models/common_components/robotiq_hand_description/robotiq_hand_no_joint_no_collision.xacro (robot description, xacro)
@@ -52,5 +52,5 @@
     <!-- joint list -->
     <!-- WARNING: LIMITS NOT CORRECT -->
-    <joint name="${prefix}joint_1" type="revolute">
+    <joint name="${prefix}joint_1" type="fixed">
       <parent link="${prefix}link_0"/>
       <child link="${prefix}link_1"/>
@@ -60,5 +60,5 @@
     </joint>
     <!-- WARNING: LIMITS NOT CORRECT -->
-    <joint name="${prefix}joint_2" type="revolute">
+    <joint name="${prefix}joint_2" type="fixed">
       <parent link="${prefix}link_1"/>
       <child link="${prefix}link_2"/>
@@ -68,5 +68,5 @@
     </joint>
     <!-- WARNING: LIMITS NOT CORRECT -->
-    <joint name="${prefix}joint_3" type="revolute">
+    <joint name="${prefix}joint_3" type="fixed">
       <parent link="${prefix}link_2"/>
       <child link="${prefix}link_3"/>
@@ -95,5 +95,5 @@
     <!-- joint list -->
     <!-- WARNING: LIMITS NOT CORRECT -->
-    <joint name="${prefix}palm_finger_1_joint" type="revolute">
+    <joint name="${prefix}palm_finger_1_joint" type="fixed">
       <parent link="${prefix}palm"/>
       <child link="${prefix}finger_1_link_0"/>
@@ -103,5 +103,5 @@
     </joint>
     <!-- WARNING: LIMITS NOT CORRECT -->
-    <joint name="${prefix}palm_finger_2_joint" type="revolute">
+    <joint name="${prefix}palm_finger_2_joint" type="fixed">
       <parent link="${prefix}palm"/>
       <child link="${prefix}finger_2_link_0"/>
