Commit message: Rotate hands to match our usual placement

File: software/models/atlas_v4/xacro/atlas_v4_LR_RR.xacro (robot description, xacro)
@@ -4,11 +4,9 @@
   <xacro:include filename="./atlas_v4_common.xacro" />
   <xacro:include filename="../../common_components/robotiq_hand_description/robotiq_hand.xacro" />
-  <!-- Set the initial hand position and orientation by changing 'rpy' and 'xyz'
-  to mach the values in your actual robot. -->
-  <xacro:robotiq_hand side="left" parent="l_hand" reflect="-1">
-    <origin rpy="3.14159 3.14159 3.14159" xyz="-0.00125 0.17 0.01"/>
+  <xacro:robotiq_hand side="left" parent="l_hand_force_torque" reflect="1">
+    <origin rpy="0 -1.57079 0" xyz="0 0.06566 0.0"/>
   </xacro:robotiq_hand>
-  <xacro:robotiq_hand side="right" parent="r_hand" reflect="1">
-    <origin rpy="3.14159 0 0" xyz="-0.00125 -0.17 0.01"/>
+  <xacro:robotiq_hand side="right" parent="r_hand_force_torque" reflect="1">
+    <origin rpy="0 -1.57079 0" xyz="0 0.06566 0.0"/>
   </xacro:robotiq_hand>
   <xacro:robotiq_camera  side_letter="l" reflect="1" parent="l_hand_force_torque" >

File: software/models/atlas_v4/xacro/atlas_v4_minimal_contact.xacro (robot description, xacro)
@@ -6,9 +6,9 @@
   <!-- Set the initial hand position and orientation by changing 'rpy' and 'xyz'
   to mach the values in your actual robot. -->
-  <xacro:robotiq_hand side="left" parent="l_hand" reflect="-1">
-    <origin rpy="3.14159 3.14159 3.14159" xyz="-0.00125 0.17 0.01"/>
+  <xacro:robotiq_hand side="left" parent="l_hand_force_torque" reflect="1">
+    <origin rpy="0 -1.57079 0" xyz="0 0.06566 0.0"/>
   </xacro:robotiq_hand>
-  <xacro:robotiq_hand side="right" parent="r_hand" reflect="1">
-    <origin rpy="3.14159 0 0" xyz="-0.00125 -0.17 0.01"/>
+  <xacro:robotiq_hand side="right" parent="r_hand_force_torque" reflect="1">
+    <origin rpy="0 -1.57079 0" xyz="0 0.06566 0.0"/>
   </xacro:robotiq_hand>
   <xacro:robotiq_camera  side_letter="l" reflect="1" parent="l_hand_force_torque" >

Commit message: Use "oven-mitt" collision geom in model_LR_RR

File: software/models/atlas_v4/xacro/atlas_v4_LR_RR.xacro (robot description, xacro)
@@ -4,4 +4,5 @@
   <xacro:include filename="./atlas_v4_common.xacro" />
   <xacro:include filename="../../common_components/robotiq_hand_description/robotiq_hand.xacro" />
+  <xacro:include filename="../../common_components/robotiq_hand_description/robotiq_hand_convex_hull.xacro" />
   <xacro:robotiq_hand side="left" parent="l_hand_force_torque" reflect="1">
     <origin rpy="0 -1.57079 0" xyz="0 0.06566 0.0"/>
@@ -10,4 +11,6 @@
     <origin rpy="0 -1.57079 0" xyz="0 0.06566 0.0"/>
   </xacro:robotiq_hand>
+  <xacro:robotiq_convex_hull side="left_convex"  is_open="1" use_visuals="0" parent="l_hand_force_torque"/>
+  <xacro:robotiq_convex_hull side="right_convex" is_open="1" use_visuals="0" parent="r_hand_force_torque"/>
   <xacro:robotiq_camera  side_letter="l" reflect="1" parent="l_hand_force_torque" >
     <origin xyz="0.0  0.0 0.0" rpy="0.0 0  0.0"/>

File: software/models/atlas_v4/xacro/atlas_v4_convex_hull_closed_hands.xacro (robot description, xacro)
@@ -6,6 +6,6 @@
   <!-- Set the initial hand position and orientation by changing 'rpy' and 'xyz'
   to mach the values in your actual robot. -->
-  <xacro:robotiq_convex_hull is_left="true" is_open="0" parent="l_hand_force_torque"/>
-  <xacro:robotiq_convex_hull is_left="false" is_open="0" parent="l_hand_force_torque"/>
+  <xacro:robotiq_convex_hull side="left"  is_open="0" use_visuals="1" parent="l_hand_force_torque"/>
+  <xacro:robotiq_convex_hull side="right" is_open="0" use_visuals="1" parent="l_hand_force_torque"/>
   <xacro:robotiq_camera  side_letter="l" reflect="1" parent="l_hand_force_torque" >
     <origin xyz="0.0  0.0 0.0" rpy="0.0 0  0.0"/>

File: software/models/atlas_v4/xacro/atlas_v4_convex_hull_open_hands.xacro (robot description, xacro)
@@ -6,6 +6,6 @@
   <!-- Set the initial hand position and orientation by changing 'rpy' and 'xyz'
   to mach the values in your actual robot. -->
-  <xacro:robotiq_convex_hull is_left="1" is_open="1" parent="l_hand_force_torque"/>
-  <xacro:robotiq_convex_hull is_left="0" is_open="1" parent="r_hand_force_torque"/>
+  <xacro:robotiq_convex_hull side="left"  is_open="1" use_visuals="1" parent="l_hand_force_torque"/>
+  <xacro:robotiq_convex_hull side="right" is_open="1" use_visuals="1" parent="r_hand_force_torque"/>
   <xacro:robotiq_camera  side_letter="l" reflect="1" parent="l_hand_force_torque" >
     <origin xyz="0.0  0.0 0.0" rpy="0.0 0  0.0"/>

File: software/models/atlas_v4/xacro/atlas_v4_minimal_contact.xacro (robot description, xacro)
@@ -3,5 +3,5 @@
   <xacro:include filename="../../common_components/multisense_sl/multisense_sl_no_collision.urdf" />
   <xacro:include filename="./atlas_v4_common.xacro" />
-  <xacro:include filename="../../common_components/robotiq_hand_description/robotiq_hand_no_collision.xacro" />
+  <xacro:include filename="../../common_components/robotiq_hand_description/robotiq_hand_no_joint_no_collision.xacro" />
   <!-- Set the initial hand position and orientation by changing 'rpy' and 'xyz'
   to mach the values in your actual robot. -->

File: software/models/atlas_v5/xacro/atlas_v5_LR_RR.xacro (robot description, xacro)
@@ -3,11 +3,14 @@
   <xacro:include filename="../../common_components/multisense_sl/multisense_sl.urdf" />
   <xacro:include filename="./atlas_v5_common.xacro" />
-  <xacro:include filename="../../common_components/robotiq_hand_description/robotiq_hand.xacro" />
+  <xacro:include filename="../../common_components/robotiq_hand_description/robotiq_hand_no_collision.xacro" />
+  <xacro:include filename="../../common_components/robotiq_hand_description/robotiq_hand_convex_hull.xacro" />
   <xacro:robotiq_hand side="left" parent="l_hand_force_torque" reflect="1">
     <origin rpy="0 -1.57079 0" xyz="0 0.06566 0.0"/>
   </xacro:robotiq_hand>
-  <xacro:robotiq_hand side="right" parent="r_hand_force_torque" reflect="1">
+  <xacro:robotiq_hand side="right" parent="r_hand_force_torque" reflect="2">
     <origin rpy="0 -1.57079 0" xyz="0 0.06566 0.0"/>
   </xacro:robotiq_hand>
+  <xacro:robotiq_convex_hull side="left_convex"  is_open="1" use_visuals="0" parent="l_hand_force_torque"/>
+  <xacro:robotiq_convex_hull side="right_convex" is_open="1" use_visuals="0" parent="r_hand_force_torque"/>
   <xacro:robotiq_camera  side_letter="l" reflect="1" parent="l_hand_force_torque" >
     <origin xyz="0.0  0.0 0.0" rpy="0.0 0  0.0"/>

File: software/models/atlas_v5/xacro/atlas_v5_convex_hull_closed_hands.xacro (robot description, xacro)
@@ -6,6 +6,6 @@
   <!-- Set the initial hand position and orientation by changing 'rpy' and 'xyz'
   to mach the values in your actual robot. -->
-  <xacro:robotiq_convex_hull is_left="true" is_open="0" parent="l_hand_force_torque"/>
-  <xacro:robotiq_convex_hull is_left="false" is_open="0" parent="l_hand_force_torque"/>
+  <xacro:robotiq_convex_hull side="left"  is_open="0" use_visuals="1" parent="l_hand_force_torque"/>
+  <xacro:robotiq_convex_hull side="right" is_open="0" use_visuals="1" parent="l_hand_force_torque"/>
   <xacro:robotiq_camera  side_letter="l" reflect="1" parent="l_hand_force_torque" >
     <origin xyz="0.0  0.0 0.0" rpy="0.0 0  0.0"/>

File: software/models/atlas_v5/xacro/atlas_v5_convex_hull_open_hands.xacro (robot description, xacro)
@@ -6,6 +6,6 @@
   <!-- Set the initial hand position and orientation by changing 'rpy' and 'xyz'
   to mach the values in your actual robot. -->
-  <xacro:robotiq_convex_hull is_left="1" is_open="1" parent="l_hand_force_torque"/>
-  <xacro:robotiq_convex_hull is_left="0" is_open="1" parent="r_hand_force_torque"/>
+  <xacro:robotiq_convex_hull side="left"  is_open="1" use_visuals="1" parent="l_hand_force_torque"/>
+  <xacro:robotiq_convex_hull side="right" is_open="1" use_visuals="1" parent="r_hand_force_torque"/>
   <xacro:robotiq_camera  side_letter="l" reflect="1" parent="l_hand_force_torque" >
     <origin xyz="0.0  0.0 0.0" rpy="0.0 0  0.0"/>

File: software/models/atlas_v5/xacro/atlas_v5_minimal_contact.xacro (robot description, xacro)
@@ -3,5 +3,5 @@
   <xacro:include filename="../../common_components/multisense_sl/multisense_sl_no_collision.urdf" />
   <xacro:include filename="./atlas_v5_common.xacro" />
-  <xacro:include filename="../../common_components/robotiq_hand_description/robotiq_hand_no_collision.xacro" />
+  <xacro:include filename="../../common_components/robotiq_hand_description/robotiq_hand_no_joint_no_collision.xacro" />
   <!-- Set the initial hand position and orientation by changing 'rpy' and 'xyz'
   to mach the values in your actual robot. -->

File: software/models/common_components/robotiq_hand_description/mit_modifications/robotiq_hand_convex_hull.xacro (robot description, xacro)
@@ -1,25 +1,19 @@
 <robot name="robotiq" xmlns:xacro="http://www.ros.org/wiki/xacro">
-  <xacro:macro name="robotiq_convex_hull" params="is_left is_open parent">
-    <xacro:if value="${is_left}">
-      <xacro:robotiq_convex_hull_local prefix="left" is_open="${is_open}" parent="${parent}"/>
-    </xacro:if>
-    <xacro:unless value="${is_left}">
-      <xacro:robotiq_convex_hull_local prefix="right" is_open="${is_open}" parent="${parent}"/>
-    </xacro:unless>
-  </xacro:macro>
-  <xacro:macro name="robotiq_convex_hull_local" params="prefix is_open parent">
-    <link name="${prefix}_palm">
-      <visual>
-        <origin rpy="-1.57079 -1.57079 0" xyz="0 0.1725 0"/>
-        <geometry>
-          <xacro:if value="${is_open}">
-            <mesh filename="package://robotiq_hand_description/meshes/s-model/visual/GRIPPER_OPEN.obj" scale="1 1 1"/>
-          </xacro:if>
-          <xacro:unless value="${is_open}">
-            <mesh filename="package://robotiq_hand_description/meshes/s-model/visual/GRIPPER_CLOSED.obj" scale="1 1 1"/>
-          </xacro:unless>
-        </geometry>
-      </visual>
-      <collision group="${prefix}_hand_robotiq">
+  <xacro:macro name="robotiq_convex_hull" params="side is_open use_visuals parent">
+    <link name="${side}_palm">
+      <xacro:if value="${use_visuals}">
+        <visual>
+          <origin rpy="-1.57079 -1.57079 0" xyz="0 0.1725 0"/>
+          <geometry>
+            <xacro:if value="${is_open}">
+              <mesh filename="package://robotiq_hand_description/meshes/s-model/visual/GRIPPER_OPEN.obj" scale="1 1 1"/>
+            </xacro:if>
+            <xacro:unless value="${is_open}">
+              <mesh filename="package://robotiq_hand_description/meshes/s-model/visual/GRIPPER_CLOSED.obj" scale="1 1 1"/>
+            </xacro:unless>
+          </geometry>
+        </visual>
+      </xacro:if>
+      <collision group="${side}_hand_robotiq">
         <origin rpy="-1.57079 -1.57079 0" xyz="0 0.1725 0"/>
         <geometry>
@@ -33,7 +27,7 @@
       </collision>
     </link>
-    <joint name="${prefix}_palm_joint" type="fixed">
+    <joint name="${side}_palm_joint" type="fixed">
       <parent link="${parent}"/>
-      <child link="${prefix}_palm"/>
+      <child link="${side}_palm"/>
     </joint>
   </xacro:macro>
