Commit message: Update generated files for atlas_v4 and atlas_v5

File: software/models/atlas_v4/components/atlas_v4_convex_hull.urdf (robot description, URDF)
Before this commit: robot drc_skeleton, 36 links, 36 joints
Joints:
- removed joint l_arm_usz
- removed joint l_arm_uwy2
- removed joint r_arm_usz
- removed joint r_arm_uwy2
- added joint l_arm_lwy: type fixed, parent l_lfarm, child l_hand, origin xyz=0 0 0 rpy=0 0 0, axis 0 1 0, limit lower=-0.001 upper=0.001 effort=5 velocity=1
- added joint l_arm_shz: type revolute, parent utorso, child l_clav, origin xyz=0.1406 0.2256 0.4776 rpy=0 -0 0, axis 0 0 1, limit lower=-1.5708 upper=0.785398 effort=87 velocity=12
- added joint r_arm_lwy: type fixed, parent r_lfarm, child r_hand, origin xyz=0 0 0 rpy=0 0 0, axis 0 1 0, limit lower=-0.001 upper=0.001 effort=5 velocity=1
- added joint r_arm_shz: type revolute, parent utorso, child r_clav, origin xyz=0.1406 -0.2256 0.4776 rpy=0 -0 0, axis 0 0 1, limit lower=-0.785398 upper=1.5708 effort=87 velocity=12

File: software/models/atlas_v4/components/atlas_v4_full_collision_geometry.urdf (robot description, URDF)
Before this commit: robot drc_skeleton, 36 links, 36 joints
Joints:
- removed joint l_arm_usz
- removed joint l_arm_uwy2
- removed joint r_arm_usz
- removed joint r_arm_uwy2
- added joint l_arm_lwy: type fixed, parent l_lfarm, child l_hand, origin xyz=0 0 0 rpy=0 0 0, axis 0 1 0, limit lower=-0.001 upper=0.001 effort=5 velocity=1
- added joint l_arm_shz: type revolute, parent utorso, child l_clav, origin xyz=0.1406 0.2256 0.4776 rpy=0 -0 0, axis 0 0 1, limit lower=-1.5708 upper=0.785398 effort=87 velocity=12
- added joint r_arm_lwy: type fixed, parent r_lfarm, child r_hand, origin xyz=0 0 0 rpy=0 0 0, axis 0 1 0, limit lower=-0.001 upper=0.001 effort=5 velocity=1
- added joint r_arm_shz: type revolute, parent utorso, child r_clav, origin xyz=0.1406 -0.2256 0.4776 rpy=0 -0 0, axis 0 0 1, limit lower=-0.785398 upper=1.5708 effort=87 velocity=12

File: software/models/atlas_v4/components/atlas_v4_minimal_contact.urdf (robot description, URDF)
Before this commit: robot drc_skeleton, 36 links, 36 joints
Joints:
- removed joint l_arm_usz
- removed joint l_arm_uwy2
- removed joint r_arm_usz
- removed joint r_arm_uwy2
- added joint l_arm_lwy: type fixed, parent l_lfarm, child l_hand, origin xyz=0 0 0 rpy=0 0 0, axis 0 1 0, limit lower=-0.001 upper=0.001 effort=5 velocity=1
- added joint l_arm_shz: type revolute, parent utorso, child l_clav, origin xyz=0.1406 0.2256 0.4776 rpy=0 -0 0, axis 0 0 1, limit lower=-1.5708 upper=0.785398 effort=87 velocity=12
- added joint r_arm_lwy: type fixed, parent r_lfarm, child r_hand, origin xyz=0 0 0 rpy=0 0 0, axis 0 1 0, limit lower=-0.001 upper=0.001 effort=5 velocity=1
- added joint r_arm_shz: type revolute, parent utorso, child r_clav, origin xyz=0.1406 -0.2256 0.4776 rpy=0 -0 0, axis 0 0 1, limit lower=-0.785398 upper=1.5708 effort=87 velocity=12

File: software/models/atlas_v4/model_LR_RR.urdf (robot description, URDF)
Before this commit: robot atlas, 96 links, 95 joints
Joints:
- removed joint l_arm_usz
- removed joint l_arm_uwy2
- removed joint r_arm_usz
- removed joint r_arm_uwy2
- added joint l_arm_lwy: type fixed, parent l_lfarm, child l_hand, origin xyz=0 0 0 rpy=0 0 0, axis 0 1 0, limit lower=-0.001 upper=0.001 effort=5 velocity=1
- added joint l_arm_shz: type revolute, parent utorso, child l_clav, origin xyz=0.1406 0.2256 0.4776 rpy=0 -0 0, axis 0 0 1, limit lower=-1.5708 upper=0.785398 effort=87 velocity=12
- added joint r_arm_lwy: type fixed, parent r_lfarm, child r_hand, origin xyz=0 0 0 rpy=0 0 0, axis 0 1 0, limit lower=-0.001 upper=0.001 effort=5 velocity=1
- added joint r_arm_shz: type revolute, parent utorso, child r_clav, origin xyz=0.1406 -0.2256 0.4776 rpy=0 -0 0, axis 0 0 1, limit lower=-0.785398 upper=1.5708 effort=87 velocity=12

File: software/models/atlas_v4/model_convex_hull.urdf (robot description, URDF)
Before this commit: robot atlas, 72 links, 71 joints
Joints:
- removed joint l_arm_usz
- removed joint l_arm_uwy2
- removed joint r_arm_usz
- removed joint r_arm_uwy2
- added joint l_arm_lwy: type fixed, parent l_lfarm, child l_hand, origin xyz=0 0 0 rpy=0 0 0, axis 0 1 0, limit lower=-0.001 upper=0.001 effort=5 velocity=1
- added joint l_arm_shz: type revolute, parent utorso, child l_clav, origin xyz=0.1406 0.2256 0.4776 rpy=0 -0 0, axis 0 0 1, limit lower=-1.5708 upper=0.785398 effort=87 velocity=12
- added joint r_arm_lwy: type fixed, parent r_lfarm, child r_hand, origin xyz=0 0 0 rpy=0 0 0, axis 0 1 0, limit lower=-0.001 upper=0.001 effort=5 velocity=1
- added joint r_arm_shz: type revolute, parent utorso, child r_clav, origin xyz=0.1406 -0.2256 0.4776 rpy=0 -0 0, axis 0 0 1, limit lower=-0.785398 upper=1.5708 effort=87 velocity=12

File: software/models/atlas_v4/model_convex_hull_closed_hands.urdf (robot description, URDF)
Before this commit: robot atlas, 72 links, 71 joints
Joints:
- removed joint l_arm_usz
- removed joint l_arm_uwy2
- removed joint r_arm_usz
- removed joint r_arm_uwy2
- added joint l_arm_lwy: type fixed, parent l_lfarm, child l_hand, origin xyz=0 0 0 rpy=0 0 0, axis 0 1 0, limit lower=-0.001 upper=0.001 effort=5 velocity=1
- added joint l_arm_shz: type revolute, parent utorso, child l_clav, origin xyz=0.1406 0.2256 0.4776 rpy=0 -0 0, axis 0 0 1, limit lower=-1.5708 upper=0.785398 effort=87 velocity=12
- added joint r_arm_lwy: type fixed, parent r_lfarm, child r_hand, origin xyz=0 0 0 rpy=0 0 0, axis 0 1 0, limit lower=-0.001 upper=0.001 effort=5 velocity=1
- added joint r_arm_shz: type revolute, parent utorso, child r_clav, origin xyz=0.1406 -0.2256 0.4776 rpy=0 -0 0, axis 0 0 1, limit lower=-0.785398 upper=1.5708 effort=87 velocity=12

File: software/models/atlas_v4/model_minimal_contact.urdf (robot description, URDF)
Before this commit: robot atlas, 96 links, 95 joints
Joints:
- removed joint l_arm_usz
- removed joint l_arm_uwy2
- removed joint r_arm_usz
- removed joint r_arm_uwy2
- added joint l_arm_lwy: type fixed, parent l_lfarm, child l_hand, origin xyz=0 0 0 rpy=0 0 0, axis 0 1 0, limit lower=-0.001 upper=0.001 effort=5 velocity=1
- added joint l_arm_shz: type revolute, parent utorso, child l_clav, origin xyz=0.1406 0.2256 0.4776 rpy=0 -0 0, axis 0 0 1, limit lower=-1.5708 upper=0.785398 effort=87 velocity=12
- added joint r_arm_lwy: type fixed, parent r_lfarm, child r_hand, origin xyz=0 0 0 rpy=0 0 0, axis 0 1 0, limit lower=-0.001 upper=0.001 effort=5 velocity=1
- added joint r_arm_shz: type revolute, parent utorso, child r_clav, origin xyz=0.1406 -0.2256 0.4776 rpy=0 -0 0, axis 0 0 1, limit lower=-0.785398 upper=1.5708 effort=87 velocity=12

File: software/models/atlas_v5/components/atlas_v5_convex_hull.urdf (robot description, URDF)
Before this commit: robot drc_skeleton, 36 links, 36 joints
Joints:
- removed joint l_arm_usz
- removed joint l_arm_uwy2
- removed joint r_arm_usz
- removed joint r_arm_uwy2
- added joint l_arm_lwy: type revolute, parent l_lfarm, child l_hand, origin xyz=0 0 0 rpy=0 0 0, axis 0 1 0, limit lower=-2.9671 upper=2.9671 effort=25 velocity=10
- added joint l_arm_shz: type revolute, parent utorso, child l_clav, origin xyz=0.1406 0.2256 0.4776 rpy=0 0 0, axis 0 0 1, limit lower=-1.5708 upper=0.785398 effort=87 velocity=12
- added joint r_arm_lwy: type revolute, parent r_lfarm, child r_hand, origin xyz=0 0 0 rpy=0 0 0, axis 0 1 0, limit lower=-2.9671 upper=2.9671 effort=25 velocity=10
- added joint r_arm_shz: type revolute, parent utorso, child r_clav, origin xyz=0.1406 -0.2256 0.4776 rpy=0 0 0, axis 0 0 1, limit lower=-0.785398 upper=1.5708 effort=87 velocity=12

File: software/models/atlas_v5/components/atlas_v5_full_collision_geometry.urdf (robot description, URDF)
Before this commit: robot drc_skeleton, 36 links, 36 joints
Joints:
- removed joint l_arm_usz
- removed joint l_arm_uwy2
- removed joint r_arm_usz
- removed joint r_arm_uwy2
- added joint l_arm_lwy: type revolute, parent l_lfarm, child l_hand, origin xyz=0 0 0 rpy=0 0 0, axis 0 1 0, limit lower=-2.9671 upper=2.9671 effort=25 velocity=10
- added joint l_arm_shz: type revolute, parent utorso, child l_clav, origin xyz=0.1406 0.2256 0.4776 rpy=0 0 0, axis 0 0 1, limit lower=-1.5708 upper=0.785398 effort=87 velocity=12
- added joint r_arm_lwy: type revolute, parent r_lfarm, child r_hand, origin xyz=0 0 0 rpy=0 0 0, axis 0 1 0, limit lower=-2.9671 upper=2.9671 effort=25 velocity=10
- added joint r_arm_shz: type revolute, parent utorso, child r_clav, origin xyz=0.1406 -0.2256 0.4776 rpy=0 0 0, axis 0 0 1, limit lower=-0.785398 upper=1.5708 effort=87 velocity=12

File: software/models/atlas_v5/components/atlas_v5_minimal_contact.urdf (robot description, URDF)
Before this commit: robot drc_skeleton, 36 links, 36 joints
Joints:
- removed joint l_arm_usz
- removed joint l_arm_uwy2
- removed joint r_arm_usz
- removed joint r_arm_uwy2
- added joint l_arm_lwy: type revolute, parent l_lfarm, child l_hand, origin xyz=0 0 0 rpy=0 0 0, axis 0 1 0, limit lower=-2.9671 upper=2.9671 effort=25 velocity=10
- added joint l_arm_shz: type revolute, parent utorso, child l_clav, origin xyz=0.1406 0.2256 0.4776 rpy=0 0 0, axis 0 0 1, limit lower=-1.5708 upper=0.785398 effort=87 velocity=12
- added joint r_arm_lwy: type revolute, parent r_lfarm, child r_hand, origin xyz=0 0 0 rpy=0 0 0, axis 0 1 0, limit lower=-2.9671 upper=2.9671 effort=25 velocity=10
- added joint r_arm_shz: type revolute, parent utorso, child r_clav, origin xyz=0.1406 -0.2256 0.4776 rpy=0 0 0, axis 0 0 1, limit lower=-0.785398 upper=1.5708 effort=87 velocity=12

File: software/models/atlas_v5/model_LR_RR.urdf (robot description, URDF)
Before this commit: robot atlas, 96 links, 95 joints
Joints:
- removed joint l_arm_usz
- removed joint l_arm_uwy2
- removed joint r_arm_usz
- removed joint r_arm_uwy2
- added joint l_arm_lwy: type revolute, parent l_lfarm, child l_hand, origin xyz=0 0 0 rpy=0 0 0, axis 0 1 0, limit lower=-2.9671 upper=2.9671 effort=25 velocity=10
- added joint l_arm_shz: type revolute, parent utorso, child l_clav, origin xyz=0.1406 0.2256 0.4776 rpy=0 0 0, axis 0 0 1, limit lower=-1.5708 upper=0.785398 effort=87 velocity=12
- added joint r_arm_lwy: type revolute, parent r_lfarm, child r_hand, origin xyz=0 0 0 rpy=0 0 0, axis 0 1 0, limit lower=-2.9671 upper=2.9671 effort=25 velocity=10
- added joint r_arm_shz: type revolute, parent utorso, child r_clav, origin xyz=0.1406 -0.2256 0.4776 rpy=0 0 0, axis 0 0 1, limit lower=-0.785398 upper=1.5708 effort=87 velocity=12

File: software/models/atlas_v5/model_convex_hull.urdf (robot description, URDF)
Before this commit: robot atlas, 72 links, 71 joints
Joints:
- removed joint l_arm_usz
- removed joint l_arm_uwy2
- removed joint r_arm_usz
- removed joint r_arm_uwy2
- added joint l_arm_lwy: type revolute, parent l_lfarm, child l_hand, origin xyz=0 0 0 rpy=0 0 0, axis 0 1 0, limit lower=-2.9671 upper=2.9671 effort=25 velocity=10
- added joint l_arm_shz: type revolute, parent utorso, child l_clav, origin xyz=0.1406 0.2256 0.4776 rpy=0 0 0, axis 0 0 1, limit lower=-1.5708 upper=0.785398 effort=87 velocity=12
- added joint r_arm_lwy: type revolute, parent r_lfarm, child r_hand, origin xyz=0 0 0 rpy=0 0 0, axis 0 1 0, limit lower=-2.9671 upper=2.9671 effort=25 velocity=10
- added joint r_arm_shz: type revolute, parent utorso, child r_clav, origin xyz=0.1406 -0.2256 0.4776 rpy=0 0 0, axis 0 0 1, limit lower=-0.785398 upper=1.5708 effort=87 velocity=12

File: software/models/atlas_v5/model_convex_hull_closed_hands.urdf (robot description, URDF)
Before this commit: robot atlas, 72 links, 71 joints
Joints:
- removed joint l_arm_usz
- removed joint l_arm_uwy2
- removed joint r_arm_usz
- removed joint r_arm_uwy2
- added joint l_arm_lwy: type revolute, parent l_lfarm, child l_hand, origin xyz=0 0 0 rpy=0 0 0, axis 0 1 0, limit lower=-2.9671 upper=2.9671 effort=25 velocity=10
- added joint l_arm_shz: type revolute, parent utorso, child l_clav, origin xyz=0.1406 0.2256 0.4776 rpy=0 0 0, axis 0 0 1, limit lower=-1.5708 upper=0.785398 effort=87 velocity=12
- added joint r_arm_lwy: type revolute, parent r_lfarm, child r_hand, origin xyz=0 0 0 rpy=0 0 0, axis 0 1 0, limit lower=-2.9671 upper=2.9671 effort=25 velocity=10
- added joint r_arm_shz: type revolute, parent utorso, child r_clav, origin xyz=0.1406 -0.2256 0.4776 rpy=0 0 0, axis 0 0 1, limit lower=-0.785398 upper=1.5708 effort=87 velocity=12

File: software/models/atlas_v5/model_minimal_contact.urdf (robot description, URDF)
Before this commit: robot atlas, 96 links, 95 joints
Joints:
- removed joint l_arm_usz
- removed joint l_arm_uwy2
- removed joint r_arm_usz
- removed joint r_arm_uwy2
- added joint l_arm_lwy: type revolute, parent l_lfarm, child l_hand, origin xyz=0 0 0 rpy=0 0 0, axis 0 1 0, limit lower=-2.9671 upper=2.9671 effort=25 velocity=10
- added joint l_arm_shz: type revolute, parent utorso, child l_clav, origin xyz=0.1406 0.2256 0.4776 rpy=0 0 0, axis 0 0 1, limit lower=-1.5708 upper=0.785398 effort=87 velocity=12
- added joint r_arm_lwy: type revolute, parent r_lfarm, child r_hand, origin xyz=0 0 0 rpy=0 0 0, axis 0 1 0, limit lower=-2.9671 upper=2.9671 effort=25 velocity=10
- added joint r_arm_shz: type revolute, parent utorso, child r_clav, origin xyz=0.1406 -0.2256 0.4776 rpy=0 0 0, axis 0 0 1, limit lower=-0.785398 upper=1.5708 effort=87 velocity=12
