Commit message: Update generated files for V4 and V5

File: software/models/atlas_v5/model_convex_hull.urdf (robot description, URDF)
Before this commit: robot atlas, 72 links, 71 joints
Links:
- link l_clav: geometry collision mesh filename=package://atlas_v5/meshes/l_clav_chull.obj; visual mesh filename=package://atlas_v5/meshes/l_clav_chull.obj
- link l_foot: geometry collision mesh filename=package://atlas_v5/meshes/l_foot_chull.obj; collision sphere radius=0.0
- link l_larm: geometry collision mesh filename=package://atlas_v5/meshes/l_larm_chull.obj; visual mesh filename=package://atlas_v5/meshes/l_larm_chull.obj
- link l_lfarm: geometry collision mesh filename=package://atlas_v5/meshes/l_hand_chull.obj; visual mesh filename=package://atlas_v5/meshes/l_hand_chull.obj
- link l_lglut: geometry collision mesh filename=package://atlas_v5/meshes/l_lglut_chull.obj; visual mesh filename=package://atlas_v5/meshes/l_lglut_chull.obj
- link l_lleg: geometry collision mesh filename=package://atlas_v5/meshes/l_lleg_chull.obj; visual mesh filename=package://atlas_v5/meshes/l_lleg_chull.obj
- link l_robotiq_convex_hull: geometry collision mesh filename=package://robotiq_hand_description/meshes/s-model/collision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 scale=1 1 1; visual mesh filename=package://robotiq_hand_description/meshes/s-model/visual/GR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 scale=1 1 1
- link l_scap: geometry collision mesh filename=package://atlas_v5/meshes/l_scap_chull.obj; visual mesh filename=package://atlas_v5/meshes/l_scap_chull.obj
- link l_situational_awareness_camera_link: geometry collision box size=0.01 0.01 0.01; visual box size=0.01 0.01 0.01
- link l_uarm: geometry collision mesh filename=package://atlas_v5/meshes/l_uarm_chull.obj; visual mesh filename=package://atlas_v5/meshes/l_uarm_chull.obj
- link l_ufarm: geometry collision mesh filename=package://atlas_v5/meshes/l_farm_chull.obj; visual mesh filename=package://atlas_v5/meshes/l_farm_chull.obj
- link l_uglut: geometry collision mesh filename=package://atlas_v5/meshes/l_uglut_chull.obj; visual mesh filename=package://atlas_v5/meshes/l_uglut_chull.obj
- link l_uleg: geometry collision mesh filename=package://atlas_v5/meshes/l_uleg_chull.obj; visual mesh filename=package://atlas_v5/meshes/l_uleg_chull.obj
- link pelvis: geometry collision mesh filename=package://atlas_v5/meshes/pelvis_chull.obj; visual mesh filename=package://atlas_v5/meshes/pelvis_chull.obj
- link r_clav: geometry collision mesh filename=package://atlas_v5/meshes/r_clav_chull.obj; visual mesh filename=package://atlas_v5/meshes/r_clav_chull.obj
- link r_foot: geometry collision mesh filename=package://atlas_v5/meshes/r_foot_chull.obj; collision sphere radius=0.0
- link r_larm: geometry collision mesh filename=package://atlas_v5/meshes/r_larm_chull.obj; visual mesh filename=package://atlas_v5/meshes/r_larm_chull.obj
- link r_lfarm: geometry collision mesh filename=package://atlas_v5/meshes/r_hand_chull.obj; visual mesh filename=package://atlas_v5/meshes/r_hand_chull.obj
- link r_lglut: geometry collision mesh filename=package://atlas_v5/meshes/r_lglut_chull.obj; visual mesh filename=package://atlas_v5/meshes/r_lglut_chull.obj
- link r_lleg: geometry collision mesh filename=package://atlas_v5/meshes/r_lleg_chull.obj; visual mesh filename=package://atlas_v5/meshes/r_lleg_chull.obj
- link r_robotiq_convex_hull: geometry collision mesh filename=package://robotiq_hand_description/meshes/s-model/collision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 scale=1 1 1; visual mesh filename=package://robotiq_hand_description/meshes/s-model/visual/GR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 scale=1 1 1
- link r_scap: geometry collision mesh filename=package://atlas_v5/meshes/r_scap_chull.obj; visual mesh filename=package://atlas_v5/meshes/r_scap_chull.obj
- link r_situational_awareness_camera_link: geometry collision box size=0.01 0.01 0.01; visual box size=0.01 0.01 0.01
- link r_uarm: geometry collision mesh filename=package://atlas_v5/meshes/r_uarm_chull.obj; visual mesh filename=package://atlas_v5/meshes/r_uarm_chull.obj
- link r_ufarm: geometry collision mesh filename=package://atlas_v5/meshes/r_farm_chull.obj; visual mesh filename=package://atlas_v5/meshes/r_farm_chull.obj
- link r_uglut: geometry collision mesh filename=package://atlas_v5/meshes/r_uglut_chull.obj; visual mesh filename=package://atlas_v5/meshes/r_uglut_chull.obj
- link r_uleg: geometry collision mesh filename=package://atlas_v5/meshes/r_uleg_chull.obj; visual mesh filename=package://atlas_v5/meshes/r_uleg_chull.obj
- link rear_situational_awareness_camera_link: geometry collision box size=0.01 0.01 0.01; visual box size=0.01 0.01 0.01
- link utorso: geometry collision mesh filename=package://atlas_v5/meshes/utorso_chull.obj; visual mesh filename=package://atlas_v5/meshes/utorso_chull.obj

File: software/models/atlas_v5/model_convex_hull_closed_hands.urdf (robot description, URDF)
Before this commit: robot atlas, 72 links, 71 joints
Links:
- link l_clav: geometry collision mesh filename=package://atlas_v5/meshes/l_clav_chull.obj; visual mesh filename=package://atlas_v5/meshes/l_clav_chull.obj
- link l_foot: geometry collision mesh filename=package://atlas_v5/meshes/l_foot_chull.obj; collision sphere radius=0.0
- link l_larm: geometry collision mesh filename=package://atlas_v5/meshes/l_larm_chull.obj; visual mesh filename=package://atlas_v5/meshes/l_larm_chull.obj
- link l_lfarm: geometry collision mesh filename=package://atlas_v5/meshes/l_hand_chull.obj; visual mesh filename=package://atlas_v5/meshes/l_hand_chull.obj
- link l_lglut: geometry collision mesh filename=package://atlas_v5/meshes/l_lglut_chull.obj; visual mesh filename=package://atlas_v5/meshes/l_lglut_chull.obj
- link l_lleg: geometry collision mesh filename=package://atlas_v5/meshes/l_lleg_chull.obj; visual mesh filename=package://atlas_v5/meshes/l_lleg_chull.obj
- link l_robotiq_convex_hull: geometry collision mesh filename=package://robotiq_hand_description/meshes/s-model/collision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 scale=1 1 1; visual mesh filename=package://robotiq_hand_description/meshes/s-model/visual/GR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 scale=1 1 1
- link l_scap: geometry collision mesh filename=package://atlas_v5/meshes/l_scap_chull.obj; visual mesh filename=package://atlas_v5/meshes/l_scap_chull.obj
- link l_situational_awareness_camera_link: geometry collision box size=0.01 0.01 0.01; visual box size=0.01 0.01 0.01
- link l_uarm: geometry collision mesh filename=package://atlas_v5/meshes/l_uarm_chull.obj; visual mesh filename=package://atlas_v5/meshes/l_uarm_chull.obj
- link l_ufarm: geometry collision mesh filename=package://atlas_v5/meshes/l_farm_chull.obj; visual mesh filename=package://atlas_v5/meshes/l_farm_chull.obj
- link l_uglut: geometry collision mesh filename=package://atlas_v5/meshes/l_uglut_chull.obj; visual mesh filename=package://atlas_v5/meshes/l_uglut_chull.obj
- link l_uleg: geometry collision mesh filename=package://atlas_v5/meshes/l_uleg_chull.obj; visual mesh filename=package://atlas_v5/meshes/l_uleg_chull.obj
- link pelvis: geometry collision mesh filename=package://atlas_v5/meshes/pelvis_chull.obj; visual mesh filename=package://atlas_v5/meshes/pelvis_chull.obj
- link r_clav: geometry collision mesh filename=package://atlas_v5/meshes/r_clav_chull.obj; visual mesh filename=package://atlas_v5/meshes/r_clav_chull.obj
- link r_foot: geometry collision mesh filename=package://atlas_v5/meshes/r_foot_chull.obj; collision sphere radius=0.0
- link r_larm: geometry collision mesh filename=package://atlas_v5/meshes/r_larm_chull.obj; visual mesh filename=package://atlas_v5/meshes/r_larm_chull.obj
- link r_lfarm: geometry collision mesh filename=package://atlas_v5/meshes/r_hand_chull.obj; visual mesh filename=package://atlas_v5/meshes/r_hand_chull.obj
- link r_lglut: geometry collision mesh filename=package://atlas_v5/meshes/r_lglut_chull.obj; visual mesh filename=package://atlas_v5/meshes/r_lglut_chull.obj
- link r_lleg: geometry collision mesh filename=package://atlas_v5/meshes/r_lleg_chull.obj; visual mesh filename=package://atlas_v5/meshes/r_lleg_chull.obj
- link r_robotiq_convex_hull: geometry collision mesh filename=package://robotiq_hand_description/meshes/s-model/collision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 scale=1 1 1; visual mesh filename=package://robotiq_hand_description/meshes/s-model/visual/GR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 scale=1 1 1
- link r_scap: geometry collision mesh filename=package://atlas_v5/meshes/r_scap_chull.obj; visual mesh filename=package://atlas_v5/meshes/r_scap_chull.obj
- link r_situational_awareness_camera_link: geometry collision box size=0.01 0.01 0.01; visual box size=0.01 0.01 0.01
- link r_uarm: geometry collision mesh filename=package://atlas_v5/meshes/r_uarm_chull.obj; visual mesh filename=package://atlas_v5/meshes/r_uarm_chull.obj
- link r_ufarm: geometry collision mesh filename=package://atlas_v5/meshes/r_farm_chull.obj; visual mesh filename=package://atlas_v5/meshes/r_farm_chull.obj
- link r_uglut: geometry collision mesh filename=package://atlas_v5/meshes/r_uglut_chull.obj; visual mesh filename=package://atlas_v5/meshes/r_uglut_chull.obj
- link r_uleg: geometry collision mesh filename=package://atlas_v5/meshes/r_uleg_chull.obj; visual mesh filename=package://atlas_v5/meshes/r_uleg_chull.obj
- link rear_situational_awareness_camera_link: geometry collision box size=0.01 0.01 0.01; visual box size=0.01 0.01 0.01
- link utorso: geometry collision mesh filename=package://atlas_v5/meshes/utorso_chull.obj; visual mesh filename=package://atlas_v5/meshes/utorso_chull.obj
