Commit message: Update v4 files for new changes from OSRF

File: software/models/atlas_v4/components/atlas_v4_convex_hull.urdf (robot description, URDF)
Before this commit: robot drc_skeleton, 36 links, 36 joints
Links:
- removed link rear_situational_awareness_camera_link
- removed link rear_situational_awareness_camera_optical_frame
- link l_clav: mass 3.45 -> 4.466
- link l_foot: mass 2.05 -> 2.41
- link l_larm: mass 2.509 -> 3.248
- link l_lglut: mass 0.866 -> 0.898
- link l_lleg: mass 5.479 -> 4.515
- link l_scap: mass 3.012 -> 3.899
- link l_uarm: mass 3.388 -> 4.386
- link l_ufarm: mass 3.388 -> 4.386
- link l_uglut: mass 0.648 -> 1.959
- link l_uleg: mass 9.209 -> 8.204
- link ltorso: mass 2.409 -> 2.270
- link mtorso: mass 0.69 -> 0.799
- link pelvis: mass 17.882 -> 9.509
- link r_clav: mass 3.45 -> 4.466
- link r_foot: mass 2.05 -> 2.41
- link r_larm: mass 2.509 -> 3.248
- link r_lglut: mass 0.866 -> 0.898
- link r_lleg: mass 5.479 -> 4.515
- link r_scap: mass 3.012 -> 3.899
- link r_uarm: mass 3.388 -> 4.386
- link r_ufarm: mass 3.388 -> 4.386
- link r_uglut: mass 0.648 -> 1.959
- link r_uleg: mass 9.209 -> 8.204
- link utorso: mass 63.73 -> 84.409
Joints:
- removed joint rear_situational_awareness_camera_joint
- removed joint rear_situational_awareness_camera_optical_frame_joint
- joint l_situational_awareness_camera_joint: origin xyz=0.216409 0.121799 0.406759 rpy=-1.57079633 0 1.30899694 -> xyz=0.155 0.121 0.785 rpy=0 0 1.309
- joint r_situational_awareness_camera_joint: origin xyz=0.216409 -0.121799 0.406759 rpy=1.57079633 0 -1.30899694 -> xyz=0.155 -0.121 0.785 rpy=0 0 -1.309

File: software/models/atlas_v4/components/atlas_v4_full_collision_geometry.urdf (robot description, URDF)
Before this commit: robot drc_skeleton, 36 links, 36 joints
Links:
- removed link rear_situational_awareness_camera_link
- removed link rear_situational_awareness_camera_optical_frame
- link l_clav: mass 3.45 -> 4.466; geometry collision box size=0.1 0.07 0.072; collision cylinder length=0.1525 radius=0.0555
- link l_foot: mass 2.05 -> 2.41; geometry collision box size=0.1 0.08 0.02; collision box size=0.227 0.133887 0.05
- link l_larm: mass 2.509 -> 3.248; geometry collision box size=0.135 0.15 0.06; collision cylinder length=0.125 radius=0.045
- link l_lfarm: geometry collision box size=0.13 0.09 0.07; collision cylinder length=0.05 radius=0.03
- link l_lglut: mass 0.866 -> 0.898
- link l_lleg: mass 5.479 -> 4.515
- link l_scap: mass 3.012 -> 3.899
- link l_uarm: mass 3.388 -> 4.386
- link l_ufarm: mass 3.388 -> 4.386; geometry collision box size=0.135 0.1 0.045; collision cylinder length=0.125 radius=0.045
- link l_uglut: mass 0.648 -> 1.959
- link l_uleg: mass 9.209 -> 8.204; geometry collision box size=0.07 0.038 0.14; collision box size=0.07 0.038 0.15
- link ltorso: mass 2.409 -> 2.270
- link mtorso: mass 0.69 -> 0.799
- link pelvis: mass 17.882 -> 9.509
- link r_clav: mass 3.45 -> 4.466; geometry collision box size=0.1 0.07 0.072; collision cylinder length=0.1525 radius=0.0555
- link r_foot: mass 2.05 -> 2.41; geometry collision box size=0.1 0.08 0.02; collision box size=0.227 0.133887 0.05
- link r_larm: mass 2.509 -> 3.248; geometry collision box size=0.135 0.15 0.06; collision cylinder length=0.125 radius=0.045
- link r_lfarm: geometry collision box size=0.13 0.09 0.07; collision cylinder length=0.05 radius=0.03
- link r_lglut: mass 0.866 -> 0.898
- link r_lleg: mass 5.479 -> 4.515
- link r_scap: mass 3.012 -> 3.899
- link r_uarm: mass 3.388 -> 4.386
- link r_ufarm: mass 3.388 -> 4.386; geometry collision box size=0.135 0.1 0.045; collision cylinder length=0.125 radius=0.045
- link r_uglut: mass 0.648 -> 1.959
- link r_uleg: mass 9.209 -> 8.204; geometry collision box size=0.07 0.038 0.14; collision box size=0.07 0.038 0.15
- link utorso: mass 63.73 -> 84.409; geometry collision box size=0.2 0.25 0.01; collision box size=0.456306 0.341719 0.12
Joints:
- removed joint rear_situational_awareness_camera_joint
- removed joint rear_situational_awareness_camera_optical_frame_joint
- joint l_situational_awareness_camera_joint: origin xyz=0.216409 0.121799 0.406759 rpy=-1.57079633 0 1.30899694 -> xyz=0.155 0.121 0.785 rpy=0 0 1.309
- joint r_situational_awareness_camera_joint: origin xyz=0.216409 -0.121799 0.406759 rpy=1.57079633 0 -1.30899694 -> xyz=0.155 -0.121 0.785 rpy=0 0 -1.309

File: software/models/atlas_v4/components/atlas_v4_minimal_contact.urdf (robot description, URDF)
Before this commit: robot drc_skeleton, 36 links, 36 joints
Links:
- removed link rear_situational_awareness_camera_link
- removed link rear_situational_awareness_camera_optical_frame
- link l_clav: mass 3.45 -> 4.466
- link l_foot: mass 2.05 -> 2.41
- link l_larm: mass 2.509 -> 3.248
- link l_lglut: mass 0.866 -> 0.898
- link l_lleg: mass 5.479 -> 4.515
- link l_scap: mass 3.012 -> 3.899
- link l_uarm: mass 3.388 -> 4.386
- link l_ufarm: mass 3.388 -> 4.386
- link l_uglut: mass 0.648 -> 1.959
- link l_uleg: mass 9.209 -> 8.204
- link ltorso: mass 2.409 -> 2.270
- link mtorso: mass 0.69 -> 0.799
- link pelvis: mass 17.882 -> 9.509
- link r_clav: mass 3.45 -> 4.466
- link r_foot: mass 2.05 -> 2.41
- link r_larm: mass 2.509 -> 3.248
- link r_lglut: mass 0.866 -> 0.898
- link r_lleg: mass 5.479 -> 4.515
- link r_scap: mass 3.012 -> 3.899
- link r_uarm: mass 3.388 -> 4.386
- link r_ufarm: mass 3.388 -> 4.386
- link r_uglut: mass 0.648 -> 1.959
- link r_uleg: mass 9.209 -> 8.204
- link utorso: mass 63.73 -> 84.409
Joints:
- removed joint rear_situational_awareness_camera_joint
- removed joint rear_situational_awareness_camera_optical_frame_joint
- joint l_situational_awareness_camera_joint: origin xyz=0.216409 0.121799 0.406759 rpy=-1.57079633 0 1.30899694 -> xyz=0.155 0.121 0.785 rpy=0 0 1.309
- joint r_situational_awareness_camera_joint: origin xyz=0.216409 -0.121799 0.406759 rpy=1.57079633 0 -1.30899694 -> xyz=0.155 -0.121 0.785 rpy=0 0 -1.309

File: software/models/atlas_v4/components/osrf_original/atlas_v4.urdf (robot description, URDF)
Before this commit: robot drc_skeleton, 36 links, 36 joints
Links:
- removed link rear_situational_awareness_camera_link
- removed link rear_situational_awareness_camera_optical_frame
- link l_clav: mass 3.45 -> 4.466; geometry collision box size=0.1 0.07 0.072; collision cylinder length=0.1525 radius=0.0555
- link l_foot: mass 2.05 -> 2.41; geometry collision box size=${0.26-0.033} ${0.124887+0.009} 0.05; collision box size=0.1 ${0.08} 0.02
- link l_larm: mass 2.509 -> 3.248; geometry collision box size=0.135 0.15 0.06; collision cylinder length=0.125 radius=0.045
- link l_lfarm: geometry collision box size=0.13 0.09 0.07; collision cylinder length=0.05 radius=0.03
- link l_lglut: mass 0.866 -> 0.898
- link l_lleg: mass 5.479 -> 4.515
- link l_scap: mass 3.012 -> 3.899
- link l_uarm: mass 3.388 -> 4.386
- link l_ufarm: mass 3.388 -> 4.386; geometry collision box size=0.135 0.1 0.045; collision cylinder length=0.125 radius=0.045
- link l_uglut: mass 0.648 -> 1.959
- link l_uleg: mass 9.209 -> 8.204; geometry collision box size=0.07 0.038 0.14; collision box size=0.07 0.038 0.15
- link ltorso: mass 2.409 -> 2.270
- link mtorso: mass 0.69 -> 0.799
- link pelvis: mass 17.882 -> 9.509
- link r_clav: mass 3.45 -> 4.466; geometry collision box size=0.1 0.07 0.072; collision cylinder length=0.1525 radius=0.0555
- link r_foot: mass 2.05 -> 2.41; geometry collision box size=${0.26-0.033} ${0.124887+0.009} 0.05; collision box size=0.1 ${0.08} 0.02
- link r_larm: mass 2.509 -> 3.248; geometry collision box size=0.135 0.15 0.06; collision cylinder length=0.125 radius=0.045
- link r_lfarm: geometry collision box size=0.13 0.09 0.07; collision cylinder length=0.05 radius=0.03
- link r_lglut: mass 0.866 -> 0.898
- link r_lleg: mass 5.479 -> 4.515
- link r_scap: mass 3.012 -> 3.899
- link r_uarm: mass 3.388 -> 4.386
- link r_ufarm: mass 3.388 -> 4.386; geometry collision box size=0.135 0.1 0.045; collision cylinder length=0.125 radius=0.045
- link r_uglut: mass 0.648 -> 1.959
- link r_uleg: mass 9.209 -> 8.204; geometry collision box size=0.07 0.038 0.14; collision box size=0.07 0.038 0.15
- link utorso: mass 63.73 -> 84.409; geometry collision box size=0.2 0.25 0.01; collision box size=0.456306 0.341719 0.12
Joints:
- removed joint rear_situational_awareness_camera_joint
- removed joint rear_situational_awareness_camera_optical_frame_joint
- joint l_situational_awareness_camera_joint: origin xyz=0.216409 0.121799 0.406759 rpy=-1.57079633 0 1.30899694 -> xyz=0.155 0.121 0.785 rpy=0 0 1.309
- joint r_situational_awareness_camera_joint: origin xyz=0.216409 -0.121799 0.406759 rpy=1.57079633 0 -1.30899694 -> xyz=0.155 -0.121 0.785 rpy=0 0 -1.309

File: software/models/atlas_v4/model_LR_RR.urdf (robot description, URDF)
Before this commit: robot atlas, 88 links, 87 joints
Links:
- removed link rear_situational_awareness_camera_link
- removed link rear_situational_awareness_camera_optical_frame
- link l_clav: mass 3.45 -> 4.466; geometry collision box size=0.1 0.07 0.072; collision cylinder length=0.1525 radius=0.0555
- link l_foot: mass 2.05 -> 2.41; geometry collision box size=0.1 0.08 0.02; collision box size=0.227 0.133887 0.05
- link l_larm: mass 2.509 -> 3.248; geometry collision box size=0.135 0.15 0.06; collision cylinder length=0.125 radius=0.045
- link l_lfarm: geometry collision box size=0.13 0.09 0.07; collision cylinder length=0.05 radius=0.03
- link l_lglut: mass 0.866 -> 0.898
- link l_lleg: mass 5.479 -> 4.515
- link l_scap: mass 3.012 -> 3.899
- link l_uarm: mass 3.388 -> 4.386
- link l_ufarm: mass 3.388 -> 4.386; geometry collision box size=0.135 0.1 0.045; collision cylinder length=0.125 radius=0.045
- link l_uglut: mass 0.648 -> 1.959
- link l_uleg: mass 9.209 -> 8.204; geometry collision box size=0.07 0.038 0.14; collision box size=0.07 0.038 0.15
- link ltorso: mass 2.409 -> 2.270
- link mtorso: mass 0.69 -> 0.799
- link pelvis: mass 17.882 -> 9.509
- link r_clav: mass 3.45 -> 4.466; geometry collision box size=0.1 0.07 0.072; collision cylinder length=0.1525 radius=0.0555
- link r_foot: mass 2.05 -> 2.41; geometry collision box size=0.1 0.08 0.02; collision box size=0.227 0.133887 0.05
- link r_larm: mass 2.509 -> 3.248; geometry collision box size=0.135 0.15 0.06; collision cylinder length=0.125 radius=0.045
- link r_lfarm: geometry collision box size=0.13 0.09 0.07; collision cylinder length=0.05 radius=0.03
- link r_lglut: mass 0.866 -> 0.898
- link r_lleg: mass 5.479 -> 4.515
- link r_scap: mass 3.012 -> 3.899
- link r_uarm: mass 3.388 -> 4.386
- link r_ufarm: mass 3.388 -> 4.386; geometry collision box size=0.135 0.1 0.045; collision cylinder length=0.125 radius=0.045
- link r_uglut: mass 0.648 -> 1.959
- link r_uleg: mass 9.209 -> 8.204; geometry collision box size=0.07 0.038 0.14; collision box size=0.07 0.038 0.15
- link utorso: mass 63.73 -> 84.409; geometry collision box size=0.2 0.25 0.01; collision box size=0.456306 0.341719 0.12
Joints:
- removed joint rear_situational_awareness_camera_joint
- removed joint rear_situational_awareness_camera_optical_frame_joint
- joint l_situational_awareness_camera_joint: origin xyz=0.216409 0.121799 0.406759 rpy=-1.57079633 0 1.30899694 -> xyz=0.155 0.121 0.785 rpy=0 0 1.309
- joint r_situational_awareness_camera_joint: origin xyz=0.216409 -0.121799 0.406759 rpy=1.57079633 0 -1.30899694 -> xyz=0.155 -0.121 0.785 rpy=0 0 -1.309

File: software/models/atlas_v4/model_convex_hull.urdf (robot description, URDF)
Before this commit: robot atlas, 72 links, 71 joints
Links:
- removed link rear_situational_awareness_camera_link
- removed link rear_situational_awareness_camera_optical_frame
- link l_clav: mass 3.45 -> 4.466
- link l_foot: mass 2.05 -> 2.41
- link l_larm: mass 2.509 -> 3.248
- link l_lglut: mass 0.866 -> 0.898
- link l_lleg: mass 5.479 -> 4.515
- link l_scap: mass 3.012 -> 3.899
- link l_uarm: mass 3.388 -> 4.386
- link l_ufarm: mass 3.388 -> 4.386
- link l_uglut: mass 0.648 -> 1.959
- link l_uleg: mass 9.209 -> 8.204
- link ltorso: mass 2.409 -> 2.270
- link mtorso: mass 0.69 -> 0.799
- link pelvis: mass 17.882 -> 9.509
- link r_clav: mass 3.45 -> 4.466
- link r_foot: mass 2.05 -> 2.41
- link r_larm: mass 2.509 -> 3.248
- link r_lglut: mass 0.866 -> 0.898
- link r_lleg: mass 5.479 -> 4.515
- link r_scap: mass 3.012 -> 3.899
- link r_uarm: mass 3.388 -> 4.386
- link r_ufarm: mass 3.388 -> 4.386
- link r_uglut: mass 0.648 -> 1.959
- link r_uleg: mass 9.209 -> 8.204
- link utorso: mass 63.73 -> 84.409
Joints:
- removed joint rear_situational_awareness_camera_joint
- removed joint rear_situational_awareness_camera_optical_frame_joint
- joint l_situational_awareness_camera_joint: origin xyz=0.216409 0.121799 0.406759 rpy=-1.57079633 0 1.30899694 -> xyz=0.155 0.121 0.785 rpy=0 0 1.309
- joint r_situational_awareness_camera_joint: origin xyz=0.216409 -0.121799 0.406759 rpy=1.57079633 0 -1.30899694 -> xyz=0.155 -0.121 0.785 rpy=0 0 -1.309

File: software/models/atlas_v4/model_convex_hull_closed_hands.urdf (robot description, URDF)
Before this commit: robot atlas, 72 links, 71 joints
Links:
- removed link rear_situational_awareness_camera_link
- removed link rear_situational_awareness_camera_optical_frame
- link l_clav: mass 3.45 -> 4.466
- link l_foot: mass 2.05 -> 2.41
- link l_larm: mass 2.509 -> 3.248
- link l_lglut: mass 0.866 -> 0.898
- link l_lleg: mass 5.479 -> 4.515
- link l_scap: mass 3.012 -> 3.899
- link l_uarm: mass 3.388 -> 4.386
- link l_ufarm: mass 3.388 -> 4.386
- link l_uglut: mass 0.648 -> 1.959
- link l_uleg: mass 9.209 -> 8.204
- link ltorso: mass 2.409 -> 2.270
- link mtorso: mass 0.69 -> 0.799
- link pelvis: mass 17.882 -> 9.509
- link r_clav: mass 3.45 -> 4.466
- link r_foot: mass 2.05 -> 2.41
- link r_larm: mass 2.509 -> 3.248
- link r_lglut: mass 0.866 -> 0.898
- link r_lleg: mass 5.479 -> 4.515
- link r_scap: mass 3.012 -> 3.899
- link r_uarm: mass 3.388 -> 4.386
- link r_ufarm: mass 3.388 -> 4.386
- link r_uglut: mass 0.648 -> 1.959
- link r_uleg: mass 9.209 -> 8.204
- link utorso: mass 63.73 -> 84.409
Joints:
- removed joint rear_situational_awareness_camera_joint
- removed joint rear_situational_awareness_camera_optical_frame_joint
- joint l_situational_awareness_camera_joint: origin xyz=0.216409 0.121799 0.406759 rpy=-1.57079633 0 1.30899694 -> xyz=0.155 0.121 0.785 rpy=0 0 1.309
- joint r_situational_awareness_camera_joint: origin xyz=0.216409 -0.121799 0.406759 rpy=1.57079633 0 -1.30899694 -> xyz=0.155 -0.121 0.785 rpy=0 0 -1.309

File: software/models/atlas_v4/model_convex_hull_fingers.urdf (robot description, URDF)
Before this commit: robot atlas, 96 links, 95 joints
Links:
- removed link rear_situational_awareness_camera_link
- removed link rear_situational_awareness_camera_optical_frame
- link l_clav: mass 3.45 -> 4.466
- link l_foot: mass 2.05 -> 2.41
- link l_larm: mass 2.509 -> 3.248
- link l_lglut: mass 0.866 -> 0.898
- link l_lleg: mass 5.479 -> 4.515
- link l_scap: mass 3.012 -> 3.899
- link l_uarm: mass 3.388 -> 4.386
- link l_ufarm: mass 3.388 -> 4.386
- link l_uglut: mass 0.648 -> 1.959
- link l_uleg: mass 9.209 -> 8.204
- link ltorso: mass 2.409 -> 2.270
- link mtorso: mass 0.69 -> 0.799
- link pelvis: mass 17.882 -> 9.509
- link r_clav: mass 3.45 -> 4.466
- link r_foot: mass 2.05 -> 2.41
- link r_larm: mass 2.509 -> 3.248
- link r_lglut: mass 0.866 -> 0.898
- link r_lleg: mass 5.479 -> 4.515
- link r_scap: mass 3.012 -> 3.899
- link r_uarm: mass 3.388 -> 4.386
- link r_ufarm: mass 3.388 -> 4.386
- link r_uglut: mass 0.648 -> 1.959
- link r_uleg: mass 9.209 -> 8.204
- link utorso: mass 63.73 -> 84.409
Joints:
- removed joint rear_situational_awareness_camera_joint
- removed joint rear_situational_awareness_camera_optical_frame_joint
- joint l_situational_awareness_camera_joint: origin xyz=0.216409 0.121799 0.406759 rpy=-1.57079633 0 1.30899694 -> xyz=0.155 0.121 0.785 rpy=0 0 1.309
- joint r_situational_awareness_camera_joint: origin xyz=0.216409 -0.121799 0.406759 rpy=1.57079633 0 -1.30899694 -> xyz=0.155 -0.121 0.785 rpy=0 0 -1.309

File: software/models/atlas_v4/model_minimal_contact.urdf (robot description, URDF)
Before this commit: robot atlas, 96 links, 95 joints
Links:
- removed link rear_situational_awareness_camera_link
- removed link rear_situational_awareness_camera_optical_frame
- link l_clav: mass 3.45 -> 4.466
- link l_foot: mass 2.05 -> 2.41
- link l_larm: mass 2.509 -> 3.248
- link l_lglut: mass 0.866 -> 0.898
- link l_lleg: mass 5.479 -> 4.515
- link l_scap: mass 3.012 -> 3.899
- link l_uarm: mass 3.388 -> 4.386
- link l_ufarm: mass 3.388 -> 4.386
- link l_uglut: mass 0.648 -> 1.959
- link l_uleg: mass 9.209 -> 8.204
- link ltorso: mass 2.409 -> 2.270
- link mtorso: mass 0.69 -> 0.799
- link pelvis: mass 17.882 -> 9.509
- link r_clav: mass 3.45 -> 4.466
- link r_foot: mass 2.05 -> 2.41
- link r_larm: mass 2.509 -> 3.248
- link r_lglut: mass 0.866 -> 0.898
- link r_lleg: mass 5.479 -> 4.515
- link r_scap: mass 3.012 -> 3.899
- link r_uarm: mass 3.388 -> 4.386
- link r_ufarm: mass 3.388 -> 4.386
- link r_uglut: mass 0.648 -> 1.959
- link r_uleg: mass 9.209 -> 8.204
- link utorso: mass 63.73 -> 84.409
Joints:
- removed joint rear_situational_awareness_camera_joint
- removed joint rear_situational_awareness_camera_optical_frame_joint
- joint l_situational_awareness_camera_joint: origin xyz=0.216409 0.121799 0.406759 rpy=-1.57079633 0 1.30899694 -> xyz=0.155 0.121 0.785 rpy=0 0 1.309
- joint r_situational_awareness_camera_joint: origin xyz=0.216409 -0.121799 0.406759 rpy=1.57079633 0 -1.30899694 -> xyz=0.155 -0.121 0.785 rpy=0 0 -1.309
