Commit message: finally found the correct left arm model

File: software/models/atlas_v4/components/atlas_v4_convex_hull.urdf (robot description, URDF)
Before this commit: robot drc_skeleton, 34 links, 34 joints
Links:
- link l_clav: geometry collision mesh filename=package://atlas_v4/meshes/r_clav_chull.obj scale=1 1 1; visual mesh filename=package://atlas_v4/meshes/r_clav.obj scale=1 1 1
- link l_larm: geometry collision mesh filename=package://atlas_v4/meshes/r_larm_chull.obj scale=1 1 1; visual mesh filename=package://atlas_v4/meshes/r_larm.obj scale=1 1 1
- link l_lfarm: geometry collision mesh filename=package://atlas_v4/meshes/r_hand_chull.obj scale=1 1 1; visual mesh filename=package://atlas_v4/meshes/r_hand.obj scale=1 1 1
- link l_scap: geometry collision mesh filename=package://atlas_v4/meshes/r_scap_chull.obj scale=1 1 1; visual mesh filename=package://atlas_v4/meshes/r_scap.obj scale=1 1 1
- link l_uarm: geometry collision mesh filename=package://atlas_v4/meshes/r_uarm_chull.obj scale=1 1 1; visual mesh filename=package://atlas_v4/meshes/r_uarm.obj scale=1 1 1
- link l_ufarm: geometry collision mesh filename=package://atlas_v4/meshes/r_farm_chull.obj scale=1 1 1; visual mesh filename=package://atlas_v4/meshes/r_farm.obj scale=1 1 1
Joints:
- joint l_arm_elx: axis 1 0 0 -> -1.0 -0.0 -0.0; origin xyz=0 0.119 0.0092 rpy=0 -0 0 -> xyz=0 -0.119 0.0092 rpy=0 -0 0
- joint l_arm_ely: axis 0 1 0 -> -0.0 -1.0 -0.0; origin xyz=0 0.187 -0.016 rpy=0 -0 0 -> xyz=0 -0.187 -0.016 rpy=0 -0 0
- joint l_arm_lwy: origin xyz=0 0 0 rpy=0 0 0 -> xyz=0 0 0 rpy=0 3.14159265359 0
- joint l_arm_mwx: origin xyz=0 0.119 0.0092 rpy=0 -0 0 -> xyz=0 -0.119 0.0092 rpy=0 -0 0
- joint l_arm_shx: axis 1 0 0 -> -1.0 -0.0 -0.0; origin xyz=0 0.11 -0.245 rpy=0 -0 0 -> xyz=0 -0.11 -0.245 rpy=0 -0 0
- joint l_arm_shz: origin xyz=0.1406 0.2256 0.4776 rpy=0 -0 0 -> xyz=0.1406 0.2256 0.4776 rpy=0 0 3.14159265359
- joint l_arm_uwy: axis 0 1 0 -> -0.0 -1.0 -0.0; origin xyz=0 0.187 -0.0092 rpy=0 -0 0 -> xyz=0 -0.187 -0.0092 rpy=0 3.14159265359 0

File: software/models/atlas_v4/components/atlas_v4_full_collision_geometry.urdf (robot description, URDF)
Before this commit: robot drc_skeleton, 34 links, 34 joints
Links:
- link l_clav: geometry collision box size=0.1 0.07 0.072; collision cylinder length=0.1525 radius=0.0555
- link l_larm: geometry collision box size=0.135 0.15 0.06; collision cylinder length=0.125 radius=0.045
- link l_lfarm: geometry collision box size=0.13 0.09 0.07; collision cylinder length=0.05 radius=0.03
- link l_scap: geometry collision box size=0.02 0.029 0.018; collision box size=0.028 0.090 0.05
- link l_uarm: geometry collision box size=0.05 0.07 0.15; collision cylinder length=0.11 radius=0.065
- link l_ufarm: geometry collision box size=0.135 0.1 0.045; collision cylinder length=0.125 radius=0.045
Joints:
- joint l_arm_elx: axis 1 0 0 -> -1.0 -0.0 -0.0; origin xyz=0 0.119 0.0092 rpy=0 -0 0 -> xyz=0 -0.119 0.0092 rpy=0 -0 0
- joint l_arm_ely: axis 0 1 0 -> -0.0 -1.0 -0.0; origin xyz=0 0.187 -0.016 rpy=0 -0 0 -> xyz=0 -0.187 -0.016 rpy=0 -0 0
- joint l_arm_lwy: origin xyz=0 0 0 rpy=0 0 0 -> xyz=0 0 0 rpy=0 3.14159265359 0
- joint l_arm_mwx: origin xyz=0 0.119 0.0092 rpy=0 -0 0 -> xyz=0 -0.119 0.0092 rpy=0 -0 0
- joint l_arm_shx: axis 1 0 0 -> -1.0 -0.0 -0.0; origin xyz=0 0.11 -0.245 rpy=0 -0 0 -> xyz=0 -0.11 -0.245 rpy=0 -0 0
- joint l_arm_shz: origin xyz=0.1406 0.2256 0.4776 rpy=0 -0 0 -> xyz=0.1406 0.2256 0.4776 rpy=0 0 3.14159265359
- joint l_arm_uwy: axis 0 1 0 -> -0.0 -1.0 -0.0; origin xyz=0 0.187 -0.0092 rpy=0 -0 0 -> xyz=0 -0.187 -0.0092 rpy=0 3.14159265359 0

File: software/models/atlas_v4/components/atlas_v4_minimal_contact.urdf (robot description, URDF)
Before this commit: robot drc_skeleton, 34 links, 34 joints
Links:
- link l_clav: geometry visual mesh filename=package://atlas_v4/meshes/r_clav.obj scale=1 1 1
- link l_larm: geometry visual mesh filename=package://atlas_v4/meshes/r_larm.obj scale=1 1 1
- link l_lfarm: geometry visual mesh filename=package://atlas_v4/meshes/r_hand.obj scale=1 1 1
- link l_scap: geometry visual mesh filename=package://atlas_v4/meshes/r_scap.obj scale=1 1 1
- link l_uarm: geometry visual mesh filename=package://atlas_v4/meshes/r_uarm.obj scale=1 1 1
- link l_ufarm: geometry visual mesh filename=package://atlas_v4/meshes/r_farm.obj scale=1 1 1
Joints:
- joint l_arm_elx: axis 1 0 0 -> -1.0 -0.0 -0.0; origin xyz=0 0.119 0.0092 rpy=0 -0 0 -> xyz=0 -0.119 0.0092 rpy=0 -0 0
- joint l_arm_ely: axis 0 1 0 -> -0.0 -1.0 -0.0; origin xyz=0 0.187 -0.016 rpy=0 -0 0 -> xyz=0 -0.187 -0.016 rpy=0 -0 0
- joint l_arm_lwy: origin xyz=0 0 0 rpy=0 0 0 -> xyz=0 0 0 rpy=0 3.14159265359 0
- joint l_arm_mwx: origin xyz=0 0.119 0.0092 rpy=0 -0 0 -> xyz=0 -0.119 0.0092 rpy=0 -0 0
- joint l_arm_shx: axis 1 0 0 -> -1.0 -0.0 -0.0; origin xyz=0 0.11 -0.245 rpy=0 -0 0 -> xyz=0 -0.11 -0.245 rpy=0 -0 0
- joint l_arm_shz: origin xyz=0.1406 0.2256 0.4776 rpy=0 -0 0 -> xyz=0.1406 0.2256 0.4776 rpy=0 0 3.14159265359
- joint l_arm_uwy: axis 0 1 0 -> -0.0 -1.0 -0.0; origin xyz=0 0.187 -0.0092 rpy=0 -0 0 -> xyz=0 -0.187 -0.0092 rpy=0 3.14159265359 0

File: software/models/atlas_v4/model_LR_RR.urdf (robot description, URDF)
Before this commit: robot atlas, 86 links, 85 joints
Links:
- link l_clav: geometry collision box size=0.1 0.07 0.072; collision cylinder length=0.1525 radius=0.0555
- link l_larm: geometry collision box size=0.135 0.15 0.06; collision cylinder length=0.125 radius=0.045
- link l_lfarm: geometry collision box size=0.13 0.09 0.07; collision cylinder length=0.05 radius=0.03
- link l_scap: geometry collision box size=0.02 0.029 0.018; collision box size=0.028 0.090 0.05
- link l_uarm: geometry collision box size=0.05 0.07 0.15; collision cylinder length=0.11 radius=0.065
- link l_ufarm: geometry collision box size=0.135 0.1 0.045; collision cylinder length=0.125 radius=0.045
Joints:
- joint l_arm_elx: axis 1 0 0 -> -1.0 -0.0 -0.0; origin xyz=0 0.119 0.0092 rpy=0 -0 0 -> xyz=0 -0.119 0.0092 rpy=0 -0 0
- joint l_arm_ely: axis 0 1 0 -> -0.0 -1.0 -0.0; origin xyz=0 0.187 -0.016 rpy=0 -0 0 -> xyz=0 -0.187 -0.016 rpy=0 -0 0
- joint l_arm_lwy: origin xyz=0 0 0 rpy=0 0 0 -> xyz=0 0 0 rpy=0 3.14159265359 0
- joint l_arm_mwx: origin xyz=0 0.119 0.0092 rpy=0 -0 0 -> xyz=0 -0.119 0.0092 rpy=0 -0 0
- joint l_arm_shx: axis 1 0 0 -> -1.0 -0.0 -0.0; origin xyz=0 0.11 -0.245 rpy=0 -0 0 -> xyz=0 -0.11 -0.245 rpy=0 -0 0
- joint l_arm_shz: origin xyz=0.1406 0.2256 0.4776 rpy=0 -0 0 -> xyz=0.1406 0.2256 0.4776 rpy=0 0 3.14159265359
- joint l_arm_uwy: axis 0 1 0 -> -0.0 -1.0 -0.0; origin xyz=0 0.187 -0.0092 rpy=0 -0 0 -> xyz=0 -0.187 -0.0092 rpy=0 3.14159265359 0
- joint l_hand_force_torque_joint: origin xyz=0 0.1245 0.0112 rpy=0 0 0 -> xyz=0 -0.1245 0.0112 rpy=0 0 3.141592
- joint r_hand_force_torque_joint: origin xyz=0 -0.1245 -0.0112 rpy=0 0 3.142 -> xyz=0 -0.1245 -0.0112 rpy=0 0 3.141592

File: software/models/atlas_v4/model_convex_hull.urdf (robot description, URDF)
Before this commit: robot atlas, 70 links, 69 joints
Links:
- link l_clav: geometry collision mesh filename=package://atlas_v4/meshes/r_clav_chull.obj scale=1 1 1; visual mesh filename=package://atlas_v4/meshes/r_clav.obj scale=1 1 1
- link l_larm: geometry collision mesh filename=package://atlas_v4/meshes/r_larm_chull.obj scale=1 1 1; visual mesh filename=package://atlas_v4/meshes/r_larm.obj scale=1 1 1
- link l_lfarm: geometry collision mesh filename=package://atlas_v4/meshes/r_hand_chull.obj scale=1 1 1; visual mesh filename=package://atlas_v4/meshes/r_hand.obj scale=1 1 1
- link l_scap: geometry collision mesh filename=package://atlas_v4/meshes/r_scap_chull.obj scale=1 1 1; visual mesh filename=package://atlas_v4/meshes/r_scap.obj scale=1 1 1
- link l_uarm: geometry collision mesh filename=package://atlas_v4/meshes/r_uarm_chull.obj scale=1 1 1; visual mesh filename=package://atlas_v4/meshes/r_uarm.obj scale=1 1 1
- link l_ufarm: geometry collision mesh filename=package://atlas_v4/meshes/r_farm_chull.obj scale=1 1 1; visual mesh filename=package://atlas_v4/meshes/r_farm.obj scale=1 1 1
Joints:
- joint l_arm_elx: axis 1 0 0 -> -1.0 -0.0 -0.0; origin xyz=0 0.119 0.0092 rpy=0 -0 0 -> xyz=0 -0.119 0.0092 rpy=0 -0 0
- joint l_arm_ely: axis 0 1 0 -> -0.0 -1.0 -0.0; origin xyz=0 0.187 -0.016 rpy=0 -0 0 -> xyz=0 -0.187 -0.016 rpy=0 -0 0
- joint l_arm_lwy: origin xyz=0 0 0 rpy=0 0 0 -> xyz=0 0 0 rpy=0 3.14159265359 0
- joint l_arm_mwx: origin xyz=0 0.119 0.0092 rpy=0 -0 0 -> xyz=0 -0.119 0.0092 rpy=0 -0 0
- joint l_arm_shx: axis 1 0 0 -> -1.0 -0.0 -0.0; origin xyz=0 0.11 -0.245 rpy=0 -0 0 -> xyz=0 -0.11 -0.245 rpy=0 -0 0
- joint l_arm_shz: origin xyz=0.1406 0.2256 0.4776 rpy=0 -0 0 -> xyz=0.1406 0.2256 0.4776 rpy=0 0 3.14159265359
- joint l_arm_uwy: axis 0 1 0 -> -0.0 -1.0 -0.0; origin xyz=0 0.187 -0.0092 rpy=0 -0 0 -> xyz=0 -0.187 -0.0092 rpy=0 3.14159265359 0
- joint l_hand_force_torque_joint: origin xyz=0 0.1245 0.0112 rpy=0 0 0 -> xyz=0 -0.1245 0.0112 rpy=0 0 3.141592
- joint r_hand_force_torque_joint: origin xyz=0 -0.1245 -0.0112 rpy=0 0 3.142 -> xyz=0 -0.1245 -0.0112 rpy=0 0 3.141592

File: software/models/atlas_v4/model_convex_hull_closed_hands.urdf (robot description, URDF)
Before this commit: robot atlas, 70 links, 69 joints
Links:
- link l_clav: geometry collision mesh filename=package://atlas_v4/meshes/r_clav_chull.obj scale=1 1 1; visual mesh filename=package://atlas_v4/meshes/r_clav.obj scale=1 1 1
- link l_larm: geometry collision mesh filename=package://atlas_v4/meshes/r_larm_chull.obj scale=1 1 1; visual mesh filename=package://atlas_v4/meshes/r_larm.obj scale=1 1 1
- link l_lfarm: geometry collision mesh filename=package://atlas_v4/meshes/r_hand_chull.obj scale=1 1 1; visual mesh filename=package://atlas_v4/meshes/r_hand.obj scale=1 1 1
- link l_scap: geometry collision mesh filename=package://atlas_v4/meshes/r_scap_chull.obj scale=1 1 1; visual mesh filename=package://atlas_v4/meshes/r_scap.obj scale=1 1 1
- link l_uarm: geometry collision mesh filename=package://atlas_v4/meshes/r_uarm_chull.obj scale=1 1 1; visual mesh filename=package://atlas_v4/meshes/r_uarm.obj scale=1 1 1
- link l_ufarm: geometry collision mesh filename=package://atlas_v4/meshes/r_farm_chull.obj scale=1 1 1; visual mesh filename=package://atlas_v4/meshes/r_farm.obj scale=1 1 1
Joints:
- joint l_arm_elx: axis 1 0 0 -> -1.0 -0.0 -0.0; origin xyz=0 0.119 0.0092 rpy=0 -0 0 -> xyz=0 -0.119 0.0092 rpy=0 -0 0
- joint l_arm_ely: axis 0 1 0 -> -0.0 -1.0 -0.0; origin xyz=0 0.187 -0.016 rpy=0 -0 0 -> xyz=0 -0.187 -0.016 rpy=0 -0 0
- joint l_arm_lwy: origin xyz=0 0 0 rpy=0 0 0 -> xyz=0 0 0 rpy=0 3.14159265359 0
- joint l_arm_mwx: origin xyz=0 0.119 0.0092 rpy=0 -0 0 -> xyz=0 -0.119 0.0092 rpy=0 -0 0
- joint l_arm_shx: axis 1 0 0 -> -1.0 -0.0 -0.0; origin xyz=0 0.11 -0.245 rpy=0 -0 0 -> xyz=0 -0.11 -0.245 rpy=0 -0 0
- joint l_arm_shz: origin xyz=0.1406 0.2256 0.4776 rpy=0 -0 0 -> xyz=0.1406 0.2256 0.4776 rpy=0 0 3.14159265359
- joint l_arm_uwy: axis 0 1 0 -> -0.0 -1.0 -0.0; origin xyz=0 0.187 -0.0092 rpy=0 -0 0 -> xyz=0 -0.187 -0.0092 rpy=0 3.14159265359 0
- joint l_hand_force_torque_joint: origin xyz=0 0.1245 0.0112 rpy=0 0 0 -> xyz=0 -0.1245 0.0112 rpy=0 0 3.141592
- joint r_hand_force_torque_joint: origin xyz=0 -0.1245 -0.0112 rpy=0 0 3.142 -> xyz=0 -0.1245 -0.0112 rpy=0 0 3.141592

File: software/models/atlas_v4/model_convex_hull_fingers.urdf (robot description, URDF)
Before this commit: robot atlas, 94 links, 93 joints
Links:
- link l_clav: geometry collision mesh filename=package://atlas_v4/meshes/r_clav_chull.obj scale=1 1 1; visual mesh filename=package://atlas_v4/meshes/r_clav.obj scale=1 1 1
- link l_larm: geometry collision mesh filename=package://atlas_v4/meshes/r_larm_chull.obj scale=1 1 1; visual mesh filename=package://atlas_v4/meshes/r_larm.obj scale=1 1 1
- link l_lfarm: geometry collision mesh filename=package://atlas_v4/meshes/r_hand_chull.obj scale=1 1 1; visual mesh filename=package://atlas_v4/meshes/r_hand.obj scale=1 1 1
- link l_scap: geometry collision mesh filename=package://atlas_v4/meshes/r_scap_chull.obj scale=1 1 1; visual mesh filename=package://atlas_v4/meshes/r_scap.obj scale=1 1 1
- link l_uarm: geometry collision mesh filename=package://atlas_v4/meshes/r_uarm_chull.obj scale=1 1 1; visual mesh filename=package://atlas_v4/meshes/r_uarm.obj scale=1 1 1
- link l_ufarm: geometry collision mesh filename=package://atlas_v4/meshes/r_farm_chull.obj scale=1 1 1; visual mesh filename=package://atlas_v4/meshes/r_farm.obj scale=1 1 1
Joints:
- joint l_arm_elx: axis 1 0 0 -> -1.0 -0.0 -0.0; origin xyz=0 0.119 0.0092 rpy=0 -0 0 -> xyz=0 -0.119 0.0092 rpy=0 -0 0
- joint l_arm_ely: axis 0 1 0 -> -0.0 -1.0 -0.0; origin xyz=0 0.187 -0.016 rpy=0 -0 0 -> xyz=0 -0.187 -0.016 rpy=0 -0 0
- joint l_arm_lwy: origin xyz=0 0 0 rpy=0 0 0 -> xyz=0 0 0 rpy=0 3.14159265359 0
- joint l_arm_mwx: origin xyz=0 0.119 0.0092 rpy=0 -0 0 -> xyz=0 -0.119 0.0092 rpy=0 -0 0
- joint l_arm_shx: axis 1 0 0 -> -1.0 -0.0 -0.0; origin xyz=0 0.11 -0.245 rpy=0 -0 0 -> xyz=0 -0.11 -0.245 rpy=0 -0 0
- joint l_arm_shz: origin xyz=0.1406 0.2256 0.4776 rpy=0 -0 0 -> xyz=0.1406 0.2256 0.4776 rpy=0 0 3.14159265359
- joint l_arm_uwy: axis 0 1 0 -> -0.0 -1.0 -0.0; origin xyz=0 0.187 -0.0092 rpy=0 -0 0 -> xyz=0 -0.187 -0.0092 rpy=0 3.14159265359 0
- joint l_hand_force_torque_joint: origin xyz=0 0.1245 0.0112 rpy=0 0 0 -> xyz=0 -0.1245 0.0112 rpy=0 0 3.141592
- joint r_hand_force_torque_joint: origin xyz=0 -0.1245 -0.0112 rpy=0 0 3.142 -> xyz=0 -0.1245 -0.0112 rpy=0 0 3.141592

File: software/models/atlas_v4/model_minimal_contact.urdf (robot description, URDF)
Before this commit: robot atlas, 94 links, 93 joints
Links:
- link l_clav: geometry visual mesh filename=package://atlas_v4/meshes/r_clav.obj scale=1 1 1
- link l_larm: geometry visual mesh filename=package://atlas_v4/meshes/r_larm.obj scale=1 1 1
- link l_lfarm: geometry visual mesh filename=package://atlas_v4/meshes/r_hand.obj scale=1 1 1
- link l_scap: geometry visual mesh filename=package://atlas_v4/meshes/r_scap.obj scale=1 1 1
- link l_uarm: geometry visual mesh filename=package://atlas_v4/meshes/r_uarm.obj scale=1 1 1
- link l_ufarm: geometry visual mesh filename=package://atlas_v4/meshes/r_farm.obj scale=1 1 1
Joints:
- joint l_arm_elx: axis 1 0 0 -> -1.0 -0.0 -0.0; origin xyz=0 0.119 0.0092 rpy=0 -0 0 -> xyz=0 -0.119 0.0092 rpy=0 -0 0
- joint l_arm_ely: axis 0 1 0 -> -0.0 -1.0 -0.0; origin xyz=0 0.187 -0.016 rpy=0 -0 0 -> xyz=0 -0.187 -0.016 rpy=0 -0 0
- joint l_arm_lwy: origin xyz=0 0 0 rpy=0 0 0 -> xyz=0 0 0 rpy=0 3.14159265359 0
- joint l_arm_mwx: origin xyz=0 0.119 0.0092 rpy=0 -0 0 -> xyz=0 -0.119 0.0092 rpy=0 -0 0
- joint l_arm_shx: axis 1 0 0 -> -1.0 -0.0 -0.0; origin xyz=0 0.11 -0.245 rpy=0 -0 0 -> xyz=0 -0.11 -0.245 rpy=0 -0 0
- joint l_arm_shz: origin xyz=0.1406 0.2256 0.4776 rpy=0 -0 0 -> xyz=0.1406 0.2256 0.4776 rpy=0 0 3.14159265359
- joint l_arm_uwy: axis 0 1 0 -> -0.0 -1.0 -0.0; origin xyz=0 0.187 -0.0092 rpy=0 -0 0 -> xyz=0 -0.187 -0.0092 rpy=0 3.14159265359 0
- joint l_hand_force_torque_joint: origin xyz=0 0.1245 0.0112 rpy=0 0 0 -> xyz=0 -0.1245 0.0112 rpy=0 0 3.141592
- joint r_hand_force_torque_joint: origin xyz=0 -0.1245 -0.0112 rpy=0 0 3.142 -> xyz=0 -0.1245 -0.0112 rpy=0 0 3.141592

File: software/models/common_components/hand_force_torque.urdf (robot description, URDF)
Before this commit: robot hand_force_torque, 2 links, 2 joints
Joints:
- joint l_hand_force_torque_joint: origin xyz=0 0.1245 0.0112 rpy=0 0 0 -> xyz=0 -0.1245 0.0112 rpy=0 0 3.141592
- joint r_hand_force_torque_joint: origin xyz=0 -0.1245 -0.0112 rpy=0 0 3.142 -> xyz=0 -0.1245 -0.0112 rpy=0 0 3.141592

Commit message: Update generated files for V4

File: software/models/atlas_v4/components/atlas_v4_convex_hull.urdf (robot description, URDF)
Before this commit: robot drc_skeleton, 34 links, 34 joints
Links:
- link l_foot: geometry collision mesh filename=package://atlas_v4/meshes/l_foot_chull.obj scale=1 1 1; collision sphere radius=0.0
- link r_foot: geometry collision mesh filename=package://atlas_v4/meshes/r_foot_chull.obj scale=1 1 1; collision sphere radius=0.0

File: software/models/atlas_v4/model_convex_hull.urdf (robot description, URDF)
Before this commit: robot atlas, 70 links, 69 joints
Links:
- link l_foot: geometry collision mesh filename=package://atlas_v4/meshes/l_foot_chull.obj scale=1 1 1; collision sphere radius=0.0
- link r_foot: geometry collision mesh filename=package://atlas_v4/meshes/r_foot_chull.obj scale=1 1 1; collision sphere radius=0.0

File: software/models/atlas_v4/model_convex_hull_closed_hands.urdf (robot description, URDF)
Before this commit: robot atlas, 70 links, 69 joints
Links:
- link l_foot: geometry collision mesh filename=package://atlas_v4/meshes/l_foot_chull.obj scale=1 1 1; collision sphere radius=0.0
- link r_foot: geometry collision mesh filename=package://atlas_v4/meshes/r_foot_chull.obj scale=1 1 1; collision sphere radius=0.0

File: software/models/atlas_v4/model_convex_hull_fingers.urdf (robot description, URDF)
Before this commit: robot atlas, 94 links, 93 joints
Links:
- link l_foot: geometry collision mesh filename=package://atlas_v4/meshes/l_foot_chull.obj scale=1 1 1; collision sphere radius=0.0
- link r_foot: geometry collision mesh filename=package://atlas_v4/meshes/r_foot_chull.obj scale=1 1 1; collision sphere radius=0.0

Commit message: add midfoot contacts we can use for walking on stairs

File: software/models/atlas_v4/components/atlas_v4_convex_hull.urdf (robot description, URDF)
Before this commit: robot drc_skeleton, 34 links, 34 joints
Links:
- link l_foot: geometry collision mesh filename=package://atlas_v4/meshes/l_foot_chull.obj scale=1 1 1; collision sphere radius=0.0
- link r_foot: geometry collision mesh filename=package://atlas_v4/meshes/r_foot_chull.obj scale=1 1 1; collision sphere radius=0.0

File: software/models/atlas_v4/components/atlas_v4_minimal_contact.urdf (robot description, URDF)
Before this commit: robot drc_skeleton, 34 links, 34 joints
Links:
- link l_foot: geometry collision sphere radius=0.0; collision sphere radius=0.0
- link r_foot: geometry collision sphere radius=0.0; collision sphere radius=0.0

File: software/models/atlas_v4/model_convex_hull.urdf (robot description, URDF)
Before this commit: robot atlas, 70 links, 69 joints
Links:
- link l_foot: geometry collision mesh filename=package://atlas_v4/meshes/l_foot_chull.obj scale=1 1 1; collision sphere radius=0.0
- link r_foot: geometry collision mesh filename=package://atlas_v4/meshes/r_foot_chull.obj scale=1 1 1; collision sphere radius=0.0

File: software/models/atlas_v4/model_convex_hull_closed_hands.urdf (robot description, URDF)
Before this commit: robot atlas, 70 links, 69 joints
Links:
- link l_foot: geometry collision mesh filename=package://atlas_v4/meshes/l_foot_chull.obj scale=1 1 1; collision sphere radius=0.0
- link r_foot: geometry collision mesh filename=package://atlas_v4/meshes/r_foot_chull.obj scale=1 1 1; collision sphere radius=0.0

File: software/models/atlas_v4/model_convex_hull_fingers.urdf (robot description, URDF)
Before this commit: robot atlas, 94 links, 93 joints
Links:
- link l_foot: geometry collision mesh filename=package://atlas_v4/meshes/l_foot_chull.obj scale=1 1 1; collision sphere radius=0.0
- link r_foot: geometry collision mesh filename=package://atlas_v4/meshes/r_foot_chull.obj scale=1 1 1; collision sphere radius=0.0

File: software/models/atlas_v4/model_minimal_contact.urdf (robot description, URDF)
Before this commit: robot atlas, 94 links, 93 joints
Links:
- link l_foot: geometry collision sphere radius=0.0; collision sphere radius=0.0
- link r_foot: geometry collision sphere radius=0.0; collision sphere radius=0.0

File: software/models/atlas_v5/components/atlas_v5_convex_hull.urdf (robot description, URDF)
Before this commit: robot drc_skeleton, 34 links, 34 joints
Links:
- link l_foot: geometry collision mesh filename=package://atlas_v5/meshes/l_foot_chull.obj; collision sphere radius=0.0
- link r_foot: geometry collision mesh filename=package://atlas_v5/meshes/r_foot_chull.obj; collision sphere radius=0.0

File: software/models/atlas_v5/components/atlas_v5_minimal_contact.urdf (robot description, URDF)
Before this commit: robot drc_skeleton, 34 links, 34 joints
Links:
- link l_foot: geometry collision sphere radius=0.0; collision sphere radius=0.0
- link r_foot: geometry collision sphere radius=0.0; collision sphere radius=0.0

File: software/models/atlas_v5/model_convex_hull.urdf (robot description, URDF)
Before this commit: robot atlas, 70 links, 69 joints
Links:
- link l_foot: geometry collision mesh filename=package://atlas_v5/meshes/l_foot_chull.obj; collision sphere radius=0.0
- link r_foot: geometry collision mesh filename=package://atlas_v5/meshes/r_foot_chull.obj; collision sphere radius=0.0

File: software/models/atlas_v5/model_convex_hull_closed_hands.urdf (robot description, URDF)
Before this commit: robot atlas, 70 links, 69 joints
Links:
- link l_foot: geometry collision mesh filename=package://atlas_v5/meshes/l_foot_chull.obj; collision sphere radius=0.0
- link r_foot: geometry collision mesh filename=package://atlas_v5/meshes/r_foot_chull.obj; collision sphere radius=0.0

File: software/models/atlas_v5/model_convex_hull_fingers.urdf (robot description, URDF)
Before this commit: robot atlas, 94 links, 93 joints
Links:
- link l_foot: geometry collision mesh filename=package://atlas_v5/meshes/l_foot_chull.obj; collision sphere radius=0.0
- link r_foot: geometry collision mesh filename=package://atlas_v5/meshes/r_foot_chull.obj; collision sphere radius=0.0

File: software/models/atlas_v5/model_minimal_contact.urdf (robot description, URDF)
Before this commit: robot atlas, 94 links, 93 joints
Links:
- link l_foot: geometry collision sphere radius=0.0; collision sphere radius=0.0
- link r_foot: geometry collision sphere radius=0.0; collision sphere radius=0.0
