Commit message: Update generated files

File: software/models/atlas_v5/components/atlas_v5_full_collision_geometry.urdf (robot description, URDF)
Before this commit: robot drc_skeleton, 34 links, 34 joints
Links:
- link l_clav: geometry collision mesh filename=package://atlas_v5/meshes/r_clav_chull.obj; visual mesh filename=package://atlas_v5/meshes/r_clav.obj
- link l_foot: geometry collision mesh filename=package://atlas_v5/meshes/l_foot_chull.obj; collision sphere radius=0.0
- link l_larm: geometry collision box size=0.15000 0.20000 0.15000; collision mesh filename=package://atlas_v5/meshes/r_larm_chull.obj
- link l_lfarm: geometry collision mesh filename=package://atlas_v5/meshes/r_hand_chull.obj; visual mesh filename=package://atlas_v5/meshes/r_hand.obj
- link l_lglut: geometry collision mesh filename=package://atlas_v5/meshes/l_lglut_chull.obj; visual mesh filename=package://atlas_v5/meshes/l_lglut.obj
- link l_lleg: geometry collision mesh filename=package://atlas_v5/meshes/l_lleg_chull.obj; visual mesh filename=package://atlas_v5/meshes/l_lleg.obj
- link l_scap: geometry collision mesh filename=package://atlas_v5/meshes/r_scap_chull.obj; visual mesh filename=package://atlas_v5/meshes/r_scap.obj
- link l_situational_awareness_camera_link: geometry collision box size=0.01 0.01 0.01; visual box size=0.01 0.01 0.01
- link l_uarm: geometry collision mesh filename=package://atlas_v5/meshes/r_uarm_chull.obj; visual mesh filename=package://atlas_v5/meshes/r_uarm.obj
- link l_ufarm: geometry collision mesh filename=package://atlas_v5/meshes/r_farm_chull.obj; visual mesh filename=package://atlas_v5/meshes/r_farm.obj
- link l_uglut: geometry collision mesh filename=package://atlas_v5/meshes/l_uglut_chull.obj; visual mesh filename=package://atlas_v5/meshes/l_uglut.obj
- link l_uleg: geometry collision mesh filename=package://atlas_v5/meshes/l_uleg_chull.obj; visual mesh filename=package://atlas_v5/meshes/l_uleg.obj
- link pelvis: geometry collision mesh filename=package://atlas_v5/meshes/pelvis_chull.obj; visual mesh filename=package://atlas_v5/meshes/pelvis.obj
- link r_clav: geometry collision mesh filename=package://atlas_v5/meshes/r_clav_chull.obj; visual mesh filename=package://atlas_v5/meshes/r_clav.obj
- link r_foot: geometry collision mesh filename=package://atlas_v5/meshes/r_foot_chull.obj; collision sphere radius=0.0
- link r_larm: geometry collision box size=0.15000 0.20000 0.15000; collision mesh filename=package://atlas_v5/meshes/r_larm_chull.obj
- link r_lfarm: geometry collision mesh filename=package://atlas_v5/meshes/r_hand_chull.obj; visual mesh filename=package://atlas_v5/meshes/r_hand.obj
- link r_lglut: geometry collision mesh filename=package://atlas_v5/meshes/r_lglut_chull.obj; visual mesh filename=package://atlas_v5/meshes/r_lglut.obj
- link r_lleg: geometry collision mesh filename=package://atlas_v5/meshes/r_lleg_chull.obj; visual mesh filename=package://atlas_v5/meshes/r_lleg.obj
- link r_scap: geometry collision mesh filename=package://atlas_v5/meshes/r_scap_chull.obj; visual mesh filename=package://atlas_v5/meshes/r_scap.obj
- link r_situational_awareness_camera_link: geometry collision box size=0.01 0.01 0.01; visual box size=0.01 0.01 0.01
- link r_uarm: geometry collision mesh filename=package://atlas_v5/meshes/r_uarm_chull.obj; visual mesh filename=package://atlas_v5/meshes/r_uarm.obj
- link r_ufarm: geometry collision mesh filename=package://atlas_v5/meshes/r_farm_chull.obj; visual mesh filename=package://atlas_v5/meshes/r_farm.obj
- link r_uglut: geometry collision mesh filename=package://atlas_v5/meshes/r_uglut_chull.obj; visual mesh filename=package://atlas_v5/meshes/r_uglut.obj
- link r_uleg: geometry collision mesh filename=package://atlas_v5/meshes/r_uleg_chull.obj; visual mesh filename=package://atlas_v5/meshes/r_uleg.obj
- link utorso: geometry collision mesh filename=package://atlas_v5/meshes/utorso_chull.obj; visual mesh filename=package://atlas_v5/meshes/utorso.obj

File: software/models/atlas_v5/model_LR_RR.urdf (robot description, URDF)
Before this commit: robot atlas, 88 links, 87 joints
Links:
- link l_clav: geometry collision mesh filename=package://atlas_v5/meshes/r_clav_chull.obj; visual mesh filename=package://atlas_v5/meshes/r_clav.obj
- link l_foot: geometry collision mesh filename=package://atlas_v5/meshes/l_foot_chull.obj; collision sphere radius=0.0
- link l_larm: geometry collision box size=0.15000 0.20000 0.15000; collision mesh filename=package://atlas_v5/meshes/r_larm_chull.obj
- link l_lfarm: geometry collision mesh filename=package://atlas_v5/meshes/r_hand_chull.obj; visual mesh filename=package://atlas_v5/meshes/r_hand.obj
- link l_lglut: geometry collision mesh filename=package://atlas_v5/meshes/l_lglut_chull.obj; visual mesh filename=package://atlas_v5/meshes/l_lglut.obj
- link l_lleg: geometry collision mesh filename=package://atlas_v5/meshes/l_lleg_chull.obj; visual mesh filename=package://atlas_v5/meshes/l_lleg.obj
- link l_scap: geometry collision mesh filename=package://atlas_v5/meshes/r_scap_chull.obj; visual mesh filename=package://atlas_v5/meshes/r_scap.obj
- link l_situational_awareness_camera_link: geometry collision box size=0.01 0.01 0.01; visual box size=0.01 0.01 0.01
- link l_uarm: geometry collision mesh filename=package://atlas_v5/meshes/r_uarm_chull.obj; visual mesh filename=package://atlas_v5/meshes/r_uarm.obj
- link l_ufarm: geometry collision mesh filename=package://atlas_v5/meshes/r_farm_chull.obj; visual mesh filename=package://atlas_v5/meshes/r_farm.obj
- link l_uglut: geometry collision mesh filename=package://atlas_v5/meshes/l_uglut_chull.obj; visual mesh filename=package://atlas_v5/meshes/l_uglut.obj
- link l_uleg: geometry collision mesh filename=package://atlas_v5/meshes/l_uleg_chull.obj; visual mesh filename=package://atlas_v5/meshes/l_uleg.obj
- link pelvis: geometry collision mesh filename=package://atlas_v5/meshes/pelvis_chull.obj; visual mesh filename=package://atlas_v5/meshes/pelvis.obj
- link r_clav: geometry collision mesh filename=package://atlas_v5/meshes/r_clav_chull.obj; visual mesh filename=package://atlas_v5/meshes/r_clav.obj
- link r_foot: geometry collision mesh filename=package://atlas_v5/meshes/r_foot_chull.obj; collision sphere radius=0.0
- link r_larm: geometry collision box size=0.15000 0.20000 0.15000; collision mesh filename=package://atlas_v5/meshes/r_larm_chull.obj
- link r_lfarm: geometry collision mesh filename=package://atlas_v5/meshes/r_hand_chull.obj; visual mesh filename=package://atlas_v5/meshes/r_hand.obj
- link r_lglut: geometry collision mesh filename=package://atlas_v5/meshes/r_lglut_chull.obj; visual mesh filename=package://atlas_v5/meshes/r_lglut.obj
- link r_lleg: geometry collision mesh filename=package://atlas_v5/meshes/r_lleg_chull.obj; visual mesh filename=package://atlas_v5/meshes/r_lleg.obj
- link r_scap: geometry collision mesh filename=package://atlas_v5/meshes/r_scap_chull.obj; visual mesh filename=package://atlas_v5/meshes/r_scap.obj
- link r_situational_awareness_camera_link: geometry collision box size=0.01 0.01 0.01; visual box size=0.01 0.01 0.01
- link r_uarm: geometry collision mesh filename=package://atlas_v5/meshes/r_uarm_chull.obj; visual mesh filename=package://atlas_v5/meshes/r_uarm.obj
- link r_ufarm: geometry collision mesh filename=package://atlas_v5/meshes/r_farm_chull.obj; visual mesh filename=package://atlas_v5/meshes/r_farm.obj
- link r_uglut: geometry collision mesh filename=package://atlas_v5/meshes/r_uglut_chull.obj; visual mesh filename=package://atlas_v5/meshes/r_uglut.obj
- link r_uleg: geometry collision mesh filename=package://atlas_v5/meshes/r_uleg_chull.obj; visual mesh filename=package://atlas_v5/meshes/r_uleg.obj
- link utorso: geometry collision mesh filename=package://atlas_v5/meshes/utorso_chull.obj; visual mesh filename=package://atlas_v5/meshes/utorso.obj

Commit message: Update generated files for removed contact pts

File: software/models/atlas_v5/components/atlas_v5_full_collision_geometry.urdf (robot description, URDF)
Before this commit: robot drc_skeleton, 34 links, 34 joints
Links:
- link l_foot: geometry collision mesh filename=package://atlas_v5/meshes/l_foot_chull.obj; visual mesh filename=package://atlas_v5/meshes/l_foot.obj
- link r_foot: geometry collision mesh filename=package://atlas_v5/meshes/r_foot_chull.obj; visual mesh filename=package://atlas_v5/meshes/r_foot.obj

File: software/models/atlas_v5/model_LR_RR.urdf (robot description, URDF)
Before this commit: robot atlas, 88 links, 87 joints
Links:
- link l_foot: geometry collision mesh filename=package://atlas_v5/meshes/l_foot_chull.obj; visual mesh filename=package://atlas_v5/meshes/l_foot.obj
- link r_foot: geometry collision mesh filename=package://atlas_v5/meshes/r_foot_chull.obj; visual mesh filename=package://atlas_v5/meshes/r_foot.obj
