Commit message: Update generated files for atlas_v4/5

File: software/models/atlas_v5/components/atlas_v5_convex_hull.urdf (robot description, URDF)
Before this commit: robot drc_skeleton, 36 links, 36 joints
Links:
- link l_clav: geometry collision mesh filename=package://atlas_v5/meshes/l_clav_chull.obj; visual mesh filename=package://atlas_v5/meshes/l_clav.obj
- link l_foot: geometry collision mesh filename=package://atlas_v5/meshes/l_foot_chull.obj; collision sphere radius=0.0
- link l_larm: geometry collision mesh filename=package://atlas_v5/meshes/l_larm_chull.obj; visual mesh filename=package://atlas_v5/meshes/l_larm.obj
- link l_lfarm: geometry collision mesh filename=package://atlas_v5/meshes/l_hand_chull.obj; visual mesh filename=package://atlas_v5/meshes/l_hand.obj
- link l_lglut: geometry collision mesh filename=package://atlas_v5/meshes/l_lglut_chull.obj; visual mesh filename=package://atlas_v5/meshes/l_lglut.obj
- link l_lleg: geometry collision mesh filename=package://atlas_v5/meshes/l_lleg_chull.obj; visual mesh filename=package://atlas_v5/meshes/l_lleg.obj
- link l_scap: geometry collision mesh filename=package://atlas_v5/meshes/l_scap_chull.obj; visual mesh filename=package://atlas_v5/meshes/l_scap.obj
- link l_uarm: geometry collision mesh filename=package://atlas_v5/meshes/l_uarm_chull.obj; visual mesh filename=package://atlas_v5/meshes/l_uarm.obj
- link l_ufarm: geometry collision mesh filename=package://atlas_v5/meshes/l_farm_chull.obj; visual mesh filename=package://atlas_v5/meshes/l_farm.obj
- link l_uglut: geometry collision mesh filename=package://atlas_v5/meshes/l_uglut_chull.obj; visual mesh filename=package://atlas_v5/meshes/l_uglut.obj
- link l_uleg: geometry collision mesh filename=package://atlas_v5/meshes/l_uleg_chull.obj; visual mesh filename=package://atlas_v5/meshes/l_uleg.obj
- link pelvis: geometry collision mesh filename=package://atlas_v5/meshes/pelvis_chull.obj; visual mesh filename=package://atlas_v5/meshes/pelvis.obj
- link r_clav: geometry collision mesh filename=package://atlas_v5/meshes/r_clav_chull.obj; visual mesh filename=package://atlas_v5/meshes/r_clav.obj
- link r_foot: geometry collision mesh filename=package://atlas_v5/meshes/r_foot_chull.obj; collision sphere radius=0.0
- link r_larm: geometry collision mesh filename=package://atlas_v5/meshes/r_larm_chull.obj; visual mesh filename=package://atlas_v5/meshes/r_larm.obj
- link r_lfarm: geometry collision mesh filename=package://atlas_v5/meshes/r_hand_chull.obj; visual mesh filename=package://atlas_v5/meshes/r_hand.obj
- link r_lglut: geometry collision mesh filename=package://atlas_v5/meshes/r_lglut_chull.obj; visual mesh filename=package://atlas_v5/meshes/r_lglut.obj
- link r_lleg: geometry collision mesh filename=package://atlas_v5/meshes/r_lleg_chull.obj; visual mesh filename=package://atlas_v5/meshes/r_lleg.obj
- link r_scap: geometry collision mesh filename=package://atlas_v5/meshes/r_scap_chull.obj; visual mesh filename=package://atlas_v5/meshes/r_scap.obj
- link r_uarm: geometry collision mesh filename=package://atlas_v5/meshes/r_uarm_chull.obj; visual mesh filename=package://atlas_v5/meshes/r_uarm.obj
- link r_ufarm: geometry collision mesh filename=package://atlas_v5/meshes/r_farm_chull.obj; visual mesh filename=package://atlas_v5/meshes/r_farm.obj
- link r_uglut: geometry collision mesh filename=package://atlas_v5/meshes/r_uglut_chull.obj; visual mesh filename=package://atlas_v5/meshes/r_uglut.obj
- link r_uleg: geometry collision mesh filename=package://atlas_v5/meshes/r_uleg_chull.obj; visual mesh filename=package://atlas_v5/meshes/r_uleg.obj
- link utorso: geometry collision mesh filename=package://atlas_v5/meshes/utorso_chull.obj; visual mesh filename=package://atlas_v5/meshes/utorso.obj

File: software/models/atlas_v5/model_convex_hull.urdf (robot description, URDF)
Before this commit: robot atlas, 72 links, 71 joints
Links:
- link l_clav: geometry collision mesh filename=package://atlas_v5/meshes/l_clav_chull.obj; visual mesh filename=package://atlas_v5/meshes/l_clav.obj
- link l_foot: geometry collision mesh filename=package://atlas_v5/meshes/l_foot_chull.obj; collision sphere radius=0.0
- link l_larm: geometry collision mesh filename=package://atlas_v5/meshes/l_larm_chull.obj; visual mesh filename=package://atlas_v5/meshes/l_larm.obj
- link l_lfarm: geometry collision mesh filename=package://atlas_v5/meshes/l_hand_chull.obj; visual mesh filename=package://atlas_v5/meshes/l_hand.obj
- link l_lglut: geometry collision mesh filename=package://atlas_v5/meshes/l_lglut_chull.obj; visual mesh filename=package://atlas_v5/meshes/l_lglut.obj
- link l_lleg: geometry collision mesh filename=package://atlas_v5/meshes/l_lleg_chull.obj; visual mesh filename=package://atlas_v5/meshes/l_lleg.obj
- link l_scap: geometry collision mesh filename=package://atlas_v5/meshes/l_scap_chull.obj; visual mesh filename=package://atlas_v5/meshes/l_scap.obj
- link l_uarm: geometry collision mesh filename=package://atlas_v5/meshes/l_uarm_chull.obj; visual mesh filename=package://atlas_v5/meshes/l_uarm.obj
- link l_ufarm: geometry collision mesh filename=package://atlas_v5/meshes/l_farm_chull.obj; visual mesh filename=package://atlas_v5/meshes/l_farm.obj
- link l_uglut: geometry collision mesh filename=package://atlas_v5/meshes/l_uglut_chull.obj; visual mesh filename=package://atlas_v5/meshes/l_uglut.obj
- link l_uleg: geometry collision mesh filename=package://atlas_v5/meshes/l_uleg_chull.obj; visual mesh filename=package://atlas_v5/meshes/l_uleg.obj
- link pelvis: geometry collision mesh filename=package://atlas_v5/meshes/pelvis_chull.obj; visual mesh filename=package://atlas_v5/meshes/pelvis.obj
- link r_clav: geometry collision mesh filename=package://atlas_v5/meshes/r_clav_chull.obj; visual mesh filename=package://atlas_v5/meshes/r_clav.obj
- link r_foot: geometry collision mesh filename=package://atlas_v5/meshes/r_foot_chull.obj; collision sphere radius=0.0
- link r_larm: geometry collision mesh filename=package://atlas_v5/meshes/r_larm_chull.obj; visual mesh filename=package://atlas_v5/meshes/r_larm.obj
- link r_lfarm: geometry collision mesh filename=package://atlas_v5/meshes/r_hand_chull.obj; visual mesh filename=package://atlas_v5/meshes/r_hand.obj
- link r_lglut: geometry collision mesh filename=package://atlas_v5/meshes/r_lglut_chull.obj; visual mesh filename=package://atlas_v5/meshes/r_lglut.obj
- link r_lleg: geometry collision mesh filename=package://atlas_v5/meshes/r_lleg_chull.obj; visual mesh filename=package://atlas_v5/meshes/r_lleg.obj
- link r_scap: geometry collision mesh filename=package://atlas_v5/meshes/r_scap_chull.obj; visual mesh filename=package://atlas_v5/meshes/r_scap.obj
- link r_uarm: geometry collision mesh filename=package://atlas_v5/meshes/r_uarm_chull.obj; visual mesh filename=package://atlas_v5/meshes/r_uarm.obj
- link r_ufarm: geometry collision mesh filename=package://atlas_v5/meshes/r_farm_chull.obj; visual mesh filename=package://atlas_v5/meshes/r_farm.obj
- link r_uglut: geometry collision mesh filename=package://atlas_v5/meshes/r_uglut_chull.obj; visual mesh filename=package://atlas_v5/meshes/r_uglut.obj
- link r_uleg: geometry collision mesh filename=package://atlas_v5/meshes/r_uleg_chull.obj; visual mesh filename=package://atlas_v5/meshes/r_uleg.obj
- link utorso: geometry collision mesh filename=package://atlas_v5/meshes/utorso_chull.obj; visual mesh filename=package://atlas_v5/meshes/utorso.obj

File: software/models/atlas_v5/model_convex_hull_closed_hands.urdf (robot description, URDF)
Before this commit: robot atlas, 72 links, 71 joints
Links:
- link l_clav: geometry collision mesh filename=package://atlas_v5/meshes/l_clav_chull.obj; visual mesh filename=package://atlas_v5/meshes/l_clav.obj
- link l_foot: geometry collision mesh filename=package://atlas_v5/meshes/l_foot_chull.obj; collision sphere radius=0.0
- link l_larm: geometry collision mesh filename=package://atlas_v5/meshes/l_larm_chull.obj; visual mesh filename=package://atlas_v5/meshes/l_larm.obj
- link l_lfarm: geometry collision mesh filename=package://atlas_v5/meshes/l_hand_chull.obj; visual mesh filename=package://atlas_v5/meshes/l_hand.obj
- link l_lglut: geometry collision mesh filename=package://atlas_v5/meshes/l_lglut_chull.obj; visual mesh filename=package://atlas_v5/meshes/l_lglut.obj
- link l_lleg: geometry collision mesh filename=package://atlas_v5/meshes/l_lleg_chull.obj; visual mesh filename=package://atlas_v5/meshes/l_lleg.obj
- link l_scap: geometry collision mesh filename=package://atlas_v5/meshes/l_scap_chull.obj; visual mesh filename=package://atlas_v5/meshes/l_scap.obj
- link l_uarm: geometry collision mesh filename=package://atlas_v5/meshes/l_uarm_chull.obj; visual mesh filename=package://atlas_v5/meshes/l_uarm.obj
- link l_ufarm: geometry collision mesh filename=package://atlas_v5/meshes/l_farm_chull.obj; visual mesh filename=package://atlas_v5/meshes/l_farm.obj
- link l_uglut: geometry collision mesh filename=package://atlas_v5/meshes/l_uglut_chull.obj; visual mesh filename=package://atlas_v5/meshes/l_uglut.obj
- link l_uleg: geometry collision mesh filename=package://atlas_v5/meshes/l_uleg_chull.obj; visual mesh filename=package://atlas_v5/meshes/l_uleg.obj
- link pelvis: geometry collision mesh filename=package://atlas_v5/meshes/pelvis_chull.obj; visual mesh filename=package://atlas_v5/meshes/pelvis.obj
- link r_clav: geometry collision mesh filename=package://atlas_v5/meshes/r_clav_chull.obj; visual mesh filename=package://atlas_v5/meshes/r_clav.obj
- link r_foot: geometry collision mesh filename=package://atlas_v5/meshes/r_foot_chull.obj; collision sphere radius=0.0
- link r_larm: geometry collision mesh filename=package://atlas_v5/meshes/r_larm_chull.obj; visual mesh filename=package://atlas_v5/meshes/r_larm.obj
- link r_lfarm: geometry collision mesh filename=package://atlas_v5/meshes/r_hand_chull.obj; visual mesh filename=package://atlas_v5/meshes/r_hand.obj
- link r_lglut: geometry collision mesh filename=package://atlas_v5/meshes/r_lglut_chull.obj; visual mesh filename=package://atlas_v5/meshes/r_lglut.obj
- link r_lleg: geometry collision mesh filename=package://atlas_v5/meshes/r_lleg_chull.obj; visual mesh filename=package://atlas_v5/meshes/r_lleg.obj
- link r_scap: geometry collision mesh filename=package://atlas_v5/meshes/r_scap_chull.obj; visual mesh filename=package://atlas_v5/meshes/r_scap.obj
- link r_uarm: geometry collision mesh filename=package://atlas_v5/meshes/r_uarm_chull.obj; visual mesh filename=package://atlas_v5/meshes/r_uarm.obj
- link r_ufarm: geometry collision mesh filename=package://atlas_v5/meshes/r_farm_chull.obj; visual mesh filename=package://atlas_v5/meshes/r_farm.obj
- link r_uglut: geometry collision mesh filename=package://atlas_v5/meshes/r_uglut_chull.obj; visual mesh filename=package://atlas_v5/meshes/r_uglut.obj
- link r_uleg: geometry collision mesh filename=package://atlas_v5/meshes/r_uleg_chull.obj; visual mesh filename=package://atlas_v5/meshes/r_uleg.obj
- link utorso: geometry collision mesh filename=package://atlas_v5/meshes/utorso_chull.obj; visual mesh filename=package://atlas_v5/meshes/utorso.obj

File: software/models/atlas_v5/model_convex_hull_fingers.urdf (robot description, URDF)
Before this commit: robot atlas, 96 links, 95 joints
Links:
- link l_clav: geometry collision mesh filename=package://atlas_v5/meshes/l_clav_chull.obj; visual mesh filename=package://atlas_v5/meshes/l_clav.obj
- link l_foot: geometry collision mesh filename=package://atlas_v5/meshes/l_foot_chull.obj; collision sphere radius=0.0
- link l_larm: geometry collision mesh filename=package://atlas_v5/meshes/l_larm_chull.obj; visual mesh filename=package://atlas_v5/meshes/l_larm.obj
- link l_lfarm: geometry collision mesh filename=package://atlas_v5/meshes/l_hand_chull.obj; visual mesh filename=package://atlas_v5/meshes/l_hand.obj
- link l_lglut: geometry collision mesh filename=package://atlas_v5/meshes/l_lglut_chull.obj; visual mesh filename=package://atlas_v5/meshes/l_lglut.obj
- link l_lleg: geometry collision mesh filename=package://atlas_v5/meshes/l_lleg_chull.obj; visual mesh filename=package://atlas_v5/meshes/l_lleg.obj
- link l_scap: geometry collision mesh filename=package://atlas_v5/meshes/l_scap_chull.obj; visual mesh filename=package://atlas_v5/meshes/l_scap.obj
- link l_uarm: geometry collision mesh filename=package://atlas_v5/meshes/l_uarm_chull.obj; visual mesh filename=package://atlas_v5/meshes/l_uarm.obj
- link l_ufarm: geometry collision mesh filename=package://atlas_v5/meshes/l_farm_chull.obj; visual mesh filename=package://atlas_v5/meshes/l_farm.obj
- link l_uglut: geometry collision mesh filename=package://atlas_v5/meshes/l_uglut_chull.obj; visual mesh filename=package://atlas_v5/meshes/l_uglut.obj
- link l_uleg: geometry collision mesh filename=package://atlas_v5/meshes/l_uleg_chull.obj; visual mesh filename=package://atlas_v5/meshes/l_uleg.obj
- link pelvis: geometry collision mesh filename=package://atlas_v5/meshes/pelvis_chull.obj; visual mesh filename=package://atlas_v5/meshes/pelvis.obj
- link r_clav: geometry collision mesh filename=package://atlas_v5/meshes/r_clav_chull.obj; visual mesh filename=package://atlas_v5/meshes/r_clav.obj
- link r_foot: geometry collision mesh filename=package://atlas_v5/meshes/r_foot_chull.obj; collision sphere radius=0.0
- link r_larm: geometry collision mesh filename=package://atlas_v5/meshes/r_larm_chull.obj; visual mesh filename=package://atlas_v5/meshes/r_larm.obj
- link r_lfarm: geometry collision mesh filename=package://atlas_v5/meshes/r_hand_chull.obj; visual mesh filename=package://atlas_v5/meshes/r_hand.obj
- link r_lglut: geometry collision mesh filename=package://atlas_v5/meshes/r_lglut_chull.obj; visual mesh filename=package://atlas_v5/meshes/r_lglut.obj
- link r_lleg: geometry collision mesh filename=package://atlas_v5/meshes/r_lleg_chull.obj; visual mesh filename=package://atlas_v5/meshes/r_lleg.obj
- link r_scap: geometry collision mesh filename=package://atlas_v5/meshes/r_scap_chull.obj; visual mesh filename=package://atlas_v5/meshes/r_scap.obj
- link r_uarm: geometry collision mesh filename=package://atlas_v5/meshes/r_uarm_chull.obj; visual mesh filename=package://atlas_v5/meshes/r_uarm.obj
- link r_ufarm: geometry collision mesh filename=package://atlas_v5/meshes/r_farm_chull.obj; visual mesh filename=package://atlas_v5/meshes/r_farm.obj
- link r_uglut: geometry collision mesh filename=package://atlas_v5/meshes/r_uglut_chull.obj; visual mesh filename=package://atlas_v5/meshes/r_uglut.obj
- link r_uleg: geometry collision mesh filename=package://atlas_v5/meshes/r_uleg_chull.obj; visual mesh filename=package://atlas_v5/meshes/r_uleg.obj
- link utorso: geometry collision mesh filename=package://atlas_v5/meshes/utorso_chull.obj; visual mesh filename=package://atlas_v5/meshes/utorso.obj
