Commit message: Update generated files for V5 models

File: software/models/atlas_v5/components/atlas_v5_convex_hull.urdf (robot description, URDF)
Before this commit: robot drc_skeleton, 34 links, 34 joints
Links:
- link l_clav: geometry collision mesh filename=package://atlas_v5/meshes/r_clav_chull.obj; visual mesh filename=package://atlas_v5/meshes/r_clav.obj
- link l_foot: geometry collision mesh filename=package://atlas_v5/meshes/l_foot_chull.obj; collision sphere radius=0.0
- link l_larm: geometry collision mesh filename=package://atlas_v5/meshes/r_larm_chull.obj; visual mesh filename=package://atlas_v5/meshes/r_larm.obj
- link l_lfarm: geometry collision mesh filename=package://atlas_v5/meshes/r_hand_chull.obj; visual mesh filename=package://atlas_v5/meshes/r_hand.obj
- link l_scap: geometry collision mesh filename=package://atlas_v5/meshes/r_scap_chull.obj; visual mesh filename=package://atlas_v5/meshes/r_scap.obj
- link l_uarm: geometry collision mesh filename=package://atlas_v5/meshes/r_uarm_chull.obj; visual mesh filename=package://atlas_v5/meshes/r_uarm.obj
- link l_ufarm: geometry collision mesh filename=package://atlas_v5/meshes/r_farm_chull.obj; visual mesh filename=package://atlas_v5/meshes/r_farm.obj
- link r_foot: geometry collision mesh filename=package://atlas_v5/meshes/r_foot_chull.obj; collision sphere radius=0.0
Joints:
- joint l_arm_elx: axis 1 0 0 -> -1.0 -0.0 -0.0; origin xyz=0 0.119 0.0092 rpy=0 0 0 -> xyz=0 -0.119 0.0092 rpy=0 0 0
- joint l_arm_ely: axis 0 1 0 -> -0.0 -1.0 -0.0; origin xyz=0 0.187 -0.016 rpy=0 0 0 -> xyz=0 -0.187 -0.016 rpy=0 0 0
- joint l_arm_lwy: axis 0 1 0 -> -0.0 -1.0 -0.0; origin xyz=0 0 0 rpy=0 0 0 -> xyz=0 0 0 rpy=0 3.14159265359 0
- joint l_arm_shx: axis 1 0 0 -> -1.0 -0.0 -0.0; origin xyz=0 0.11 -0.245 rpy=0 0 0 -> xyz=0 -0.11 -0.245 rpy=0 0 0
- joint l_arm_shz: origin xyz=0.1406 0.2256 0.4776 rpy=0 0 0 -> xyz=0.1406 0.2256 0.4776 rpy=0 0 3.14159265359
- joint l_arm_uwy: axis 0 1 0 -> -0.0 -1.0 -0.0; origin xyz=0 0.29955 -0.00921 rpy=0 0 0 -> xyz=0 -0.29955 -0.00921 rpy=0 3.14159265359 0

File: software/models/atlas_v5/components/atlas_v5_full_collision_geometry.urdf (robot description, URDF)
Before this commit: robot drc_skeleton, 34 links, 34 joints
Links:
- link l_clav: geometry collision box size=0.1 0.07 0.072; collision cylinder length=0.1525 radius=0.0555
- link l_larm: geometry collision box size=0.025 0.06 0.06; collision box size=0.025 0.155 0.07
- link l_lfarm: geometry collision cylinder length=0.015 radius=0.045; collision cylinder length=0.015 radius=0.052
- link l_scap: geometry collision box size=0.02 0.029 0.018; collision box size=0.028 0.090 0.05
- link l_uarm: geometry collision box size=0.05 0.07 0.15; collision cylinder length=0.11 radius=0.065
- link l_ufarm: geometry collision box size=0.08 0.09 0.11; collision cylinder length=0.1 radius=0.053
Joints:
- joint l_arm_elx: axis 1 0 0 -> -1.0 -0.0 -0.0; origin xyz=0 0.119 0.0092 rpy=0 0 0 -> xyz=0 -0.119 0.0092 rpy=0 0 0
- joint l_arm_ely: axis 0 1 0 -> -0.0 -1.0 -0.0; origin xyz=0 0.187 -0.016 rpy=0 0 0 -> xyz=0 -0.187 -0.016 rpy=0 0 0
- joint l_arm_lwy: axis 0 1 0 -> -0.0 -1.0 -0.0; origin xyz=0 0 0 rpy=0 0 0 -> xyz=0 0 0 rpy=0 3.14159265359 0
- joint l_arm_shx: axis 1 0 0 -> -1.0 -0.0 -0.0; origin xyz=0 0.11 -0.245 rpy=0 0 0 -> xyz=0 -0.11 -0.245 rpy=0 0 0
- joint l_arm_shz: origin xyz=0.1406 0.2256 0.4776 rpy=0 0 0 -> xyz=0.1406 0.2256 0.4776 rpy=0 0 3.14159265359
- joint l_arm_uwy: axis 0 1 0 -> -0.0 -1.0 -0.0; origin xyz=0 0.29955 -0.00921 rpy=0 0 0 -> xyz=0 -0.29955 -0.00921 rpy=0 3.14159265359 0

File: software/models/atlas_v5/components/atlas_v5_minimal_contact.urdf (robot description, URDF)
Before this commit: robot drc_skeleton, 34 links, 34 joints
Links:
- link l_clav: geometry visual mesh filename=package://atlas_v5/meshes/r_clav.obj
- link l_larm: geometry visual mesh filename=package://atlas_v5/meshes/r_larm.obj
- link l_lfarm: geometry visual mesh filename=package://atlas_v5/meshes/r_hand.obj
- link l_scap: geometry visual mesh filename=package://atlas_v5/meshes/r_scap.obj
- link l_uarm: geometry visual mesh filename=package://atlas_v5/meshes/r_uarm.obj
- link l_ufarm: geometry visual mesh filename=package://atlas_v5/meshes/r_farm.obj
Joints:
- joint l_arm_elx: axis 1 0 0 -> -1.0 -0.0 -0.0; origin xyz=0 0.119 0.0092 rpy=0 0 0 -> xyz=0 -0.119 0.0092 rpy=0 0 0
- joint l_arm_ely: axis 0 1 0 -> -0.0 -1.0 -0.0; origin xyz=0 0.187 -0.016 rpy=0 0 0 -> xyz=0 -0.187 -0.016 rpy=0 0 0
- joint l_arm_lwy: axis 0 1 0 -> -0.0 -1.0 -0.0; origin xyz=0 0 0 rpy=0 0 0 -> xyz=0 0 0 rpy=0 3.14159265359 0
- joint l_arm_shx: axis 1 0 0 -> -1.0 -0.0 -0.0; origin xyz=0 0.11 -0.245 rpy=0 0 0 -> xyz=0 -0.11 -0.245 rpy=0 0 0
- joint l_arm_shz: origin xyz=0.1406 0.2256 0.4776 rpy=0 0 0 -> xyz=0.1406 0.2256 0.4776 rpy=0 0 3.14159265359
- joint l_arm_uwy: axis 0 1 0 -> -0.0 -1.0 -0.0; origin xyz=0 0.29955 -0.00921 rpy=0 0 0 -> xyz=0 -0.29955 -0.00921 rpy=0 3.14159265359 0

File: software/models/atlas_v5/model_LR_RR.urdf (robot description, URDF)
Before this commit: robot atlas, 86 links, 85 joints
Links:
- link l_clav: geometry collision box size=0.1 0.07 0.072; collision cylinder length=0.1525 radius=0.0555
- link l_larm: geometry collision box size=0.025 0.06 0.06; collision box size=0.025 0.155 0.07
- link l_lfarm: geometry collision cylinder length=0.015 radius=0.045; collision cylinder length=0.015 radius=0.052
- link l_scap: geometry collision box size=0.02 0.029 0.018; collision box size=0.028 0.090 0.05
- link l_uarm: geometry collision box size=0.05 0.07 0.15; collision cylinder length=0.11 radius=0.065
- link l_ufarm: geometry collision box size=0.08 0.09 0.11; collision cylinder length=0.1 radius=0.053
Joints:
- joint l_arm_elx: axis 1 0 0 -> -1.0 -0.0 -0.0; origin xyz=0 0.119 0.0092 rpy=0 0 0 -> xyz=0 -0.119 0.0092 rpy=0 0 0
- joint l_arm_ely: axis 0 1 0 -> -0.0 -1.0 -0.0; origin xyz=0 0.187 -0.016 rpy=0 0 0 -> xyz=0 -0.187 -0.016 rpy=0 0 0
- joint l_arm_lwy: axis 0 1 0 -> -0.0 -1.0 -0.0; origin xyz=0 0 0 rpy=0 0 0 -> xyz=0 0 0 rpy=0 3.14159265359 0
- joint l_arm_shx: axis 1 0 0 -> -1.0 -0.0 -0.0; origin xyz=0 0.11 -0.245 rpy=0 0 0 -> xyz=0 -0.11 -0.245 rpy=0 0 0
- joint l_arm_shz: origin xyz=0.1406 0.2256 0.4776 rpy=0 0 0 -> xyz=0.1406 0.2256 0.4776 rpy=0 0 3.14159265359
- joint l_arm_uwy: axis 0 1 0 -> -0.0 -1.0 -0.0; origin xyz=0 0.29955 -0.00921 rpy=0 0 0 -> xyz=0 -0.29955 -0.00921 rpy=0 3.14159265359 0
- joint l_hand_force_torque_joint: origin xyz=0 0.1245 0.0112 rpy=0 0 0 -> xyz=0 -0.1245 0.0112 rpy=0 0 3.141592
- joint r_hand_force_torque_joint: origin xyz=0 -0.1245 -0.0112 rpy=0 0 3.142 -> xyz=0 -0.1245 -0.0112 rpy=0 0 3.141592

File: software/models/atlas_v5/model_convex_hull.urdf (robot description, URDF)
Before this commit: robot atlas, 70 links, 69 joints
Links:
- link l_clav: geometry collision mesh filename=package://atlas_v5/meshes/r_clav_chull.obj; visual mesh filename=package://atlas_v5/meshes/r_clav.obj
- link l_foot: geometry collision mesh filename=package://atlas_v5/meshes/l_foot_chull.obj; collision sphere radius=0.0
- link l_larm: geometry collision mesh filename=package://atlas_v5/meshes/r_larm_chull.obj; visual mesh filename=package://atlas_v5/meshes/r_larm.obj
- link l_lfarm: geometry collision mesh filename=package://atlas_v5/meshes/r_hand_chull.obj; visual mesh filename=package://atlas_v5/meshes/r_hand.obj
- link l_scap: geometry collision mesh filename=package://atlas_v5/meshes/r_scap_chull.obj; visual mesh filename=package://atlas_v5/meshes/r_scap.obj
- link l_uarm: geometry collision mesh filename=package://atlas_v5/meshes/r_uarm_chull.obj; visual mesh filename=package://atlas_v5/meshes/r_uarm.obj
- link l_ufarm: geometry collision mesh filename=package://atlas_v5/meshes/r_farm_chull.obj; visual mesh filename=package://atlas_v5/meshes/r_farm.obj
- link r_foot: geometry collision mesh filename=package://atlas_v5/meshes/r_foot_chull.obj; collision sphere radius=0.0
Joints:
- joint l_arm_elx: axis 1 0 0 -> -1.0 -0.0 -0.0; origin xyz=0 0.119 0.0092 rpy=0 0 0 -> xyz=0 -0.119 0.0092 rpy=0 0 0
- joint l_arm_ely: axis 0 1 0 -> -0.0 -1.0 -0.0; origin xyz=0 0.187 -0.016 rpy=0 0 0 -> xyz=0 -0.187 -0.016 rpy=0 0 0
- joint l_arm_lwy: axis 0 1 0 -> -0.0 -1.0 -0.0; origin xyz=0 0 0 rpy=0 0 0 -> xyz=0 0 0 rpy=0 3.14159265359 0
- joint l_arm_shx: axis 1 0 0 -> -1.0 -0.0 -0.0; origin xyz=0 0.11 -0.245 rpy=0 0 0 -> xyz=0 -0.11 -0.245 rpy=0 0 0
- joint l_arm_shz: origin xyz=0.1406 0.2256 0.4776 rpy=0 0 0 -> xyz=0.1406 0.2256 0.4776 rpy=0 0 3.14159265359
- joint l_arm_uwy: axis 0 1 0 -> -0.0 -1.0 -0.0; origin xyz=0 0.29955 -0.00921 rpy=0 0 0 -> xyz=0 -0.29955 -0.00921 rpy=0 3.14159265359 0
- joint l_hand_force_torque_joint: origin xyz=0 0.1245 0.0112 rpy=0 0 0 -> xyz=0 -0.1245 0.0112 rpy=0 0 3.141592
- joint r_hand_force_torque_joint: origin xyz=0 -0.1245 -0.0112 rpy=0 0 3.142 -> xyz=0 -0.1245 -0.0112 rpy=0 0 3.141592

File: software/models/atlas_v5/model_convex_hull_closed_hands.urdf (robot description, URDF)
Before this commit: robot atlas, 70 links, 69 joints
Links:
- link l_clav: geometry collision mesh filename=package://atlas_v5/meshes/r_clav_chull.obj; visual mesh filename=package://atlas_v5/meshes/r_clav.obj
- link l_foot: geometry collision mesh filename=package://atlas_v5/meshes/l_foot_chull.obj; collision sphere radius=0.0
- link l_larm: geometry collision mesh filename=package://atlas_v5/meshes/r_larm_chull.obj; visual mesh filename=package://atlas_v5/meshes/r_larm.obj
- link l_lfarm: geometry collision mesh filename=package://atlas_v5/meshes/r_hand_chull.obj; visual mesh filename=package://atlas_v5/meshes/r_hand.obj
- link l_scap: geometry collision mesh filename=package://atlas_v5/meshes/r_scap_chull.obj; visual mesh filename=package://atlas_v5/meshes/r_scap.obj
- link l_uarm: geometry collision mesh filename=package://atlas_v5/meshes/r_uarm_chull.obj; visual mesh filename=package://atlas_v5/meshes/r_uarm.obj
- link l_ufarm: geometry collision mesh filename=package://atlas_v5/meshes/r_farm_chull.obj; visual mesh filename=package://atlas_v5/meshes/r_farm.obj
- link r_foot: geometry collision mesh filename=package://atlas_v5/meshes/r_foot_chull.obj; collision sphere radius=0.0
Joints:
- joint l_arm_elx: axis 1 0 0 -> -1.0 -0.0 -0.0; origin xyz=0 0.119 0.0092 rpy=0 0 0 -> xyz=0 -0.119 0.0092 rpy=0 0 0
- joint l_arm_ely: axis 0 1 0 -> -0.0 -1.0 -0.0; origin xyz=0 0.187 -0.016 rpy=0 0 0 -> xyz=0 -0.187 -0.016 rpy=0 0 0
- joint l_arm_lwy: axis 0 1 0 -> -0.0 -1.0 -0.0; origin xyz=0 0 0 rpy=0 0 0 -> xyz=0 0 0 rpy=0 3.14159265359 0
- joint l_arm_shx: axis 1 0 0 -> -1.0 -0.0 -0.0; origin xyz=0 0.11 -0.245 rpy=0 0 0 -> xyz=0 -0.11 -0.245 rpy=0 0 0
- joint l_arm_shz: origin xyz=0.1406 0.2256 0.4776 rpy=0 0 0 -> xyz=0.1406 0.2256 0.4776 rpy=0 0 3.14159265359
- joint l_arm_uwy: axis 0 1 0 -> -0.0 -1.0 -0.0; origin xyz=0 0.29955 -0.00921 rpy=0 0 0 -> xyz=0 -0.29955 -0.00921 rpy=0 3.14159265359 0
- joint l_hand_force_torque_joint: origin xyz=0 0.1245 0.0112 rpy=0 0 0 -> xyz=0 -0.1245 0.0112 rpy=0 0 3.141592
- joint r_hand_force_torque_joint: origin xyz=0 -0.1245 -0.0112 rpy=0 0 3.142 -> xyz=0 -0.1245 -0.0112 rpy=0 0 3.141592

File: software/models/atlas_v5/model_convex_hull_fingers.urdf (robot description, URDF)
Before this commit: robot atlas, 94 links, 93 joints
Links:
- link l_clav: geometry collision mesh filename=package://atlas_v5/meshes/r_clav_chull.obj; visual mesh filename=package://atlas_v5/meshes/r_clav.obj
- link l_foot: geometry collision mesh filename=package://atlas_v5/meshes/l_foot_chull.obj; collision sphere radius=0.0
- link l_larm: geometry collision mesh filename=package://atlas_v5/meshes/r_larm_chull.obj; visual mesh filename=package://atlas_v5/meshes/r_larm.obj
- link l_lfarm: geometry collision mesh filename=package://atlas_v5/meshes/r_hand_chull.obj; visual mesh filename=package://atlas_v5/meshes/r_hand.obj
- link l_scap: geometry collision mesh filename=package://atlas_v5/meshes/r_scap_chull.obj; visual mesh filename=package://atlas_v5/meshes/r_scap.obj
- link l_uarm: geometry collision mesh filename=package://atlas_v5/meshes/r_uarm_chull.obj; visual mesh filename=package://atlas_v5/meshes/r_uarm.obj
- link l_ufarm: geometry collision mesh filename=package://atlas_v5/meshes/r_farm_chull.obj; visual mesh filename=package://atlas_v5/meshes/r_farm.obj
- link r_foot: geometry collision mesh filename=package://atlas_v5/meshes/r_foot_chull.obj; collision sphere radius=0.0
Joints:
- joint l_arm_elx: axis 1 0 0 -> -1.0 -0.0 -0.0; origin xyz=0 0.119 0.0092 rpy=0 0 0 -> xyz=0 -0.119 0.0092 rpy=0 0 0
- joint l_arm_ely: axis 0 1 0 -> -0.0 -1.0 -0.0; origin xyz=0 0.187 -0.016 rpy=0 0 0 -> xyz=0 -0.187 -0.016 rpy=0 0 0
- joint l_arm_lwy: axis 0 1 0 -> -0.0 -1.0 -0.0; origin xyz=0 0 0 rpy=0 0 0 -> xyz=0 0 0 rpy=0 3.14159265359 0
- joint l_arm_shx: axis 1 0 0 -> -1.0 -0.0 -0.0; origin xyz=0 0.11 -0.245 rpy=0 0 0 -> xyz=0 -0.11 -0.245 rpy=0 0 0
- joint l_arm_shz: origin xyz=0.1406 0.2256 0.4776 rpy=0 0 0 -> xyz=0.1406 0.2256 0.4776 rpy=0 0 3.14159265359
- joint l_arm_uwy: axis 0 1 0 -> -0.0 -1.0 -0.0; origin xyz=0 0.29955 -0.00921 rpy=0 0 0 -> xyz=0 -0.29955 -0.00921 rpy=0 3.14159265359 0
- joint l_hand_force_torque_joint: origin xyz=0 0.1245 0.0112 rpy=0 0 0 -> xyz=0 -0.1245 0.0112 rpy=0 0 3.141592
- joint r_hand_force_torque_joint: origin xyz=0 -0.1245 -0.0112 rpy=0 0 3.142 -> xyz=0 -0.1245 -0.0112 rpy=0 0 3.141592

File: software/models/atlas_v5/model_minimal_contact.urdf (robot description, URDF)
Before this commit: robot atlas, 94 links, 93 joints
Links:
- link l_clav: geometry visual mesh filename=package://atlas_v5/meshes/r_clav.obj
- link l_larm: geometry visual mesh filename=package://atlas_v5/meshes/r_larm.obj
- link l_lfarm: geometry visual mesh filename=package://atlas_v5/meshes/r_hand.obj
- link l_scap: geometry visual mesh filename=package://atlas_v5/meshes/r_scap.obj
- link l_uarm: geometry visual mesh filename=package://atlas_v5/meshes/r_uarm.obj
- link l_ufarm: geometry visual mesh filename=package://atlas_v5/meshes/r_farm.obj
Joints:
- joint l_arm_elx: axis 1 0 0 -> -1.0 -0.0 -0.0; origin xyz=0 0.119 0.0092 rpy=0 0 0 -> xyz=0 -0.119 0.0092 rpy=0 0 0
- joint l_arm_ely: axis 0 1 0 -> -0.0 -1.0 -0.0; origin xyz=0 0.187 -0.016 rpy=0 0 0 -> xyz=0 -0.187 -0.016 rpy=0 0 0
- joint l_arm_lwy: axis 0 1 0 -> -0.0 -1.0 -0.0; origin xyz=0 0 0 rpy=0 0 0 -> xyz=0 0 0 rpy=0 3.14159265359 0
- joint l_arm_shx: axis 1 0 0 -> -1.0 -0.0 -0.0; origin xyz=0 0.11 -0.245 rpy=0 0 0 -> xyz=0 -0.11 -0.245 rpy=0 0 0
- joint l_arm_shz: origin xyz=0.1406 0.2256 0.4776 rpy=0 0 0 -> xyz=0.1406 0.2256 0.4776 rpy=0 0 3.14159265359
- joint l_arm_uwy: axis 0 1 0 -> -0.0 -1.0 -0.0; origin xyz=0 0.29955 -0.00921 rpy=0 0 0 -> xyz=0 -0.29955 -0.00921 rpy=0 3.14159265359 0
- joint l_hand_force_torque_joint: origin xyz=0 0.1245 0.0112 rpy=0 0 0 -> xyz=0 -0.1245 0.0112 rpy=0 0 3.141592
- joint r_hand_force_torque_joint: origin xyz=0 -0.1245 -0.0112 rpy=0 0 3.142 -> xyz=0 -0.1245 -0.0112 rpy=0 0 3.141592

Commit message: Update V5 for changes from OSRF
Fixes head position.

File: software/models/atlas_v5/components/atlas_v5_convex_hull.urdf (robot description, URDF)
Before this commit: robot drc_skeleton, 34 links, 34 joints
Joints:
- joint neck_ay: origin xyz=0.2946 0 0.5765 rpy=0 0 0 -> xyz=0.2546 0 0.6215 rpy=0 0 0

File: software/models/atlas_v5/components/atlas_v5_full_collision_geometry.urdf (robot description, URDF)
Before this commit: robot drc_skeleton, 34 links, 34 joints
Links:
- link l_lglut: geometry collision box size=0.0975 0.069 0.103; collision box size=0.125 0.05 0.08
- link l_uglut: geometry collision box size=0.05 0.1 0.1; collision cylinder length=0.080842 radius=0.019841
- link r_lglut: geometry collision box size=0.0975 0.069 0.103; collision box size=0.125 0.05 0.08
- link r_uglut: geometry collision box size=0.05 0.1 0.1; collision cylinder length=0.080842 radius=0.019841
- link utorso: geometry collision box size=0.13 0.50 0.10; collision box size=0.2 0.18 0.10
Joints:
- joint neck_ay: origin xyz=0.2946 0 0.5765 rpy=0 0 0 -> xyz=0.2546 0 0.6215 rpy=0 0 0

File: software/models/atlas_v5/components/atlas_v5_minimal_contact.urdf (robot description, URDF)
Before this commit: robot drc_skeleton, 34 links, 34 joints
Joints:
- joint neck_ay: origin xyz=0.2946 0 0.5765 rpy=0 0 0 -> xyz=0.2546 0 0.6215 rpy=0 0 0

File: software/models/atlas_v5/components/osrf_original/atlas_v5.urdf (robot description, URDF)
Before this commit: robot drc_skeleton, 34 links, 34 joints
Links:
- link l_lglut: geometry collision box size=0.0975 0.069 0.103; collision box size=0.125 0.05 0.08
- link l_uglut: geometry collision box size=0.05 0.1 0.1; collision cylinder length=0.080842 radius=0.019841
- link r_lglut: geometry collision box size=0.0975 0.069 0.103; collision box size=0.125 0.05 0.08
- link r_uglut: geometry collision box size=0.05 0.1 0.1; collision cylinder length=0.080842 radius=0.019841
- link utorso: geometry collision box size=0.13 0.50 0.10; collision box size=0.2 0.18 0.10
Joints:
- joint neck_ry: origin xyz=${0.2546+0.04} 0 ${0.6215-0.045} rpy=0 0 0 -> xyz=0.2546 0 0.6215 rpy=0 0 0

File: software/models/atlas_v5/model_LR_RR.urdf (robot description, URDF)
Before this commit: robot atlas, 86 links, 85 joints
Links:
- link l_lglut: geometry collision box size=0.0975 0.069 0.103; collision box size=0.125 0.05 0.08
- link l_uglut: geometry collision box size=0.05 0.1 0.1; collision cylinder length=0.080842 radius=0.019841
- link r_lglut: geometry collision box size=0.0975 0.069 0.103; collision box size=0.125 0.05 0.08
- link r_uglut: geometry collision box size=0.05 0.1 0.1; collision cylinder length=0.080842 radius=0.019841
- link utorso: geometry collision box size=0.13 0.50 0.10; collision box size=0.2 0.18 0.10
Joints:
- joint neck_ay: origin xyz=0.2946 0 0.5765 rpy=0 0 0 -> xyz=0.2546 0 0.6215 rpy=0 0 0

File: software/models/atlas_v5/model_convex_hull.urdf (robot description, URDF)
Before this commit: robot atlas, 70 links, 69 joints
Joints:
- joint neck_ay: origin xyz=0.2946 0 0.5765 rpy=0 0 0 -> xyz=0.2546 0 0.6215 rpy=0 0 0

File: software/models/atlas_v5/model_convex_hull_closed_hands.urdf (robot description, URDF)
Before this commit: robot atlas, 70 links, 69 joints
Joints:
- joint neck_ay: origin xyz=0.2946 0 0.5765 rpy=0 0 0 -> xyz=0.2546 0 0.6215 rpy=0 0 0

File: software/models/atlas_v5/model_convex_hull_fingers.urdf (robot description, URDF)
Before this commit: robot atlas, 94 links, 93 joints
Joints:
- joint neck_ay: origin xyz=0.2946 0 0.5765 rpy=0 0 0 -> xyz=0.2546 0 0.6215 rpy=0 0 0

File: software/models/atlas_v5/model_minimal_contact.urdf (robot description, URDF)
Before this commit: robot atlas, 94 links, 93 joints
Joints:
- joint neck_ay: origin xyz=0.2946 0 0.5765 rpy=0 0 0 -> xyz=0.2546 0 0.6215 rpy=0 0 0
