Commit message: update a subset of joint limits on v5 (importantly: electric joints) based on measurements

File: software/models/atlas_v5/components/atlas_v5_convex_hull.urdf (robot description, URDF)
Before this commit: robot drc_skeleton, 34 links, 34 joints
Joints:
- joint l_arm_lwy: limit lower=-2.9671 upper=2.9671 effort=25 velocity=10 -> lower=-2.82 upper=2.82 effort=25 velocity=10
- joint l_arm_mwx: limit lower=-1.7628 upper=1.7628 effort=25 velocity=10 -> lower=-1.76 upper=1.76 effort=25 velocity=10
- joint l_arm_uwy: limit lower=-3.011 upper=3.011 effort=25 velocity=10 -> lower=-2.98 upper=2.98 effort=25 velocity=10
- joint l_leg_akx: limit lower=-0.8 upper=0.8 effort=360 velocity=12 -> lower=-0.7 upper=0.7 effort=360 velocity=12
- joint l_leg_aky: limit lower=-1 upper=0.7 effort=740 velocity=12 -> lower=-1.06 upper=0.72 effort=740 velocity=12
- joint l_leg_hpx: limit lower=-0.523599 upper=0.523599 effort=530 velocity=12 -> lower=-0.23 upper=0.52 effort=530 velocity=12
- joint l_leg_hpz: limit lower=-0.174358 upper=0.786794 effort=275 velocity=12 -> lower=-0.2 upper=0.82 effort=275 velocity=12
- joint neck_ay: limit lower=-0.602139 upper=1.14319 effort=25 velocity=6.28 -> lower=-0.605 upper=1.16 effort=25 velocity=6.28
- joint r_arm_lwy: limit lower=-2.9671 upper=2.9671 effort=25 velocity=10 -> lower=-2.82 upper=2.82 effort=25 velocity=10
- joint r_arm_mwx: limit lower=-1.7628 upper=1.7628 effort=25 velocity=10 -> lower=-1.76 upper=1.76 effort=25 velocity=10
- joint r_arm_uwy: limit lower=-3.011 upper=3.011 effort=25 velocity=10 -> lower=-2.98 upper=2.98 effort=25 velocity=10
- joint r_leg_akx: limit lower=-0.8 upper=0.8 effort=360 velocity=12 -> lower=-0.7 upper=0.7 effort=360 velocity=12
- joint r_leg_aky: limit lower=-1 upper=0.7 effort=740 velocity=12 -> lower=-1.06 upper=0.72 effort=740 velocity=12
- joint r_leg_hpx: limit lower=-0.523599 upper=0.523599 effort=530 velocity=12 -> lower=-0.52 upper=0.23 effort=530 velocity=12
- joint r_leg_hpz: limit lower=-0.786794 upper=0.174358 effort=275 velocity=12 -> lower=-0.82 upper=0.2 effort=275 velocity=12

File: software/models/atlas_v5/components/atlas_v5_full_collision_geometry.urdf (robot description, URDF)
Before this commit: robot drc_skeleton, 34 links, 34 joints
Joints:
- joint l_arm_lwy: limit lower=-2.9671 upper=2.9671 effort=25 velocity=10 -> lower=-2.82 upper=2.82 effort=25 velocity=10
- joint l_arm_mwx: limit lower=-1.7628 upper=1.7628 effort=25 velocity=10 -> lower=-1.76 upper=1.76 effort=25 velocity=10
- joint l_arm_uwy: limit lower=-3.011 upper=3.011 effort=25 velocity=10 -> lower=-2.98 upper=2.98 effort=25 velocity=10
- joint l_leg_akx: limit lower=-0.8 upper=0.8 effort=360 velocity=12 -> lower=-0.7 upper=0.7 effort=360 velocity=12
- joint l_leg_aky: limit lower=-1 upper=0.7 effort=740 velocity=12 -> lower=-1.06 upper=0.72 effort=740 velocity=12
- joint l_leg_hpx: limit lower=-0.523599 upper=0.523599 effort=530 velocity=12 -> lower=-0.23 upper=0.52 effort=530 velocity=12
- joint l_leg_hpz: limit lower=-0.174358 upper=0.786794 effort=275 velocity=12 -> lower=-0.2 upper=0.82 effort=275 velocity=12
- joint neck_ay: limit lower=-0.602139 upper=1.14319 effort=25 velocity=6.28 -> lower=-0.605 upper=1.16 effort=25 velocity=6.28
- joint r_arm_lwy: limit lower=-2.9671 upper=2.9671 effort=25 velocity=10 -> lower=-2.82 upper=2.82 effort=25 velocity=10
- joint r_arm_mwx: limit lower=-1.7628 upper=1.7628 effort=25 velocity=10 -> lower=-1.76 upper=1.76 effort=25 velocity=10
- joint r_arm_uwy: limit lower=-3.011 upper=3.011 effort=25 velocity=10 -> lower=-2.98 upper=2.98 effort=25 velocity=10
- joint r_leg_akx: limit lower=-0.8 upper=0.8 effort=360 velocity=12 -> lower=-0.7 upper=0.7 effort=360 velocity=12
- joint r_leg_aky: limit lower=-1 upper=0.7 effort=740 velocity=12 -> lower=-1.06 upper=0.72 effort=740 velocity=12
- joint r_leg_hpx: limit lower=-0.523599 upper=0.523599 effort=530 velocity=12 -> lower=-0.52 upper=0.23 effort=530 velocity=12
- joint r_leg_hpz: limit lower=-0.786794 upper=0.174358 effort=275 velocity=12 -> lower=-0.82 upper=0.2 effort=275 velocity=12

File: software/models/atlas_v5/components/atlas_v5_minimal_contact.urdf (robot description, URDF)
Before this commit: robot drc_skeleton, 34 links, 34 joints
Joints:
- joint l_arm_lwy: limit lower=-2.9671 upper=2.9671 effort=25 velocity=10 -> lower=-2.82 upper=2.82 effort=25 velocity=10
- joint l_arm_mwx: limit lower=-1.7628 upper=1.7628 effort=25 velocity=10 -> lower=-1.76 upper=1.76 effort=25 velocity=10
- joint l_arm_uwy: limit lower=-3.011 upper=3.011 effort=25 velocity=10 -> lower=-2.98 upper=2.98 effort=25 velocity=10
- joint l_leg_akx: limit lower=-0.8 upper=0.8 effort=360 velocity=12 -> lower=-0.7 upper=0.7 effort=360 velocity=12
- joint l_leg_aky: limit lower=-1 upper=0.7 effort=740 velocity=12 -> lower=-1.06 upper=0.72 effort=740 velocity=12
- joint l_leg_hpx: limit lower=-0.523599 upper=0.523599 effort=530 velocity=12 -> lower=-0.23 upper=0.52 effort=530 velocity=12
- joint l_leg_hpz: limit lower=-0.174358 upper=0.786794 effort=275 velocity=12 -> lower=-0.2 upper=0.82 effort=275 velocity=12
- joint neck_ay: limit lower=-0.602139 upper=1.14319 effort=25 velocity=6.28 -> lower=-0.605 upper=1.16 effort=25 velocity=6.28
- joint r_arm_lwy: limit lower=-2.9671 upper=2.9671 effort=25 velocity=10 -> lower=-2.82 upper=2.82 effort=25 velocity=10
- joint r_arm_mwx: limit lower=-1.7628 upper=1.7628 effort=25 velocity=10 -> lower=-1.76 upper=1.76 effort=25 velocity=10
- joint r_arm_uwy: limit lower=-3.011 upper=3.011 effort=25 velocity=10 -> lower=-2.98 upper=2.98 effort=25 velocity=10
- joint r_leg_akx: limit lower=-0.8 upper=0.8 effort=360 velocity=12 -> lower=-0.7 upper=0.7 effort=360 velocity=12
- joint r_leg_aky: limit lower=-1 upper=0.7 effort=740 velocity=12 -> lower=-1.06 upper=0.72 effort=740 velocity=12
- joint r_leg_hpx: limit lower=-0.523599 upper=0.523599 effort=530 velocity=12 -> lower=-0.52 upper=0.23 effort=530 velocity=12
- joint r_leg_hpz: limit lower=-0.786794 upper=0.174358 effort=275 velocity=12 -> lower=-0.82 upper=0.2 effort=275 velocity=12

File: software/models/atlas_v5/model_LR_RR.urdf (robot description, URDF)
Before this commit: robot atlas, 88 links, 87 joints
Joints:
- joint l_arm_lwy: limit lower=-2.9671 upper=2.9671 effort=25 velocity=10 -> lower=-2.82 upper=2.82 effort=25 velocity=10
- joint l_arm_mwx: limit lower=-1.7628 upper=1.7628 effort=25 velocity=10 -> lower=-1.76 upper=1.76 effort=25 velocity=10
- joint l_arm_uwy: limit lower=-3.011 upper=3.011 effort=25 velocity=10 -> lower=-2.98 upper=2.98 effort=25 velocity=10
- joint l_leg_akx: limit lower=-0.8 upper=0.8 effort=360 velocity=12 -> lower=-0.7 upper=0.7 effort=360 velocity=12
- joint l_leg_aky: limit lower=-1 upper=0.7 effort=740 velocity=12 -> lower=-1.06 upper=0.72 effort=740 velocity=12
- joint l_leg_hpx: limit lower=-0.523599 upper=0.523599 effort=530 velocity=12 -> lower=-0.23 upper=0.52 effort=530 velocity=12
- joint l_leg_hpz: limit lower=-0.174358 upper=0.786794 effort=275 velocity=12 -> lower=-0.2 upper=0.82 effort=275 velocity=12
- joint neck_ay: limit lower=-0.602139 upper=1.14319 effort=25 velocity=6.28 -> lower=-0.605 upper=1.16 effort=25 velocity=6.28
- joint r_arm_lwy: limit lower=-2.9671 upper=2.9671 effort=25 velocity=10 -> lower=-2.82 upper=2.82 effort=25 velocity=10
- joint r_arm_mwx: limit lower=-1.7628 upper=1.7628 effort=25 velocity=10 -> lower=-1.76 upper=1.76 effort=25 velocity=10
- joint r_arm_uwy: limit lower=-3.011 upper=3.011 effort=25 velocity=10 -> lower=-2.98 upper=2.98 effort=25 velocity=10
- joint r_leg_akx: limit lower=-0.8 upper=0.8 effort=360 velocity=12 -> lower=-0.7 upper=0.7 effort=360 velocity=12
- joint r_leg_aky: limit lower=-1 upper=0.7 effort=740 velocity=12 -> lower=-1.06 upper=0.72 effort=740 velocity=12
- joint r_leg_hpx: limit lower=-0.523599 upper=0.523599 effort=530 velocity=12 -> lower=-0.52 upper=0.23 effort=530 velocity=12
- joint r_leg_hpz: limit lower=-0.786794 upper=0.174358 effort=275 velocity=12 -> lower=-0.82 upper=0.2 effort=275 velocity=12

File: software/models/atlas_v5/model_convex_hull.urdf (robot description, URDF)
Before this commit: robot atlas, 70 links, 69 joints
Joints:
- joint l_arm_lwy: limit lower=-2.9671 upper=2.9671 effort=25 velocity=10 -> lower=-2.82 upper=2.82 effort=25 velocity=10
- joint l_arm_mwx: limit lower=-1.7628 upper=1.7628 effort=25 velocity=10 -> lower=-1.76 upper=1.76 effort=25 velocity=10
- joint l_arm_uwy: limit lower=-3.011 upper=3.011 effort=25 velocity=10 -> lower=-2.98 upper=2.98 effort=25 velocity=10
- joint l_leg_akx: limit lower=-0.8 upper=0.8 effort=360 velocity=12 -> lower=-0.7 upper=0.7 effort=360 velocity=12
- joint l_leg_aky: limit lower=-1 upper=0.7 effort=740 velocity=12 -> lower=-1.06 upper=0.72 effort=740 velocity=12
- joint l_leg_hpx: limit lower=-0.523599 upper=0.523599 effort=530 velocity=12 -> lower=-0.23 upper=0.52 effort=530 velocity=12
- joint l_leg_hpz: limit lower=-0.174358 upper=0.786794 effort=275 velocity=12 -> lower=-0.2 upper=0.82 effort=275 velocity=12
- joint neck_ay: limit lower=-0.602139 upper=1.14319 effort=25 velocity=6.28 -> lower=-0.605 upper=1.16 effort=25 velocity=6.28
- joint r_arm_lwy: limit lower=-2.9671 upper=2.9671 effort=25 velocity=10 -> lower=-2.82 upper=2.82 effort=25 velocity=10
- joint r_arm_mwx: limit lower=-1.7628 upper=1.7628 effort=25 velocity=10 -> lower=-1.76 upper=1.76 effort=25 velocity=10
- joint r_arm_uwy: limit lower=-3.011 upper=3.011 effort=25 velocity=10 -> lower=-2.98 upper=2.98 effort=25 velocity=10
- joint r_leg_akx: limit lower=-0.8 upper=0.8 effort=360 velocity=12 -> lower=-0.7 upper=0.7 effort=360 velocity=12
- joint r_leg_aky: limit lower=-1 upper=0.7 effort=740 velocity=12 -> lower=-1.06 upper=0.72 effort=740 velocity=12
- joint r_leg_hpx: limit lower=-0.523599 upper=0.523599 effort=530 velocity=12 -> lower=-0.52 upper=0.23 effort=530 velocity=12
- joint r_leg_hpz: limit lower=-0.786794 upper=0.174358 effort=275 velocity=12 -> lower=-0.82 upper=0.2 effort=275 velocity=12

File: software/models/atlas_v5/model_convex_hull_closed_hands.urdf (robot description, URDF)
Before this commit: robot atlas, 70 links, 69 joints
Joints:
- joint l_arm_lwy: limit lower=-2.9671 upper=2.9671 effort=25 velocity=10 -> lower=-2.82 upper=2.82 effort=25 velocity=10
- joint l_arm_mwx: limit lower=-1.7628 upper=1.7628 effort=25 velocity=10 -> lower=-1.76 upper=1.76 effort=25 velocity=10
- joint l_arm_uwy: limit lower=-3.011 upper=3.011 effort=25 velocity=10 -> lower=-2.98 upper=2.98 effort=25 velocity=10
- joint l_leg_akx: limit lower=-0.8 upper=0.8 effort=360 velocity=12 -> lower=-0.7 upper=0.7 effort=360 velocity=12
- joint l_leg_aky: limit lower=-1 upper=0.7 effort=740 velocity=12 -> lower=-1.06 upper=0.72 effort=740 velocity=12
- joint l_leg_hpx: limit lower=-0.523599 upper=0.523599 effort=530 velocity=12 -> lower=-0.23 upper=0.52 effort=530 velocity=12
- joint l_leg_hpz: limit lower=-0.174358 upper=0.786794 effort=275 velocity=12 -> lower=-0.2 upper=0.82 effort=275 velocity=12
- joint neck_ay: limit lower=-0.602139 upper=1.14319 effort=25 velocity=6.28 -> lower=-0.605 upper=1.16 effort=25 velocity=6.28
- joint r_arm_lwy: limit lower=-2.9671 upper=2.9671 effort=25 velocity=10 -> lower=-2.82 upper=2.82 effort=25 velocity=10
- joint r_arm_mwx: limit lower=-1.7628 upper=1.7628 effort=25 velocity=10 -> lower=-1.76 upper=1.76 effort=25 velocity=10
- joint r_arm_uwy: limit lower=-3.011 upper=3.011 effort=25 velocity=10 -> lower=-2.98 upper=2.98 effort=25 velocity=10
- joint r_leg_akx: limit lower=-0.8 upper=0.8 effort=360 velocity=12 -> lower=-0.7 upper=0.7 effort=360 velocity=12
- joint r_leg_aky: limit lower=-1 upper=0.7 effort=740 velocity=12 -> lower=-1.06 upper=0.72 effort=740 velocity=12
- joint r_leg_hpx: limit lower=-0.523599 upper=0.523599 effort=530 velocity=12 -> lower=-0.52 upper=0.23 effort=530 velocity=12
- joint r_leg_hpz: limit lower=-0.786794 upper=0.174358 effort=275 velocity=12 -> lower=-0.82 upper=0.2 effort=275 velocity=12

File: software/models/atlas_v5/model_convex_hull_fingers.urdf (robot description, URDF)
Before this commit: robot atlas, 94 links, 93 joints
Joints:
- joint l_arm_lwy: limit lower=-2.9671 upper=2.9671 effort=25 velocity=10 -> lower=-2.82 upper=2.82 effort=25 velocity=10
- joint l_arm_mwx: limit lower=-1.7628 upper=1.7628 effort=25 velocity=10 -> lower=-1.76 upper=1.76 effort=25 velocity=10
- joint l_arm_uwy: limit lower=-3.011 upper=3.011 effort=25 velocity=10 -> lower=-2.98 upper=2.98 effort=25 velocity=10
- joint l_leg_akx: limit lower=-0.8 upper=0.8 effort=360 velocity=12 -> lower=-0.7 upper=0.7 effort=360 velocity=12
- joint l_leg_aky: limit lower=-1 upper=0.7 effort=740 velocity=12 -> lower=-1.06 upper=0.72 effort=740 velocity=12
- joint l_leg_hpx: limit lower=-0.523599 upper=0.523599 effort=530 velocity=12 -> lower=-0.23 upper=0.52 effort=530 velocity=12
- joint l_leg_hpz: limit lower=-0.174358 upper=0.786794 effort=275 velocity=12 -> lower=-0.2 upper=0.82 effort=275 velocity=12
- joint neck_ay: limit lower=-0.602139 upper=1.14319 effort=25 velocity=6.28 -> lower=-0.605 upper=1.16 effort=25 velocity=6.28
- joint r_arm_lwy: limit lower=-2.9671 upper=2.9671 effort=25 velocity=10 -> lower=-2.82 upper=2.82 effort=25 velocity=10
- joint r_arm_mwx: limit lower=-1.7628 upper=1.7628 effort=25 velocity=10 -> lower=-1.76 upper=1.76 effort=25 velocity=10
- joint r_arm_uwy: limit lower=-3.011 upper=3.011 effort=25 velocity=10 -> lower=-2.98 upper=2.98 effort=25 velocity=10
- joint r_leg_akx: limit lower=-0.8 upper=0.8 effort=360 velocity=12 -> lower=-0.7 upper=0.7 effort=360 velocity=12
- joint r_leg_aky: limit lower=-1 upper=0.7 effort=740 velocity=12 -> lower=-1.06 upper=0.72 effort=740 velocity=12
- joint r_leg_hpx: limit lower=-0.523599 upper=0.523599 effort=530 velocity=12 -> lower=-0.52 upper=0.23 effort=530 velocity=12
- joint r_leg_hpz: limit lower=-0.786794 upper=0.174358 effort=275 velocity=12 -> lower=-0.82 upper=0.2 effort=275 velocity=12

File: software/models/atlas_v5/model_minimal_contact.urdf (robot description, URDF)
Before this commit: robot atlas, 94 links, 93 joints
Joints:
- joint l_arm_lwy: limit lower=-2.9671 upper=2.9671 effort=25 velocity=10 -> lower=-2.82 upper=2.82 effort=25 velocity=10
- joint l_arm_mwx: limit lower=-1.7628 upper=1.7628 effort=25 velocity=10 -> lower=-1.76 upper=1.76 effort=25 velocity=10
- joint l_arm_uwy: limit lower=-3.011 upper=3.011 effort=25 velocity=10 -> lower=-2.98 upper=2.98 effort=25 velocity=10
- joint l_leg_akx: limit lower=-0.8 upper=0.8 effort=360 velocity=12 -> lower=-0.7 upper=0.7 effort=360 velocity=12
- joint l_leg_aky: limit lower=-1 upper=0.7 effort=740 velocity=12 -> lower=-1.06 upper=0.72 effort=740 velocity=12
- joint l_leg_hpx: limit lower=-0.523599 upper=0.523599 effort=530 velocity=12 -> lower=-0.23 upper=0.52 effort=530 velocity=12
- joint l_leg_hpz: limit lower=-0.174358 upper=0.786794 effort=275 velocity=12 -> lower=-0.2 upper=0.82 effort=275 velocity=12
- joint neck_ay: limit lower=-0.602139 upper=1.14319 effort=25 velocity=6.28 -> lower=-0.605 upper=1.16 effort=25 velocity=6.28
- joint r_arm_lwy: limit lower=-2.9671 upper=2.9671 effort=25 velocity=10 -> lower=-2.82 upper=2.82 effort=25 velocity=10
- joint r_arm_mwx: limit lower=-1.7628 upper=1.7628 effort=25 velocity=10 -> lower=-1.76 upper=1.76 effort=25 velocity=10
- joint r_arm_uwy: limit lower=-3.011 upper=3.011 effort=25 velocity=10 -> lower=-2.98 upper=2.98 effort=25 velocity=10
- joint r_leg_akx: limit lower=-0.8 upper=0.8 effort=360 velocity=12 -> lower=-0.7 upper=0.7 effort=360 velocity=12
- joint r_leg_aky: limit lower=-1 upper=0.7 effort=740 velocity=12 -> lower=-1.06 upper=0.72 effort=740 velocity=12
- joint r_leg_hpx: limit lower=-0.523599 upper=0.523599 effort=530 velocity=12 -> lower=-0.52 upper=0.23 effort=530 velocity=12
- joint r_leg_hpz: limit lower=-0.786794 upper=0.174358 effort=275 velocity=12 -> lower=-0.82 upper=0.2 effort=275 velocity=12

Commit message: WIP from on-robot tests

File: software/models/atlas_v5/components/atlas_v5_convex_hull.urdf (robot description, URDF)
Before this commit: robot drc_skeleton, 34 links, 34 joints
Links:
- link pelvis: geometry collision mesh filename=package://atlas_v5/meshes/pelvis_chull.obj; collision sphere radius=0.0

File: software/models/atlas_v5/components/atlas_v5_minimal_contact.urdf (robot description, URDF)
Before this commit: robot drc_skeleton, 34 links, 34 joints
Links:
- link pelvis: geometry collision sphere radius=0.0; collision sphere radius=0.0

File: software/models/atlas_v5/model_convex_hull.urdf (robot description, URDF)
Before this commit: robot atlas, 70 links, 69 joints
Links:
- link pelvis: geometry collision mesh filename=package://atlas_v5/meshes/pelvis_chull.obj; collision sphere radius=0.0

File: software/models/atlas_v5/model_convex_hull_closed_hands.urdf (robot description, URDF)
Before this commit: robot atlas, 70 links, 69 joints
Links:
- link pelvis: geometry collision mesh filename=package://atlas_v5/meshes/pelvis_chull.obj; collision sphere radius=0.0

File: software/models/atlas_v5/model_convex_hull_fingers.urdf (robot description, URDF)
Before this commit: robot atlas, 94 links, 93 joints
Links:
- link pelvis: geometry collision mesh filename=package://atlas_v5/meshes/pelvis_chull.obj; collision sphere radius=0.0

File: software/models/atlas_v5/model_minimal_contact.urdf (robot description, URDF)
Before this commit: robot atlas, 94 links, 93 joints
Links:
- link pelvis: geometry collision sphere radius=0.0; collision sphere radius=0.0
