Commit message: Add mass to robotiq hand models. What?!

File: software/models/atlas_v5/model_LR_RR.urdf (robot description, URDF)
Before this commit: robot atlas, 88 links, 87 joints
Links:
- link left_palm: mass None -> 2.3002
- link right_palm: mass None -> 2.3002

File: software/models/atlas_v5/model_convex_hull_fingers.urdf (robot description, URDF)
Before this commit: robot atlas, 94 links, 93 joints
Links:
- link left_palm: mass None -> 2.3002
- link right_palm: mass None -> 2.3002

File: software/models/atlas_v5/model_minimal_contact.urdf (robot description, URDF)
Before this commit: robot atlas, 94 links, 93 joints
Links:
- removed link left_finger_1_link_0
- removed link left_finger_1_link_1
- removed link left_finger_1_link_2
- removed link left_finger_1_link_3
- removed link left_finger_2_link_0
- removed link left_finger_2_link_1
- removed link left_finger_2_link_2
- removed link left_finger_2_link_3
- removed link left_finger_middle_link_0
- removed link left_finger_middle_link_1
- removed link left_finger_middle_link_2
- removed link left_finger_middle_link_3
- removed link left_palm
- removed link right_finger_1_link_0
- removed link right_finger_1_link_1
- removed link right_finger_1_link_2
- removed link right_finger_1_link_3
- removed link right_finger_2_link_0
- removed link right_finger_2_link_1
- removed link right_finger_2_link_2
- removed link right_finger_2_link_3
- removed link right_finger_middle_link_0
- removed link right_finger_middle_link_1
- removed link right_finger_middle_link_2
- removed link right_finger_middle_link_3
- removed link right_palm
Joints:
- removed joint left_finger_1_joint_1
- removed joint left_finger_1_joint_2
- removed joint left_finger_1_joint_3
- removed joint left_finger_2_joint_1
- removed joint left_finger_2_joint_2
- removed joint left_finger_2_joint_3
- removed joint left_finger_middle_joint_1
- removed joint left_finger_middle_joint_2
- removed joint left_finger_middle_joint_3
- removed joint left_palm_finger_1_joint
- removed joint left_palm_finger_2_joint
- removed joint left_palm_finger_middle_joint
- removed joint left_robotiq_hand_joint
- removed joint right_finger_1_joint_1
- removed joint right_finger_1_joint_2
- removed joint right_finger_1_joint_3
- removed joint right_finger_2_joint_1
- removed joint right_finger_2_joint_2
- removed joint right_finger_2_joint_3
- removed joint right_finger_middle_joint_1
- removed joint right_finger_middle_joint_2
- removed joint right_finger_middle_joint_3
- removed joint right_palm_finger_1_joint
- removed joint right_palm_finger_2_joint
- removed joint right_palm_finger_middle_joint
- removed joint right_robotiq_hand_joint

File: software/models/atlas_v5/xacro/atlas_v5_minimal_contact.xacro (robot description, xacro)
@@ -3,13 +3,4 @@
   <xacro:include filename="../../common_components/multisense_sl/multisense_sl_no_collision.urdf" />
   <xacro:include filename="./atlas_v5_common.xacro" />
-  <xacro:include filename="../../common_components/robotiq_hand_description/robotiq_hand_no_joint_no_collision.xacro" />
-  <!-- Set the initial hand position and orientation by changing 'rpy' and 'xyz'
-  to mach the values in your actual robot. -->
-  <xacro:robotiq_hand side="left" parent="l_hand_force_torque" reflect="1">
-    <origin rpy="0 -1.57079 0" xyz="0 0.06566 0.0"/>
-  </xacro:robotiq_hand>
-  <xacro:robotiq_hand side="right" parent="r_hand_force_torque" reflect="1">
-    <origin rpy="0 -1.57079 0" xyz="0 0.06566 0.0"/>
-  </xacro:robotiq_hand>
   <xacro:robotiq_camera  side_letter="l" reflect="1" parent="l_hand_force_torque" >
     <origin xyz="0.0  0.0 0.0" rpy="0.0 0  0.0"/>

File: software/models/common_components/robotiq_hand_description/cfg/s-model_articulated_macro.xacro (robot description, xacro)
@@ -13,4 +13,10 @@
 		<!-- link list -->
 		<link name="${prefix}palm">
+		    <inertial>
+		      <!-- Total mass of robotiq hand -->
+		      <mass value="2.3002"/>
+		      <origin xyz="0 0 0"/>
+		      <inertia ixx="0.001" ixy="0.0" ixz="0.0" iyy="0.001" iyz="0.0" izz="0.001"/>
+		    </inertial>
 			<visual>
 				<geometry>

File: software/models/common_components/robotiq_hand_description/robotiq_hand.xacro (robot description, xacro)
@@ -113,4 +113,10 @@
     <!-- link list -->
     <link name="${prefix}palm">
+      <inertial>
+        <!-- Total mass of robotiq hand from the associated urdf -->
+        <mass value="2.3002"/>
+        <origin xyz="0 0 0"/>
+        <inertia ixx="0.001" ixy="0.0" ixz="0.0" iyy="0.001" iyz="0.0" izz="0.001"/>
+      </inertial>
       <visual>
         <geometry>

File: software/models/common_components/robotiq_hand_description/robotiq_hand_no_collision.xacro (robot description, xacro)
@@ -83,4 +83,10 @@
     <!-- link list -->
     <link name="${prefix}palm">
+      <inertial>
+        <!-- Total mass of robotiq hand from the associated urdf -->
+        <mass value="2.3002"/>
+        <origin xyz="0 0 0"/>
+        <inertia ixx="0.001" ixy="0.0" ixz="0.0" iyy="0.001" iyz="0.0" izz="0.001"/>
+      </inertial>
       <visual>
         <geometry>

File: software/models/common_components/robotiq_hand_description/robotiq_hand_no_joint.xacro (robot description, xacro)
@@ -113,4 +113,10 @@
     <!-- link list -->
     <link name="${prefix}palm">
+      <inertial>
+        <!-- Total mass of robotiq hand from the associated urdf -->
+        <mass value="2.3002"/>
+        <origin xyz="0 0 0"/>
+        <inertia ixx="0.001" ixy="0.0" ixz="0.0" iyy="0.001" iyz="0.0" izz="0.001"/>
+      </inertial>
       <visual>
         <geometry>

File: software/models/common_components/robotiq_hand_description/robotiq_hand_no_joint_no_collision.xacro (robot description, xacro)
@@ -83,4 +83,10 @@
     <!-- link list -->
     <link name="${prefix}palm">
+      <inertial>
+        <!-- Total mass of robotiq hand from the associated urdf -->
+        <mass value="2.3002"/>
+        <origin xyz="0 0 0"/>
+        <inertia ixx="0.001" ixy="0.0" ixz="0.0" iyy="0.001" iyz="0.0" izz="0.001"/>
+      </inertial>
       <visual>
         <geometry>
