Commit message: working on the new official val model from nasa
this urdf was imported after generation within the valkyrie description

File: software/models/val_description/model.urdf (robot description, URDF)
Before this commit: robot valkyrie, 78 links, 77 joints
Links:
- removed link Ensenso_Frame
- removed link HeadIMU_Frame
- removed link HeadWebcam_Frame
- added link head_hokuyo_frame_offset, mass 1e-07
- added link hokuyo_link, mass 0.057664; collision mesh filename=package://val_description/meshes/multisense_hokuyo.stl; visual mesh filename=package://val_description/meshes/multisense_hokuyo.stl
- added link left_camera_frame_offset, mass 1e-07
- added link right_camera_frame_offset, mass 1e-07
- link Head: geometry collision mesh filename=package://val_description/meshes/head_multisense_no_visor.s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; visual mesh filename=package://val_description/meshes/head_multisense_no_visor.s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
Joints:
- removed joint Ensenso_Offset
- removed joint HeadIMU_Offset
- removed joint HeadWebcam_Offset
- added joint MultisenseSLSpinnyJointFrame: type continuous, parent Head, child hokuyo_link, origin xyz=0.001654 0.0 0.012564 rpy=0.0 0.1309 0.0, axis 1 0 0
- added joint head_hokuyo_frame_joint: type fixed, parent hokuyo_link, child head_hokuyo_frame_offset, origin xyz=0.16018 0.0 -0.015 rpy=3.14 0.0 0.0, axis 0 0 1
- added joint left_camera_frame_joint: type fixed, parent Head, child left_camera_frame_offset, origin xyz=0.18335 0.035 0.0774 rpy=-3.14 0.1309 0.0, axis 0 0 1
- added joint right_camera_frame_joint: type fixed, parent Head, child right_camera_frame_offset, origin xyz=0.18335 -0.035 0.0774 rpy=-3.14 0.1309 0.0, axis 0 0 1
- joint LeftElbowPitch: limit lower=-1.92 upper=0.087 effort=65 velocity=11.5 -> lower=-1.92 upper=-0.087 effort=65 velocity=11.5
- joint LeftForearmYaw: limit lower=-2.36 upper=2.356 effort=26 velocity=5 -> lower=-0.7853 upper=3.9269 effort=26 velocity=5
- joint LeftHipRoll: limit lower=-0.524 upper=0.262 effort=350 velocity=7 -> lower=-0.262 upper=0.524 effort=350 velocity=7
- joint LeftHipYaw: limit lower=-0.524 upper=0.169 effort=190 velocity=5.89 -> lower=-0.169 upper=0.524 effort=190 velocity=5.89
- joint LeftKneePitch: limit lower=-1.902 upper=0.218 effort=350 velocity=6.11 -> lower=-0.218 upper=1.902 effort=350 velocity=6.11
- joint LeftShoulderRoll: limit lower=-3.05 upper=0.155 effort=190 velocity=5.89 -> lower=-1.3962 upper=1.4835 effort=190 velocity=5.89
- joint LeftShoulderYaw: limit lower=-1.57 upper=1.7 effort=65 velocity=11.5 -> lower=-1.57 upper=1.5707 effort=65 velocity=11.5
- joint LeftWristPitch: limit lower=-0.524 upper=0.436 effort=14 velocity=1 -> lower=-0.873 upper=0.698 effort=14 velocity=1
- joint LeftWristRoll: limit lower=-0.873 upper=0.698 effort=14 velocity=1 -> lower=-0.436 upper=0.524 effort=14 velocity=1
- joint LowerNeckPitch: limit lower=-1.57 upper=0 effort=26 velocity=5 -> lower=0 upper=1.57 effort=26 velocity=5
- joint RightElbowPitch: limit lower=-1.92 upper=0.087 effort=65 velocity=11.5 -> lower=0.087 upper=1.92 effort=65 velocity=11.5
- joint RightForearmYaw: limit lower=-2.36 upper=2.356 effort=26 velocity=5 -> lower=-0.7853 upper=3.9269 effort=26 velocity=5
- joint RightKneePitch: limit lower=-1.902 upper=0.218 effort=350 velocity=6.11 -> lower=-0.218 upper=1.902 effort=350 velocity=6.11
- joint RightShoulderRoll: limit lower=-3.05 upper=0.155 effort=190 velocity=5.89 -> lower=-1.4835 upper=1.3962 effort=190 velocity=5.89
- joint RightShoulderYaw: limit lower=-1.57 upper=1.7 effort=65 velocity=11.5 -> lower=-1.57 upper=1.5707 effort=65 velocity=11.5
- joint RightWristPitch: limit lower=-0.524 upper=0.436 effort=14 velocity=1 -> lower=-0.698 upper=0.873 effort=14 velocity=1
- joint RightWristRoll: limit lower=-0.873 upper=0.698 effort=14 velocity=1 -> lower=-0.524 upper=0.436 effort=14 velocity=1

Commit message: made the fingers and multisense fixed for now.
this allows simple joint planning to work in ddapp. next: ik

File: software/models/val_description/model.urdf (robot description, URDF)
Before this commit: robot valkyrie, 79 links, 78 joints
Joints:
- joint LeftIndexFingerPitch1: limit lower=-0.087 upper=0.087 effort=10 velocity=1 -> (none); type revolute -> fixed
- joint LeftIndexFingerPitch2: limit lower=-1.658 upper=0.175 effort=10 velocity=1 -> (none); type revolute -> fixed
- joint LeftIndexFingerPitch3: limit lower=-1.92 upper=0 effort=10 velocity=1 -> (none); type revolute -> fixed
- joint LeftMiddleFingerPitch1: limit lower=-1.658 upper=0.175 effort=10 velocity=1 -> (none); type revolute -> fixed
- joint LeftMiddleFingerPitch2: limit lower=-1.92 upper=0 effort=10 velocity=1 -> (none); type revolute -> fixed
- joint LeftMiddleFingerPitch3: limit lower=-1.57 upper=0.175 effort=10 velocity=1 -> (none); type revolute -> fixed
- joint LeftPinkyPitch1: limit lower=-0.262 upper=0.0 effort=10 velocity=1 -> (none); type revolute -> fixed
- joint LeftPinkyPitch2: limit lower=-1.658 upper=0.175 effort=10 velocity=1 -> (none); type revolute -> fixed
- joint LeftPinkyPitch3: limit lower=-1.92 upper=0 effort=10 velocity=1 -> (none); type revolute -> fixed
- joint LeftThumbPitch1: axis 1 0 0 -> 0 0 1; limit lower=-1.658 upper=0.175 effort=10 velocity=1 -> (none); type revolute -> fixed
- joint LeftThumbPitch2: axis 1 0 0 -> 0 0 1; limit lower=-1.92 upper=0.0 effort=10 velocity=1 -> (none); type revolute -> fixed
- joint LeftThumbPitch3: axis 1 0 0 -> 0 0 1; limit lower=-1.57 upper=0.175 effort=10 velocity=1 -> (none); type revolute -> fixed
- joint LeftThumbRoll: axis 0 1 0 -> 0 0 1; limit lower=-0.087 upper=2.356 effort=10 velocity=1 -> (none); type revolute -> fixed
- joint MultisenseSLSpinnyJointFrame: axis 1 0 0 -> 0 0 1; type continuous -> fixed
- joint RightIndexFingerPitch1: limit lower=-0.087 upper=0.087 effort=10 velocity=1 -> (none); type revolute -> fixed
- joint RightIndexFingerPitch2: limit lower=-1.658 upper=0.175 effort=10 velocity=1 -> (none); type revolute -> fixed
- joint RightIndexFingerPitch3: limit lower=-1.92 upper=0 effort=10 velocity=1 -> (none); type revolute -> fixed
- joint RightMiddleFingerPitch1: limit lower=-1.658 upper=0.175 effort=10 velocity=1 -> (none); type revolute -> fixed
- joint RightMiddleFingerPitch2: limit lower=-1.92 upper=0 effort=10 velocity=1 -> (none); type revolute -> fixed
- joint RightMiddleFingerPitch3: limit lower=-1.57 upper=0.175 effort=10 velocity=1 -> (none); type revolute -> fixed
- joint RightPinkyPitch1: limit lower=-0.262 upper=0.0 effort=10 velocity=1 -> (none); type revolute -> fixed
- joint RightPinkyPitch2: limit lower=-1.658 upper=0.175 effort=10 velocity=1 -> (none); type revolute -> fixed
- joint RightPinkyPitch3: limit lower=-1.92 upper=0 effort=10 velocity=1 -> (none); type revolute -> fixed
- joint RightThumbPitch1: axis 1 0 0 -> 0 0 1; limit lower=-1.658 upper=0.175 effort=10 velocity=1 -> (none); type revolute -> fixed
- joint RightThumbPitch2: axis 1 0 0 -> 0 0 1; limit lower=-1.92 upper=0.0 effort=10 velocity=1 -> (none); type revolute -> fixed
- joint RightThumbPitch3: axis 1 0 0 -> 0 0 1; limit lower=-1.57 upper=0.175 effort=10 velocity=1 -> (none); type revolute -> fixed
- joint RightThumbRoll: axis 0 1 0 -> 0 0 1; limit lower=-0.087 upper=2.356 effort=10 velocity=1 -> (none); type revolute -> fixed

Commit message: further changes to the urdf which are needed for quasi static balancing

File: software/models/val_description/model.urdf (robot description, URDF)
Before this commit: robot valkyrie, 79 links, 78 joints
Links:
- link LeftFoot: geometry collision mesh filename=package://val_description/meshes/foot_Left.stl; collision sphere radius=0.0
- link RightFoot: geometry collision mesh filename=package://val_description/meshes/foot_Right.stl; collision sphere radius=0.0

Commit message: moving meshes around to match NASA

File: software/models/val_description/model.urdf (robot description, URDF)
Before this commit: robot valkyrie, 79 links, 78 joints
Links:
- link Head: geometry collision mesh filename=package://val_description/meshes/head/head_multisense_no_vi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; visual mesh filename=package://val_description/meshes/head/head_multisense_no_vi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
- link LeftAnklePitchLink: geometry collision mesh filename=package://val_description/meshes/legs/lj5.stl; visual mesh filename=package://val_description/meshes/legs/lj5.stl
- link LeftElbowPitchLink: geometry collision mesh filename=package://val_description/meshes/arms/aj4_Left.stl; visual mesh filename=package://val_description/meshes/arms/aj4_Left.stl
- link LeftFoot: geometry collision mesh filename=package://val_description/meshes/legs/foot_Left.stl; collision sphere radius=0.0
- link LeftForearmLink: geometry collision mesh filename=package://val_description/meshes/arms/aj5_Left.stl; visual mesh filename=package://val_description/meshes/arms/aj5_Left.stl
- link LeftHipPitchLink: geometry collision mesh filename=package://val_description/meshes/legs/lj3_Left.stl; visual mesh filename=package://val_description/meshes/legs/lj3_Left.stl
- link LeftHipRollLink: geometry collision mesh filename=package://val_description/meshes/legs/lj2_Left.stl; visual mesh filename=package://val_description/meshes/legs/lj2_Left.stl
- link LeftHipYawLink: geometry collision mesh filename=package://val_description/meshes/legs/lj1_Left.stl; visual mesh filename=package://val_description/meshes/legs/lj1_Left.stl
- link LeftIndexFingerPitch1Link: geometry collision mesh filename=package://val_description/meshes/fingers/indexj1_Left.stl; visual mesh filename=package://val_description/meshes/fingers/indexj1_Left.stl
- link LeftIndexFingerPitch2Link: geometry collision mesh filename=package://val_description/meshes/fingers/indexj2_Left.stl; visual mesh filename=package://val_description/meshes/fingers/indexj2_Left.stl
- link LeftIndexFingerPitch3Link: geometry collision mesh filename=package://val_description/meshes/fingers/indexj3_Left.stl; visual mesh filename=package://val_description/meshes/fingers/indexj3_Left.stl
- link LeftKneePitchLink: geometry collision mesh filename=package://val_description/meshes/legs/lj4_Left.stl; visual mesh filename=package://val_description/meshes/legs/lj4_Left.stl
- link LeftMiddleFingerPitch1Link: geometry collision mesh filename=package://val_description/meshes/fingers/middlej1_Left.stl; visual mesh filename=package://val_description/meshes/fingers/middlej1_Left.stl
- link LeftMiddleFingerPitch2Link: geometry collision mesh filename=package://val_description/meshes/fingers/middlej2_Left.stl; visual mesh filename=package://val_description/meshes/fingers/middlej2_Left.stl
- link LeftMiddleFingerPitch3Link: geometry collision mesh filename=package://val_description/meshes/fingers/middlej3_Left.stl; visual mesh filename=package://val_description/meshes/fingers/middlej3_Left.stl
- link LeftPalm: geometry collision mesh filename=package://val_description/meshes/arms/palm_Left.stl; visual mesh filename=package://val_description/meshes/arms/palm_Left.stl
- link LeftPinkyPitch1Link: geometry collision mesh filename=package://val_description/meshes/fingers/pinkyj1_Left.stl; visual mesh filename=package://val_description/meshes/fingers/pinkyj1_Left.stl
- link LeftPinkyPitch2Link: geometry collision mesh filename=package://val_description/meshes/fingers/pinkyj2_Left.stl; visual mesh filename=package://val_description/meshes/fingers/pinkyj2_Left.stl
- link LeftPinkyPitch3Link: geometry collision mesh filename=package://val_description/meshes/fingers/pinkyj3_Left.stl; visual mesh filename=package://val_description/meshes/fingers/pinkyj3_Left.stl
- link LeftShoulderPitchLink: geometry collision mesh filename=package://val_description/meshes/arms/aj1_Left.stl; visual mesh filename=package://val_description/meshes/arms/aj1_Left.stl
- link LeftShoulderRollLink: geometry collision mesh filename=package://val_description/meshes/arms/aj2_Left.stl; visual mesh filename=package://val_description/meshes/arms/aj2_Left.stl
- link LeftShoulderYawLink: geometry collision mesh filename=package://val_description/meshes/arms/aj3_Left.stl; visual mesh filename=package://val_description/meshes/arms/aj3_Left.stl
- link LeftThumbPitch1Link: geometry collision mesh filename=package://val_description/meshes/fingers/thumbj2_Left.stl; visual mesh filename=package://val_description/meshes/fingers/thumbj2_Left.stl
- link LeftThumbPitch2Link: geometry collision mesh filename=package://val_description/meshes/fingers/thumbj3_Left.stl; visual mesh filename=package://val_description/meshes/fingers/thumbj3_Left.stl
- link LeftThumbPitch3Link: geometry collision mesh filename=package://val_description/meshes/fingers/thumbj4_Left.stl; visual mesh filename=package://val_description/meshes/fingers/thumbj4_Left.stl
- link LeftThumbRollLink: geometry collision mesh filename=package://val_description/meshes/fingers/thumbj1_Left.stl; visual mesh filename=package://val_description/meshes/fingers/thumbj1_Left.stl
- link LeftWristRollLink: geometry collision mesh filename=package://val_description/meshes/arms/aj6_Left.stl; visual mesh filename=package://val_description/meshes/arms/aj6_Left.stl
- link LowerNeckPitchLink: geometry collision mesh filename=package://val_description/meshes/head/neckj1.stl; visual mesh filename=package://val_description/meshes/head/neckj1.stl
- link NeckYawLink: geometry collision mesh filename=package://val_description/meshes/head/neckj2.stl; visual mesh filename=package://val_description/meshes/head/neckj2.stl
- link Pelvis: geometry collision mesh filename=package://val_description/meshes/pelvis/pelvis.stl; visual mesh filename=package://val_description/meshes/pelvis/pelvis.stl
- link RightAnklePitchLink: geometry collision mesh filename=package://val_description/meshes/legs/lj5.stl; visual mesh filename=package://val_description/meshes/legs/lj5.stl
- link RightElbowPitchLink: geometry collision mesh filename=package://val_description/meshes/arms/aj4_Right.stl; visual mesh filename=package://val_description/meshes/arms/aj4_Right.stl
- link RightFoot: geometry collision mesh filename=package://val_description/meshes/legs/foot_Right.stl; collision sphere radius=0.0
- link RightForearmLink: geometry collision mesh filename=package://val_description/meshes/arms/aj5_Right.stl; visual mesh filename=package://val_description/meshes/arms/aj5_Right.stl
- link RightHipPitchLink: geometry collision mesh filename=package://val_description/meshes/legs/lj3_Right.stl; visual mesh filename=package://val_description/meshes/legs/lj3_Right.stl
- link RightHipRollLink: geometry collision mesh filename=package://val_description/meshes/legs/lj2_Right.stl; visual mesh filename=package://val_description/meshes/legs/lj2_Right.stl
- link RightHipYawLink: geometry collision mesh filename=package://val_description/meshes/legs/lj1_Right.stl; visual mesh filename=package://val_description/meshes/legs/lj1_Right.stl
- link RightIndexFingerPitch1Link: geometry collision mesh filename=package://val_description/meshes/fingers/indexj1_Right.stl; visual mesh filename=package://val_description/meshes/fingers/indexj1_Right.stl
- link RightIndexFingerPitch2Link: geometry collision mesh filename=package://val_description/meshes/fingers/indexj2_Right.stl; visual mesh filename=package://val_description/meshes/fingers/indexj2_Right.stl
- link RightIndexFingerPitch3Link: geometry collision mesh filename=package://val_description/meshes/fingers/indexj3_Right.stl; visual mesh filename=package://val_description/meshes/fingers/indexj3_Right.stl
- link RightKneePitchLink: geometry collision mesh filename=package://val_description/meshes/legs/lj4_Right.stl; visual mesh filename=package://val_description/meshes/legs/lj4_Right.stl
- link RightMiddleFingerPitch1Link: geometry collision mesh filename=package://val_description/meshes/fingers/middlej1_Right.stl; visual mesh filename=package://val_description/meshes/fingers/middlej1_Right.stl
- link RightMiddleFingerPitch2Link: geometry collision mesh filename=package://val_description/meshes/fingers/middlej2_Right.stl; visual mesh filename=package://val_description/meshes/fingers/middlej2_Right.stl
- link RightMiddleFingerPitch3Link: geometry collision mesh filename=package://val_description/meshes/fingers/middlej3_Right.stl; visual mesh filename=package://val_description/meshes/fingers/middlej3_Right.stl
- link RightPalm: geometry collision mesh filename=package://val_description/meshes/arms/palm_Right.stl; visual mesh filename=package://val_description/meshes/arms/palm_Right.stl
- link RightPinkyPitch1Link: geometry collision mesh filename=package://val_description/meshes/fingers/pinkyj1_Right.stl; visual mesh filename=package://val_description/meshes/fingers/pinkyj1_Right.stl
- link RightPinkyPitch2Link: geometry collision mesh filename=package://val_description/meshes/fingers/pinkyj2_Right.stl; visual mesh filename=package://val_description/meshes/fingers/pinkyj2_Right.stl
- link RightPinkyPitch3Link: geometry collision mesh filename=package://val_description/meshes/fingers/pinkyj3_Right.stl; visual mesh filename=package://val_description/meshes/fingers/pinkyj3_Right.stl
- link RightShoulderPitchLink: geometry collision mesh filename=package://val_description/meshes/arms/aj1_Right.stl; visual mesh filename=package://val_description/meshes/arms/aj1_Right.stl
- link RightShoulderRollLink: geometry collision mesh filename=package://val_description/meshes/arms/aj2_Right.stl; visual mesh filename=package://val_description/meshes/arms/aj2_Right.stl
- link RightShoulderYawLink: geometry collision mesh filename=package://val_description/meshes/arms/aj3_Right.stl; visual mesh filename=package://val_description/meshes/arms/aj3_Right.stl
- link RightThumbPitch1Link: geometry collision mesh filename=package://val_description/meshes/fingers/thumbj2_Right.stl; visual mesh filename=package://val_description/meshes/fingers/thumbj2_Right.stl
- link RightThumbPitch2Link: geometry collision mesh filename=package://val_description/meshes/fingers/thumbj3_Right.stl; visual mesh filename=package://val_description/meshes/fingers/thumbj3_Right.stl
- link RightThumbPitch3Link: geometry collision mesh filename=package://val_description/meshes/fingers/thumbj4_Right.stl; visual mesh filename=package://val_description/meshes/fingers/thumbj4_Right.stl
- link RightThumbRollLink: geometry collision mesh filename=package://val_description/meshes/fingers/thumbj1_Right.stl; visual mesh filename=package://val_description/meshes/fingers/thumbj1_Right.stl
- link RightWristRollLink: geometry collision mesh filename=package://val_description/meshes/arms/aj6_Right.stl; visual mesh filename=package://val_description/meshes/arms/aj6_Right.stl
- link Torso: geometry collision mesh filename=package://val_description/meshes/torso/torso.stl; visual mesh filename=package://val_description/meshes/torso/torso.stl
- link TorsoPitchLink: geometry collision mesh filename=package://val_description/meshes/torso/torsopitch.stl; visual mesh filename=package://val_description/meshes/torso/torsopitch.stl
- link TorsoYawLink: geometry collision mesh filename=package://val_description/meshes/torso/torsoyaw.stl; visual mesh filename=package://val_description/meshes/torso/torsoyaw.stl
- link hokuyo_link: geometry collision mesh filename=package://val_description/meshes/head/multisense_hokuyo.stl; visual mesh filename=package://val_description/meshes/head/multisense_hokuyo.stl
Joints:
- joint LeftElbowPitch: limit lower=-1.92 upper=-0.087 effort=65 velocity=11.5 -> lower=-1.92 upper=0.0 effort=65 velocity=11.5
- joint RightElbowPitch: limit lower=0.087 upper=1.92 effort=65 velocity=11.5 -> lower=-0.0 upper=1.92 effort=65 velocity=11.5
- joint TorsoPitch: limit lower=-0.698 upper=0.087 effort=150 velocity=9 -> lower=-0.087 upper=0.698 effort=150 velocity=9
