Commit message: final version provided in vtp and dae format with png textures

File: software/models/val_description/model.urdf (robot description, URDF)
Before this commit: robot valkyrie, 79 links, 78 joints
Links:
- link Head: geometry collision mesh filename=package://val_description/meshes/head/head_multisense.obj; visual mesh filename=package://val_description/meshes/head/head_multisense.obj
- link LeftAnklePitchLink: geometry collision mesh filename=package://val_description/meshes/legs/lj5.obj; visual mesh filename=package://val_description/meshes/legs/lj5.obj
- link LeftElbowPitchLink: geometry collision mesh filename=package://val_description/meshes/arms/aj4_Left.obj; visual mesh filename=package://val_description/meshes/arms/aj4_Left.obj
- link LeftFoot: geometry collision mesh filename=package://val_description/meshes/legs/foot_Left.obj; collision sphere radius=0.0
- link LeftForearmLink: geometry collision mesh filename=package://val_description/meshes/arms/aj5_Left.obj; visual mesh filename=package://val_description/meshes/arms/aj5_Left.obj
- link LeftHipPitchLink: geometry collision mesh filename=package://val_description/meshes/legs/lj3_Left.obj; visual mesh filename=package://val_description/meshes/legs/lj3_Left.obj
- link LeftHipRollLink: geometry collision mesh filename=package://val_description/meshes/legs/lj2_Left.obj; visual mesh filename=package://val_description/meshes/legs/lj2_Left.obj
- link LeftHipYawLink: geometry collision mesh filename=package://val_description/meshes/legs/lj1_Left.obj; visual mesh filename=package://val_description/meshes/legs/lj1_Left.obj
- link LeftIndexFingerPitch1Link: geometry collision mesh filename=package://val_description/meshes/fingers/indexj1_Left.obj; visual mesh filename=package://val_description/meshes/fingers/indexj1_Left.obj
- link LeftIndexFingerPitch2Link: geometry collision mesh filename=package://val_description/meshes/fingers/indexj2_Left.obj; visual mesh filename=package://val_description/meshes/fingers/indexj2_Left.obj
- link LeftIndexFingerPitch3Link: geometry collision mesh filename=package://val_description/meshes/fingers/indexj3_Left.obj; visual mesh filename=package://val_description/meshes/fingers/indexj3_Left.obj
- link LeftKneePitchLink: geometry collision mesh filename=package://val_description/meshes/legs/lj4_Left.obj; visual mesh filename=package://val_description/meshes/legs/lj4_Left.obj
- link LeftMiddleFingerPitch1Link: geometry collision mesh filename=package://val_description/meshes/fingers/middlej1_Left.obj; visual mesh filename=package://val_description/meshes/fingers/middlej1_Left.obj
- link LeftMiddleFingerPitch2Link: geometry collision mesh filename=package://val_description/meshes/fingers/middlej2_Left.obj; visual mesh filename=package://val_description/meshes/fingers/middlej2_Left.obj
- link LeftMiddleFingerPitch3Link: geometry collision mesh filename=package://val_description/meshes/fingers/middlej3_Left.obj; visual mesh filename=package://val_description/meshes/fingers/middlej3_Left.obj
- link LeftPalm: geometry collision mesh filename=package://val_description/meshes/arms/palm_Left.obj; visual mesh filename=package://val_description/meshes/arms/palm_Left.obj
- link LeftPinkyPitch1Link: geometry collision mesh filename=package://val_description/meshes/fingers/pinkyj1_Left.obj; visual mesh filename=package://val_description/meshes/fingers/pinkyj1_Left.obj
- link LeftPinkyPitch2Link: geometry collision mesh filename=package://val_description/meshes/fingers/pinkyj2_Left.obj; visual mesh filename=package://val_description/meshes/fingers/pinkyj2_Left.obj
- link LeftPinkyPitch3Link: geometry collision mesh filename=package://val_description/meshes/fingers/pinkyj3_Left.obj; visual mesh filename=package://val_description/meshes/fingers/pinkyj3_Left.obj
- link LeftShoulderPitchLink: geometry collision mesh filename=package://val_description/meshes/arms/aj1_Left.obj; visual mesh filename=package://val_description/meshes/arms/aj1_Left.obj
- link LeftShoulderRollLink: geometry collision mesh filename=package://val_description/meshes/arms/aj2_Left.obj; visual mesh filename=package://val_description/meshes/arms/aj2_Left.obj
- link LeftShoulderYawLink: geometry collision mesh filename=package://val_description/meshes/arms/aj3_Left.obj; visual mesh filename=package://val_description/meshes/arms/aj3_Left.obj
- link LeftThumbPitch1Link: geometry collision mesh filename=package://val_description/meshes/fingers/thumbj2_Left.obj; visual mesh filename=package://val_description/meshes/fingers/thumbj2_Left.obj
- link LeftThumbPitch2Link: geometry collision mesh filename=package://val_description/meshes/fingers/thumbj3_Left.obj; visual mesh filename=package://val_description/meshes/fingers/thumbj3_Left.obj
- link LeftThumbPitch3Link: geometry collision mesh filename=package://val_description/meshes/fingers/thumbj4_Left.obj; visual mesh filename=package://val_description/meshes/fingers/thumbj4_Left.obj
- link LeftThumbRollLink: geometry collision mesh filename=package://val_description/meshes/fingers/thumbj1_Left.obj; visual mesh filename=package://val_description/meshes/fingers/thumbj1_Left.obj
- link LeftWristRollLink: geometry collision mesh filename=package://val_description/meshes/arms/aj6_Left.obj; visual mesh filename=package://val_description/meshes/arms/aj6_Left.obj
- link LowerNeckPitchLink: geometry collision mesh filename=package://val_description/meshes/head/neckj1.obj; visual mesh filename=package://val_description/meshes/head/neckj1.obj
- link NeckYawLink: geometry collision mesh filename=package://val_description/meshes/head/neckj2.obj; visual mesh filename=package://val_description/meshes/head/neckj2.obj
- link Pelvis: geometry collision mesh filename=package://val_description/meshes/pelvis/pelvis.obj; visual mesh filename=package://val_description/meshes/pelvis/pelvis.obj
- link RightAnklePitchLink: geometry collision mesh filename=package://val_description/meshes/legs/lj5.obj; visual mesh filename=package://val_description/meshes/legs/lj5.obj
- link RightElbowPitchLink: geometry collision mesh filename=package://val_description/meshes/arms/aj4_Right.obj; visual mesh filename=package://val_description/meshes/arms/aj4_Right.obj
- link RightFoot: geometry collision mesh filename=package://val_description/meshes/legs/foot_Right.obj; collision sphere radius=0.0
- link RightForearmLink: geometry collision mesh filename=package://val_description/meshes/arms/aj5_Right.obj; visual mesh filename=package://val_description/meshes/arms/aj5_Right.obj
- link RightHipPitchLink: geometry collision mesh filename=package://val_description/meshes/legs/lj3_Right.obj; visual mesh filename=package://val_description/meshes/legs/lj3_Right.obj
- link RightHipRollLink: geometry collision mesh filename=package://val_description/meshes/legs/lj2_Right.obj; visual mesh filename=package://val_description/meshes/legs/lj2_Right.obj
- link RightHipYawLink: geometry collision mesh filename=package://val_description/meshes/legs/lj1_Right.obj; visual mesh filename=package://val_description/meshes/legs/lj1_Right.obj
- link RightIndexFingerPitch1Link: geometry collision mesh filename=package://val_description/meshes/fingers/indexj1_Right.obj; visual mesh filename=package://val_description/meshes/fingers/indexj1_Right.obj
- link RightIndexFingerPitch2Link: geometry collision mesh filename=package://val_description/meshes/fingers/indexj2_Right.obj; visual mesh filename=package://val_description/meshes/fingers/indexj2_Right.obj
- link RightIndexFingerPitch3Link: geometry collision mesh filename=package://val_description/meshes/fingers/indexj3_Right.obj; visual mesh filename=package://val_description/meshes/fingers/indexj3_Right.obj
- link RightKneePitchLink: geometry collision mesh filename=package://val_description/meshes/legs/lj4_Right.obj; visual mesh filename=package://val_description/meshes/legs/lj4_Right.obj
- link RightMiddleFingerPitch1Link: geometry collision mesh filename=package://val_description/meshes/fingers/middlej1_Right.obj; visual mesh filename=package://val_description/meshes/fingers/middlej1_Right.obj
- link RightMiddleFingerPitch2Link: geometry collision mesh filename=package://val_description/meshes/fingers/middlej2_Right.obj; visual mesh filename=package://val_description/meshes/fingers/middlej2_Right.obj
- link RightMiddleFingerPitch3Link: geometry collision mesh filename=package://val_description/meshes/fingers/middlej3_Right.obj; visual mesh filename=package://val_description/meshes/fingers/middlej3_Right.obj
- link RightPalm: geometry collision mesh filename=package://val_description/meshes/arms/palm_Right.obj; visual mesh filename=package://val_description/meshes/arms/palm_Right.obj
- link RightPinkyPitch1Link: geometry collision mesh filename=package://val_description/meshes/fingers/pinkyj1_Right.obj; visual mesh filename=package://val_description/meshes/fingers/pinkyj1_Right.obj
- link RightPinkyPitch2Link: geometry collision mesh filename=package://val_description/meshes/fingers/pinkyj2_Right.obj; visual mesh filename=package://val_description/meshes/fingers/pinkyj2_Right.obj
- link RightPinkyPitch3Link: geometry collision mesh filename=package://val_description/meshes/fingers/pinkyj3_Right.obj; visual mesh filename=package://val_description/meshes/fingers/pinkyj3_Right.obj
- link RightShoulderPitchLink: geometry collision mesh filename=package://val_description/meshes/arms/aj1_Right.obj; visual mesh filename=package://val_description/meshes/arms/aj1_Right.obj
- link RightShoulderRollLink: geometry collision mesh filename=package://val_description/meshes/arms/aj2_Right.obj; visual mesh filename=package://val_description/meshes/arms/aj2_Right.obj
- link RightShoulderYawLink: geometry collision mesh filename=package://val_description/meshes/arms/aj3_Right.obj; visual mesh filename=package://val_description/meshes/arms/aj3_Right.obj
- link RightThumbPitch1Link: geometry collision mesh filename=package://val_description/meshes/fingers/thumbj2_Right.obj; visual mesh filename=package://val_description/meshes/fingers/thumbj2_Right.obj
- link RightThumbPitch2Link: geometry collision mesh filename=package://val_description/meshes/fingers/thumbj3_Right.obj; visual mesh filename=package://val_description/meshes/fingers/thumbj3_Right.obj
- link RightThumbPitch3Link: geometry collision mesh filename=package://val_description/meshes/fingers/thumbj4_Right.obj; visual mesh filename=package://val_description/meshes/fingers/thumbj4_Right.obj
- link RightThumbRollLink: geometry collision mesh filename=package://val_description/meshes/fingers/thumbj1_Right.obj; visual mesh filename=package://val_description/meshes/fingers/thumbj1_Right.obj
- link RightWristRollLink: geometry collision mesh filename=package://val_description/meshes/arms/aj6_Right.obj; visual mesh filename=package://val_description/meshes/arms/aj6_Right.obj
- link Torso: geometry collision mesh filename=package://val_description/meshes/torso/torso.obj; visual mesh filename=package://val_description/meshes/torso/torso.obj
- link TorsoPitchLink: geometry collision mesh filename=package://val_description/meshes/torso/torsopitch.obj; visual mesh filename=package://val_description/meshes/torso/torsopitch.obj
- link TorsoYawLink: geometry collision mesh filename=package://val_description/meshes/torso/torsoyaw.obj; visual mesh filename=package://val_description/meshes/torso/torsoyaw.obj
- link hokuyo_link: geometry collision mesh filename=package://val_description/meshes/head/multisense_hokuyo.obj; visual mesh filename=package://val_description/meshes/head/multisense_hokuyo.obj

Commit message: some of the new urdf mods

File: software/models/val_description/model.urdf (robot description, URDF)
Before this commit: robot valkyrie, 79 links, 78 joints
Joints:
- joint MultisenseSLSpinnyJointFrame: axis 0 0 1 -> 1 0 0

Commit message: minor change

File: software/models/val_description/model.urdf (robot description, URDF)
Before this commit: robot valkyrie, 79 links, 78 joints
Joints:
- joint LeftLegSixAxis_Offset: origin xyz=0.022 0.0 -0.059 rpy=3.14 0.0 -1.047 -> xyz=0.0215594 0.0 -0.0585488 rpy=3.14 0.0 -1.047
- joint RightLegSixAxis_Offset: origin xyz=0.022 0.0 -0.059 rpy=3.14 0.0 -1.047 -> xyz=0.0215594 0.0 -0.0585488 rpy=3.14 0.0 -1.047
