Commit message: generalize robot to use original valkyrie joint names - except for feet

File: software/models/common_components/hand_factory/valkyrie_hand_left.urdf (robot description, URDF)
Before this commit: robot valkyrie_hand_left, 17 links, 16 joints
Links:
- link /v1/LeftLittleDistalPhalanx: geometry collision mesh filename=package://valkyrie_original/meshes/sf3_ssf4.stl; visual mesh filename=package://valkyrie_original/meshes/sf3_ssf4.stl
- link /v1/LeftLittleMedialPhalanx: geometry collision mesh filename=package://valkyrie_original/meshes/sf2_ssf3.stl; visual mesh filename=package://valkyrie_original/meshes/sf2_ssf3.stl
- link /v1/LeftLittleProximalPhalanx: geometry collision mesh filename=package://valkyrie_original/meshes/ssf2_Left.stl; visual mesh filename=package://valkyrie_original/meshes/ssf2_Left.stl
- link /v1/LeftMedialMetacarpal: geometry collision mesh filename=package://valkyrie_original/meshes/ssf1_Left.stl; visual mesh filename=package://valkyrie_original/meshes/ssf1_Left.stl
- link /v1/LeftMiddleDistalPhalanx: geometry collision mesh filename=package://valkyrie_original/meshes/sf3_ssf4.stl; visual mesh filename=package://valkyrie_original/meshes/sf3_ssf4.stl
- link /v1/LeftMiddleMedialPhalanx: geometry collision mesh filename=package://valkyrie_original/meshes/sf2_ssf3.stl; visual mesh filename=package://valkyrie_original/meshes/sf2_ssf3.stl
- link /v1/LeftMiddleProximalPhalanx: geometry collision mesh filename=package://valkyrie_original/meshes/sf1.stl; visual mesh filename=package://valkyrie_original/meshes/sf1.stl
- link /v1/LeftPrimaryDistalPhalanx: geometry collision mesh filename=package://valkyrie_original/meshes/pf4.stl; visual mesh filename=package://valkyrie_original/meshes/pf4.stl
- link /v1/LeftPrimaryMedialPhalanx: geometry collision mesh filename=package://valkyrie_original/meshes/pf3.stl; visual mesh filename=package://valkyrie_original/meshes/pf3.stl
- link /v1/LeftPrimaryMetacarpal: geometry collision mesh filename=package://valkyrie_original/meshes/pf1.stl; visual mesh filename=package://valkyrie_original/meshes/pf1.stl
- link /v1/LeftPrimaryProximalPhalanx: geometry collision mesh filename=package://valkyrie_original/meshes/pf2.stl; visual mesh filename=package://valkyrie_original/meshes/pf2.stl
- link /v1/LeftThumbDistalPhalanx: geometry collision mesh filename=package://valkyrie_original/meshes/tf4.stl; visual mesh filename=package://valkyrie_original/meshes/tf4.stl
- link /v1/LeftThumbMedialPhalanx: geometry collision mesh filename=package://valkyrie_original/meshes/tf3.stl; visual mesh filename=package://valkyrie_original/meshes/tf3.stl
- link /v1/LeftThumbMetacarpal: geometry collision mesh filename=package://valkyrie_original/meshes/tf1_Left.stl; visual mesh filename=package://valkyrie_original/meshes/tf1_Left.stl
- link /v1/LeftThumbProximalPhalanx: geometry collision mesh filename=package://valkyrie_original/meshes/tf2.stl; visual mesh filename=package://valkyrie_original/meshes/tf2.stl
- link left_palm: geometry collision mesh filename=package://valkyrie_original/meshes/palm_Left.stl; visual mesh filename=package://valkyrie_original/meshes/palm_Left.stl

File: software/models/common_components/hand_factory/valkyrie_hand_right.urdf (robot description, URDF)
Before this commit: robot valkyrie_hand_right, 17 links, 16 joints
Links:
- link /v1/RightLittleDistalPhalanx: geometry collision mesh filename=package://valkyrie_original/meshes/sf3_ssf4.stl; visual mesh filename=package://valkyrie_original/meshes/sf3_ssf4.stl
- link /v1/RightLittleMedialPhalanx: geometry collision mesh filename=package://valkyrie_original/meshes/sf2_ssf3.stl; visual mesh filename=package://valkyrie_original/meshes/sf2_ssf3.stl
- link /v1/RightLittleProximalPhalanx: geometry collision mesh filename=package://valkyrie_original/meshes/ssf2_Right.stl; visual mesh filename=package://valkyrie_original/meshes/ssf2_Right.stl
- link /v1/RightMedialMetacarpal: geometry collision mesh filename=package://valkyrie_original/meshes/ssf1_Right.stl; visual mesh filename=package://valkyrie_original/meshes/ssf1_Right.stl
- link /v1/RightMiddleDistalPhalanx: geometry collision mesh filename=package://valkyrie_original/meshes/sf3_ssf4.stl; visual mesh filename=package://valkyrie_original/meshes/sf3_ssf4.stl
- link /v1/RightMiddleMedialPhalanx: geometry collision mesh filename=package://valkyrie_original/meshes/sf2_ssf3.stl; visual mesh filename=package://valkyrie_original/meshes/sf2_ssf3.stl
- link /v1/RightMiddleProximalPhalanx: geometry collision mesh filename=package://valkyrie_original/meshes/sf1.stl; visual mesh filename=package://valkyrie_original/meshes/sf1.stl
- link /v1/RightPrimaryDistalPhalanx: geometry collision mesh filename=package://valkyrie_original/meshes/pf4.stl; visual mesh filename=package://valkyrie_original/meshes/pf4.stl
- link /v1/RightPrimaryMedialPhalanx: geometry collision mesh filename=package://valkyrie_original/meshes/pf3.stl; visual mesh filename=package://valkyrie_original/meshes/pf3.stl
- link /v1/RightPrimaryMetacarpal: geometry collision mesh filename=package://valkyrie_original/meshes/pf1.stl; visual mesh filename=package://valkyrie_original/meshes/pf1.stl
- link /v1/RightPrimaryProximalPhalanx: geometry collision mesh filename=package://valkyrie_original/meshes/pf2.stl; visual mesh filename=package://valkyrie_original/meshes/pf2.stl
- link /v1/RightThumbDistalPhalanx: geometry collision mesh filename=package://valkyrie_original/meshes/tf4.stl; visual mesh filename=package://valkyrie_original/meshes/tf4.stl
- link /v1/RightThumbMedialPhalanx: geometry collision mesh filename=package://valkyrie_original/meshes/tf3.stl; visual mesh filename=package://valkyrie_original/meshes/tf3.stl
- link /v1/RightThumbMetacarpal: geometry collision mesh filename=package://valkyrie_original/meshes/tf1_Right.stl; visual mesh filename=package://valkyrie_original/meshes/tf1_Right.stl
- link /v1/RightThumbProximalPhalanx: geometry collision mesh filename=package://valkyrie_original/meshes/tf2.stl; visual mesh filename=package://valkyrie_original/meshes/tf2.stl
- link right_palm: geometry collision mesh filename=package://valkyrie_original/meshes/palm_Right.stl; visual mesh filename=package://valkyrie_original/meshes/palm_Right.stl

File: software/models/valkyrie/V1_sim_shells_reduced_polygon_count_mit.urdf (robot description, URDF)
Before this commit: robot V1, 101 links, 100 joints
Links:
- link l_foot: geometry collision box size=0.082 0.128 0.3; collision sphere radius=0.0
- link r_foot: geometry collision box size=0.082 0.128 0.3; collision sphere radius=0.0

Commit message: reordering the main robot urdf to that the hand urdf is identical

File: software/models/common_components/hand_factory/valkyrie_hand_left.urdf (robot description, URDF)
Before this commit: robot valkyrie_hand_left, 17 links, 16 joints
Links:
- removed link /v1/LeftLittleDistalPhalanx
- removed link /v1/LeftLittleMedialPhalanx
- removed link /v1/LeftLittleProximalPhalanx
- removed link /v1/LeftMedialMetacarpal
- removed link /v1/LeftMiddleDistalPhalanx
- removed link /v1/LeftMiddleMedialPhalanx
- removed link /v1/LeftMiddleProximalPhalanx
- removed link /v1/LeftPrimaryDistalPhalanx
- removed link /v1/LeftPrimaryMedialPhalanx
- removed link /v1/LeftPrimaryMetacarpal
- removed link /v1/LeftPrimaryProximalPhalanx
- removed link /v1/LeftThumbDistalPhalanx
- removed link /v1/LeftThumbMedialPhalanx
- removed link /v1/LeftThumbMetacarpal
- removed link /v1/LeftThumbProximalPhalanx
- removed link left_palm
- added link LeftLittleDistalPhalanx, mass 0.006; collision mesh filename=package://V1/meshes/reduced_polygon_meshes/sf3_ssf4.stl; visual mesh filename=package://V1/meshes/reduced_polygon_meshes/sf3_ssf4.stl
- added link LeftLittleMedialPhalanx, mass 0.011; collision mesh filename=package://V1/meshes/reduced_polygon_meshes/sf2_ssf3.stl; visual mesh filename=package://V1/meshes/reduced_polygon_meshes/sf2_ssf3.stl
- added link LeftLittleProximalPhalanx, mass 0.02; collision mesh filename=package://V1/meshes/reduced_polygon_meshes/ssf2_Left.stl; visual mesh filename=package://V1/meshes/reduced_polygon_meshes/ssf2_Left.stl
- added link LeftMedialMetacarpal, mass 0.047; collision mesh filename=package://V1/meshes/reduced_polygon_meshes/ssf1_Left.stl; visual mesh filename=package://V1/meshes/reduced_polygon_meshes/ssf1_Left.stl
- added link LeftMiddleDistalPhalanx, mass 0.006; collision mesh filename=package://V1/meshes/reduced_polygon_meshes/sf3_ssf4.stl; visual mesh filename=package://V1/meshes/reduced_polygon_meshes/sf3_ssf4.stl
- added link LeftMiddleMedialPhalanx, mass 0.011; collision mesh filename=package://V1/meshes/reduced_polygon_meshes/sf2_ssf3.stl; visual mesh filename=package://V1/meshes/reduced_polygon_meshes/sf2_ssf3.stl
- added link LeftMiddleProximalPhalanx, mass 0.02; collision mesh filename=package://V1/meshes/reduced_polygon_meshes/sf1.stl; visual mesh filename=package://V1/meshes/reduced_polygon_meshes/sf1.stl
- added link LeftPalm, mass 0.712; collision mesh filename=package://V1/meshes/reduced_polygon_meshes/palm_Left.stl; visual mesh filename=package://V1/meshes/reduced_polygon_meshes/palm_Left.stl
- added link LeftPrimaryDistalPhalanx, mass 0.005; collision mesh filename=package://V1/meshes/reduced_polygon_meshes/pf4.stl; visual mesh filename=package://V1/meshes/reduced_polygon_meshes/pf4.stl
- added link LeftPrimaryMedialPhalanx, mass 0.01; collision mesh filename=package://V1/meshes/reduced_polygon_meshes/pf3.stl; visual mesh filename=package://V1/meshes/reduced_polygon_meshes/pf3.stl
- added link LeftPrimaryMetacarpal, mass 0.006; collision mesh filename=package://V1/meshes/reduced_polygon_meshes/pf1.stl; visual mesh filename=package://V1/meshes/reduced_polygon_meshes/pf1.stl
- added link LeftPrimaryProximalPhalanx, mass 0.018; collision mesh filename=package://V1/meshes/reduced_polygon_meshes/pf2.stl; visual mesh filename=package://V1/meshes/reduced_polygon_meshes/pf2.stl
- added link LeftThumbDistalPhalanx, mass 0.006; collision mesh filename=package://V1/meshes/reduced_polygon_meshes/tf4.stl; visual mesh filename=package://V1/meshes/reduced_polygon_meshes/tf4.stl
- added link LeftThumbMedialPhalanx, mass 0.013; collision mesh filename=package://V1/meshes/reduced_polygon_meshes/tf3.stl; visual mesh filename=package://V1/meshes/reduced_polygon_meshes/tf3.stl
- added link LeftThumbMetacarpal, mass 0.017; collision mesh filename=package://V1/meshes/reduced_polygon_meshes/tf1_Left.stl; visual mesh filename=package://V1/meshes/reduced_polygon_meshes/tf1_Left.stl
- added link LeftThumbProximalPhalanx, mass 0.02; collision mesh filename=package://V1/meshes/reduced_polygon_meshes/tf2.stl; visual mesh filename=package://V1/meshes/reduced_polygon_meshes/tf2.stl
Joints:
- joint LeftLittleDIPExtensor: child /v1/LeftLittleDistalPhalanx -> LeftLittleDistalPhalanx; parent /v1/LeftLittleMedialPhalanx -> LeftLittleMedialPhalanx
- joint LeftLittleMPExtensor: child /v1/LeftLittleProximalPhalanx -> LeftLittleProximalPhalanx; parent /v1/LeftMedialMetacarpal -> LeftMedialMetacarpal
- joint LeftLittleMPYaw: child /v1/LeftMedialMetacarpal -> LeftMedialMetacarpal; parent left_palm -> LeftPalm
- joint LeftLittlePIPExtensor: child /v1/LeftLittleMedialPhalanx -> LeftLittleMedialPhalanx; parent /v1/LeftLittleProximalPhalanx -> LeftLittleProximalPhalanx
- joint LeftMiddleDIPExtensor: child /v1/LeftMiddleDistalPhalanx -> LeftMiddleDistalPhalanx; parent /v1/LeftMiddleMedialPhalanx -> LeftMiddleMedialPhalanx
- joint LeftMiddleMPExtensor: child /v1/LeftMiddleProximalPhalanx -> LeftMiddleProximalPhalanx; parent left_palm -> LeftPalm
- joint LeftMiddlePIPExtensor: child /v1/LeftMiddleMedialPhalanx -> LeftMiddleMedialPhalanx; parent /v1/LeftMiddleProximalPhalanx -> LeftMiddleProximalPhalanx
- joint LeftPrimaryDIPExtensor: child /v1/LeftPrimaryDistalPhalanx -> LeftPrimaryDistalPhalanx; parent /v1/LeftPrimaryMedialPhalanx -> LeftPrimaryMedialPhalanx
- joint LeftPrimaryMPExtensor: child /v1/LeftPrimaryProximalPhalanx -> LeftPrimaryProximalPhalanx; parent /v1/LeftPrimaryMetacarpal -> LeftPrimaryMetacarpal
- joint LeftPrimaryMPYaw: child /v1/LeftPrimaryMetacarpal -> LeftPrimaryMetacarpal; parent left_palm -> LeftPalm
- joint LeftPrimaryPIPExtensor: child /v1/LeftPrimaryMedialPhalanx -> LeftPrimaryMedialPhalanx; parent /v1/LeftPrimaryProximalPhalanx -> LeftPrimaryProximalPhalanx
- joint LeftThumbDIPExtensor: child /v1/LeftThumbDistalPhalanx -> LeftThumbDistalPhalanx; parent /v1/LeftThumbMedialPhalanx -> LeftThumbMedialPhalanx
- joint LeftThumbMPExtensor: child /v1/LeftThumbProximalPhalanx -> LeftThumbProximalPhalanx; parent /v1/LeftThumbMetacarpal -> LeftThumbMetacarpal
- joint LeftThumbMPYaw: child /v1/LeftThumbMetacarpal -> LeftThumbMetacarpal; parent left_palm -> LeftPalm
- joint LeftThumbPIPExtensor: child /v1/LeftThumbMedialPhalanx -> LeftThumbMedialPhalanx; parent /v1/LeftThumbProximalPhalanx -> LeftThumbProximalPhalanx
- joint left_valkyrie_hand_joint: child left_palm -> LeftPalm

File: software/models/common_components/hand_factory/valkyrie_hand_right.urdf (robot description, URDF)
Before this commit: robot valkyrie_hand_right, 17 links, 16 joints
Links:
- removed link /v1/RightLittleDistalPhalanx
- removed link /v1/RightLittleMedialPhalanx
- removed link /v1/RightLittleProximalPhalanx
- removed link /v1/RightMedialMetacarpal
- removed link /v1/RightMiddleDistalPhalanx
- removed link /v1/RightMiddleMedialPhalanx
- removed link /v1/RightMiddleProximalPhalanx
- removed link /v1/RightPrimaryDistalPhalanx
- removed link /v1/RightPrimaryMedialPhalanx
- removed link /v1/RightPrimaryMetacarpal
- removed link /v1/RightPrimaryProximalPhalanx
- removed link /v1/RightThumbDistalPhalanx
- removed link /v1/RightThumbMedialPhalanx
- removed link /v1/RightThumbMetacarpal
- removed link /v1/RightThumbProximalPhalanx
- removed link right_palm
- added link RightLittleDistalPhalanx, mass 0.006; collision mesh filename=package://V1/meshes/reduced_polygon_meshes/sf3_ssf4.stl; visual mesh filename=package://V1/meshes/reduced_polygon_meshes/sf3_ssf4.stl
- added link RightLittleMedialPhalanx, mass 0.011; collision mesh filename=package://V1/meshes/reduced_polygon_meshes/sf2_ssf3.stl; visual mesh filename=package://V1/meshes/reduced_polygon_meshes/sf2_ssf3.stl
- added link RightLittleProximalPhalanx, mass 0.02; collision mesh filename=package://V1/meshes/reduced_polygon_meshes/ssf2_Right.stl; visual mesh filename=package://V1/meshes/reduced_polygon_meshes/ssf2_Right.stl
- added link RightMedialMetacarpal, mass 0.047; collision mesh filename=package://V1/meshes/reduced_polygon_meshes/ssf1_Right.stl; visual mesh filename=package://V1/meshes/reduced_polygon_meshes/ssf1_Right.stl
- added link RightMiddleDistalPhalanx, mass 0.006; collision mesh filename=package://V1/meshes/reduced_polygon_meshes/sf3_ssf4.stl; visual mesh filename=package://V1/meshes/reduced_polygon_meshes/sf3_ssf4.stl
- added link RightMiddleMedialPhalanx, mass 0.011; collision mesh filename=package://V1/meshes/reduced_polygon_meshes/sf2_ssf3.stl; visual mesh filename=package://V1/meshes/reduced_polygon_meshes/sf2_ssf3.stl
- added link RightMiddleProximalPhalanx, mass 0.02; collision mesh filename=package://V1/meshes/reduced_polygon_meshes/sf1.stl; visual mesh filename=package://V1/meshes/reduced_polygon_meshes/sf1.stl
- added link RightPalm, mass 0.712; collision mesh filename=package://V1/meshes/reduced_polygon_meshes/palm_Right.stl; visual mesh filename=package://V1/meshes/reduced_polygon_meshes/palm_Right.stl
- added link RightPrimaryDistalPhalanx, mass 0.005; collision mesh filename=package://V1/meshes/reduced_polygon_meshes/pf4.stl; visual mesh filename=package://V1/meshes/reduced_polygon_meshes/pf4.stl
- added link RightPrimaryMedialPhalanx, mass 0.01; collision mesh filename=package://V1/meshes/reduced_polygon_meshes/pf3.stl; visual mesh filename=package://V1/meshes/reduced_polygon_meshes/pf3.stl
- added link RightPrimaryMetacarpal, mass 0.006; collision mesh filename=package://V1/meshes/reduced_polygon_meshes/pf1.stl; visual mesh filename=package://V1/meshes/reduced_polygon_meshes/pf1.stl
- added link RightPrimaryProximalPhalanx, mass 0.018; collision mesh filename=package://V1/meshes/reduced_polygon_meshes/pf2.stl; visual mesh filename=package://V1/meshes/reduced_polygon_meshes/pf2.stl
- added link RightThumbDistalPhalanx, mass 0.006; collision mesh filename=package://V1/meshes/reduced_polygon_meshes/tf4.stl; visual mesh filename=package://V1/meshes/reduced_polygon_meshes/tf4.stl
- added link RightThumbMedialPhalanx, mass 0.013; collision mesh filename=package://V1/meshes/reduced_polygon_meshes/tf3.stl; visual mesh filename=package://V1/meshes/reduced_polygon_meshes/tf3.stl
- added link RightThumbMetacarpal, mass 0.017; collision mesh filename=package://V1/meshes/reduced_polygon_meshes/tf1_Right.stl; visual mesh filename=package://V1/meshes/reduced_polygon_meshes/tf1_Right.stl
- added link RightThumbProximalPhalanx, mass 0.02; collision mesh filename=package://V1/meshes/reduced_polygon_meshes/tf2.stl; visual mesh filename=package://V1/meshes/reduced_polygon_meshes/tf2.stl
Joints:
- joint RightLittleDIPExtensor: child /v1/RightLittleDistalPhalanx -> RightLittleDistalPhalanx; parent /v1/RightLittleMedialPhalanx -> RightLittleMedialPhalanx
- joint RightLittleMPExtensor: child /v1/RightLittleProximalPhalanx -> RightLittleProximalPhalanx; parent /v1/RightMedialMetacarpal -> RightMedialMetacarpal
- joint RightLittleMPYaw: child /v1/RightMedialMetacarpal -> RightMedialMetacarpal; parent right_palm -> RightPalm
- joint RightLittlePIPExtensor: child /v1/RightLittleMedialPhalanx -> RightLittleMedialPhalanx; parent /v1/RightLittleProximalPhalanx -> RightLittleProximalPhalanx
- joint RightMiddleDIPExtensor: child /v1/RightMiddleDistalPhalanx -> RightMiddleDistalPhalanx; parent /v1/RightMiddleMedialPhalanx -> RightMiddleMedialPhalanx
- joint RightMiddleMPExtensor: child /v1/RightMiddleProximalPhalanx -> RightMiddleProximalPhalanx; parent right_palm -> RightPalm
- joint RightMiddlePIPExtensor: child /v1/RightMiddleMedialPhalanx -> RightMiddleMedialPhalanx; parent /v1/RightMiddleProximalPhalanx -> RightMiddleProximalPhalanx
- joint RightPrimaryDIPExtensor: child /v1/RightPrimaryDistalPhalanx -> RightPrimaryDistalPhalanx; parent /v1/RightPrimaryMedialPhalanx -> RightPrimaryMedialPhalanx
- joint RightPrimaryMPExtensor: child /v1/RightPrimaryProximalPhalanx -> RightPrimaryProximalPhalanx; parent /v1/RightPrimaryMetacarpal -> RightPrimaryMetacarpal
- joint RightPrimaryMPYaw: child /v1/RightPrimaryMetacarpal -> RightPrimaryMetacarpal; parent right_palm -> RightPalm
- joint RightPrimaryPIPExtensor: child /v1/RightPrimaryMedialPhalanx -> RightPrimaryMedialPhalanx; parent /v1/RightPrimaryProximalPhalanx -> RightPrimaryProximalPhalanx
- joint RightThumbDIPExtensor: child /v1/RightThumbDistalPhalanx -> RightThumbDistalPhalanx; parent /v1/RightThumbMedialPhalanx -> RightThumbMedialPhalanx
- joint RightThumbMPExtensor: child /v1/RightThumbProximalPhalanx -> RightThumbProximalPhalanx; parent /v1/RightThumbMetacarpal -> RightThumbMetacarpal
- joint RightThumbMPYaw: child /v1/RightThumbMetacarpal -> RightThumbMetacarpal; parent right_palm -> RightPalm
- joint RightThumbPIPExtensor: child /v1/RightThumbMedialPhalanx -> RightThumbMedialPhalanx; parent /v1/RightThumbProximalPhalanx -> RightThumbProximalPhalanx
- joint right_valkyrie_hand_joint: child right_palm -> RightPalm
