Commit message: fixed issues in director config and valkyrie hand right urdf

File: software/models/common_components/hand_factory/valkyrie_hand_right.urdf (robot description, URDF)
Before this commit: robot valkyrie_hand_right, 15 links, 14 joints
Links:
- link rightIndexFingerPitch1Link: geometry collision mesh filename=package://val_description/model/meshes/fingers/indexj1_righ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; visual mesh filename=package://val_description/model/meshes/fingers/indexj1_righ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
- link rightIndexFingerPitch2Link: geometry collision mesh filename=package://val_description/model/meshes/fingers/indexj2_righ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; visual mesh filename=package://val_description/model/meshes/fingers/indexj2_righ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
- link rightIndexFingerPitch3Link: geometry collision mesh filename=package://val_description/model/meshes/fingers/indexj3_righ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; visual mesh filename=package://val_description/model/meshes/fingers/indexj3_righ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
- link rightMiddleFingerPitch1Link: geometry collision mesh filename=package://val_description/model/meshes/fingers/middlej1_rig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; visual mesh filename=package://val_description/model/meshes/fingers/middlej1_rig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
- link rightMiddleFingerPitch2Link: geometry collision mesh filename=package://val_description/model/meshes/fingers/middlej2_rig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; visual mesh filename=package://val_description/model/meshes/fingers/middlej2_rig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
- link rightMiddleFingerPitch3Link: geometry collision mesh filename=package://val_description/model/meshes/fingers/middlej3_rig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; visual mesh filename=package://val_description/model/meshes/fingers/middlej3_rig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
- link rightPalm: geometry collision mesh filename=package://val_description/model/meshes/arms/palm_right.obj; visual mesh filename=package://val_description/model/meshes/arms/palm_right.obj
- link rightPinkyPitch1Link: geometry collision mesh filename=package://val_description/model/meshes/fingers/pinkyj1_righ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; visual mesh filename=package://val_description/model/meshes/fingers/pinkyj1_righ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
- link rightPinkyPitch2Link: geometry collision mesh filename=package://val_description/model/meshes/fingers/pinkyj2_righ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; visual mesh filename=package://val_description/model/meshes/fingers/pinkyj2_righ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
- link rightPinkyPitch3Link: geometry collision mesh filename=package://val_description/model/meshes/fingers/pinkyj3_righ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; visual mesh filename=package://val_description/model/meshes/fingers/pinkyj3_righ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
- link rightThumbPitch1Link: geometry collision mesh filename=package://val_description/model/meshes/fingers/thumbj2_righ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; visual mesh filename=package://val_description/model/meshes/fingers/thumbj2_righ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
- link rightThumbPitch2Link: geometry collision mesh filename=package://val_description/model/meshes/fingers/thumbj3_righ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; visual mesh filename=package://val_description/model/meshes/fingers/thumbj3_righ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
- link rightThumbPitch3Link: geometry collision mesh filename=package://val_description/model/meshes/fingers/thumbj4_righ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; visual mesh filename=package://val_description/model/meshes/fingers/thumbj4_righ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
- link rightThumbRollLink: geometry collision mesh filename=package://val_description/model/meshes/fingers/thumbj1_righ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; visual mesh filename=package://val_description/model/meshes/fingers/thumbj1_righ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
