Commit message: new urdf but fails to be read by drake

File: software/models/val_description/urdf/valkyrie_A_sim.urdf (robot description, URDF)
Before this commit: robot valkyrie, 79 links, 78 joints
Links:
- removed link Head
- removed link LeftIMU_Frame
- removed link RightIMU_Frame
- removed link head_hokuyo_frame_offset
- removed link left_camera_frame_offset
- removed link right_camera_frame_offset
- added link LeftTorsoIMU_Frame, mass 1e-07
- added link RightTorsoIMU_Frame, mass 1e-07
- added link UpperNeckPitchLink, mass 4.59; collision mesh filename=package://val_description/meshes/head/head_multisense_no_vi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; visual mesh filename=package://val_description/meshes/head/head_multisense_no_vi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
- added link center_bottom_led_frame, mass 1e-5
- added link center_top_led_frame, mass 1e-5
- added link head, mass 1.41984; collision box size=0.0468 0.12 0.1184; collision box size=0.1311 0.12 0.0591
- added link head_hokuyo_frame, mass 1e-5
- added link head_imu_link, mass 1e-5; visual box size=0.01 0.01 0.01
- added link left_camera_frame, mass 1e-5
- added link left_camera_optical_frame
- added link left_led_frame, mass 1e-5
- added link right_camera_frame, mass 1e-5
- added link right_camera_optical_frame
- added link right_led_frame, mass 1e-5
- link LeftAnklePitchLink: mass 0.395 -> 0.06
- link LeftElbowPitchLink: mass 2.367 -> 1.83
- link LeftFoot: mass 1.888 -> 3.255
- link LeftForearmLink: mass 2.903 -> 2.476
- link LeftHipPitchLink: mass 10.3 -> 10.2
- link LeftHipRollLink: mass 5.95 -> 3.665
- link LeftIndexFingerPitch1Link: mass 0.006 -> 0.02
- link LeftKneePitchLink: mass 7.4 -> 6.6
- link LeftPinkyPitch1Link: mass 0.047 -> 0.02
- link LeftPinkyPitch2Link: mass 0.02 -> 0.011
- link LeftPinkyPitch3Link: mass 0.011 -> 0.006
- link LeftShoulderRollLink: mass 2.87 -> 3.97
- link LeftShoulderYawLink: mass 2.575 -> 3.085
- link LeftWristRollLink: mass 0.1 -> 0.14
- link LowerNeckPitchLink: mass 0.1 -> 1.05
- link NeckYawLink: mass 0.1 -> 1.4
- link Pelvis: mass 6.986 -> 8.22
- link RightAnklePitchLink: mass 0.395 -> 0.06
- link RightElbowPitchLink: mass 2.367 -> 1.83
- link RightFoot: mass 1.888 -> 3.255
- link RightForearmLink: mass 2.903 -> 2.476
- link RightHipPitchLink: mass 10.3 -> 10.2
- link RightHipRollLink: mass 5.95 -> 3.665
- link RightIndexFingerPitch1Link: mass 0.006 -> 0.02
- link RightKneePitchLink: mass 7.4 -> 6.6
- link RightPinkyPitch1Link: mass 0.047 -> 0.02
- link RightPinkyPitch2Link: mass 0.02 -> 0.011
- link RightPinkyPitch3Link: mass 0.011 -> 0.006
- link RightShoulderRollLink: mass 2.87 -> 3.97
- link RightShoulderYawLink: mass 2.575 -> 3.085
- link RightWristRollLink: mass 0.1 -> 0.14
- link Torso: mass 42.6 -> 39.47
- link TorsoPitchLink: mass 1e-05 -> 0.1
- link TorsoYawLink: mass 1e-05 -> 0.5
- link hokuyo_link: mass 0.057664 -> 0.057654; geometry collision box size=0.08 0.06 0.04238; collision cylinder length=0.047 radius=0.024425
Joints:
- removed joint LeftIMU_Offset
- removed joint MultisenseSLSpinnyJointFrame
- removed joint RightIMU_Offset
- removed joint head_hokuyo_frame_joint
- added joint LeftTorsoIMU_Offset: type fixed, parent Torso, child LeftTorsoIMU_Frame, origin xyz=-0.047 0.134 0.363 rpy=1.57 0.0 3.14, axis 0 0 1
- added joint RightTorsoIMU_Offset: type fixed, parent Torso, child RightTorsoIMU_Frame, origin xyz=-0.047 -0.134 0.363 rpy=-1.57 0.0 3.14, axis 0 0 1
- added joint center_bottom_led_frame_joint: type fixed, parent head, child center_bottom_led_frame, origin xyz=0.01125 0.0 -0.0155
- added joint center_top_led_frame_joint: type fixed, parent head, child center_top_led_frame, origin xyz=0.01125 0.0 0.0105
- added joint head_hokuyo_joint: type fixed, parent hokuyo_link, child head_hokuyo_frame, origin xyz=0.03 0 0.015 rpy=0 0 0, axis 0 1 0
- added joint head_imu_joint: type fixed, parent head, child head_imu_link, origin xyz=-0.0475 0.035 0.0 rpy=0 0 0
- added joint hokuyo_joint: type continuous, parent head, child hokuyo_link, origin xyz=-0.0446 0 0.0880 rpy=0 0 0, axis 1 0 0
- added joint left_camera_optical_frame_joint: type fixed, parent left_camera_frame, child left_camera_optical_frame, origin xyz=0 0 0 rpy=-1.5708 0.0 -1.5708
- added joint left_led_frame_joint: type fixed, parent head, child left_led_frame, origin xyz=-0.01443 0.07452 0.050346 rpy=0 -0.15 0.53
- added joint multisense_head_root_joint: type fixed, parent UpperNeckPitchLink, child head, origin xyz=0.183585961 0.0 0.075353826 rpy=-3.14159 0.130899694 0.0, axis 0 0 1
- added joint right_camera_optical_frame_joint: type fixed, parent right_camera_frame, child right_camera_optical_frame, origin xyz=0 0 0 rpy=-1.5708 0.0 -1.5708
- added joint right_led_frame_joint: type fixed, parent head, child right_led_frame, origin xyz=-0.01443 -0.07452 0.050346 rpy=0 -0.15 -0.53
- joint LeftAnklePitch: limit lower=-0.873 upper=0.873 effort=205 velocity=11 -> lower=-0.8644 upper=0.875 effort=205 velocity=11
- joint LeftAnkleRoll: limit lower=-0.349 upper=0.349 effort=205 velocity=11 -> lower=-0.349 upper=0.348 effort=205 velocity=11
- joint LeftElbowPitch: limit lower=-1.92 upper=0.0 effort=65 velocity=11.5 -> lower=-2.174 upper=0.12 effort=65 velocity=11.5
- joint LeftForearmYaw: limit lower=-0.7853 upper=3.9269 effort=26 velocity=5 -> lower=-2.019 upper=3.14 effort=26 velocity=5
- joint LeftHipPitch: limit lower=-2.356 upper=1.71 effort=350 velocity=6.11 -> lower=-2.42 upper=1.619 effort=350 velocity=6.11
- joint LeftHipRoll: limit lower=-0.262 upper=0.524 effort=350 velocity=7 -> lower=-0.467 upper=0.5515 effort=350 velocity=7
- joint LeftHipYaw: limit lower=-0.169 upper=0.524 effort=190 velocity=5.89 -> lower=-0.4141 upper=1.1 effort=190 velocity=5.89
- joint LeftKneePitch: limit lower=-0.218 upper=1.902 effort=350 velocity=6.11 -> lower=-0.083 upper=2.057 effort=350 velocity=6.11
- joint LeftShoulderPitch: limit lower=-3.14 upper=3.14 effort=190 velocity=5.89 -> lower=-2.85 upper=2.0 effort=190 velocity=5.89
- joint LeftShoulderRoll: limit lower=-1.3962 upper=1.4835 effort=190 velocity=5.89 -> lower=-1.519 upper=1.266 effort=190 velocity=5.89
- joint LeftShoulderYaw: limit lower=-1.57 upper=1.5707 effort=65 velocity=11.5 -> lower=-3.1 upper=2.18 effort=65 velocity=11.5
- joint LeftWristPitch: limit lower=-0.873 upper=0.698 effort=14 velocity=1 -> lower=-0.36 upper=0.49 effort=14 velocity=1
- joint LeftWristRoll: limit lower=-0.436 upper=0.524 effort=14 velocity=1 -> lower=-0.62 upper=0.625 effort=14 velocity=1
- joint LowerNeckPitch: limit lower=0 upper=1.57 effort=26 velocity=5 -> lower=0 upper=1.162 effort=26 velocity=5
- joint NeckYaw: limit lower=-1.57 upper=1.57 effort=26 velocity=5 -> lower=-1.04719755 upper=1.04719755 effort=26 velocity=5
- joint RightAnklePitch: limit lower=-0.873 upper=0.873 effort=205 velocity=11 -> lower=-0.8644 upper=0.875 effort=205 velocity=11
- joint RightAnkleRoll: limit lower=-0.349 upper=0.349 effort=205 velocity=11 -> lower=-0.349 upper=0.348 effort=205 velocity=11
- joint RightElbowPitch: limit lower=-0.0 upper=1.92 effort=65 velocity=11.5 -> lower=-0.12 upper=2.174 effort=65 velocity=11.5
- joint RightForearmYaw: limit lower=-0.7853 upper=3.9269 effort=26 velocity=5 -> lower=-2.019 upper=3.14 effort=26 velocity=5
- joint RightHipPitch: limit lower=-2.356 upper=1.71 effort=350 velocity=6.11 -> lower=-2.42 upper=1.619 effort=350 velocity=6.11
- joint RightHipRoll: limit lower=-0.524 upper=0.262 effort=350 velocity=7 -> lower=-0.5515 upper=0.467 effort=350 velocity=7
- joint RightHipYaw: limit lower=-0.524 upper=0.169 effort=190 velocity=5.89 -> lower=-1.1 upper=0.4141 effort=190 velocity=5.89
- joint RightKneePitch: limit lower=-0.218 upper=1.902 effort=350 velocity=6.11 -> lower=-0.083 upper=2.057 effort=350 velocity=6.11
- joint RightShoulderPitch: limit lower=-3.14 upper=3.14 effort=190 velocity=5.89 -> lower=-2.85 upper=2.0 effort=190 velocity=5.89
- joint RightShoulderRoll: limit lower=-1.4835 upper=1.3962 effort=190 velocity=5.89 -> lower=-1.266 upper=1.519 effort=190 velocity=5.89
- joint RightShoulderYaw: limit lower=-1.57 upper=1.5707 effort=65 velocity=11.5 -> lower=-3.1 upper=2.18 effort=65 velocity=11.5
- joint RightWristPitch: limit lower=-0.698 upper=0.873 effort=14 velocity=1 -> lower=-0.49 upper=0.36 effort=14 velocity=1
- joint RightWristRoll: limit lower=-0.524 upper=0.436 effort=14 velocity=1 -> lower=-0.625 upper=0.62 effort=14 velocity=1
- joint TorsoPitch: limit lower=-0.087 upper=0.698 effort=150 velocity=9 -> lower=-0.13 upper=0.666 effort=150 velocity=9
- joint TorsoRoll: limit lower=-0.262 upper=0.262 effort=150 velocity=9 -> lower=-0.23 upper=0.255 effort=150 velocity=9
- joint TorsoYaw: limit lower=-0.698 upper=0.698 effort=190 velocity=5.89 -> lower=-1.329 upper=1.181 effort=190 velocity=5.89
- joint UpperNeckPitch: child Head -> UpperNeckPitchLink; limit lower=-0.087 upper=0.785 effort=26 velocity=5 -> lower=-0.872 upper=0.0 effort=26 velocity=5
- joint left_camera_frame_joint: axis 0 0 1 -> (none); child left_camera_frame_offset -> left_camera_frame; origin xyz=0.18335 0.035 0.0774 rpy=-3.14 0.1309 0.0 -> xyz=0.0 0.035 -0.002; parent Head -> head
- joint right_camera_frame_joint: axis 0 0 1 -> (none); child right_camera_frame_offset -> right_camera_frame; origin xyz=0.18335 -0.035 0.0774 rpy=-3.14 0.1309 0.0 -> xyz=0.0 -0.035 -0.002; parent Head -> head

Commit message: minor mods to support multiRRT planning: move palm point
this should be temporary

File: software/models/val_description/urdf/valkyrie_A_sim.urdf (robot description, URDF)
Before this commit: robot valkyrie, 87 links, 86 joints
Joints:
- joint l_hand_face_joint: origin xyz=0.08 0.0 -0.04 rpy=3.14159265359 0 1.57079632679 -> xyz=0.07 0.0 -0.08 rpy=3.14159265359 0 1.57079632679
- joint r_hand_face_joint: origin xyz=0.08 0 0.04 rpy=0 0 -1.57079632679 -> xyz=0.07 0 0.08 rpy=0 0 -1.57079632679

File: software/models/val_description/urdf/valkyrie_A_sim_drake.urdf (robot description, URDF)
Before this commit: robot valkyrie, 87 links, 86 joints
Joints:
- joint l_hand_face_joint: origin xyz=0.08 0.0 -0.04 rpy=3.14159265359 0 1.57079632679 -> xyz=0.07 0.0 -0.08 rpy=3.14159265359 0 1.57079632679
- joint r_hand_face_joint: origin xyz=0.08 0 0.04 rpy=0 0 -1.57079632679 -> xyz=0.07 0 0.08 rpy=0 0 -1.57079632679

Commit message: Added midfoot_front and midfoot_rear to Valkyrie urdf.

File: software/models/val_description/urdf/valkyrie_A_sim.urdf (robot description, URDF)
Before this commit: robot valkyrie, 87 links, 86 joints
Links:
- link leftFoot: geometry collision box size=0.27 0.16 0.064; collision sphere radius=0.0
- link rightFoot: geometry collision box size=0.27 0.16 0.064; collision sphere radius=0.0

File: software/models/val_description/urdf/valkyrie_A_sim_drake.urdf (robot description, URDF)
Before this commit: robot valkyrie, 87 links, 86 joints
Links:
- link leftFoot: geometry collision box size=0.27 0.16 0.064; collision sphere radius=0.0
- link rightFoot: geometry collision box size=0.27 0.16 0.064; collision sphere radius=0.0
