Commit message: new working versions of the urdf

File: software/models/val_description/urdf/valkyrie_sim.urdf (robot description, URDF)
Before this commit: robot valkyrie, 87 links, 86 joints
Links:
- removed link leftLegSixAxis_Frame
- removed link leftPelvisIMU_Frame
- removed link rightLegSixAxis_Frame
- removed link rightPelvisIMU_Frame
- removed link rightTorsoIMU_Frame
- added link pelvisMiddleImu_Frame, mass 1e-07
- added link pelvisRearImu_Frame, mass 1e-07
- link leftAnklePitchLink: mass 0.06 -> 0.03
- link leftFoot: mass 3.255 -> 2.27
- link leftKneePitchLink: mass 6.6 -> 6.2
- link rightAnklePitchLink: mass 0.06 -> 0.03
- link rightFoot: mass 3.255 -> 2.27
- link rightKneePitchLink: mass 6.6 -> 6.2
- link upperNeckPitchLink: mass 4.59 -> 3.89
Joints:
- removed joint leftLegSixAxis_Offset
- removed joint leftPelvisIMU_Offset
- removed joint rightLegSixAxis_Offset
- removed joint rightPelvisIMU_Offset
- removed joint rightTorsoIMU_Offset
- added joint pelvisMiddleImu_Offset: type fixed, parent pelvis, child pelvisMiddleImu_Frame, origin xyz=0.0 0.0 -0.108184035 rpy=3.14159 0.0 0.0, axis 0 0 1
- added joint pelvisRearImu_Offset: type fixed, parent pelvis, child pelvisRearImu_Frame, origin xyz=-0.075844901 0.0 -0.111056426 rpy=-3.14159 0.476467 -3.14159, axis 0 0 1
- joint leftCOP_Offset: origin xyz=0.0189 0.0 -0.0783 rpy=0.0 0.13 0.0 -> xyz=0.0189 0.0 -0.0783 rpy=0.0 0.0 0.0
- joint leftTorsoIMU_Offset: origin xyz=-0.047 0.134 0.363 rpy=1.57 0.0 3.14 -> xyz=-0.046863 0.134239 0.3630676 rpy=1.57 0 3.14
- joint rightCOP_Offset: origin xyz=0.0189 0.0 -0.0783 rpy=0.0 0.13 0.0 -> xyz=0.0189 0.0 -0.0783 rpy=0.0 0.0 0.0

File: software/models/val_description/urdf/valkyrie_sim_drake.urdf (robot description, URDF)
Before this commit: robot valkyrie, 87 links, 86 joints
Links:
- removed link leftLegSixAxis_Frame
- removed link leftPelvisIMU_Frame
- removed link rightLegSixAxis_Frame
- removed link rightPelvisIMU_Frame
- removed link rightTorsoIMU_Frame
- added link pelvisMiddleImu_Frame, mass 1e-07
- added link pelvisRearImu_Frame, mass 1e-07
- link leftAnklePitchLink: mass 0.06 -> 0.03
- link leftFoot: mass 3.255 -> 2.27
- link leftKneePitchLink: mass 6.6 -> 6.2
- link rightAnklePitchLink: mass 0.06 -> 0.03
- link rightFoot: mass 3.255 -> 2.27
- link rightKneePitchLink: mass 6.6 -> 6.2
- link upperNeckPitchLink: mass 4.59 -> 3.89
Joints:
- removed joint leftLegSixAxis_Offset
- removed joint leftPelvisIMU_Offset
- removed joint rightLegSixAxis_Offset
- removed joint rightPelvisIMU_Offset
- removed joint rightTorsoIMU_Offset
- added joint pelvisMiddleImu_Offset: type fixed, parent pelvis, child pelvisMiddleImu_Frame, origin xyz=0.0 0.0 -0.108184035 rpy=3.14159 0.0 0.0, axis 0 0 1
- added joint pelvisRearImu_Offset: type fixed, parent pelvis, child pelvisRearImu_Frame, origin xyz=-0.075844901 0.0 -0.111056426 rpy=-3.14159 0.476467 -3.14159, axis 0 0 1
- joint leftCOP_Offset: origin xyz=0.0189 0.0 -0.0783 rpy=0.0 0.13 0.0 -> xyz=0.0189 0.0 -0.0783 rpy=0.0 0.0 0.0
- joint leftTorsoIMU_Offset: origin xyz=-0.047 0.134 0.363 rpy=1.57 0.0 3.14 -> xyz=-0.046863 0.134239 0.3630676 rpy=1.57 0 3.14
- joint rightCOP_Offset: origin xyz=0.0189 0.0 -0.0783 rpy=0.0 0.13 0.0 -> xyz=0.0189 0.0 -0.0783 rpy=0.0 0.0 0.0

Commit message: valkyrie_sim.urdf: un-fix hand joints

File: software/models/val_description/urdf/valkyrie_sim.urdf (robot description, URDF)
Before this commit: robot valkyrie, 84 links, 83 joints
Joints:
- joint leftIndexFingerPitch1: limit (none) -> lower=-1.57 upper=-0.0 effort=10 velocity=1; type fixed -> revolute
- joint leftIndexFingerPitch2: limit (none) -> lower=-1.658 upper=-0.0 effort=10 velocity=1; type fixed -> revolute
- joint leftIndexFingerPitch3: limit (none) -> lower=-1.92 upper=-0.0 effort=10 velocity=1; type fixed -> revolute
- joint leftMiddleFingerPitch1: limit (none) -> lower=-1.658 upper=-0.0 effort=10 velocity=1; type fixed -> revolute
- joint leftMiddleFingerPitch2: limit (none) -> lower=-1.92 upper=-0.0 effort=10 velocity=1; type fixed -> revolute
- joint leftMiddleFingerPitch3: limit (none) -> lower=-1.57 upper=-0.0 effort=10 velocity=1; type fixed -> revolute
- joint leftPinkyPitch1: limit (none) -> lower=-1.57 upper=-0.0 effort=10 velocity=1; type fixed -> revolute
- joint leftPinkyPitch2: limit (none) -> lower=-1.658 upper=-0.0 effort=10 velocity=1; type fixed -> revolute
- joint leftPinkyPitch3: limit (none) -> lower=-1.92 upper=-0.0 effort=10 velocity=1; type fixed -> revolute
- joint leftThumbPitch1: axis 0 0 1 -> 1 0 0; limit (none) -> lower=-1.658 upper=-0.0 effort=10 velocity=1; type fixed -> revolute
- joint leftThumbPitch2: axis 0 0 1 -> 1 0 0; limit (none) -> lower=-1.92 upper=-0.0 effort=10 velocity=1; type fixed -> revolute
- joint leftThumbPitch3: axis 0 0 1 -> 1 0 0; limit (none) -> lower=-1.57 upper=-0.0 effort=10 velocity=1; type fixed -> revolute
- joint leftThumbRoll: axis 0 0 1 -> 0 1 0; limit (none) -> lower=0.0 upper=2.356 effort=10 velocity=1; type fixed -> revolute
- joint rightIndexFingerPitch1: limit (none) -> lower=0.0 upper=1.57 effort=10 velocity=1; type fixed -> revolute
- joint rightIndexFingerPitch2: limit (none) -> lower=0.0 upper=1.658 effort=10 velocity=1; type fixed -> revolute
- joint rightIndexFingerPitch3: limit (none) -> lower=0.0 upper=1.92 effort=10 velocity=1; type fixed -> revolute
- joint rightMiddleFingerPitch1: limit (none) -> lower=0.0 upper=1.658 effort=10 velocity=1; type fixed -> revolute
- joint rightMiddleFingerPitch2: limit (none) -> lower=0.0 upper=1.92 effort=10 velocity=1; type fixed -> revolute
- joint rightMiddleFingerPitch3: limit (none) -> lower=0.0 upper=1.57 effort=10 velocity=1; type fixed -> revolute
- joint rightPinkyPitch1: limit (none) -> lower=0.0 upper=1.57 effort=10 velocity=1; type fixed -> revolute
- joint rightPinkyPitch2: limit (none) -> lower=0.0 upper=1.658 effort=10 velocity=1; type fixed -> revolute
- joint rightPinkyPitch3: limit (none) -> lower=0.0 upper=1.92 effort=10 velocity=1; type fixed -> revolute
- joint rightThumbPitch1: axis 0 0 1 -> 1 0 0; limit (none) -> lower=0.0 upper=1.658 effort=10 velocity=1; type fixed -> revolute
- joint rightThumbPitch2: axis 0 0 1 -> 1 0 0; limit (none) -> lower=0.0 upper=1.92 effort=10 velocity=1; type fixed -> revolute
- joint rightThumbPitch3: axis 0 0 1 -> 1 0 0; limit (none) -> lower=0.0 upper=1.57 effort=10 velocity=1; type fixed -> revolute
- joint rightThumbRoll: axis 0 0 1 -> 0 1 0; limit (none) -> lower=0.0 upper=2.356 effort=10 velocity=1; type fixed -> revolute

Commit message: reliable and working version

File: software/models/val_description/urdf/valkyrie_sim.urdf (robot description, URDF)
Before this commit: robot valkyrie, 84 links, 83 joints
Joints:
- joint leftShoulderRoll: limit lower=-1.519 upper=1.266 effort=190 velocity=5.89 -> lower=-1.509 upper=1.266 effort=190 velocity=5.89
- joint leftWristPitch: limit lower=-0.36 upper=0.49 effort=14 velocity=1 -> lower=-0.36 upper=0.48 effort=14 velocity=1
- joint rightShoulderRoll: limit lower=-1.266 upper=1.519 effort=190 velocity=5.89 -> lower=-1.266 upper=1.509 effort=190 velocity=5.89
- joint rightWristPitch: limit lower=-0.49 upper=0.36 effort=14 velocity=1 -> lower=-0.48 upper=0.36 effort=14 velocity=1

File: software/models/val_description/urdf/valkyrie_sim_drake.urdf (robot description, URDF)
Before this commit: robot valkyrie, 84 links, 83 joints
Joints:
- joint leftShoulderRoll: limit lower=-1.519 upper=1.266 effort=190 velocity=5.89 -> lower=-1.509 upper=1.266 effort=190 velocity=5.89
- joint leftWristPitch: limit lower=-0.36 upper=0.49 effort=14 velocity=1 -> lower=-0.36 upper=0.48 effort=14 velocity=1
- joint rightShoulderRoll: limit lower=-1.266 upper=1.519 effort=190 velocity=5.89 -> lower=-1.266 upper=1.509 effort=190 velocity=5.89
- joint rightWristPitch: limit lower=-0.49 upper=0.36 effort=14 velocity=1 -> lower=-0.48 upper=0.36 effort=14 velocity=1

Commit message: revert ROM changes

File: software/models/val_description/urdf/valkyrie_sim.urdf (robot description, URDF)
Before this commit: robot valkyrie, 84 links, 83 joints
Joints:
- joint leftShoulderRoll: limit lower=-1.509 upper=1.266 effort=190 velocity=5.89 -> lower=-1.519 upper=1.266 effort=190 velocity=5.89
- joint leftWristPitch: limit lower=-0.36 upper=0.48 effort=14 velocity=1 -> lower=-0.36 upper=0.49 effort=14 velocity=1
- joint rightShoulderRoll: limit lower=-1.266 upper=1.509 effort=190 velocity=5.89 -> lower=-1.266 upper=1.519 effort=190 velocity=5.89
- joint rightWristPitch: limit lower=-0.48 upper=0.36 effort=14 velocity=1 -> lower=-0.49 upper=0.36 effort=14 velocity=1

File: software/models/val_description/urdf/valkyrie_sim_drake.urdf (robot description, URDF)
Before this commit: robot valkyrie, 84 links, 83 joints
Joints:
- joint leftShoulderRoll: limit lower=-1.509 upper=1.266 effort=190 velocity=5.89 -> lower=-1.519 upper=1.266 effort=190 velocity=5.89
- joint leftWristPitch: limit lower=-0.36 upper=0.48 effort=14 velocity=1 -> lower=-0.36 upper=0.49 effort=14 velocity=1
- joint rightShoulderRoll: limit lower=-1.266 upper=1.509 effort=190 velocity=5.89 -> lower=-1.266 upper=1.519 effort=190 velocity=5.89
- joint rightWristPitch: limit lower=-0.48 upper=0.36 effort=14 velocity=1 -> lower=-0.49 upper=0.36 effort=14 velocity=1

Commit message: move the hand goal frame to somewhere useful

File: software/models/val_description/urdf/valkyrie_sim.urdf (robot description, URDF)
Before this commit: robot valkyrie, 84 links, 83 joints
Joints:
- joint l_hand_face_joint: origin xyz=0.07 0.0 -0.08 rpy=3.14159265359 0 1.57079632679 -> xyz=0.06 0.0 -0.045 rpy=3.14159265359 0 1.57079632679
- joint r_hand_face_joint: origin xyz=0.07 0 0.08 rpy=0 0 -1.57079632679 -> xyz=0.06 0 0.045 rpy=0 0 -1.57079632679

File: software/models/val_description/urdf/valkyrie_sim_drake.urdf (robot description, URDF)
Before this commit: robot valkyrie, 84 links, 83 joints
Joints:
- joint l_hand_face_joint: origin xyz=0.07 0.0 -0.08 rpy=3.14159265359 0 1.57079632679 -> xyz=0.06 0.0 -0.045 rpy=3.14159265359 0 1.57079632679
- joint r_hand_face_joint: origin xyz=0.07 0 0.08 rpy=0 0 -1.57079632679 -> xyz=0.06 0 0.045 rpy=0 0 -1.57079632679
