Commit message: adding config for husky playback

File: software/models/husky_description/model.urdf (robot description, URDF)
Before this commit: robot husky, 13 links, 12 joints
Links:
- added link pelvis
Joints:
- added joint pelvis_joint: type fixed, parent base_link, child pelvis, origin xyz=0 0 0 rpy=0 0 0
